Commit message: modifications for cob3-2

File: ros/robots/cob_platform.urdf.xacro (robot description, xacro)
@@ -9,9 +9,9 @@
   <include filename="$(find cob_description)/ros/urdf/common.xacro" />
   <!-- cob base -->
-  <include filename="$(find cob_description)/ros/urdf/base_v0/base.urdf.xacro" />
+  <!--include filename="$(find cob_description)/ros/urdf/base_v0/base.urdf.xacro" /-->
   <!-- cob torse-->
   <include filename="$(find cob_description)/ros/urdf/torso_v0/torso.urdf.xacro" />
   <!-- cob eyes-->
-  <include filename="$(find cob_description)/ros/urdf/headeyes_v0/headeyes.urdf.xacro" />
+  <!--include filename="$(find cob_description)/ros/urdf/headeyes_v0/headeyes.urdf.xacro" /-->
   <!-- cob arm-->
   <!--include filename="$(find cob_description)/ros/urdf/arm_v0/arm.urdf.xacro" /-->

File: ros/urdf/torso_v0/torso.urdf.xacro (robot description, xacro)
@@ -48,5 +48,5 @@
       <axis xyz="0 0 1" />
       <dynamics damping="0.1" />
-      <calibration reference_position="0.0344"/>
+      <calibration reference_position="-0.5149"/>
       <limit effort="24" lower="-6.2831" upper="6.2831" velocity="0.5"/>
     </joint>
@@ -73,5 +73,5 @@
     <!--joint between torso_neckZ_link and torso_neck_link-->
     <joint name="${name}_neck_joint" type="revolute">
-      <origin xyz="0 0 0" rpy="0 0.293 0" />   <!--FIX pitch angle Later-->
+      <origin xyz="0 0 0" rpy="0 0 0" />   <!--FIX pitch angle Later-->
       <parent link="${name}_neckZ_link"/>
       <child link="${name}_neck_link"/>
@@ -109,5 +109,5 @@
       <axis xyz="0 0 1" />
       <dynamics damping="0.1" />
-      <calibration reference_position="0.022078"/>
+      <calibration reference_position="0.0247"/>
       <limit effort="24" lower="-1.5" upper="1.5" velocity="0.5"/>
     </joint>
@@ -134,5 +134,5 @@
     <!--joint between torso_headZ_link and torso_headbase_link-->
     <joint name="${name}_headbase_joint" type="revolute">
-      <origin xyz="0 0 0" rpy="0 -0.26 0" /> <!---0.392699075-->
+      <origin xyz="0 0 0" rpy="0 0 0" /> <!---0.392699075-->
       <parent link="${name}_headZ_link"/>
       <child link="${name}_headbase_link"/>

Commit message: new urdf desciption

File: ros/robots/cob_platform.urdf.xacro (robot description, xacro)
@@ -13,5 +13,5 @@
   <include filename="$(find cob_description)/ros/urdf/torso_v0/torso.urdf.xacro" />
   <!-- cob eyes-->
-  <include filename="$(find cob_description)/ros/urdf/headeyes_v0/headeyes.urdf.xacro" />
+  <include filename="$(find cob_description)/ros/urdf/head_cameras_v0/head_cameras.urdf.xacro" />
   <!-- cob arm-->
   <!--include filename="$(find cob_description)/ros/urdf/arm_v0/arm.urdf.xacro" /-->
@@ -32,6 +32,6 @@
     <origin xyz="0.24627 0 0.7798" rpy="0 0 0" />
   </xacro:cob_torso_v0>
-  <xacro:cob_headeyes_v0 name="headeyes" parent="torso_headbase_link">
+  <xacro:cob_head_cameras_v0 name="head" parent="torso_upper_neck_tilt_link">
     <origin xyz="0 0 0.154" rpy="0 0 0" />
-  </xacro:cob_headeyes_v0>
+  </xacro:cob_head_cameras_v0>
 </robot>

File: ros/urdf/sensors/cameraone.urdf.xacro (robot description, xacro)
@@ -7,5 +7,5 @@
   <include filename="$(find cob_description)/ros/urdf/sensors/cameraone.gazebo.xacro" />
   <xacro:macro name="cob_cameraone_v0" params="name parent *origin">
-    <joint name="${name}_frame_joint" type="fixed">
+    <joint name="${name}_joint" type="fixed">
       <insert_block name="origin" />
       <parent link="${parent}"/>

File: ros/urdf/torso_v0/torso.gazebo.xacro (robot description, xacro)
@@ -9,21 +9,21 @@
       <turnGravityOff>false</turnGravityOff>
     </gazebo>
-    <gazebo reference="${name}_neckZ_link">
+    <gazebo reference="${name}_lower_neck_pan_link">
       <material value="PR2/Blue" />
       <turnGravityOff>false</turnGravityOff>
     </gazebo>
-    <gazebo reference="${name}_neck_link">
+    <gazebo reference="${name}_lower_neck_tilt_link">
       <material value="PR2/Red" />
       <turnGravityOff>false</turnGravityOff>
     </gazebo>
-    <gazebo reference="${name}_headZ_link">
+    <gazebo reference="${name}_upper_neck_pan_link">
       <material value="PR2/Blue" />
       <turnGravityOff>false</turnGravityOff>
     </gazebo>
-    <gazebo reference="${name}_headbase_link">
+    <gazebo reference="${name}_upper_neck_tilt_link">
       <material value="PR2/Grey" />
       <turnGravityOff>false</turnGravityOff>
     </gazebo>
-    <gazebo reference="${name}_headcover_link">
+    <gazebo reference="head_cover_link">
       <material value="PR2/Blue" />
       <turnGravityOff>false</turnGravityOff>

File: ros/urdf/torso_v0/torso.transmission.xacro (robot description, xacro)
@@ -5,14 +5,4 @@
        xmlns:xacro="http://ros.org/wiki/xacro">
   <xacro:macro name="cob_torso_transmission_v0" params="name">
-    <transmission name="${name}_neckZ_trans" type="SimpleTransmission">
-		<actuator name="${name}_neckZ_motor"/>
-		<joint name="${name}_neckZ_joint"/>
-		<mechanicalReduction>1</mechanicalReduction>
-    </transmission>
-    <transmission name="${name}_neck_trans" type="SimpleTransmission">
-		<actuator name="${name}_neck_motor"/>
-		<joint name="${name}_neck_joint"/>
-		<mechanicalReduction>1</mechanicalReduction>
-    </transmission>
     <transmission name="${name}_tray_trans" type="SimpleTransmission">
 		<actuator name="${name}_tray_motor"/>
@@ -20,12 +10,22 @@
 		<mechanicalReduction>1</mechanicalReduction>
     </transmission>
-    <transmission name="${name}_headZ_trans" type="SimpleTransmission">
-		<actuator name="${name}_headZ_motor"/>
-		<joint name="${name}_headZ_joint"/>
+    <transmission name="${name}_lower_neck_pan_trans" type="SimpleTransmission">
+		<actuator name="${name}_lower_neck_pan_motor"/>
+		<joint name="${name}_lower_neck_pan_joint"/>
 		<mechanicalReduction>1</mechanicalReduction>
     </transmission>
-    <transmission name="${name}_headbase_trans" type="SimpleTransmission">
-		<actuator name="${name}_headbase_motor"/>
-		<joint name="${name}_headbase_joint"/>
+    <transmission name="${name}_lower_neck_tilt_trans" type="SimpleTransmission">
+		<actuator name="${name}_lower_neck_tilt_motor"/>
+		<joint name="${name}_lower_neck_tilt_joint"/>
+		<mechanicalReduction>1</mechanicalReduction>
+    </transmission>
+    <transmission name="${name}_upper_neck_pan_trans" type="SimpleTransmission">
+		<actuator name="${name}_upper_neck_pan_motor"/>
+		<joint name="${name}_upper_neck_pan_joint"/>
+		<mechanicalReduction>1</mechanicalReduction>
+    </transmission>
+    <transmission name="${name}_upper_neck_tilt_trans" type="SimpleTransmission">
+		<actuator name="${name}_upper_neck_tilt_motor"/>
+		<joint name="${name}_upper_neck_tilt_joint"/>
 		<mechanicalReduction>1</mechanicalReduction>
     </transmission>

File: ros/urdf/torso_v0/torso.urdf.xacro (robot description, xacro)
@@ -41,15 +41,15 @@
        </collision>
     </link>
-    <!--joint between base_link and torso_neckZ_link-->
-    <joint name="${name}_neckZ_joint" type="revolute">
+    <!--joint between base_link and torso_lower_neck_pan_link-->
+    <joint name="${name}_lower_neck_pan_joint" type="revolute">
       <insert_block name="origin" />
       <parent link="${parent}"/>
-      <child link="${name}_neckZ_link"/>
+      <child link="${name}_lower_neck_pan_link"/>
       <axis xyz="0 0 1" />
       <dynamics damping="0.1" />
-      <calibration reference_position="0.0344"/>
+      <calibration reference_position="-0.5149"/>
       <limit effort="24" lower="-6.2831" upper="6.2831" velocity="0.5"/>
     </joint>
-    <link name="${name}_neckZ_link">
+    <link name="${name}_lower_neck_pan_link">
 	<inertial>
 	   <origin xyz="0 0 0" rpy="0 0 0"/>
@@ -71,9 +71,9 @@
 	</collision>
     </link>
-    <!--joint between torso_neckZ_link and torso_neck_link-->
-    <joint name="${name}_neck_joint" type="revolute">
+    <!--joint between torso_lower_neck_pan_link and torso_lower_neck_tilt_link-->
+    <joint name="${name}_lower_neck_tilt_joint" type="revolute">
       <origin xyz="0 0 0" rpy="0 0.293 0" />   <!--FIX pitch angle Later-->
-      <parent link="${name}_neckZ_link"/>
-      <child link="${name}_neck_link"/>
+      <parent link="${name}_lower_neck_pan_link"/>
+      <child link="${name}_lower_neck_tilt_link"/>
       <axis xyz="0 1 0" />
       <dynamics damping="0.1" />
@@ -81,5 +81,5 @@
       <limit effort="46" lower="-1.5" upper="1.5" velocity="0.5"/>
     </joint>
-    <link name="${name}_neck_link">
+    <link name="${name}_lower_neck_tilt_link">
        <inertial>
 	  <origin xyz="0 0 0" rpy="0 0 0"/>
@@ -102,15 +102,15 @@
        </collision>
     </link>
-    <!--joint between torso_neck_link and torso_headZ_link-->
-    <joint name="${name}_headZ_joint" type="revolute">
+    <!--joint between torso_lower_neck_tilt_link and torso_upper_neck_pan_link-->
+    <joint name="${name}_upper_neck_pan_joint" type="revolute">
       <origin xyz="-0.09039 0 0.30489" rpy="0 0 0" />
-      <parent link="${name}_neck_link"/>
-      <child link="${name}_headZ_link"/>
+      <parent link="${name}_lower_neck_tilt_link"/>
+      <child link="${name}_upper_neck_pan_link"/>
       <axis xyz="0 0 1" />
       <dynamics damping="0.1" />
-      <calibration reference_position="0.022078"/>
-      <limit effort="24" lower="-1.5" upper="1.5" velocity="0.5"/>
+      <calibration reference_position="0.0247"/>
+      <limit effort="4" lower="-6.2831" upper="6.2831" velocity="0.5"/>
     </joint>
-    <link name="${name}_headZ_link">
+    <link name="${name}_upper_neck_pan_link">
 	<inertial>
 	   <origin xyz="0 0 0" rpy="0 0 0"/>
@@ -132,9 +132,9 @@
 	</collision>
     </link>
-    <!--joint between torso_headZ_link and torso_headbase_link-->
-    <joint name="${name}_headbase_joint" type="revolute">
+    <!--joint between torso_upper_neck_pan_link and torso_upper_neck_tilt_link-->
+    <joint name="${name}_upper_neck_tilt_joint" type="revolute">
       <origin xyz="0 0 0" rpy="0 -0.26 0" /> <!---0.392699075-->
-      <parent link="${name}_headZ_link"/>
-      <child link="${name}_headbase_link"/>
+      <parent link="${name}_upper_neck_pan_link"/>
+      <child link="${name}_upper_neck_tilt_link"/>
       <axis xyz="0 1 0" />
       <dynamics damping="0.1" />
@@ -142,5 +142,5 @@
       <limit effort="24" lower="-1.5" upper="1.5" velocity="0.5"/>
     </joint>
-    <link name="${name}_headbase_link">
+    <link name="${name}_upper_neck_tilt_link">
 	<inertial>
 	   <origin xyz="0 0 0" rpy="0 0 0"/>
@@ -162,11 +162,11 @@
 	</collision>
     </link>
-    <!--joint between torso_headbase_link and torso_headcover_link-->
-    <joint name="${name}_headcover_joint" type="fixed">
+    <!--joint between torso_upper_neck_tilt_link and head_cover_link-->
+    <joint name="head_cover_joint" type="fixed">
       <origin xyz="0 0 0" rpy="0 0 0" />
-      <parent link="${name}_headbase_link"/>
-      <child link="${name}_headcover_link"/>
+      <parent link="${name}_upper_neck_tilt_link"/>
+      <child link="head_cover_link"/>
     </joint>
-    <link name="${name}_headcover_link">
+    <link name="head_cover_link">
 	<inertial>
 	   <origin xyz="0 0 0" rpy="0 0 0"/>

Commit message: included arm

File: ros/robots/cob_platform.urdf.xacro (robot description, xacro)
@@ -15,5 +15,5 @@
   <include filename="$(find cob_description)/ros/urdf/head_cameras_v0/head_cameras.urdf.xacro" />
   <!-- cob arm-->
-  <!--include filename="$(find cob_description)/ros/urdf/arm_v0/arm.urdf.xacro" /-->
+  <include filename="$(find cob_description)/ros/urdf/arm_v0/arm.urdf.xacro" />
   <!-- generic simulator_gazebo plugins for starting mechanism control, ros time, ros battery -->
   <include filename="$(find cob_description)/ros/gazebo/gazebo.urdf.xacro" />
@@ -35,3 +35,6 @@
     <origin xyz="0 0 0.154" rpy="0 0 0" />
   </xacro:cob_head_cameras_v0>
+  <xacro:cob_arm_v0 name="arm" parent="base_link">
+    <origin xyz="0.040 -0.005 0.83637" rpy="3.1415926 0.7854 -1.8326" />
+  </xacro:cob_arm_v0>
 </robot>

File: ros/urdf/torso_v0/torso.urdf.xacro (robot description, xacro)
@@ -54,11 +54,11 @@
 	<inertial>
 	   <origin xyz="0 0 0" rpy="0 0 0"/>
-	   <mass value="0.1"/>
-	   <inertia ixx="0.001"  ixy="0"  ixz="0" iyy="0.001" iyz="0" izz="0.001" />
+	   <mass value="1.0"/>
+	   <inertia ixx="0.01"  ixy="0"  ixz="0" iyy="0.01" iyz="0" izz="0.01" />
 	</inertial>
 	<visual>
-	   <origin xyz="0 0 0.0005" rpy="0 0 0" />
+	   <origin xyz="0 0 0.005" rpy="0 0 0" />
 	   <geometry>
-	      <box size="0.001 0.001 0.001"/>
+	      <box size="0.01 0.01 0.01"/>
 	   </geometry>
            <material name="Blue" />
@@ -115,16 +115,16 @@
 	<inertial>
 	   <origin xyz="0 0 0" rpy="0 0 0"/>
-	   <mass value="1"/>
-	   <inertia ixx="0.001"  ixy="0"  ixz="0" iyy="0.001" iyz="0" izz="0.001" />
+	   <mass value="1.0"/>
+	   <inertia ixx="0.01"  ixy="0"  ixz="0" iyy="0.01" iyz="0" izz="0.01" />
         </inertial>
 	<visual>
-	   <origin xyz="0 0 0" rpy="0 0 0" />
+	   <origin xyz="0 0 0.005" rpy="0 0 0" />
 	   <geometry>
-              <box size="0.001 0.001 0.001"/>
+              <box size="0.01 0.01 0.01"/>
 	   </geometry>
            <material name="Blue" />
 	</visual>
 	<collision>
-	   <origin xyz="0 0 0" rpy="0 0 0" />
+	   <origin xyz="0 0 0.0005" rpy="0 0 0" />
 	   <geometry>
               <box size="0.001 0.001 0.001"/>
