Commit message: included calibration files

File: ros/robots/cob_platform.urdf.xacro (robot description, xacro)
@@ -8,12 +8,16 @@
   <!-- misc common stuff? -->
   <include filename="$(find cob_description)/ros/urdf/common.xacro" />
+  <!-- cob calibration -->
+  <include filename="$(find cob_description)/ros/calibration/cob3-1.urdf.xacro" />
   <!-- cob base -->
   <include filename="$(find cob_description)/ros/urdf/base_v0/base.urdf.xacro" />
   <!-- cob torse-->
   <include filename="$(find cob_description)/ros/urdf/torso_v0/torso.urdf.xacro" />
-  <!-- cob eyes-->
+  <!-- cob cameras-->
   <include filename="$(find cob_description)/ros/urdf/head_cameras_v0/head_cameras.urdf.xacro" />
   <!-- cob arm-->
   <include filename="$(find cob_description)/ros/urdf/arm_v0/arm.urdf.xacro" />
+  <!-- cob sdh-->
+  <include filename="$(find cob_description)/ros/urdf/sdh_v0/sdh.urdf.xacro" />
   <!-- generic simulator_gazebo plugins for starting mechanism control, ros time, ros battery -->
   <include filename="$(find cob_description)/ros/gazebo/gazebo.urdf.xacro" />
@@ -38,3 +42,6 @@
     <origin xyz="0.040 -0.005 0.83637" rpy="3.1415926 0.7854 -1.8326" />
   </xacro:cob_arm_v0>
+  <xacro:cob_sdh_v0 name="sdh" parent="arm_7_link">
+    <origin xyz="0 0 0" rpy="0 3.1415926 0" />
+  </xacro:cob_sdh_v0>
 </robot>

File: ros/urdf/arm_v0/arm.urdf.xacro (robot description, xacro)
@@ -42,12 +42,12 @@
 		<child link="${name}_1_link"/>
 		<axis xyz="0 0 1"/>
-	        <calibration reference_position="1.47881"/>
+	        <calibration reference_position="${arm_1_ref}"/>
 		<limit effort="370" velocity="0.4363" lower="-2.0943951" upper="2.0943951"/>
 	</joint>
 	<link name="${name}_1_link">
 		<inertial>
-			<origin xyz="0 0 0" rpy="0 0 0" />
-			<mass value="5.4"/>
-			<inertia ixx="0.01"  ixy="0"  ixz="0" iyy="0.01" iyz="0" izz="0.01" />
+			<origin xyz="0 0.00923 0.1564" rpy="0 0 0" />
+			<mass value="5.9907"/>
+			<inertia ixx="0.184545"  ixy="0"  ixz="0" iyy="0.180577" iyz="0.000420" izz="0.016081" />
 		</inertial>
 		<visual>
@@ -71,12 +71,12 @@
 		<child link="${name}_2_link"/>
 		<axis xyz="0 0 1"/>
-	        <calibration reference_position="1.47881"/>
+	        <calibration reference_position="${arm_2_ref}"/>
 		<limit effort="370" velocity="0.4363" lower="-2.0943951" upper="2.0943951"/>
 	</joint>
 	<link name="${name}_2_link">
 		<inertial>
-			<origin xyz="0 0 0" rpy="0 0 0"/>
-			<mass value="2.8"/>
-			<inertia ixx="0.01"  ixy="0"  ixz="0" iyy="0.01" iyz="0" izz="0.01" />
+			<origin xyz="0 -0.006249 0.008252" rpy="0 0 0"/>
+			<mass value="5.734939"/>
+			<inertia ixx="0.020715"  ixy="0"  ixz="0" iyy="0.017585" iyz="-0.000460" izz="0.014454" />
 		</inertial>
 		<visual>
@@ -100,12 +100,12 @@
 		<child link="${name}_3_link"/>
 		<axis xyz="0 0 1"/>
-	        <calibration reference_position="-6.28087"/>
+	        <calibration reference_position="${arm_3_ref}"/>
 		<limit effort="176" velocity="0.4189" lower="-6.2831853" upper="6.2831853"/>
 	</joint>
 	<link name="${name}_3_link">
 		<inertial>
-			<origin xyz="0 0 0" rpy="0 0 0"/>
-			<mass value="2.0"/>
-			<inertia ixx="0.01"  ixy="0"  ixz="0" iyy="0.01" iyz="0" izz="0.01" />
+			<origin xyz="0 0.007908 0.192805" rpy="0 0 0"/>
+			<mass value="4.214668"/>
+			<inertia ixx="0.192416"  ixy="0"  ixz="0" iyy="0.190323" iyz="0.000310" izz="0.008570" />
 		</inertial>
 		<visual>
@@ -129,12 +129,12 @@
 		<child link="${name}_4_link"/>
 		<axis xyz="0 0 1" />
-	        <calibration reference_position="0.0192641"/>
+	        <calibration reference_position="${arm_4_ref}"/>
 		<limit effort="176" velocity="0.4189" upper="2.0943951" lower="-2.0943951" />
 	</joint>
 	<link name="${name}_4_link">
 		<inertial>
-			<origin xyz="0 0 0" rpy="0 0 0"/>
-			<mass value="1.6"/>
-			<inertia ixx="0.01"  ixy="0"  ixz="0" iyy="0.01" iyz="0" izz="0.01" />
+			<origin xyz="0 -0.006319 0.009681" rpy="0 0 0"/>
+			<mass value="3.669819"/>
+			<inertia ixx="0.010547"  ixy="0"  ixz="0" iyy="0.008708" iyz="-0.000335" izz="0.006913" />
 		</inertial>
 		<visual>
@@ -158,12 +158,12 @@
 		<child link="${name}_5_link"/>
 		<axis xyz="0 0 1" />
-	        <calibration reference_position="-2.86457"/>
+	        <calibration reference_position="${arm_5_ref}"/>
 		<limit effort="41.6" velocity="0.4363" upper="6.2831853" lower="-6.2831853" />
 	</joint>
 	<link name="${name}_5_link">
 		<inertial>
-			<origin xyz="0 0 0" rpy="0 0 0"/>
-			<mass value="1.2"/>
-			<inertia ixx="0.01"  ixy="0"  ixz="0" iyy="0.01" iyz="0" izz="0.01" />
+			<origin xyz="0 -0.004963 0.008394" rpy="0 0 0"/>
+			<mass value="2.313272"/>
+			<inertia ixx="0.004108"  ixy="0"  ixz="0" iyy="0.003468" iyz="-0.000103" izz="0.002507" />
 		</inertial>
 		<visual>
@@ -187,5 +187,5 @@
 		<child link="${name}_6_link"/>
 		<axis xyz="0 0 1" />
-	        <calibration reference_position="0.00414364"/>
+	        <calibration reference_position="${arm_6_ref}"/>
 		<limit effort="20.1" velocity="0.4363" upper="2.0943951" lower="-2.0943951" />
 	</joint>
@@ -216,5 +216,5 @@
 		<child link="${name}_7_link"/>
 		<axis xyz="0 0 1" />
-	        <calibration reference_position="-0.000421242"/>
+	        <calibration reference_position="${arm_7_ref}"/>
 		<limit effort="9.6" velocity="0.8727" upper="6.2831853" lower="-6.2831853" />
 	</joint>

File: ros/urdf/base_v0/base.gazebo.xacro (robot description, xacro)
@@ -31,5 +31,5 @@
         </controller:gazebo_ros_bumper>
       </sensor:contact>
-      <material value="PR2/Grey" />
+      <material>Gazebo/Grey</material>
     </gazebo>
     <gazebo>

File: ros/urdf/base_v0/base.urdf.xacro (robot description, xacro)
@@ -178,14 +178,14 @@
     </joint>
     <!--modify here for test: front,base and top lasers -->
-    <!-- base laser front -->
-    <xacro:hokuyo_lx30_laser_v0 name="${name}_laser_front" parent="${name}" ros_topic="base_scan_front" update_rate="20" min_angle="-1.35" max_angle="1.35" >
+    <!-- base scanner front -->
+    <xacro:hokuyo_lx30_laser_v0 name="${name}_scanner_front" parent="${name}" ros_topic="base_scan_front" update_rate="20" min_angle="-1.35" max_angle="1.35" >
       <origin xyz="${base_laser_x} ${base_laser_y} ${base_laser_z}" rpy="0 0 0" />
     </xacro:hokuyo_lx30_laser_v0>
-    <!-- base laser back -->
-    <xacro:hokuyo_lx30_laser_v0 name="${name}_laser_back" parent="${name}" ros_topic="base_scan_back" update_rate="20" min_angle="-1.35" max_angle="1.35" >
+    <!-- base scanner rear -->
+    <xacro:hokuyo_lx30_laser_v0 name="${name}_scanner_rear" parent="${name}" ros_topic="base_scan_back" update_rate="20" min_angle="-1.35" max_angle="1.35" >
       <origin xyz="${-base_laser_x} ${base_laser_y} ${base_laser_z}" rpy="0 0 ${M_PI}" />
     </xacro:hokuyo_lx30_laser_v0>
-    <!-- base laser top -->
-    <xacro:hokuyo_lx30_laser_v0 name="${name}_laser_top" parent="${name}" ros_topic="base_scan_top" update_rate="10" min_angle="-2.094" max_angle="2.094" >
+    <!-- base scanner top -->
+    <xacro:hokuyo_lx30_laser_v0 name="${name}_scanner_top" parent="${name}" ros_topic="base_scan_top" update_rate="10" min_angle="-2.094" max_angle="2.094" >
       <origin xyz="-0.252 0 0.42" rpy="0 0 ${M_PI}" />
     </xacro:hokuyo_lx30_laser_v0>

File: ros/urdf/head_cameras_v0/head_cameras.urdf.xacro (robot description, xacro)
@@ -19,5 +19,5 @@
        <axis xyz="0 1 0" />
        <dynamics damping="0.1" />
-       <calibration reference_position="-3.14"/>
+       <calibration reference_position="${head_camera_axis_ref}"/>
        <limit effort="100" lower="-0.1745" upper="3.316" velocity="0.5"/>
     </joint>

File: ros/urdf/materials.urdf.xacro (robot description, xacro)
@@ -19,4 +19,7 @@
     <color rgba="1.0 1.0 1.0 1.0"/>
   </material>
+  <material name="Black">
+    <color rgba="0.0 0.0 0.0 1.0"/>
+  </material>
   <material name="Caster">
     <texture filename="package://pr2_ogre/Media/materials/textures/pr2_caster_texture.png" />

File: ros/urdf/torso_v0/torso.gazebo.xacro (robot description, xacro)
@@ -6,25 +6,25 @@
   <xacro:macro name="cob_torso_gazebo_v0" params="name">
     <gazebo reference="${name}_tray_link">
-      <material>PR2/Green</material>
+      <material>Gazebo/Green</material>
       <turnGravityOff>false</turnGravityOff>
     </gazebo>
     <gazebo reference="${name}_lower_neck_pan_link">
-      <material value="PR2/Blue" />
+      <material>Gazebo/Blue</material>
       <turnGravityOff>false</turnGravityOff>
     </gazebo>
     <gazebo reference="${name}_lower_neck_tilt_link">
-      <material value="PR2/Red" />
+      <material>Gazebo/Red</material>
       <turnGravityOff>false</turnGravityOff>
     </gazebo>
     <gazebo reference="${name}_upper_neck_pan_link">
-      <material value="PR2/Blue" />
+      <material>Gazebo/Blue</material>
       <turnGravityOff>false</turnGravityOff>
     </gazebo>
     <gazebo reference="${name}_upper_neck_tilt_link">
-      <material value="PR2/Grey" />
+      <material>Gazebo/Grey</material>
       <turnGravityOff>false</turnGravityOff>
     </gazebo>
     <gazebo reference="head_cover_link">
-      <material value="PR2/Blue" />
+      <material>Gazebo/Blue</material>
       <turnGravityOff>false</turnGravityOff>
     </gazebo>

File: ros/urdf/torso_v0/torso.urdf.xacro (robot description, xacro)
@@ -16,5 +16,5 @@
        <child link="${name}_tray_link"/>
        <axis xyz="0 0 1" />
-       <calibration reference_position="0.0"/>
+       <calibration reference_position="${torso_tray_ref}"/>
        <dynamics damping="1.0" />
        <limit effort="100" lower="0" upper="3.31612" velocity="5"/>
@@ -47,6 +47,6 @@
       <child link="${name}_lower_neck_pan_link"/>
       <axis xyz="0 0 1" />
+      <calibration reference_position="${torso_lower_neck_pan_ref}"/>
       <dynamics damping="0.1" />
-      <calibration reference_position="-0.5149"/>
       <limit effort="24" lower="-6.2831" upper="6.2831" velocity="0.5"/>
     </joint>
@@ -78,5 +78,5 @@
       <axis xyz="0 1 0" />
       <dynamics damping="0.1" />
-      <calibration reference_position="0.0344"/>
+      <calibration reference_position="${torso_lower_neck_tilt_ref}"/>
       <limit effort="46" lower="-1.5" upper="1.5" velocity="0.5"/>
     </joint>
@@ -109,5 +109,5 @@
       <axis xyz="0 0 1" />
       <dynamics damping="0.1" />
-      <calibration reference_position="0.0247"/>
+      <calibration reference_position="${torso_upper_neck_pan_ref}"/>
       <limit effort="4" lower="-6.2831" upper="6.2831" velocity="0.5"/>
     </joint>
@@ -139,5 +139,5 @@
       <axis xyz="0 1 0" />
       <dynamics damping="0.1" />
-      <calibration reference_position="0.022078"/>
+      <calibration reference_position="${torso_upper_neck_tilt_ref}"/>
       <limit effort="24" lower="-1.5" upper="1.5" velocity="0.5"/>
     </joint>

Commit message: modified urdf to have less shaking

File: ros/robots/cob_platform.urdf.xacro (robot description, xacro)
@@ -36,10 +36,10 @@
     <origin xyz="0.24627 0 0.7798" rpy="3.1415926 0 0" />
   </xacro:cob_torso_v0>
-  <xacro:cob_head_cameras_v0 name="head" parent="torso_upper_neck_tilt_link">
-    <origin xyz="0 0 0.154" rpy="0 0 0" />
-  </xacro:cob_head_cameras_v0>
   <xacro:cob_arm_v0 name="arm" parent="base_link">
     <origin xyz="0.040 -0.005 0.83637" rpy="3.1415926 0.7854 -1.8326" />
   </xacro:cob_arm_v0>
+  <xacro:cob_head_cameras_v0 name="head" parent="torso_upper_neck_tilt_link">
+    <origin xyz="0 -0.154 0" rpy="-1.5708 0 0" />
+  </xacro:cob_head_cameras_v0>
   <xacro:cob_sdh_v0 name="sdh" parent="arm_7_link">
     <origin xyz="0 0 0" rpy="0 3.1415926 0" />

File: ros/urdf/arm_v0/arm.urdf.xacro (robot description, xacro)
@@ -30,7 +30,7 @@
 		</visual>
 		<collision>
-		   <origin xyz="0 0 0.0005" rpy="0 0 0" />
+		   <origin xyz="0 0 0.005" rpy="0 0 0" />
 		   <geometry>
-		      <box size="0.001 0.001 0.001"/>
+		      <box size="0.01 0.01 0.01"/>
 		   </geometry>
 		</collision>
@@ -47,7 +47,7 @@
 	<link name="${name}_1_link">
 		<inertial>
-			<origin xyz="0 0.00923 0.1564" rpy="0 0 0" />
+			<origin xyz="0 0 0" rpy="0 0 0" />
 			<mass value="5.9907"/>
-			<inertia ixx="0.184545"  ixy="0"  ixz="0" iyy="0.180577" iyz="0.000420" izz="0.016081" />
+			<inertia ixx="5"  ixy="0"  ixz="0" iyy="5" iyz="0" izz="5" />
 		</inertial>
 		<visual>
@@ -76,7 +76,7 @@
 	<link name="${name}_2_link">
 		<inertial>
-			<origin xyz="0 -0.00629 0.008252" rpy="0 0 0"/>
+			<origin xyz="0 0 0" rpy="0 0 0"/>
 			<mass value="5.734939"/>
-			<inertia ixx="0.020715"  ixy="0"  ixz="0" iyy="0.017585" iyz="-0.000460" izz="0.01454" />
+			<inertia ixx="0.03"  ixy="0"  ixz="0" iyy="0.03" iyz="0" izz="0.03" />
 		</inertial>
 		<visual>
@@ -106,6 +106,6 @@
 		<inertial>
 			<origin xyz="0 0 0" rpy="0 0 0"/>
-			<mass value="2.0"/>
-			<inertia ixx="0.01"  ixy="0"  ixz="0" iyy="0.01" iyz="0" izz="0.01" />
+			<mass value="4.214668"/>
+			<inertia ixx="0.03"  ixy="0"  ixz="0" iyy="0.03" iyz="0" izz="0.03" />
 		</inertial>
 		<visual>
@@ -135,6 +135,6 @@
 		<inertial>
 			<origin xyz="0 0 0" rpy="0 0 0"/>
-			<mass value="1.6"/>
-			<inertia ixx="0.01"  ixy="0"  ixz="0" iyy="0.01" iyz="0" izz="0.01" />
+			<mass value="3.669819"/>
+			<inertia ixx="0.03"  ixy="0"  ixz="0" iyy="0.03" iyz="0" izz="0.03" />
 		</inertial>
 		<visual>
@@ -164,6 +164,6 @@
 		<inertial>
 			<origin xyz="0 0 0" rpy="0 0 0"/>
-			<mass value="1.2"/>
-			<inertia ixx="0.01"  ixy="0"  ixz="0" iyy="0.01" iyz="0" izz="0.01" />
+			<mass value="2.313272"/>
+			<inertia ixx="0.03"  ixy="0"  ixz="0" iyy="0.03" iyz="0" izz="0.03" />
 		</inertial>
 		<visual>
@@ -193,5 +193,5 @@
 		<inertial>
 			<origin xyz="0 0 0" rpy="0 0 0"/>
-			<mass value="1.1"/>
+			<mass value="2.057856"/>
 			<inertia ixx="0.01"  ixy="0"  ixz="0" iyy="0.01" iyz="0" izz="0.01" />
 		</inertial>
@@ -222,5 +222,5 @@
 		<inertial>
 			<origin xyz="0 0 0" rpy="0 0 0"/>
-			<mass value="0.5"/>
+			<mass value="1.120198"/>
 			<inertia ixx="0.01"  ixy="0"  ixz="0" iyy="0.01" iyz="0" izz="0.01" />
 		</inertial>

File: ros/urdf/base_v0/base.urdf.xacro (robot description, xacro)
@@ -74,5 +74,5 @@
     <xacro:cob_wheel_transmission_v0 parent="${parent}" suffix="${suffix}" reflect="${reflect}" />
   </xacro:macro>
-  <!-- Macro for PR2 Caster hub only -->
+  <!-- Macro for Caster hub only -->
   <xacro:macro name="cob_caster_hub_v0" params="suffix parent *origin ref_position" >
     <joint name="${suffix}_rotation_joint" type="continuous">
@@ -173,5 +173,5 @@
     </link>
     <joint name="${name}_footprint_joint" type="fixed">
-      <origin xyz="0 0 0" rpy="0 0 0" />
+      <origin xyz="0 0 0.051" rpy="0 0 0" />
       <child link="${name}_link" />
       <parent link="${name}_footprint"/>
@@ -183,5 +183,5 @@
     </xacro:hokuyo_lx30_laser_v0>
     <!-- base scanner rear -->
-    <xacro:hokuyo_lx30_laser_v0 name="${name}_scanner_rear" parent="${name}" ros_topic="base_scan_back" update_rate="20" min_angle="-1.35" max_angle="1.35" >
+    <xacro:hokuyo_lx30_laser_v0 name="${name}_scanner_rear" parent="${name}" ros_topic="base_scan_rear" update_rate="20" min_angle="-1.35" max_angle="1.35" >
       <origin xyz="${-base_laser_x} ${base_laser_y} ${base_laser_z}" rpy="0 0 ${M_PI}" />
     </xacro:hokuyo_lx30_laser_v0>

File: ros/urdf/torso_v0/torso.urdf.xacro (robot description, xacro)
@@ -17,5 +17,5 @@
        <axis xyz="0 0 1" />
        <calibration reference_position="${torso_tray_ref}"/>
-       <dynamics damping="1.0" />
+       <dynamics damping="5.0" friction="0.5"/>
        <limit effort="100" lower="0" upper="3.31612" velocity="5"/>
     </joint>
@@ -24,6 +24,5 @@
 	  <origin xyz="0 0 0" rpy="0 0 0"/>
 	  <mass value="0.1"/>
-	  <inertia ixx="0.000482611007"  ixy="-0.000144683999"  ixz="0.000110076136"
-                 iyy="0.0005218991412"  iyz="-0.000314239509"  izz="0.0008618784925" />
+	  <inertia ixx="0.01"  ixy="0"  ixz="0" iyy="0.01"  iyz="0"  izz="0.01" />
        </inertial>
        <visual>
@@ -48,5 +47,5 @@
       <axis xyz="0 0 1" />
       <calibration reference_position="${torso_lower_neck_pan_ref}"/>
-      <dynamics damping="0.1" />
+      <dynamics damping="15.0" friction="10.0"/>
       <limit effort="24" lower="-6.2831" upper="6.2831" velocity="0.5"/>
     </joint>
@@ -55,5 +54,5 @@
 	   <origin xyz="0 0 0" rpy="0 0 0"/>
 	   <mass value="1.0"/>
-	   <inertia ixx="0.01"  ixy="0"  ixz="0" iyy="0.01" iyz="0" izz="0.01" />
+	   <inertia ixx="0.200549"  ixy="0.001322"  ixz="-0.000000" iyy="0.123664" iyz="-0.000000" izz="0.104101" />
 	</inertial>
 	<visual>
@@ -77,5 +76,5 @@
       <child link="${name}_lower_neck_tilt_link"/>
       <axis xyz="0 0 1" />
-      <dynamics damping="0.1" />
+      <dynamics damping="15.0" friction="10.0"/>
       <calibration reference_position="${torso_lower_neck_tilt_ref}"/>
       <limit effort="46" lower="-1.5" upper="1.5" velocity="0.5"/>
@@ -84,7 +83,7 @@
        <inertial>
 	  <origin xyz="0 0 0" rpy="0 0 0"/>
-	  <mass value="3"/>
-	  <inertia ixx="0.0001"  ixy="0"  ixz="0"
-                 iyy="0.0001"  iyz="0"  izz="0.0001" />
+	  <mass value="6.209720"/>
+	  <inertia ixx="0.171118"  ixy="0.002544"  ixz="-0.000000"
+                 iyy="0.083077"  iyz="0.000000"  izz="0.120948" />
        </inertial>
        <visual>
@@ -108,5 +107,5 @@
       <child link="${name}_upper_neck_pan_link"/>
       <axis xyz="0 0 1" />
-      <dynamics damping="0.1" />
+      <dynamics damping="15.0" friction="10.0"/>
       <calibration reference_position="${torso_upper_neck_pan_ref}"/>
       <limit effort="4" lower="-6.2831" upper="6.2831" velocity="0.5"/>
@@ -134,9 +133,9 @@
     <!--joint between torso_upper_neck_pan_link and torso_upper_neck_tilt_link-->
     <joint name="${name}_upper_neck_tilt_joint" type="revolute">
-      <origin xyz="0 0 0" rpy="1.5708 0 0" /> <!---0.392699075-->
+      <origin xyz="0 0 0" rpy="1.5708 0 0" />
       <parent link="${name}_upper_neck_pan_link"/>
       <child link="${name}_upper_neck_tilt_link"/>
       <axis xyz="0 0 1" />
-      <dynamics damping="0.1" />
+      <dynamics damping="15.0" friction="10.0"/>
       <calibration reference_position="${torso_upper_neck_tilt_ref}"/>
       <limit effort="24" lower="-1.5" upper="1.5" velocity="0.5"/>
@@ -145,6 +144,6 @@
 	<inertial>
 	   <origin xyz="0 0 0" rpy="0 0 0"/>
-	   <mass value="1"/>
-	   <inertia ixx="0.001"  ixy="0"  ixz="0" iyy="0.001" iyz="0" izz="0.001" />
+	   <mass value="6.744238"/>
+	   <inertia ixx="0.01"  ixy="0"  ixz="0" iyy="0.01" iyz="0" izz="0.01" />
         </inertial>
 	<visual>
@@ -172,10 +171,10 @@
 	   <origin xyz="0 0 0" rpy="0 0 0"/>
 	   <mass value="0.5"/>
-	   <inertia ixx="0.001"  ixy="0"  ixz="0" iyy="0.001" iyz="0" izz="0.001" />
+	   <inertia ixx="0.01"  ixy="0"  ixz="0" iyy="0.01" iyz="0" izz="0.01" />
         </inertial>
 	<visual>
 	   <origin xyz="0 0 0" rpy="0 0 0" />
 	   <geometry>
-			<mesh filename="package://cob_description/ros/meshes/torso_v0/head_cover.stl" />
+              <mesh filename="package://cob_description/ros/meshes/torso_v0/head_cover.stl" />
 	   </geometry>
            <material name="Blue" />
@@ -184,5 +183,5 @@
 	   <origin xyz="0 0 0" rpy="0 0 0" />
 	   <geometry>
-			<mesh filename="package://cob_description/ros/meshes/torso_v0/head_cover.stl" />
+	      <mesh filename="package://cob_description/ros/meshes/torso_v0/head_cover.stl" />
 	   </geometry>
 	</collision>
