Commit message: small fixes for simulation

File: ros/robots/sdh.urdf.xacro (robot description, xacro)
@@ -15,7 +15,28 @@
   <!-- materials for visualization -->
   <include filename="$(find cob_description)/ros/urdf/materials.urdf.xacro" />
+  <!-- foot for sdh-->
+	<link name="base_link">
+		<inertial>
+		   <origin xyz="0 0 0" rpy="0 0 0"/>
+		   <mass value="100.0"/>
+		   <inertia ixx="10.0"  ixy="0"  ixz="0" iyy="100.0" iyz="0" izz="100.0" />
+		</inertial>
+		<visual>
+		   <origin xyz="0 0 0.25" rpy="0 0 0" />
+		   <geometry>
+			  <cylinder radius="0.1" length="0.5"/>
+		   </geometry>
+		   <material name="Grey" />
+		</visual>
+		<collision>
+		   <origin xyz="0 0 0.25" rpy="0 0 0" />
+		   <geometry>
+			  <cylinder radius="0.1" length="0.5"/>
+		   </geometry>
+		</collision>
+	</link>
   <!-- sdh -->
-  <xacro:cob_sdh_v0 name="sdh" parent="world">
-    <origin xyz="0 0 0.01" rpy="0 0 0" />
+  <xacro:cob_sdh_v0 name="sdh" parent="base_link">
+    <origin xyz="0 0 0.5" rpy="0 0 0" />
   </xacro:cob_sdh_v0>
 </robot>
