Commit message: updated lbr description, is now correct

File: ros/robots/cob3-lbr.urdf.xacro (robot description, xacro)
@@ -37,5 +37,5 @@
   </xacro:cob_torso_v0>
   <xacro:cob_lbr_v0 name="lbr" parent="base_link">
-    <origin xyz="0.040 -0.005 0.83637" rpy="3.1415926 0.7854 -1.8326" />
+    <origin xyz="0.040 -0.005 0.83637" rpy="0 0.7854 -1.8326" />
   </xacro:cob_lbr_v0>
   <xacro:cob_head_cameras_v0 name="head" parent="torso_upper_neck_tilt_link">
@@ -43,5 +43,5 @@
   </xacro:cob_head_cameras_v0>
   <xacro:cob_sdh_v0 name="sdh" parent="lbr_7_link">
-    <origin xyz="0 0 -0.02" rpy="0 3.1415926 0" />
+    <origin xyz="0 0 0.02" rpy="0 0 0" />
   </xacro:cob_sdh_v0>
 </robot>

File: ros/robots/lbr.urdf.xacro (robot description, xacro)
@@ -38,5 +38,5 @@
   <!-- cob lbr-->
   <xacro:cob_lbr_v0 name="lbr" parent="base_link">
-    <origin xyz="0 0 0.5" rpy="3.1415926 0 0" />
+    <origin xyz="0 0 1.5" rpy="0 0 0" />
   </xacro:cob_lbr_v0>
 </robot>

File: ros/urdf/lbr_v0/lbr.urdf.xacro (robot description, xacro)
@@ -30,7 +30,7 @@
 		</visual>
 		<collision>
-		   <origin xyz="0 0 0.005" rpy="0 0 0" />
+		   <origin xyz="0 0 0.09" rpy="0 0 0" />
 		   <geometry>
-		      <box size="0.01 0.01 0.01"/>
+		      <cylinder radius="0.045" length="0.18"/>
 		   </geometry>
 		</collision>
@@ -38,5 +38,5 @@
        <!--joint between lbr_0_link and lbr_1_link -->
 	<joint name="${name}_1_joint" type="revolute">
-		<origin xyz="0 0 0" rpy="0 0 0"/>
+		<origin xyz="0 0 0.18" rpy="0 0 0"/>
 		<parent link="${name}_0_link"/>
 		<child link="${name}_1_link"/>
@@ -68,5 +68,5 @@
         <!--joint between lbr_1_link and lbr_2_link-->
 	<joint name="${name}_2_joint" type="revolute">
-		<origin xyz="0 0 -0.1915" rpy="1.5708 0 0"/>
+		<origin xyz="0 -0.002 0.1915" rpy="1.5708 0 0"/>
 		<parent link="${name}_1_link"/>
 		<child link="${name}_2_link"/>
@@ -98,5 +98,5 @@
         <!--joint between lbr_2_link and lbr_3_link-->
 	<joint name="${name}_3_joint" type="revolute">
-		<origin xyz="0 -0.1915 0" rpy="-1.5708 0 0"/>
+		<origin xyz="0 0.2085 0" rpy="-1.5708 0 0"/>
 		<parent link="${name}_2_link"/>
 		<child link="${name}_3_link"/>
@@ -128,5 +128,5 @@
          <!--joint between lbr_3_link and lbr_4_link-->
 	<joint name="${name}_4_joint" type="revolute">
-		<origin xyz="0 0 -0.1915" rpy="1.5708 0 0" />
+		<origin xyz="0 0.002 0.1915" rpy="-1.5708 0 0" />
 		<parent link="${name}_3_link"/>
 		<child link="${name}_4_link"/>
@@ -158,5 +158,5 @@
         <!--joint between lbr_4_link and lbr_5_link-->
 	<joint name="${name}_5_joint" type="revolute">
-		<origin xyz="0 -0.1915 0" rpy="-1.5708 0 0" />
+		<origin xyz="0 -0.2085 0" rpy="1.5708 0 0" />
 		<parent link="${name}_4_link"/>
 		<child link="${name}_5_link"/>
@@ -188,5 +188,5 @@
 	<!--joint between lbr_5_link and lbr_6_link-->
 	<joint name="${name}_6_joint" type="revolute">
-		<origin xyz="0 0 -0.15" rpy="1.5708 0 0" />
+		<origin xyz="0 0.046 0.1815" rpy="1.5708 0 0" />
 		<parent link="${name}_5_link"/>
 		<child link="${name}_6_link"/>
@@ -218,5 +218,5 @@
 	<!--joint between lbr_6_link and lbr_7_link-->
 	<joint name="${name}_7_joint" type="revolute">
-		<origin xyz="0 -0.13 0" rpy="-1.5708 0 0" />
+		<origin xyz="0 0.057 0.0455" rpy="-1.5708 0 0" />
 		<parent link="${name}_6_link"/>
 		<child link="${name}_7_link"/>
