Commit message: dual arm cob3 simulation and modified controllers for schunk simulation

File: ros/robots/lbr_sdh.urdf.xacro (robot description, xacro)
@@ -11,4 +11,6 @@
   <!-- cob lbr-->
   <include filename="$(find cob_description)/ros/urdf/lbr_v0/lbr.urdf.xacro" />
+  <!-- cob sdh-->
+  <include filename="$(find cob_description)/ros/urdf/sdh_v0/sdh.urdf.xacro" />
   <!-- generic simulator_gazebo plugins for starting mechanism control, ros time, ros battery -->
   <include filename="$(find cob_description)/ros/gazebo/gazebo.urdf.xacro" />
@@ -40,3 +42,6 @@
     <origin xyz="0 0 0.5" rpy="0 0 0" />
   </xacro:cob_lbr_v0>
+  <xacro:cob_sdh_v0 name="sdh" parent="lbr_7_link">
+    <origin xyz="0 0 0.02" rpy="0 0 0" />
+  </xacro:cob_sdh_v0>
 </robot>

File: ros/urdf/arm_v0/arm.urdf.xacro (robot description, xacro)
@@ -43,5 +43,5 @@
 		<axis xyz="0 0 1"/>
 	        <calibration reference_position="${arm_1_ref}"/>
-                <dynamics damping="20" />
+                <dynamics damping="30" />
 		<limit effort="370" velocity="0.4363" lower="-6.2831853" upper="6.2831853"/>
 	</joint>
@@ -73,5 +73,5 @@
 		<axis xyz="0 0 1"/>
 	        <calibration reference_position="${arm_2_ref}"/>
-                <dynamics damping="20" />
+                <dynamics damping="30" />
 		<limit effort="370" velocity="0.4363" lower="-2.0943951" upper="2.0943951"/>
 	</joint>
@@ -103,5 +103,5 @@
 		<axis xyz="0 0 1"/>
 	        <calibration reference_position="${arm_3_ref}"/>
-                <dynamics damping="20" />
+                <dynamics damping="30" />
 		<limit effort="176" velocity="0.4189" lower="-6.2831853" upper="6.2831853"/>
 	</joint>
@@ -133,5 +133,5 @@
 		<axis xyz="0 0 1" />
 	        <calibration reference_position="${arm_4_ref}"/>
-                <dynamics damping="20" />
+                <dynamics damping="30" />
 		<limit effort="176" velocity="0.4189" upper="2.0943951" lower="-2.0943951" />
 	</joint>
@@ -163,5 +163,5 @@
 		<axis xyz="0 0 1" />
 	        <calibration reference_position="${arm_5_ref}"/>
-                <dynamics damping="10" />
+                <dynamics damping="30" />
 		<limit effort="41.6" velocity="0.4363" upper="6.2831853" lower="-6.2831853" />
 	</joint>
@@ -193,5 +193,5 @@
 		<axis xyz="0 0 1" />
 	        <calibration reference_position="${arm_6_ref}"/>
-                <dynamics damping="10" />
+                <dynamics damping="30" />
 		<limit effort="20.1" velocity="0.4363" upper="2.0943951" lower="-2.0943951" />
 	</joint>
@@ -223,5 +223,5 @@
 		<axis xyz="0 0 1" />
 	        <calibration reference_position="${arm_7_ref}"/>
-                <dynamics damping="10" />
+                <dynamics damping="30" />
 		<limit effort="9.6" velocity="0.8727" upper="6.2831853" lower="-6.2831853" />
 	</joint>
