Commit message: improvements of lbr simulation

File: ros/robots/lbr.urdf.xacro (robot description, xacro)
@@ -25,5 +25,5 @@
 		   <origin xyz="0 0 0.25" rpy="0 0 0" />
 		   <geometry>
-			  <cylinder radius="0.1" length="0.5"/>
+			  <cylinder radius="0.075" length="0.5"/>
 		   </geometry>
 		   <material name="Grey" />
@@ -32,5 +32,5 @@
 		   <origin xyz="0 0 0.25" rpy="0 0 0" />
 		   <geometry>
-			  <cylinder radius="0.1" length="0.5"/>
+			  <cylinder radius="0.075" length="0.5"/>
 		   </geometry>
 		</collision>

Commit message: fixed error in lbr

File: ros/robots/lbr.urdf.xacro (robot description, xacro)
@@ -11,4 +11,6 @@
   <!-- cob lbr-->
   <include filename="$(find cob_description)/ros/urdf/lbr_v0/lbr.urdf.xacro" />
+  <!-- cob sdh-->
+  <include filename="$(find cob_description)/ros/urdf/sdh_v0/sdh.urdf.xacro" />
   <!-- generic simulator_gazebo plugins for starting mechanism control, ros time, ros battery -->
   <include filename="$(find cob_description)/ros/gazebo/gazebo.urdf.xacro" />
@@ -40,3 +42,6 @@
     <origin xyz="0 0 0.5" rpy="0 0 0" />
   </xacro:cob_lbr_v0>
+  <xacro:cob_sdh_v0 name="sdh" parent="arm_7_link">
+    <origin xyz="0 0 0.02" rpy="0 0 0" />
+  </xacro:cob_sdh_v0>
 </robot>

File: ros/urdf/lbr_v0/lbr.urdf.xacro (robot description, xacro)
@@ -6,6 +6,4 @@
 	<include filename="$(find cob_description)/ros/urdf/lbr_v0/lbr.gazebo.xacro" />
 	<include filename="$(find cob_description)/ros/urdf/lbr_v0/lbr.transmission.xacro" />
-  <!-- cob sdh-->
-  <include filename="$(find cob_description)/ros/urdf/sdh_v0/sdh.urdf.xacro" />
 	<xacro:macro name="cob_lbr_v0" params="parent name *origin">
 		<!-- joint between base_link and arm_0_link -->
@@ -245,7 +243,4 @@
 			</collision>
 		</link>
-  <xacro:cob_sdh_v0 name="sdh" parent="arm_7_link">
-    <origin xyz="0 0 0.02" rpy="0 0 0" />
-  </xacro:cob_sdh_v0>
 		<!-- extensions -->
 		<xacro:cob_lbr_gazebo_v0 name="${name}" />
