Commit message: fixed voxelization + now including sdh

File: ros/robots/lbr_voxelization.urdf.xacro (robot description, xacro)
@@ -12,5 +12,5 @@
   <include filename="$(find cob_description)/ros/urdf/lbr_v0/lbr_voxelization.urdf.xacro" />
   <!-- cob sdh-->
-  <!--include filename="$(find cob_description)/ros/urdf/sdh_v0/sdh_voxelization.urdf.xacro" /-->
+  <include filename="$(find cob_description)/ros/urdf/sdh_v0/sdh_voxelization.urdf.xacro" />
   <!-- generic simulator_gazebo plugins for starting mechanism control, ros time, ros battery -->
   <include filename="$(find cob_description)/ros/gazebo/gazebo.urdf.xacro" />
@@ -44,8 +44,6 @@
     <origin xyz="-0.015982 -0.080992 0.875995" rpy="0.7854 0.0 -0.2618" />
   </xacro:cob_lbr_v0>
-<!--
   <xacro:cob_sdh_v0 name="sdh" parent="arm_7_link">
     <origin xyz="0 0 0.02" rpy="0 0 0" />
   </xacro:cob_sdh_v0>
--->
 </robot>

File: ros/urdf/sdh_v0/sdh.urdf.xacro (robot description, xacro)
@@ -43,5 +43,5 @@
 		<!-- joint between sdh_palm_link and sdh_finger_11_link -->
 		<joint name="${name}_finger_11_joint" type="revolute">
-			<origin xyz="0.01905 0.033 0.0745" rpy="0 0 3.159265" />
+			<origin xyz="0.01905 0.033 0.0745" rpy="0 0 3.14159265" />
 			<parent link="${name}_palm_link"/>
 			<child link="${name}_finger_11_link"/>

File: ros/urdf/sdh_v0/sdh_voxelization.urdf.xacro (robot description, xacro)
@@ -34,19 +34,19 @@
 		</link>
 		<!-- grasp link -->
-		<joint name="${name}_grasp_joint" type="fixed" >
+<!--		<joint name="${name}_grasp_joint" type="fixed" >
 			<origin xyz="0 0 0.15" rpy="0 0 0"/>
 			<parent link="${name}_palm_link" />
 			<child link="${name}_grasp_link" />
 		</joint>
-		<link name="${name}_grasp_link"/>
+		<link name="${name}_grasp_link"/>	-->
 		<!-- finger1 -->
 		<!-- joint between sdh_palm_link and sdh_finger_11_link -->
-		<joint name="${name}_finger_11_joint" type="revolute">
+		<joint name="${name}_finger_1_joint" type="fixed">
 			<origin xyz="0.01905 0.033 0.0745" rpy="0 0 3.159265" />
 			<parent link="${name}_palm_link"/>
 			<child link="${name}_finger_11_link"/>
-			<axis xyz="0 0 1" />
-			<dynamics damping="1" />
-			<limit effort="100" lower="-2" upper="2" velocity="5"/>
+<!--			<axis xyz="0 0 1" />
+			<dynamics damping="1" />
+			<limit effort="100" lower="-2" upper="2" velocity="5"/>		-->
 		</joint>
 		<link name="${name}_finger_11_link">
@@ -61,15 +61,15 @@
 					<mesh filename="package://cob_description/ros/meshes/sdh_v0/knuckle.stl" />
 				</geometry>
-				<material name="Black" />
-			</visual>
-			<collision>
-				<origin xyz="0 0 0.015" rpy="0 0 0" />
-				<geometry>
-					<cylinder radius="0.03" length="0.03"/>
+				<material name="Grey" />
+			</visual>
+			<collision>
+				<origin xyz="0 0 0.09" rpy="0 0 0" />
+				<geometry>
+					<cylinder radius="0.03" length="0.18"/>
 				</geometry>
 			</collision>
 		</link>
 		<!-- joint between sdh_finger_11_link and sdh_finger_12_link -->
-		<joint name="${name}_finger_12_joint" type="revolute">
+<!--		<joint name="${name}_finger_12_joint" type="revolute">
 			<origin xyz="0 0 0.0165" rpy="0 0 0" />
 			<parent link="${name}_finger_11_link"/>
@@ -98,7 +98,7 @@
 				</geometry>
 			</collision>
-		</link>
+		</link>		-->
 		<!-- joint between sdh_finger_12_link and sdh_finger_13_link -->
-		<joint name="${name}_finger_13_joint" type="revolute">
+<!--		<joint name="${name}_finger_13_joint" type="revolute">
 			<origin xyz="0 0 0.0865" rpy="0 0 0" />
 			<parent link="${name}_finger_12_link"/>
@@ -127,14 +127,14 @@
 				</geometry>
 			</collision>
-		</link>
+		</link>		-->
 		<!-- finger2 -->
 		<!-- joint between sdh_palm_link and sdh_finger_21_link -->
-		<joint name="${name}_finger_21_joint" type="revolute">
+		<joint name="${name}_finger_2_joint" type="fixed">
 			<origin xyz="0.01905 -0.033 0.0745" rpy="0 0 3.14159265" />
 			<parent link="${name}_palm_link"/>
 			<child link="${name}_finger_21_link"/>
-			<axis xyz="0 0 1" />
-			<dynamics damping="1" />
-			<limit effort="100" lower="-2" upper="2" velocity="5"/>
+<!--			<axis xyz="0 0 1" />
+			<dynamics damping="1" />
+			<limit effort="100" lower="-2" upper="2" velocity="5"/>		-->
 		</joint>
 		<link name="${name}_finger_21_link">
@@ -149,15 +149,15 @@
 					<mesh filename="package://cob_description/ros/meshes/sdh_v0/knuckle.stl" />
 				</geometry>
-				<material name="Black" />
-			</visual>
-			<collision>
-				<origin xyz="0 0 0.015" rpy="0 0 0" />
-				<geometry>
-					<cylinder radius="0.03" length="0.03"/>
+				<material name="Grey" />
+			</visual>
+			<collision>
+				<origin xyz="0 0 0.09" rpy="0 0 0" />
+				<geometry>
+					<cylinder radius="0.03" length="0.18"/>
 				</geometry>
 			</collision>
 		</link>
 		<!-- joint between sdh_finger_21_link and sdh_finger_22_link -->
-		<joint name="${name}_finger_22_joint" type="revolute">
+<!--		<joint name="${name}_finger_22_joint" type="revolute">
 			<origin xyz="0 0 0.0165" rpy="0 0 0" />
 			<parent link="${name}_finger_21_link"/>
@@ -186,7 +186,7 @@
 				</geometry>
 			</collision>
-		</link>
+		</link>		-->
 		<!-- joint between sdh_finger_22_link and sdh_finger_23_link -->
-		<joint name="${name}_finger_23_joint" type="revolute">
+<!--		<joint name="${name}_finger_23_joint" type="revolute">
 			<origin xyz="0 0 0.0865" rpy="0 0 0" />
 			<parent link="${name}_finger_22_link"/>
@@ -215,5 +215,5 @@
 				</geometry>
 			</collision>
-		</link>
+		</link>		-->
 		<!-- thumb -->
 		<!-- joint between sdh_palm_link and sdh_thumb_1_link -->
@@ -234,15 +234,15 @@
 					<mesh filename="package://cob_description/ros/meshes/sdh_v0/knuckle.stl" />
 				</geometry>
-				<material name="Black" />
-			</visual>
-			<collision>
-				<origin xyz="0 0 0.015" rpy="0 0 0" />
-				<geometry>
-					<cylinder radius="0.03" length="0.03"/>
+				<material name="Grey" />
+			</visual>
+			<collision>
+				<origin xyz="0 0 0.09" rpy="0 0 0" />
+				<geometry>
+					<cylinder radius="0.03" length="0.18"/>
 				</geometry>
 			</collision>
 		</link>
 		<!-- joint between sdh_thumb_1_link and shd_thumb_2_link -->
-		<joint name="${name}_thumb_2_joint" type="revolute">
+<!--		<joint name="${name}_thumb_2_joint" type="revolute">
 		<origin xyz="0 0 0.0165" rpy="0 0 0" />
 		<parent link="${name}_thumb_1_link"/>
@@ -271,7 +271,7 @@
 				</geometry>
 			</collision>
-		</link>
+		</link>		-->
 		<!-- joint between sdh_thumb_2_link and sdh_thumb_3_link -->
-		<joint name="${name}_thumb_3_joint" type="revolute">
+<!--		<joint name="${name}_thumb_3_joint" type="revolute">
 			<origin xyz="0 0 0.0865" rpy="0 0 0" />
 			<parent link="${name}_thumb_2_link"/>
@@ -300,5 +300,5 @@
 				</geometry>
 			</collision>
-		</link>
+		</link>		-->
 		<!-- extensions -->
 		<xacro:cob_sdh_gazebo_v0 name="${name}" />
