Commit message: added virtual camera support

File: ros/robots/cob3-1.urdf.xacro (robot description, xacro)
@@ -40,5 +40,5 @@
   </xacro:cob_arm_v0>
   <xacro:cob_head_cameras_v0 name="head" parent="torso_upper_neck_tilt_link">
-    <origin xyz="0 -0.154 0" rpy="-1.5708 0 0" />
+    <origin xyz="0 -0.154 0" rpy="3.14159 0 0" />
   </xacro:cob_head_cameras_v0>
   <xacro:cob_sdh_v0 name="sdh" parent="arm_7_link">

Commit message: grasp from cooler scenarion running

File: ros/robots/cob3-1.urdf.xacro (robot description, xacro)
@@ -37,5 +37,5 @@
   </xacro:cob_torso_v0>
   <xacro:cob_lbr_v0 name="arm" parent="base_link">
-    <origin xyz="0.040 -0.005 0.83637" rpy="3.1415926 0.7854 -1.8326" />
+    <origin xyz="0.040 -0.005 0.83637" rpy="0.0 0.7854 -1.8326" />
   </xacro:cob_lbr_v0>
   <xacro:cob_head_cameras_v0 name="head" parent="torso_upper_neck_tilt_link">
@@ -43,5 +43,5 @@
   </xacro:cob_head_cameras_v0>
   <xacro:cob_sdh_v0 name="sdh" parent="arm_7_link">
-    <origin xyz="0 0 0" rpy="0 3.1415926 0" />
+    <origin xyz="0 0 0.02" rpy="0 0 0" />
   </xacro:cob_sdh_v0>
 </robot>

Commit message: changed transformation based on box-style-calibration

File: ros/robots/cob3-1.urdf.xacro (robot description, xacro)
@@ -37,5 +37,5 @@
   </xacro:cob_torso_v0>
   <xacro:cob_lbr_v0 name="arm" parent="base_link">
-    <origin xyz="0.040 -0.005 0.83637" rpy="0.0 0.7854 -1.8326" />
+    <origin xyz="0.040 -0.005 0.83637" rpy="0.0 0.7854 -1.6326" />
   </xacro:cob_lbr_v0>
   <xacro:cob_head_cameras_v0 name="head" parent="torso_upper_neck_tilt_link">

Commit message: lbr working on cob

File: ros/robots/cob3-1.urdf.xacro (robot description, xacro)
@@ -44,5 +44,5 @@
   </xacro:cob_head_v0>
   <xacro:cob_sdh_v0 name="sdh" parent="arm_7_link">
-    <origin xyz="0 0 0.02" rpy="0 0 0" />
+    <origin xyz="0 0 0.02" rpy="0 0 1.5708" />
   </xacro:cob_sdh_v0>
 </robot>

File: ros/urdf/lbr_v0/lbr.urdf.xacro (robot description, xacro)
@@ -15,19 +15,19 @@
 		<link name="${name}_0_link">
 			<inertial>
-				<origin xyz="0 0 0.004" rpy="0 0 0"/>
+				<origin xyz="0 0 0.07" rpy="0 0 0"/>
 				<mass value="1.0"/>
 				<inertia ixx="0.01" ixy="0" ixz="0" iyy="0.01" iyz="0" izz="0.01" />
 			</inertial>
 			<visual>
-				<origin xyz="0 0 0.004" rpy="0 0 0" />
-				<geometry>
-					<cylinder radius="0.045" length="0.08"/>
-				</geometry>
-				<material name="Red" />
-			</visual>
-			<collision>
-				<origin xyz="0 0 0.004" rpy="0 0 0" />
-				<geometry>
-					<cylinder radius="0.045" length="0.08"/>
+				<origin xyz="0 0 0.07" rpy="0 0 0" />
+				<geometry>
+					<cylinder radius="0.060" length="0.14"/>
+				</geometry>
+				<material name="Red" />
+			</visual>
+			<collision>
+				<origin xyz="0 0 0.07" rpy="0 0 0" />
+				<geometry>
+					<cylinder radius="0.060" length="0.14"/>
 				</geometry>
 			</collision>
@@ -35,5 +35,5 @@
 		<!-- joint between arm_0_link and arm_1_link -->
 		<joint name="${name}_1_joint" type="revolute">
-		<origin xyz="0 0 0.08" rpy="0 0 -2.7407"/>
+		<origin xyz="0 0 0.14" rpy="0 0 -2.8407"/>
 			<parent link="${name}_0_link"/>
 			<child link="${name}_1_link"/>

Commit message: new stl models for collision added and implemented

File: ros/robots/cob3-1.urdf.xacro (robot description, xacro)
@@ -11,5 +11,5 @@
   <include filename="$(find cob_description)/ros/calibration/cob3-1.urdf.xacro" />
   <!-- cob base -->
-  <include filename="$(find cob_description)/ros/urdf/base_v0/base.urdf.xacro" />
+  <include filename="$(find cob_description)/ros/urdf/base_v1/base.urdf.xacro" />
   <!-- cob torse-->
   <include filename="$(find cob_description)/ros/urdf/torso_v0/torso.urdf.xacro" />

File: ros/urdf/base_v1/base.urdf.xacro (robot description, xacro)
@@ -4,6 +4,6 @@
        xmlns:interface="http://playerstage.sourceforge.net/gazebo/xmlschema/#interface"
        xmlns:xacro="http://ros.org/wiki/xacro">
-  <include filename="$(find cob_description)/ros/urdf/base_v1/base.gazebo.xacro" />
-  <include filename="$(find cob_description)/ros/urdf/base_v1/base.transmission.xacro" />
+  <include filename="$(find cob_description)/ros/urdf/base_v0/base.gazebo.xacro" />
+  <include filename="$(find cob_description)/ros/urdf/base_v0/base.transmission.xacro" />
   <!-- modify here for test -->
   <include filename="$(find cob_description)/ros/urdf/sensors/hokuyo_lx30_laser.urdf.xacro"/>
@@ -15,6 +15,6 @@
   <property name="caster_offset_x" value="0.235" />  <!--modify here-->
   <property name="caster_offset_y" value="0.185" />
-  <property name="caster_offset_z" value="0.0282" />
-  <property name="caster_wheel_offset_y" value="0.049" />
+  <property name="caster_offset_z" value="0.075" />
+  <property name="caster_wheel_offset_y" value="0.000" />
   <property name="wheel_length" value="0.034" />
   <property name="wheel_radius" value="0.074792" />   <!-- This is the 'effective' wheel radius. Wheel radius for uncompressed wheel is 0.079.  mp 20080801 -->
@@ -103,7 +103,7 @@
       </visual>
       <collision>
-        <origin xyz="0 0 0.07" rpy="0.0 0.0 0.0" />
-        <geometry>
-          <box size="0.192 0.164 0.013" />
+        <origin xyz="0 0 0.002" rpy="0.0 0.0 0.0" />
+        <geometry>
+          <box size="0.001 0.001 0.001" />
         </geometry>
       </collision>
@@ -143,5 +143,5 @@
         <origin xyz="0 0 0" rpy="0 0 0" />
         <geometry>
-	      <mesh filename="package://cob_description/ros/meshes/base_v0/base.stl"/>
+	      <mesh filename="package://cob_description/ros/meshes/base_v0/base_collision.stl"/>
           <!--box size="${base_size_x} ${base_size_y} ${base_collision_size_z}" /-->
         </geometry>

File: ros/urdf/lbr_v0/lbr.urdf.xacro (robot description, xacro)
@@ -6,4 +6,6 @@
 	<include filename="$(find cob_description)/ros/urdf/lbr_v0/lbr.gazebo.xacro" />
 	<include filename="$(find cob_description)/ros/urdf/lbr_v0/lbr.transmission.xacro" />
+  <!-- cob sdh-->
+  <include filename="$(find cob_description)/ros/urdf/sdh_v0/sdh.urdf.xacro" />
 	<xacro:macro name="cob_lbr_v0" params="parent name *origin">
 		<!-- joint between base_link and arm_0_link -->
@@ -52,12 +54,12 @@
 				<origin xyz="0 0 0" rpy="0 0 0" />
 				<geometry>
-					<mesh filename="package://cob_description/ros/meshes/lbr_v0/lbr1.stl" />
-				</geometry>
-				<material name="Blue" />
-			</visual>
-			<collision>
-				<origin xyz="0 0 0" rpy="0 0 0" />
-				<geometry>
-					<mesh filename="package://cob_description/ros/meshes/lbr_v0/lbr1.stl" />
+					<mesh filename="package://cob_description/ros/meshes/lbr_v0/joint_1.stl" />
+				</geometry>
+				<material name="Blue" />
+			</visual>
+			<collision>
+				<origin xyz="0 0 0" rpy="0 0 0" />
+				<geometry>
+					<mesh filename="package://cob_description/ros/meshes/lbr_v0/joint_1_collision.stl" />
 				</geometry>
 			</collision>
@@ -82,12 +84,12 @@
 				<origin xyz="0 0 0" rpy="0 0 0" />
 				<geometry>
-					<mesh filename="package://cob_description/ros/meshes/lbr_v0/lbr2.stl" />
-				</geometry>
-				<material name="Red" />
-			</visual>
-			<collision>
-				<origin xyz="0 0 0" rpy="0 0 0" />
-				<geometry>
-					<mesh filename="package://cob_description/ros/meshes/lbr_v0/lbr2.stl"/>
+					<mesh filename="package://cob_description/ros/meshes/lbr_v0/joint_2.stl" />
+				</geometry>
+				<material name="Red" />
+			</visual>
+			<collision>
+				<origin xyz="0 0 0" rpy="0 0 0" />
+				<geometry>
+					<mesh filename="package://cob_description/ros/meshes/lbr_v0/joint_2_collision.stl"/>
 				</geometry>
 			</collision>
@@ -112,12 +114,12 @@
 				<origin xyz="0 0 0" rpy="0 0 0" />
 				<geometry>
-					<mesh filename="package://cob_description/ros/meshes/lbr_v0/lbr3.stl" />
-				</geometry>
-				<material name="Blue" />
-			</visual>
-			<collision>
-				<origin xyz="0 0 0" rpy="0 0 0" />
-				<geometry>
-					<mesh filename="package://cob_description/ros/meshes/lbr_v0/lbr3.stl"/>
+					<mesh filename="package://cob_description/ros/meshes/lbr_v0/joint_3.stl" />
+				</geometry>
+				<material name="Blue" />
+			</visual>
+			<collision>
+				<origin xyz="0 0 0" rpy="0 0 0" />
+				<geometry>
+					<mesh filename="package://cob_description/ros/meshes/lbr_v0/joint_3_collision.stl"/>
 				</geometry>
 			</collision>
@@ -142,12 +144,12 @@
 				<origin xyz="0 0 0" rpy="0 0 0" />
 				<geometry>
-					<mesh filename="package://cob_description/ros/meshes/lbr_v0/lbr4.stl" />
-				</geometry>
-				<material name="Red" />
-			</visual>
-			<collision>
-				<origin xyz="0 0 0" rpy="0 0 0" />
-				<geometry>
-					<mesh filename="package://cob_description/ros/meshes/lbr_v0/lbr4.stl"/>
+					<mesh filename="package://cob_description/ros/meshes/lbr_v0/joint_4.stl" />
+				</geometry>
+				<material name="Red" />
+			</visual>
+			<collision>
+				<origin xyz="0 0 0" rpy="0 0 0" />
+				<geometry>
+					<mesh filename="package://cob_description/ros/meshes/lbr_v0/joint_4_collision.stl"/>
 				</geometry>
 			</collision>
@@ -172,12 +174,12 @@
 				<origin xyz="0 0 0" rpy="0 0 0" />
 				<geometry>
-					<mesh filename="package://cob_description/ros/meshes/lbr_v0/lbr5.stl" />
-				</geometry>
-				<material name="Blue" />
-			</visual>
-			<collision>
-				<origin xyz="0 0 0" rpy="0 0 0" />
-				<geometry>
-					<mesh filename="package://cob_description/ros/meshes/lbr_v0/lbr5.stl"/>
+					<mesh filename="package://cob_description/ros/meshes/lbr_v0/joint_5.stl" />
+				</geometry>
+				<material name="Blue" />
+			</visual>
+			<collision>
+				<origin xyz="0 0 0" rpy="0 0 0" />
+				<geometry>
+					<mesh filename="package://cob_description/ros/meshes/lbr_v0/joint_5_collision.stl"/>
 				</geometry>
 			</collision>
@@ -202,12 +204,12 @@
 				<origin xyz="0 0 0" rpy="0 0 0" />
 				<geometry>
-					<mesh filename="package://cob_description/ros/meshes/lbr_v0/lbr6.stl" />
-				</geometry>
-				<material name="Red" />
-			</visual>
-			<collision>
-				<origin xyz="0 0 0" rpy="0 0 0" />
-				<geometry>
-					<mesh filename="package://cob_description/ros/meshes/lbr_v0/lbr6.stl"/>
+					<mesh filename="package://cob_description/ros/meshes/lbr_v0/joint_6.stl" />
+				</geometry>
+				<material name="Red" />
+			</visual>
+			<collision>
+				<origin xyz="0 0 0" rpy="0 0 0" />
+				<geometry>
+					<mesh filename="package://cob_description/ros/meshes/lbr_v0/joint_6_collision.stl"/>
 				</geometry>
 			</collision>
@@ -232,15 +234,18 @@
 				<origin xyz="0 0 0" rpy="0 0 0" />
 				<geometry>
-					<mesh filename="package://cob_description/ros/meshes/lbr_v0/lbr7.stl" />
-				</geometry>
-				<material name="Blue" />
-			</visual>
-			<collision>
-				<origin xyz="0 0 0" rpy="0 0 0" />
-				<geometry>
-					<mesh filename="package://cob_description/ros/meshes/lbr_v0/lbr7.stl"/>
-				</geometry>
-			</collision>
-		</link>
+					<mesh filename="package://cob_description/ros/meshes/lbr_v0/joint_7.stl" />
+				</geometry>
+				<material name="Blue" />
+			</visual>
+			<collision>
+				<origin xyz="0 0 0" rpy="0 0 0" />
+				<geometry>
+					<mesh filename="package://cob_description/ros/meshes/lbr_v0/joint_7_collision.stl"/>
+				</geometry>
+			</collision>
+		</link>
+  <xacro:cob_sdh_v0 name="sdh" parent="arm_7_link">
+    <origin xyz="0 0 0.02" rpy="0 0 0" />
+  </xacro:cob_sdh_v0>
 		<!-- extensions -->
 		<xacro:cob_lbr_gazebo_v0 name="${name}" />

File: ros/urdf/torso_v0/torso.urdf.xacro (robot description, xacro)
@@ -33,5 +33,5 @@
 				<origin xyz="0 0 0" rpy="0 0 0" />
 				<geometry>
-					<mesh filename="package://cob_description/ros/meshes/torso_v0/tray.stl" />
+					<mesh filename="package://cob_description/ros/meshes/torso_v0/tray_collision.stl" />
 				</geometry>
 			</collision>
@@ -93,5 +93,5 @@
 				<origin xyz="0 0 0" rpy="0 0 0" />
 				<geometry>
-					<mesh filename="package://cob_description/ros/meshes/torso_v0/lower_neck.stl" />
+					<mesh filename="package://cob_description/ros/meshes/torso_v0/lower_neck_collision.stl" />
 				</geometry>
 			</collision>
@@ -153,5 +153,5 @@
 				<origin xyz="0 0 0" rpy="0 0 0" />
 				<geometry>
-					<mesh filename="package://cob_description/ros/meshes/torso_v0/upper_neck.stl" />
+					<mesh filename="package://cob_description/ros/meshes/torso_v0/upper_neck_collision.stl" />
 				</geometry>
 			</collision>
@@ -179,5 +179,5 @@
 				<origin xyz="0 0 0" rpy="0 0 0" />
 				<geometry>
-					<mesh filename="package://cob_description/ros/meshes/torso_v0/head_cover.stl" />
+					<mesh filename="package://cob_description/ros/meshes/torso_v0/head_cover_collision.stl" />
 				</geometry>
 			</collision>

Commit message: alltest launch file

File: ros/robots/cob3-1.urdf.xacro (robot description, xacro)
@@ -8,16 +8,16 @@
   <!-- misc common stuff? -->
   <include filename="$(find cob_description)/ros/urdf/common.xacro" />
-  <!-- cob calibration -->
+  <!-- calibration -->
   <include filename="$(find cob_description)/ros/calibration/cob3-1.urdf.xacro" />
-  <!-- cob base -->
+  <!-- base -->
   <!--include filename="$(find cob_description)/ros/urdf/base_v0/base.urdf.xacro" /-->		<!-- with BOX base-collision model only -->
   <include filename="$(find cob_description)/ros/urdf/base_v1/base.urdf.xacro" />	<!-- new version; platform_controller and platform_navigation not yet working -->
   <!-- torso -->
   <include filename="$(find cob_description)/ros/urdf/torso_v0/torso.urdf.xacro" />
-  <!-- cob head-->
+  <!-- head -->
   <include filename="$(find cob_description)/ros/urdf/head_v0/head.urdf.xacro" />
-  <!-- cob arm-->
+  <!-- arm -->
   <include filename="$(find cob_description)/ros/urdf/lbr_v0/lbr.urdf.xacro" />
-  <!-- cob sdh-->
+  <!-- sdh -->
   <include filename="$(find cob_description)/ros/urdf/sdh_v0/sdh.urdf.xacro" />
   <!-- generic simulator_gazebo plugins for starting mechanism control, ros time, ros battery -->

File: ros/robots/cob3-3.urdf.xacro (robot description, xacro)
@@ -4,5 +4,5 @@
        xmlns:interface="http://playerstage.sourceforge.net/gazebo/xmlschema/#interface"
        xmlns:xacro="http://playerstage.sourceforge.net/gazebo/xmlschema/#interface"
-       name="cob3-2" >
+       name="cob3-3" >
   <!-- The following included files set up definitions of parts of the robot body -->
   <!-- misc common stuff? -->
@@ -11,6 +11,6 @@
   <include filename="$(find cob_description)/ros/calibration/cob3-3.urdf.xacro" />
   <!-- base -->
-  <include filename="$(find cob_description)/ros/urdf/base_v0/base.urdf.xacro" />		<!-- with BOX base-collision model only -->
-  <!--include filename="$(find cob_description)/ros/urdf/base_v1/base.urdf.xacro" /-->	<!-- new version; platform_controller and platform_navigation not yet working -->
+  <!--include filename="$(find cob_description)/ros/urdf/base_v0/base.urdf.xacro" /-->		<!-- with BOX base-collision model only -->
+  <include filename="$(find cob_description)/ros/urdf/base_v1/base.urdf.xacro" />	<!-- new version; platform_controller and platform_navigation not yet working -->
   <!-- torso -->
   <include filename="$(find cob_description)/ros/urdf/torso_v0/torso.urdf.xacro" />
@@ -18,5 +18,5 @@
   <include filename="$(find cob_description)/ros/urdf/head_v0/head.urdf.xacro" />
   <!-- arm -->
-  <include filename="$(find cob_description)/ros/urdf/arm_v0/arm.urdf.xacro" />
+  <include filename="$(find cob_description)/ros/urdf/lbr_v0/lbr.urdf.xacro" />
   <!-- sdh -->
   <include filename="$(find cob_description)/ros/urdf/sdh_v0/sdh.urdf.xacro" />
@@ -33,17 +33,17 @@
        the origin block defines where the component is w.r.t its parent (in this case the parent
        is the world frame). For more, see http://www.ros.org/wiki/xacro -->
-  <xacro:cob_base_v0 name="base"/>
-  <!--xacro:cob_base_v1 name="base"/-->	<!--with new collision_model, but no platform_controller available yet-->
+  <!--<xacro:cob_base_v0 name="base"/-->
+  <xacro:cob_base_v1 name="base"/>	<!--with new collision_model, but no platform_controller available yet-->
   <xacro:cob_torso_v0 name="torso" parent="base_link">
     <origin xyz="0.155 0 0.892" rpy="3.1415926 0 0" />
   </xacro:cob_torso_v0>
-  <xacro:cob_arm_v0 name="arm" parent="base_link">
-    <origin xyz="0.040 -0.005 0.83637" rpy="3.1415926 0.7854 -1.8326" />
-  </xacro:cob_arm_v0>
+  <xacro:cob_lbr_v0 name="arm" parent="base_link">
+    <origin xyz="-0.015982 -0.080992 0.875995" rpy="0.7854 0.0 -0.2618" />
+  </xacro:cob_lbr_v0>
   <xacro:cob_head_v0 name="head" parent="torso_upper_neck_tilt_link">
     <origin xyz="0 -0.154 0" rpy="3.14159 0 0" />
   </xacro:cob_head_v0>
   <xacro:cob_sdh_v0 name="sdh" parent="arm_7_link">
-    <origin xyz="0 0 0" rpy="0 3.1415926 0" />
+    <origin xyz="0 0 0.02" rpy="0 0 1.5708" />
   </xacro:cob_sdh_v0>
 </robot>
