Commit message: fix urdf of cob3-3

File: ros/robots/cob3-3.urdf.xacro (robot description, xacro)
@@ -34,5 +34,5 @@
   <xacro:cob_base_v1 name="base"/>	<!--with new collision_model, but no platform_controller available yet-->
   <xacro:cob_torso_v1 name="torso" parent="base_link">
-    <origin xyz="0.155 0 0.892" rpy="3.1415926 0 0" />
+    <origin xyz="0.155 0 0.892" rpy="1.5708 0 0" />
   </xacro:cob_torso_v1>
   <xacro:cob_lbr_v0 name="arm" parent="base_link">
@@ -40,5 +40,5 @@
   </xacro:cob_lbr_v0>
   <xacro:cob_head_v0 name="head" parent="torso_upper_neck_tilt_link">
-    <origin xyz="0 -0.154 0" rpy="3.14159 0 0" />
+    <origin xyz="0 0.154 0" rpy="3.14159 0 0" />
   </xacro:cob_head_v0>
   <xacro:cob_sdh_v0 name="sdh" parent="arm_7_link">

File: ros/urdf/torso_v1/torso.urdf.xacro (robot description, xacro)
@@ -39,15 +39,14 @@
 		<!-- joint between base_link and torso_lower_neck_tilt_link -->
 		<joint name="${name}_lower_neck_tilt_joint" type="revolute">
-			<!--insert_block name="origin" /-->
-			<origin xyz="0.155 0 0.892" rpy="1.5708 0 0" />
+			<insert_block name="origin" />
 			<parent link="${parent}"/>
 			<child link="${name}_lower_neck_tilt_link"/>
 			<axis xyz="0 0 1" />
+			<dynamics damping="25.0" friction="10.0"/>
 			<calibration rising="${torso_lower_neck_tilt_ref}"/>
-			<dynamics damping="25.0" friction="10.0"/>
 			<limit effort="41.4" lower="-6.2831" upper="6.2831" velocity="0.5"/>
 		</joint>
 		<link name="${name}_lower_neck_tilt_link">
-		<inertial>
+			<inertial>
 				<origin xyz="0 0 0" rpy="0 0 0"/>
 				<mass value="6.209720"/>
@@ -79,5 +78,5 @@
 		</joint>
 		<link name="${name}_pan_link">
-		         <inertial>
+			<inertial>
 				<origin xyz="0 0 0" rpy="0 0 0"/>
 				<mass value="1.0"/>
@@ -98,5 +97,5 @@
 			</collision>
 		</link>
-		<!-- joint between torso_pan_link and torso_upper_neck_link -->
+		<!-- joint between torso_pan_link and torso_upper_neck_tilt_link -->
 		<joint name="${name}_upper_neck_tilt_joint" type="revolute">
 			<origin xyz="0 0 -0.237" rpy="-1.5708 0 0" />
@@ -155,6 +154,6 @@
 		</link>
 		<!-- extensions -->
-		<xacro:cob_torso_gazebo_v0 name="${name}" />
-		<xacro:cob_torso_transmission_v0 name="${name}" />
+		<xacro:cob_torso_gazebo_v1 name="${name}" />
+		<xacro:cob_torso_transmission_v1 name="${name}" />
 	</xacro:macro>
 </robot>
