Commit message: changed angle offset after calibration

File: ros/urdf/lbr_v0/lbr.urdf.xacro (robot description, xacro)
@@ -38,5 +38,5 @@
        <!--joint between arm_0_link and arm_1_link -->
 	<joint name="${name}_1_joint" type="revolute">
-		<origin xyz="0 0 0.18" rpy="0 0 0"/>
+		<origin xyz="0 0 0.18" rpy="0 0 -1.7407"/>
 		<parent link="${name}_0_link"/>
 		<child link="${name}_1_link"/>

Commit message: optimized controllers for simulation

File: ros/urdf/lbr_v0/lbr.urdf.xacro (robot description, xacro)
@@ -43,5 +43,5 @@
 		<axis xyz="0 0 1"/>
 	        <calibration reference_position="${arm_1_ref}"/>
-                <dynamics damping="20" />
+                <dynamics damping="25" />
 		<limit effort="370" velocity="0.4363" lower="-6.2831853" upper="6.2831853"/>
 	</joint>
@@ -73,5 +73,5 @@
 		<axis xyz="0 0 1"/>
 	        <calibration reference_position="${arm_2_ref}"/>
-                <dynamics damping="20" />
+                <dynamics damping="25" />
 		<limit effort="370" velocity="0.4363" lower="-2.0943951" upper="2.0943951"/>
 	</joint>
@@ -103,5 +103,5 @@
 		<axis xyz="0 0 1"/>
 	        <calibration reference_position="${arm_3_ref}"/>
-                <dynamics damping="20" />
+                <dynamics damping="25" />
 		<limit effort="176" velocity="0.4189" lower="-6.2831853" upper="6.2831853"/>
 	</joint>
@@ -133,5 +133,5 @@
 		<axis xyz="0 0 1" />
 	        <calibration reference_position="${arm_4_ref}"/>
-                <dynamics damping="20" />
+                <dynamics damping="25" />
 		<limit effort="176" velocity="0.4189" upper="2.0943951" lower="-2.0943951" />
 	</joint>
@@ -163,5 +163,5 @@
 		<axis xyz="0 0 1" />
 	        <calibration reference_position="${arm_5_ref}"/>
-                <dynamics damping="10" />
+                <dynamics damping="25" />
 		<limit effort="41.6" velocity="0.4363" upper="6.2831853" lower="-6.2831853" />
 	</joint>
@@ -193,5 +193,5 @@
 		<axis xyz="0 0 1" />
 	        <calibration reference_position="${arm_6_ref}"/>
-                <dynamics damping="10" />
+                <dynamics damping="25" />
 		<limit effort="20.1" velocity="0.4363" upper="2.0943951" lower="-2.0943951" />
 	</joint>
@@ -223,5 +223,5 @@
 		<axis xyz="0 0 1" />
 	        <calibration reference_position="${arm_7_ref}"/>
-                <dynamics damping="10" />
+                <dynamics damping="25" />
 		<limit effort="9.6" velocity="0.8727" upper="6.2831853" lower="-6.2831853" />
 	</joint>

Commit message: new trnasformation for base lbr

File: ros/urdf/lbr_v0/lbr.urdf.xacro (robot description, xacro)
@@ -15,19 +15,19 @@
 		<link name="${name}_0_link">
 			<inertial>
-				<origin xyz="0 0 0" rpy="0 0 0"/>
+				<origin xyz="0 0 0.004" rpy="0 0 0"/>
 				<mass value="1.0"/>
 				<inertia ixx="0.01" ixy="0" ixz="0" iyy="0.01" iyz="0" izz="0.01" />
 			</inertial>
 			<visual>
-				<origin xyz="0 0 0.09" rpy="0 0 0" />
-				<geometry>
-					<cylinder radius="0.045" length="0.18"/>
-				</geometry>
-				<material name="Red" />
-			</visual>
-			<collision>
-				<origin xyz="0 0 0.09" rpy="0 0 0" />
-				<geometry>
-					<cylinder radius="0.045" length="0.18"/>
+				<origin xyz="0 0 0.004" rpy="0 0 0" />
+				<geometry>
+					<cylinder radius="0.045" length="0.08"/>
+				</geometry>
+				<material name="Red" />
+			</visual>
+			<collision>
+				<origin xyz="0 0 0.004" rpy="0 0 0" />
+				<geometry>
+					<cylinder radius="0.045" length="0.08"/>
 				</geometry>
 			</collision>
@@ -35,5 +35,5 @@
 		<!-- joint between arm_0_link and arm_1_link -->
 		<joint name="${name}_1_joint" type="revolute">
-		<origin xyz="0 0 0.18" rpy="0 0 -1.7407"/>
+		<origin xyz="0 0 0.08" rpy="0 0 -2.7407"/>
 			<parent link="${name}_0_link"/>
 			<child link="${name}_1_link"/>

Commit message: update joint limits for lbr

File: ros/urdf/lbr_v0/lbr.urdf.xacro (robot description, xacro)
@@ -41,5 +41,5 @@
 			<calibration rising="${arm_1_ref}" falling="${arm_1_ref}"/>
 			<dynamics damping="25" />
-			<limit effort="370" velocity="0.4363" lower="-6.2831853" upper="6.2831853"/>
+			<limit effort="200" velocity="1.9634" lower="-2.9670" upper="2.9670"/>
 		</joint>
 		<link name="${name}_1_link">
@@ -71,5 +71,5 @@
 			<calibration rising="${arm_2_ref}" falling="${arm_2_ref}"/>
 			<dynamics damping="25" />
-			<limit effort="370" velocity="0.4363" lower="-2.0943951" upper="2.0943951"/>
+			<limit effort="200" velocity="1.9634" lower="-2.0943" upper="2.0943"/>
 		</joint>
 		<link name="${name}_2_link">
@@ -101,5 +101,5 @@
 			<calibration rising="${arm_3_ref}" falling="${arm_3_ref}"/>
 			<dynamics damping="25" />
-			<limit effort="176" velocity="0.4189" lower="-6.2831853" upper="6.2831853"/>
+			<limit effort="100" velocity="1.9634" lower="-2.9670" upper="2.9670"/>
 		</joint>
 		<link name="${name}_3_link">
@@ -131,5 +131,5 @@
 			<calibration rising="${arm_4_ref}" falling="${arm_4_ref}"/>
 			<dynamics damping="25" />
-			<limit effort="176" velocity="0.4189" upper="2.0943951" lower="-2.0943951" />
+			<limit effort="100" velocity="1.9634" lower="-2.0943" upper="2.0943" />
 		</joint>
 		<link name="${name}_4_link">
@@ -161,5 +161,5 @@
 			<calibration rising="${arm_5_ref}" falling="${arm_5_ref}"/>
 			<dynamics damping="25" />
-			<limit effort="41.6" velocity="0.4363" upper="6.2831853" lower="-6.2831853" />
+			<limit effort="100" velocity="3.1415926" lower="-2.9670" upper="2.9670" />
 		</joint>
 		<link name="${name}_5_link">
@@ -191,5 +191,5 @@
 			<calibration rising="${arm_6_ref}" falling="${arm_6_ref}"/>
 			<dynamics damping="25" />
-			<limit effort="20.1" velocity="0.4363" upper="2.0943951" lower="-2.0943951" />
+			<limit effort="30" velocity="1.9634" lower="-2.0943951" upper="2.0943951" />
 		</joint>
 		<link name="${name}_6_link">
@@ -221,5 +221,5 @@
 			<calibration rising="${arm_7_ref}" falling="${arm_7_ref}"/>
 			<dynamics damping="25" />
-			<limit effort="9.6" velocity="0.8727" upper="6.2831853" lower="-6.2831853" />
+			<limit effort="30" velocity="1.9634" lower="-2.9670" upper="2.9670" />
 		</joint>
 		<link name="${name}_7_link">

Commit message: added safety_controller for pr2_kinematics

File: ros/urdf/lbr_v0/lbr.urdf.xacro (robot description, xacro)
@@ -42,4 +42,6 @@
 			<dynamics damping="25" />
 			<limit effort="200" velocity="1.9634" lower="-2.9670" upper="2.9670"/>
+			<!--limit effort="370" velocity="0.4363" lower="-6.2831853" upper="6.2831853"/-->
+			<safety_controller k_position="20" k_velocity="25" soft_upper_limit="${2.9670 - 0.10}" soft_lower_limit="${-2.9670 + 0.10}" />
 		</joint>
 		<link name="${name}_1_link">
@@ -72,4 +74,6 @@
 			<dynamics damping="25" />
 			<limit effort="200" velocity="1.9634" lower="-2.0943" upper="2.0943"/>
+			<!--limit effort="370" velocity="0.4363" lower="-2.0943951" upper="2.0943951"/-->
+			<safety_controller k_position="20" k_velocity="50" soft_upper_limit="${2.0943 - 0.10}" 	soft_lower_limit="${-2.0943 + 0.10}" />
 		</joint>
 		<link name="${name}_2_link">
@@ -102,4 +106,6 @@
 			<dynamics damping="25" />
 			<limit effort="100" velocity="1.9634" lower="-2.9670" upper="2.9670"/>
+			<!--limit effort="176" velocity="0.4189" lower="-6.2831853" upper="6.2831853"/-->
+			<safety_controller k_position="20" k_velocity="25" soft_upper_limit="${2.9670 - 0.10}" soft_lower_limit="${-2.9670 + 0.10}" />
 		</joint>
 		<link name="${name}_3_link">
@@ -131,5 +137,7 @@
 			<calibration rising="${arm_4_ref}" falling="${arm_4_ref}"/>
 			<dynamics damping="25" />
-			<limit effort="100" velocity="1.9634" lower="-2.0943" upper="2.0943" />
+			<limit effort="100" velocity="1.9634" lower="-2.0943" upper="2.0943"/>
+			<!--limit effort="176" velocity="0.4189" upper="2.0943951" lower="-2.0943951"/-->
+			<safety_controller k_position="20" k_velocity="25" soft_upper_limit="${2.0943 - 0.10}" soft_lower_limit="${-2.0943 + 0.10}" />
 		</joint>
 		<link name="${name}_4_link">
@@ -162,4 +170,6 @@
 			<dynamics damping="25" />
 			<limit effort="100" velocity="3.1415926" lower="-2.9670" upper="2.9670" />
+			<!--limit effort="41.6" velocity="0.4363" upper="6.2831853" lower="-6.2831853" /-->
+			<safety_controller k_position="20" k_velocity="25" soft_upper_limit="${2.9670 - 0.10}" soft_lower_limit="${-2.9670 + 0.10}" />
 		</joint>
 		<link name="${name}_5_link">
@@ -192,4 +202,6 @@
 			<dynamics damping="25" />
 			<limit effort="30" velocity="1.9634" lower="-2.0943951" upper="2.0943951" />
+			<!--limit effort="20.1" velocity="0.4363" upper="2.0943951" lower="-2.0943951" /-->
+			<safety_controller k_position="20" k_velocity="25" soft_upper_limit="${2.0943951 - 0.10}" soft_lower_limit="${-2.0943951 + 0.10}" />
 		</joint>
 		<link name="${name}_6_link">
@@ -222,4 +234,6 @@
 			<dynamics damping="25" />
 			<limit effort="30" velocity="1.9634" lower="-2.9670" upper="2.9670" />
+			<!--limit effort="20.1" velocity="0.4363" upper="2.0943951" lower="-2.0943951" /-->
+			<safety_controller k_position="20" k_velocity="25" soft_upper_limit="${2.9670 - 0.10}" soft_lower_limit="${-2.9670 + 0.10}" />
 		</joint>
 		<link name="${name}_7_link">

Commit message: tuned gazebo controller

File: ros/urdf/lbr_v0/lbr.urdf.xacro (robot description, xacro)
@@ -40,8 +40,8 @@
 			<axis xyz="0 0 1"/>
 			<calibration rising="${arm_1_ref}"/>
-			<dynamics damping="1" />
+			<dynamics damping="10" />
 			<limit effort="200" velocity="1.9634" lower="-2.9670" upper="2.9670"/>
 			<!--limit effort="370" velocity="0.4363" lower="-6.2831853" upper="6.2831853"/-->
-			<safety_controller k_position="20" k_velocity="25" soft_lower_limit="${-2.9670 + 0.10}" soft_upper_limit="${2.9670 - 0.10}" />
+			<safety_controller k_position="20" k_velocity="50" soft_lower_limit="${-2.9670 + 0.01}" soft_upper_limit="${2.9670 - 0.01}" />
 		</joint>
 		<link name="${name}_1_link">
@@ -72,7 +72,7 @@
 			<axis xyz="0 0 1"/>
 			<calibration rising="${arm_2_ref}"/>
-			<dynamics damping="1" />
+			<dynamics damping="10" />
 			<limit effort="200" velocity="1.9634" lower="-2.0943" upper="2.0943"/>
-			<safety_controller k_position="20" k_velocity="50" soft_lower_limit="${-2.0943 + 0.10}" 	soft_upper_limit="${2.0943 - 0.10}" />
+			<safety_controller k_position="20" k_velocity="50" soft_lower_limit="${-2.0943 + 0.01}" 	soft_upper_limit="${2.0943 - 0.01}" />
 		</joint>
 		<link name="${name}_2_link">
@@ -103,8 +103,8 @@
 			<axis xyz="0 0 1"/>
 			<calibration rising="${arm_3_ref}"/>
-			<dynamics damping="1" />
+			<dynamics damping="5" />
 			<limit effort="100" velocity="1.9634" lower="-2.9670" upper="2.9670"/>
 			<!--limit effort="176" velocity="0.4189" lower="-6.2831853" upper="6.2831853"/-->
-			<safety_controller k_position="20" k_velocity="25" soft_lower_limit="${-2.9670 + 0.10}" soft_upper_limit="${2.9670 - 0.10}" />
+			<safety_controller k_position="20" k_velocity="25" soft_lower_limit="${-2.9670 + 0.01}" soft_upper_limit="${2.9670 - 0.01}" />
 		</joint>
 		<link name="${name}_3_link">
@@ -135,8 +135,8 @@
 			<axis xyz="0 0 1" />
 			<calibration rising="${arm_4_ref}"/>
-			<dynamics damping="1" />
+			<dynamics damping="5" />
 			<limit effort="100" velocity="1.9634" lower="-2.0943" upper="2.0943"/>
 			<!--limit effort="176" velocity="0.4189" upper="2.0943951" lower="-2.0943951"/-->
-			<safety_controller k_position="20" k_velocity="25" soft_lower_limit="${-2.0943 + 0.10}" soft_upper_limit="${2.0943 - 0.10}" />
+			<safety_controller k_position="20" k_velocity="25" soft_lower_limit="${-2.0943 + 0.01}" soft_upper_limit="${2.0943 - 0.01}" />
 		</joint>
 		<link name="${name}_4_link">
@@ -167,8 +167,8 @@
 			<axis xyz="0 0 1" />
 			<calibration rising="${arm_5_ref}"/>
-			<dynamics damping="1" />
+			<dynamics damping="5" />
 			<limit effort="100" velocity="1.9634" lower="-2.9670" upper="2.9670" />
 			<!--limit effort="41.6" velocity="0.4363" upper="6.2831853" lower="-6.2831853" /-->
-			<safety_controller k_position="20" k_velocity="25" soft_lower_limit="${-2.9670 + 0.10}" soft_upper_limit="${2.9670 - 0.10}" />
+			<safety_controller k_position="20" k_velocity="25" soft_lower_limit="${-2.9670 + 0.01}" soft_upper_limit="${2.9670 - 0.01}" />
 		</joint>
 		<link name="${name}_5_link">
@@ -199,8 +199,8 @@
 			<axis xyz="0 0 1" />
 			<calibration rising="${arm_6_ref}"/>
-			<dynamics damping="1" />
+			<dynamics damping="5" />
 			<limit effort="30" velocity="1.9634" lower="-2.0943951" upper="2.0943951" />
 			<!--limit effort="20.1" velocity="0.4363" upper="2.0943951" lower="-2.0943951" /-->
-			<safety_controller k_position="20" k_velocity="25" soft_lower_limit="${-2.0943951 + 0.10}" soft_upper_limit="${2.0943951 - 0.10}" />
+			<safety_controller k_position="20" k_velocity="25" soft_lower_limit="${-2.0943951 + 0.01}" soft_upper_limit="${2.0943951 - 0.01}" />
 		</joint>
 		<link name="${name}_6_link">
@@ -231,8 +231,8 @@
 			<axis xyz="0 0 1" />
 			<calibration rising="${arm_7_ref}"/>
-			<dynamics damping="1" />
+			<dynamics damping="5" />
 			<limit effort="30" velocity="1.9634" lower="-2.9670" upper="2.9670" />
 			<!--limit effort="20.1" velocity="0.4363" upper="2.0943951" lower="-2.0943951" /-->
-			<safety_controller k_position="20" k_velocity="25" soft_lower_limit="${-2.9670 + 0.10}" soft_upper_limit="${2.9670 - 0.10}" />
+			<safety_controller k_position="20" k_velocity="25" soft_lower_limit="${-2.9670 + 0.01}" soft_upper_limit="${2.9670 - 0.01}" />
 		</joint>
 		<link name="${name}_7_link">

Commit message: reduced mass for simulation

File: ros/urdf/lbr_v0/lbr.urdf.xacro (robot description, xacro)
@@ -48,5 +48,6 @@
 			<inertial>
 				<origin xyz="0 0 0" rpy="0 0 0" />
-				<mass value="5.9907"/>
+				<!--mass value="5.9907"/-->
+				<mass value="2.0"/>
 				<inertia ixx="0.01" ixy="0" ixz="0" iyy="0.01" iyz="0" izz="0.01" />
 			</inertial>
@@ -79,5 +80,6 @@
 			<inertial>
 				<origin xyz="0 0 0" rpy="0 0 0"/>
-				<mass value="5.734939"/>
+				<!--mass value="5.734939"/-->
+				<mass value="2.0"/>
 				<inertia ixx="0.03" ixy="0" ixz="0" iyy="0.03" iyz="0" izz="0.03" />
 			</inertial>
@@ -111,5 +113,6 @@
 			<inertial>
 				<origin xyz="0 0 0" rpy="0 0 0"/>
-				<mass value="4.214668"/>
+				<!--mass value="4.214668"/-->
+				<mass value="2.0"/>
 				<inertia ixx="0.03" ixy="0" ixz="0" iyy="0.03" iyz="0" izz="0.03" />
 			</inertial>
@@ -143,5 +146,6 @@
 			<inertial>
 				<origin xyz="0 0 0" rpy="0 0 0"/>
-				<mass value="3.669819"/>
+				<!--mass value="3.669819"/-->
+				<mass value="2.0"/>
 				<inertia ixx="0.03" ixy="0" ixz="0" iyy="0.03" iyz="0" izz="0.03" />
 			</inertial>
