Commit message: modified camera coordinate systems

File: ros/calibration/cob3-2.urdf.xacro (robot description, xacro)
@@ -19,3 +19,21 @@
   <property name="arm_6_ref" value="-1.6167" />
   <property name="arm_7_ref" value="8.1075" />
+  <property name="cam_r_x" value="0.0" />
+  <property name="cam_r_y" value="0.0" />
+  <property name="cam_r_z" value="0.0" />
+  <property name="cam_r_roll" value="0.0" />
+  <property name="cam_r_pitch" value="0.0" />
+  <property name="cam_r_yaw" value="0.0" />
+  <property name="cam_l_x" value="0.0" />
+  <property name="cam_l_y" value="0.0" />
+  <property name="cam_l_z" value="0.0" />
+  <property name="cam_l_roll" value="0.0" />
+  <property name="cam_l_pitch" value="0.0" />
+  <property name="cam_l_yaw" value="0.0" />
+  <property name="tof_x" value="0.0" />
+  <property name="tof_y" value="0.0" />
+  <property name="tof_z" value="0.0" />
+  <property name="tof_roll" value="0.0" />
+  <property name="tof_pitch" value="0.0" />
+  <property name="tof_yaw" value="0.0" />
 </robot>

File: ros/robots/cob3-2.urdf.xacro (robot description, xacro)
@@ -40,5 +40,5 @@
   </xacro:cob_arm_v0>
   <xacro:cob_head_cameras_v0 name="head" parent="torso_upper_neck_tilt_link">
-    <origin xyz="0 -0.154 0" rpy="-1.5708 0 0" />
+    <origin xyz="0 -0.154 0" rpy="3.14159 0 0" />
   </xacro:cob_head_cameras_v0>
   <xacro:cob_sdh_v0 name="sdh" parent="arm_7_link">

File: ros/urdf/head_cameras_v0/head_cameras.urdf.xacro (robot description, xacro)
@@ -44,13 +44,13 @@
     <!--##################################################-->
     <!-- camera test here -->
-    <xacro:cob_cameraone_v0 name="${name}_color_camera_l" parent="${name}_camera_axis_link">
-      <origin xyz="0 0.03 -0.003" rpy="0 0 0" />
+    <xacro:cob_cameraone_v0 name="${name}_color_camera_l" parent="${name}_color_camera_r_link">
+      <origin xyz="${cam_l_x-0.12} ${cam_l_y} ${cam_l_z}" rpy="${cam_l_roll} ${cam_l_pitch} ${cam_l_yaw}" />
     </xacro:cob_cameraone_v0>
     <xacro:cob_cameraone_v0 name="${name}_color_camera_r" parent="${name}_camera_axis_link">
-      <origin xyz="0 -0.03 -0.003" rpy="0 0 0" />
+      <origin xyz="${cam_r_x} ${cam_r_y} ${cam_r_z+0.06}" rpy="${cam_r_roll} ${cam_r_pitch-1.5708} ${cam_r_yaw+3.14159}" />
     </xacro:cob_cameraone_v0>
     <!-- hokuyo_SR400_laser test here-->
-    <xacro:hokuyo_SR400_laser_v0 name="${name}_tof_camera" parent="${name}_camera_axis" ros_topic="head_scan" update_rate="54" min_angle="-0.302" max_angle="0.302" >
-      <origin xyz="0 0 0" rpy="0 0 0" />
+    <xacro:hokuyo_SR400_laser_v0 name="${name}_tof_camera" parent="${name}_color_camera_r_link" ros_topic="head_scan" update_rate="54" min_angle="-0.302" max_angle="0.302" >
+      <origin xyz="${tof_x-0.06} ${tof_y} ${tof_z}" rpy="${tof_roll} ${tof_pitch} ${tof_yaw}" />
     </xacro:hokuyo_SR400_laser_v0>
     <!-- extensions -->

File: ros/urdf/sensors/cameraone.gazebo.xacro (robot description, xacro)
@@ -5,5 +5,5 @@
       xmlns:xacro="http://ros.org/wiki/xacro">
 <xacro:macro name="cob_cameraone_gazebo_v0" params="name">
-  <gazebo reference="${name}_frame">
+  <gazebo reference="${name}_link">
     <sensor:camera name="${name}_sensor">
       <imageFormat>R8G8B8</imageFormat>

File: ros/urdf/sensors/cameraone.urdf.xacro (robot description, xacro)
@@ -10,7 +10,7 @@
       <insert_block name="origin" />
       <parent link="${parent}"/>
-      <child link="${name}_frame"/>
+      <child link="${name}_link"/>
     </joint>
-    <link name="${name}_frame">
+    <link name="${name}_link">
       <inertial>
         <mass value="0.01" />

File: ros/urdf/sensors/hokuyo_SR400_laser.urdf.xacro (robot description, xacro)
@@ -9,5 +9,5 @@
       <axis xyz="0 1 0" />
       <insert_block name="origin" />
-      <parent link="${parent}_link"/>
+      <parent link="${parent}"/>
       <child link="${name}_link"/>
     </joint>

Commit message: update on robot

File: ros/calibration/cob3-2.urdf.xacro (robot description, xacro)
@@ -13,11 +13,11 @@
 	<property name="head_camera_axis_ref" value="-3.14" />
 	<!-- arm reference positions -->
-	<property name="arm_1_ref" value="8.1252" />
-	<property name="arm_2_ref" value="0.6454" />
-	<property name="arm_3_ref" value="-4.9119" />
-	<property name="arm_4_ref" value="-0.8774" />
-	<property name="arm_5_ref" value="-0.3908" />
-	<property name="arm_6_ref" value="-1.6167" />
-	<property name="arm_7_ref" value="8.1075" />
+	<property name="arm_1_ref" value="-2.8761" />
+	<property name="arm_2_ref" value="-0.1687" />
+	<property name="arm_3_ref" value="-0.0274" />
+	<property name="arm_4_ref" value="-1.7193" />
+	<property name="arm_5_ref" value="0.0342" />
+	<property name="arm_6_ref" value="-1.6959" />
+	<property name="arm_7_ref" value="1.8707" />
 	<!-- camera calibration properties -->
 	<property name="cam_r_x" value="0.0" />

File: ros/urdf/arm_v0/arm.urdf.xacro (robot description, xacro)
@@ -38,5 +38,5 @@
        <!--joint between arm_0_link and arm_1_link -->
 	<joint name="${name}_1_joint" type="revolute">
-		<origin xyz="0 0 -0.250" rpy="0 0 0"/>
+		<origin xyz="0 0 -0.250" rpy="0 0 3.1415926"/>
 		<parent link="${name}_0_link"/>
 		<child link="${name}_1_link"/>
