Commit message: new stl files for torso

File: ros/calibration/cob3-1.urdf.xacro (robot description, xacro)
@@ -3,8 +3,8 @@
   <property name="M_PI" value="3.1415926535897931" />
   <!-- torso reference position -->
-  <property name="torso_lower_neck_pan_ref" value="-0.5149" />
-  <property name="torso_lower_neck_tilt_ref" value="0.0344" />
-  <property name="torso_upper_neck_pan_ref" value="0.0247" />
-  <property name="torso_upper_neck_tilt_ref" value="0.022078" />
+  <property name="torso_lower_neck_pan_ref" value="-0.5306" />
+  <property name="torso_lower_neck_tilt_ref" value="0.0320" />
+  <property name="torso_upper_neck_pan_ref" value="0.5481" />
+  <property name="torso_upper_neck_tilt_ref" value="0.0229" />
   <!-- tray reference position -->
   <property name="torso_tray_ref" value="0.0" />

File: ros/robots/cob_platform.urdf.xacro (robot description, xacro)
@@ -34,5 +34,5 @@
   <xacro:cob_base_v0 name="base"/>
   <xacro:cob_torso_v0 name="torso" parent="base_link">
-    <origin xyz="0.24627 0 0.7798" rpy="0 0 0" />
+    <origin xyz="0.24627 0 0.7798" rpy="3.1415926 0 0" />
   </xacro:cob_torso_v0>
   <xacro:cob_head_cameras_v0 name="head" parent="torso_upper_neck_tilt_link">

File: ros/urdf/torso_v0/torso.urdf.xacro (robot description, xacro)
@@ -73,8 +73,8 @@
     <!--joint between torso_lower_neck_pan_link and torso_lower_neck_tilt_link-->
     <joint name="${name}_lower_neck_tilt_joint" type="revolute">
-      <origin xyz="0 0 0" rpy="0 0.293 0" />   <!--FIX pitch angle Later-->
+      <origin xyz="0 0 0" rpy="1.5708 0 0" />   <!--FIX pitch angle Later-->
       <parent link="${name}_lower_neck_pan_link"/>
       <child link="${name}_lower_neck_tilt_link"/>
-      <axis xyz="0 1 0" />
+      <axis xyz="0 0 1" />
       <dynamics damping="0.1" />
       <calibration reference_position="${torso_lower_neck_tilt_ref}"/>
@@ -91,5 +91,5 @@
 	 <origin xyz="0 0 0" rpy="0 0 0" />
 	 <geometry>
-	    <mesh filename="package://cob_defs/common/files/meshes/neck.stl" />
+	    <mesh filename="package://cob_description/ros/meshes/torso_v0/lower_neck.stl" />
 	 </geometry>
          <material name="Red" />
@@ -98,5 +98,5 @@
 	 <origin xyz="0 0 0" rpy="0 0 0" />
 	 <geometry>
-	    <mesh filename="package://cob_defs/common/files/meshes/neck.stl" />
+	    <mesh filename="package://cob_description/ros/meshes/torso_v0/lower_neck.stl" />
 	 </geometry>
        </collision>
@@ -104,5 +104,5 @@
     <!--joint between torso_lower_neck_tilt_link and torso_upper_neck_pan_link-->
     <joint name="${name}_upper_neck_pan_joint" type="revolute">
-      <origin xyz="-0.09039 0 0.30489" rpy="0 0 0" />
+      <origin xyz="-0.09039 -0.30489 0" rpy="-1.5708 0 0" />
       <parent link="${name}_lower_neck_tilt_link"/>
       <child link="${name}_upper_neck_pan_link"/>
@@ -134,8 +134,8 @@
     <!--joint between torso_upper_neck_pan_link and torso_upper_neck_tilt_link-->
     <joint name="${name}_upper_neck_tilt_joint" type="revolute">
-      <origin xyz="0 0 0" rpy="0 -0.26 0" /> <!---0.392699075-->
+      <origin xyz="0 0 0" rpy="1.5708 0 0" /> <!---0.392699075-->
       <parent link="${name}_upper_neck_pan_link"/>
       <child link="${name}_upper_neck_tilt_link"/>
-      <axis xyz="0 1 0" />
+      <axis xyz="0 0 1" />
       <dynamics damping="0.1" />
       <calibration reference_position="${torso_upper_neck_tilt_ref}"/>
@@ -151,5 +151,5 @@
 	   <origin xyz="0 0 0" rpy="0 0 0" />
 	   <geometry>
-              <mesh filename="package://cob_defs/common/files/meshes/head.stl" />
+			<mesh filename="package://cob_description/ros/meshes/torso_v0/upper_neck.stl" />
 	   </geometry>
            <material name="Grey" />
@@ -158,5 +158,5 @@
 	   <origin xyz="0 0 0" rpy="0 0 0" />
 	   <geometry>
-              <mesh filename="package://cob_defs/common/files/meshes/head.stl" />
+			<mesh filename="package://cob_description/ros/meshes/torso_v0/upper_neck.stl" />
 	   </geometry>
 	</collision>

Commit message: adaptions to urdf for tray

File: ros/calibration/cob3-1.urdf.xacro (robot description, xacro)
@@ -8,5 +8,5 @@
   <property name="torso_upper_neck_tilt_ref" value="0.0229" />
   <!-- tray reference position -->
-  <property name="torso_tray_ref" value="0.0" />
+  <property name="torso_tray_ref" value="2.5541" />
   <!-- head cameras reference position -->
   <property name="head_camera_axis_ref" value="-3.14" />

File: ros/urdf/torso_v0/torso.urdf.xacro (robot description, xacro)
@@ -12,5 +12,5 @@
     <!--joint between base_link and torso_tray_link -->
     <joint name="${name}_tray_joint" type="revolute">
-       <origin xyz="0.21864 0.20061 0.83196" rpy="-0.707 0 0" />
+       <origin xyz="0.016 0.192 0.680" rpy="2.4346 0 0" />
        <parent link="${parent}"/>
        <child link="${name}_tray_link"/>
@@ -18,5 +18,5 @@
        <calibration reference_position="${torso_tray_ref}"/>
        <dynamics damping="5.0" friction="0.5"/>
-       <limit effort="100" lower="0" upper="3.31612" velocity="5"/>
+       <limit effort="100" lower="-3.31612" upper="0" velocity="5"/>
     </joint>
     <link name="${name}_tray_link">
@@ -29,5 +29,5 @@
 	 <origin xyz="0 0 0" rpy="0.707 0 0" />
 	 <geometry>
-	    <mesh filename="package://cob_defs/common/files/meshes/tray.stl" />
+	    <mesh filename="package://cob_description/ros/meshes/torso_v0/tray.stl" />
 	 </geometry>
          <material name="Green" />
@@ -36,5 +36,5 @@
 	 <origin xyz="0 0 0" rpy="0.707 0 0" />
 	 <geometry>
-	  <mesh filename="package://cob_defs/common/files/meshes/tray.stl" />
+	    <mesh filename="package://cob_description/ros/meshes/torso_v0/tray.stl" />
 	 </geometry>
        </collision>

Commit message: preparations for cameras and tof in simulation

File: ros/calibration/cob3-1.urdf.xacro (robot description, xacro)
@@ -11,5 +11,5 @@
 	<property name="torso_tray_ref" value="2.5541" />
 	<!-- head camera axis reference position -->
-	<property name="head_camera_axis_ref" value="-3.14" />
+	<property name="head_axis_ref" value="-3.14" />
 	<!-- arm reference positions -->
 	<property name="arm_1_ref" value="1.47881" />

File: ros/robots/cob3-1.urdf.xacro (robot description, xacro)
@@ -14,6 +14,6 @@
   <!-- cob torse-->
   <include filename="$(find cob_description)/ros/urdf/torso_v0/torso.urdf.xacro" />
-  <!-- cob cameras-->
-  <include filename="$(find cob_description)/ros/urdf/head_cameras_v0/head_cameras.urdf.xacro" />
+  <!-- cob head-->
+  <include filename="$(find cob_description)/ros/urdf/head_v0/head.urdf.xacro" />
   <!-- cob arm-->
   <include filename="$(find cob_description)/ros/urdf/lbr_v0/lbr.urdf.xacro" />
@@ -39,7 +39,7 @@
     <origin xyz="0.040 -0.005 0.83637" rpy="0.0 0.7854 -1.6326" />
   </xacro:cob_lbr_v0>
-  <xacro:cob_head_cameras_v0 name="head" parent="torso_upper_neck_tilt_link">
+  <xacro:cob_head_v0 name="head" parent="torso_upper_neck_tilt_link">
     <origin xyz="0 -0.154 0" rpy="3.14159 0 0" />
-  </xacro:cob_head_cameras_v0>
+  </xacro:cob_head_v0>
   <xacro:cob_sdh_v0 name="sdh" parent="arm_7_link">
     <origin xyz="0 0 0.02" rpy="0 0 0" />

File: ros/urdf/head_v0/head.gazebo.xacro (robot description, xacro)
@@ -4,10 +4,9 @@
        xmlns:interface="http://playerstage.sourceforge.net/gazebo/xmlschema/#interface"
        xmlns:xacro="http://ros.org/wiki/xacro">
-  <xacro:macro name="cob_head_cameras_transmission_v0" params="name">
-    <transmission name="${name}_camera_axis_trans" type="pr2_mechanism_model/SimpleTransmission">
-		<actuator name="${name}_camera_axis_motor"/>
-		<joint name="${name}_camera_axis_joint"/>
-		<mechanicalReduction>1</mechanicalReduction>
-    </transmission>
+  <xacro:macro name="cob_head_gazebo_v0" params="name">
+    <gazebo reference="${name}_axis_link">
+      <material>Gazebo/Green</material>
+      <turnGravityOff>false</turnGravityOff>
+    </gazebo>
   </xacro:macro>
 </robot>

File: ros/urdf/head_v0/head.transmission.xacro (robot description, xacro)
@@ -4,9 +4,10 @@
        xmlns:interface="http://playerstage.sourceforge.net/gazebo/xmlschema/#interface"
        xmlns:xacro="http://ros.org/wiki/xacro">
-  <xacro:macro name="cob_head_cameras_gazebo_v0" params="name">
-    <gazebo reference="${name}_camera_axis_link">
-      <material>PR2/Green</material>
-      <turnGravityOff>false</turnGravityOff>
-    </gazebo>
+  <xacro:macro name="cob_head_transmission_v0" params="name">
+    <transmission name="${name}_axis_trans" type="pr2_mechanism_model/SimpleTransmission">
+		<actuator name="${name}_axis_motor"/>
+		<joint name="${name}_axis_joint"/>
+		<mechanicalReduction>1</mechanicalReduction>
+    </transmission>
   </xacro:macro>
 </robot>

File: ros/urdf/head_v0/head.urdf.xacro (robot description, xacro)
@@ -4,6 +4,6 @@
        xmlns:interface="http://playerstage.sourceforge.net/gazebo/xmlschema/#interface"
        xmlns:xacro="http://ros.org/wiki/xacro">
-  <include filename="$(find cob_description)/ros/urdf/head_cameras_v0/head_cameras.gazebo.xacro" />
-  <include filename="$(find cob_description)/ros/urdf/head_cameras_v0/head_cameras.transmission.xacro" />
+  <include filename="$(find cob_description)/ros/urdf/head_v0/head.gazebo.xacro" />
+  <include filename="$(find cob_description)/ros/urdf/head_v0/head.transmission.xacro" />
   <include filename="$(find cob_description)/ros/urdf/sensors/cameraone.urdf.xacro" />
   <include filename="$(find cob_description)/ros/urdf/sensors/hokuyo_SR400_laser.urdf.xacro" />
@@ -11,16 +11,16 @@
                        <!--Fix Some Parameters Later-->
 <!--####################################################################-->
-  <xacro:macro name="cob_head_cameras_v0" params="name parent *origin">
-    <!--joint between torso_upper_neck_tilt_link and head_camera_axis_link-->
-    <joint name="${name}_camera_axis_joint" type="revolute">
+  <xacro:macro name="cob_head_v0" params="name parent *origin">
+    <!--joint between torso_upper_neck_tilt_link and head_axis_link-->
+    <joint name="${name}_axis_joint" type="revolute">
        <insert_block name="origin" />
        <parent link="${parent}"/>
-       <child link="${name}_camera_axis_link"/>
-       <axis xyz="0 1 0" />
+       <child link="${name}_axis_link"/>
+       <axis xyz="0 0 1" />
        <dynamics damping="0.1" />
-       <calibration rising="${head_camera_axis_ref}" falling="${head_camera_axis_ref}"/>
+       <calibration rising="${head_axis_ref}" falling="${head_axis_ref}"/>
        <limit effort="100" lower="-1.5" upper="3.316" velocity="0.5"/>
     </joint>
-	<link name="${name}_camera_axis_link">
+	<link name="${name}_axis_link">
 		<inertial>
 			<origin xyz="0 0 0" rpy="0 0 0"/>
@@ -42,4 +42,34 @@
 		</collision>
 	</link>
+	<!--joint between head_axis_link and head_tof_axis_link-->
+	<joint name="${name}_tof_tilt_joint" type="revolute">
+		<origin xyz="0 0 0" rpy="0 0 0" />
+		<parent link="${name}_tof_camera_link"/>
+		<child link="${name}_tof_axis_link"/>
+		<axis xyz="0 0 1" />
+		<dynamics damping="25.0" friction="10.0"/>
+		<calibration rising="0" falling="0"/>
+		<limit effort="46" lower="-1.5" upper="1.5" velocity="0.5"/>
+	</joint>
+	<link name="${name}_tof_tilt_link">
+		<inertial>
+			<origin xyz="0 0 0" rpy="0 0 0"/>
+			<mass value="1.0"/>
+			<inertia ixx="0.1" ixy="0.0" ixz="0.0" iyy="0.1" iyz="0.0" izz="0.1" />
+		</inertial>
+		<visual>
+			<origin xyz="0 0 0" rpy="0 0 0" />
+			<geometry>
+				<box size="0.1 0.1 0.01"/>
+			</geometry>
+			<material name="Red" />
+		</visual>
+		<collision>
+			<origin xyz="0 0 0" rpy="0 0 0" />
+			<geometry>
+				<box size="0.1 0.1 0.01"/>
+			</geometry>
+		</collision>
+	</link>
     <!--##################################################-->
     <!-- camera test here -->
@@ -47,5 +77,5 @@
       <origin xyz="${cam_l_x-0.12} ${cam_l_y} ${cam_l_z}" rpy="${cam_l_roll} ${cam_l_pitch} ${cam_l_yaw}" />
     </xacro:cob_cameraone_v0>
-    <xacro:cob_cameraone_v0 name="${name}_color_camera_r" parent="${name}_camera_axis_link">
+    <xacro:cob_cameraone_v0 name="${name}_color_camera_r" parent="${name}_axis_link">
       <origin xyz="${cam_r_x} ${cam_r_y} ${cam_r_z-0.06}" rpy="${cam_r_roll} ${cam_r_pitch+1.5708} ${cam_r_yaw+3.14159}" />
     </xacro:cob_cameraone_v0>
@@ -55,6 +85,6 @@
     </xacro:hokuyo_SR400_laser_v0>
     <!-- extensions -->
-    <xacro:cob_head_cameras_gazebo_v0 name="${name}" />
-    <xacro:cob_head_cameras_transmission_v0 name="${name}" />
+    <xacro:cob_head_gazebo_v0 name="${name}" />
+    <xacro:cob_head_transmission_v0 name="${name}" />
   </xacro:macro>
 </robot>

Commit message: small modification for dashboard

File: ros/calibration/cob3-1.urdf.xacro (robot description, xacro)
@@ -39,3 +39,10 @@
 	<property name="tof_pitch" value="-0.0029" />
 	<property name="tof_yaw" value="-0.0058" />
+	<!-- head_kinect_link is identical to head_tof_link -->
+	<property name="kinect_x" value="0.0" />
+	<property name="kinect_y" value="0.0" />
+	<property name="kinect_z" value="0.0" />
+	<property name="kinect_roll" value="0.0" />
+	<property name="kinect_pitch" value="0.0" />
+	<property name="kinect_yaw" value="0.0" />
 </robot>

File: ros/urdf/head_v0/head.urdf.xacro (robot description, xacro)
@@ -8,4 +8,5 @@
 	<include filename="$(find cob_description)/ros/urdf/sensors/prosilica.urdf.xacro" />
 	<include filename="$(find cob_description)/ros/urdf/sensors/tof.urdf.xacro" />
+	<include filename="$(find cob_description)/ros/urdf/sensors/kinect.urdf.xacro" />
 	<!--include filename="$(find cob_description)/ros/urdf/sensors/hokuyo_SR400_laser.urdf.xacro" /-->
 	<xacro:macro name="cob_head_v0" params="name parent *origin">
@@ -52,4 +53,8 @@
 			<origin xyz="${tof_x-0.06} ${tof_y} ${tof_z}" rpy="${tof_roll} ${tof_pitch} ${tof_yaw}" />
 		</xacro:cob_tof_v0>
+		<!-- kinect_trial -->
+		<xacro:cob_kinect_v0 name="${name}_kinect" parent="${name}_tof_link" ros_topic="/pseudo_kinect_topic">
+			<origin xyz="${kinect_x} ${kinect_y} ${kinect_z}" rpy="${kinect_roll} ${kinect_pitch} ${kinect_yaw}" />
+		</xacro:cob_kinect_v0>
 		<!-- extensions -->
 		<xacro:cob_head_gazebo_v0 name="${name}" />

Commit message: update head description with general tof

File: ros/calibration/cob3-1.urdf.xacro (robot description, xacro)
@@ -39,10 +39,3 @@
 	<property name="tof_pitch" value="-0.0029" />
 	<property name="tof_yaw" value="-0.0058" />
-	<!-- head_kinect_link is identical to head_tof_link -->
-	<property name="kinect_x" value="0.0" />
-	<property name="kinect_y" value="0.0" />
-	<property name="kinect_z" value="0.0" />
-	<property name="kinect_roll" value="0.0" />
-	<property name="kinect_pitch" value="0.0" />
-	<property name="kinect_yaw" value="0.0" />
 </robot>

File: ros/urdf/head_v0/head.urdf.xacro (robot description, xacro)
@@ -8,5 +8,4 @@
 	<include filename="$(find cob_description)/ros/urdf/sensors/prosilica.urdf.xacro" />
 	<include filename="$(find cob_description)/ros/urdf/sensors/tof.urdf.xacro" />
-	<include filename="$(find cob_description)/ros/urdf/sensors/kinect.urdf.xacro" />
 	<!--include filename="$(find cob_description)/ros/urdf/sensors/hokuyo_SR400_laser.urdf.xacro" /-->
 	<xacro:macro name="cob_head_v0" params="name parent *origin">
@@ -53,8 +52,4 @@
 			<origin xyz="${tof_x-0.06} ${tof_y} ${tof_z}" rpy="${tof_roll} ${tof_pitch} ${tof_yaw}" />
 		</xacro:cob_tof_v0>
-		<!-- kinect_trial -->
-		<xacro:cob_kinect_v0 name="${name}_kinect" parent="${name}_tof_link" ros_topic="/pseudo_kinect_topic">
-			<origin xyz="${kinect_x} ${kinect_y} ${kinect_z}" rpy="${kinect_roll} ${kinect_pitch} ${kinect_yaw}" />
-		</xacro:cob_kinect_v0>
 		<!-- extensions -->
 		<xacro:cob_head_gazebo_v0 name="${name}" />
