Commit message: update for cob3-3

File: ros/calibration/cob3-3.urdf.xacro (robot description, xacro)
@@ -4,12 +4,11 @@
 	<property name="M_PI" value="3.1415926535897931" />
 	<!-- torso reference positions -->
-	<property name="torso_lower_neck_pan_ref" value="-0.5306" />
-	<property name="torso_lower_neck_tilt_ref" value="0.0320" />
-	<property name="torso_upper_neck_pan_ref" value="0.5481" />
-	<property name="torso_upper_neck_tilt_ref" value="0.0229" />
+	<property name="torso_lower_neck_tilt_ref" value="0" />
+	<property name="torso_pan_ref" value="0" />
+	<property name="torso_upper_neck_tilt_ref" value="0" />
 	<!-- tray reference position -->
-	<property name="torso_tray_ref" value="2.5541" />
+	<property name="torso_tray_ref" value="0" />
 	<!-- head camera axis reference position -->
-	<property name="head_axis_ref" value="-3.266798" />
+	<property name="head_axis_ref" value="0.0" />
 	<!-- arm reference positions -->
 	<property name="arm_1_ref" value="0" />
@@ -21,21 +20,21 @@
 	<property name="arm_7_ref" value="0" />
 	<!-- camera calibration properties -->
-	<property name="cam_r_x" value="-0.0854" />
-	<property name="cam_r_y" value="0.0148" />
-	<property name="cam_r_z" value="0.0032" />
-	<property name="cam_r_roll" value="2.4734" />
-	<property name="cam_r_pitch" value="-0.0151" />
-	<property name="cam_r_yaw" value="-3.8144" />
-	<property name="cam_l_x" value="-0.0007" />
-	<property name="cam_l_y" value="0.0008" />
-	<property name="cam_l_z" value="-0.0021" />
-	<property name="cam_l_roll" value="0.00036" />
-	<property name="cam_l_pitch" value="-0.00733" />
-	<property name="cam_l_yaw" value="-0.00069" />
-	<property name="tof_x" value="-0.0016" />
-	<property name="tof_y" value="-0.0015" />
-	<property name="tof_z" value="-0.0078" />
-	<property name="tof_roll" value="-0.0058" />
-	<property name="tof_pitch" value="-0.0029" />
-	<property name="tof_yaw" value="-0.0058" />
+	<property name="cam_r_x" value="0" />
+	<property name="cam_r_y" value="0" />
+	<property name="cam_r_z" value="0" />
+	<property name="cam_r_roll" value="0" />
+	<property name="cam_r_pitch" value="0" />
+	<property name="cam_r_yaw" value="0" />
+	<property name="cam_l_x" value="0" />
+	<property name="cam_l_y" value="0" />
+	<property name="cam_l_z" value="0" />
+	<property name="cam_l_roll" value="0" />
+	<property name="cam_l_pitch" value="0" />
+	<property name="cam_l_yaw" value="0" />
+	<property name="tof_x" value="0" />
+	<property name="tof_y" value="0" />
+	<property name="tof_z" value="0" />
+	<property name="tof_roll" value="0" />
+	<property name="tof_pitch" value="0" />
+	<property name="tof_yaw" value="0" />
 </robot>

File: ros/robots/cob3-1.urdf.xacro (robot description, xacro)
@@ -8,16 +8,15 @@
   <!-- misc common stuff? -->
   <include filename="$(find cob_description)/ros/urdf/common.xacro" />
-  <!-- cob calibration -->
+  <!-- calibration -->
   <include filename="$(find cob_description)/ros/calibration/cob3-1.urdf.xacro" />
-  <!-- cob base -->
-  <!--include filename="$(find cob_description)/ros/urdf/base_v0/base.urdf.xacro" /-->		<!-- with BOX base-collision model only -->
+  <!-- base -->
   <include filename="$(find cob_description)/ros/urdf/base_v1/base.urdf.xacro" />	<!-- new version; platform_controller and platform_navigation not yet working -->
   <!-- torso -->
   <include filename="$(find cob_description)/ros/urdf/torso_v0/torso.urdf.xacro" />
-  <!-- cob head-->
+  <!-- head -->
   <include filename="$(find cob_description)/ros/urdf/head_v0/head.urdf.xacro" />
-  <!-- cob arm-->
+  <!-- arm -->
   <include filename="$(find cob_description)/ros/urdf/lbr_v0/lbr.urdf.xacro" />
-  <!-- cob sdh-->
+  <!-- sdh -->
   <include filename="$(find cob_description)/ros/urdf/sdh_v0/sdh.urdf.xacro" />
   <!-- generic simulator_gazebo plugins for starting mechanism control, ros time, ros battery -->
@@ -33,5 +32,4 @@
        the origin block defines where the component is w.r.t its parent (in this case the parent
        is the world frame). For more, see http://www.ros.org/wiki/xacro -->
-  <!--<xacro:cob_base_v0 name="base"/-->
   <xacro:cob_base_v1 name="base"/>	<!--with new collision_model, but no platform_controller available yet-->
   <xacro:cob_torso_v0 name="torso" parent="base_link">

File: ros/robots/cob3-3.urdf.xacro (robot description, xacro)
@@ -4,5 +4,5 @@
        xmlns:interface="http://playerstage.sourceforge.net/gazebo/xmlschema/#interface"
        xmlns:xacro="http://playerstage.sourceforge.net/gazebo/xmlschema/#interface"
-       name="cob3-2" >
+       name="cob3-3" >
   <!-- The following included files set up definitions of parts of the robot body -->
   <!-- misc common stuff? -->
@@ -11,6 +11,5 @@
   <include filename="$(find cob_description)/ros/calibration/cob3-3.urdf.xacro" />
   <!-- base -->
-  <include filename="$(find cob_description)/ros/urdf/base_v0/base.urdf.xacro" />		<!-- with BOX base-collision model only -->
-  <!--include filename="$(find cob_description)/ros/urdf/base_v1/base.urdf.xacro" /-->	<!-- new version; platform_controller and platform_navigation not yet working -->
+  <include filename="$(find cob_description)/ros/urdf/base_v1/base.urdf.xacro" />	<!-- new version; platform_controller and platform_navigation not yet working -->
   <!-- torso -->
   <include filename="$(find cob_description)/ros/urdf/torso_v1/torso.urdf.xacro" />
@@ -18,5 +17,5 @@
   <include filename="$(find cob_description)/ros/urdf/head_v0/head.urdf.xacro" />
   <!-- arm -->
-  <include filename="$(find cob_description)/ros/urdf/arm_v0/arm.urdf.xacro" />
+  <include filename="$(find cob_description)/ros/urdf/lbr_v0/lbr.urdf.xacro" />
   <!-- sdh -->
   <include filename="$(find cob_description)/ros/urdf/sdh_v0/sdh.urdf.xacro" />
@@ -33,17 +32,16 @@
        the origin block defines where the component is w.r.t its parent (in this case the parent
        is the world frame). For more, see http://www.ros.org/wiki/xacro -->
-  <xacro:cob_base_v0 name="base"/>
-  <!--xacro:cob_base_v1 name="base"/-->	<!--with new collision_model, but no platform_controller available yet-->
+  <xacro:cob_base_v1 name="base"/>	<!--with new collision_model, but no platform_controller available yet-->
   <xacro:cob_torso_v1 name="torso" parent="base_link">
     <origin xyz="0.155 0 0.892" rpy="3.1415926 0 0" />
   </xacro:cob_torso_v1>
-  <xacro:cob_arm_v0 name="arm" parent="base_link">
-    <origin xyz="0.040 -0.005 0.83637" rpy="3.1415926 0.7854 -1.8326" />
-  </xacro:cob_arm_v0>
+  <xacro:cob_lbr_v0 name="arm" parent="base_link">
+    <origin xyz="-0.015982 -0.080992 0.875995" rpy="0.7854 0.0 -0.2618" />
+  </xacro:cob_lbr_v0>
   <xacro:cob_head_v0 name="head" parent="torso_upper_neck_tilt_link">
     <origin xyz="0 -0.154 0" rpy="3.14159 0 0" />
   </xacro:cob_head_v0>
   <xacro:cob_sdh_v0 name="sdh" parent="arm_7_link">
-    <origin xyz="0 0 0" rpy="0 3.1415926 0" />
+    <origin xyz="0 0 0.02" rpy="0 0 1.5708" />
   </xacro:cob_sdh_v0>
 </robot>

File: ros/urdf/torso_v1/torso.urdf.xacro (robot description, xacro)
@@ -40,9 +40,9 @@
 		<joint name="${name}_lower_neck_tilt_joint" type="revolute">
 			<!--insert_block name="origin" /-->
-			<origin xyz="0.155 0 0.892" rpy="4.7123926 0 0" />
+			<origin xyz="0.155 0 0.892" rpy="1.5708 0 0" />
 			<parent link="${parent}"/>
 			<child link="${name}_lower_neck_tilt_link"/>
 			<axis xyz="0 0 1" />
-			<calibration rising="-0.536"/>
+			<calibration rising="${torso_lower_neck_tilt_ref}"/>
 			<dynamics damping="25.0" friction="10.0"/>
 			<limit effort="41.4" lower="-6.2831" upper="6.2831" velocity="0.5"/>
@@ -55,5 +55,5 @@
 			</inertial>
 			<visual>
-				<origin xyz="0 0 0" rpy="0 0 0" />
+				<origin xyz="0 0 0" rpy="3.14 0 0" />
 				<geometry>
 					<mesh filename="package://cob_description/ros/meshes/torso_v0/lower_neck.stl" />
@@ -62,5 +62,5 @@
 			</visual>
 			<collision>
-				<origin xyz="0 0 0" rpy="0 0 0" />
+				<origin xyz="0 0 0" rpy="3.14 0 0" />
 				<geometry>
 					<mesh filename="package://cob_description/ros/meshes/torso_v0/lower_neck_collision.stlb" />
@@ -70,10 +70,10 @@
 		<!-- joint between torso_lower_neck_tilt_link and torso_pan_link -->
 		<joint name="${name}_pan_joint" type="revolute">
-			<origin xyz="0 0 0" rpy="0 0 0" />
+			<origin xyz="0 0 0" rpy="1.5708 0 0" />
 			<parent link="${name}_lower_neck_tilt_link"/>
 			<child link="${name}_pan_link"/>
 			<axis xyz="0 0 1" />
 			<dynamics damping="25.0" friction="10.0"/>
-			<calibration rising="0.0870"/>
+			<calibration rising="${torso_pan_ref}"/>
 			<limit effort="41.4" lower="-6.2831" upper="6.2831" velocity="0.5"/>
 		</joint>
@@ -100,10 +100,10 @@
 		<!-- joint between torso_pan_link and torso_upper_neck_link -->
 		<joint name="${name}_upper_neck_tilt_joint" type="revolute">
-			<origin xyz="0 -0.237 0" rpy="0 0 0" />
+			<origin xyz="0 0 -0.237" rpy="-1.5708 0 0" />
 			<parent link="${name}_pan_link"/>
 			<child link="${name}_upper_neck_tilt_link"/>
 			<axis xyz="0 0 1" />
 			<dynamics damping="25.0" friction="10.0"/>
-			<calibration rising="0.5481"/>
+			<calibration rising="${torso_upper_neck_tilt_ref}"/>
 			<limit effort="41.4" lower="-6.2831" upper="6.2831" velocity="0.5"/>
 		</joint>
@@ -115,5 +115,5 @@
 			</inertial>
 			<visual>
-				<origin xyz="0 0 0" rpy="0 0 0" />
+				<origin xyz="0 0 0" rpy="3.1415926 0 0" />
 				<geometry>
 					<mesh filename="package://cob_description/ros/meshes/torso_v0/upper_neck.stl" />
@@ -122,5 +122,5 @@
 			</visual>
 			<collision>
-				<origin xyz="0 0 0" rpy="0 0 0" />
+				<origin xyz="0 0 0" rpy="1.5708 0 0" />
 				<geometry>
 					<mesh filename="package://cob_description/ros/meshes/torso_v0/upper_neck_collision.stlb" />
@@ -130,5 +130,5 @@
 		<!-- joint between torso_upper_neck_tilt_link and head_cover_link -->
 		<joint name="head_cover_joint" type="fixed">
-			<origin xyz="0 0 0" rpy="0 0 0" />
+			<origin xyz="0 0 0" rpy="3.1415926 0 0" />
 			<parent link="${name}_upper_neck_tilt_link"/>
 			<child link="head_cover_link"/>

Commit message: Left tp right camera change in urdf

File: ros/calibration/cob3-3.urdf.xacro (robot description, xacro)
@@ -28,5 +28,5 @@
 	<property name="cam_l_yaw" value="0" />
 	<!-- right to left calibration -->
-	<property name="cam_r_x" value="-0.00008029" />
+	<property name="cam_r_x" value="-0.00002029" />
 	<property name="cam_r_y" value="0.00058637" />
 	<property name="cam_r_z" value="-0.00018271" />
@@ -35,5 +35,5 @@
 	<property name="cam_r_yaw" value="0.00299" />
 	<!-- cam3d to left calibration -->
-	<property name="cam3d_x" value="-0.01928202" />
+	<property name="cam3d_x" value="0.01928202" />
 	<property name="cam3d_y" value="0.03176335" />
 	<property name="cam3d_z" value="-0.00067414" />

File: ros/urdf/head_v0/head.urdf.xacro (robot description, xacro)
@@ -42,13 +42,13 @@
 		<!-- left camera -->
 		<xacro:cob_prosilica_v0 name="${name}_color_camera_l" ros_topic="stereo/left" parent="${name}_axis_link">
-			<origin xyz="${cam_l_x} ${cam_l_y} ${cam_l_z-0.06}" rpy="${cam_l_roll} ${cam_l_pitch+1.5708} ${cam_l_yaw+3.14159}" />
+			<origin xyz="${cam_l_x} ${cam_l_y} ${cam_l_z-0.06+0.12}" rpy="${cam_l_roll} ${cam_l_pitch+1.5708} ${cam_l_yaw+3.14159}" />
 		</xacro:cob_prosilica_v0>
 		<!-- right camera -->
 		<xacro:cob_prosilica_v0 name="${name}_color_camera_r" ros_topic="stereo/right" parent="${name}_color_camera_l_link">
-			<origin xyz="${cam_r_x-0.12} ${cam_r_y} ${cam_r_z}" rpy="${cam_r_roll} ${cam_r_pitch} ${cam_r_yaw}" />
+			<origin xyz="${cam_r_x+0.12} ${cam_r_y} ${cam_r_z}" rpy="${cam_r_roll} ${cam_r_pitch} ${cam_r_yaw}" />
 		</xacro:cob_prosilica_v0>
 		<!-- cam3d -->
 		<xacro:cob_kinect_v0 name="${name}_cam3d" ros_topic="cam3d/depth" parent="${name}_color_camera_l_link">
-			<origin xyz="${cam3d_x-0.06} ${cam3d_y} ${cam3d_z}" rpy="${cam3d_roll} ${cam3d_pitch} ${cam3d_yaw}" />
+			<origin xyz="${cam3d_x+0.06} ${cam3d_y} ${cam3d_z}" rpy="${cam3d_roll} ${cam3d_pitch} ${cam3d_yaw}" />
 		</xacro:cob_kinect_v0>
 		<!-- extensions -->

Commit message: fix cob3-3 tf

File: ros/calibration/cob3-3.urdf.xacro (robot description, xacro)
@@ -28,5 +28,5 @@
 	<property name="cam_l_yaw" value="0" />
 	<!-- right to left calibration -->
-	<property name="cam_r_x" value="-0.00002029" />
+	<property name="cam_r_x" value="0.00002029" />
 	<property name="cam_r_y" value="0.00058637" />
 	<property name="cam_r_z" value="-0.00018271" />
@@ -35,5 +35,5 @@
 	<property name="cam_r_yaw" value="0.00299" />
 	<!-- cam3d to left calibration -->
-	<property name="cam3d_x" value="0.01928202" />
+	<property name="cam3d_x" value="-0.01928202" />
 	<property name="cam3d_y" value="0.03176335" />
 	<property name="cam3d_z" value="-0.00067414" />

File: ros/robots/cob3-3.urdf.xacro (robot description, xacro)
@@ -40,5 +40,5 @@
   </xacro:cob_lbr_v0>
   <xacro:cob_head_v0 name="head" parent="torso_upper_neck_tilt_link">
-    <origin xyz="0 0.154 0" rpy="3.14159 0 0" />
+    <origin xyz="0 0.154 0" rpy="0 0 0" />
   </xacro:cob_head_v0>
   <xacro:cob_sdh_v0 name="sdh" parent="arm_7_link">

Commit message: added helper coordinate system for calibration, added calibration values

File: ros/calibration/cob3-3.urdf.xacro (robot description, xacro)
@@ -21,10 +21,10 @@
 	<!-- camera calibration properties -->
 	<!-- hand eye calibration -->
-	<property name="cam_l_x" value="0" />
-	<property name="cam_l_y" value="0" />
-	<property name="cam_l_z" value="0" />
-	<property name="cam_l_roll" value="0" />
-	<property name="cam_l_pitch" value="0" />
-	<property name="cam_l_yaw" value="0" />
+	<property name="cam_l_x" value="-0.00319" />
+	<property name="cam_l_y" value="0.03363" />
+	<property name="cam_l_z" value="0.05452" />
+	<property name="cam_l_roll" value="-0.0094" />
+	<property name="cam_l_pitch" value="-0.0003" />
+	<property name="cam_l_yaw" value="-0.0082" />
 	<!-- right to left calibration -->
 	<property name="cam_r_x" value="-0.00008258" />

File: ros/urdf/head_v3/head.urdf.xacro (robot description, xacro)
@@ -40,7 +40,32 @@
 			</collision>
 		</link>
+		<joint name="${name}_calib_joint" type="fixed">
+			<origin xyz="0 0 -0.06" rpy="0 -1.5708 0" />
+			<parent link="${name}_axis_link"/>
+			<child link="${name}_calib_link"/>
+		</joint>
+		<link name="${name}_calib_link">
+			<inertial>
+				<origin xyz="0 0 0" rpy="0 0 0"/>
+				<mass value="0.1"/>
+				<inertia ixx="0.0001" ixy="0" ixz="0" iyy="0.0001" iyz="0" izz="0.0001" />
+			</inertial>
+			<visual>
+				<origin xyz="0 0 0" rpy="0 0 0" />
+				<geometry>
+					<box size="0.01 0.01 0.12"/>
+				</geometry>
+				<material name="Green" />
+			</visual>
+			<collision>
+				<origin xyz="0 0 0" rpy="0 0 0" />
+				<geometry>
+					<box size="0.01 0.01 0.12"/>
+				</geometry>
+			</collision>
+		</link>
 		<!-- left camera -->
-		<xacro:cob_prosilica_v0 name="${name}_color_camera_l" ros_topic="stereo/left" parent="${name}_axis_link">
-			<origin xyz="${cam_l_x} ${cam_l_y} ${cam_l_z-0.06}" rpy="${cam_l_roll} ${cam_l_pitch-1.5708} ${cam_l_yaw}" />
+		<xacro:cob_prosilica_v0 name="${name}_color_camera_l" ros_topic="stereo/left" parent="${name}_calib_link">
+			<origin xyz="${cam_l_x} ${cam_l_y} ${cam_l_z}" rpy="${cam_l_roll} ${cam_l_pitch} ${cam_l_yaw}" />
 		</xacro:cob_prosilica_v0>
 		<!-- right camera -->

Commit message: new calibration for cob3-3 and cob3-4

File: ros/calibration/cob3-3.urdf.xacro (robot description, xacro)
@@ -26,5 +26,5 @@
 	<property name="cam_l_roll" value="0" />
 	<property name="cam_l_pitch" value="0" />
-	<property name="cam_l_yaw" value="0" />
+	<property name="cam_l_yaw" value="0.05" />
 	<!-- right to left calibration -->
 	<property name="cam_r_x" value="0.0000281" />
@@ -35,7 +35,7 @@
 	<property name="cam_r_yaw" value="-0.00272" />
 	<!-- cam3d to left calibration -->
-	<property name="cam3d_x" value="-0.01899859" />
-	<property name="cam3d_y" value="0.03048727" />
-	<property name="cam3d_z" value="-0.00303078" />
+	<property name="cam3d_x" value="0.06099859" />
+	<property name="cam3d_y" value="-0.04048727" />
+	<property name="cam3d_z" value="0.05303078" />
 	<property name="cam3d_roll" value="0.00641" />
 	<property name="cam3d_pitch" value="0.00728" />

File: ros/calibration/cob3-4.urdf.xacro (robot description, xacro)
@@ -26,5 +26,5 @@
 	<property name="cam_l_roll" value="0" />
 	<property name="cam_l_pitch" value="0" />
-	<property name="cam_l_yaw" value="0" />
+	<property name="cam_l_yaw" value="0.05" />
 	<!-- right to left calibration -->
 	<property name="cam_r_x" value="0.0000281" />
@@ -35,7 +35,7 @@
 	<property name="cam_r_yaw" value="-0.00272" />
 	<!-- cam3d to left calibration -->
-	<property name="cam3d_x" value="-0.01899859" />
-	<property name="cam3d_y" value="0.03048727" />
-	<property name="cam3d_z" value="-0.00303078" />
+	<property name="cam3d_x" value="0.01099859" />
+	<property name="cam3d_y" value="-0.04048727" />
+	<property name="cam3d_z" value="0.03303078" />
 	<property name="cam3d_roll" value="0.00641" />
 	<property name="cam3d_pitch" value="0.00728" />

File: ros/robots/cob3-4.urdf.xacro (robot description, xacro)
@@ -37,5 +37,6 @@
   </xacro:cob_torso_v1>
   <xacro:cob_arm_v1 name="arm" parent="base_link">
-    <origin xyz="0.040 -0.005 0.83637" rpy="3.1415926 0.7854 -1.8326" />
+    <!--origin xyz="0.040 -0.005 0.83637" rpy="3.1415926 0.7854 -1.8326" /-->
+    <origin xyz="0.040 -0.005 0.77637" rpy="3.1415926 0.7854 -1.8326" />
   </xacro:cob_arm_v1>
   <xacro:cob_head_v3 name="head" parent="torso_upper_neck_tilt_link">

File: ros/urdf/arm_v1/arm.urdf.xacro (robot description, xacro)
@@ -225,5 +225,5 @@
 		<!-- joint between arm_6_link and arm_7_link -->
 		<joint name="${name}_7_joint" type="revolute">
-			<origin xyz="0 -0.237448 0" rpy="-1.5708 0 0" />
+			<origin xyz="0 -0.197448 0" rpy="-1.5708 0 0" />
 			<parent link="${name}_6_link"/>
 			<child link="${name}_7_link"/>
