Commit message: big changes to simulation structure

File: ros/urdf/arm_v0/arm.gazebo.xacro (robot description, xacro)
@@ -6,34 +6,34 @@
   <xacro:macro name="cob_arm_gazebo_v0" params="name">
 	<gazebo reference="${name}_0_link">
-		<material value="PR2/Red" />
-		<turnGravityOff>false</turnGravityOff>
+		<material value="Gazebo/Red" />
+		<turnGravityOff>true</turnGravityOff>
 	</gazebo>
 	<gazebo reference="${name}_1_link">
-		<material value="PR2/Blue" />
-		<turnGravityOff>false</turnGravityOff>
+		<material value="Gazebo/Blue" />
+		<turnGravityOff>true</turnGravityOff>
 	</gazebo>
 	<gazebo reference="${name}_2_link">
-		<material value="PR2/Red" />
-		<turnGravityOff>false</turnGravityOff>
+		<material value="Gazebo/Red" />
+		<turnGravityOff>true</turnGravityOff>
 	</gazebo>
 	<gazebo reference="${name}_3_link">
-		<material value="PR2/Blue" />
-		<turnGravityOff>false</turnGravityOff>
+		<material value="Gazebo/Blue" />
+		<turnGravityOff>true</turnGravityOff>
 	</gazebo>
 	<gazebo reference="${name}_4_link">
-		<material value="PR2/Red" />
-		<turnGravityOff>false</turnGravityOff>
+		<material value="Gazebo/Red" />
+		<turnGravityOff>true</turnGravityOff>
 	</gazebo>
 	<gazebo reference="${name}_5_link">
-		<material value="PR2/Blue" />
-		<turnGravityOff>false</turnGravityOff>
+		<material value="Gazebo/Blue" />
+		<turnGravityOff>true</turnGravityOff>
 	</gazebo>
 	<gazebo reference="${name}_6_link">
-		<material value="PR2/Red" />
-		<turnGravityOff>false</turnGravityOff>
+		<material value="Gazebo/Red" />
+		<turnGravityOff>true</turnGravityOff>
 	</gazebo>
 	<gazebo reference="${name}_7_link">
-		<material value="PR2/Blue" />
-		<turnGravityOff>false</turnGravityOff>
+		<material value="Gazebo/Blue" />
+		<turnGravityOff>true</turnGravityOff>
 	</gazebo>
   </xacro:macro>

File: ros/urdf/arm_v0/arm.urdf.xacro (robot description, xacro)
@@ -43,4 +43,5 @@
 		<axis xyz="0 0 1"/>
 	        <calibration reference_position="${arm_1_ref}"/>
+                <dynamics damping="20" />
 		<limit effort="370" velocity="0.4363" lower="-2.0943951" upper="2.0943951"/>
 	</joint>
@@ -49,5 +50,5 @@
 			<origin xyz="0 0 0" rpy="0 0 0" />
 			<mass value="5.9907"/>
-			<inertia ixx="5"  ixy="0"  ixz="0" iyy="5" iyz="0" izz="5" />
+			<inertia ixx="0.01"  ixy="0"  ixz="0" iyy="0.01" iyz="0" izz="0.01" />
 		</inertial>
 		<visual>
@@ -72,4 +73,5 @@
 		<axis xyz="0 0 1"/>
 	        <calibration reference_position="${arm_2_ref}"/>
+                <dynamics damping="20" />
 		<limit effort="370" velocity="0.4363" lower="-2.0943951" upper="2.0943951"/>
 	</joint>
@@ -101,4 +103,5 @@
 		<axis xyz="0 0 1"/>
 	        <calibration reference_position="${arm_3_ref}"/>
+                <dynamics damping="20" />
 		<limit effort="176" velocity="0.4189" lower="-6.2831853" upper="6.2831853"/>
 	</joint>
@@ -130,4 +133,5 @@
 		<axis xyz="0 0 1" />
 	        <calibration reference_position="${arm_4_ref}"/>
+                <dynamics damping="20" />
 		<limit effort="176" velocity="0.4189" upper="2.0943951" lower="-2.0943951" />
 	</joint>
@@ -159,4 +163,5 @@
 		<axis xyz="0 0 1" />
 	        <calibration reference_position="${arm_5_ref}"/>
+                <dynamics damping="10" />
 		<limit effort="41.6" velocity="0.4363" upper="6.2831853" lower="-6.2831853" />
 	</joint>
@@ -188,4 +193,5 @@
 		<axis xyz="0 0 1" />
 	        <calibration reference_position="${arm_6_ref}"/>
+                <dynamics damping="10" />
 		<limit effort="20.1" velocity="0.4363" upper="2.0943951" lower="-2.0943951" />
 	</joint>
@@ -217,4 +223,5 @@
 		<axis xyz="0 0 1" />
 	        <calibration reference_position="${arm_7_ref}"/>
+                <dynamics damping="10" />
 		<limit effort="9.6" velocity="0.8727" upper="6.2831853" lower="-6.2831853" />
 	</joint>

File: ros/urdf/head_cameras_v0/head_cameras.urdf.xacro (robot description, xacro)
@@ -45,8 +45,8 @@
     <!-- camera test here -->
     <xacro:cob_cameraone_v0 name="${name}_color_camera_l" parent="${name}_camera_axis_link">
-      <origin xyz="0 0.05 0" rpy="0 0 0" />
+      <origin xyz="0 0.03 -0.003" rpy="0 0 0" />
     </xacro:cob_cameraone_v0>
     <xacro:cob_cameraone_v0 name="${name}_color_camera_r" parent="${name}_camera_axis_link">
-      <origin xyz="0 -0.05 0" rpy="0 0 0" />
+      <origin xyz="0 -0.03 -0.003" rpy="0 0 0" />
     </xacro:cob_cameraone_v0>
     <!-- hokuyo_SR400_laser test here-->

File: ros/urdf/sdh_v0/sdh.gazebo.xacro (robot description, xacro)
@@ -14,6 +14,17 @@
 	</gazebo>
 	<gazebo reference="${name}_finger_12_link">
-		<material>Gazebo/Red</material>
-		<turnGravityOff>false</turnGravityOff>
+           <selfCollide>true</selfCollide>
+              <sensor:contact name="${name}_finger_12_contact_sensor">
+                 <geom>${name}_finger_12_link_geom</geom>
+                 <updateRate>100.0</updateRate>
+                 <controller:gazebo_ros_bumper name="${name}_finger_12_gazebo_ros_bumper_controller" plugin="libgazebo_ros_bumper.so">
+                    <alwaysOn>true</alwaysOn>
+                    <updateRate>100.0</updateRate>
+                    <bumperTopicName>${name}_finger_12_bumper</bumperTopicName>
+                    <interface:bumper name="${name}_finger_12_bumper_iface" />
+                 </controller:gazebo_ros_bumper>
+              </sensor:contact>
+              <material>Gazebo/Red</material>
+	      <turnGravityOff>false</turnGravityOff>
 	</gazebo>
         <gazebo reference="${name}_finger_13_link">
@@ -36,6 +47,17 @@
 	</gazebo>
 	<gazebo reference="${name}_finger_22_link">
-		<material>Gazebo/Red</material>
-		<turnGravityOff>false</turnGravityOff>
+           <selfCollide>true</selfCollide>
+              <sensor:contact name="${name}_finger_22_contact_sensor">
+                 <geom>${name}_finger_22_link_geom</geom>
+                 <updateRate>100.0</updateRate>
+                 <controller:gazebo_ros_bumper name="${name}_finger_22_gazebo_ros_bumper_controller" plugin="libgazebo_ros_bumper.so">
+                    <alwaysOn>true</alwaysOn>
+                    <updateRate>100.0</updateRate>
+                    <bumperTopicName>${name}_finger_22_bumper</bumperTopicName>
+                    <interface:bumper name="${name}_finger_22_bumper_iface" />
+                 </controller:gazebo_ros_bumper>
+              </sensor:contact>
+	      <material>Gazebo/Red</material>
+	      <turnGravityOff>false</turnGravityOff>
 	</gazebo>
         <gazebo reference="${name}_finger_23_link">
@@ -58,6 +80,17 @@
 	</gazebo>
 	<gazebo reference="${name}_thumb_2_link">
-		<material>Gazebo/Red</material>
-		<turnGravityOff>false</turnGravityOff>
+           <selfCollide>true</selfCollide>
+              <sensor:contact name="${name}_thumb_2_contact_sensor">
+                 <geom>${name}_thumb_2_link_geom</geom>
+                 <updateRate>100.0</updateRate>
+                 <controller:gazebo_ros_bumper name="${name}_thumb_2_gazebo_ros_bumper_controller" plugin="libgazebo_ros_bumper.so">
+                    <alwaysOn>true</alwaysOn>
+                    <updateRate>100.0</updateRate>
+                    <bumperTopicName>${name}_thumb_2_bumper</bumperTopicName>
+                    <interface:bumper name="${name}_thumb_2_bumper_iface" />
+                 </controller:gazebo_ros_bumper>
+              </sensor:contact>
+	      <material>Gazebo/Red</material>
+	      <turnGravityOff>false</turnGravityOff>
 	</gazebo>
         <gazebo reference="${name}_thumb_3_link">

File: ros/urdf/sdh_v0/sdh.urdf.xacro (robot description, xacro)
@@ -20,10 +20,10 @@
 			<origin xyz="0 0 0" rpy="0 0 0"/>
 			<mass value="1"/>
-			<inertia ixx="1"  ixy="0"  ixz="0" iyy="1" iyz="0" izz="1" />
-		</inertial>
-		<visual>
-			<origin xyz="0 0 0" rpy="0 0 0" />
-			<geometry>
-				<mesh filename="package://cob_defs/common/files/meshes/palm.stl" />
+			<inertia ixx="0.01"  ixy="0"  ixz="0" iyy="0.01" iyz="0" izz="0.01" />
+		</inertial>
+		<visual>
+			<origin xyz="0 0 0" rpy="0 0 0" />
+			<geometry>
+				<mesh filename="package://cob_description/ros/meshes/sdh_v0/palm.stl" />
 			</geometry>
                         <material name="Grey" />
@@ -32,5 +32,5 @@
 			<origin xyz="0 0 0" rpy="0 0 0" />
 			<geometry>
-				<mesh filename="package://cob_defs/common/files/meshes/palm.stl"/>
+				<mesh filename="package://cob_description/ros/meshes/sdh_v0/palm.stl"/>
 			</geometry>
 		</collision>
@@ -43,4 +43,5 @@
 		<child link="${name}_finger_11_link"/>
 		<axis xyz="0 0 1" />
+                <dynamics damping="1" />
 	        <calibration reference_position="0.0"/>
 		<limit effort="100" lower="-2" upper="2" velocity="5"/>
@@ -50,10 +51,10 @@
 			<origin xyz="0 0 0" rpy="0 0 0"/>
 			<mass value="0.1"/>
-			<inertia ixx="1"  ixy="0"  ixz="0" iyy="1" iyz="0" izz="1" />
-		</inertial>
-		<visual>
-			<origin xyz="0 0 0" rpy="0 0 0" />
-			<geometry>
-				<mesh filename="package://cob_defs/common/files/meshes/knuckle.stl" />
+			<inertia ixx="0.01"  ixy="0"  ixz="0" iyy="0.01" iyz="0" izz="0.01" />
+		</inertial>
+		<visual>
+			<origin xyz="0 0 0" rpy="0 0 0" />
+			<geometry>
+				<mesh filename="package://cob_description/ros/meshes/sdh_v0/knuckle.stl" />
 			</geometry>
                         <material name="Black" />
@@ -62,5 +63,5 @@
 			<origin xyz="0 0 0" rpy="0 0 0" />
 			<geometry>
-				<mesh filename="package://cob_defs/common/files/meshes/knuckle.stl"/>
+				<mesh filename="package://cob_description/ros/meshes/sdh_v0/knuckle.stl"/>
 			</geometry>
 		</collision>
@@ -72,4 +73,5 @@
 		<child link="${name}_finger_12_link"/>
 		<axis xyz="0 1 0" />
+                <dynamics damping="1" />
 	        <calibration reference_position="0.0"/>
 		<limit effort="100" lower="-2" upper="2" velocity="5"/>
@@ -79,10 +81,10 @@
 			<origin xyz="0 0 0" rpy="0 0 0"/>
 			<mass value="0.1"/>
-			<inertia ixx="1"  ixy="0"  ixz="0" iyy="1" iyz="0" izz="1" />
-		</inertial>
-		<visual>
-			<origin xyz="0 0 0" rpy="0 0 0" />
-			<geometry>
-				<mesh filename="package://cob_defs/common/files/meshes/finger.stl" />
+			<inertia ixx="0.01"  ixy="0"  ixz="0" iyy="0.01" iyz="0" izz="0.01" />
+		</inertial>
+		<visual>
+			<origin xyz="0 0 0" rpy="0 0 0" />
+			<geometry>
+				<mesh filename="package://cob_description/ros/meshes/sdh_v0/finger.stl" />
 			</geometry>
                         <material name="Red" />
@@ -91,5 +93,5 @@
 			<origin xyz="0 0 0" rpy="0 0 0" />
 			<geometry>
-				<mesh filename="package://cob_defs/common/files/meshes/finger.stl"/>
+				<mesh filename="package://cob_description/ros/meshes/sdh_v0/finger.stl"/>
 			</geometry>
 		</collision>
@@ -101,4 +103,5 @@
 		<child link="${name}_finger_13_link"/>
 		<axis xyz="0 1 0" />
+                <dynamics damping="1" />
 	        <calibration reference_position="0.0"/>
 		<limit effort="100" lower="-2" upper="2" velocity="5"/>
@@ -108,10 +111,10 @@
 			<origin xyz="0 0 0" rpy="0 0 0"/>
 			<mass value="0.1"/>
-			<inertia ixx="1"  ixy="0"  ixz="0" iyy="1" iyz="0" izz="1" />
-		</inertial>
-		<visual>
-			<origin xyz="0 0 0" rpy="0 0 0" />
-			<geometry>
-				<mesh filename="package://cob_defs/common/files/meshes/finger_tip.stl" />
+			<inertia ixx="0.01"  ixy="0"  ixz="0" iyy="0.01" iyz="0" izz="0.01" />
+		</inertial>
+		<visual>
+			<origin xyz="0 0 0" rpy="0 0 0" />
+			<geometry>
+				<mesh filename="package://cob_description/ros/meshes/sdh_v0/finger_tip.stl" />
 			</geometry>
                         <material name="Blue" />
@@ -120,5 +123,5 @@
 			<origin xyz="0 0 0" rpy="0 0 0" />
 			<geometry>
-				<mesh filename="package://cob_defs/common/files/meshes/finger_tip.stl"/>
+				<mesh filename="package://cob_description/ros/meshes/sdh_v0/finger_tip.stl"/>
 			</geometry>
 		</collision>
@@ -131,4 +134,5 @@
 		<child link="${name}_finger_21_link"/>
 		<axis xyz="0 0 1" />
+                <dynamics damping="1" />
 	        <calibration reference_position="0.0"/>
 		<limit effort="100" lower="-2" upper="2" velocity="5"/>
@@ -138,10 +142,10 @@
 			<origin xyz="0 0 0" rpy="0 0 0"/>
 			<mass value="0.1"/>
-			<inertia ixx="1"  ixy="0"  ixz="0" iyy="1" iyz="0" izz="1" />
-		</inertial>
-		<visual>
-			<origin xyz="0 0 0" rpy="0 0 0" />
-			<geometry>
-				<mesh filename="package://cob_defs/common/files/meshes/knuckle.stl" />
+			<inertia ixx="0.01"  ixy="0"  ixz="0" iyy="0.01" iyz="0" izz="0.01" />
+		</inertial>
+		<visual>
+			<origin xyz="0 0 0" rpy="0 0 0" />
+			<geometry>
+				<mesh filename="package://cob_description/ros/meshes/sdh_v0/knuckle.stl" />
 			</geometry>
                         <material name="Black" />
@@ -150,5 +154,5 @@
 			<origin xyz="0 0 0" rpy="1.57079633 0 0" />
 			<geometry>
-				<mesh filename="package://cob_defs/common/files/meshes/knuckle.stl"/>
+				<mesh filename="package://cob_description/ros/meshes/sdh_v0/knuckle.stl"/>
 			</geometry>
 		</collision>
@@ -160,4 +164,5 @@
 		<child link="${name}_finger_22_link"/>
 		<axis xyz="0 1 0" />
+                <dynamics damping="1" />
 	        <calibration reference_position="0.0"/>
 		<limit effort="100" lower="-2" upper="2" velocity="5"/>
@@ -167,10 +172,10 @@
 			<origin xyz="0 0 0" rpy="0 0 0"/>
 			<mass value="0.1"/>
-			<inertia ixx="1"  ixy="0"  ixz="0" iyy="1" iyz="0" izz="1" />
-		</inertial>
-		<visual>
-			<origin xyz="0 0 0" rpy="0 0 0" />
-			<geometry>
-				<mesh filename="package://cob_defs/common/files/meshes/finger.stl" />
+			<inertia ixx="0.01"  ixy="0"  ixz="0" iyy="0.01" iyz="0" izz="0.01" />
+		</inertial>
+		<visual>
+			<origin xyz="0 0 0" rpy="0 0 0" />
+			<geometry>
+				<mesh filename="package://cob_description/ros/meshes/sdh_v0/finger.stl" />
 			</geometry>
                         <material name="Red" />
@@ -179,5 +184,5 @@
 			<origin xyz="0 0 0" rpy="0 0 0" />
 			<geometry>
-				<mesh filename="package://cob_defs/common/files/meshes/finger.stl"/>
+				<mesh filename="package://cob_description/ros/meshes/sdh_v0/finger.stl"/>
 			</geometry>
 		</collision>
@@ -189,4 +194,5 @@
 		<child link="${name}_finger_23_link"/>
 		<axis xyz="0 1 0" />
+                <dynamics damping="1" />
 	        <calibration reference_position="0.0"/>
 		<limit effort="100" lower="-2" upper="2" velocity="5"/>
@@ -196,10 +202,10 @@
 			<origin xyz="0 0 0" rpy="0 0 0"/>
 			<mass value="0.1"/>
-			<inertia ixx="1"  ixy="0"  ixz="0" iyy="1" iyz="0" izz="1" />
-		</inertial>
-		<visual>
-			<origin xyz="0 0 0" rpy="0 0 0" />
-			<geometry>
-				<mesh filename="package://cob_defs/common/files/meshes/finger_tip.stl" />
+			<inertia ixx="0.01"  ixy="0"  ixz="0" iyy="0.01" iyz="0" izz="0.01" />
+		</inertial>
+		<visual>
+			<origin xyz="0 0 0" rpy="0 0 0" />
+			<geometry>
+				<mesh filename="package://cob_description/ros/meshes/sdh_v0/finger_tip.stl" />
 			</geometry>
                         <material name="Blue" />
@@ -208,5 +214,5 @@
 			<origin xyz="0 0 0" rpy="0 0 0" />
 			<geometry>
-				<mesh filename="package://cob_defs/common/files/meshes/finger_tip.stl"/>
+				<mesh filename="package://cob_description/ros/meshes/sdh_v0/finger_tip.stl"/>
 			</geometry>
 		</collision>
@@ -224,10 +230,10 @@
 			<origin xyz="0 0 0" rpy="0 0 0"/>
 			<mass value="0.1"/>
-			<inertia ixx="1"  ixy="0"  ixz="0" iyy="1" iyz="0" izz="1" />
-		</inertial>
-		<visual>
-			<origin xyz="0 0 0" rpy="0 0 0" />
-			<geometry>
-				<mesh filename="package://cob_defs/common/files/meshes/knuckle.stl" />
+			<inertia ixx="0.01"  ixy="0"  ixz="0" iyy="0.01" iyz="0" izz="0.01" />
+		</inertial>
+		<visual>
+			<origin xyz="0 0 0" rpy="0 0 0" />
+			<geometry>
+				<mesh filename="package://cob_description/ros/meshes/sdh_v0/knuckle.stl" />
 			</geometry>
                         <material name="Black" />
@@ -236,5 +242,5 @@
 			<origin xyz="0 0 0" rpy="0 0 0" />
 			<geometry>
-				<mesh filename="package://cob_defs/common/files/meshes/knuckle.stl"/>
+				<mesh filename="package://cob_description/ros/meshes/sdh_v0/knuckle.stl"/>
 			</geometry>
 		</collision>
@@ -246,4 +252,5 @@
 		<child link="${name}_thumb_2_link"/>
 		<axis xyz="0 1 0" />
+                <dynamics damping="1" />
 	        <calibration reference_position="0.0"/>
 		<limit effort="100" lower="-2" upper="2" velocity="5"/>
@@ -253,10 +260,10 @@
 			<origin xyz="0 0 0" rpy="0 0 0"/>
 			<mass value="0.1"/>
-			<inertia ixx="1"  ixy="0"  ixz="0" iyy="1" iyz="0" izz="1" />
-		</inertial>
-		<visual>
-			<origin xyz="0 0 0" rpy="0 0 0" />
-			<geometry>
-				<mesh filename="package://cob_defs/common/files/meshes/finger.stl" />
+			<inertia ixx="0.01"  ixy="0"  ixz="0" iyy="0.01" iyz="0" izz="0.01" />
+		</inertial>
+		<visual>
+			<origin xyz="0 0 0" rpy="0 0 0" />
+			<geometry>
+				<mesh filename="package://cob_description/ros/meshes/sdh_v0/finger.stl" />
 			</geometry>
                         <material name="Red" />
@@ -265,5 +272,5 @@
 			<origin xyz="0 0 0" rpy="0 0 0" />
 			<geometry>
-				<mesh filename="package://cob_defs/common/files/meshes/finger.stl"/>
+				<mesh filename="package://cob_description/ros/meshes/sdh_v0/finger.stl"/>
 			</geometry>
 		</collision>
@@ -275,4 +282,5 @@
 		<child link="${name}_thumb_3_link"/>
 		<axis xyz="0 1 0" />
+                <dynamics damping="1" />
 	        <calibration reference_position="0.0"/>
 		<limit effort="100" lower="-2" upper="2" velocity="5"/>
@@ -282,10 +290,10 @@
 			<origin xyz="0 0 0" rpy="0 0 0"/>
 			<mass value="0.1"/>
-			<inertia ixx="1"  ixy="0"  ixz="0" iyy="1" iyz="0" izz="1" />
-		</inertial>
-		<visual>
-			<origin xyz="0 0 0" rpy="0 0 0" />
-			<geometry>
-				<mesh filename="package://cob_defs/common/files/meshes/finger_tip.stl" />
+			<inertia ixx="0.01"  ixy="0"  ixz="0" iyy="0.01" iyz="0" izz="0.01" />
+		</inertial>
+		<visual>
+			<origin xyz="0 0 0" rpy="0 0 0" />
+			<geometry>
+				<mesh filename="package://cob_description/ros/meshes/sdh_v0/finger_tip.stl" />
 			</geometry>
                         <material name="Blue" />
@@ -294,5 +302,5 @@
 			<origin xyz="0 0 0" rpy="0 0 0" />
 			<geometry>
-				<mesh filename="package://cob_defs/common/files/meshes/finger_tip.stl"/>
+				<mesh filename="package://cob_description/ros/meshes/sdh_v0/finger_tip.stl"/>
 			</geometry>
 		</collision>

File: ros/urdf/sensors/cameraone.urdf.xacro (robot description, xacro)
@@ -21,5 +21,5 @@
         <origin xyz="0 0 0" rpy="0 0 0" />
         <geometry>
-          <cylinder radius="0.01" length="0.01"/>
+          <cylinder radius="0.005" length="0.005"/>
         </geometry>
         <material name="Red" />
@@ -28,5 +28,5 @@
         <origin xyz="0 0 0" rpy="0 0 0" />
         <geometry>
-           <cylinder radius="0.01" length="0.01"/>
+           <cylinder radius="0.001" length="0.001"/>
         </geometry>
       </collision >

File: ros/urdf/torso_v0/torso.urdf.xacro (robot description, xacro)
@@ -29,5 +29,5 @@
 	 <origin xyz="0 0 0" rpy="0.707 0 0" />
 	 <geometry>
-	    <mesh filename="package://cob_defs/common/files/meshes/tray.stl" />
+	    <mesh filename="package://cob_description/ros/meshes/torso_v0/tray.stl" />
 	 </geometry>
          <material name="Green" />
@@ -36,5 +36,5 @@
 	 <origin xyz="0 0 0" rpy="0.707 0 0" />
 	 <geometry>
-	  <mesh filename="package://cob_defs/common/files/meshes/tray.stl" />
+	  <mesh filename="package://cob_description/ros/meshes/torso_v0/tray.stl" />
 	 </geometry>
        </collision>
@@ -47,5 +47,5 @@
       <axis xyz="0 0 1" />
       <calibration reference_position="${torso_lower_neck_pan_ref}"/>
-      <dynamics damping="15.0" friction="10.0"/>
+      <dynamics damping="25.0" friction="10.0"/>
       <limit effort="24" lower="-6.2831" upper="6.2831" velocity="0.5"/>
     </joint>
@@ -76,5 +76,5 @@
       <child link="${name}_lower_neck_tilt_link"/>
       <axis xyz="0 0 1" />
-      <dynamics damping="15.0" friction="10.0"/>
+      <dynamics damping="25.0" friction="10.0"/>
       <calibration reference_position="${torso_lower_neck_tilt_ref}"/>
       <limit effort="46" lower="-1.5" upper="1.5" velocity="0.5"/>
@@ -107,5 +107,5 @@
       <child link="${name}_upper_neck_pan_link"/>
       <axis xyz="0 0 1" />
-      <dynamics damping="15.0" friction="10.0"/>
+      <dynamics damping="25.0" friction="10.0"/>
       <calibration reference_position="${torso_upper_neck_pan_ref}"/>
       <limit effort="4" lower="-6.2831" upper="6.2831" velocity="0.5"/>
@@ -137,5 +137,5 @@
       <child link="${name}_upper_neck_tilt_link"/>
       <axis xyz="0 0 1" />
-      <dynamics damping="15.0" friction="10.0"/>
+      <dynamics damping="25.0" friction="10.0"/>
       <calibration reference_position="${torso_upper_neck_tilt_ref}"/>
       <limit effort="24" lower="-1.5" upper="1.5" velocity="0.5"/>
