Commit message: improved simulation for schunk arm and cleanup in 2dnav package

File: ros/urdf/arm_v0/arm.gazebo.xacro (robot description, xacro)
@@ -6,34 +6,34 @@
   <xacro:macro name="cob_arm_gazebo_v0" params="name">
 	<gazebo reference="${name}_0_link">
-		<material value="Gazebo/Red" />
-		<turnGravityOff>true</turnGravityOff>
+		<material value="PR2/Red" />
+		<turnGravityOff>false</turnGravityOff>
 	</gazebo>
 	<gazebo reference="${name}_1_link">
-		<material value="Gazebo/Blue" />
-		<turnGravityOff>true</turnGravityOff>
+		<material value="PR2/Blue" />
+		<turnGravityOff>false</turnGravityOff>
 	</gazebo>
 	<gazebo reference="${name}_2_link">
-		<material value="Gazebo/Red" />
-		<turnGravityOff>true</turnGravityOff>
+		<material value="PR2/Red" />
+		<turnGravityOff>false</turnGravityOff>
 	</gazebo>
 	<gazebo reference="${name}_3_link">
-		<material value="Gazebo/Blue" />
-		<turnGravityOff>true</turnGravityOff>
+		<material value="PR2/Blue" />
+		<turnGravityOff>false</turnGravityOff>
 	</gazebo>
 	<gazebo reference="${name}_4_link">
-		<material value="Gazebo/Red" />
-		<turnGravityOff>true</turnGravityOff>
+		<material value="PR2/Red" />
+		<turnGravityOff>false</turnGravityOff>
 	</gazebo>
 	<gazebo reference="${name}_5_link">
-		<material value="Gazebo/Blue" />
-		<turnGravityOff>true</turnGravityOff>
+		<material value="PR2/Blue" />
+		<turnGravityOff>false</turnGravityOff>
 	</gazebo>
 	<gazebo reference="${name}_6_link">
-		<material value="Gazebo/Red" />
-		<turnGravityOff>true</turnGravityOff>
+		<material value="PR2/Red" />
+		<turnGravityOff>false</turnGravityOff>
 	</gazebo>
 	<gazebo reference="${name}_7_link">
-		<material value="Gazebo/Blue" />
-		<turnGravityOff>true</turnGravityOff>
+		<material value="PR2/Blue" />
+		<turnGravityOff>false</turnGravityOff>
 	</gazebo>
   </xacro:macro>

File: ros/urdf/arm_v0/arm.urdf.xacro (robot description, xacro)
@@ -42,6 +42,6 @@
 		<child link="${name}_1_link"/>
 		<axis xyz="0 0 1"/>
-	        <calibration reference_position="${arm_1_ref}"/>
-                <dynamics damping="30" />
+		<calibration reference_position="${arm_1_ref}"/>
+		<dynamics damping="10.0" friction="10.0" />
 		<limit effort="370" velocity="0.4363" lower="-6.2831853" upper="6.2831853"/>
 	</joint>
@@ -72,6 +72,6 @@
 		<child link="${name}_2_link"/>
 		<axis xyz="0 0 1"/>
-	        <calibration reference_position="${arm_2_ref}"/>
-                <dynamics damping="30" />
+		<calibration reference_position="${arm_2_ref}"/>
+		<dynamics damping="10.0" friction="10.0" />
 		<limit effort="370" velocity="0.4363" lower="-2.0943951" upper="2.0943951"/>
 	</joint>
@@ -102,6 +102,6 @@
 		<child link="${name}_3_link"/>
 		<axis xyz="0 0 1"/>
-	        <calibration reference_position="${arm_3_ref}"/>
-                <dynamics damping="30" />
+		<calibration reference_position="${arm_3_ref}"/>
+		<dynamics damping="10.0" friction="10.0" />
 		<limit effort="176" velocity="0.4189" lower="-6.2831853" upper="6.2831853"/>
 	</joint>
@@ -132,7 +132,7 @@
 		<child link="${name}_4_link"/>
 		<axis xyz="0 0 1" />
-	        <calibration reference_position="${arm_4_ref}"/>
-                <dynamics damping="30" />
-		<limit effort="176" velocity="0.4189" upper="2.0943951" lower="-2.0943951" />
+		<calibration reference_position="${arm_4_ref}"/>
+		<dynamics damping="10.0" friction="10.0" />
+		<limit effort="176" velocity="0.4189" lower="-2.0943951" upper="2.0943951"/>
 	</joint>
 	<link name="${name}_4_link">
@@ -162,7 +162,7 @@
 		<child link="${name}_5_link"/>
 		<axis xyz="0 0 1" />
-	        <calibration reference_position="${arm_5_ref}"/>
-                <dynamics damping="30" />
-		<limit effort="41.6" velocity="0.4363" upper="6.2831853" lower="-6.2831853" />
+		<calibration reference_position="${arm_5_ref}"/>
+		<dynamics damping="10.0" friction="10.0" />
+		<limit effort="41.6" velocity="0.4363" lower="-6.2831853" upper="6.2831853" />
 	</joint>
 	<link name="${name}_5_link">
@@ -192,7 +192,7 @@
 		<child link="${name}_6_link"/>
 		<axis xyz="0 0 1" />
-	        <calibration reference_position="${arm_6_ref}"/>
-                <dynamics damping="30" />
-		<limit effort="20.1" velocity="0.4363" upper="2.0943951" lower="-2.0943951" />
+		<calibration reference_position="${arm_6_ref}"/>
+		<dynamics damping="10.0" friction="10.0" />
+		<limit effort="20.1" velocity="0.4363" lower="-2.0943951" upper="2.0943951" />
 	</joint>
 	<link name="${name}_6_link">
@@ -222,7 +222,7 @@
 		<child link="${name}_7_link"/>
 		<axis xyz="0 0 1" />
-	        <calibration reference_position="${arm_7_ref}"/>
-                <dynamics damping="30" />
-		<limit effort="9.6" velocity="0.8727" upper="6.2831853" lower="-6.2831853" />
+		<calibration reference_position="${arm_7_ref}"/>
+		<dynamics damping="10.0" friction="10.0" />
+		<limit effort="9.6" velocity="0.8727" lower="-6.2831853" upper="6.2831853" />
 	</joint>
 	<link name="${name}_7_link">
