Commit message: modified urdf

File: ros/urdf/arm_v0/arm.urdf.xacro (robot description, xacro)
@@ -76,7 +76,7 @@
 	<link name="${name}_2_link">
 		<inertial>
-			<origin xyz="0 -0.006249 0.008252" rpy="0 0 0"/>
+			<origin xyz="0 -0.00629 0.008252" rpy="0 0 0"/>
 			<mass value="5.734939"/>
-			<inertia ixx="0.020715"  ixy="0"  ixz="0" iyy="0.017585" iyz="-0.000460" izz="0.014454" />
+			<inertia ixx="0.020715"  ixy="0"  ixz="0" iyy="0.017585" iyz="-0.000460" izz="0.01454" />
 		</inertial>
 		<visual>
@@ -105,7 +105,7 @@
 	<link name="${name}_3_link">
 		<inertial>
-			<origin xyz="0 0.007908 0.192805" rpy="0 0 0"/>
-			<mass value="4.214668"/>
-			<inertia ixx="0.192416"  ixy="0"  ixz="0" iyy="0.190323" iyz="0.000310" izz="0.008570" />
+			<origin xyz="0 0 0" rpy="0 0 0"/>
+			<mass value="2.0"/>
+			<inertia ixx="0.01"  ixy="0"  ixz="0" iyy="0.01" iyz="0" izz="0.01" />
 		</inertial>
 		<visual>
@@ -134,7 +134,7 @@
 	<link name="${name}_4_link">
 		<inertial>
-			<origin xyz="0 -0.006319 0.009681" rpy="0 0 0"/>
-			<mass value="3.669819"/>
-			<inertia ixx="0.010547"  ixy="0"  ixz="0" iyy="0.008708" iyz="-0.000335" izz="0.006913" />
+			<origin xyz="0 0 0" rpy="0 0 0"/>
+			<mass value="1.6"/>
+			<inertia ixx="0.01"  ixy="0"  ixz="0" iyy="0.01" iyz="0" izz="0.01" />
 		</inertial>
 		<visual>
@@ -163,7 +163,7 @@
 	<link name="${name}_5_link">
 		<inertial>
-			<origin xyz="0 -0.004963 0.008394" rpy="0 0 0"/>
-			<mass value="2.313272"/>
-			<inertia ixx="0.004108"  ixy="0"  ixz="0" iyy="0.003468" iyz="-0.000103" izz="0.002507" />
+			<origin xyz="0 0 0" rpy="0 0 0"/>
+			<mass value="1.2"/>
+			<inertia ixx="0.01"  ixy="0"  ixz="0" iyy="0.01" iyz="0" izz="0.01" />
 		</inertial>
 		<visual>

Commit message: small fix

File: ros/urdf/arm_v0/arm.urdf.xacro (robot description, xacro)
@@ -55,12 +55,12 @@
 			<origin xyz="0 0 0" rpy="0 0 0" />
 			<geometry>
-				<mesh filename="package://cob_description/ros/meshes/arm_v0/J1.STL" />
-			</geometry>
-                        <material name="Blue" />
-		</visual>
-		<collision>
-			<origin xyz="0 0 0" rpy="0 0 0" />
-			<geometry>
-				<mesh filename="package://cob_description/ros/meshes/arm_v0/J1.STL" />
+				<mesh filename="package://cob_description/ros/meshes/arm_v0/arm1.stl" />
+			</geometry>
+                        <material name="Blue" />
+		</visual>
+		<collision>
+			<origin xyz="0 0 0" rpy="0 0 0" />
+			<geometry>
+				<mesh filename="package://cob_description/ros/meshes/arm_v0/arm1.stl" />
 			</geometry>
 		</collision>
@@ -85,5 +85,5 @@
 			<origin xyz="0 0 0" rpy="0 0 0" />
 			<geometry>
-				<mesh filename="package://cob_description/ros/meshes/arm_v0/J2.STL" />
+				<mesh filename="package://cob_description/ros/meshes/arm_v0/arm2.stl" />
 			</geometry>
                         <material name="Red" />
@@ -92,5 +92,5 @@
 			<origin xyz="0 0 0" rpy="0 0 0" />
 			<geometry>
-				<mesh filename="package://cob_description/ros/meshes/arm_v0/J2.STL"/>
+				<mesh filename="package://cob_description/ros/meshes/arm_v0/arm2.stl"/>
 			</geometry>
 		</collision>
@@ -115,12 +115,12 @@
 			<origin xyz="0 0 0" rpy="0 0 0" />
 			<geometry>
-				<mesh filename="package://cob_description/ros/meshes/arm_v0/J3.STL" />
-			</geometry>
-                        <material name="Blue" />
-		</visual>
-		<collision>
-			<origin xyz="0 0 0" rpy="0 0 0" />
-			<geometry>
-				<mesh filename="package://cob_description/ros/meshes/arm_v0/J3.STL"/>
+				<mesh filename="package://cob_description/ros/meshes/arm_v0/arm3.stl" />
+			</geometry>
+                        <material name="Blue" />
+		</visual>
+		<collision>
+			<origin xyz="0 0 0" rpy="0 0 0" />
+			<geometry>
+				<mesh filename="package://cob_description/ros/meshes/arm_v0/arm3.stl"/>
 			</geometry>
 		</collision>
@@ -145,5 +145,5 @@
 			<origin xyz="0 0 0" rpy="0 0 0" />
 			<geometry>
-				<mesh filename="package://cob_description/ros/meshes/arm_v0/J4.STL" />
+				<mesh filename="package://cob_description/ros/meshes/arm_v0/arm4.stl" />
 			</geometry>
                         <material name="Red" />
@@ -152,5 +152,5 @@
 			<origin xyz="0 0 0" rpy="0 0 0" />
 			<geometry>
-				<mesh filename="package://cob_description/ros/meshes/arm_v0/J4.STL"/>
+				<mesh filename="package://cob_description/ros/meshes/arm_v0/arm4.stl"/>
 			</geometry>
 		</collision>
@@ -175,12 +175,12 @@
 			<origin xyz="0 0 0" rpy="0 0 0" />
 			<geometry>
-				<mesh filename="package://cob_description/ros/meshes/arm_v0/J5.STL" />
-			</geometry>
-                        <material name="Blue" />
-		</visual>
-		<collision>
-			<origin xyz="0 0 0" rpy="0 0 0" />
-			<geometry>
-				<mesh filename="package://cob_description/ros/meshes/arm_v0/J5.STL"/>
+				<mesh filename="package://cob_description/ros/meshes/arm_v0/arm5.stl" />
+			</geometry>
+                        <material name="Blue" />
+		</visual>
+		<collision>
+			<origin xyz="0 0 0" rpy="0 0 0" />
+			<geometry>
+				<mesh filename="package://cob_description/ros/meshes/arm_v0/arm5.stl"/>
 			</geometry>
 		</collision>
@@ -205,5 +205,5 @@
 			<origin xyz="0 0 0" rpy="0 0 0" />
 			<geometry>
-				<mesh filename="package://cob_description/ros/meshes/arm_v0/J6.STL" />
+				<mesh filename="package://cob_description/ros/meshes/arm_v0/arm6.stl" />
 			</geometry>
                         <material name="Red" />
@@ -212,5 +212,5 @@
 			<origin xyz="0 0 0" rpy="0 0 0" />
 			<geometry>
-				<mesh filename="package://cob_description/ros/meshes/arm_v0/J6.STL"/>
+				<mesh filename="package://cob_description/ros/meshes/arm_v0/arm6.stl"/>
 			</geometry>
 		</collision>
@@ -235,12 +235,12 @@
 			<origin xyz="0 0 0" rpy="0 0 0" />
 			<geometry>
-				<mesh filename="package://cob_description/ros/meshes/arm_v0/J7.STL" />
-			</geometry>
-                        <material name="Blue" />
-		</visual>
-		<collision>
-			<origin xyz="0 0 0" rpy="0 0 0" />
-			<geometry>
-				<mesh filename="package://cob_description/ros/meshes/arm_v0/J7.STL"/>
+				<mesh filename="package://cob_description/ros/meshes/arm_v0/arm7.stl" />
+			</geometry>
+                        <material name="Blue" />
+		</visual>
+		<collision>
+			<origin xyz="0 0 0" rpy="0 0 0" />
+			<geometry>
+				<mesh filename="package://cob_description/ros/meshes/arm_v0/arm7.stl"/>
 			</geometry>
 		</collision>

Commit message: extended limits of joint 1

File: ros/urdf/arm_v0/arm.urdf.xacro (robot description, xacro)
@@ -44,5 +44,5 @@
 	        <calibration reference_position="${arm_1_ref}"/>
                 <dynamics damping="20" />
-		<limit effort="370" velocity="0.4363" lower="-2.0943951" upper="2.0943951"/>
+		<limit effort="370" velocity="0.4363" lower="-6.2831853" upper="6.2831853"/>
 	</joint>
 	<link name="${name}_1_link">

Commit message: modified urdf to work with hokuyo simulation

File: ros/urdf/arm_v0/arm.urdf.xacro (robot description, xacro)
@@ -23,7 +23,7 @@
 		</inertial>
 		<visual>
-		   <origin xyz="0 0 0.005" rpy="0 0 0" />
+		   <origin xyz="0 0 0.09" rpy="0 0 0" />
 		   <geometry>
-		      <box size="0.01 0.01 0.01"/>
+		      <cylinder radius="0.045" length="0.18"/>
 		   </geometry>
 		   <material name="Red" />

File: ros/urdf/head_cameras_v0/head_cameras.urdf.xacro (robot description, xacro)
@@ -20,5 +20,5 @@
        <dynamics damping="0.1" />
        <calibration reference_position="${head_camera_axis_ref}"/>
-       <limit effort="100" lower="-0.1745" upper="3.316" velocity="0.5"/>
+       <limit effort="100" lower="-1.5" upper="3.316" velocity="0.5"/>
     </joint>
     <link name="${name}_camera_axis_link">

File: ros/urdf/sensors/hokuyo_SR400_laser.gazebo.xacro (robot description, xacro)
@@ -14,5 +14,5 @@
         <minAngle>${min_angle*180.0/M_PI}</minAngle>
         <maxAngle>${max_angle*180.0/M_PI}</maxAngle>
-        <minRange>0.8</minRange>
+        <minRange>0.30</minRange>
         <maxRange>5.0</maxRange>
         <resRange>0.01</resRange>

Commit message: use stlb files in collision now

File: ros/urdf/arm_v0/arm.urdf.xacro (robot description, xacro)
@@ -59,5 +59,5 @@
 				<origin xyz="0 0 0" rpy="0 0 0" />
 				<geometry>
-					<mesh filename="package://cob_description/ros/meshes/arm_v0/arm1.stl" />
+					<mesh filename="package://cob_description/ros/meshes/arm_v0/arm1.stlb" />
 				</geometry>
 			</collision>
@@ -89,5 +89,5 @@
 				<origin xyz="0 0 0" rpy="0 0 0" />
 				<geometry>
-					<mesh filename="package://cob_description/ros/meshes/arm_v0/arm2.stl"/>
+					<mesh filename="package://cob_description/ros/meshes/arm_v0/arm2.stlb"/>
 				</geometry>
 			</collision>
@@ -119,5 +119,5 @@
 				<origin xyz="0 0 0" rpy="0 0 0" />
 				<geometry>
-					<mesh filename="package://cob_description/ros/meshes/arm_v0/arm3.stl"/>
+					<mesh filename="package://cob_description/ros/meshes/arm_v0/arm3.stlb"/>
 				</geometry>
 			</collision>
@@ -149,5 +149,5 @@
 				<origin xyz="0 0 0" rpy="0 0 0" />
 				<geometry>
-					<mesh filename="package://cob_description/ros/meshes/arm_v0/arm4.stl"/>
+					<mesh filename="package://cob_description/ros/meshes/arm_v0/arm4.stlb"/>
 				</geometry>
 			</collision>
@@ -179,5 +179,5 @@
 				<origin xyz="0 0 0" rpy="0 0 0" />
 				<geometry>
-					<mesh filename="package://cob_description/ros/meshes/arm_v0/arm5.stl"/>
+					<mesh filename="package://cob_description/ros/meshes/arm_v0/arm5.stlb"/>
 				</geometry>
 			</collision>
@@ -209,5 +209,5 @@
 				<origin xyz="0 0 0" rpy="0 0 0" />
 				<geometry>
-					<mesh filename="package://cob_description/ros/meshes/arm_v0/arm6.stl"/>
+					<mesh filename="package://cob_description/ros/meshes/arm_v0/arm6.stlb"/>
 				</geometry>
 			</collision>
@@ -239,5 +239,5 @@
 				<origin xyz="0 0 0" rpy="0 0 0" />
 				<geometry>
-					<mesh filename="package://cob_description/ros/meshes/arm_v0/arm7.stl"/>
+					<mesh filename="package://cob_description/ros/meshes/arm_v0/arm7.stlb"/>
 				</geometry>
 			</collision>

File: ros/urdf/base_v0/base.urdf.xacro (robot description, xacro)
@@ -147,14 +147,19 @@
         <!-- represent base collision with a simple rectangular model, positioned by base_size_z s.t. top
              surface of the collision box matches the top surface of the PR2 base -->
-<!--original model: works for platform-navigation
-        <origin xyz="0 0 ${base_size_z-base_collision_size_z/2}" rpy="0 0 0" />
+		<!--original box-shaped model: works for platform-navigation -->
+        <!--<origin xyz="0 0 ${base_size_z-base_collision_size_z/2}" rpy="0 0 0" />
         <geometry>
           <box size="${base_size_x} ${base_size_y} ${base_collision_size_z}" />
-        </geometry>
--->
+        </geometry>-->
+		<!--second box-shaped model:-->
 		<origin xyz="${base_size_x2/2} 0 ${base_size_z2}" rpy="0 0 0" />
         <geometry>
           <box size="${base_size_x2} ${base_size_y2} ${base_collision_size_z2}" />
         </geometry>
+		<!--latest collision model using meshes -->
+		<!--<origin xyz="0 0 0" rpy="0 0 0" />
+        <geometry>
+	      <mesh filename="package://cob_description/ros/meshes/base_v0/base_collision.stlb"/>
+        </geometry>-->
       </collision>
     </link>

File: ros/urdf/base_v1/base.urdf.xacro (robot description, xacro)
@@ -147,5 +147,5 @@
         <geometry>
 		  <!--box size="0.001 0.001 0.001" /-->
-	      <mesh filename="package://cob_description/ros/meshes/base_v0/base_collision.stl"/>
+	      <mesh filename="package://cob_description/ros/meshes/base_v0/base_collision.stlb"/>
           <!--box size="${base_size_x} ${base_size_y} ${base_collision_size_z}" /-->
         </geometry>

File: ros/urdf/lbr_v0/lbr.urdf.xacro (robot description, xacro)
@@ -61,5 +61,5 @@
 				<origin xyz="0 0 0" rpy="0 0 0" />
 				<geometry>
-					<mesh filename="package://cob_description/ros/meshes/lbr_v0/joint_1_collision.stl" />
+					<mesh filename="package://cob_description/ros/meshes/lbr_v0/joint_1_collision.stlb" />
 				</geometry>
 			</collision>
@@ -93,5 +93,5 @@
 				<origin xyz="0 0 0" rpy="0 0 0" />
 				<geometry>
-					<mesh filename="package://cob_description/ros/meshes/lbr_v0/joint_2_collision.stl"/>
+					<mesh filename="package://cob_description/ros/meshes/lbr_v0/joint_2_collision.stlb"/>
 				</geometry>
 			</collision>
@@ -125,5 +125,5 @@
 				<origin xyz="0 0 0" rpy="0 0 0" />
 				<geometry>
-					<mesh filename="package://cob_description/ros/meshes/lbr_v0/joint_3_collision.stl"/>
+					<mesh filename="package://cob_description/ros/meshes/lbr_v0/joint_3_collision.stlb"/>
 				</geometry>
 			</collision>
@@ -157,5 +157,5 @@
 				<origin xyz="0 0 0" rpy="0 0 0" />
 				<geometry>
-					<mesh filename="package://cob_description/ros/meshes/lbr_v0/joint_4_collision.stl"/>
+					<mesh filename="package://cob_description/ros/meshes/lbr_v0/joint_4_collision.stlb"/>
 				</geometry>
 			</collision>
@@ -189,5 +189,5 @@
 				<origin xyz="0 0 0" rpy="0 0 0" />
 				<geometry>
-					<mesh filename="package://cob_description/ros/meshes/lbr_v0/joint_5_collision.stl"/>
+					<mesh filename="package://cob_description/ros/meshes/lbr_v0/joint_5_collision.stlb"/>
 				</geometry>
 			</collision>
@@ -221,5 +221,5 @@
 				<origin xyz="0 0 0" rpy="0 0 0" />
 				<geometry>
-					<mesh filename="package://cob_description/ros/meshes/lbr_v0/joint_6_collision.stl"/>
+					<mesh filename="package://cob_description/ros/meshes/lbr_v0/joint_6_collision.stlb"/>
 				</geometry>
 			</collision>
@@ -253,5 +253,5 @@
 				<origin xyz="0 0 0" rpy="0 0 0" />
 				<geometry>
-					<mesh filename="package://cob_description/ros/meshes/lbr_v0/joint_7_collision.stl"/>
+					<mesh filename="package://cob_description/ros/meshes/lbr_v0/joint_7_collision.stlb"/>
 				</geometry>
 			</collision>

File: ros/urdf/sdh_v0/sdh.urdf.xacro (robot description, xacro)
@@ -29,5 +29,5 @@
 				<origin xyz="0 0 0" rpy="0 0 0" />
 				<geometry>
-					<mesh filename="package://cob_description/ros/meshes/sdh_v0/palm.stl"/>
+					<mesh filename="package://cob_description/ros/meshes/sdh_v0/palm.stlb"/>
 				</geometry>
 			</collision>
@@ -66,5 +66,5 @@
 				<origin xyz="0 0 0" rpy="0 0 0" />
 				<geometry>
-				<mesh filename="package://cob_description/ros/meshes/sdh_v0/knuckle.stl"/>
+				<mesh filename="package://cob_description/ros/meshes/sdh_v0/knuckle.stlb"/>
 				</geometry>
 			</collision>
@@ -95,5 +95,5 @@
 				<origin xyz="0 0 0" rpy="0 0 0" />
 				<geometry>
-					<mesh filename="package://cob_description/ros/meshes/sdh_v0/finger.stl"/>
+					<mesh filename="package://cob_description/ros/meshes/sdh_v0/finger.stlb"/>
 				</geometry>
 			</collision>
@@ -124,5 +124,5 @@
 				<origin xyz="0 0 0" rpy="0 0 0" />
 				<geometry>
-					<mesh filename="package://cob_description/ros/meshes/sdh_v0/finger_tip.stl"/>
+					<mesh filename="package://cob_description/ros/meshes/sdh_v0/finger_tip.stlb"/>
 				</geometry>
 			</collision>
@@ -154,5 +154,5 @@
 				<origin xyz="0 0 0" rpy="1.57079633 0 0" />
 				<geometry>
-					<mesh filename="package://cob_description/ros/meshes/sdh_v0/knuckle.stl"/>
+					<mesh filename="package://cob_description/ros/meshes/sdh_v0/knuckle.stlb"/>
 				</geometry>
 			</collision>
@@ -183,5 +183,5 @@
 				<origin xyz="0 0 0" rpy="0 0 0" />
 				<geometry>
-					<mesh filename="package://cob_description/ros/meshes/sdh_v0/finger.stl"/>
+					<mesh filename="package://cob_description/ros/meshes/sdh_v0/finger.stlb"/>
 				</geometry>
 			</collision>
@@ -212,5 +212,5 @@
 				<origin xyz="0 0 0" rpy="0 0 0" />
 				<geometry>
-					<mesh filename="package://cob_description/ros/meshes/sdh_v0/finger_tip.stl"/>
+					<mesh filename="package://cob_description/ros/meshes/sdh_v0/finger_tip.stlb"/>
 				</geometry>
 			</collision>
@@ -239,5 +239,5 @@
 				<origin xyz="0 0 0" rpy="0 0 0" />
 				<geometry>
-					<mesh filename="package://cob_description/ros/meshes/sdh_v0/knuckle.stl"/>
+					<mesh filename="package://cob_description/ros/meshes/sdh_v0/knuckle.stlb"/>
 				</geometry>
 			</collision>
@@ -268,5 +268,5 @@
 				<origin xyz="0 0 0" rpy="0 0 0" />
 				<geometry>
-					<mesh filename="package://cob_description/ros/meshes/sdh_v0/finger.stl"/>
+					<mesh filename="package://cob_description/ros/meshes/sdh_v0/finger.stlb"/>
 				</geometry>
 			</collision>
@@ -297,5 +297,5 @@
 				<origin xyz="0 0 0" rpy="0 0 0" />
 				<geometry>
-					<mesh filename="package://cob_description/ros/meshes/sdh_v0/finger_tip.stl"/>
+					<mesh filename="package://cob_description/ros/meshes/sdh_v0/finger_tip.stlb"/>
 				</geometry>
 			</collision>

File: ros/urdf/torso_v0/torso.urdf.xacro (robot description, xacro)
@@ -33,5 +33,5 @@
 				<origin xyz="0 0 0" rpy="0 0 0" />
 				<geometry>
-					<mesh filename="package://cob_description/ros/meshes/torso_v0/tray_collision.stl" />
+					<mesh filename="package://cob_description/ros/meshes/torso_v0/tray_collision.stlb" />
 				</geometry>
 			</collision>
@@ -93,5 +93,5 @@
 				<origin xyz="0 0 0" rpy="0 0 0" />
 				<geometry>
-					<mesh filename="package://cob_description/ros/meshes/torso_v0/lower_neck_collision.stl" />
+					<mesh filename="package://cob_description/ros/meshes/torso_v0/lower_neck_collision.stlb" />
 				</geometry>
 			</collision>
@@ -153,5 +153,5 @@
 				<origin xyz="0 0 0" rpy="0 0 0" />
 				<geometry>
-					<mesh filename="package://cob_description/ros/meshes/torso_v0/upper_neck_collision.stl" />
+					<mesh filename="package://cob_description/ros/meshes/torso_v0/upper_neck_collision.stlb" />
 				</geometry>
 			</collision>
@@ -179,5 +179,5 @@
 				<origin xyz="0 0 0" rpy="0 0 0" />
 				<geometry>
-					<mesh filename="package://cob_description/ros/meshes/torso_v0/head_cover_collision.stl" />
+					<mesh filename="package://cob_description/ros/meshes/torso_v0/head_cover_collision.stlb" />
 				</geometry>
 			</collision>
