Commit message: modified urdf and adapted xaml files

File: ros/urdf/head_cameras_v0/head_cameras.urdf.xacro (robot description, xacro)
@@ -13,5 +13,5 @@
   <xacro:macro name="cob_head_cameras_v0" params="name parent *origin">
     <!--joint between torso_upper_neck_tilt_link and head_camera_axis_link-->
-    <joint name="${name}_camera_axis_joint" type="revolute">
+    <joint name="${name}_camera_axis_joint" type="fixed">
        <insert_block name="origin" />
        <parent link="${parent}"/>
@@ -22,24 +22,24 @@
        <limit effort="100" lower="-1.5" upper="3.316" velocity="0.5"/>
     </joint>
-    <link name="${name}_camera_axis_link">
-       <inertial>
-	  <origin xyz="0 0 0" rpy="0 0 0"/>
-	  <mass value="0.1"/>
-	  <inertia ixx="0.0001"  ixy="0"  ixz="0" iyy="0.0001" iyz="0" izz="0.0001" />
-       </inertial>
-       <visual>
-	 <origin xyz="0 0 0" rpy="0 0 0" />
-	 <geometry>
-	    <box size="0.1 0.1 0.01"/>
-	 </geometry>
-         <material name="Green" />
-       </visual>
-       <collision>
-	 <origin xyz="0 0 0" rpy="0 0 0" />
-	 <geometry>
-            <box size="0.1 0.1 0.01"/>
-	 </geometry>
-       </collision>
-    </link>
+	<link name="${name}_camera_axis_link">
+		<inertial>
+			<origin xyz="0 0 0" rpy="0 0 0"/>
+			<mass value="0.1"/>
+			<inertia ixx="0.0001"  ixy="0"  ixz="0" iyy="0.0001" iyz="0" izz="0.0001" />
+		</inertial>
+		<visual>
+			<origin xyz="0 0 0" rpy="0 0 0" />
+			<geometry>
+				<box size="0.1 0.1 0.01"/>
+			</geometry>
+			<material name="Green" />
+		</visual>
+		<collision>
+			<origin xyz="0 0 0" rpy="0 0 0" />
+			<geometry>
+				<box size="0.1 0.1 0.01"/>
+			</geometry>
+		</collision>
+	</link>
     <!--##################################################-->
     <!-- camera test here -->
@@ -48,5 +48,5 @@
     </xacro:cob_cameraone_v0>
     <xacro:cob_cameraone_v0 name="${name}_color_camera_r" parent="${name}_camera_axis_link">
-      <origin xyz="${cam_r_x} ${cam_r_y} ${cam_r_z+0.06}" rpy="${cam_r_roll} ${cam_r_pitch-1.5708} ${cam_r_yaw+3.14159}" />
+      <origin xyz="${cam_r_x} ${cam_r_y} ${cam_r_z-0.06}" rpy="${cam_r_roll} ${cam_r_pitch+1.5708} ${cam_r_yaw+3.14159}" />
     </xacro:cob_cameraone_v0>
     <!-- hokuyo_SR400_laser test here-->

Commit message: fixed bug with fixed joint

File: ros/urdf/head_cameras_v0/head_cameras.urdf.xacro (robot description, xacro)
@@ -13,5 +13,5 @@
   <xacro:macro name="cob_head_cameras_v0" params="name parent *origin">
     <!--joint between torso_upper_neck_tilt_link and head_camera_axis_link-->
-    <joint name="${name}_camera_axis_joint" type="fixed">
+    <joint name="${name}_camera_axis_joint" type="revolute">
        <insert_block name="origin" />
        <parent link="${parent}"/>
