Commit message: simulated cameras working

File: ros/urdf/sensors/cameraone.gazebo.xacro (robot description, xacro)
@@ -5,5 +5,5 @@
       xmlns:xacro="http://ros.org/wiki/xacro">
 <xacro:macro name="cob_cameraone_gazebo_v0" params="name">
-  <gazebo reference="${name}_link">
+  <gazebo reference="${name}_frame">
     <sensor:camera name="${name}_sensor">
       <imageFormat>R8G8B8</imageFormat>

File: ros/urdf/sensors/cameraone.urdf.xacro (robot description, xacro)
@@ -32,4 +32,29 @@
       </collision >
     </link>
+    <joint name="${name}_frame_joint" type="fixed">
+      <origin xyz="0 0 0" rpy="1.5708 -1.5708 0" />
+      <parent link="${name}_link"/>
+      <child link="${name}_frame"/>
+    </joint>
+    <link name="${name}_frame">
+      <inertial>
+        <mass value="0.01" />
+        <origin xyz="0 0 0" rpy="0 0 0"/>
+        <inertia ixx="0.0001" ixy="0" ixz="0" iyy="0.0001" iyz="0" izz="0.0001" />
+      </inertial>
+      <visual>
+        <origin xyz="0 0 0" rpy="0 0 0" />
+        <geometry>
+          <cylinder radius="0.005" length="0.005"/>
+        </geometry>
+        <material name="Red" />
+      </visual>
+      <collision>
+        <origin xyz="0 0 0" rpy="0 0 0" />
+        <geometry>
+           <cylinder radius="0.001" length="0.001"/>
+        </geometry>
+      </collision >
+    </link>
    <xacro:cob_cameraone_gazebo_v0 name="${name}"/>
   </xacro:macro>
