Commit message: inserted new stl files

File: ros/urdf/base_v0/base.urdf.xacro (robot description, xacro)
@@ -173,5 +173,5 @@
     </link>
     <joint name="${name}_footprint_joint" type="fixed">
-      <origin xyz="0 0 0.051" rpy="0 0 0" />
+      <origin xyz="0 0 0" rpy="0 0 0" />
       <child link="${name}_link" />
       <parent link="${name}_footprint"/>

File: ros/urdf/torso_v0/torso.urdf.xacro (robot description, xacro)
@@ -104,5 +104,5 @@
     <!--joint between torso_lower_neck_tilt_link and torso_upper_neck_pan_link-->
     <joint name="${name}_upper_neck_pan_joint" type="revolute">
-      <origin xyz="-0.09039 -0.30489 0" rpy="-1.5708 0 0" />
+      <origin xyz="0 -0.30489 0" rpy="-1.5708 0 0" />
       <parent link="${name}_lower_neck_tilt_link"/>
       <child link="${name}_upper_neck_pan_link"/>
@@ -177,5 +177,5 @@
 	   <origin xyz="0 0 0" rpy="0 0 0" />
 	   <geometry>
-              <mesh filename="package://cob_defs/common/files/meshes/head_cover.stl" />
+			<mesh filename="package://cob_description/ros/meshes/torso_v0/head_cover.stl" />
 	   </geometry>
            <material name="Blue" />
@@ -184,5 +184,5 @@
 	   <origin xyz="0 0 0" rpy="0 0 0" />
 	   <geometry>
-              <mesh filename="package://cob_defs/common/files/meshes/head_cover.stl" />
+			<mesh filename="package://cob_description/ros/meshes/torso_v0/head_cover.stl" />
 	   </geometry>
 	</collision>

Commit message: new files for navigation, e.g. maps and launch files

File: ros/urdf/base_v0/base.urdf.xacro (robot description, xacro)
@@ -131,5 +131,5 @@
       </inertial>
       <visual>
-        <origin xyz="0 0 ${base_collision_size_z/2}" rpy="0 0 0" />
+        <origin xyz="0 0 0" rpy="0 0 0" />
         <!-- modify here for test-->
         <geometry>
@@ -173,19 +173,19 @@
     </link>
     <joint name="${name}_footprint_joint" type="fixed">
-      <origin xyz="0 0 0.051" rpy="0 0 0" />
+      <origin xyz="0 0 0" rpy="0 0 0" />
       <child link="${name}_link" />
       <parent link="${name}_footprint"/>
     </joint>
     <!--modify here for test: front,base and top lasers -->
-    <!-- base scanner front -->
-    <xacro:hokuyo_lx30_laser_v0 name="${name}_scanner_front" parent="${name}" ros_topic="base_scan_front" update_rate="20" min_angle="-1.35" max_angle="1.35" >
+    <!-- base laser front -->
+    <xacro:hokuyo_lx30_laser_v0 name="${name}_laser_front" parent="${name}" ros_topic="base_scan_front" update_rate="20" min_angle="-1.35" max_angle="1.35" >
       <origin xyz="${base_laser_x} ${base_laser_y} ${base_laser_z}" rpy="0 0 0" />
     </xacro:hokuyo_lx30_laser_v0>
-    <!-- base scanner rear -->
-    <xacro:hokuyo_lx30_laser_v0 name="${name}_scanner_rear" parent="${name}" ros_topic="base_scan_rear" update_rate="20" min_angle="-1.35" max_angle="1.35" >
+    <!-- base laser rear -->
+    <xacro:hokuyo_lx30_laser_v0 name="${name}_laser_rear" parent="${name}" ros_topic="base_scan_rear" update_rate="20" min_angle="-1.35" max_angle="1.35" >
       <origin xyz="${-base_laser_x} ${base_laser_y} ${base_laser_z}" rpy="0 0 ${M_PI}" />
     </xacro:hokuyo_lx30_laser_v0>
-    <!-- base scanner top -->
-    <xacro:hokuyo_lx30_laser_v0 name="${name}_scanner_top" parent="${name}" ros_topic="base_scan_top" update_rate="10" min_angle="-2.094" max_angle="2.094" >
+    <!-- base laser top -->
+    <xacro:hokuyo_lx30_laser_v0 name="${name}_laser_top" parent="${name}" ros_topic="base_scan_top" update_rate="10" min_angle="-2.094" max_angle="2.094" >
       <origin xyz="-0.252 0 0.42" rpy="0 0 ${M_PI}" />
     </xacro:hokuyo_lx30_laser_v0>

Commit message: changed mesh files for new transformations

File: ros/urdf/base_v0/base.urdf.xacro (robot description, xacro)
@@ -134,5 +134,5 @@
         <!-- modify here for test-->
         <geometry>
-          <mesh filename="package://cob_defs/common/files/meshes/platform.stl"/>
+          <mesh filename="package://cob_description/ros/meshes/base_v0/base.stl"/>
         </geometry>
         <material name="Grey"/>

File: ros/urdf/base_v0_ipa/base.urdf.xacro (robot description, xacro)
@@ -136,5 +136,5 @@
         <!-- modify here for test-->
         <geometry>
-          <mesh filename="package://cob_defs/common/files/meshes/platform.stl"/>
+          <mesh filename="package://cob_description/ros/meshes/base_v0/base.stl"/>
           <!--box size="0.6 0.8 0.1" /-->
         </geometry>
@@ -146,5 +146,5 @@
         <origin xyz="0 0 0" rpy="0 0 0" />
         <geometry>
-          <!--mesh filename="package://cob_defs/common/files/meshes/platform.stl"/-->
+          <!--mesh filename="package://cob_description/ros/meshes/base_v0/base.stl"/-->
           <box size="0.6 0.8 0.1" />
         </geometry>

File: ros/urdf/base_v1/base.urdf.xacro (robot description, xacro)
@@ -135,5 +135,5 @@
         <origin xyz="0 0 0" rpy="0 0 0" />
         <geometry>
-          <mesh filename="package://cob_defs/common/files/meshes/platform.stl"/>
+          <mesh filename="package://cob_description/ros/meshes/base_v0/base.stl"/>
           <!--box size="${base_size_x} ${base_size_y} ${base_collision_size_z}" /-->
         </geometry>
@@ -143,5 +143,5 @@
         <origin xyz="0 0 0" rpy="0 0 0" />
         <geometry>
-	      <mesh filename="package://cob_defs/common/files/meshes/platform.stl"/>
+	      <mesh filename="package://cob_description/ros/meshes/base_v0/base.stl"/>
           <!--box size="${base_size_x} ${base_size_y} ${base_collision_size_z}" /-->
         </geometry>

Commit message: simple base collision model

File: ros/urdf/base_v0/base.urdf.xacro (robot description, xacro)
@@ -17,6 +17,9 @@
   <property name="caster_offset_y" value="0.185" />
   <property name="caster_offset_z" value="0.0282" />
+<!--TODO: adjust base collision model and wheel values -->
+  <!--property name="caster_wheel_offset_y" value="0.01" /-->
   <property name="caster_wheel_offset_y" value="0.049" />
   <property name="wheel_length" value="0.034" />
+  <!--property name="wheel_radius" value="0.05" /-->
   <property name="wheel_radius" value="0.074792" />   <!-- This is the 'effective' wheel radius. Wheel radius for uncompressed wheel is 0.079.  mp 20080801 -->
   <property name="base_cg_x" value="-0.061" />
@@ -24,5 +27,10 @@
   <property name="base_cg_z" value="0.293" />
   <property name="base_mass" value="116.0" />
-  <!-- simplified box collision geometry for base -->
+<!-- uhr-messmerf -->
+  <property name="base_size_x2" value="0.4" />
+  <property name="base_size_y2" value="0.5" />
+  <property name="base_size_z2" value="0.4" />
+  <property name="base_collision_size_z2" value="0.6" />
+<!-- simplified box collision geometry for base -->
   <property name="base_size_x" value="0.8" />
   <property name="base_size_y" value="0.6" />
@@ -104,5 +112,5 @@
         <origin xyz="0 0 0.07" rpy="0.0 0.0 0.0" />
         <geometry>
-          <box size="0.192 0.164 0.013" />
+          <box size="0.01 0.01 0.01" />
         </geometry>
       </collision>
@@ -142,8 +150,21 @@
         <!-- represent base collision with a simple rectangular model, positioned by base_size_z s.t. top
              surface of the collision box matches the top surface of the PR2 base -->
+		<!--
+		<origin xyz="0 0 0" rpy="0 0 0" />
+        <geometry>
+          <mesh filename="package://cob_description/ros/meshes/base_v0/base.stl"/>
+        </geometry>
+		-->
+        <origin xyz="${base_size_x2/2} 0 ${base_size_z2}" rpy="0 0 0" />
+        <geometry>
+          <box size="${base_size_x2} ${base_size_y2} ${base_collision_size_z2}" />
+        </geometry>
+		<!--
+		OLD collision model
         <origin xyz="0 0 ${base_size_z-base_collision_size_z/2}" rpy="0 0 0" />
         <geometry>
           <box size="${base_size_x} ${base_size_y} ${base_collision_size_z}" />
         </geometry>
+		-->
       </collision>
     </link>

Commit message: modified base collision model for 2dnav_ipa

File: ros/urdf/base_v0/base.urdf.xacro (robot description, xacro)
@@ -17,9 +17,6 @@
   <property name="caster_offset_y" value="0.185" />
   <property name="caster_offset_z" value="0.0282" />
-<!--TODO: adjust base collision model and wheel values -->
-  <!--property name="caster_wheel_offset_y" value="0.01" /-->
   <property name="caster_wheel_offset_y" value="0.049" />
   <property name="wheel_length" value="0.034" />
-  <!--property name="wheel_radius" value="0.05" /-->
   <property name="wheel_radius" value="0.074792" />   <!-- This is the 'effective' wheel radius. Wheel radius for uncompressed wheel is 0.079.  mp 20080801 -->
   <property name="base_cg_x" value="-0.061" />
@@ -27,10 +24,10 @@
   <property name="base_cg_z" value="0.293" />
   <property name="base_mass" value="116.0" />
-<!-- uhr-messmerf -->
+  <!-- uhr-messmerf -->
   <property name="base_size_x2" value="0.4" />
   <property name="base_size_y2" value="0.5" />
-  <property name="base_size_z2" value="0.4" />
-  <property name="base_collision_size_z2" value="0.6" />
-<!-- simplified box collision geometry for base -->
+  <property name="base_size_z2" value="0.5" />
+  <property name="base_collision_size_z2" value="0.4" />
+  <!-- simplified box collision geometry for base -->
   <property name="base_size_x" value="0.8" />
   <property name="base_size_y" value="0.6" />
@@ -112,5 +109,5 @@
         <origin xyz="0 0 0.07" rpy="0.0 0.0 0.0" />
         <geometry>
-          <box size="0.01 0.01 0.01" />
+          <box size="0.192 0.164 0.013" />
         </geometry>
       </collision>
@@ -150,21 +147,14 @@
         <!-- represent base collision with a simple rectangular model, positioned by base_size_z s.t. top
              surface of the collision box matches the top surface of the PR2 base -->
-		<!--
-		<origin xyz="0 0 0" rpy="0 0 0" />
-        <geometry>
-          <mesh filename="package://cob_description/ros/meshes/base_v0/base.stl"/>
-        </geometry>
-		-->
-        <origin xyz="${base_size_x2/2} 0 ${base_size_z2}" rpy="0 0 0" />
+<!--original model: works for platform-navigation
+        <origin xyz="0 0 ${base_size_z-base_collision_size_z/2}" rpy="0 0 0" />
+        <geometry>
+          <box size="${base_size_x} ${base_size_y} ${base_collision_size_z}" />
+        </geometry>
+-->
+		<origin xyz="${base_size_x2/2} 0 ${base_size_z2}" rpy="0 0 0" />
         <geometry>
           <box size="${base_size_x2} ${base_size_y2} ${base_collision_size_z2}" />
         </geometry>
-		<!--
-		OLD collision model
-        <origin xyz="0 0 ${base_size_z-base_collision_size_z/2}" rpy="0 0 0" />
-        <geometry>
-          <box size="${base_size_x} ${base_size_y} ${base_collision_size_z}" />
-        </geometry>
-		-->
       </collision>
     </link>
