Commit message: head axis working in simulation

File: ros/urdf/head_v0/head.urdf.xacro (robot description, xacro)
@@ -20,5 +20,5 @@
        <dynamics damping="0.1" />
        <calibration rising="${head_axis_ref}" falling="${head_axis_ref}"/>
-       <limit effort="100" lower="-1.5" upper="3.316" velocity="0.5"/>
+       <limit effort="100" lower="-3.2" upper="0.1" velocity="0.5"/>
     </joint>
 	<link name="${name}_axis_link">
@@ -45,6 +45,6 @@
 	<joint name="${name}_tof_tilt_joint" type="revolute">
 		<origin xyz="0 0 0" rpy="0 0 0" />
-		<parent link="${name}_tof_camera_link"/>
-		<child link="${name}_tof_axis_link"/>
+		<parent link="${name}_tof_link"/>
+		<child link="${name}_tof_tilt_link"/>
 		<axis xyz="0 0 1" />
 		<dynamics damping="25.0" friction="10.0"/>
@@ -81,5 +81,5 @@
     </xacro:cob_cameraone_v0>
     <!-- hokuyo_SR400_laser test here-->
-    <xacro:hokuyo_SR400_laser_v0 name="${name}_tof_camera" parent="${name}_color_camera_r_link" ros_topic="head_scan" update_rate="54" min_angle="-0.302" max_angle="0.302" >
+    <xacro:hokuyo_SR400_laser_v0 name="${name}_tof" parent="${name}_color_camera_r_link" ros_topic="head_scan" update_rate="54" min_angle="-0.302" max_angle="0.302" >
       <origin xyz="${tof_x-0.06} ${tof_y} ${tof_z}" rpy="${tof_roll} ${tof_pitch} ${tof_yaw}" />
     </xacro:hokuyo_SR400_laser_v0>

Commit message: preparation for blocklaser

File: ros/urdf/head_v0/head.urdf.xacro (robot description, xacro)
@@ -7,4 +7,5 @@
   <include filename="$(find cob_description)/ros/urdf/head_v0/head.transmission.xacro" />
   <include filename="$(find cob_description)/ros/urdf/sensors/cameraone.urdf.xacro" />
+  <include filename="$(find cob_description)/ros/urdf/sensors/tof.urdf.xacro" />
   <include filename="$(find cob_description)/ros/urdf/sensors/hokuyo_SR400_laser.urdf.xacro" />
 <!--####################################################################-->
@@ -42,46 +43,17 @@
 		</collision>
 	</link>
-	<!--joint between head_axis_link and head_tof_axis_link-->
-	<joint name="${name}_tof_tilt_joint" type="revolute">
-		<origin xyz="0 0 0" rpy="0 0 0" />
-		<parent link="${name}_tof_link"/>
-		<child link="${name}_tof_tilt_link"/>
-		<axis xyz="0 0 1" />
-		<dynamics damping="25.0" friction="10.0"/>
-		<calibration rising="0" falling="0"/>
-		<limit effort="46" lower="-1.5" upper="1.5" velocity="0.5"/>
-	</joint>
-	<link name="${name}_tof_tilt_link">
-		<inertial>
-			<origin xyz="0 0 0" rpy="0 0 0"/>
-			<mass value="1.0"/>
-			<inertia ixx="0.1" ixy="0.0" ixz="0.0" iyy="0.1" iyz="0.0" izz="0.1" />
-		</inertial>
-		<visual>
-			<origin xyz="0 0 0" rpy="0 0 0" />
-			<geometry>
-				<box size="0.1 0.1 0.01"/>
-			</geometry>
-			<material name="Red" />
-		</visual>
-		<collision>
-			<origin xyz="0 0 0" rpy="0 0 0" />
-			<geometry>
-				<box size="0.1 0.1 0.01"/>
-			</geometry>
-		</collision>
-	</link>
     <!--##################################################-->
-    <!-- camera test here -->
+    <!-- right camera -->
+    <xacro:cob_cameraone_v0 name="${name}_color_camera_r" parent="${name}_axis_link">
+      <origin xyz="${cam_r_x} ${cam_r_y} ${cam_r_z-0.06}" rpy="${cam_r_roll} ${cam_r_pitch+1.5708} ${cam_r_yaw+3.14159}" />
+    </xacro:cob_cameraone_v0>
+    <!-- right camera -->
     <xacro:cob_cameraone_v0 name="${name}_color_camera_l" parent="${name}_color_camera_r_link">
       <origin xyz="${cam_l_x-0.12} ${cam_l_y} ${cam_l_z}" rpy="${cam_l_roll} ${cam_l_pitch} ${cam_l_yaw}" />
     </xacro:cob_cameraone_v0>
-    <xacro:cob_cameraone_v0 name="${name}_color_camera_r" parent="${name}_axis_link">
-      <origin xyz="${cam_r_x} ${cam_r_y} ${cam_r_z-0.06}" rpy="${cam_r_roll} ${cam_r_pitch+1.5708} ${cam_r_yaw+3.14159}" />
-    </xacro:cob_cameraone_v0>
-    <!-- hokuyo_SR400_laser test here-->
-    <xacro:hokuyo_SR400_laser_v0 name="${name}_tof" parent="${name}_color_camera_r_link" ros_topic="head_scan" update_rate="54" min_angle="-0.302" max_angle="0.302" >
+    <!-- tof -->
+    <xacro:cob_tof_v0 name="${name}_tof" parent="${name}_color_camera_r_link">
       <origin xyz="${tof_x-0.06} ${tof_y} ${tof_z}" rpy="${tof_roll} ${tof_pitch} ${tof_yaw}" />
-    </xacro:hokuyo_SR400_laser_v0>
+    </xacro:cob_tof_v0>
     <!-- extensions -->
     <xacro:cob_head_gazebo_v0 name="${name}" />

Commit message: fixed camera topics for simulation

File: ros/urdf/head_v0/head.urdf.xacro (robot description, xacro)
@@ -41,9 +41,9 @@
 		</link>
 		<!-- right camera -->
-		<xacro:cob_cameraone_v0 name="${name}_color_camera_r" parent="${name}_axis_link">
+		<xacro:cob_cameraone_v0 name="${name}_color_camera_r" ros_topic="stereo/right" parent="${name}_axis_link">
 			<origin xyz="${cam_r_x} ${cam_r_y} ${cam_r_z-0.06}" rpy="${cam_r_roll} ${cam_r_pitch+1.5708} ${cam_r_yaw+3.14159}" />
 		</xacro:cob_cameraone_v0>
 		<!-- right camera -->
-		<xacro:cob_cameraone_v0 name="${name}_color_camera_l" parent="${name}_color_camera_r_link">
+		<xacro:cob_cameraone_v0 name="${name}_color_camera_l" ros_topic="stereo/left" parent="${name}_color_camera_r_link">
 			<origin xyz="${cam_l_x-0.12} ${cam_l_y} ${cam_l_z}" rpy="${cam_l_roll} ${cam_l_pitch} ${cam_l_yaw}" />
 		</xacro:cob_cameraone_v0>

File: ros/urdf/sensors/cameraone.gazebo.xacro (robot description, xacro)
@@ -4,5 +4,5 @@
       xmlns:interface="http://playerstage.sourceforge.net/gazebo/xmlschema/#interface"
       xmlns:xacro="http://ros.org/wiki/xacro">
-	<xacro:macro name="cob_cameraone_gazebo_v0" params="name">
+	<xacro:macro name="cob_cameraone_gazebo_v0" params="name ros_topic">
 		<gazebo reference="${name}_frame">
 			<sensor:camera name="${name}_sensor">
@@ -16,7 +16,7 @@
 					<alwaysOn>true</alwaysOn>
 					<updateRate>20.0</updateRate>
-					<topicName>${name}_image_data</topicName>
-					<imageTopicName>/${name}/image_raw</imageTopicName>
-					<cameraInfoTopicName>/${name}/camera_info</cameraInfoTopicName>
+					<topicName>${ros_topic}_image_data</topicName>
+					<imageTopicName>/${ros_topic}/image_raw</imageTopicName>
+					<cameraInfoTopicName>/${ros_topic}/camera_info</cameraInfoTopicName>
 					<pollServiceName>/${name}/request_image</pollServiceName>
 					<frameName>/${name}_link</frameName>

File: ros/urdf/sensors/cameraone.urdf.xacro (robot description, xacro)
@@ -6,5 +6,5 @@
        name="LaserBlock">
 	<include filename="$(find cob_description)/ros/urdf/sensors/cameraone.gazebo.xacro" />
-	<xacro:macro name="cob_cameraone_v0" params="name parent *origin">
+	<xacro:macro name="cob_cameraone_v0" params="name parent *origin ros_topic">
 		<joint name="${name}_joint" type="fixed">
 			<insert_block name="origin" />
@@ -57,5 +57,5 @@
 			</collision>
 		</link>
-	<xacro:cob_cameraone_gazebo_v0 name="${name}"/>
+	<xacro:cob_cameraone_gazebo_v0 name="${name}" ros_topic="${ros_topic}"/>
 	</xacro:macro>
 </robot>

Commit message: renamed cameraone to prosilica

File: ros/urdf/head_v0/head.urdf.xacro (robot description, xacro)
@@ -6,5 +6,5 @@
 	<include filename="$(find cob_description)/ros/urdf/head_v0/head.gazebo.xacro" />
 	<include filename="$(find cob_description)/ros/urdf/head_v0/head.transmission.xacro" />
-	<include filename="$(find cob_description)/ros/urdf/sensors/cameraone.urdf.xacro" />
+	<include filename="$(find cob_description)/ros/urdf/sensors/prosilica.urdf.xacro" />
 	<include filename="$(find cob_description)/ros/urdf/sensors/tof.urdf.xacro" />
 	<!--include filename="$(find cob_description)/ros/urdf/sensors/hokuyo_SR400_laser.urdf.xacro" /-->
@@ -41,11 +41,11 @@
 		</link>
 		<!-- right camera -->
-		<xacro:cob_cameraone_v0 name="${name}_color_camera_r" ros_topic="stereo/right" parent="${name}_axis_link">
+		<xacro:cob_prosilica_v0 name="${name}_color_camera_r" ros_topic="stereo/right" parent="${name}_axis_link">
 			<origin xyz="${cam_r_x} ${cam_r_y} ${cam_r_z-0.06}" rpy="${cam_r_roll} ${cam_r_pitch+1.5708} ${cam_r_yaw+3.14159}" />
-		</xacro:cob_cameraone_v0>
+		</xacro:cob_prosilica_v0>
 		<!-- right camera -->
-		<xacro:cob_cameraone_v0 name="${name}_color_camera_l" ros_topic="stereo/left" parent="${name}_color_camera_r_link">
+		<xacro:cob_prosilica_v0 name="${name}_color_camera_l" ros_topic="stereo/left" parent="${name}_color_camera_r_link">
 			<origin xyz="${cam_l_x-0.12} ${cam_l_y} ${cam_l_z}" rpy="${cam_l_roll} ${cam_l_pitch} ${cam_l_yaw}" />
-		</xacro:cob_cameraone_v0>
+		</xacro:cob_prosilica_v0>
 		<!-- tof -->
 		<xacro:cob_tof_v0 name="${name}_tof" parent="${name}_color_camera_r_link">

File: ros/urdf/sensors/prosilica.gazebo.xacro (robot description, xacro)
@@ -4,5 +4,5 @@
       xmlns:interface="http://playerstage.sourceforge.net/gazebo/xmlschema/#interface"
       xmlns:xacro="http://ros.org/wiki/xacro">
-	<xacro:macro name="cob_cameraone_gazebo_v0" params="name ros_topic">
+	<xacro:macro name="cob_prosilica_gazebo_v0" params="name ros_topic">
 		<gazebo reference="${name}_frame">
 			<sensor:camera name="${name}_sensor">

File: ros/urdf/sensors/prosilica.urdf.xacro (robot description, xacro)
@@ -5,6 +5,6 @@
        xmlns:xacro="http://playerstage.sourceforge.net/gazebo/xmlschema/#interface"
        name="LaserBlock">
-	<include filename="$(find cob_description)/ros/urdf/sensors/cameraone.gazebo.xacro" />
-	<xacro:macro name="cob_cameraone_v0" params="name parent *origin ros_topic">
+	<include filename="$(find cob_description)/ros/urdf/sensors/prosilica.gazebo.xacro" />
+	<xacro:macro name="cob_prosilica_v0" params="name parent *origin ros_topic">
 		<joint name="${name}_joint" type="fixed">
 			<insert_block name="origin" />
@@ -57,5 +57,5 @@
 			</collision>
 		</link>
-	<xacro:cob_cameraone_gazebo_v0 name="${name}" ros_topic="${ros_topic}"/>
+	<xacro:cob_prosilica_gazebo_v0 name="${name}" ros_topic="${ros_topic}"/>
 	</xacro:macro>
 </robot>
