Commit message: fix head_v3 simulation error

File: ros/urdf/head_v3/head.gazebo.xacro (robot description, xacro)
@@ -4,5 +4,5 @@
        xmlns:interface="http://playerstage.sourceforge.net/gazebo/xmlschema/#interface"
        xmlns:xacro="http://ros.org/wiki/xacro">
-	<xacro:macro name="cob_head_gazebo_v0" params="name">
+	<xacro:macro name="cob_head_gazebo_v3" params="name">
 		<gazebo reference="${name}_axis_link">
 			<material>Gazebo/Green</material>

File: ros/urdf/head_v3/head.transmission.xacro (robot description, xacro)
@@ -4,5 +4,5 @@
        xmlns:interface="http://playerstage.sourceforge.net/gazebo/xmlschema/#interface"
        xmlns:xacro="http://ros.org/wiki/xacro">
-	<xacro:macro name="cob_head_transmission_v0" params="name">
+	<xacro:macro name="cob_head_transmission_v3" params="name">
 		<transmission name="${name}_axis_trans" type="pr2_mechanism_model/SimpleTransmission">
 			<actuator name="${name}_axis_motor"/>
