Commit message: modifications for fetch and carry

File: ros/urdf/head_v3/head.urdf.xacro (robot description, xacro)
@@ -18,5 +18,5 @@
 			<dynamics damping="0.1" />
 			<calibration rising="${head_axis_ref}"/>
-			<limit effort="100" lower="-3.2" upper="0.1" velocity="0.5"/>
+			<limit effort="100" lower="-3.2" upper="0.1" velocity="1.4"/>
 		</joint>
 		<link name="${name}_axis_link">

Commit message: Kinect rgb configuration

File: ros/urdf/head_v3/head.urdf.xacro (robot description, xacro)
@@ -8,4 +8,5 @@
 	<include filename="$(find cob_description)/ros/urdf/sensors/prosilica.urdf.xacro" />
 	<include filename="$(find cob_description)/ros/urdf/sensors/kinect.urdf.xacro" />
+	<include filename="$(find cob_description)/ros/urdf/sensors/kinect.rgb.urdf.xacro" />
 	<!--include filename="$(find cob_description)/ros/urdf/sensors/hokuyo_SR400_laser.urdf.xacro" /-->
 	<xacro:macro name="cob_head_v3" params="name parent *origin">
@@ -52,4 +53,8 @@
 			<origin xyz="${cam3d_x+0.06} ${cam3d_y} ${cam3d_z}" rpy="${cam3d_roll} ${cam3d_pitch} ${cam3d_yaw}" />
 		</xacro:cob_kinect_v0>
+		<!-- cam3d -->
+                <xacro:cob_kinect_rgb_v0 name="${name}_cam3d_rgb" ros_topic="cam3d/rgb" parent="${name}_color_camera_l_link">
+                        <origin xyz="${cam3d_x-0.06} ${cam3d_y} ${cam3d_z}" rpy="${cam3d_roll} ${cam3d_pitch} ${cam3d_yaw+3.14}" />
+                </xacro:cob_kinect_rgb_v0>
 		<!-- extensions -->
 		<xacro:cob_head_gazebo_v3 name="${name}" />

File: ros/urdf/sensors/kinect.gazebo.xacro (robot description, xacro)
@@ -7,23 +7,30 @@
   <gazebo reference="${name}_frame">
     <sensor:ray name="${name}_sensor">
-          <rayCount>160</rayCount> <!--true value 640-->
-          <rangeCount>160</rangeCount>
+          <rayCount>210</rayCount> <!--old value 160-->
+          <rangeCount>210</rangeCount>
           <laserCount>1</laserCount>
           <origin>0.0 0.0 0.05</origin>
           <displayRays>false</displayRays>
-          <minAngle>-31.63</minAngle>
-          <maxAngle>31.63</maxAngle>
-          <minRange>1.00</minRange> <!--0.8m min calibrated range-->
-          <maxRange>5.0</maxRange> <!--5.0m max calibrated range-->
-          <resRange>0.010</resRange>
-          <updateRate>10</updateRate> <!-- true value 30Hz -->
-          <verticalRayCount>120</verticalRayCount> <!--true value 480 -->
-          <verticalRangeCount>120</verticalRangeCount>
-          <verticalMinAngle>-25.74</verticalMinAngle>
-          <verticalMaxAngle>25.74</verticalMaxAngle>
+          <minAngle>-28.50</minAngle>
+	  <!--minAngle>-31.63</minAngle-->
+          <maxAngle>28.50</maxAngle>
+	  <!--maxAngle>31.63</maxAngle-->
+          <!--minRange>1.00</minRange--> <!--0.8m min calibrated range-->
+          <minRange>1</minRange>  <!--original value 1.2-->
+	  <!--maxRange>5.0</maxRange--> <!--5.0m max calibrated range-->
+          <maxRange>10</maxRange><!--real value 3.5-->
+	  <resRange>0.010</resRange>
+          <updateRate>30</updateRate> <!-- old value 10Hz -->
+          <verticalRayCount>220</verticalRayCount> <!--old value 120 -->
+          <verticalRangeCount>220</verticalRangeCount>
+          <verticalMinAngle>-21.50</verticalMinAngle>
+	  <!--verticalMinAngle>-25.74</verticalMinAngle-->
+          <verticalMaxAngle>21.50</verticalMaxAngle>
+	  <!--verticalMaxAngle>25.74</verticalMaxAngle-->
           <controller:gazebo_ros_block_laser name="kinect_controller" plugin="libgazebo_ros_block_laser.so">
-            <gaussianNoise>0.005</gaussianNoise>
+            <focal_length>580</focal_length>
+	    <gaussianNoise>0.005</gaussianNoise>
             <alwaysOn>true</alwaysOn>
-            <updateRate>10</updateRate> <!-- true value 30Hz -->
+            <updateRate>30</updateRate> <!-- old value 10Hz -->
             <topicName>${ros_topic}</topicName>
             <frameName>/${name}_frame</frameName>

Commit message: fixed origin offset

File: ros/urdf/head_v3/head.urdf.xacro (robot description, xacro)
@@ -79,7 +79,7 @@
 		</xacro:cob_kinect_v0>
 		<!-- cam3d -->
-                <xacro:cob_kinect_rgb_v0 name="${name}_cam3d_rgb" ros_topic="cam3d/rgb" parent="${name}_color_camera_l_link">
-                        <origin xyz="${cam3d_x-0.06} ${cam3d_y} ${cam3d_z}" rpy="${cam3d_roll} ${cam3d_pitch} ${cam3d_yaw+3.14}" />
-                </xacro:cob_kinect_rgb_v0>
+    <xacro:cob_kinect_rgb_v0 name="${name}_cam3d_rgb" ros_topic="cam3d/rgb" parent="${name}_color_camera_l_link">
+    	<origin xyz="${cam3d_x+0.06} ${cam3d_y} ${cam3d_z}" rpy="${cam3d_roll} ${cam3d_pitch} ${cam3d_yaw}" />
+    </xacro:cob_kinect_rgb_v0>
 		<!-- extensions -->
 		<xacro:cob_head_gazebo_v3 name="${name}" />

Commit message: using now kinect plugin from pr2_gazebo

File: ros/urdf/head_v3/head.urdf.xacro (robot description, xacro)
@@ -8,5 +8,4 @@
 	<include filename="$(find cob_description)/ros/urdf/sensors/prosilica.urdf.xacro" />
 	<include filename="$(find cob_description)/ros/urdf/sensors/kinect.urdf.xacro" />
-	<include filename="$(find cob_description)/ros/urdf/sensors/kinect.rgb.urdf.xacro" />
 	<!--include filename="$(find cob_description)/ros/urdf/sensors/hokuyo_SR400_laser.urdf.xacro" /-->
 	<xacro:macro name="cob_head_v3" params="name parent *origin">
@@ -75,11 +74,7 @@
 		</xacro:cob_prosilica_v0>
 		<!-- cam3d -->
-		<xacro:cob_kinect_v0 name="${name}_cam3d" ros_topic="cam3d/depth/points1" parent="${name}_color_camera_l_link">
+		<xacro:cob_kinect_v0 name="${name}_cam3d" ros_topic="cam3d" parent="${name}_color_camera_l_link">
 			<origin xyz="${cam3d_x+0.06} ${cam3d_y} ${cam3d_z}" rpy="${cam3d_roll} ${cam3d_pitch} ${cam3d_yaw}" />
 		</xacro:cob_kinect_v0>
-		<!-- cam3d -->
-    <xacro:cob_kinect_rgb_v0 name="${name}_cam3d_rgb" ros_topic="cam3d/rgb" parent="${name}_color_camera_l_link">
-    	<origin xyz="${cam3d_x+0.06} ${cam3d_y} ${cam3d_z}" rpy="${cam3d_roll} ${cam3d_pitch} ${cam3d_yaw}" />
-    </xacro:cob_kinect_rgb_v0>
 		<!-- extensions -->
 		<xacro:cob_head_gazebo_v3 name="${name}" />

File: ros/urdf/sensors/kinect.gazebo.xacro (robot description, xacro)
@@ -6,38 +6,27 @@
 <xacro:macro name="cob_kinect_gazebo_v0" params="name ros_topic">
   <gazebo reference="${name}_frame">
-    <sensor:ray name="${name}_sensor">
-          <rayCount>210</rayCount> <!--old value 160-->
-          <rangeCount>210</rangeCount>
-          <laserCount>1</laserCount>
-          <origin>0.0 0.0 0.05</origin>
-          <displayRays>false</displayRays>
-          <minAngle>-28.50</minAngle>
-	  <!--minAngle>-31.63</minAngle-->
-          <maxAngle>28.50</maxAngle>
-	  <!--maxAngle>31.63</maxAngle-->
-          <!--minRange>1.00</minRange--> <!--0.8m min calibrated range-->
-          <minRange>1</minRange>  <!--original value 1.2-->
-	  <!--maxRange>5.0</maxRange--> <!--5.0m max calibrated range-->
-          <maxRange>10</maxRange><!--real value 3.5-->
-	  <resRange>0.010</resRange>
-          <updateRate>30</updateRate> <!-- old value 10Hz -->
-          <verticalRayCount>220</verticalRayCount> <!--old value 120 -->
-          <verticalRangeCount>220</verticalRangeCount>
-          <verticalMinAngle>-21.50</verticalMinAngle>
-	  <!--verticalMinAngle>-25.74</verticalMinAngle-->
-          <verticalMaxAngle>21.50</verticalMaxAngle>
-	  <!--verticalMaxAngle>25.74</verticalMaxAngle-->
-          <controller:gazebo_ros_block_laser name="kinect_controller" plugin="libgazebo_ros_block_laser.so">
-            <focal_length>580</focal_length>
-	    <gaussianNoise>0.005</gaussianNoise>
-            <alwaysOn>true</alwaysOn>
-            <updateRate>30</updateRate> <!-- old value 10Hz -->
-            <topicName>${ros_topic}</topicName>
-            <frameName>/${name}_frame</frameName>
-            <interface:laser name="${name}_ray_block_iface" />
-          </controller:gazebo_ros_block_laser>
-        </sensor:ray>
-    <material value="Gazebo/Red" />
-    <turnGravityOff>true</turnGravityOff>
+    <sensor:camera name="${name}_frame_sensor">
+      <imageFormat>R8G8B8</imageFormat>
+      <imageSize>640 480</imageSize>
+      <hfov>57</hfov>
+      <nearClip>0.01</nearClip>
+      <farClip>5</farClip>
+      <updateRate>20.0</updateRate>
+      <baseline>0.2</baseline>
+      <controller:gazebo_ros_camera name="${name}_frame_controller" plugin="libgazebo_ros_camera.so">
+        <alwaysOn>true</alwaysOn>
+        <updateRate>20.0</updateRate>
+        <imageTopicName>${ros_topic}/rgb/image_raw</imageTopicName>
+        <pointCloudTopicName>${ros_topic}/depth/points</pointCloudTopicName>
+        <cameraInfoTopicName>${ros_topic}/camera_info</cameraInfoTopicName>
+        <frameName>/${name}_link</frameName>
+        <pointCloudCutoff>0.5</pointCloudCutoff>
+        <distortion_k1>0.00000001</distortion_k1>
+        <distortion_k2>0.00000001</distortion_k2>
+        <distortion_k3>0.00000001</distortion_k3>
+        <distortion_t1>0.00000001</distortion_t1>
+        <distortion_t2>0.00000001</distortion_t2>
+      </controller:gazebo_ros_camera>
+    </sensor:camera>
   </gazebo>
 </xacro:macro>

File: ros/urdf/sensors/kinect.urdf.xacro (robot description, xacro)
@@ -1,8 +1,7 @@
 <?xml version="1.0"?>
-<robot xmlns:sensor="http://playerstage.sourceforge.net/gazebo/xmlschema/#sensor"
-       xmlns:controller="http://playerstage.sourceforge.net/gazebo/xmlschema/#controller"
-       xmlns:interface="http://playerstage.sourceforge.net/gazebo/xmlschema/#interface"
-       xmlns:xacro="http://playerstage.sourceforge.net/gazebo/xmlschema/#interface"
-       name="LaserBlock">
+<root xmlns:sensor="http://playerstage.sourceforge.net/gazebo/xmlschema/#sensor"
+      xmlns:controller="http://playerstage.sourceforge.net/gazebo/xmlschema/#controller"
+      xmlns:interface="http://playerstage.sourceforge.net/gazebo/xmlschema/#interface"
+      xmlns:xacro="http://ros.org/wiki/xacro">
   <include filename="$(find cob_description)/ros/urdf/sensors/kinect.gazebo.xacro" />
   <xacro:macro name="cob_kinect_v0" params="name parent *origin ros_topic">
@@ -57,6 +56,6 @@
       </collision >
     </link>
-   <!-- for simulation -->
-   <xacro:cob_kinect_gazebo_v0 name="${name}" ros_topic="${ros_topic}"/>
+    <!-- extensions -->
+    <xacro:cob_kinect_gazebo_v0 name="${name}" ros_topic="${ros_topic}" />
   </xacro:macro>
-</robot>
+</root>

Commit message: removed calib_joint

File: ros/urdf/head_v3/head.urdf.xacro (robot description, xacro)
@@ -29,5 +29,5 @@
 				<origin xyz="0 0 0" rpy="0 0 0" />
 				<geometry>
-					<box size="0.01 0.01 0.12"/>
+					<box size="0.01 0.01 0.01"/>
 				</geometry>
 				<material name="Green" />
@@ -36,36 +36,11 @@
 				<origin xyz="0 0 0" rpy="0 0 0" />
 				<geometry>
-					<box size="0.01 0.01 0.12"/>
-				</geometry>
-			</collision>
-		</link>
-		<joint name="${name}_calib_joint" type="fixed">
-			<origin xyz="0 0 -0.06" rpy="0 -1.5708 0" />
-			<parent link="${name}_axis_link"/>
-			<child link="${name}_calib_link"/>
-		</joint>
-		<link name="${name}_calib_link">
-			<inertial>
-				<origin xyz="0 0 0" rpy="0 0 0"/>
-				<mass value="0.1"/>
-				<inertia ixx="0.0001" ixy="0" ixz="0" iyy="0.0001" iyz="0" izz="0.0001" />
-			</inertial>
-			<visual>
-				<origin xyz="0 0 0" rpy="0 0 0" />
-				<geometry>
-					<box size="0.01 0.01 0.12"/>
-				</geometry>
-				<material name="Green" />
-			</visual>
-			<collision>
-				<origin xyz="0 0 0" rpy="0 0 0" />
-				<geometry>
-					<box size="0.01 0.01 0.12"/>
+					<box size="0.01 0.01 0.01"/>
 				</geometry>
 			</collision>
 		</link>
 		<!-- left camera -->
-		<xacro:cob_prosilica_v0 name="${name}_color_camera_l" ros_topic="stereo/left" parent="${name}_calib_link">
-			<origin xyz="${cam_l_x} ${cam_l_y} ${cam_l_z}" rpy="${cam_l_roll} ${cam_l_pitch} ${cam_l_yaw}" />
+		<xacro:cob_prosilica_v0 name="${name}_color_camera_l" ros_topic="stereo/left" parent="${name}_axis_link">
+			<origin xyz="${cam_l_x} ${cam_l_y} ${cam_l_z}-0.06" rpy="${cam_l_roll} ${cam_l_pitch}-1.5708 ${cam_l_yaw}" />
 		</xacro:cob_prosilica_v0>
 		<!-- right camera -->
