Commit message: beautify sdh transmissions

File: ros/urdf/sdh_v0/sdh.transmission.xacro (robot description, xacro)
@@ -6,10 +6,5 @@
 	<xacro:macro name="cob_sdh_transmission_v0" params="name">
 		<transmission name="${name}_knuckle_trans" type="pr2_mechanism_model/SimpleTransmission">
-		    	<actuator name="${name}_knuckle_motor"/>
-			<joint name="${name}_finger_21_joint"/>
-			<mechanicalReduction>1</mechanicalReduction>
-		</transmission>
-	        <transmission name="${name}_knuckle_trans" type="pr2_mechanism_model/SimpleTransmission">
-		    	<actuator name="${name}_knuckle_motor"/>
+			<actuator name="${name}_knuckle_motor"/>
 			<joint name="${name}_knuckle_joint"/>
 			<mechanicalReduction>1</mechanicalReduction>
