Commit message: inserted cob base mesh file

File: ros/urdf/base_v1/base.urdf.xacro (robot description, xacro)
@@ -128,20 +128,21 @@
       <inertial>
         <mass value="${base_mass}" />
-        <origin xyz="${base_cg_x} ${base_cg_y} ${base_cg_z}" />
+        <origin xyz="0 0 0" />
         <inertia ixx="5.652232699207" ixy="-0.009719934438" ixz="1.293988226423"
                  iyy="5.669473158652" iyz="-0.007379583694" izz="3.683196351726" />
       </inertial>
       <visual>
-        <origin xyz="0 0 0.15" rpy="0 0 0" />
-        <geometry>
-          <!--mesh filename="package://cob_defs/common/files/meshes/platform.stl"/-->  <!--modified by jie-->
-          <box size="${base_size_x} ${base_size_y} ${base_collision_size_z}" />
+        <origin xyz="0 0 0" rpy="0 0 0" />
+        <geometry>
+          <mesh filename="package://cob_defs/common/files/meshes/platform.stl"/>
+          <!--box size="${base_size_x} ${base_size_y} ${base_collision_size_z}" /-->
         </geometry>
         <material name="Grey"/>
       </visual>
       <collision>
-        <origin xyz="0 0 ${base_size_z-base_collision_size_z/2}" rpy="0 0 0" />
-        <geometry>
-          <box size="${base_size_x} ${base_size_y} ${base_collision_size_z}" />
+        <origin xyz="0 0 0" rpy="0 0 0" />
+        <geometry>
+	      <mesh filename="package://cob_defs/common/files/meshes/platform.stl"/>
+          <!--box size="${base_size_x} ${base_size_y} ${base_collision_size_z}" /-->
         </geometry>
       </collision>

Commit message: fixed laser sensor names, version number and visual model

File: ros/urdf/base_v1/base.urdf.xacro (robot description, xacro)
@@ -7,4 +7,5 @@
   <include filename="$(find cob_description)/ros/urdf/base_v0/base.transmission.xacro" />
   <!-- modify here for test -->
+  <include filename="$(find cob_description)/ros/urdf/sensors/sick_s300_laser.urdf.xacro"/>
   <include filename="$(find cob_description)/ros/urdf/sensors/hokuyo_lx30_laser.urdf.xacro"/>
   <!-- DATA SOURCES -->
@@ -95,8 +96,10 @@
       </inertial>
       <visual>
-        <origin xyz="0 0 0.085" rpy="0 0 0" />  <!--modified by jie-->
+        <!--origin xyz="0 0 0.085" rpy="0 0 0" /-->  <!--modified by jie-->
+		<origin xyz="0 0 0.002" rpy="0.0 0.0 0.0" />
         <geometry>
           <!--mesh filename="package://cob_description/ros/meshes/base_v0/caster.stl" /-->  <!--modified by jie-->
-          <box size="0.192 0.164 0.013" />
+          <!--box size="0.192 0.164 0.013" /-->
+		  <box size="0.001 0.001 0.001" />
         </geometry>
         <material name="Green" />
@@ -124,5 +127,5 @@
   </xacro:macro>
   <!-- The xacro macro xacro:cob_base contains: base, casters and wheels -->
-  <xacro:macro name="cob_base_v0" params="name">
+  <xacro:macro name="cob_base_v1" params="name">
   <link name="${name}_link">
       <inertial>
@@ -143,4 +146,5 @@
         <origin xyz="0 0 0" rpy="0 0 0" />
         <geometry>
+		  <!--box size="0.001 0.001 0.001" /-->
 	      <mesh filename="package://cob_description/ros/meshes/base_v0/base_collision.stl"/>
           <!--box size="${base_size_x} ${base_size_y} ${base_collision_size_z}" /-->
@@ -180,14 +184,14 @@
     <!--modify here for test: front,base and top lasers -->
     <!-- base laser front -->
-    <xacro:hokuyo_lx30_laser_v0 name="${name}_laser_front" parent="${name}" ros_topic="scan_front" update_rate="20" min_angle="-1.35" max_angle="1.35" >
+    <xacro:sick_s300_laser_v0 name="${name}_laser_front" parent="${name}" ros_topic="scan_front_raw" update_rate="10" min_angle="-2.3562" max_angle="2.3562" >
       <origin xyz="${base_laser_x} ${base_laser_y} ${base_laser_z}" rpy="0 0 0" />
-    </xacro:hokuyo_lx30_laser_v0>
+    </xacro:sick_s300_laser_v0>
     <!-- base laser rear -->
-    <xacro:hokuyo_lx30_laser_v0 name="${name}_laser_rear" parent="${name}" ros_topic="scan_rear" update_rate="20" min_angle="-1.35" max_angle="1.35" >
+    <xacro:sick_s300_laser_v0 name="${name}_laser_rear" parent="${name}" ros_topic="scan_rear_raw" update_rate="10" min_angle="-2.3562" max_angle="2.3562" >
       <origin xyz="${-base_laser_x} ${base_laser_y} ${base_laser_z}" rpy="0 0 ${M_PI}" />
-    </xacro:hokuyo_lx30_laser_v0>
+    </xacro:sick_s300_laser_v0>
     <!-- base laser top -->
-    <xacro:hokuyo_lx30_laser_v0 name="${name}_laser_top" parent="${name}" ros_topic="scan_top" update_rate="10" min_angle="-2.094" max_angle="2.094" >
-      <origin xyz="-0.252 0 0.42" rpy="0 0 ${M_PI}" />
+    <xacro:hokuyo_lx30_laser_v0 name="${name}_laser_top" parent="${name}" ros_topic="scan_top" update_rate="10" min_angle="-2.3562" max_angle="2.3562" >
+      <origin xyz="-0.252 0 0.42" rpy="0 0 0" />
     </xacro:hokuyo_lx30_laser_v0>
     <!-- all four caster macros -->

Commit message: temporary fix for urdf collision model

File: ros/urdf/base_v1/base.urdf.xacro (robot description, xacro)
@@ -28,5 +28,5 @@
   <property name="base_size_y" value="0.6" />
   <property name="base_size_z" value="0.23" />
-  <property name="base_collision_size_z" value="0.04" />
+  <property name="base_collision_size_z" value="0.4" />
   <!-- simplified box collision geometry for hokuyo laser -->
   <property name="base_laser_x" value="0.325" />
@@ -148,5 +148,31 @@
 		  <!--box size="0.001 0.001 0.001" /-->
 	      <mesh filename="package://cob_description/ros/meshes/base_v0/base_collision.stlb"/>
-          <!--box size="${base_size_x} ${base_size_y} ${base_collision_size_z}" /-->
+        </geometry>
+      </collision>
+    </link>
+<!-- FIXME remove this -->
+    <joint name="${name}_link2_joint" type="fixed">
+      <origin xyz="0 0 0" rpy="0 0 0" />
+      <child link="${name}_link2" />
+      <parent link="${name}_footprint"/>
+    </joint>
+  <link name="${name}_link2">
+      <inertial>
+        <mass value="${base_mass}" />
+        <origin xyz="0 0 0" />
+        <inertia ixx="5.652232699207" ixy="-0.009719934438" ixz="1.293988226423"
+                 iyy="5.669473158652" iyz="-0.007379583694" izz="3.683196351726" />
+      </inertial>
+      <visual>
+        <origin xyz="0 0 0" rpy="0 0 0" />
+        <geometry>
+          <box size="0.01 0.01 0.01" />
+        </geometry>
+        <material name="Grey"/>
+      </visual>
+      <collision>
+        <origin xyz="0 0 0.2" rpy="0 0 0" />
+        <geometry>
+          <box size="0.8 0.6 0.4" />
         </geometry>
       </collision>

File: ros/urdf/sdh_v0/sdh.urdf.xacro (robot description, xacro)
@@ -160,5 +160,5 @@
 			</visual>
 			<collision>
-				<origin xyz="0 0 0" rpy="1.57079633 0 0" />
+				<origin xyz="0 0 0" rpy="0 0 0" />
 				<geometry>
 					<mesh filename="package://cob_description/ros/meshes/sdh_v0/knuckle.stlb"/>

File: ros/urdf/torso_v1/torso.urdf.xacro (robot description, xacro)
@@ -9,5 +9,5 @@
 		<!-- joint between base_link and torso_tray_link -->
 		<joint name="${name}_tray_joint" type="revolute">
-			<origin xyz="0.2406 0.1900 0.7320" rpy="2.3561 0 0" />
+			<origin xyz="0.2406 0.1900 0.7920" rpy="2.3561 0 0" />
 			<parent link="${parent}"/>
 			<child link="${name}_tray_link"/>
@@ -34,4 +34,30 @@
 				<geometry>
 					<mesh filename="package://cob_description/ros/meshes/torso_v0/tray_collision.stlb" />
+				</geometry>
+			</collision>
+		</link>
+		<!-- FIXME additional tray colission box, should be removed -->
+		<joint name="${name}_tray_joint2" type="fixed">
+			<origin xyz="0.25 0.25 0.1" rpy="0.78 0 0" />
+			<parent link="${name}_tray_link"/>
+			<child link="${name}_tray_link2"/>
+		</joint>
+		<link name="${name}_tray_link2">
+			<inertial>
+				<origin xyz="0 0 0" rpy="0 0 0"/>
+				<mass value="0.1"/>
+				<inertia ixx="0.01" ixy="0" ixz="0" iyy="0.01" iyz="0" izz="0.01" />
+			</inertial>
+			<visual>
+				<origin xyz="0 0 0" rpy="0 0 0" />
+				<geometry>
+					<box size="0.01 0.01 0.01"/>
+				</geometry>
+				<material name="Green" />
+			</visual>
+			<collision>
+				<origin xyz="0 0 0" rpy="0 0 0" />
+				<geometry>
+					<box size="0.3 0.4 0.1"/>
 				</geometry>
 			</collision>
@@ -121,5 +147,5 @@
 			</visual>
 			<collision>
-				<origin xyz="0 0 0" rpy="1.5708 0 0" />
+				<origin xyz="0 0 0" rpy="3.1415926 0 0" />
 				<geometry>
 					<mesh filename="package://cob_description/ros/meshes/torso_v0/upper_neck_collision.stlb" />
