Commit message: revert urdf changes because of arm planning collisions

File: ros/urdf/arm_v1/arm.urdf.xacro (robot description, xacro)
@@ -225,5 +225,5 @@
 		<!-- joint between arm_6_link and arm_7_link -->
 		<joint name="${name}_7_joint" type="revolute">
-			<origin xyz="0 -0.197448 0" rpy="-1.5708 0 0" />
+			<origin xyz="0 -0.237448 0" rpy="-1.5708 0 0" />
 			<parent link="${name}_6_link"/>
 			<child link="${name}_7_link"/>

File: ros/urdf/base_v1/base.urdf.xacro (robot description, xacro)
@@ -28,5 +28,5 @@
   <property name="base_size_y" value="0.6" />
   <property name="base_size_z" value="0.23" />
-  <property name="base_collision_size_z" value="0.4" />
+  <property name="base_collision_size_z" value="0.04" />
   <!-- simplified box collision geometry for hokuyo laser -->
   <property name="base_laser_x" value="0.325" />
@@ -148,31 +148,5 @@
 		  <!--box size="0.001 0.001 0.001" /-->
 	      <mesh filename="package://cob_description/ros/meshes/base_v0/base_collision.stlb"/>
-        </geometry>
-      </collision>
-    </link>
-<!-- FIXME remove this -->
-    <joint name="${name}_link2_joint" type="fixed">
-      <origin xyz="0 0 0" rpy="0 0 0" />
-      <child link="${name}_link2" />
-      <parent link="${name}_footprint"/>
-    </joint>
-  <link name="${name}_link2">
-      <inertial>
-        <mass value="${base_mass}" />
-        <origin xyz="0 0 0" />
-        <inertia ixx="5.652232699207" ixy="-0.009719934438" ixz="1.293988226423"
-                 iyy="5.669473158652" iyz="-0.007379583694" izz="3.683196351726" />
-      </inertial>
-      <visual>
-        <origin xyz="0 0 0" rpy="0 0 0" />
-        <geometry>
-          <box size="0.01 0.01 0.01" />
-        </geometry>
-        <material name="Grey"/>
-      </visual>
-      <collision>
-        <origin xyz="0 0 0.2" rpy="0 0 0" />
-        <geometry>
-          <box size="0.8 0.6 0.4" />
+          <!--box size="${base_size_x} ${base_size_y} ${base_collision_size_z}" /-->
         </geometry>
       </collision>

File: ros/urdf/sdh_v0/sdh.transmission.xacro (robot description, xacro)
@@ -5,4 +5,9 @@
        xmlns:xacro="http://ros.org/wiki/xacro">
 	<xacro:macro name="cob_sdh_transmission_v0" params="name">
+		<transmission name="${name}_knuckle_trans" type="pr2_mechanism_model/SimpleTransmission">
+		<actuator name="${name}_knuckle_motor"/>
+			<joint name="${name}_finger_21_joint"/>
+			<mechanicalReduction>1</mechanicalReduction>
+		</transmission>
 		<transmission name="${name}_knuckle_trans" type="pr2_mechanism_model/SimpleTransmission">
 			<actuator name="${name}_knuckle_motor"/>

File: ros/urdf/torso_v1/torso.urdf.xacro (robot description, xacro)
@@ -9,5 +9,5 @@
 		<!-- joint between base_link and torso_tray_link -->
 		<joint name="${name}_tray_joint" type="revolute">
-			<origin xyz="0.2406 0.1900 0.7920" rpy="2.3561 0 0" />
+			<origin xyz="0.2406 0.1900 0.7320" rpy="2.3561 0 0" />
 			<parent link="${parent}"/>
 			<child link="${name}_tray_link"/>
@@ -34,30 +34,4 @@
 				<geometry>
 					<mesh filename="package://cob_description/ros/meshes/torso_v0/tray_collision.stlb" />
-				</geometry>
-			</collision>
-		</link>
-		<!-- FIXME additional tray colission box, should be removed -->
-		<joint name="${name}_tray_joint2" type="fixed">
-			<origin xyz="0.25 0.25 0.1" rpy="0.78 0 0" />
-			<parent link="${name}_tray_link"/>
-			<child link="${name}_tray_link2"/>
-		</joint>
-		<link name="${name}_tray_link2">
-			<inertial>
-				<origin xyz="0 0 0" rpy="0 0 0"/>
-				<mass value="0.1"/>
-				<inertia ixx="0.01" ixy="0" ixz="0" iyy="0.01" iyz="0" izz="0.01" />
-			</inertial>
-			<visual>
-				<origin xyz="0 0 0" rpy="0 0 0" />
-				<geometry>
-					<box size="0.01 0.01 0.01"/>
-				</geometry>
-				<material name="Green" />
-			</visual>
-			<collision>
-				<origin xyz="0 0 0" rpy="0 0 0" />
-				<geometry>
-					<box size="0.3 0.4 0.1"/>
 				</geometry>
 			</collision>
