Commit message: rename from arm to lwa

File: schunk_description/ros/robots/lwa_sdh.urdf.xacro (robot description, xacro)
@@ -4,44 +4,47 @@
        xmlns:interface="http://playerstage.sourceforge.net/gazebo/xmlschema/#interface"
        xmlns:xacro="http://playerstage.sourceforge.net/gazebo/xmlschema/#interface"
-       name="lbr" >
+       name="arm_sdh" >
   <!-- The following included files set up definitions of parts of the robot body -->
   <!-- misc common stuff? -->
   <include filename="$(find cob_description)/ros/urdf/common.xacro" />
-  <include filename="$(find cob_description)/ros/calibration/$(env ROBOT).urdf.xacro" />
-  <!-- cob lbr-->
-  <include filename="$(find cob_description)/ros/urdf/lbr_v0/lbr.urdf.xacro" />
+  <include filename="$(find schunk_description)/ros/calibration/lwa.urdf.xacro" />
+  <!-- cob arm-->
+  <include filename="$(find schunk_description)/ros/urdf/lwa_v0/lwa.urdf.xacro" />
   <!-- cob sdh-->
-  <include filename="$(find cob_description)/ros/urdf/sdh_v0/sdh.urdf.xacro" />
+  <include filename="$(find schunk_description)/ros/urdf/sdh_v0/sdh.urdf.xacro" />
   <!-- generic simulator_gazebo plugins for starting mechanism control, ros time, ros battery -->
   <include filename="$(find cob_description)/ros/gazebo/gazebo.urdf.xacro" />
   <!-- materials for visualization -->
   <include filename="$(find cob_description)/ros/urdf/materials.urdf.xacro" />
-  <!-- foot for lbr-->
-	<link name="base_link">
+  <!-- foot for arm-->
+	<link name="dummy_link">
 		<inertial>
 		   <origin xyz="0 0 -10" rpy="0 0 0"/>
-		   <mass value="100.0"/>
-		   <inertia ixx="10.0"  ixy="0"  ixz="0" iyy="100.0" iyz="0" izz="100.0" />
+		   <mass value="1000.0"/>
+		   <inertia ixx="100.0"  ixy="0"  ixz="0" iyy="100.0" iyz="0" izz="100.0" />
 		</inertial>
 		<visual>
 		   <origin xyz="0 0 0.25" rpy="0 0 0" />
 		   <geometry>
-			  <cylinder radius="0.075" length="0.5"/>
+		   	  <box size="0.6 0.4 0.4"/>
+			  <!--cylinder radius="0.1" length="0.5"/-->
 		   </geometry>
-		   <material name="Grey" />
+		   <material name="Blue" />
 		</visual>
 		<collision>
 		   <origin xyz="0 0 0.25" rpy="0 0 0" />
 		   <geometry>
-			  <cylinder radius="0.075" length="0.5"/>
+		   	  <box size="0.6 0.4 0.4"/>
+			  <!--cylinder radius="0.1" length="0.5"/-->
 		   </geometry>
 		</collision>
 	</link>
-  <!-- cob lbr-->
-  <xacro:cob_lbr_v0 name="arm" parent="base_link">
-    <origin xyz="0 0 0.5" rpy="0 0 0" />
-  </xacro:cob_lbr_v0>
-  <xacro:cob_sdh_v0 name="sdh" parent="arm_7_link">
-    <origin xyz="0 0 0.02" rpy="0 0 0" />
-  </xacro:cob_sdh_v0>
+  <!-- arm -->
+  <xacro:schunk_lwa_v0 name="lwa" parent="dummy_link">
+    <origin xyz="0 0 0.5" rpy="3.1415926 0 0" />
+  </xacro:schunk_lwa_v0>
+  <!-- sdh -->
+  <xacro:schunk_sdh_v0 name="sdh" parent="arm_7_link">
+    <origin xyz="0 0 0" rpy="0 3.1415926 0" />
+  </xacro:schunk_sdh_v0>
 </robot>
