Commit message: changed stl files not using solid

File: schunk_description/urdf/lwa_extended/lwa_extended.urdf.xacro (robot description, xacro)
@@ -61,5 +61,5 @@
 				<origin xyz="0 0 0" rpy="0 0 0" />
 				<geometry>
-					<mesh filename="package://schunk_description/meshes/lwa/lwa1.stlb" />
+					<mesh filename="package://schunk_description/meshes/lwa/lwa1.stl" />
 				</geometry>
 			</collision>
@@ -93,5 +93,5 @@
 				<origin xyz="0 0 0" rpy="0 0 0" />
 				<geometry>
-					<mesh filename="package://schunk_description/meshes/lwa/lwa2.stlb"/>
+					<mesh filename="package://schunk_description/meshes/lwa/lwa2.stl"/>
 				</geometry>
 			</collision>
@@ -125,5 +125,5 @@
 				<origin xyz="0 0 0" rpy="0 0 0" />
 				<geometry>
-					<mesh filename="package://schunk_description/meshes/lwa/lwa3.stlb"/>
+					<mesh filename="package://schunk_description/meshes/lwa/lwa3.stl"/>
 				</geometry>
 			</collision>
@@ -157,5 +157,5 @@
 				<origin xyz="0 0 0" rpy="0 0 0" />
 				<geometry>
-					<mesh filename="package://schunk_description/meshes/lwa/lwa4.stlb"/>
+					<mesh filename="package://schunk_description/meshes/lwa/lwa4.stl"/>
 				</geometry>
 			</collision>
@@ -188,5 +188,5 @@
 				<origin xyz="0 0 0" rpy="0 0 0" />
 				<geometry>
-					<mesh filename="package://schunk_description/meshes/lwa/lwa5.stlb"/>
+					<mesh filename="package://schunk_description/meshes/lwa/lwa5.stl"/>
 				</geometry>
 			</collision>
@@ -219,5 +219,5 @@
 				<origin xyz="0 0 0" rpy="0 0 0" />
 				<geometry>
-					<mesh filename="package://schunk_description/meshes/lwa/lwa6.stlb"/>
+					<mesh filename="package://schunk_description/meshes/lwa/lwa6.stl"/>
 				</geometry>
 			</collision>
@@ -250,5 +250,5 @@
 				<origin xyz="0 0 0" rpy="0 0 0" />
 				<geometry>
-					<mesh filename="package://schunk_description/meshes/lwa/lwa7.stlb"/>
+					<mesh filename="package://schunk_description/meshes/lwa/lwa7.stl"/>
 				</geometry>
 			</collision>

File: schunk_description/urdf/powerball/powerball.urdf.xacro (robot description, xacro)
@@ -29,5 +29,5 @@
 				<origin xyz="0 0 0" rpy="0 0 0" />
 				<geometry>
-					<mesh filename="package://schunk_description/meshes/powerball/powerball0.stlb" />
+					<mesh filename="package://schunk_description/meshes/powerball/powerball0.stl" />
 				</geometry>
 			</collision>
@@ -60,5 +60,5 @@
 				<origin xyz="0 0 0" rpy="0 0 0" />
 				<geometry>
-					<mesh filename="package://schunk_description/meshes/powerball/powerball1.stlb" />
+					<mesh filename="package://schunk_description/meshes/powerball/powerball1.stl" />
 				</geometry>
 			</collision>
@@ -91,5 +91,5 @@
 				<origin xyz="0 0 0" rpy="0 0 0" />
 				<geometry>
-					<mesh filename="package://schunk_description/meshes/powerball/powerball2.stlb"/>
+					<mesh filename="package://schunk_description/meshes/powerball/powerball2.stl"/>
 				</geometry>
 			</collision>
@@ -122,5 +122,5 @@
 				<origin xyz="0 0 0" rpy="0 0 0" />
 				<geometry>
-					<mesh filename="package://schunk_description/meshes/powerball/powerball3.stlb"/>
+					<mesh filename="package://schunk_description/meshes/powerball/powerball3.stl"/>
 				</geometry>
 			</collision>
@@ -153,5 +153,5 @@
 				<origin xyz="0 0 0" rpy="0 0 0" />
 				<geometry>
-					<mesh filename="package://schunk_description/meshes/powerball/powerball4.stlb"/>
+					<mesh filename="package://schunk_description/meshes/powerball/powerball4.stl"/>
 				</geometry>
 			</collision>
@@ -184,5 +184,5 @@
 				<origin xyz="0 0 0" rpy="0 0 0" />
 				<geometry>
-					<mesh filename="package://schunk_description/meshes/powerball/powerball5.stlb"/>
+					<mesh filename="package://schunk_description/meshes/powerball/powerball5.stl"/>
 				</geometry>
 			</collision>
@@ -215,5 +215,5 @@
 				<origin xyz="0 0 0" rpy="0 0 0" />
 				<geometry>
-					<mesh filename="package://schunk_description/meshes/powerball/powerball6.stlb"/>
+					<mesh filename="package://schunk_description/meshes/powerball/powerball6.stl"/>
 				</geometry>
 			</collision>
