Commit message: New meshes files for powerball

File: schunk_description/urdf/powerball/powerball.urdf.xacro (robot description, xacro)
@@ -35,5 +35,5 @@
 		<!-- joint between arm_0_link and arm_1_link -->
 		<joint name="${name}_1_joint" type="revolute">
-			<origin xyz="0 0 -0.0897" rpy="0 0 0"/>
+			<origin xyz="0 0 0" rpy="0 3.14159 0"/>
 			<parent link="${name}_0_link"/>
 			<child link="${name}_1_link"/>
@@ -53,5 +53,5 @@
 				<origin xyz="0 0 0" rpy="0 0 0" />
 				<geometry>
-					<mesh filename="package://schunk_description/meshes/powerball/powerball1.stl" />
+					<mesh filename="package://schunk_description/meshes/powerball/powerball3.stl" />
 				</geometry>
 				<material name="Blue" />
@@ -60,5 +60,5 @@
 				<origin xyz="0 0 0" rpy="0 0 0" />
 				<geometry>
-					<mesh filename="package://schunk_description/meshes/powerball/powerball1.stl" />
+					<mesh filename="package://schunk_description/meshes/powerball/powerball3.stl" />
 				</geometry>
 			</collision>
@@ -66,5 +66,5 @@
 		<!-- joint between arm_1_link and arm_2_link -->
 		<joint name="${name}_2_joint" type="revolute">
-			<origin xyz="0 0 0" rpy="1.5708 0 0"/>
+			<origin xyz="0 -0.02 -0.05" rpy="1.5708 0 0"/>
 			<parent link="${name}_1_link"/>
 			<child link="${name}_2_link"/>
@@ -97,5 +97,5 @@
 		<!-- joint between arm_2_link and arm_3_link -->
 		<joint name="${name}_3_joint" type="revolute">
-			<origin xyz="0 -0.350 0" rpy="3.14159 0 0"/>
+			<origin xyz="0 -0.350 -0.05" rpy="0 3.14159 3.14159"/>
 			<parent link="${name}_2_link"/>
 			<child link="${name}_3_link"/>
@@ -128,5 +128,5 @@
 		<!-- joint between arm_3_link and arm_4_link -->
 		<joint name="${name}_4_joint" type="revolute">
-			<origin xyz="0 0 0" rpy="1.5708 0 0" />
+			<origin xyz="0 0 -0.05" rpy="1.5708 0 0" />
 			<parent link="${name}_3_link"/>
 			<child link="${name}_4_link"/>
@@ -159,5 +159,5 @@
 		<!-- joint between arm_4_link and arm_5_link -->
 		<joint name="${name}_5_joint" type="revolute">
-			<origin xyz="0 0.005 -0.3049" rpy="1.5708 0 0" />
+			<origin xyz="0 -0.07 -0.3049" rpy="1.5708 1.5708 0" />
 			<parent link="${name}_4_link"/>
 			<child link="${name}_5_link"/>
@@ -190,5 +190,5 @@
 		<!-- joint between arm_5_link and arm_6_link -->
 		<joint name="${name}_6_joint" type="revolute">
-			<origin xyz="0 0 0" rpy="-1.5708 0 0" />
+			<origin xyz="0 0 -0.08" rpy="-1.5708 0 1.5708" />
 			<parent link="${name}_5_link"/>
 			<child link="${name}_6_link"/>

Commit message: Revised powerball  urdf and mesh files

File: schunk_description/urdf/powerball/powerball.urdf.xacro (robot description, xacro)
@@ -22,12 +22,12 @@
 				<origin xyz="0 0 0" rpy="0 0 0" />
 				<geometry>
-					<mesh filename="package://schunk_description/meshes/powerball/powerball0.stl" />
-				</geometry>
-				<material name="Grey" />
-			</visual>
-			<collision>
-				<origin xyz="0 0 0" rpy="0 0 0" />
-				<geometry>
-					<mesh filename="package://schunk_description/meshes/powerball/powerball0.stl" />
+					<mesh filename="package://schunk_description/meshes/powerball/arm_0_link.stl" />
+				</geometry>
+				<material name="Grey" />
+			</visual>
+			<collision>
+				<origin xyz="0 0 0" rpy="0 0 0" />
+				<geometry>
+					<mesh filename="package://schunk_description/meshes/powerball/arm_0_link.stl" />
 				</geometry>
 			</collision>
@@ -35,5 +35,5 @@
 		<!-- joint between arm_0_link and arm_1_link -->
 		<joint name="${name}_1_joint" type="revolute">
-			<origin xyz="0 0 0" rpy="0 3.14159 0"/>
+			<origin xyz="0 0 0" rpy="0 0 0"/>
 			<parent link="${name}_0_link"/>
 			<child link="${name}_1_link"/>
@@ -53,5 +53,5 @@
 				<origin xyz="0 0 0" rpy="0 0 0" />
 				<geometry>
-					<mesh filename="package://schunk_description/meshes/powerball/powerball3.stl" />
+					<mesh filename="package://schunk_description/meshes/powerball/arm_1_link.stl" />
 				</geometry>
 				<material name="Blue" />
@@ -60,5 +60,5 @@
 				<origin xyz="0 0 0" rpy="0 0 0" />
 				<geometry>
-					<mesh filename="package://schunk_description/meshes/powerball/powerball3.stl" />
+					<mesh filename="package://schunk_description/meshes/powerball/arm_1_link.stl" />
 				</geometry>
 			</collision>
@@ -66,5 +66,5 @@
 		<!-- joint between arm_1_link and arm_2_link -->
 		<joint name="${name}_2_joint" type="revolute">
-			<origin xyz="0 -0.02 -0.05" rpy="1.5708 0 0"/>
+			<origin xyz="0 0 0" rpy="1.5708 0 0"/>
 			<parent link="${name}_1_link"/>
 			<child link="${name}_2_link"/>
@@ -73,5 +73,5 @@
 			<dynamics damping="10" />
 			<limit effort="370" velocity="2.0" lower="-2.0943951" upper="2.0943951"/>
-			<safety_controller k_position="20" k_velocity="50" soft_lower_limit="${-2.0943 + 0.01}" 	soft_upper_limit="${2.0943 - 0.01}" />
+			<safety_controller k_position="20" k_velocity="50" soft_lower_limit="${-2.0943 + 0.01}" soft_upper_limit="${2.0943 - 0.01}" />
 		</joint>
 		<link name="${name}_2_link">
@@ -84,12 +84,12 @@
 				<origin xyz="0 0 0" rpy="0 0 0" />
 				<geometry>
-					<mesh filename="package://schunk_description/meshes/powerball/powerball2.stl" />
-				</geometry>
-				<material name="Grey" />
-			</visual>
-			<collision>
-				<origin xyz="0 0 0" rpy="0 0 0" />
-				<geometry>
-					<mesh filename="package://schunk_description/meshes/powerball/powerball2.stl"/>
+					<mesh filename="package://schunk_description/meshes/powerball/arm_2_link.stl" />
+				</geometry>
+				<material name="Grey" />
+			</visual>
+			<collision>
+				<origin xyz="0 0 0" rpy="0 0 0" />
+				<geometry>
+					<mesh filename="package://schunk_description/meshes/powerball/arm_2_link.stl" />
 				</geometry>
 			</collision>
@@ -97,5 +97,5 @@
 		<!-- joint between arm_2_link and arm_3_link -->
 		<joint name="${name}_3_joint" type="revolute">
-			<origin xyz="0 -0.350 -0.05" rpy="0 3.14159 3.14159"/>
+			<origin xyz="0 0.350 0" rpy="0 3.14159 0"/>
 			<parent link="${name}_2_link"/>
 			<child link="${name}_3_link"/>
@@ -115,5 +115,5 @@
 				<origin xyz="0 0 0" rpy="0 0 0" />
 				<geometry>
-					<mesh filename="package://schunk_description/meshes/powerball/powerball3.stl" />
+					<mesh filename="package://schunk_description/meshes/powerball/arm_3_link.stl" />
 				</geometry>
 				<material name="Blue" />
@@ -122,5 +122,5 @@
 				<origin xyz="0 0 0" rpy="0 0 0" />
 				<geometry>
-					<mesh filename="package://schunk_description/meshes/powerball/powerball3.stl"/>
+					<mesh filename="package://schunk_description/meshes/powerball/arm_3_link.stl" />
 				</geometry>
 			</collision>
@@ -128,5 +128,5 @@
 		<!-- joint between arm_3_link and arm_4_link -->
 		<joint name="${name}_4_joint" type="revolute">
-			<origin xyz="0 0 -0.05" rpy="1.5708 0 0" />
+			<origin xyz="0 0 0" rpy="-1.5708 3.14159 0" />
 			<parent link="${name}_3_link"/>
 			<child link="${name}_4_link"/>
@@ -146,12 +146,12 @@
 				<origin xyz="0 0 0" rpy="0 0 0" />
 				<geometry>
-					<mesh filename="package://schunk_description/meshes/powerball/powerball4.stl" />
-				</geometry>
-				<material name="Grey" />
-			</visual>
-			<collision>
-				<origin xyz="0 0 0" rpy="0 0 0" />
-				<geometry>
-					<mesh filename="package://schunk_description/meshes/powerball/powerball4.stl"/>
+					<mesh filename="package://schunk_description/meshes/powerball/arm_4_link.stl" />
+				</geometry>
+				<material name="Grey" />
+			</visual>
+			<collision>
+				<origin xyz="0 0 0" rpy="0 0 0" />
+				<geometry>
+					<mesh filename="package://schunk_description/meshes/powerball/arm_4_link.stl" />
 				</geometry>
 			</collision>
@@ -159,5 +159,5 @@
 		<!-- joint between arm_4_link and arm_5_link -->
 		<joint name="${name}_5_joint" type="revolute">
-			<origin xyz="0 -0.07 -0.3049" rpy="1.5708 1.5708 0" />
+			<origin xyz="0 0.05263 0.3049" rpy="1.5708 0 3.14159" />
 			<parent link="${name}_4_link"/>
 			<child link="${name}_5_link"/>
@@ -177,5 +177,5 @@
 				<origin xyz="0 0 0" rpy="0 0 0" />
 				<geometry>
-					<mesh filename="package://schunk_description/meshes/powerball/powerball5.stl" />
+					<mesh filename="package://schunk_description/meshes/powerball/arm_5_link.stl" />
 				</geometry>
 				<material name="Blue" />
@@ -184,5 +184,5 @@
 				<origin xyz="0 0 0" rpy="0 0 0" />
 				<geometry>
-					<mesh filename="package://schunk_description/meshes/powerball/powerball5.stl"/>
+					<mesh filename="package://schunk_description/meshes/powerball/arm_5_link.stl" />
 				</geometry>
 			</collision>
@@ -190,5 +190,5 @@
 		<!-- joint between arm_5_link and arm_6_link -->
 		<joint name="${name}_6_joint" type="revolute">
-			<origin xyz="0 0 -0.08" rpy="-1.5708 0 1.5708" />
+			<origin xyz="0 0 0" rpy="-1.5708 0 0" />
 			<parent link="${name}_5_link"/>
 			<child link="${name}_6_link"/>
@@ -208,12 +208,12 @@
 				<origin xyz="0 0 0" rpy="0 0 0" />
 				<geometry>
-					<mesh filename="package://schunk_description/meshes/powerball/powerball6.stl" />
-				</geometry>
-				<material name="Grey" />
-			</visual>
-			<collision>
-				<origin xyz="0 0 0" rpy="0 0 0" />
-				<geometry>
-					<mesh filename="package://schunk_description/meshes/powerball/powerball6.stl"/>
+					<mesh filename="package://schunk_description/meshes/powerball/arm_6_link.stl" />
+				</geometry>
+				<material name="Grey" />
+			</visual>
+			<collision>
+				<origin xyz="0 0 0" rpy="0 0 0" />
+				<geometry>
+					<mesh filename="package://schunk_description/meshes/powerball/arm_6_link.stl" />
 				</geometry>
 			</collision>

Commit message: Fixed arm_0_link origin

File: schunk_description/urdf/powerball/powerball.urdf.xacro (robot description, xacro)
@@ -35,5 +35,5 @@
 		<!-- joint between arm_0_link and arm_1_link -->
 		<joint name="${name}_1_joint" type="revolute">
-			<origin xyz="0 0 0" rpy="0 0 0"/>
+			<origin xyz="0 0 0.11" rpy="0 0 0"/>
 			<parent link="${name}_0_link"/>
 			<child link="${name}_1_link"/>
@@ -159,5 +159,5 @@
 		<!-- joint between arm_4_link and arm_5_link -->
 		<joint name="${name}_5_joint" type="revolute">
-			<origin xyz="0 0.05263 0.3049" rpy="1.5708 0 3.14159" />
+			<origin xyz="0 0.005263 0.365" rpy="1.5708 0 3.14159" />
 			<parent link="${name}_4_link"/>
 			<child link="${name}_5_link"/>
