Commit message: added meshes files for lwa4p_extended

File: schunk_description/urdf/lwa4p_extended/lwa4p_extended.gazebo.xacro (robot description, xacro)
@@ -11,5 +11,5 @@
 		</gazebo>
 		<gazebo reference="${name}_1_link">
-			<material value="Schunk/Blue" />
+			<material value="Schunk/LightGrey" />
 			<turnGravityOff>false</turnGravityOff>
 			<selfCollide>true</selfCollide>
@@ -21,5 +21,5 @@
 		</gazebo>
 		<gazebo reference="${name}_3_link">
-			<material value="Schunk/Blue" />
+			<material value="Schunk/LightGrey" />
 			<turnGravityOff>false</turnGravityOff>
 			<selfCollide>true</selfCollide>
@@ -31,5 +31,5 @@
 		</gazebo>
 		<gazebo reference="${name}_5_link">
-			<material value="Schunk/Blue" />
+			<material value="Schunk/LightGrey" />
 			<turnGravityOff>false</turnGravityOff>
 			<selfCollide>true</selfCollide>

File: schunk_description/urdf/lwa4p_extended/lwa4p_extended.urdf.xacro (robot description, xacro)
@@ -13,5 +13,11 @@
 			<child link="${name}_base_link"/>
 		</joint>
-		<link name="${name}_base_link"/>
+		<link name="${name}_base_link">
+			<inertial>
+				<origin xyz="0 0 0" rpy="0 0 0"/>
+				<mass value="0.1"/>
+				<inertia ixx="0.01" ixy="0" ixz="0" iyy="0.01" iyz="0" izz="0.01" />
+			</inertial>
+		</link>
 		<!-- joint between arm_base_link and arm_1_link -->
 		<joint name="${name}_1_joint" type="revolute" >
@@ -25,5 +31,11 @@
 			<safety_controller k_position="20" k_velocity="50" soft_lower_limit="${-6.2831853 + 0.01}" soft_upper_limit="${6.2831853 - 0.01}" />
 		</joint>
-		<link name="${name}_1_link"/>
+		<link name="${name}_1_link">
+			<inertial>
+				<origin xyz="0 0 0" rpy="0 0 0"/>
+				<mass value="0.1"/>
+				<inertia ixx="0.01" ixy="0" ixz="0" iyy="0.01" iyz="0" izz="0.01" />
+			</inertial>
+		</link>
 		<!-- joint between arm_1_link and arm_2_link -->
 		<joint name="${name}_2_joint" type="revolute">
@@ -37,5 +49,24 @@
 			<safety_controller k_position="20" k_velocity="50" soft_lower_limit="${-2.0943 + 0.01}" soft_upper_limit="${2.0943 - 0.01}" />
 		</joint>
-		<link name="${name}_2_link"/>
+		<link name="${name}_2_link">
+			<inertial>
+				<origin xyz="0 0 0" rpy="0 0 0"/>
+				<mass value="0.1"/>
+				<inertia ixx="0.01" ixy="0" ixz="0" iyy="0.01" iyz="0" izz="0.01" />
+			</inertial>
+		<visual>
+				<origin xyz="0 0 0" rpy="0 0 0" />
+				<geometry>
+					<mesh filename="package://schunk_description/meshes/lwa4p_extended/arm_1_link.stl" />
+				</geometry>
+				<material name="Schunk/LightGrey" />
+			</visual>
+			<collision>
+				<origin xyz="0 0 0" rpy="0 0 0" />
+				<geometry>
+					<mesh filename="package://schunk_description/meshes/lwa4p_extended/arm_1_link.stl" />
+				</geometry>
+			</collision>
+		</link>
 		<!-- joint between arm_2_link and arm_3_link -->
 		<joint name="${name}_3_joint" type="revolute">
@@ -49,5 +80,29 @@
 			<safety_controller k_position="20" k_velocity="25" soft_lower_limit="${-6.2831853 + 0.01}" soft_upper_limit="${6.2831853 - 0.01}" />
 		</joint>
-		<link name="${name}_3_link"/>
+		<link name="${name}_3_link">
+			<inertial>
+				<origin xyz="0 0 0" rpy="0 0 0"/>
+				<mass value="0.1"/>
+				<inertia ixx="0.01" ixy="0" ixz="0" iyy="0.01" iyz="0" izz="0.01" />
+			</inertial>
+			<inertial>
+				<origin xyz="0 0 0" rpy="0 0 0"/>
+				<mass value="0.1"/>
+				<inertia ixx="0.01" ixy="0" ixz="0" iyy="0.01" iyz="0" izz="0.01" />
+			</inertial>
+		<visual>
+				<origin xyz="0 0 0" rpy="0 0 0" />
+				<geometry>
+					<mesh filename="package://schunk_description/meshes/lwa4p_extended/arm_2_link.stl" />
+				</geometry>
+				<material name="Schunk/LightGrey" />
+			</visual>
+			<collision>
+				<origin xyz="0 0 0" rpy="0 0 0" />
+				<geometry>
+					<mesh filename="package://schunk_description/meshes/lwa4p_extended/arm_2_link.stl" />
+				</geometry>
+			</collision>
+		</link>
 		<!-- joint between arm_3_link and arm_4_link -->
 		<joint name="${name}_4_joint" type="revolute">
@@ -61,5 +116,24 @@
 			<safety_controller k_position="20" k_velocity="25" soft_lower_limit="${-2.0943951 + 0.01}" soft_upper_limit="${2.0943951 - 0.01}" />
 		</joint>
-		<link name="${name}_4_link"/>
+		<link name="${name}_4_link">
+			<inertial>
+				<origin xyz="0 0 0" rpy="0 0 0"/>
+				<mass value="0.1"/>
+				<inertia ixx="0.01" ixy="0" ixz="0" iyy="0.01" iyz="0" izz="0.01" />
+			</inertial>
+			<visual>
+				<origin xyz="0 0 0" rpy="0 0 0" />
+				<geometry>
+					<mesh filename="package://schunk_description/meshes/lwa4p_extended/arm_3_link.stl" />
+				</geometry>
+				<material name="Schunk/LightGrey" />
+			</visual>
+			<collision>
+				<origin xyz="0 0 0" rpy="0 0 0" />
+				<geometry>
+					<mesh filename="package://schunk_description/meshes/lwa4p_extended/arm_3_link.stl" />
+				</geometry>
+			</collision>
+		</link>
 		<!-- joint between arm_4_link and arm_5_link -->
 		<joint name="${name}_5_joint" type="revolute">
@@ -73,5 +147,24 @@
 			<safety_controller k_position="20" k_velocity="25" soft_lower_limit="${-6.2831853 + 0.01}" soft_upper_limit="${6.2831853 - 0.01}" />
 		</joint>
-		<link name="${name}_5_link"/>
+		<link name="${name}_5_link">
+			<inertial>
+				<origin xyz="0 0 0" rpy="0 0 0"/>
+				<mass value="0.1"/>
+				<inertia ixx="0.01" ixy="0" ixz="0" iyy="0.01" iyz="0" izz="0.01" />
+			</inertial>
+			<visual>
+				<origin xyz="0 0 0" rpy="0 0 0" />
+				<geometry>
+					<mesh filename="package://schunk_description/meshes/lwa4p_extended/arm_4_link.stl" />
+				</geometry>
+				<material name="Schunk/LightGrey" />
+			</visual>
+			<collision>
+				<origin xyz="0 0 0" rpy="0 0 0" />
+				<geometry>
+					<mesh filename="package://schunk_description/meshes/lwa4p_extended/arm_4_link.stl" />
+				</geometry>
+			</collision>
+		</link>
 		<!-- joint between arm_5_link and arm_6_link -->
 		<joint name="${name}_6_joint" type="revolute">
@@ -85,5 +178,24 @@
 			<safety_controller k_position="20" k_velocity="25" soft_lower_limit="${-2.0943951 + 0.01}" soft_upper_limit="${2.0943951 - 0.01}" />
 		</joint>
-		<link name="${name}_6_link"/>
+		<link name="${name}_6_link">
+			<inertial>
+				<origin xyz="0 0 0" rpy="0 0 0"/>
+				<mass value="0.1"/>
+				<inertia ixx="0.01" ixy="0" ixz="0" iyy="0.01" iyz="0" izz="0.01" />
+			</inertial>
+			<visual>
+				<origin xyz="0 0 0" rpy="0 0 0" />
+				<geometry>
+					<mesh filename="package://schunk_description/meshes/lwa4p_extended/arm_5_link.stl" />
+				</geometry>
+				<material name="Schunk/LightGrey" />
+			</visual>
+			<collision>
+				<origin xyz="0 0 0" rpy="0 0 0" />
+				<geometry>
+					<mesh filename="package://schunk_description/meshes/lwa4p_extended/arm_5_link.stl" />
+				</geometry>
+			</collision>
+		</link>
 		<!-- joint between arm_6_link and arm_7_link -->
 		<joint name="${name}_7_joint" type="revolute">
@@ -97,5 +209,11 @@
 			<safety_controller k_position="20" k_velocity="25" soft_lower_limit="${-2.0943951 + 0.01}" soft_upper_limit="${2.0943951 - 0.01}" />
 		</joint>
-		<link name="${name}_7_link"/>
+		<link name="${name}_7_link">
+			<inertial>
+				<origin xyz="0 0 0" rpy="0 0 0"/>
+				<mass value="0.1"/>
+				<inertia ixx="0.01" ixy="0" ixz="0" iyy="0.01" iyz="0" izz="0.01" />
+			</inertial>
+		</link>
 		<!-- extensions -->
 		<xacro:schunk_lwa4p_extended_gazebo name="${name}" />

Commit message: update xacro file format

File: schunk_description/urdf/lwa4p_extended/lwa4p_extended.gazebo.xacro (robot description, xacro)
@@ -1,48 +1,45 @@
 <?xml version="1.0"?>
-<robot xmlns:sensor="http://playerstage.sourceforge.net/gazebo/xmlschema/#sensor"
-       xmlns:controller="http://playerstage.sourceforge.net/gazebo/xmlschema/#controller"
-       xmlns:interface="http://playerstage.sourceforge.net/gazebo/xmlschema/#interface"
-       xmlns:xacro="http://ros.org/wiki/xacro">
-	<xacro:macro name="schunk_lwa4p_extended_gazebo" params="name">
-		<gazebo reference="${name}_0_link">
-			<material value="Schunk/LightGrey" />
-			<turnGravityOff>false</turnGravityOff>
-			<selfCollide>true</selfCollide>
-		</gazebo>
-		<gazebo reference="${name}_1_link">
-			<material value="Schunk/LightGrey" />
-			<turnGravityOff>false</turnGravityOff>
-			<selfCollide>true</selfCollide>
-		</gazebo>
-		<gazebo reference="${name}_2_link">
-			<material value="Schunk/LightGrey" />
-			<turnGravityOff>false</turnGravityOff>
-			<selfCollide>true</selfCollide>
-		</gazebo>
-		<gazebo reference="${name}_3_link">
-			<material value="Schunk/LightGrey" />
-			<turnGravityOff>false</turnGravityOff>
-			<selfCollide>true</selfCollide>
-		</gazebo>
-		<gazebo reference="${name}_4_link">
-			<material value="Schunk/LightGrey" />
-			<turnGravityOff>false</turnGravityOff>
-			<selfCollide>true</selfCollide>
-		</gazebo>
-		<gazebo reference="${name}_5_link">
-			<material value="Schunk/LightGrey" />
-			<turnGravityOff>false</turnGravityOff>
-			<selfCollide>true</selfCollide>
-		</gazebo>
-		<gazebo reference="${name}_6_link">
-			<material value="Schunk/LightGrey" />
-			<turnGravityOff>false</turnGravityOff>
-			<selfCollide>true</selfCollide>
-		</gazebo>
-		<gazebo reference="${name}_7_link">
-			<material value="Schunk/LightGrey" />
-			<turnGravityOff>false</turnGravityOff>
-			<selfCollide>true</selfCollide>
-		</gazebo>
-	</xacro:macro>
+<robot xmlns:xacro="http://www.ros.org/wiki/xacro">
+  <xacro:macro name="schunk_lwa4p_extended_gazebo" params="name">
+    <gazebo reference="${name}_0_link">
+      <material value="Schunk/LightGrey" />
+      <turnGravityOff>false</turnGravityOff>
+      <selfCollide>true</selfCollide>
+    </gazebo>
+    <gazebo reference="${name}_1_link">
+      <material value="Schunk/LightGrey" />
+      <turnGravityOff>false</turnGravityOff>
+      <selfCollide>true</selfCollide>
+    </gazebo>
+    <gazebo reference="${name}_2_link">
+      <material value="Schunk/LightGrey" />
+      <turnGravityOff>false</turnGravityOff>
+      <selfCollide>true</selfCollide>
+    </gazebo>
+    <gazebo reference="${name}_3_link">
+      <material value="Schunk/LightGrey" />
+      <turnGravityOff>false</turnGravityOff>
+      <selfCollide>true</selfCollide>
+    </gazebo>
+    <gazebo reference="${name}_4_link">
+      <material value="Schunk/LightGrey" />
+      <turnGravityOff>false</turnGravityOff>
+      <selfCollide>true</selfCollide>
+    </gazebo>
+    <gazebo reference="${name}_5_link">
+      <material value="Schunk/LightGrey" />
+      <turnGravityOff>false</turnGravityOff>
+      <selfCollide>true</selfCollide>
+    </gazebo>
+    <gazebo reference="${name}_6_link">
+      <material value="Schunk/LightGrey" />
+      <turnGravityOff>false</turnGravityOff>
+      <selfCollide>true</selfCollide>
+    </gazebo>
+    <gazebo reference="${name}_7_link">
+      <material value="Schunk/LightGrey" />
+      <turnGravityOff>false</turnGravityOff>
+      <selfCollide>true</selfCollide>
+    </gazebo>
+  </xacro:macro>
 </robot>

File: schunk_description/urdf/lwa4p_extended/lwa4p_extended.transmission.xacro (robot description, xacro)
@@ -1,43 +1,61 @@
 <?xml version="1.0"?>
-<robot xmlns:sensor="http://playerstage.sourceforge.net/gazebo/xmlschema/#sensor"
-       xmlns:controller="http://playerstage.sourceforge.net/gazebo/xmlschema/#controller"
-       xmlns:interface="http://playerstage.sourceforge.net/gazebo/xmlschema/#interface"
-       xmlns:xacro="http://ros.org/wiki/xacro">
-	<xacro:macro name="schunk_lwa4p_extended_transmission" params="name">
-		<transmission name="${name}_1_trans" type="pr2_mechanism_model/SimpleTransmission">
-			<actuator name="${name}_1_motor"/>
-			<joint name="${name}_1_joint"/>
-			<mechanicalReduction>1</mechanicalReduction>
-		</transmission>
-		<transmission name="${name}_2_trans" type="pr2_mechanism_model/SimpleTransmission">
-			<actuator name="${name}_2_motor"/>
-			<joint name="${name}_2_joint"/>
-			<mechanicalReduction>1</mechanicalReduction>
-		</transmission>
-		<transmission name="${name}_3_trans" type="pr2_mechanism_model/SimpleTransmission">
-			<actuator name="${name}_3_motor"/>
-			<joint name="${name}_3_joint"/>
-			<mechanicalReduction>1</mechanicalReduction>
-		</transmission>
-		<transmission name="${name}_4_trans" type="pr2_mechanism_model/SimpleTransmission">
-			<actuator name="${name}_4_motor"/>
-			<joint name="${name}_4_joint"/>
-			<mechanicalReduction>1</mechanicalReduction>
-		</transmission>
-		<transmission name="${name}_5_trans" type="pr2_mechanism_model/SimpleTransmission">
-			<actuator name="${name}_5_motor"/>
-			<joint name="${name}_5_joint"/>
-			<mechanicalReduction>1</mechanicalReduction>
-		</transmission>
-		<transmission name="${name}_6_trans" type="pr2_mechanism_model/SimpleTransmission">
-			<actuator name="${name}_6_motor"/>
-			<joint name="${name}_6_joint"/>
-			<mechanicalReduction>1</mechanicalReduction>
-		</transmission>
-		<transmission name="${name}_7_trans" type="pr2_mechanism_model/SimpleTransmission">
-			<actuator name="${name}_7_motor"/>
-			<joint name="${name}_7_joint"/>
-			<mechanicalReduction>1</mechanicalReduction>
-		</transmission>
-	</xacro:macro>
+<robot xmlns:xacro="http://www.ros.org/wiki/xacro">
+  <xacro:macro name="schunk_lwa4p_extended_transmission" params="name">
+    <transmission name="${name}_1_trans">
+      <type>transmission_interface/SimpleTransmission</type>
+      <joint name="${name}_1_joint"/>
+      <actuator name="${name}_1_motor">
+        <hardwareInterface>EffortJointInterface</hardwareInterface>
+        <mechanicalReduction>1</mechanicalReduction>
+      </actuator>
+    </transmission>
+    <transmission name="${name}_2_trans">
+      <type>transmission_interface/SimpleTransmission</type>
+      <joint name="${name}_2_joint"/>
+      <actuator name="${name}_2_motor">
+        <hardwareInterface>EffortJointInterface</hardwareInterface>
+        <mechanicalReduction>1</mechanicalReduction>
+      </actuator>
+    </transmission>
+    <transmission name="${name}_3_trans">
+      <type>transmission_interface/SimpleTransmission</type>
+      <joint name="${name}_3_joint"/>
+      <actuator name="${name}_3_motor">
+        <hardwareInterface>EffortJointInterface</hardwareInterface>
+        <mechanicalReduction>1</mechanicalReduction>
+      </actuator>
+    </transmission>
+    <transmission name="${name}_4_trans">
+      <type>transmission_interface/SimpleTransmission</type>
+      <joint name="${name}_4_joint"/>
+      <actuator name="${name}_4_motor">
+        <hardwareInterface>EffortJointInterface</hardwareInterface>
+        <mechanicalReduction>1</mechanicalReduction>
+      </actuator>
+    </transmission>
+    <transmission name="${name}_5_trans">
+      <type>transmission_interface/SimpleTransmission</type>
+      <joint name="${name}_5_joint"/>
+      <actuator name="${name}_5_motor">
+        <hardwareInterface>EffortJointInterface</hardwareInterface>
+        <mechanicalReduction>1</mechanicalReduction>
+      </actuator>
+    </transmission>
+    <transmission name="${name}_6_trans">
+      <type>transmission_interface/SimpleTransmission</type>
+      <joint name="${name}_6_joint"/>
+      <actuator name="${name}_6_motor">
+        <hardwareInterface>EffortJointInterface</hardwareInterface>
+        <mechanicalReduction>1</mechanicalReduction>
+      </actuator>
+    </transmission>
+    <transmission name="${name}_7_trans">
+      <type>transmission_interface/SimpleTransmission</type>
+      <joint name="${name}_7_joint"/>
+      <actuator name="${name}_7_motor">
+        <hardwareInterface>EffortJointInterface</hardwareInterface>
+        <mechanicalReduction>1</mechanicalReduction>
+      </actuator>
+    </transmission>
+  </xacro:macro>
 </robot>
