Commit message: update xacro file format

File: schunk_description/urdf/lwa4p_extended/lwa4p_extended.urdf.xacro (robot description, xacro)
@@ -1,222 +1,219 @@
 <?xml version="1.0"?>
-<robot xmlns:sensor="http://playerstage.sourceforge.net/gazebo/xmlschema/#sensor"
-       xmlns:controller="http://playerstage.sourceforge.net/gazebo/xmlschema/#controller"
-       xmlns:interface="http://playerstage.sourceforge.net/gazebo/xmlschema/#interface"
-       xmlns:xacro="http://ros.org/wiki/xacro">
-	<include filename="$(find schunk_description)/urdf/lwa4p_extended/lwa4p_extended.gazebo.xacro" />
-	<include filename="$(find schunk_description)/urdf/lwa4p_extended/lwa4p_extended.transmission.xacro" />
-	<xacro:macro name="schunk_lwa4p_extended" params="parent name *origin arm_1_ref arm_2_ref arm_3_ref arm_4_ref arm_5_ref arm_6_ref arm_7_ref">
-		<!-- joint between base_link and lwa4p_extended_connector_link -->
-		<joint name="${name}_base_joint" type="fixed">
-			<insert_block name="origin" />
-			<parent link="${parent}"/>
-			<child link="${name}_base_link"/>
-		</joint>
-		<link name="${name}_base_link">
-			<inertial>
-				<origin xyz="0 0 0" rpy="0 0 0"/>
-				<mass value="0.1"/>
-				<inertia ixx="0.01" ixy="0" ixz="0" iyy="0.01" iyz="0" izz="0.01" />
-			</inertial>
-		</link>
-		<!-- joint between arm_base_link and arm_1_link -->
-		<joint name="${name}_1_joint" type="revolute" >
-			<origin xyz="0 0 0" rpy="0 0 0" />
-			<parent link="${name}_base_link" />
-			<child link="${name}_1_link" />
-			<axis xyz="0 0 1"/>
-			<calibration rising="${arm_1_ref}"/>
-			<dynamics damping="10" />
-			<limit effort="370" velocity="2.0" lower="-6.2831853" upper="6.2831853"/>
-			<safety_controller k_position="20" k_velocity="50" soft_lower_limit="${-6.2831853 + 0.01}" soft_upper_limit="${6.2831853 - 0.01}" />
-		</joint>
-		<link name="${name}_1_link">
-			<inertial>
-				<origin xyz="0 0 0" rpy="0 0 0"/>
-				<mass value="0.1"/>
-				<inertia ixx="0.01" ixy="0" ixz="0" iyy="0.01" iyz="0" izz="0.01" />
-			</inertial>
-		</link>
-		<!-- joint between arm_1_link and arm_2_link -->
-		<joint name="${name}_2_joint" type="revolute">
-			<origin xyz="0 0 0.0915" rpy="1.5708 0 0"/>
-			<parent link="${name}_1_link"/>
-			<child link="${name}_2_link"/>
-			<axis xyz="0 0 1"/>
-			<calibration rising="${arm_2_ref}"/>
-			<dynamics damping="10" />
-			<limit effort="370" velocity="2.0" lower="-2.0943951" upper="2.0943951"/>
-			<safety_controller k_position="20" k_velocity="50" soft_lower_limit="${-2.0943 + 0.01}" soft_upper_limit="${2.0943 - 0.01}" />
-		</joint>
-		<link name="${name}_2_link">
-			<inertial>
-				<origin xyz="0 0 0" rpy="0 0 0"/>
-				<mass value="0.1"/>
-				<inertia ixx="0.01" ixy="0" ixz="0" iyy="0.01" iyz="0" izz="0.01" />
-			</inertial>
-		<visual>
-				<origin xyz="0 0 0" rpy="0 0 0" />
-				<geometry>
-					<mesh filename="package://schunk_description/meshes/lwa4p_extended/arm_1_link.stl" />
-				</geometry>
-				<material name="Schunk/LightGrey" />
-			</visual>
-			<collision>
-				<origin xyz="0 0 0" rpy="0 0 0" />
-				<geometry>
-					<mesh filename="package://schunk_description/meshes/lwa4p_extended/arm_1_link.stl" />
-				</geometry>
-			</collision>
-		</link>
-		<!-- joint between arm_2_link and arm_3_link -->
-		<joint name="${name}_3_joint" type="revolute">
-			<origin xyz="0 0 0" rpy="-1.5708 0 0"/>
-			<parent link="${name}_2_link"/>
-			<child link="${name}_3_link"/>
-			<axis xyz="0 0 1"/>
-			<calibration rising="${arm_3_ref}"/>
-			<dynamics damping="5" />
-			<limit effort="176" velocity="2.0" lower="-6.2831853" upper="6.2831853"/>
-			<safety_controller k_position="20" k_velocity="25" soft_lower_limit="${-6.2831853 + 0.01}" soft_upper_limit="${6.2831853 - 0.01}" />
-		</joint>
-		<link name="${name}_3_link">
-			<inertial>
-				<origin xyz="0 0 0" rpy="0 0 0"/>
-				<mass value="0.1"/>
-				<inertia ixx="0.01" ixy="0" ixz="0" iyy="0.01" iyz="0" izz="0.01" />
-			</inertial>
-			<inertial>
-				<origin xyz="0 0 0" rpy="0 0 0"/>
-				<mass value="0.1"/>
-				<inertia ixx="0.01" ixy="0" ixz="0" iyy="0.01" iyz="0" izz="0.01" />
-			</inertial>
-		<visual>
-				<origin xyz="0 0 0" rpy="0 0 0" />
-				<geometry>
-					<mesh filename="package://schunk_description/meshes/lwa4p_extended/arm_2_link.stl" />
-				</geometry>
-				<material name="Schunk/LightGrey" />
-			</visual>
-			<collision>
-				<origin xyz="0 0 0" rpy="0 0 0" />
-				<geometry>
-					<mesh filename="package://schunk_description/meshes/lwa4p_extended/arm_2_link.stl" />
-				</geometry>
-			</collision>
-		</link>
-		<!-- joint between arm_3_link and arm_4_link -->
-		<joint name="${name}_4_joint" type="revolute">
-			<origin xyz="0 0 0.45360" rpy="1.5708 0 0" />
-			<parent link="${name}_3_link"/>
-			<child link="${name}_4_link"/>
-			<axis xyz="0 0 1" />
-			<calibration rising="${arm_4_ref}"/>
-			<dynamics damping="5" />
-			<limit effort="176" velocity="2.0" lower="-2.0943951" upper="2.0943951"/>
-			<safety_controller k_position="20" k_velocity="25" soft_lower_limit="${-2.0943951 + 0.01}" soft_upper_limit="${2.0943951 - 0.01}" />
-		</joint>
-		<link name="${name}_4_link">
-			<inertial>
-				<origin xyz="0 0 0" rpy="0 0 0"/>
-				<mass value="0.1"/>
-				<inertia ixx="0.01" ixy="0" ixz="0" iyy="0.01" iyz="0" izz="0.01" />
-			</inertial>
-			<visual>
-				<origin xyz="0 0 0" rpy="0 0 0" />
-				<geometry>
-					<mesh filename="package://schunk_description/meshes/lwa4p_extended/arm_3_link.stl" />
-				</geometry>
-				<material name="Schunk/LightGrey" />
-			</visual>
-			<collision>
-				<origin xyz="0 0 0" rpy="0 0 0" />
-				<geometry>
-					<mesh filename="package://schunk_description/meshes/lwa4p_extended/arm_3_link.stl" />
-				</geometry>
-			</collision>
-		</link>
-		<!-- joint between arm_4_link and arm_5_link -->
-		<joint name="${name}_5_joint" type="revolute">
-			<origin xyz="0 0 0" rpy="-1.5708 0 0" />
-			<parent link="${name}_4_link"/>
-			<child link="${name}_5_link"/>
-			<axis xyz="0 0 1" />
-			<calibration rising="${arm_5_ref}"/>
-			<dynamics damping="5" />
-			<limit effort="41.6" velocity="2.0" lower="-6.2831853" upper="6.2831853" />
-			<safety_controller k_position="20" k_velocity="25" soft_lower_limit="${-6.2831853 + 0.01}" soft_upper_limit="${6.2831853 - 0.01}" />
-		</joint>
-		<link name="${name}_5_link">
-			<inertial>
-				<origin xyz="0 0 0" rpy="0 0 0"/>
-				<mass value="0.1"/>
-				<inertia ixx="0.01" ixy="0" ixz="0" iyy="0.01" iyz="0" izz="0.01" />
-			</inertial>
-			<visual>
-				<origin xyz="0 0 0" rpy="0 0 0" />
-				<geometry>
-					<mesh filename="package://schunk_description/meshes/lwa4p_extended/arm_4_link.stl" />
-				</geometry>
-				<material name="Schunk/LightGrey" />
-			</visual>
-			<collision>
-				<origin xyz="0 0 0" rpy="0 0 0" />
-				<geometry>
-					<mesh filename="package://schunk_description/meshes/lwa4p_extended/arm_4_link.stl" />
-				</geometry>
-			</collision>
-		</link>
-		<!-- joint between arm_5_link and arm_6_link -->
-		<joint name="${name}_6_joint" type="revolute">
-			<origin xyz="0 0 0.2986" rpy="1.5708 0 0" />
-			<parent link="${name}_5_link"/>
-			<child link="${name}_6_link"/>
-			<axis xyz="0 0 1" />
-			<calibration rising="${arm_6_ref}"/>
-			<dynamics damping="5" />
-			<limit effort="20.1" velocity="2.0" lower="-2.0943951" upper="2.0943951" />
-			<safety_controller k_position="20" k_velocity="25" soft_lower_limit="${-2.0943951 + 0.01}" soft_upper_limit="${2.0943951 - 0.01}" />
-		</joint>
-		<link name="${name}_6_link">
-			<inertial>
-				<origin xyz="0 0 0" rpy="0 0 0"/>
-				<mass value="0.1"/>
-				<inertia ixx="0.01" ixy="0" ixz="0" iyy="0.01" iyz="0" izz="0.01" />
-			</inertial>
-			<visual>
-				<origin xyz="0 0 0" rpy="0 0 0" />
-				<geometry>
-					<mesh filename="package://schunk_description/meshes/lwa4p_extended/arm_5_link.stl" />
-				</geometry>
-				<material name="Schunk/LightGrey" />
-			</visual>
-			<collision>
-				<origin xyz="0 0 0" rpy="0 0 0" />
-				<geometry>
-					<mesh filename="package://schunk_description/meshes/lwa4p_extended/arm_5_link.stl" />
-				</geometry>
-			</collision>
-		</link>
-		<!-- joint between arm_6_link and arm_7_link -->
-		<joint name="${name}_7_joint" type="revolute">
-			<origin xyz="0 0 0" rpy="-1.5708 0 0" />
-			<parent link="${name}_6_link"/>
-			<child link="${name}_7_link"/>
-			<axis xyz="0 0 1" />
-			<calibration rising="${arm_7_ref}"/>
-			<dynamics damping="5" />
-			<limit effort="20.1" velocity="2.0" lower="-2.0943951" upper="2.0943951" />
-			<safety_controller k_position="20" k_velocity="25" soft_lower_limit="${-2.0943951 + 0.01}" soft_upper_limit="${2.0943951 - 0.01}" />
-		</joint>
-		<link name="${name}_7_link">
-			<inertial>
-				<origin xyz="0 0 0" rpy="0 0 0"/>
-				<mass value="0.1"/>
-				<inertia ixx="0.01" ixy="0" ixz="0" iyy="0.01" iyz="0" izz="0.01" />
-			</inertial>
-		</link>
-		<!-- extensions -->
-		<xacro:schunk_lwa4p_extended_gazebo name="${name}" />
-		<xacro:schunk_lwa4p_extended_transmission name="${name}" />
-	</xacro:macro>
+<robot xmlns:xacro="http://www.ros.org/wiki/xacro">
+  <xacro:include filename="$(find schunk_description)/urdf/lwa4p_extended/lwa4p_extended.gazebo.xacro" />
+  <xacro:include filename="$(find schunk_description)/urdf/lwa4p_extended/lwa4p_extended.transmission.xacro" />
+  <xacro:macro name="schunk_lwa4p_extended" params="parent name *origin arm_1_ref arm_2_ref arm_3_ref arm_4_ref arm_5_ref arm_6_ref arm_7_ref">
+    <!-- joint between base_link and lwa4p_extended_connector_link -->
+    <joint name="${name}_base_joint" type="fixed">
+      <insert_block name="origin" />
+      <parent link="${parent}"/>
+      <child link="${name}_base_link"/>
+    </joint>
+    <link name="${name}_base_link">
+      <inertial>
+        <origin xyz="0 0 0" rpy="0 0 0"/>
+        <mass value="0.1"/>
+        <inertia ixx="0.01" ixy="0" ixz="0" iyy="0.01" iyz="0" izz="0.01" />
+      </inertial>
+    </link>
+    <!-- joint between arm_base_link and arm_1_link -->
+    <joint name="${name}_1_joint" type="revolute" >
+      <origin xyz="0 0 0" rpy="0 0 0" />
+      <parent link="${name}_base_link" />
+      <child link="${name}_1_link" />
+      <axis xyz="0 0 1"/>
+      <calibration rising="${arm_1_ref}"/>
+      <dynamics damping="10" />
+      <limit effort="370" velocity="2.0" lower="-6.2831853" upper="6.2831853"/>
+      <safety_controller k_position="20" k_velocity="50" soft_lower_limit="${-6.2831853 + 0.01}" soft_upper_limit="${6.2831853 - 0.01}" />
+    </joint>
+    <link name="${name}_1_link">
+      <inertial>
+        <origin xyz="0 0 0" rpy="0 0 0"/>
+        <mass value="0.1"/>
+        <inertia ixx="0.01" ixy="0" ixz="0" iyy="0.01" iyz="0" izz="0.01" />
+      </inertial>
+    </link>
+    <!-- joint between arm_1_link and arm_2_link -->
+    <joint name="${name}_2_joint" type="revolute">
+      <origin xyz="0 0 0.0915" rpy="1.5708 0 0"/>
+      <parent link="${name}_1_link"/>
+      <child link="${name}_2_link"/>
+      <axis xyz="0 0 1"/>
+      <calibration rising="${arm_2_ref}"/>
+      <dynamics damping="10" />
+      <limit effort="370" velocity="2.0" lower="-2.0943951" upper="2.0943951"/>
+      <safety_controller k_position="20" k_velocity="50" soft_lower_limit="${-2.0943 + 0.01}" soft_upper_limit="${2.0943 - 0.01}" />
+    </joint>
+    <link name="${name}_2_link">
+      <inertial>
+        <origin xyz="0 0 0" rpy="0 0 0"/>
+        <mass value="0.1"/>
+        <inertia ixx="0.01" ixy="0" ixz="0" iyy="0.01" iyz="0" izz="0.01" />
+      </inertial>
+    <visual>
+        <origin xyz="0 0 0" rpy="0 0 0" />
+        <geometry>
+          <mesh filename="package://schunk_description/meshes/lwa4p_extended/arm_1_link.stl" />
+        </geometry>
+        <material name="Schunk/LightGrey" />
+      </visual>
+      <collision>
+        <origin xyz="0 0 0" rpy="0 0 0" />
+        <geometry>
+          <mesh filename="package://schunk_description/meshes/lwa4p_extended/arm_1_link.stl" />
+        </geometry>
+      </collision>
+    </link>
+    <!-- joint between arm_2_link and arm_3_link -->
+    <joint name="${name}_3_joint" type="revolute">
+      <origin xyz="0 0 0" rpy="-1.5708 0 0"/>
+      <parent link="${name}_2_link"/>
+      <child link="${name}_3_link"/>
+      <axis xyz="0 0 1"/>
+      <calibration rising="${arm_3_ref}"/>
+      <dynamics damping="5" />
+      <limit effort="176" velocity="2.0" lower="-6.2831853" upper="6.2831853"/>
+      <safety_controller k_position="20" k_velocity="25" soft_lower_limit="${-6.2831853 + 0.01}" soft_upper_limit="${6.2831853 - 0.01}" />
+    </joint>
+    <link name="${name}_3_link">
+      <inertial>
+        <origin xyz="0 0 0" rpy="0 0 0"/>
+        <mass value="0.1"/>
+        <inertia ixx="0.01" ixy="0" ixz="0" iyy="0.01" iyz="0" izz="0.01" />
+      </inertial>
+      <inertial>
+        <origin xyz="0 0 0" rpy="0 0 0"/>
+        <mass value="0.1"/>
+        <inertia ixx="0.01" ixy="0" ixz="0" iyy="0.01" iyz="0" izz="0.01" />
+      </inertial>
+    <visual>
+        <origin xyz="0 0 0" rpy="0 0 0" />
+        <geometry>
+          <mesh filename="package://schunk_description/meshes/lwa4p_extended/arm_2_link.stl" />
+        </geometry>
+        <material name="Schunk/LightGrey" />
+      </visual>
+      <collision>
+        <origin xyz="0 0 0" rpy="0 0 0" />
+        <geometry>
+          <mesh filename="package://schunk_description/meshes/lwa4p_extended/arm_2_link.stl" />
+        </geometry>
+      </collision>
+    </link>
+    <!-- joint between arm_3_link and arm_4_link -->
+    <joint name="${name}_4_joint" type="revolute">
+      <origin xyz="0 0 0.45360" rpy="1.5708 0 0" />
+      <parent link="${name}_3_link"/>
+      <child link="${name}_4_link"/>
+      <axis xyz="0 0 1" />
+      <calibration rising="${arm_4_ref}"/>
+      <dynamics damping="5" />
+      <limit effort="176" velocity="2.0" lower="-2.0943951" upper="2.0943951"/>
+      <safety_controller k_position="20" k_velocity="25" soft_lower_limit="${-2.0943951 + 0.01}" soft_upper_limit="${2.0943951 - 0.01}" />
+    </joint>
+    <link name="${name}_4_link">
+      <inertial>
+        <origin xyz="0 0 0" rpy="0 0 0"/>
+        <mass value="0.1"/>
+        <inertia ixx="0.01" ixy="0" ixz="0" iyy="0.01" iyz="0" izz="0.01" />
+      </inertial>
+      <visual>
+        <origin xyz="0 0 0" rpy="0 0 0" />
+        <geometry>
+          <mesh filename="package://schunk_description/meshes/lwa4p_extended/arm_3_link.stl" />
+        </geometry>
+        <material name="Schunk/LightGrey" />
+      </visual>
+      <collision>
+        <origin xyz="0 0 0" rpy="0 0 0" />
+        <geometry>
+          <mesh filename="package://schunk_description/meshes/lwa4p_extended/arm_3_link.stl" />
+        </geometry>
+      </collision>
+    </link>
+    <!-- joint between arm_4_link and arm_5_link -->
+    <joint name="${name}_5_joint" type="revolute">
+      <origin xyz="0 0 0" rpy="-1.5708 0 0" />
+      <parent link="${name}_4_link"/>
+      <child link="${name}_5_link"/>
+      <axis xyz="0 0 1" />
+      <calibration rising="${arm_5_ref}"/>
+      <dynamics damping="5" />
+      <limit effort="41.6" velocity="2.0" lower="-6.2831853" upper="6.2831853" />
+      <safety_controller k_position="20" k_velocity="25" soft_lower_limit="${-6.2831853 + 0.01}" soft_upper_limit="${6.2831853 - 0.01}" />
+    </joint>
+    <link name="${name}_5_link">
+      <inertial>
+        <origin xyz="0 0 0" rpy="0 0 0"/>
+        <mass value="0.1"/>
+        <inertia ixx="0.01" ixy="0" ixz="0" iyy="0.01" iyz="0" izz="0.01" />
+      </inertial>
+      <visual>
+        <origin xyz="0 0 0" rpy="0 0 0" />
+        <geometry>
+          <mesh filename="package://schunk_description/meshes/lwa4p_extended/arm_4_link.stl" />
+        </geometry>
+        <material name="Schunk/LightGrey" />
+      </visual>
+      <collision>
+        <origin xyz="0 0 0" rpy="0 0 0" />
+        <geometry>
+          <mesh filename="package://schunk_description/meshes/lwa4p_extended/arm_4_link.stl" />
+        </geometry>
+      </collision>
+    </link>
+    <!-- joint between arm_5_link and arm_6_link -->
+    <joint name="${name}_6_joint" type="revolute">
+      <origin xyz="0 0 0.2986" rpy="1.5708 0 0" />
+      <parent link="${name}_5_link"/>
+      <child link="${name}_6_link"/>
+      <axis xyz="0 0 1" />
+      <calibration rising="${arm_6_ref}"/>
+      <dynamics damping="5" />
+      <limit effort="20.1" velocity="2.0" lower="-2.0943951" upper="2.0943951" />
+      <safety_controller k_position="20" k_velocity="25" soft_lower_limit="${-2.0943951 + 0.01}" soft_upper_limit="${2.0943951 - 0.01}" />
+    </joint>
+    <link name="${name}_6_link">
+      <inertial>
+        <origin xyz="0 0 0" rpy="0 0 0"/>
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
File: schunk_description/urdf/pg70/pg70.gazebo.xacro (robot description, xacro)
@@ -1,20 +1,17 @@
 <?xml version="1.0"?>
-<robot xmlns:sensor="http://playerstage.sourceforge.net/gazebo/xmlschema/#sensor"
-       xmlns:controller="http://playerstage.sourceforge.net/gazebo/xmlschema/#controller"
-       xmlns:interface="http://playerstage.sourceforge.net/gazebo/xmlschema/#interface"
-       xmlns:xacro="http://ros.org/wiki/xacro">
-	<xacro:macro name="schunk_pg70_gazebo" params="name">
-		<gazebo reference="${name}_palm_link">
-			<material>Schunk/LightGrey</material>
-			<turnGravityOff>false</turnGravityOff>
-		</gazebo>
-		<gazebo reference="${name}_finger_1_link">
-			<material>Schunk/LightGrey</material>
-			<turnGravityOff>false</turnGravityOff>
-		</gazebo>
-		<gazebo reference="${name}_finger_2_link">
-			<material>Schunk/LightGrey</material>
-			<turnGravityOff>false</turnGravityOff>
-		</gazebo>
-	</xacro:macro>
+<robot xmlns:xacro="http://www.ros.org/wiki/xacro">
+  <xacro:macro name="schunk_pg70_gazebo" params="name">
+    <gazebo reference="${name}_palm_link">
+      <material>Schunk/LightGrey</material>
+      <turnGravityOff>false</turnGravityOff>
+    </gazebo>
+    <gazebo reference="${name}_finger_1_link">
+      <material>Schunk/LightGrey</material>
+      <turnGravityOff>false</turnGravityOff>
+    </gazebo>
+    <gazebo reference="${name}_finger_2_link">
+      <material>Schunk/LightGrey</material>
+      <turnGravityOff>false</turnGravityOff>
+    </gazebo>
+  </xacro:macro>
 </robot>

File: schunk_description/urdf/pg70/pg70.transmission.xacro (robot description, xacro)
@@ -1,20 +1,23 @@
 <?xml version="1.0"?>
-<robot xmlns:sensor="http://playerstage.sourceforge.net/gazebo/xmlschema/#sensor"
-       xmlns:controller="http://playerstage.sourceforge.net/gazebo/xmlschema/#controller"
-       xmlns:interface="http://playerstage.sourceforge.net/gazebo/xmlschema/#interface"
-       xmlns:xacro="http://ros.org/wiki/xacro">
-	<xacro:macro name="schunk_pg70_transmission" params="name">
-		<!-- finger1 -->
-		<transmission name="${name}_finger_trans" type="pr2_mechanism_model/SimpleTransmission">
-			<actuator name="${name}_finger_motor"/>
-			<joint name="${name}_finger_joint"/>
-			<mechanicalReduction>1</mechanicalReduction>
-		</transmission>
-		<!-- finger2 -->
-		<transmission name="${name}_finger_mimic_trans" type="pr2_mechanism_model/SimpleTransmission">
-			<actuator name="${name}_finger_mimic_motor"/>
-			<joint name="${name}_finger_mimic_joint"/>
-			<mechanicalReduction>1</mechanicalReduction>
-		</transmission>
-	</xacro:macro>
+<robot xmlns:xacro="http://www.ros.org/wiki/xacro">
+  <xacro:macro name="schunk_pg70_transmission" params="name">
+    <!-- finger1 -->
+    <transmission name="${name}_finger_trans">
+      <type>transmission_interface/SimpleTransmission</type>
+      <joint name="${name}_finger_joint"/>
+      <actuator name="${name}_finger_motor">
+        <hardwareInterface>EffortJointInterface</hardwareInterface>
+        <mechanicalReduction>1</mechanicalReduction>
+      </actuator>
+    </transmission>
+    <!-- finger2 -->
+    <transmission name="${name}_finger_mimic_trans">
+      <type>transmission_interface/SimpleTransmission</type>
+      <joint name="${name}_finger_mimic_joint"/>
+      <actuator name="${name}_finger_mimic_motor">
+        <hardwareInterface>EffortJointInterface</hardwareInterface>
+        <mechanicalReduction>1</mechanicalReduction>
+      </actuator>
+    </transmission>
+  </xacro:macro>
 </robot>
