Commit message: use inertias and physic properties from controller_tuning tests

File: schunk_description/urdf/lwa4p_extended/lwa4p_extended.gazebo.xacro (robot description, xacro)
@@ -2,38 +2,118 @@
 <robot xmlns:xacro="http://www.ros.org/wiki/xacro">
   <xacro:macro name="schunk_lwa4p_extended_gazebo" params="name">
-    <gazebo reference="${name}_0_link">
-      <material value="Schunk/LightGrey" />
-      <turnGravityOff>false</turnGravityOff>
+    <!--
+      Gazebo tags example for links
+      <gazebo reference="name">
+        <material value="Schunk/LightGrey"/>
+        <selfCollide>true</selfCollide>
+        <gravity>false</gravity>
+        <dampingFactor>1</dampingFactor>
+        <maxVel>1.0</maxVel>
+        <minDepth>0.0</minDepth>
+        <mu1>1</mu1>
+        <mu2>1</mu2>
+        <fdir1>1 0 0</fdir1>
+        <kp>1000000</kp>
+        <kd>100</kd>
+        <maxContacts>50</maxContacts>
+        <laserRetro>1</laserRetro>
+      </gazebo>
+    -->
+    <gazebo reference="${name}_base_link">
+      <material value="Schunk/LightGrey"/>
       <selfCollide>true</selfCollide>
+      <!--gravity>false</gravity-->
+<!--
+      <mu1>1.0</mu1>
+      <mu2>1.0</mu2>
+-->
     </gazebo>
     <gazebo reference="${name}_1_link">
       <material value="Schunk/LightGrey" />
-      <turnGravityOff>false</turnGravityOff>
       <selfCollide>true</selfCollide>
+      <!--gravity>false</gravity-->
+<!--
+      <mu1>1.0</mu1>
+      <mu2>1.0</mu2>
+-->
     </gazebo>
     <gazebo reference="${name}_2_link">
-      <turnGravityOff>false</turnGravityOff>
       <selfCollide>true</selfCollide>
+      <!--gravity>false</gravity-->
+<!--
+      <mu1>1.0</mu1>
+      <mu2>1.0</mu2>
+-->
     </gazebo>
     <gazebo reference="${name}_3_link">
-      <turnGravityOff>false</turnGravityOff>
       <selfCollide>true</selfCollide>
+      <!--gravity>false</gravity-->
+<!--
+      <mu1>1.0</mu1>
+      <mu2>1.0</mu2>
+-->
     </gazebo>
     <gazebo reference="${name}_4_link">
-      <turnGravityOff>false</turnGravityOff>
       <selfCollide>true</selfCollide>
+      <!--gravity>false</gravity-->
+<!--
+      <mu1>1.0</mu1>
+      <mu2>1.0</mu2>
+-->
     </gazebo>
     <gazebo reference="${name}_5_link">
-      <turnGravityOff>false</turnGravityOff>
       <selfCollide>true</selfCollide>
+      <!--gravity>false</gravity-->
+<!--
+      <mu1>1.0</mu1>
+      <mu2>1.0</mu2>
+-->
     </gazebo>
     <gazebo reference="${name}_6_link">
-      <turnGravityOff>false</turnGravityOff>
       <selfCollide>true</selfCollide>
+      <!--gravity>false</gravity-->
+<!--
+      <mu1>1.0</mu1>
+      <mu2>1.0</mu2>
+-->
     </gazebo>
     <gazebo reference="${name}_7_link">
       <material value="Schunk/LightGrey" />
-      <turnGravityOff>false</turnGravityOff>
-      <selfCollide>true</selfCollide>
+      <!--gravity>false</gravity-->
+<!--
+      <mu1>1.0</mu1>
+      <mu2>1.0</mu2>
+-->
+    </gazebo>
+    <!--
+    Gazebo tags example for joints
+    <gazebo reference="name">
+      <stopCfm>1</stopCfm>
+      <stopErp>1</stopErp>
+      <provideFeedback>1</provideFeedback>
+      <implicitSpringDamper>1</implicitSpringDamper>
+      <fudgeFactor>1</fudgeFactor>
+    </gazebo>
+    -->
+    <gazebo reference="${name}_1_joint">
+      <implicitSpringDamper>true</implicitSpringDamper>
+    </gazebo>
+    <gazebo reference="${name}_2_joint">
+      <implicitSpringDamper>true</implicitSpringDamper>
+    </gazebo>
+    <gazebo reference="${name}_3_joint">
+      <implicitSpringDamper>true</implicitSpringDamper>
+    </gazebo>
+    <gazebo reference="${name}_4_joint">
+      <implicitSpringDamper>true</implicitSpringDamper>
+    </gazebo>
+    <gazebo reference="${name}_5_joint">
+      <implicitSpringDamper>true</implicitSpringDamper>
+    </gazebo>
+    <gazebo reference="${name}_6_joint">
+      <implicitSpringDamper>true</implicitSpringDamper>
+    </gazebo>
+    <gazebo reference="${name}_7_joint">
+      <implicitSpringDamper>true</implicitSpringDamper>
     </gazebo>
   </xacro:macro>

File: schunk_description/urdf/lwa4p_extended/lwa4p_extended.transmission.xacro (robot description, xacro)
@@ -1,57 +1,9 @@
 <?xml version="1.0"?>
 <robot xmlns:xacro="http://www.ros.org/wiki/xacro">
-  <xacro:macro name="schunk_lwa4p_extended_transmission" params="name">
-    <transmission name="${name}_1_trans">
+  <xacro:macro name="schunk_lwa4p_extended_SimpleTransmission" params="jname number">
+    <transmission name="${jname}_${number}_trans">
       <type>transmission_interface/SimpleTransmission</type>
-      <joint name="${name}_1_joint"/>
-      <actuator name="${name}_1_motor">
-        <hardwareInterface>EffortJointInterface</hardwareInterface>
-        <mechanicalReduction>1</mechanicalReduction>
-      </actuator>
-    </transmission>
-    <transmission name="${name}_2_trans">
-      <type>transmission_interface/SimpleTransmission</type>
-      <joint name="${name}_2_joint"/>
-      <actuator name="${name}_2_motor">
-        <hardwareInterface>EffortJointInterface</hardwareInterface>
-        <mechanicalReduction>1</mechanicalReduction>
-      </actuator>
-    </transmission>
-    <transmission name="${name}_3_trans">
-      <type>transmission_interface/SimpleTransmission</type>
-      <joint name="${name}_3_joint"/>
-      <actuator name="${name}_3_motor">
-        <hardwareInterface>EffortJointInterface</hardwareInterface>
-        <mechanicalReduction>1</mechanicalReduction>
-      </actuator>
-    </transmission>
-    <transmission name="${name}_4_trans">
-      <type>transmission_interface/SimpleTransmission</type>
-      <joint name="${name}_4_joint"/>
-      <actuator name="${name}_4_motor">
-        <hardwareInterface>EffortJointInterface</hardwareInterface>
-        <mechanicalReduction>1</mechanicalReduction>
-      </actuator>
-    </transmission>
-    <transmission name="${name}_5_trans">
-      <type>transmission_interface/SimpleTransmission</type>
-      <joint name="${name}_5_joint"/>
-      <actuator name="${name}_5_motor">
-        <hardwareInterface>EffortJointInterface</hardwareInterface>
-        <mechanicalReduction>1</mechanicalReduction>
-      </actuator>
-    </transmission>
-    <transmission name="${name}_6_trans">
-      <type>transmission_interface/SimpleTransmission</type>
-      <joint name="${name}_6_joint"/>
-      <actuator name="${name}_6_motor">
-        <hardwareInterface>EffortJointInterface</hardwareInterface>
-        <mechanicalReduction>1</mechanicalReduction>
-      </actuator>
-    </transmission>
-    <transmission name="${name}_7_trans">
-      <type>transmission_interface/SimpleTransmission</type>
-      <joint name="${name}_7_joint"/>
-      <actuator name="${name}_7_motor">
+      <joint name="${jname}_${number}_joint"/>
+      <actuator name="${jname}_${number}_motor">
         <hardwareInterface>EffortJointInterface</hardwareInterface>
         <mechanicalReduction>1</mechanicalReduction>
@@ -59,3 +11,12 @@
     </transmission>
   </xacro:macro>
+  <xacro:macro name="schunk_lwa4p_extended_transmission" params="name">
+    <xacro:schunk_lwa4p_extended_SimpleTransmission jname="${name}" number="1"></xacro:schunk_lwa4p_extended_SimpleTransmission>
+    <xacro:schunk_lwa4p_extended_SimpleTransmission jname="${name}" number="2"></xacro:schunk_lwa4p_extended_SimpleTransmission>
+    <xacro:schunk_lwa4p_extended_SimpleTransmission jname="${name}" number="3"></xacro:schunk_lwa4p_extended_SimpleTransmission>
+    <xacro:schunk_lwa4p_extended_SimpleTransmission jname="${name}" number="4"></xacro:schunk_lwa4p_extended_SimpleTransmission>
+    <xacro:schunk_lwa4p_extended_SimpleTransmission jname="${name}" number="5"></xacro:schunk_lwa4p_extended_SimpleTransmission>
+    <xacro:schunk_lwa4p_extended_SimpleTransmission jname="${name}" number="6"></xacro:schunk_lwa4p_extended_SimpleTransmission>
+    <xacro:schunk_lwa4p_extended_SimpleTransmission jname="${name}" number="7"></xacro:schunk_lwa4p_extended_SimpleTransmission>
+  </xacro:macro>
 </robot>

File: schunk_description/urdf/lwa4p_extended/lwa4p_extended.urdf.xacro (robot description, xacro)
@@ -11,19 +11,29 @@
     </joint>
     <link name="${name}_base_link">
-      <inertial>
-        <origin xyz="0 0 0" rpy="0 0 0"/>
-        <mass value="0.1"/>
-        <inertia ixx="0.01" ixy="0" ixz="0" iyy="0.01" iyz="0" izz="0.01" />
-      </inertial>
+      <xacro:cylinder_inertial radius="0.056" length="0.134" mass="2.0">
+        <origin xyz="0 0 ${0.134/2}" rpy="0 0 0" />
+      </xacro:cylinder_inertial>
+      <visual>
+        <origin xyz="0 0 0" rpy="0 0 0" />
+        <geometry>
+          <mesh filename="package://schunk_description/meshes/lwa4p_extended/arm_base_link.stl" />
+        </geometry>
+      </visual>
+      <collision>
+        <origin xyz="0 0 0" rpy="0 0 0" />
+        <geometry>
+          <mesh filename="package://schunk_description/meshes/lwa4p_extended/arm_base_link.stl" />
+        </geometry>
+      </collision>
     </link>
     <!-- joint between arm_base_link and arm_1_link -->
     <joint name="${name}_1_joint" type="revolute" >
-      <origin xyz="0 0 0" rpy="0 0 0" />
+      <origin xyz="0 0 ${0.134+0.005}" rpy="0 0 0" />
       <parent link="${name}_base_link" />
       <child link="${name}_1_link" />
       <axis xyz="0 0 1"/>
       <calibration rising="${arm_1_ref}"/>
-      <dynamics damping="10" />
-      <limit effort="370" velocity="2.0" lower="-6.2831853" upper="6.2831853"/>
+      <dynamics damping="0" friction="0"/>
+      <limit effort="81.5" velocity="0.42" lower="-6.2831853" upper="6.2831853"/>
       <safety_controller k_position="20" k_velocity="50" soft_lower_limit="${-6.2831853 + 0.01}" soft_upper_limit="${6.2831853 - 0.01}" />
     </joint>
@@ -54,13 +64,13 @@
       <axis xyz="0 0 1"/>
       <calibration rising="${arm_2_ref}"/>
-      <dynamics damping="10" />
-      <limit effort="370" velocity="2.0" lower="-2.0943951" upper="2.0943951"/>
+      <dynamics damping="0" friction="0"/>
+      <limit effort="48" velocity="1.2566" lower="-2.0943951" upper="2.0943951"/>
       <safety_controller k_position="20" k_velocity="50" soft_lower_limit="${-2.0943 + 0.01}" soft_upper_limit="${2.0943 - 0.01}" />
     </joint>
     <link name="${name}_2_link">
       <inertial>
-        <origin xyz="0 0 0" rpy="0 0 0"/>
-        <mass value="0.1"/>
-        <inertia ixx="0.01" ixy="0" ixz="0" iyy="0.01" iyz="0" izz="0.01" />
+        <origin xyz="0 0.018 0.018" rpy="0 0 0"/>
+        <mass value="3.9"/>
+        <inertia ixx="0.009780" ixy="0.0" ixz="0.0" iyy="0.013300" iyz="0.0" izz="0.009780" />
       </inertial>
       <visual>
@@ -84,9 +94,14 @@
       <axis xyz="0 0 1"/>
       <calibration rising="${arm_3_ref}"/>
-      <dynamics damping="5" />
-      <limit effort="176" velocity="2.0" lower="-6.2831853" upper="6.2831853"/>
+      <dynamics damping="0" friction="0"/>
+      <limit effort="48" velocity="1.2566" lower="-6.2831853" upper="6.2831853"/>
       <safety_controller k_position="20" k_velocity="25" soft_lower_limit="${-6.2831853 + 0.01}" soft_upper_limit="${6.2831853 - 0.01}" />
     </joint>
     <link name="${name}_3_link">
+      <inertial>
+        <origin xyz="0.0 0.06247 0.23425" rpy="0 0 0"/>
+        <mass value="1.94533"/>
+        <inertia ixx="0.0344" ixy="0.0" ixz="0.0077" iyy="0.0362" iyz="0.0" izz="0.0052" />
+      </inertial>
       <inertial>
         <origin xyz="0 0 0" rpy="0 0 0"/>
@@ -94,10 +109,5 @@
         <inertia ixx="0.01" ixy="0" ixz="0" iyy="0.01" iyz="0" izz="0.01" />
       </inertial>
-      <inertial>
-        <origin xyz="0 0 0" rpy="0 0 0"/>
-        <mass value="0.1"/>
-        <inertia ixx="0.01" ixy="0" ixz="0" iyy="0.01" iyz="0" izz="0.01" />
-      </inertial>
-      <visual>
+    <visual>
         <origin xyz="0 0 0" rpy="0 0 0" />
         <geometry>
@@ -119,13 +129,13 @@
       <axis xyz="0 0 1" />
       <calibration rising="${arm_4_ref}"/>
-      <dynamics damping="5" />
-      <limit effort="176" velocity="2.0" lower="-2.0943951" upper="2.0943951"/>
+      <dynamics damping="0" friction="0"/>
+      <limit effort="48" velocity="1.2566" lower="-2.0943951" upper="2.0943951"/>
       <safety_controller k_position="20" k_velocity="25" soft_lower_limit="${-2.0943951 + 0.01}" soft_upper_limit="${2.0943951 - 0.01}" />
     </joint>
     <link name="${name}_4_link">
       <inertial>
-        <origin xyz="0 0 0" rpy="0 0 0"/>
-        <mass value="0.1"/>
-        <inertia ixx="0.01" ixy="0" ixz="0" iyy="0.01" iyz="0" izz="0.01" />
+        <origin xyz="0 0.018 -0.018" rpy="0 0 0"/>
+        <mass value="3.9"/>
+        <inertia ixx="0.009780" ixy="0.0" ixz="0.0" iyy="0.013300" iyz="0.0" izz="0.009780" />
       </inertial>
       <visual>
@@ -149,13 +159,13 @@
       <axis xyz="0 0 1" />
       <calibration rising="${arm_5_ref}"/>
-      <dynamics damping="5" />
-      <limit effort="41.6" velocity="2.0" lower="-6.2831853" upper="6.2831853" />
+      <dynamics damping="0" friction="0"/>
+      <limit effort="48" velocity="1.2566" lower="-6.2831853" upper="6.2831853" />
       <safety_controller k_position="20" k_velocity="25" soft_lower_limit="${-6.2831853 + 0.01}" soft_upper_limit="${6.2831853 - 0.01}" />
     </joint>
     <link name="${name}_5_link">
       <inertial>
-        <origin xyz="0 0 0" rpy="0 0 0"/>
-        <mass value="0.1"/>
-        <inertia ixx="0.01" ixy="0" ixz="0" iyy="0.01" iyz="0" izz="0.01" />
+        <origin xyz="0.0 0.04175 0.17026" rpy="0 0 0"/>
+        <mass value="1.3297"/>
+        <inertia ixx="0.01" ixy="0.0" ixz="-0.0031" iyy="0.0111" iyz="0.0" izz="0.0031" />
       </inertial>
       <visual>
@@ -179,13 +189,13 @@
       <axis xyz="0 0 1" />
       <calibration rising="${arm_6_ref}"/>
-      <dynamics damping="5" />
-      <limit effort="20.1" velocity="2.0" lower="-2.0943951" upper="2.0943951" />
+      <dynamics damping="0" friction="0"/>
+      <limit effort="15" velocity="1.2566" lower="-2.0943951" upper="2.0943951" />
       <safety_controller k_position="20" k_velocity="25" soft_lower_limit="${-2.0943951 + 0.01}" soft_upper_limit="${2.0943951 - 0.01}" />
     </joint>
     <link name="${name}_6_link">
       <inertial>
-        <origin xyz="0 0 0" rpy="0 0 0"/>
-        <mass value="0.1"/>
-        <inertia ixx="0.01" ixy="0" ixz="0" iyy="0.01" iyz="0" izz="0.01" />
+        <origin xyz="0 0.012 -0.012" rpy="0 0 0"/>
+        <mass value="1.9"/>
+        <inertia ixx="0.002750" ixy="0.0" ixz="0.0" iyy="0.004002" iyz="0.0" izz="0.002830" />
       </inertial>
       <visual>
@@ -209,6 +219,6 @@
       <axis xyz="0 0 1" />
       <calibration rising="${arm_7_ref}"/>
-      <dynamics damping="5" />
-      <limit effort="20.1" velocity="2.0" lower="-2.0943951" upper="2.0943951" />
+      <dynamics damping="0" friction="0"/>
+      <limit effort="15" velocity="1.2566" lower="-2.0943951" upper="2.0943951" />
       <safety_controller k_position="20" k_velocity="25" soft_lower_limit="${-2.0943951 + 0.01}" soft_upper_limit="${2.0943951 - 0.01}" />
     </joint>

Commit message: temporary modifications for easier controller tuning

File: schunk_description/urdf/lwa4p_extended/lwa4p_extended.gazebo.xacro (robot description, xacro)
@@ -96,4 +96,5 @@
     </gazebo>
     -->
+<!--
     <gazebo reference="${name}_1_joint">
       <implicitSpringDamper>true</implicitSpringDamper>
@@ -117,4 +118,5 @@
       <implicitSpringDamper>true</implicitSpringDamper>
     </gazebo>
+-->
   </xacro:macro>
 </robot>

File: schunk_description/urdf/lwa4p_extended/lwa4p_extended.transmission.xacro (robot description, xacro)
@@ -12,4 +12,6 @@
   </xacro:macro>
   <xacro:macro name="schunk_lwa4p_extended_transmission" params="name">
+    <xacro:schunk_lwa4p_extended_SimpleTransmission jname="${name}" number="2"></xacro:schunk_lwa4p_extended_SimpleTransmission>
+<!--
     <xacro:schunk_lwa4p_extended_SimpleTransmission jname="${name}" number="1"></xacro:schunk_lwa4p_extended_SimpleTransmission>
     <xacro:schunk_lwa4p_extended_SimpleTransmission jname="${name}" number="2"></xacro:schunk_lwa4p_extended_SimpleTransmission>
@@ -19,4 +21,5 @@
     <xacro:schunk_lwa4p_extended_SimpleTransmission jname="${name}" number="6"></xacro:schunk_lwa4p_extended_SimpleTransmission>
     <xacro:schunk_lwa4p_extended_SimpleTransmission jname="${name}" number="7"></xacro:schunk_lwa4p_extended_SimpleTransmission>
+-->
   </xacro:macro>
 </robot>

File: schunk_description/urdf/lwa4p_extended/lwa4p_extended.urdf.xacro (robot description, xacro)
@@ -28,8 +28,9 @@
     </link>
     <!-- joint between arm_base_link and arm_1_link -->
-    <joint name="${name}_1_joint" type="revolute" >
+    <joint name="${name}_1_joint" type="fixed">
       <origin xyz="0 0 ${0.134+0.005}" rpy="0 0 0" />
       <parent link="${name}_base_link" />
       <child link="${name}_1_link" />
+<!--
       <axis xyz="0 0 1"/>
       <calibration rising="${arm_1_ref}"/>
@@ -37,4 +38,5 @@
       <limit effort="81.5" velocity="0.42" lower="-6.2831853" upper="6.2831853"/>
       <safety_controller k_position="20" k_velocity="50" soft_lower_limit="${-6.2831853 + 0.01}" soft_upper_limit="${6.2831853 - 0.01}" />
+-->
     </joint>
     <link name="${name}_1_link">
@@ -88,8 +90,9 @@
     </link>
     <!-- joint between arm_2_link and arm_3_link -->
-    <joint name="${name}_3_joint" type="revolute">
+    <joint name="${name}_3_joint" type="fixed">
       <origin xyz="0 0 0" rpy="-1.5708 0 0"/>
       <parent link="${name}_2_link"/>
       <child link="${name}_3_link"/>
+<!--
       <axis xyz="0 0 1"/>
       <calibration rising="${arm_3_ref}"/>
@@ -97,4 +100,5 @@
       <limit effort="48" velocity="1.2566" lower="-6.2831853" upper="6.2831853"/>
       <safety_controller k_position="20" k_velocity="25" soft_lower_limit="${-6.2831853 + 0.01}" soft_upper_limit="${6.2831853 - 0.01}" />
+-->
     </joint>
     <link name="${name}_3_link">
@@ -123,8 +127,9 @@
     </link>
     <!-- joint between arm_3_link and arm_4_link -->
-    <joint name="${name}_4_joint" type="revolute">
+    <joint name="${name}_4_joint" type="fixed">
       <origin xyz="0 0 0.45360" rpy="1.5708 0 0" />
       <parent link="${name}_3_link"/>
       <child link="${name}_4_link"/>
+<!--
       <axis xyz="0 0 1" />
       <calibration rising="${arm_4_ref}"/>
@@ -132,4 +137,5 @@
       <limit effort="48" velocity="1.2566" lower="-2.0943951" upper="2.0943951"/>
       <safety_controller k_position="20" k_velocity="25" soft_lower_limit="${-2.0943951 + 0.01}" soft_upper_limit="${2.0943951 - 0.01}" />
+-->
     </joint>
     <link name="${name}_4_link">
@@ -153,8 +159,9 @@
     </link>
     <!-- joint between arm_4_link and arm_5_link -->
-    <joint name="${name}_5_joint" type="revolute">
+    <joint name="${name}_5_joint" type="fixed">
       <origin xyz="0 0 0" rpy="-1.5708 0 0" />
       <parent link="${name}_4_link"/>
       <child link="${name}_5_link"/>
+<!--
       <axis xyz="0 0 1" />
       <calibration rising="${arm_5_ref}"/>
@@ -162,4 +169,5 @@
       <limit effort="48" velocity="1.2566" lower="-6.2831853" upper="6.2831853" />
       <safety_controller k_position="20" k_velocity="25" soft_lower_limit="${-6.2831853 + 0.01}" soft_upper_limit="${6.2831853 - 0.01}" />
+-->
     </joint>
     <link name="${name}_5_link">
@@ -183,8 +191,9 @@
     </link>
     <!-- joint between arm_5_link and arm_6_link -->
-    <joint name="${name}_6_joint" type="revolute">
+    <joint name="${name}_6_joint" type="fixed">
       <origin xyz="0 0 0.2986" rpy="1.5708 0 0" />
       <parent link="${name}_5_link"/>
       <child link="${name}_6_link"/>
+<!--
       <axis xyz="0 0 1" />
       <calibration rising="${arm_6_ref}"/>
@@ -192,4 +201,5 @@
       <limit effort="15" velocity="1.2566" lower="-2.0943951" upper="2.0943951" />
       <safety_controller k_position="20" k_velocity="25" soft_lower_limit="${-2.0943951 + 0.01}" soft_upper_limit="${2.0943951 - 0.01}" />
+-->
     </joint>
     <link name="${name}_6_link">
@@ -213,8 +223,9 @@
     </link>
     <!-- joint between arm_6_link and arm_7_link -->
-    <joint name="${name}_7_joint" type="revolute">
+    <joint name="${name}_7_joint" type="fixed">
       <origin xyz="0 0 0" rpy="-1.5708 0 0" />
       <parent link="${name}_6_link"/>
       <child link="${name}_7_link"/>
+<!--
       <axis xyz="0 0 1" />
       <calibration rising="${arm_7_ref}"/>
@@ -222,4 +233,5 @@
       <limit effort="15" velocity="1.2566" lower="-2.0943951" upper="2.0943951" />
       <safety_controller k_position="20" k_velocity="25" soft_lower_limit="${-2.0943951 + 0.01}" soft_upper_limit="${2.0943951 - 0.01}" />
+-->
     </joint>
     <link name="${name}_7_link">
