Commit message: cleaning up after testing

File: schunk_description/urdf/lwa4p_extended/lwa4p_extended.gazebo.xacro (robot description, xacro)
@@ -23,100 +23,28 @@
       <material value="Schunk/LightGrey"/>
       <selfCollide>true</selfCollide>
-      <!--gravity>false</gravity-->
-<!--
-      <mu1>1.0</mu1>
-      <mu2>1.0</mu2>
--->
     </gazebo>
     <gazebo reference="${name}_1_link">
       <material value="Schunk/LightGrey" />
       <selfCollide>true</selfCollide>
-      <!--gravity>false</gravity-->
-<!--
-      <mu1>1.0</mu1>
-      <mu2>1.0</mu2>
--->
     </gazebo>
     <gazebo reference="${name}_2_link">
       <selfCollide>true</selfCollide>
-      <!--gravity>false</gravity-->
-<!--
-      <mu1>1.0</mu1>
-      <mu2>1.0</mu2>
--->
     </gazebo>
     <gazebo reference="${name}_3_link">
       <selfCollide>true</selfCollide>
-      <!--gravity>false</gravity-->
-<!--
-      <mu1>1.0</mu1>
-      <mu2>1.0</mu2>
--->
     </gazebo>
     <gazebo reference="${name}_4_link">
       <selfCollide>true</selfCollide>
-      <!--gravity>false</gravity-->
-<!--
-      <mu1>1.0</mu1>
-      <mu2>1.0</mu2>
--->
     </gazebo>
     <gazebo reference="${name}_5_link">
       <selfCollide>true</selfCollide>
-      <!--gravity>false</gravity-->
-<!--
-      <mu1>1.0</mu1>
-      <mu2>1.0</mu2>
--->
     </gazebo>
     <gazebo reference="${name}_6_link">
       <selfCollide>true</selfCollide>
-      <!--gravity>false</gravity-->
-<!--
-      <mu1>1.0</mu1>
-      <mu2>1.0</mu2>
--->
     </gazebo>
     <gazebo reference="${name}_7_link">
       <material value="Schunk/LightGrey" />
-      <!--gravity>false</gravity-->
-<!--
-      <mu1>1.0</mu1>
-      <mu2>1.0</mu2>
--->
+      <selfCollide>true</selfCollide>
     </gazebo>
-    <!--
-    Gazebo tags example for joints
-    <gazebo reference="name">
-      <stopCfm>1</stopCfm>
-      <stopErp>1</stopErp>
-      <provideFeedback>1</provideFeedback>
-      <implicitSpringDamper>1</implicitSpringDamper>
-      <fudgeFactor>1</fudgeFactor>
-    </gazebo>
-    -->
-<!--
-    <gazebo reference="${name}_1_joint">
-      <implicitSpringDamper>true</implicitSpringDamper>
-    </gazebo>
-    <gazebo reference="${name}_2_joint">
-      <implicitSpringDamper>true</implicitSpringDamper>
-    </gazebo>
-    <gazebo reference="${name}_3_joint">
-      <implicitSpringDamper>true</implicitSpringDamper>
-    </gazebo>
-    <gazebo reference="${name}_4_joint">
-      <implicitSpringDamper>true</implicitSpringDamper>
-    </gazebo>
-    <gazebo reference="${name}_5_joint">
-      <implicitSpringDamper>true</implicitSpringDamper>
-    </gazebo>
-    <gazebo reference="${name}_6_joint">
-      <implicitSpringDamper>true</implicitSpringDamper>
-    </gazebo>
-    <gazebo reference="${name}_7_joint">
-      <implicitSpringDamper>true</implicitSpringDamper>
-    </gazebo>
--->
   </xacro:macro>
 </robot>

File: schunk_description/urdf/lwa4p_extended/lwa4p_extended.transmission.xacro (robot description, xacro)
@@ -12,6 +12,4 @@
   </xacro:macro>
   <xacro:macro name="schunk_lwa4p_extended_transmission" params="name">
-    <xacro:schunk_lwa4p_extended_SimpleTransmission jname="${name}" number="2"></xacro:schunk_lwa4p_extended_SimpleTransmission>
-<!--
     <xacro:schunk_lwa4p_extended_SimpleTransmission jname="${name}" number="1"></xacro:schunk_lwa4p_extended_SimpleTransmission>
     <xacro:schunk_lwa4p_extended_SimpleTransmission jname="${name}" number="2"></xacro:schunk_lwa4p_extended_SimpleTransmission>
@@ -21,5 +19,4 @@
     <xacro:schunk_lwa4p_extended_SimpleTransmission jname="${name}" number="6"></xacro:schunk_lwa4p_extended_SimpleTransmission>
     <xacro:schunk_lwa4p_extended_SimpleTransmission jname="${name}" number="7"></xacro:schunk_lwa4p_extended_SimpleTransmission>
--->
   </xacro:macro>
 </robot>

File: schunk_description/urdf/lwa4p_extended/lwa4p_extended.urdf.xacro (robot description, xacro)
@@ -29,9 +29,8 @@
     </link>
     <!-- joint between arm_base_link and arm_1_link -->
-    <joint name="${name}_1_joint" type="fixed">
+    <joint name="${name}_1_joint" type="revolute">
       <origin xyz="0 0 ${0.134+0.005}" rpy="0 0 0" />
       <parent link="${name}_base_link" />
       <child link="${name}_1_link" />
-<!--
       <axis xyz="0 0 1"/>
       <calibration rising="${arm_1_ref}"/>
@@ -39,5 +38,4 @@
       <limit effort="81.5" velocity="0.42" lower="-6.2831853" upper="6.2831853"/>
       <safety_controller k_position="20" k_velocity="50" soft_lower_limit="${-6.2831853 + 0.01}" soft_upper_limit="${6.2831853 - 0.01}" />
--->
     </joint>
     <!-- prl100 rototor + shoulder flansh -->
@@ -92,9 +90,8 @@
     </link>
     <!-- joint between arm_2_link and arm_3_link -->
-    <joint name="${name}_3_joint" type="fixed">
+    <joint name="${name}_3_joint" type="revolute">
       <origin xyz="0 0 0" rpy="-1.5708 0 0"/>
       <parent link="${name}_2_link"/>
       <child link="${name}_3_link"/>
-<!--
       <axis xyz="0 0 1"/>
       <calibration rising="${arm_3_ref}"/>
@@ -102,5 +99,4 @@
       <limit effort="48" velocity="1.2566" lower="-6.2831853" upper="6.2831853"/>
       <safety_controller k_position="20" k_velocity="25" soft_lower_limit="${-6.2831853 + 0.01}" soft_upper_limit="${6.2831853 - 0.01}" />
--->
     </joint>
     <link name="${name}_3_link">
@@ -129,9 +125,8 @@
     </link>
     <!-- joint between arm_3_link and arm_4_link -->
-    <joint name="${name}_4_joint" type="fixed">
+    <joint name="${name}_4_joint" type="revolute">
       <origin xyz="0 0 0.45360" rpy="1.5708 0 0" />
       <parent link="${name}_3_link"/>
       <child link="${name}_4_link"/>
-<!--
       <axis xyz="0 0 1" />
       <calibration rising="${arm_4_ref}"/>
@@ -139,5 +134,4 @@
       <limit effort="48" velocity="1.2566" lower="-2.0943951" upper="2.0943951"/>
       <safety_controller k_position="20" k_velocity="25" soft_lower_limit="${-2.0943951 + 0.01}" soft_upper_limit="${2.0943951 - 0.01}" />
--->
     </joint>
     <link name="${name}_4_link">
@@ -161,9 +155,8 @@
     </link>
     <!-- joint between arm_4_link and arm_5_link -->
-    <joint name="${name}_5_joint" type="fixed">
+    <joint name="${name}_5_joint" type="revolute">
       <origin xyz="0 0 0" rpy="-1.5708 0 0" />
       <parent link="${name}_4_link"/>
       <child link="${name}_5_link"/>
-<!--
       <axis xyz="0 0 1" />
       <calibration rising="${arm_5_ref}"/>
@@ -171,5 +164,4 @@
       <limit effort="48" velocity="1.2566" lower="-6.2831853" upper="6.2831853" />
       <safety_controller k_position="20" k_velocity="25" soft_lower_limit="${-6.2831853 + 0.01}" soft_upper_limit="${6.2831853 - 0.01}" />
--->
     </joint>
     <link name="${name}_5_link">
@@ -193,9 +185,8 @@
     </link>
     <!-- joint between arm_5_link and arm_6_link -->
-    <joint name="${name}_6_joint" type="fixed">
+    <joint name="${name}_6_joint" type="revolute">
       <origin xyz="0 0 0.2986" rpy="1.5708 0 0" />
       <parent link="${name}_5_link"/>
       <child link="${name}_6_link"/>
-<!--
       <axis xyz="0 0 1" />
       <calibration rising="${arm_6_ref}"/>
@@ -203,5 +194,4 @@
       <limit effort="15" velocity="1.2566" lower="-2.0943951" upper="2.0943951" />
       <safety_controller k_position="20" k_velocity="25" soft_lower_limit="${-2.0943951 + 0.01}" soft_upper_limit="${2.0943951 - 0.01}" />
--->
     </joint>
     <link name="${name}_6_link">
@@ -225,9 +215,8 @@
     </link>
     <!-- joint between arm_6_link and arm_7_link -->
-    <joint name="${name}_7_joint" type="fixed">
+    <joint name="${name}_7_joint" type="revolute">
       <origin xyz="0 0 0" rpy="-1.5708 0 0" />
       <parent link="${name}_6_link"/>
       <child link="${name}_7_link"/>
-<!--
       <axis xyz="0 0 1" />
       <calibration rising="${arm_7_ref}"/>
@@ -235,5 +224,4 @@
       <limit effort="15" velocity="1.2566" lower="-2.0943951" upper="2.0943951" />
       <safety_controller k_position="20" k_velocity="25" soft_lower_limit="${-2.0943951 + 0.01}" soft_upper_limit="${2.0943951 - 0.01}" />
--->
     </joint>
     <link name="${name}_7_link">

Commit message: use meshes with reduced vertices and reduce joint_limits for moveit_config

File: schunk_description/urdf/lwa4p_extended/lwa4p_extended.gazebo.xacro (robot description, xacro)
@@ -2,22 +2,4 @@
 <robot xmlns:xacro="http://www.ros.org/wiki/xacro">
   <xacro:macro name="schunk_lwa4p_extended_gazebo" params="name">
-    <!--
-      Gazebo tags example for links
-      <gazebo reference="name">
-        <material value="Schunk/LightGrey"/>
-        <selfCollide>true</selfCollide>
-        <gravity>false</gravity>
-        <dampingFactor>1</dampingFactor>
-        <maxVel>1.0</maxVel>
-        <minDepth>0.0</minDepth>
-        <mu1>1</mu1>
-        <mu2>1</mu2>
-        <fdir1>1 0 0</fdir1>
-        <kp>1000000</kp>
-        <kd>100</kd>
-        <maxContacts>50</maxContacts>
-        <laserRetro>1</laserRetro>
-      </gazebo>
-    -->
     <gazebo reference="${name}_base_link">
       <material value="Schunk/LightGrey"/>

File: schunk_description/urdf/lwa4p_extended/lwa4p_extended.urdf.xacro (robot description, xacro)
@@ -36,6 +36,7 @@
       <calibration rising="${arm_1_ref}"/>
       <dynamics damping="0" friction="0"/>
-      <limit effort="81.5" velocity="0.42" lower="-6.2831853" upper="6.2831853"/>
-      <safety_controller k_position="20" k_velocity="50" soft_lower_limit="${-6.2831853 + 0.01}" soft_upper_limit="${6.2831853 - 0.01}" />
+      <!--limit effort="81.5" velocity="0.42" lower="-6.2831853" upper="6.2831853"/-->
+      <limit effort="81.5" velocity="0.42" lower="-${M_PI}" upper="${M_PI}"/>
+      <safety_controller k_position="20" k_velocity="50" soft_lower_limit="${-M_PI + 0.01}" soft_upper_limit="${M_PI - 0.01}" />
     </joint>
     <!-- prl100 rototor + shoulder flansh -->
@@ -55,5 +56,5 @@
         <origin xyz="0 0 0" rpy="0 0 0" />
         <geometry>
-          <mesh filename="package://schunk_description/meshes/lwa4p_extended/arm_1_link.stl" />
+          <mesh filename="package://schunk_description/meshes/lwa4p_extended/arm_1_link_reduced.stl" />
         </geometry>
       </collision>
@@ -97,6 +98,7 @@
       <calibration rising="${arm_3_ref}"/>
       <dynamics damping="0" friction="0"/>
-      <limit effort="48" velocity="1.2566" lower="-6.2831853" upper="6.2831853"/>
-      <safety_controller k_position="20" k_velocity="25" soft_lower_limit="${-6.2831853 + 0.01}" soft_upper_limit="${6.2831853 - 0.01}" />
+      <!--limit effort="48" velocity="1.2566" lower="-6.2831853" upper="6.2831853"/-->
+      <limit effort="48" velocity="1.2566" lower="-${M_PI}" upper="${M_PI}"/>
+      <safety_controller k_position="20" k_velocity="25" soft_lower_limit="${-M_PI + 0.01}" soft_upper_limit="${M_PI - 0.01}" />
     </joint>
     <link name="${name}_3_link">
@@ -120,5 +122,5 @@
         <origin xyz="0 0 0" rpy="0 0 0" />
         <geometry>
-          <mesh filename="package://schunk_description/meshes/lwa4p_extended/arm_3_link.dae" />
+          <mesh filename="package://schunk_description/meshes/lwa4p_extended/arm_3_link_reduced.stl" />
         </geometry>
       </collision>
@@ -162,6 +164,7 @@
       <calibration rising="${arm_5_ref}"/>
       <dynamics damping="0" friction="0"/>
-      <limit effort="48" velocity="1.2566" lower="-6.2831853" upper="6.2831853" />
-      <safety_controller k_position="20" k_velocity="25" soft_lower_limit="${-6.2831853 + 0.01}" soft_upper_limit="${6.2831853 - 0.01}" />
+      <!--limit effort="48" velocity="1.2566" lower="-6.2831853" upper="6.2831853" /-->
+      <limit effort="48" velocity="1.2566" lower="-${M_PI}" upper="${M_PI}" />
+      <safety_controller k_position="20" k_velocity="25" soft_lower_limit="${-M_PI + 0.01}" soft_upper_limit="${M_PI - 0.01}" />
     </joint>
     <link name="${name}_5_link">
@@ -180,5 +183,5 @@
         <origin xyz="0 0 0" rpy="0 0 0" />
         <geometry>
-          <mesh filename="package://schunk_description/meshes/lwa4p_extended/arm_5_link.dae" />
+          <mesh filename="package://schunk_description/meshes/lwa4p_extended/arm_5_link_reduced.stl" />
         </geometry>
       </collision>

Commit message: get rid off safety_controller and gazebo tags for more intuitive testing

File: schunk_description/urdf/lwa4p_extended/lwa4p_extended.gazebo.xacro (robot description, xacro)
@@ -2,4 +2,5 @@
 <robot xmlns:xacro="http://www.ros.org/wiki/xacro">
   <xacro:macro name="schunk_lwa4p_extended_gazebo" params="name">
+<!--
     <gazebo reference="${name}_base_link">
       <gravity>true</gravity>
@@ -35,4 +36,5 @@
       <material value="Schunk/LightGrey" />
     </gazebo>
+-->
   </xacro:macro>
 </robot>

File: schunk_description/urdf/lwa4p_extended/lwa4p_extended.urdf.xacro (robot description, xacro)
@@ -38,5 +38,5 @@
       <!--limit effort="81.5" velocity="0.42" lower="-6.2831853" upper="6.2831853"/-->
       <limit effort="81.5" velocity="0.42" lower="-${M_PI}" upper="${M_PI}"/>
-      <safety_controller k_position="20" k_velocity="50" soft_lower_limit="${-M_PI + 0.01}" soft_upper_limit="${M_PI - 0.01}" />
+      <!--safety_controller k_position="20" k_velocity="50" soft_lower_limit="${-M_PI + 0.01}" soft_upper_limit="${M_PI - 0.01}" /-->
     </joint>
     <!-- prl100 rototor + shoulder flansh -->
@@ -69,5 +69,5 @@
       <dynamics damping="0" friction="0"/>
       <limit effort="48" velocity="1.2566" lower="-2.0943951" upper="2.0943951"/>
-      <safety_controller k_position="20" k_velocity="50" soft_lower_limit="${-2.0943 + 0.01}" soft_upper_limit="${2.0943 - 0.01}" />
+      <!--safety_controller k_position="20" k_velocity="50" soft_lower_limit="${-2.0943 + 0.01}" soft_upper_limit="${2.0943 - 0.01}" /-->
     </joint>
     <link name="${name}_2_link">
@@ -100,5 +100,5 @@
       <!--limit effort="48" velocity="1.2566" lower="-6.2831853" upper="6.2831853"/-->
       <limit effort="48" velocity="1.2566" lower="-${M_PI}" upper="${M_PI}"/>
-      <safety_controller k_position="20" k_velocity="25" soft_lower_limit="${-M_PI + 0.01}" soft_upper_limit="${M_PI - 0.01}" />
+      <!--safety_controller k_position="20" k_velocity="25" soft_lower_limit="${-M_PI + 0.01}" soft_upper_limit="${M_PI - 0.01}" /-->
     </joint>
     <link name="${name}_3_link">
@@ -113,5 +113,5 @@
         <inertia ixx="0.01" ixy="0" ixz="0" iyy="0.01" iyz="0" izz="0.01" />
       </inertial>
-    <visual>
+      <visual>
         <origin xyz="0 0 0" rpy="0 0 0" />
         <geometry>
@@ -135,5 +135,5 @@
       <dynamics damping="0" friction="0"/>
       <limit effort="48" velocity="1.2566" lower="-2.0943951" upper="2.0943951"/>
-      <safety_controller k_position="20" k_velocity="25" soft_lower_limit="${-2.0943951 + 0.01}" soft_upper_limit="${2.0943951 - 0.01}" />
+      <!--safety_controller k_position="20" k_velocity="25" soft_lower_limit="${-2.0943951 + 0.01}" soft_upper_limit="${2.0943951 - 0.01}" /-->
     </joint>
     <link name="${name}_4_link">
@@ -166,5 +166,5 @@
       <!--limit effort="48" velocity="1.2566" lower="-6.2831853" upper="6.2831853" /-->
       <limit effort="48" velocity="1.2566" lower="-${M_PI}" upper="${M_PI}" />
-      <safety_controller k_position="20" k_velocity="25" soft_lower_limit="${-M_PI + 0.01}" soft_upper_limit="${M_PI - 0.01}" />
+      <!--safety_controller k_position="20" k_velocity="25" soft_lower_limit="${-M_PI + 0.01}" soft_upper_limit="${M_PI - 0.01}" /-->
     </joint>
     <link name="${name}_5_link">
@@ -196,5 +196,5 @@
       <dynamics damping="0" friction="0"/>
       <limit effort="15" velocity="1.2566" lower="-2.0943951" upper="2.0943951" />
-      <safety_controller k_position="20" k_velocity="25" soft_lower_limit="${-2.0943951 + 0.01}" soft_upper_limit="${2.0943951 - 0.01}" />
+      <!--safety_controller k_position="20" k_velocity="25" soft_lower_limit="${-2.0943951 + 0.01}" soft_upper_limit="${2.0943951 - 0.01}" /-->
     </joint>
     <link name="${name}_6_link">
@@ -226,12 +226,10 @@
       <dynamics damping="0" friction="0"/>
       <limit effort="15" velocity="1.2566" lower="-2.0943951" upper="2.0943951" />
-      <safety_controller k_position="20" k_velocity="25" soft_lower_limit="${-2.0943951 + 0.01}" soft_upper_limit="${2.0943951 - 0.01}" />
+      <!--safety_controller k_position="20" k_velocity="25" soft_lower_limit="${-2.0943951 + 0.01}" soft_upper_limit="${2.0943951 - 0.01}" /-->
     </joint>
     <link name="${name}_7_link">
-      <inertial>
-        <origin xyz="0 0 0" rpy="0 0 0"/>
-        <mass value="0.1"/>
-        <inertia ixx="0.01" ixy="0" ixz="0" iyy="0.01" iyz="0" izz="0.01" />
-      </inertial>
+      <xacro:box_inertial x="0.01" y="0.01" z="0.01" mass="0.01">
+        <origin xyz="0 0 0" rpy="0 0 0" />
+      </xacro:box_inertial>
     </link>
     <!-- extensions -->

Commit message: get rid off safety_controller and gazebo tags for more intuitive testing

File: schunk_description/urdf/lwa4p_extended/lwa4p_extended.gazebo.xacro (robot description, xacro)
@@ -2,4 +2,5 @@
 <robot xmlns:xacro="http://www.ros.org/wiki/xacro">
   <xacro:macro name="schunk_lwa4p_extended_gazebo" params="name">
+<!--
     <gazebo reference="${name}_base_link">
       <material value="Schunk/LightGrey"/>
@@ -29,4 +30,5 @@
       <selfCollide>true</selfCollide>
     </gazebo>
+-->
   </xacro:macro>
 </robot>

File: schunk_description/urdf/lwa4p_extended/lwa4p_extended.urdf.xacro (robot description, xacro)
@@ -38,5 +38,5 @@
       <!--limit effort="81.5" velocity="0.42" lower="-6.2831853" upper="6.2831853"/-->
       <limit effort="81.5" velocity="0.42" lower="-${M_PI}" upper="${M_PI}"/>
-      <safety_controller k_position="20" k_velocity="50" soft_lower_limit="${-M_PI + 0.01}" soft_upper_limit="${M_PI - 0.01}" />
+      <!--safety_controller k_position="20" k_velocity="50" soft_lower_limit="${-M_PI + 0.01}" soft_upper_limit="${M_PI - 0.01}" /-->
     </joint>
     <!-- prl100 rototor + shoulder flansh -->
@@ -69,5 +69,5 @@
       <dynamics damping="0" friction="0"/>
       <limit effort="48" velocity="1.2566" lower="-2.0943951" upper="2.0943951"/>
-      <safety_controller k_position="20" k_velocity="50" soft_lower_limit="${-2.0943 + 0.01}" soft_upper_limit="${2.0943 - 0.01}" />
+      <!--safety_controller k_position="20" k_velocity="50" soft_lower_limit="${-2.0943 + 0.01}" soft_upper_limit="${2.0943 - 0.01}" /-->
     </joint>
     <link name="${name}_2_link">
@@ -100,5 +100,5 @@
       <!--limit effort="48" velocity="1.2566" lower="-6.2831853" upper="6.2831853"/-->
       <limit effort="48" velocity="1.2566" lower="-${M_PI}" upper="${M_PI}"/>
-      <safety_controller k_position="20" k_velocity="25" soft_lower_limit="${-M_PI + 0.01}" soft_upper_limit="${M_PI - 0.01}" />
+      <!--safety_controller k_position="20" k_velocity="25" soft_lower_limit="${-M_PI + 0.01}" soft_upper_limit="${M_PI - 0.01}" /-->
     </joint>
     <link name="${name}_3_link">
@@ -113,5 +113,5 @@
         <inertia ixx="0.01" ixy="0" ixz="0" iyy="0.01" iyz="0" izz="0.01" />
       </inertial>
-    <visual>
+      <visual>
         <origin xyz="0 0 0" rpy="0 0 0" />
         <geometry>
@@ -135,5 +135,5 @@
       <dynamics damping="0" friction="0"/>
       <limit effort="48" velocity="1.2566" lower="-2.0943951" upper="2.0943951"/>
-      <safety_controller k_position="20" k_velocity="25" soft_lower_limit="${-2.0943951 + 0.01}" soft_upper_limit="${2.0943951 - 0.01}" />
+      <!--safety_controller k_position="20" k_velocity="25" soft_lower_limit="${-2.0943951 + 0.01}" soft_upper_limit="${2.0943951 - 0.01}" /-->
     </joint>
     <link name="${name}_4_link">
@@ -166,5 +166,5 @@
       <!--limit effort="48" velocity="1.2566" lower="-6.2831853" upper="6.2831853" /-->
       <limit effort="48" velocity="1.2566" lower="-${M_PI}" upper="${M_PI}" />
-      <safety_controller k_position="20" k_velocity="25" soft_lower_limit="${-M_PI + 0.01}" soft_upper_limit="${M_PI - 0.01}" />
+      <!--safety_controller k_position="20" k_velocity="25" soft_lower_limit="${-M_PI + 0.01}" soft_upper_limit="${M_PI - 0.01}" /-->
     </joint>
     <link name="${name}_5_link">
@@ -196,5 +196,5 @@
       <dynamics damping="0" friction="0"/>
       <limit effort="15" velocity="1.2566" lower="-2.0943951" upper="2.0943951" />
-      <safety_controller k_position="20" k_velocity="25" soft_lower_limit="${-2.0943951 + 0.01}" soft_upper_limit="${2.0943951 - 0.01}" />
+      <!--safety_controller k_position="20" k_velocity="25" soft_lower_limit="${-2.0943951 + 0.01}" soft_upper_limit="${2.0943951 - 0.01}" /-->
     </joint>
     <link name="${name}_6_link">
@@ -226,12 +226,10 @@
       <dynamics damping="0" friction="0"/>
       <limit effort="15" velocity="1.2566" lower="-2.0943951" upper="2.0943951" />
-      <safety_controller k_position="20" k_velocity="25" soft_lower_limit="${-2.0943951 + 0.01}" soft_upper_limit="${2.0943951 - 0.01}" />
+      <!--safety_controller k_position="20" k_velocity="25" soft_lower_limit="${-2.0943951 + 0.01}" soft_upper_limit="${2.0943951 - 0.01}" /-->
     </joint>
     <link name="${name}_7_link">
-      <inertial>
-        <origin xyz="0 0 0" rpy="0 0 0"/>
-        <mass value="0.1"/>
-        <inertia ixx="0.01" ixy="0" ixz="0" iyy="0.01" iyz="0" izz="0.01" />
-      </inertial>
+      <xacro:box_inertial x="0.01" y="0.01" z="0.01" mass="0.01">
+        <origin xyz="0 0 0" rpy="0 0 0" />
+      </xacro:box_inertial>
     </link>
     <!-- extensions -->

Commit message: Coloured mesh files

File: schunk_description/urdf/lwa4p_extended/lwa4p_extended.gazebo.xacro (robot description, xacro)
@@ -3,10 +3,8 @@
   <xacro:macro name="schunk_lwa4p_extended_gazebo" params="name">
     <gazebo reference="${name}_0_link">
-      <material value="Schunk/LightGrey" />
       <turnGravityOff>false</turnGravityOff>
       <selfCollide>true</selfCollide>
     </gazebo>
     <gazebo reference="${name}_1_link">
-      <material value="Schunk/LightGrey" />
       <turnGravityOff>false</turnGravityOff>
       <selfCollide>true</selfCollide>

File: schunk_description/urdf/lwa4p_extended/lwa4p_extended.urdf.xacro (robot description, xacro)
@@ -37,11 +37,11 @@
         <origin xyz="0 0 0" rpy="0 0 0" />
         <geometry>
-          <mesh filename="package://schunk_description/meshes/lwa4p_extended/arm_1_link.stl" />
-        </geometry>
-      </visual>
-      <collision>
-        <origin xyz="0 0 0" rpy="0 0 0" />
-        <geometry>
-          <mesh filename="package://schunk_description/meshes/lwa4p_extended/arm_1_link.stl" />
+          <mesh filename="package://schunk_description/meshes/lwa4p_extended/arm_1_link.dae" />
+        </geometry>
+      </visual>
+      <collision>
+        <origin xyz="0 0 0" rpy="0 0 0" />
+        <geometry>
+          <mesh filename="package://schunk_description/meshes/lwa4p_extended/arm_1_link.dae" />
         </geometry>
       </collision>
