Commit message: Added calibration arm_1_calibrationg_rising

File: schunk_description/urdf/lwa4p_extended/lwa4p_extended.urdf.xacro (robot description, xacro)
@@ -6,5 +6,5 @@
 	<include filename="$(find schunk_description)/urdf/lwa4p_extended/lwa4p_extended.gazebo.xacro" />
 	<include filename="$(find schunk_description)/urdf/lwa4p_extended/lwa4p_extended.transmission.xacro" />
-	<xacro:macro name="schunk_lwa4p_extended" params="parent name *origin arm_2_ref arm_3_ref arm_4_ref arm_5_ref arm_6_ref arm_7_ref arm_8_ref">
+	<xacro:macro name="schunk_lwa4p_extended" params="parent name *origin arm_1_ref arm_2_ref arm_3_ref arm_4_ref arm_5_ref arm_6_ref arm_7_ref">
 		<!-- joint between base_link and lwa4p_extended_connector_link -->
 		<joint name="${name}_base_joint" type="fixed">
@@ -20,4 +20,5 @@
 			<child link="${name}_1_link" />
 			<axis xyz="0 0 1"/>
+			<calibration rising="${arm_1_ref}"/>
 			<dynamics damping="10" />
 			<limit effort="370" velocity="2.0" lower="-6.2831853" upper="6.2831853"/>
@@ -27,5 +28,5 @@
 		<!-- joint between arm_1_link and arm_2_link -->
 		<joint name="${name}_2_joint" type="revolute">
-			<origin xyz="0 0 0" rpy="1.5708 0 0"/> <!--z=91,5+?-->
+			<origin xyz="0 0 0.0915" rpy="1.5708 0 0"/>
 			<parent link="${name}_1_link"/>
 			<child link="${name}_2_link"/>

Commit message: Add inercia paraters in urdf

File: schunk_description/urdf/lwa4p_extended/lwa4p_extended.urdf.xacro (robot description, xacro)
@@ -13,5 +13,11 @@
 			<child link="${name}_base_link"/>
 		</joint>
-		<link name="${name}_base_link"/>
+		<link name="${name}_base_link">
+			<inertial>
+				<origin xyz="0 0 0" rpy="0 0 0"/>
+				<mass value="0.1"/>
+				<inertia ixx="0.01" ixy="0" ixz="0" iyy="0.01" iyz="0" izz="0.01" />
+			</inertial>
+		</link>
 		<!-- joint between arm_base_link and arm_1_link -->
 		<joint name="${name}_1_joint" type="revolute" >
@@ -25,5 +31,11 @@
 			<safety_controller k_position="20" k_velocity="50" soft_lower_limit="${-6.2831853 + 0.01}" soft_upper_limit="${6.2831853 - 0.01}" />
 		</joint>
-		<link name="${name}_1_link"/>
+		<link name="${name}_1_link">
+			<inertial>
+				<origin xyz="0 0 0" rpy="0 0 0"/>
+				<mass value="0.1"/>
+				<inertia ixx="0.01" ixy="0" ixz="0" iyy="0.01" iyz="0" izz="0.01" />
+			</inertial>
+		</link>
 		<!-- joint between arm_1_link and arm_2_link -->
 		<joint name="${name}_2_joint" type="revolute">
@@ -37,5 +49,24 @@
 			<safety_controller k_position="20" k_velocity="50" soft_lower_limit="${-2.0943 + 0.01}" soft_upper_limit="${2.0943 - 0.01}" />
 		</joint>
-		<link name="${name}_2_link"/>
+		<link name="${name}_2_link">
+			<inertial>
+				<origin xyz="0 0 0" rpy="0 0 0"/>
+				<mass value="0.1"/>
+				<inertia ixx="0.01" ixy="0" ixz="0" iyy="0.01" iyz="0" izz="0.01" />
+			</inertial>
+		<visual>
+				<origin xyz="0 0 0" rpy="0 0 0" />
+				<geometry>
+					<mesh filename="package://schunk_description/meshes/lwa4p_extended/arm_1_link.stl" />
+				</geometry>
+				<material name="Schunk/Blue" />
+			</visual>
+			<collision>
+				<origin xyz="0 0 0" rpy="0 0 0" />
+				<geometry>
+					<mesh filename="package://schunk_description/meshes/lwa4p_extended/arm_1_link.stl" />
+				</geometry>
+			</collision>
+		</link>
 		<!-- joint between arm_2_link and arm_3_link -->
 		<joint name="${name}_3_joint" type="revolute">
@@ -49,5 +80,11 @@
 			<safety_controller k_position="20" k_velocity="25" soft_lower_limit="${-6.2831853 + 0.01}" soft_upper_limit="${6.2831853 - 0.01}" />
 		</joint>
-		<link name="${name}_3_link"/>
+		<link name="${name}_3_link">
+			<inertial>
+				<origin xyz="0 0 0" rpy="0 0 0"/>
+				<mass value="0.1"/>
+				<inertia ixx="0.01" ixy="0" ixz="0" iyy="0.01" iyz="0" izz="0.01" />
+			</inertial>
+		</link>
 		<!-- joint between arm_3_link and arm_4_link -->
 		<joint name="${name}_4_joint" type="revolute">
@@ -61,5 +98,11 @@
 			<safety_controller k_position="20" k_velocity="25" soft_lower_limit="${-2.0943951 + 0.01}" soft_upper_limit="${2.0943951 - 0.01}" />
 		</joint>
-		<link name="${name}_4_link"/>
+		<link name="${name}_4_link">
+			<inertial>
+				<origin xyz="0 0 0" rpy="0 0 0"/>
+				<mass value="0.1"/>
+				<inertia ixx="0.01" ixy="0" ixz="0" iyy="0.01" iyz="0" izz="0.01" />
+			</inertial>
+		</link>
 		<!-- joint between arm_4_link and arm_5_link -->
 		<joint name="${name}_5_joint" type="revolute">
@@ -73,5 +116,11 @@
 			<safety_controller k_position="20" k_velocity="25" soft_lower_limit="${-6.2831853 + 0.01}" soft_upper_limit="${6.2831853 - 0.01}" />
 		</joint>
-		<link name="${name}_5_link"/>
+		<link name="${name}_5_link">
+			<inertial>
+				<origin xyz="0 0 0" rpy="0 0 0"/>
+				<mass value="0.1"/>
+				<inertia ixx="0.01" ixy="0" ixz="0" iyy="0.01" iyz="0" izz="0.01" />
+			</inertial>
+		</link>
 		<!-- joint between arm_5_link and arm_6_link -->
 		<joint name="${name}_6_joint" type="revolute">
@@ -85,5 +134,11 @@
 			<safety_controller k_position="20" k_velocity="25" soft_lower_limit="${-2.0943951 + 0.01}" soft_upper_limit="${2.0943951 - 0.01}" />
 		</joint>
-		<link name="${name}_6_link"/>
+		<link name="${name}_6_link">
+			<inertial>
+				<origin xyz="0 0 0" rpy="0 0 0"/>
+				<mass value="0.1"/>
+				<inertia ixx="0.01" ixy="0" ixz="0" iyy="0.01" iyz="0" izz="0.01" />
+			</inertial>
+		</link>
 		<!-- joint between arm_6_link and arm_7_link -->
 		<joint name="${name}_7_joint" type="revolute">
@@ -97,5 +152,11 @@
 			<safety_controller k_position="20" k_velocity="25" soft_lower_limit="${-2.0943951 + 0.01}" soft_upper_limit="${2.0943951 - 0.01}" />
 		</joint>
-		<link name="${name}_7_link"/>
+		<link name="${name}_7_link">
+			<inertial>
+				<origin xyz="0 0 0" rpy="0 0 0"/>
+				<mass value="0.1"/>
+				<inertia ixx="0.01" ixy="0" ixz="0" iyy="0.01" iyz="0" izz="0.01" />
+			</inertial>
+		</link>
 		<!-- extensions -->
 		<xacro:schunk_lwa4p_extended_gazebo name="${name}" />

Commit message: New inertia and mass values

File: schunk_description/urdf/lwa4p_extended/lwa4p_extended.urdf.xacro (robot description, xacro)
@@ -16,6 +16,6 @@
 			<inertial>
 				<origin xyz="0 0 0" rpy="0 0 0"/>
-				<mass value="0.1"/>
-				<inertia ixx="0.01" ixy="0" ixz="0" iyy="0.01" iyz="0" izz="0.01" />
+				<mass value="1.68311"/>    <!--TODO!-->
+				<inertia ixx="0.03" ixy="0" ixz="0" iyy="0.03" iyz="0" izz="0.03" />
 			</inertial>
 		</link>
@@ -34,5 +34,5 @@
 			<inertial>
 				<origin xyz="0 0 0" rpy="0 0 0"/>
-				<mass value="0.1"/>
+				<mass value="0.29364"/>
 				<inertia ixx="0.01" ixy="0" ixz="0" iyy="0.01" iyz="0" izz="0.01" />
 			</inertial>
@@ -52,6 +52,6 @@
 			<inertial>
 				<origin xyz="0 0 0" rpy="0 0 0"/>
-				<mass value="0.1"/>
-				<inertia ixx="0.01" ixy="0" ixz="0" iyy="0.01" iyz="0" izz="0.01" />
+				<mass value="1.68311"/>
+				<inertia ixx="0.03" ixy="0" ixz="0" iyy="0.03" iyz="0" izz="0.03" />
 			</inertial>
 		<visual>
@@ -83,6 +83,6 @@
 			<inertial>
 				<origin xyz="0 0 0" rpy="0 0 0"/>
-				<mass value="0.1"/>
-				<inertia ixx="0.01" ixy="0" ixz="0" iyy="0.01" iyz="0" izz="0.01" />
+				<mass value="2.1"/>
+				<inertia ixx="0.03" ixy="0" ixz="0" iyy="0.03" iyz="0" izz="0.03" />
 			</inertial>
 			<inertial>
@@ -119,6 +119,6 @@
 			<inertial>
 				<origin xyz="0 0 0" rpy="0 0 0"/>
-				<mass value="0.1"/>
-				<inertia ixx="0.01" ixy="0" ixz="0" iyy="0.01" iyz="0" izz="0.01" />
+				<mass value="1.68311"/>
+				<inertia ixx="0.03" ixy="0" ixz="0" iyy="0.03" iyz="0" izz="0.03" />
 			</inertial>
 			<visual>
@@ -150,6 +150,6 @@
 			<inertial>
 				<origin xyz="0 0 0" rpy="0 0 0"/>
-				<mass value="0.1"/>
-				<inertia ixx="0.01" ixy="0" ixz="0" iyy="0.01" iyz="0" izz="0.01" />
+				<mass value="0.807"/>
+				<inertia ixx="0.03" ixy="0" ixz="0" iyy="0.03" iyz="0" izz="0.03" />
 			</inertial>
 			<visual>
@@ -181,6 +181,6 @@
 			<inertial>
 				<origin xyz="0 0 0" rpy="0 0 0"/>
-				<mass value="0.1"/>
-				<inertia ixx="0.01" ixy="0" ixz="0" iyy="0.01" iyz="0" izz="0.01" />
+				<mass value="0.807"/>
+				<inertia ixx="0.03" ixy="0" ixz="0" iyy="0.03" iyz="0" izz="0.03" />
 			</inertial>
 			<visual>
@@ -211,6 +211,5 @@
 		<link name="${name}_7_link">
 			<inertial>
-				<origin xyz="0 0 0" rpy="0 0 0"/>
-				<mass value="0.1"/>
+				<mass value="0.819"/>
 				<inertia ixx="0.01" ixy="0" ixz="0" iyy="0.01" iyz="0" izz="0.01" />
 			</inertial>

Commit message: Renamed links and added shoulder model

File: schunk_description/urdf/lwa4p_extended/lwa4p_extended.urdf.xacro (robot description, xacro)
@@ -34,4 +34,16 @@
         <inertia ixx="0.01" ixy="0" ixz="0" iyy="0.01" iyz="0" izz="0.01" />
       </inertial>
+      <visual>
+        <origin xyz="0 0 0" rpy="0 0 0" />
+        <geometry>
+          <mesh filename="package://schunk_description/meshes/lwa4p_extended/arm_1_link.stl" />
+        </geometry>
+      </visual>
+      <collision>
+        <origin xyz="0 0 0" rpy="0 0 0" />
+        <geometry>
+          <mesh filename="package://schunk_description/meshes/lwa4p_extended/arm_1_link.stl" />
+        </geometry>
+      </collision>
     </link>
     <!-- joint between arm_1_link and arm_2_link -->
@@ -52,14 +64,14 @@
         <inertia ixx="0.01" ixy="0" ixz="0" iyy="0.01" iyz="0" izz="0.01" />
       </inertial>
-    <visual>
-        <origin xyz="0 0 0" rpy="0 0 0" />
-        <geometry>
-          <mesh filename="package://schunk_description/meshes/lwa4p_extended/arm_1_link.dae" />
-        </geometry>
-      </visual>
-      <collision>
-        <origin xyz="0 0 0" rpy="0 0 0" />
-        <geometry>
-          <mesh filename="package://schunk_description/meshes/lwa4p_extended/arm_1_link.dae" />
+      <visual>
+        <origin xyz="0 0 0" rpy="0 0 0" />
+        <geometry>
+          <mesh filename="package://schunk_description/meshes/lwa4p_extended/arm_2_link.dae" />
+        </geometry>
+      </visual>
+      <collision>
+        <origin xyz="0 0 0" rpy="0 0 0" />
+        <geometry>
+          <mesh filename="package://schunk_description/meshes/lwa4p_extended/arm_2_link.dae" />
         </geometry>
       </collision>
@@ -87,14 +99,14 @@
         <inertia ixx="0.01" ixy="0" ixz="0" iyy="0.01" iyz="0" izz="0.01" />
       </inertial>
-    <visual>
-        <origin xyz="0 0 0" rpy="0 0 0" />
-        <geometry>
-          <mesh filename="package://schunk_description/meshes/lwa4p_extended/arm_2_link.dae" />
-        </geometry>
-      </visual>
-      <collision>
-        <origin xyz="0 0 0" rpy="0 0 0" />
-        <geometry>
-          <mesh filename="package://schunk_description/meshes/lwa4p_extended/arm_2_link.dae" />
+      <visual>
+        <origin xyz="0 0 0" rpy="0 0 0" />
+        <geometry>
+          <mesh filename="package://schunk_description/meshes/lwa4p_extended/arm_3_link.dae" />
+        </geometry>
+      </visual>
+      <collision>
+        <origin xyz="0 0 0" rpy="0 0 0" />
+        <geometry>
+          <mesh filename="package://schunk_description/meshes/lwa4p_extended/arm_3_link.dae" />
         </geometry>
       </collision>
@@ -120,11 +132,11 @@
         <origin xyz="0 0 0" rpy="0 0 0" />
         <geometry>
-          <mesh filename="package://schunk_description/meshes/lwa4p_extended/arm_3_link.dae" />
-        </geometry>
-      </visual>
-      <collision>
-        <origin xyz="0 0 0" rpy="0 0 0" />
-        <geometry>
-          <mesh filename="package://schunk_description/meshes/lwa4p_extended/arm_3_link.dae" />
+          <mesh filename="package://schunk_description/meshes/lwa4p_extended/arm_4_link.dae" />
+        </geometry>
+      </visual>
+      <collision>
+        <origin xyz="0 0 0" rpy="0 0 0" />
+        <geometry>
+          <mesh filename="package://schunk_description/meshes/lwa4p_extended/arm_4_link.dae" />
         </geometry>
       </collision>
@@ -150,11 +162,11 @@
         <origin xyz="0 0 0" rpy="0 0 0" />
         <geometry>
-          <mesh filename="package://schunk_description/meshes/lwa4p_extended/arm_4_link.dae" />
-        </geometry>
-      </visual>
-      <collision>
-        <origin xyz="0 0 0" rpy="0 0 0" />
-        <geometry>
-          <mesh filename="package://schunk_description/meshes/lwa4p_extended/arm_4_link.dae" />
+          <mesh filename="package://schunk_description/meshes/lwa4p_extended/arm_5_link.dae" />
+        </geometry>
+      </visual>
+      <collision>
+        <origin xyz="0 0 0" rpy="0 0 0" />
+        <geometry>
+          <mesh filename="package://schunk_description/meshes/lwa4p_extended/arm_5_link.dae" />
         </geometry>
       </collision>
@@ -180,11 +192,11 @@
         <origin xyz="0 0 0" rpy="0 0 0" />
         <geometry>
-          <mesh filename="package://schunk_description/meshes/lwa4p_extended/arm_5_link.dae" />
-        </geometry>
-      </visual>
-      <collision>
-        <origin xyz="0 0 0" rpy="0 0 0" />
-        <geometry>
-          <mesh filename="package://schunk_description/meshes/lwa4p_extended/arm_5_link.dae" />
+          <mesh filename="package://schunk_description/meshes/lwa4p_extended/arm_6_link.dae" />
+        </geometry>
+      </visual>
+      <collision>
+        <origin xyz="0 0 0" rpy="0 0 0" />
+        <geometry>
+          <mesh filename="package://schunk_description/meshes/lwa4p_extended/arm_6_link.dae" />
         </geometry>
       </collision>

Commit message: inertias for arm_1_link

File: schunk_description/urdf/lwa4p_extended/lwa4p_extended.urdf.xacro (robot description, xacro)
@@ -10,4 +10,5 @@
       <child link="${name}_base_link"/>
     </joint>
+    <!-- static part of PRL100 -->
     <link name="${name}_base_link">
       <xacro:cylinder_inertial radius="0.056" length="0.134" mass="2.0">
@@ -40,9 +41,10 @@
 -->
     </joint>
+    <!-- prl100 rototor + shoulder flansh -->
     <link name="${name}_1_link">
       <inertial>
-        <origin xyz="0 0 0" rpy="0 0 0"/>
-        <mass value="0.1"/>
-        <inertia ixx="0.01" ixy="0" ixz="0" iyy="0.01" iyz="0" izz="0.01" />
+        <origin xyz="0.0 -0.0662 -0.0473" rpy="0 0 0"/>
+        <mass value="0.8"/>
+        <inertia ixx="0.002034" ixy="0.0" ixz="0.0" iyy="0.001437" iyz="0.000784" izz="0.00161" />
       </inertial>
       <visual>

Commit message: fix center of mass

File: schunk_description/urdf/lwa4p_extended/lwa4p_extended.urdf.xacro (robot description, xacro)
@@ -73,5 +73,5 @@
     <link name="${name}_2_link">
       <inertial>
-        <origin xyz="0 0.018 0.018" rpy="0 0 0"/>
+        <origin xyz="0 0.018 -0.018" rpy="0 0 0"/>
         <mass value="3.9"/>
         <inertia ixx="0.009780" ixy="0.0" ixz="0.0" iyy="0.013300" iyz="0.0" izz="0.009780" />
@@ -230,5 +230,5 @@
     <link name="${name}_7_link">
       <xacro:box_inertial x="0.01" y="0.01" z="0.01" mass="0.01">
-        <origin xyz="0 0 0" rpy="0 0 0" />
+        <origin xyz="0 0 0.1" rpy="0 0 0" />
       </xacro:box_inertial>
     </link>

Commit message: changed inertia of link 5

File: schunk_description/urdf/lwa4p_extended/lwa4p_extended.urdf.xacro (robot description, xacro)
@@ -108,9 +108,4 @@
         <inertia ixx="0.0344" ixy="0.0" ixz="0.0077" iyy="0.0362" iyz="0.0" izz="0.0052" />
       </inertial>
-      <inertial>
-        <origin xyz="0 0 0" rpy="0 0 0"/>
-        <mass value="0.1"/>
-        <inertia ixx="0.01" ixy="0" ixz="0" iyy="0.01" iyz="0" izz="0.01" />
-      </inertial>
       <visual>
         <origin xyz="0 0 0" rpy="0 0 0" />
@@ -172,5 +167,5 @@
         <origin xyz="0.0 0.04175 0.17026" rpy="0 0 0"/>
         <mass value="1.3297"/>
-        <inertia ixx="0.01" ixy="0.0" ixz="-0.0031" iyy="0.0111" iyz="0.0" izz="0.0031" />
+        <inertia ixx="0.0058555" ixy="0.000005805" ixz="-0.0018259" iyy="0.0065955" iyz="0.000006485" izz="0.0016198" />
       </inertial>
       <visual>

Commit message: back to CAD inertia

File: schunk_description/urdf/lwa4p_extended/lwa4p_extended.urdf.xacro (robot description, xacro)
@@ -167,5 +167,5 @@
         <origin xyz="0.0 0.04175 0.17026" rpy="0 0 0"/>
         <mass value="1.3297"/>
-        <inertia ixx="0.0058555" ixy="0.000005805" ixz="-0.0018259" iyy="0.0065955" iyz="0.000006485" izz="0.0016198" />
+        <inertia ixx="0.01" ixy="0.0" ixz="-0.0031" iyy="0.0111" iyz="0.0" izz="0.0031" />
       </inertial>
       <visual>

Commit message: extend limits for axis 1

File: schunk_description/urdf/lwa4p_extended/lwa4p_extended.urdf.xacro (robot description, xacro)
@@ -39,5 +39,5 @@
       <calibration rising="${arm_1_ref}"/>
       <dynamics damping="0" friction="0"/>
-      <limit effort="81.5" velocity="0.42" lower="-${M_PI}" upper="${M_PI}"/>
+      <limit effort="81.5" velocity="0.42" lower="-${3/2*M_PI}" upper="${3/2*M_PI}"/>
       <!--safety_controller k_position="20" k_velocity="50" soft_lower_limit="${-M_PI + 0.01}" soft_upper_limit="${M_PI - 0.01}" /-->
     </joint>

Commit message: defined real limits

File: schunk_description/urdf/lwa4p_extended/lwa4p_extended.urdf.xacro (robot description, xacro)
@@ -73,5 +73,5 @@
       <calibration rising="${arm_2_ref}"/>
       <dynamics damping="0" friction="0"/>
-      <limit effort="48" velocity="1.2566" lower="-2.0943951" upper="2.0943951"/>
+      <limit effort="48" velocity="1.2566" lower="-1.92" upper="1.92"/>   <!--Theoricarl limit +/-170 , Real Limit +/- 110 (self collision)-->
       <!--safety_controller k_position="20" k_velocity="50" soft_lower_limit="${-2.0943 + 0.01}" soft_upper_limit="${2.0943 - 0.01}" /-->
     </joint>
@@ -106,5 +106,5 @@
       <calibration rising="${arm_3_ref}"/>
       <dynamics damping="0" friction="0"/>
-      <limit effort="48" velocity="1.2566" lower="-${M_PI}" upper="${M_PI}"/>
+      <limit effort="48" velocity="1.2566" lower="-2.967" upper="2.967"/>   <!--Theoricarl limit +/-170 , Real Limit +/- 170-->
       <!--safety_controller k_position="20" k_velocity="25" soft_lower_limit="${-M_PI + 0.01}" soft_upper_limit="${M_PI - 0.01}" /-->
     </joint>
@@ -139,5 +139,5 @@
       <calibration rising="${arm_4_ref}"/>
       <dynamics damping="0" friction="0"/>
-      <limit effort="48" velocity="1.2566" lower="-2.0943951" upper="2.0943951"/>
+      <limit effort="48" velocity="1.2566" lower="-2.618" upper="2.618"/>   <!--Theoricarl limit +/-170 , Real Limit +/- 150 (self collision)-->
       <!--safety_controller k_position="20" k_velocity="25" soft_lower_limit="${-2.0943951 + 0.01}" soft_upper_limit="${2.0943951 - 0.01}" /-->
     </joint>
@@ -172,5 +172,5 @@
       <calibration rising="${arm_5_ref}"/>
       <dynamics damping="0" friction="0"/>
-      <limit effort="48" velocity="1.2566" lower="-${M_PI}" upper="${M_PI}" />
+      <limit effort="48" velocity="1.2566" lower="-2.967" upper="2.967"/>   <!--Theoricarl limit +/-170 , Real Limit +/- 170-->
       <!--safety_controller k_position="20" k_velocity="25" soft_lower_limit="${-M_PI + 0.01}" soft_upper_limit="${M_PI - 0.01}" /-->
     </joint>
@@ -205,5 +205,5 @@
       <calibration rising="${arm_6_ref}"/>
       <dynamics damping="0" friction="0"/>
-      <limit effort="15" velocity="1.2566" lower="-2.0943951" upper="2.0943951" />
+      <limit effort="15" velocity="1.2566" lower="-2.443" upper="2.967"/>   <!--Theoricarl limit +/-170 , Real Limit -140/+170 (self collision)-->
       <!--safety_controller k_position="20" k_velocity="25" soft_lower_limit="${-2.0943951 + 0.01}" soft_upper_limit="${2.0943951 - 0.01}" /-->
     </joint>
@@ -238,5 +238,5 @@
       <calibration rising="${arm_7_ref}"/>
       <dynamics damping="0" friction="0"/>
-      <limit effort="15" velocity="1.2566" lower="-2.0943951" upper="2.0943951" />
+      <limit effort="15" velocity="1.2566" lower="-2.967" upper="2.967"/>   <!--Theoricarl limit +/-170 , Real Limit +/- 170-->
       <!--safety_controller k_position="20" k_velocity="25" soft_lower_limit="${-2.0943951 + 0.01}" soft_upper_limit="${2.0943951 - 0.01}" /-->
     </joint>

Commit message: defined real limits

File: schunk_description/urdf/lwa4p_extended/lwa4p_extended.urdf.xacro (robot description, xacro)
@@ -39,5 +39,5 @@
       <calibration rising="${arm_1_ref}"/>
       <dynamics damping="0" friction="0"/>
-      <limit effort="81.5" velocity="0.42" lower="-${M_PI}" upper="${M_PI}"/>
+      <limit effort="81.5" velocity="0.42" lower="-4,712" upper="4,712"/>   <!--Theoricarl limit +/-270 , Real Limit +/- 270-->
       <!--safety_controller k_position="20" k_velocity="50" soft_lower_limit="${-M_PI + 0.01}" soft_upper_limit="${M_PI - 0.01}" /-->
     </joint>

Commit message: type error

File: schunk_description/urdf/lwa4p_extended/lwa4p_extended.urdf.xacro (robot description, xacro)
@@ -39,5 +39,5 @@
       <calibration rising="${arm_1_ref}"/>
       <dynamics damping="0" friction="0"/>
-      <limit effort="81.5" velocity="0.42" lower="-4,712" upper="4,712"/>   <!--Theoricarl limit +/-270 , Real Limit +/- 270-->
+      <limit effort="81.5" velocity="0.42" lower="-4.712" upper="4.712"/>   <!--Theoricarl limit +/-270 , Real Limit +/- 270-->
       <!--safety_controller k_position="20" k_velocity="50" soft_lower_limit="${-M_PI + 0.01}" soft_upper_limit="${M_PI - 0.01}" /-->
     </joint>
