Commit message: Update lwa4p_extended.urdf.xacro
Proposing this as according to the tests on the Schunk LWA4D, the limits should be reduced from the HW limit in a range of 0.01 radians

File: schunk_description/urdf/lwa4p_extended/lwa4p_extended.urdf.xacro (robot description, xacro)
@@ -39,5 +39,5 @@
       <calibration rising="${arm_1_ref}"/>
       <dynamics damping="0" friction="0"/>
-      <limit effort="81.5" velocity="0.42" lower="-4.712" upper="4.712"/>   <!--Theoricarl limit +/-270 , Real Limit +/- 270-->
+      <limit effort="81.5" velocity="0.42" lower="-4.702" upper="4.702"/>   <!--Theoricarl limit +/-270 , Real Limit +/- 270-->
       <!--safety_controller k_position="20" k_velocity="50" soft_lower_limit="${-M_PI + 0.01}" soft_upper_limit="${M_PI - 0.01}" /-->
     </joint>
@@ -73,5 +73,5 @@
       <calibration rising="${arm_2_ref}"/>
       <dynamics damping="0" friction="0"/>
-      <limit effort="48" velocity="1.2566" lower="-1.92" upper="1.92"/>   <!--Theoricarl limit +/-170 , Real Limit +/- 110 (self collision)-->
+      <limit effort="48" velocity="1.2566" lower="-1.91" upper="1.91"/>   <!--Theoricarl limit +/-170 , Real Limit +/- 110 (self collision)-->
       <!--safety_controller k_position="20" k_velocity="50" soft_lower_limit="${-2.0943 + 0.01}" soft_upper_limit="${2.0943 - 0.01}" /-->
     </joint>
@@ -106,5 +106,5 @@
       <calibration rising="${arm_3_ref}"/>
       <dynamics damping="0" friction="0"/>
-      <limit effort="48" velocity="1.2566" lower="-2.967" upper="2.967"/>   <!--Theoricarl limit +/-170 , Real Limit +/- 170-->
+      <limit effort="48" velocity="1.2566" lower="-2.957" upper="2.957"/>   <!--Theoricarl limit +/-170 , Real Limit +/- 170-->
       <!--safety_controller k_position="20" k_velocity="25" soft_lower_limit="${-M_PI + 0.01}" soft_upper_limit="${M_PI - 0.01}" /-->
     </joint>
@@ -139,5 +139,5 @@
       <calibration rising="${arm_4_ref}"/>
       <dynamics damping="0" friction="0"/>
-      <limit effort="48" velocity="1.2566" lower="-2.618" upper="2.618"/>   <!--Theoricarl limit +/-170 , Real Limit +/- 150 (self collision)-->
+      <limit effort="48" velocity="1.2566" lower="-2.608" upper="2.608"/>   <!--Theoricarl limit +/-170 , Real Limit +/- 150 (self collision)-->
       <!--safety_controller k_position="20" k_velocity="25" soft_lower_limit="${-2.0943951 + 0.01}" soft_upper_limit="${2.0943951 - 0.01}" /-->
     </joint>
@@ -172,5 +172,5 @@
       <calibration rising="${arm_5_ref}"/>
       <dynamics damping="0" friction="0"/>
-      <limit effort="48" velocity="1.2566" lower="-2.967" upper="2.967"/>   <!--Theoricarl limit +/-170 , Real Limit +/- 170-->
+      <limit effort="48" velocity="1.2566" lower="-2.957" upper="2.957"/>   <!--Theoricarl limit +/-170 , Real Limit +/- 170-->
       <!--safety_controller k_position="20" k_velocity="25" soft_lower_limit="${-M_PI + 0.01}" soft_upper_limit="${M_PI - 0.01}" /-->
     </joint>
@@ -205,5 +205,5 @@
       <calibration rising="${arm_6_ref}"/>
       <dynamics damping="0" friction="0"/>
-      <limit effort="15" velocity="1.2566" lower="-2.443" upper="2.967"/>   <!--Theoricarl limit +/-170 , Real Limit -140/+170 (self collision)-->
+      <limit effort="15" velocity="1.2566" lower="-2.433" upper="2.957"/>   <!--Theoricarl limit +/-170 , Real Limit -140/+170 (self collision)-->
       <!--safety_controller k_position="20" k_velocity="25" soft_lower_limit="${-2.0943951 + 0.01}" soft_upper_limit="${2.0943951 - 0.01}" /-->
     </joint>
@@ -238,5 +238,5 @@
       <calibration rising="${arm_7_ref}"/>
       <dynamics damping="0" friction="0"/>
-      <limit effort="15" velocity="1.2566" lower="-2.967" upper="2.967"/>   <!--Theoricarl limit +/-170 , Real Limit +/- 170-->
+      <limit effort="15" velocity="1.2566" lower="-2.957" upper="2.957"/>   <!--Theoricarl limit +/-170 , Real Limit +/- 170-->
       <!--safety_controller k_position="20" k_velocity="25" soft_lower_limit="${-2.0943951 + 0.01}" soft_upper_limit="${2.0943951 - 0.01}" /-->
     </joint>

Commit message: Update lwa4p_extended.urdf.xacro
Velocity and Positions limits updated according to firmware settings

File: schunk_description/urdf/lwa4p_extended/lwa4p_extended.urdf.xacro (robot description, xacro)
@@ -70,5 +70,5 @@
       <calibration rising="${arm_1_ref}"/>
       <dynamics damping="0" friction="0"/>
-      <limit effort="81.5" velocity="0.42" lower="${-4.712 + safety_offset}" upper="${4.712 - safety_offset}"/>   <!--Theoretical limit +/-270 , Real Limit +/- 270-->
+      <limit effort="81.5" velocity="0.66" lower="${-4.712 + safety_offset}" upper="${4.712 - safety_offset}"/>   <!--Theoretical limit +/-270 , Real Limit +/- 270-->
       <!--safety_controller k_position="20" k_velocity="50" soft_lower_limit="${-M_PI + 0.01}" soft_upper_limit="${M_PI - 0.01}" /-->
     </joint>
@@ -104,5 +104,5 @@
       <calibration rising="${arm_2_ref}"/>
       <dynamics damping="0" friction="0"/>
-      <limit effort="48" velocity="1.2566" lower="${-1.92 + safety_offset}" upper="${1.92 - safety_offset}"/>   <!--Theoretical limit +/-170 , Real Limit +/- 110 (self collision)-->
+      <limit effort="48" velocity="1.57" lower="${-1.91 + safety_offset}" upper="${1.91 - safety_offset}"/>   <!--Theoretical limit +/-170 , Real Limit +/- 110 (self collision)-->
       <!--safety_controller k_position="20" k_velocity="50" soft_lower_limit="${-2.0943 + 0.01}" soft_upper_limit="${2.0943 - 0.01}" /-->
     </joint>
@@ -137,5 +137,5 @@
       <calibration rising="${arm_3_ref}"/>
       <dynamics damping="0" friction="0"/>
-      <limit effort="48" velocity="1.2566" lower="${-2.967 + safety_offset}" upper="${2.967 - safety_offset}"/>   <!--Theoretical limit +/-170 , Real Limit +/- 170-->
+      <limit effort="48" velocity="1.57" lower="${-2.967 + safety_offset}" upper="${2.967 - safety_offset}"/>   <!--Theoretical limit +/-170 , Real Limit +/- 170-->
       <!--safety_controller k_position="20" k_velocity="25" soft_lower_limit="${-M_PI + 0.01}" soft_upper_limit="${M_PI - 0.01}" /-->
     </joint>
@@ -170,5 +170,5 @@
       <calibration rising="${arm_4_ref}"/>
       <dynamics damping="0" friction="0"/>
-      <limit effort="48" velocity="1.2566" lower="${-2.618 + safety_offset}" upper="${2.618 - safety_offset}"/>   <!--Theoretical limit +/-170 , Real Limit +/- 150 (self collision)-->
+      <limit effort="48" velocity="1.57" lower="${-2.618 + safety_offset}" upper="${2.618 - safety_offset}"/>   <!--Theoretical limit +/-170 , Real Limit +/- 150 (self collision)-->
       <!--safety_controller k_position="20" k_velocity="25" soft_lower_limit="${-2.0943951 + 0.01}" soft_upper_limit="${2.0943951 - 0.01}" /-->
     </joint>
@@ -203,5 +203,5 @@
       <calibration rising="${arm_5_ref}"/>
       <dynamics damping="0" friction="0"/>
-      <limit effort="48" velocity="1.2566" lower="${-2.967 + safety_offset}" upper="${2.967 - safety_offset}"/>   <!--Theoretical limit +/-170 , Real Limit +/- 170-->
+      <limit effort="48" velocity="1.57" lower="${-2.967 + safety_offset}" upper="${2.967 - safety_offset}"/>   <!--Theoretical limit +/-170 , Real Limit +/- 170-->
       <!--safety_controller k_position="20" k_velocity="25" soft_lower_limit="${-M_PI + 0.01}" soft_upper_limit="${M_PI - 0.01}" /-->
     </joint>
@@ -236,5 +236,5 @@
       <calibration rising="${arm_6_ref}"/>
       <dynamics damping="0" friction="0"/>
-      <limit effort="15" velocity="1.2566" lower="${-2.443 + safety_offset}" upper="${2.967 - safety_offset}"/>   <!--Theoretical limit +/-170 , Real Limit -140/+170 (self collision)-->
+      <limit effort="15" velocity="2.09" lower="${-2.967 + safety_offset}" upper="${2.967 - safety_offset}"/>   <!--Theoretical limit +/-170 , Real Limit -140/+170 (self collision)-->
       <!--safety_controller k_position="20" k_velocity="25" soft_lower_limit="${-2.0943951 + 0.01}" soft_upper_limit="${2.0943951 - 0.01}" /-->
     </joint>
@@ -269,5 +269,5 @@
       <calibration rising="${arm_7_ref}"/>
       <dynamics damping="0" friction="0"/>
-      <limit effort="15" velocity="1.2566" lower="${-2.967 + safety_offset}" upper="${2.967 - safety_offset}"/>   <!--Theoretical limit +/-170 , Real Limit +/- 170-->
+      <limit effort="15" velocity="2.09" lower="${-3.75 + safety_offset}" upper="${2.21 - safety_offset}"/>   <!--Theoretical limit +127/-215 , Real Limit +127/-215-->
       <!--safety_controller k_position="20" k_velocity="25" soft_lower_limit="${-2.0943951 + 0.01}" soft_upper_limit="${2.0943951 - 0.01}" /-->
     </joint>
