Commit message: renamed to schunk names

File: schunk_description/urdf/lwa/lwa.gazebo.xacro (robot description, xacro)
@@ -4,5 +4,5 @@
        xmlns:interface="http://playerstage.sourceforge.net/gazebo/xmlschema/#interface"
        xmlns:xacro="http://ros.org/wiki/xacro">
-	<xacro:macro name="schunk_lwa_gazebo_v0" params="name">
+	<xacro:macro name="schunk_lwa_gazebo" params="name">
 		<gazebo reference="${name}_0_link">
 			<material value="PR2/Red" />

File: schunk_description/urdf/lwa/lwa.transmission.xacro (robot description, xacro)
@@ -4,5 +4,5 @@
        xmlns:interface="http://playerstage.sourceforge.net/gazebo/xmlschema/#interface"
        xmlns:xacro="http://ros.org/wiki/xacro">
-	<xacro:macro name="schunk_lwa_transmission_v1" params="name">
+	<xacro:macro name="schunk_lwa_transmission" params="name">
 		<transmission name="${name}_1_trans" type="pr2_mechanism_model/SimpleTransmission">
 			<actuator name="${name}_1_motor"/>

File: schunk_description/urdf/lwa/lwa.urdf.xacro (robot description, xacro)
@@ -4,7 +4,7 @@
        xmlns:interface="http://playerstage.sourceforge.net/gazebo/xmlschema/#interface"
        xmlns:xacro="http://ros.org/wiki/xacro">
-	<include filename="$(find schunk_description)/ros/urdf/arm_v1/arm.gazebo.xacro" />
-	<include filename="$(find schunk_description)/ros/urdf/arm_v1/arm.transmission.xacro" />
-	<xacro:macro name="schunk_lwa_v1" params="parent name *origin">
+	<include filename="$(find schunk_description)/urdf/lwa/lwa.gazebo.xacro" />
+	<include filename="$(find schunk_description)/urdf/lwa/lwa.transmission.xacro" />
+	<xacro:macro name="schunk_lwa" params="parent name *origin">
 		<!-- joint between base_link and arm_0_link -->
 		<joint name="${name}_0_joint" type="fixed" >
@@ -35,5 +35,5 @@
 		<!-- joint between arm_0_link and arm_1_link -->
 		<joint name="${name}_1_joint" type="revolute">
-			<origin xyz="0 0 -0.30" rpy="0 0 3.1415926"/>
+			<origin xyz="0 0 -0.250" rpy="0 0 3.1415926"/>
 			<parent link="${name}_0_link"/>
 			<child link="${name}_1_link"/>
@@ -54,12 +54,12 @@
 				<origin xyz="0 0 0" rpy="0 0 0" />
 				<geometry>
-					<mesh filename="package://schunk_description/ros/meshes/arm_v0/arm1.stl" />
-				</geometry>
-				<material name="Blue" />
-			</visual>
-			<collision>
-				<origin xyz="0 0 0" rpy="0 0 0" />
-				<geometry>
-					<mesh filename="package://schunk_description/ros/meshes/arm_v0/arm1.stlb" />
+					<mesh filename="package://schunk_description/meshes/lwa/arm1.stl" />
+				</geometry>
+				<material name="Blue" />
+			</visual>
+			<collision>
+				<origin xyz="0 0 0" rpy="0 0 0" />
+				<geometry>
+					<mesh filename="package://schunk_description/meshes/lwa/arm1.stlb" />
 				</geometry>
 			</collision>
@@ -86,12 +86,12 @@
 				<origin xyz="0 0 0" rpy="0 0 0" />
 				<geometry>
-					<mesh filename="package://schunk_description/ros/meshes/arm_v0/arm2.stl" />
-				</geometry>
-				<material name="Red" />
-			</visual>
-			<collision>
-				<origin xyz="0 0 0" rpy="0 0 0" />
-				<geometry>
-					<mesh filename="package://schunk_description/ros/meshes/arm_v0/arm2.stlb"/>
+					<mesh filename="package://schunk_description/meshes/lwa/arm2.stl" />
+				</geometry>
+				<material name="Red" />
+			</visual>
+			<collision>
+				<origin xyz="0 0 0" rpy="0 0 0" />
+				<geometry>
+					<mesh filename="package://schunk_description/meshes/lwa/arm2.stlb"/>
 				</geometry>
 			</collision>
@@ -99,5 +99,5 @@
 		<!-- joint between arm_2_link and arm_3_link -->
 		<joint name="${name}_3_joint" type="revolute">
-			<origin xyz="0 -0.328 0" rpy="-1.5708 0 0"/>
+			<origin xyz="0 -0.408 0" rpy="-1.5708 0 0"/>
 			<parent link="${name}_2_link"/>
 			<child link="${name}_3_link"/>
@@ -118,12 +118,12 @@
 				<origin xyz="0 0 0" rpy="0 0 0" />
 				<geometry>
-					<mesh filename="package://schunk_description/ros/meshes/arm_v0/arm3.stl" />
-				</geometry>
-				<material name="Blue" />
-			</visual>
-			<collision>
-				<origin xyz="0 0 0" rpy="0 0 0" />
-				<geometry>
-					<mesh filename="package://schunk_description/ros/meshes/arm_v0/arm3.stlb"/>
+					<mesh filename="package://schunk_description/meshes/lwa/arm3.stl" />
+				</geometry>
+				<material name="Blue" />
+			</visual>
+			<collision>
+				<origin xyz="0 0 0" rpy="0 0 0" />
+				<geometry>
+					<mesh filename="package://schunk_description/meshes/lwa/arm3.stlb"/>
 				</geometry>
 			</collision>
@@ -150,12 +150,12 @@
 				<origin xyz="0 0 0" rpy="0 0 0" />
 				<geometry>
-					<mesh filename="package://schunk_description/ros/meshes/arm_v0/arm4.stl" />
-				</geometry>
-				<material name="Red" />
-			</visual>
-			<collision>
-				<origin xyz="0 0 0" rpy="0 0 0" />
-				<geometry>
-					<mesh filename="package://schunk_description/ros/meshes/arm_v0/arm4.stlb"/>
+					<mesh filename="package://schunk_description/meshes/lwa/arm4.stl" />
+				</geometry>
+				<material name="Red" />
+			</visual>
+			<collision>
+				<origin xyz="0 0 0" rpy="0 0 0" />
+				<geometry>
+					<mesh filename="package://schunk_description/meshes/lwa/arm4.stlb"/>
 				</geometry>
 			</collision>
@@ -163,5 +163,5 @@
 		<!-- joint between arm_4_link and arm_5_link -->
 		<joint name="${name}_5_joint" type="revolute">
-			<origin xyz="0 -0.2765 0" rpy="-1.5708 0 0" />
+			<origin xyz="0 -0.3165 0" rpy="-1.5708 0 0" />
 			<parent link="${name}_4_link"/>
 			<child link="${name}_5_link"/>
@@ -181,12 +181,12 @@
 				<origin xyz="0 0 0" rpy="0 0 0" />
 				<geometry>
-					<mesh filename="package://schunk_description/ros/meshes/arm_v0/arm5.stl" />
-				</geometry>
-				<material name="Blue" />
-			</visual>
-			<collision>
-				<origin xyz="0 0 0" rpy="0 0 0" />
-				<geometry>
-					<mesh filename="package://schunk_description/ros/meshes/arm_v0/arm5.stlb"/>
+					<mesh filename="package://schunk_description/meshes/lwa/arm5.stl" />
+				</geometry>
+				<material name="Blue" />
+			</visual>
+			<collision>
+				<origin xyz="0 0 0" rpy="0 0 0" />
+				<geometry>
+					<mesh filename="package://schunk_description/meshes/lwa/arm5.stlb"/>
 				</geometry>
 			</collision>
@@ -212,12 +212,12 @@
 				<origin xyz="0 0 0" rpy="0 0 0" />
 				<geometry>
-					<mesh filename="package://schunk_description/ros/meshes/arm_v0/arm6.stl" />
-				</geometry>
-				<material name="Red" />
-			</visual>
-			<collision>
-				<origin xyz="0 0 0" rpy="0 0 0" />
-				<geometry>
-					<mesh filename="package://schunk_description/ros/meshes/arm_v0/arm6.stlb"/>
+					<mesh filename="package://schunk_description/meshes/lwa/arm6.stl" />
+				</geometry>
+				<material name="Red" />
+			</visual>
+			<collision>
+				<origin xyz="0 0 0" rpy="0 0 0" />
+				<geometry>
+					<mesh filename="package://schunk_description/meshes/lwa/arm6.stlb"/>
 				</geometry>
 			</collision>
@@ -225,5 +225,5 @@
 		<!-- joint between arm_6_link and arm_7_link -->
 		<joint name="${name}_7_joint" type="revolute">
-			<origin xyz="0 -0.237448 0" rpy="-1.5708 0 0" />
+			<origin xyz="0 -0.1927 0" rpy="-1.5708 0 0" />
 			<parent link="${name}_6_link"/>
 			<child link="${name}_7_link"/>
@@ -243,18 +243,18 @@
 				<origin xyz="0 0 0" rpy="0 0 0" />
 				<geometry>
-					<mesh filename="package://schunk_description/ros/meshes/arm_v0/arm7.stl" />
-				</geometry>
-				<material name="Blue" />
-			</visual>
-			<collision>
-				<origin xyz="0 0 0" rpy="0 0 0" />
-				<geometry>
-					<mesh filename="package://schunk_description/ros/meshes/arm_v0/arm7.stlb"/>
+					<mesh filename="package://schunk_description/meshes/lwa/arm7.stl" />
+				</geometry>
+				<material name="Blue" />
+			</visual>
+			<collision>
+				<origin xyz="0 0 0" rpy="0 0 0" />
+				<geometry>
+					<mesh filename="package://schunk_description/meshes/lwa/arm7.stlb"/>
 				</geometry>
 			</collision>
 		</link>
 		<!-- extensions -->
-		<xacro:schunk_lwa_gazebo_v1 name="${name}" />
-		<xacro:schunk_lwa_transmission_v1 name="${name}" />
+		<xacro:schunk_lwa_gazebo name="${name}" />
+		<xacro:schunk_lwa_transmission name="${name}" />
 	</xacro:macro>
 </robot>

File: schunk_description/urdf/lwa_extended/lwa_extended.gazebo.xacro (robot description, xacro)
@@ -4,5 +4,5 @@
        xmlns:interface="http://playerstage.sourceforge.net/gazebo/xmlschema/#interface"
        xmlns:xacro="http://ros.org/wiki/xacro">
-	<xacro:macro name="schunk_lwa_gazebo_v1" params="name">
+	<xacro:macro name="schunk_lwa_extended_gazebo" params="name">
 		<gazebo reference="${name}_0_link">
 			<material value="PR2/Red" />

File: schunk_description/urdf/lwa_extended/lwa_extended.transmission.xacro (robot description, xacro)
@@ -4,5 +4,5 @@
        xmlns:interface="http://playerstage.sourceforge.net/gazebo/xmlschema/#interface"
        xmlns:xacro="http://ros.org/wiki/xacro">
-	<xacro:macro name="schunk_lwa_transmission_v0" params="name">
+	<xacro:macro name="schunk_lwa_extended_transmission" params="name">
 		<transmission name="${name}_1_trans" type="pr2_mechanism_model/SimpleTransmission">
 			<actuator name="${name}_1_motor"/>

File: schunk_description/urdf/lwa_extended/lwa_extended.urdf.xacro (robot description, xacro)
@@ -4,7 +4,7 @@
        xmlns:interface="http://playerstage.sourceforge.net/gazebo/xmlschema/#interface"
        xmlns:xacro="http://ros.org/wiki/xacro">
-	<include filename="$(find schunk_description)/ros/urdf/arm_v0/arm.gazebo.xacro" />
-	<include filename="$(find schunk_description)/ros/urdf/arm_v0/arm.transmission.xacro" />
-	<xacro:macro name="schunk_lwa_v0" params="parent name *origin">
+	<include filename="$(find schunk_description)/urdf/lwa_extended/lwa_extended.gazebo.xacro" />
+	<include filename="$(find schunk_description)/urdf/lwa_extended/lwa_extended.transmission.xacro" />
+	<xacro:macro name="schunk_lwa_extended" params="parent name *origin">
 		<!-- joint between base_link and arm_0_link -->
 		<joint name="${name}_0_joint" type="fixed" >
@@ -35,5 +35,5 @@
 		<!-- joint between arm_0_link and arm_1_link -->
 		<joint name="${name}_1_joint" type="revolute">
-			<origin xyz="0 0 -0.250" rpy="0 0 3.1415926"/>
+			<origin xyz="0 0 -0.30" rpy="0 0 3.1415926"/>
 			<parent link="${name}_0_link"/>
 			<child link="${name}_1_link"/>
@@ -54,12 +54,12 @@
 				<origin xyz="0 0 0" rpy="0 0 0" />
 				<geometry>
-					<mesh filename="package://schunk_description/ros/meshes/arm_v0/arm1.stl" />
-				</geometry>
-				<material name="Blue" />
-			</visual>
-			<collision>
-				<origin xyz="0 0 0" rpy="0 0 0" />
-				<geometry>
-					<mesh filename="package://schunk_description/ros/meshes/arm_v0/arm1.stlb" />
+					<mesh filename="package://schunk_description/meshes/lwa/lwa1.stl" />
+				</geometry>
+				<material name="Blue" />
+			</visual>
+			<collision>
+				<origin xyz="0 0 0" rpy="0 0 0" />
+				<geometry>
+					<mesh filename="package://schunk_description/meshes/lwa/lwa1.stlb" />
 				</geometry>
 			</collision>
@@ -86,12 +86,12 @@
 				<origin xyz="0 0 0" rpy="0 0 0" />
 				<geometry>
-					<mesh filename="package://schunk_description/ros/meshes/arm_v0/arm2.stl" />
-				</geometry>
-				<material name="Red" />
-			</visual>
-			<collision>
-				<origin xyz="0 0 0" rpy="0 0 0" />
-				<geometry>
-					<mesh filename="package://schunk_description/ros/meshes/arm_v0/arm2.stlb"/>
+					<mesh filename="package://schunk_description/meshes/lwa/lwa2.stl" />
+				</geometry>
+				<material name="Red" />
+			</visual>
+			<collision>
+				<origin xyz="0 0 0" rpy="0 0 0" />
+				<geometry>
+					<mesh filename="package://schunk_description/meshes/lwa/lwa2.stlb"/>
 				</geometry>
 			</collision>
@@ -99,5 +99,5 @@
 		<!-- joint between arm_2_link and arm_3_link -->
 		<joint name="${name}_3_joint" type="revolute">
-			<origin xyz="0 -0.408 0" rpy="-1.5708 0 0"/>
+			<origin xyz="0 -0.328 0" rpy="-1.5708 0 0"/>
 			<parent link="${name}_2_link"/>
 			<child link="${name}_3_link"/>
@@ -118,12 +118,12 @@
 				<origin xyz="0 0 0" rpy="0 0 0" />
 				<geometry>
-					<mesh filename="package://schunk_description/ros/meshes/arm_v0/arm3.stl" />
-				</geometry>
-				<material name="Blue" />
-			</visual>
-			<collision>
-				<origin xyz="0 0 0" rpy="0 0 0" />
-				<geometry>
-					<mesh filename="package://schunk_description/ros/meshes/arm_v0/arm3.stlb"/>
+					<mesh filename="package://schunk_description/meshes/lwa/lwa3.stl" />
+				</geometry>
+				<material name="Blue" />
+			</visual>
+			<collision>
+				<origin xyz="0 0 0" rpy="0 0 0" />
+				<geometry>
+					<mesh filename="package://schunk_description/meshes/lwa/lwa3.stlb"/>
 				</geometry>
 			</collision>
@@ -150,12 +150,12 @@
 				<origin xyz="0 0 0" rpy="0 0 0" />
 				<geometry>
-					<mesh filename="package://schunk_description/ros/meshes/arm_v0/arm4.stl" />
-				</geometry>
-				<material name="Red" />
-			</visual>
-			<collision>
-				<origin xyz="0 0 0" rpy="0 0 0" />
-				<geometry>
-					<mesh filename="package://schunk_description/ros/meshes/arm_v0/arm4.stlb"/>
+					<mesh filename="package://schunk_description/meshes/lwa/lwa4.stl" />
+				</geometry>
+				<material name="Red" />
+			</visual>
+			<collision>
+				<origin xyz="0 0 0" rpy="0 0 0" />
+				<geometry>
+					<mesh filename="package://schunk_description/meshes/lwa/lwa4.stlb"/>
 				</geometry>
 			</collision>
@@ -163,5 +163,5 @@
 		<!-- joint between arm_4_link and arm_5_link -->
 		<joint name="${name}_5_joint" type="revolute">
-			<origin xyz="0 -0.3165 0" rpy="-1.5708 0 0" />
+			<origin xyz="0 -0.2765 0" rpy="-1.5708 0 0" />
 			<parent link="${name}_4_link"/>
 			<child link="${name}_5_link"/>
@@ -181,12 +181,12 @@
 				<origin xyz="0 0 0" rpy="0 0 0" />
 				<geometry>
-					<mesh filename="package://schunk_description/ros/meshes/arm_v0/arm5.stl" />
-				</geometry>
-				<material name="Blue" />
-			</visual>
-			<collision>
-				<origin xyz="0 0 0" rpy="0 0 0" />
-				<geometry>
-					<mesh filename="package://schunk_description/ros/meshes/arm_v0/arm5.stlb"/>
+					<mesh filename="package://schunk_description/meshes/lwa/lwa5.stl" />
+				</geometry>
+				<material name="Blue" />
+			</visual>
+			<collision>
+				<origin xyz="0 0 0" rpy="0 0 0" />
+				<geometry>
+					<mesh filename="package://schunk_description/meshes/lwa/lwa5.stlb"/>
 				</geometry>
 			</collision>
@@ -212,12 +212,12 @@
 				<origin xyz="0 0 0" rpy="0 0 0" />
 				<geometry>
-					<mesh filename="package://schunk_description/ros/meshes/arm_v0/arm6.stl" />
-				</geometry>
-				<material name="Red" />
-			</visual>
-			<collision>
-				<origin xyz="0 0 0" rpy="0 0 0" />
-				<geometry>
-					<mesh filename="package://schunk_description/ros/meshes/arm_v0/arm6.stlb"/>
+					<mesh filename="package://schunk_description/meshes/lwa/lwa6.stl" />
+				</geometry>
+				<material name="Red" />
+			</visual>
+			<collision>
+				<origin xyz="0 0 0" rpy="0 0 0" />
+				<geometry>
+					<mesh filename="package://schunk_description/meshes/lwa/lwa6.stlb"/>
 				</geometry>
 			</collision>
@@ -225,5 +225,5 @@
 		<!-- joint between arm_6_link and arm_7_link -->
 		<joint name="${name}_7_joint" type="revolute">
-			<origin xyz="0 -0.1927 0" rpy="-1.5708 0 0" />
+			<origin xyz="0 -0.237448 0" rpy="-1.5708 0 0" />
 			<parent link="${name}_6_link"/>
 			<child link="${name}_7_link"/>
@@ -243,18 +243,18 @@
 				<origin xyz="0 0 0" rpy="0 0 0" />
 				<geometry>
-					<mesh filename="package://schunk_description/ros/meshes/arm_v0/arm7.stl" />
-				</geometry>
-				<material name="Blue" />
-			</visual>
-			<collision>
-				<origin xyz="0 0 0" rpy="0 0 0" />
-				<geometry>
-					<mesh filename="package://schunk_description/ros/meshes/arm_v0/arm7.stlb"/>
+					<mesh filename="package://schunk_description/meshes/lwa/lwa7.stl" />
+				</geometry>
+				<material name="Blue" />
+			</visual>
+			<collision>
+				<origin xyz="0 0 0" rpy="0 0 0" />
+				<geometry>
+					<mesh filename="package://schunk_description/meshes/lwa/lwa7.stlb"/>
 				</geometry>
 			</collision>
 		</link>
 		<!-- extensions -->
-		<xacro:schunk_lwa_gazebo_v0 name="${name}" />
-		<xacro:schunk_lwa_transmission_v0 name="${name}" />
+		<xacro:schunk_lwa_extended_gazebo name="${name}" />
+		<xacro:schunk_lwa_extended_transmission name="${name}" />
 	</xacro:macro>
 </robot>

File: schunk_description/urdf/sdh/sdh.gazebo.xacro (robot description, xacro)
@@ -4,5 +4,5 @@
        xmlns:interface="http://playerstage.sourceforge.net/gazebo/xmlschema/#interface"
        xmlns:xacro="http://ros.org/wiki/xacro">
-	<xacro:macro name="schunk_sdh_gazebo_v0" params="name">
+	<xacro:macro name="schunk_sdh_gazebo" params="name">
 		<gazebo reference="${name}_palm_link">
 			<material>Gazebo/Grey</material>

File: schunk_description/urdf/sdh/sdh.transmission.xacro (robot description, xacro)
@@ -4,5 +4,5 @@
        xmlns:interface="http://playerstage.sourceforge.net/gazebo/xmlschema/#interface"
        xmlns:xacro="http://ros.org/wiki/xacro">
-	<xacro:macro name="schunk_sdh_transmission_v0" params="name">
+	<xacro:macro name="schunk_sdh_transmission" params="name">
 		<transmission name="${name}_knuckle_trans" type="pr2_mechanism_model/SimpleTransmission">
 		<actuator name="${name}_knuckle_motor"/>
