Commit message: renamed to schunk names

File: schunk_description/urdf/sdh/sdh.urdf.xacro (robot description, xacro)
@@ -4,7 +4,7 @@
        xmlns:interface="http://playerstage.sourceforge.net/gazebo/xmlschema/#interface"
        xmlns:xacro="http://ros.org/wiki/xacro">
-	<include filename="$(find schunk_description)/ros/urdf/sdh_v0/sdh.gazebo.xacro" />
-	<include filename="$(find schunk_description)/ros/urdf/sdh_v0/sdh.transmission.xacro" />
-	<xacro:macro name="schunk_sdh_v0" params="parent name *origin">
+	<include filename="$(find schunk_description)/urdf/sdh/sdh.gazebo.xacro" />
+	<include filename="$(find schunk_description)/urdf/sdh/sdh.transmission.xacro" />
+	<xacro:macro name="schunk_sdh" params="parent name *origin">
 		<!-- joint between arm_7_link and sdh_palm_link -->
 		<joint name="${name}_palm_joint" type="fixed" >
@@ -22,5 +22,5 @@
 				<origin xyz="0 0 0" rpy="0 0 0" />
 				<geometry>
-					<mesh filename="package://schunk_description/ros/meshes/sdh_v0/palm.stl" />
+					<mesh filename="package://schunk_description/meshes/sdh/palm.stl" />
 				</geometry>
 				<material name="Grey" />
@@ -29,5 +29,5 @@
 				<origin xyz="0 0 0" rpy="0 0 0" />
 				<geometry>
-					<mesh filename="package://schunk_description/ros/meshes/sdh_v0/palm.stlb"/>
+					<mesh filename="package://schunk_description/meshes/sdh/palm.stlb"/>
 				</geometry>
 			</collision>
@@ -66,5 +66,5 @@
 				<origin xyz="0 0 0" rpy="0 0 0" />
 				<geometry>
-					<mesh filename="package://schunk_description/ros/meshes/sdh_v0/knuckle.stl" />
+					<mesh filename="package://schunk_description/meshes/sdh/knuckle.stl" />
 				</geometry>
 				<material name="Black" />
@@ -73,5 +73,5 @@
 				<origin xyz="0 0 0" rpy="0 0 0" />
 				<geometry>
-				<mesh filename="package://schunk_description/ros/meshes/sdh_v0/knuckle.stlb"/>
+				<mesh filename="package://schunk_description/meshes/sdh/knuckle.stlb"/>
 				</geometry>
 			</collision>
@@ -95,5 +95,5 @@
 				<origin xyz="0 0 0" rpy="0 0 0" />
 				<geometry>
-					<mesh filename="package://schunk_description/ros/meshes/sdh_v0/finger.stl" />
+					<mesh filename="package://schunk_description/meshes/sdh/finger.stl" />
 				</geometry>
 			<material name="Red" />
@@ -102,5 +102,5 @@
 				<origin xyz="0 0 0" rpy="0 0 0" />
 				<geometry>
-					<mesh filename="package://schunk_description/ros/meshes/sdh_v0/finger.stlb"/>
+					<mesh filename="package://schunk_description/meshes/sdh/finger.stlb"/>
 				</geometry>
 			</collision>
@@ -124,5 +124,5 @@
 				<origin xyz="0 0 0" rpy="0 0 0" />
 				<geometry>
-					<mesh filename="package://schunk_description/ros/meshes/sdh_v0/finger_tip.stl" />
+					<mesh filename="package://schunk_description/meshes/sdh/finger_tip.stl" />
 				</geometry>
 				<material name="Blue" />
@@ -131,5 +131,5 @@
 				<origin xyz="0 0 0" rpy="0 0 0" />
 				<geometry>
-					<mesh filename="package://schunk_description/ros/meshes/sdh_v0/finger_tip.stlb"/>
+					<mesh filename="package://schunk_description/meshes/sdh/finger_tip.stlb"/>
 				</geometry>
 			</collision>
@@ -155,5 +155,5 @@
 				<origin xyz="0 0 0" rpy="0 0 0" />
 				<geometry>
-					<mesh filename="package://schunk_description/ros/meshes/sdh_v0/knuckle.stl" />
+					<mesh filename="package://schunk_description/meshes/sdh/knuckle.stl" />
 				</geometry>
 				<material name="Black" />
@@ -162,5 +162,5 @@
 				<origin xyz="0 0 0" rpy="0 0 0" />
 				<geometry>
-					<mesh filename="package://schunk_description/ros/meshes/sdh_v0/knuckle.stlb"/>
+					<mesh filename="package://schunk_description/meshes/sdh/knuckle.stlb"/>
 				</geometry>
 			</collision>
@@ -184,5 +184,5 @@
 				<origin xyz="0 0 0" rpy="0 0 0" />
 				<geometry>
-					<mesh filename="package://schunk_description/ros/meshes/sdh_v0/finger.stl" />
+					<mesh filename="package://schunk_description/meshes/sdh/finger.stl" />
 				</geometry>
 				<material name="Red" />
@@ -191,5 +191,5 @@
 				<origin xyz="0 0 0" rpy="0 0 0" />
 				<geometry>
-					<mesh filename="package://schunk_description/ros/meshes/sdh_v0/finger.stlb"/>
+					<mesh filename="package://schunk_description/meshes/sdh/finger.stlb"/>
 				</geometry>
 			</collision>
@@ -213,5 +213,5 @@
 				<origin xyz="0 0 0" rpy="0 0 0" />
 				<geometry>
-					<mesh filename="package://schunk_description/ros/meshes/sdh_v0/finger_tip.stl" />
+					<mesh filename="package://schunk_description/meshes/sdh/finger_tip.stl" />
 				</geometry>
 				<material name="Blue" />
@@ -220,5 +220,5 @@
 				<origin xyz="0 0 0" rpy="0 0 0" />
 				<geometry>
-					<mesh filename="package://schunk_description/ros/meshes/sdh_v0/finger_tip.stlb"/>
+					<mesh filename="package://schunk_description/meshes/sdh/finger_tip.stlb"/>
 				</geometry>
 			</collision>
@@ -240,5 +240,5 @@
 				<origin xyz="0 0 0" rpy="0 0 0" />
 				<geometry>
-					<mesh filename="package://schunk_description/ros/meshes/sdh_v0/knuckle.stl" />
+					<mesh filename="package://schunk_description/meshes/sdh/knuckle.stl" />
 				</geometry>
 				<material name="Black" />
@@ -247,5 +247,5 @@
 				<origin xyz="0 0 0" rpy="0 0 0" />
 				<geometry>
-					<mesh filename="package://schunk_description/ros/meshes/sdh_v0/knuckle.stlb"/>
+					<mesh filename="package://schunk_description/meshes/sdh/knuckle.stlb"/>
 				</geometry>
 			</collision>
@@ -269,5 +269,5 @@
 				<origin xyz="0 0 0" rpy="0 0 0" />
 				<geometry>
-					<mesh filename="package://schunk_description/ros/meshes/sdh_v0/finger.stl" />
+					<mesh filename="package://schunk_description/meshes/sdh/finger.stl" />
 				</geometry>
 				<material name="Red" />
@@ -276,5 +276,5 @@
 				<origin xyz="0 0 0" rpy="0 0 0" />
 				<geometry>
-					<mesh filename="package://schunk_description/ros/meshes/sdh_v0/finger.stlb"/>
+					<mesh filename="package://schunk_description/meshes/sdh/finger.stlb"/>
 				</geometry>
 			</collision>
@@ -298,5 +298,5 @@
 				<origin xyz="0 0 0" rpy="0 0 0" />
 				<geometry>
-					<mesh filename="package://schunk_description/ros/meshes/sdh_v0/finger_tip.stl" />
+					<mesh filename="package://schunk_description/meshes/sdh/finger_tip.stl" />
 				</geometry>
 				<material name="Blue" />
@@ -305,11 +305,11 @@
 				<origin xyz="0 0 0" rpy="0 0 0" />
 				<geometry>
-					<mesh filename="package://schunk_description/ros/meshes/sdh_v0/finger_tip.stlb"/>
+					<mesh filename="package://schunk_description/meshes/sdh/finger_tip.stlb"/>
 				</geometry>
 			</collision>
 		</link>
 		<!-- extensions -->
-		<xacro:schunk_sdh_gazebo_v0 name="${name}" />
-		<xacro:schunk_sdh_transmission_v0 name="${name}" />
+		<xacro:schunk_sdh_gazebo name="${name}" />
+		<xacro:schunk_sdh_transmission name="${name}" />
 	</xacro:macro>
 </robot>

Commit message: Redefined Schunk component colors for gazebo and rviz

File: schunk_description/urdf/lwa/lwa.gazebo.xacro (robot description, xacro)
@@ -6,33 +6,33 @@
 	<xacro:macro name="schunk_lwa_gazebo" params="name">
 		<gazebo reference="${name}_0_link">
-			<material value="PR2/Red" />
+			<material value="IPA/DarkGolden" />
 			<turnGravityOff>false</turnGravityOff>
 		</gazebo>
 		<gazebo reference="${name}_1_link">
-			<material value="PR2/Blue" />
+			<material value="IPA/DarkGolden" />
 			<turnGravityOff>false</turnGravityOff>
 		</gazebo>
 		<gazebo reference="${name}_2_link">
-			<material value="PR2/Red" />
+			<material value="IPA/DarkGolden" />
 			<turnGravityOff>false</turnGravityOff>
 		</gazebo>
 		<gazebo reference="${name}_3_link">
-			<material value="PR2/Blue" />
+			<material value="IPA/DarkGolden" />
 			<turnGravityOff>false</turnGravityOff>
 		</gazebo>
 		<gazebo reference="${name}_4_link">
-			<material value="PR2/Red" />
+			<material value="IPA/DarkGolden" />
 			<turnGravityOff>false</turnGravityOff>
 		</gazebo>
 		<gazebo reference="${name}_5_link">
-			<material value="PR2/Blue" />
+			<material value="IPA/DarkGolden" />
 			<turnGravityOff>false</turnGravityOff>
 		</gazebo>
 		<gazebo reference="${name}_6_link">
-			<material value="PR2/Red" />
+			<material value="IPA/DarkGolden" />
 			<turnGravityOff>false</turnGravityOff>
 		</gazebo>
 		<gazebo reference="${name}_7_link">
-			<material value="PR2/Blue" />
+			<material value="IPA/DarkGolden" />
 			<turnGravityOff>false</turnGravityOff>
 		</gazebo>

File: schunk_description/urdf/lwa/lwa.urdf.xacro (robot description, xacro)
@@ -24,5 +24,5 @@
 					<cylinder radius="0.045" length="0.08"/>
 				</geometry>
-				<material name="Red" />
+				<material name="DarkGolden" />
 			</visual>
 			<collision>
@@ -56,5 +56,5 @@
 					<mesh filename="package://schunk_description/meshes/lwa/lwa1.stl" />
 				</geometry>
-				<material name="Blue" />
+				<material name="DarkGolden" />
 			</visual>
 			<collision>
@@ -88,5 +88,5 @@
 					<mesh filename="package://schunk_description/meshes/lwa/lwa2.stl" />
 				</geometry>
-				<material name="Red" />
+				<material name="DarkGolden" />
 			</visual>
 			<collision>
@@ -120,5 +120,5 @@
 					<mesh filename="package://schunk_description/meshes/lwa/lwa3.stl" />
 				</geometry>
-				<material name="Blue" />
+				<material name="DarkGolden" />
 			</visual>
 			<collision>
@@ -152,5 +152,5 @@
 					<mesh filename="package://schunk_description/meshes/lwa/lwa4.stl" />
 				</geometry>
-				<material name="Red" />
+				<material name="DarkGolden" />
 			</visual>
 			<collision>
@@ -183,5 +183,5 @@
 					<mesh filename="package://schunk_description/meshes/lwa/lwa5.stl" />
 				</geometry>
-				<material name="Blue" />
+				<material name="DarkGolden" />
 			</visual>
 			<collision>
@@ -214,5 +214,5 @@
 					<mesh filename="package://schunk_description/meshes/lwa/lwa6.stl" />
 				</geometry>
-				<material name="Red" />
+				<material name="DarkGolden" />
 			</visual>
 			<collision>
@@ -245,5 +245,5 @@
 					<mesh filename="package://schunk_description/meshes/lwa/lwa7.stl" />
 				</geometry>
-				<material name="Blue" />
+				<material name="DarkGolden" />
 			</visual>
 			<collision>

File: schunk_description/urdf/sdh/sdh.gazebo.xacro (robot description, xacro)
@@ -26,5 +26,5 @@
 				</controller:gazebo_ros_bumper>
 			</sensor:contact>
-			<material>Gazebo/Red</material>
+			<material>IPA/Grey1</material>
 			<turnGravityOff>false</turnGravityOff>
 		</gazebo>
@@ -42,5 +42,5 @@
 				</controller:gazebo_ros_bumper>
 			</sensor:contact>
-			<material>Gazebo/Blue</material>
+			<material>IPA/Grey2</material>
 		</gazebo>
 		<gazebo reference="${name}_finger_21_link">
@@ -61,5 +61,5 @@
 				</controller:gazebo_ros_bumper>
 			</sensor:contact>
-			<material>Gazebo/Red</material>
+			<material>IPA/Grey1</material>
 			<turnGravityOff>false</turnGravityOff>
 		</gazebo>
@@ -77,5 +77,5 @@
 				</controller:gazebo_ros_bumper>
 			</sensor:contact>
-			<material>Gazebo/Blue</material>
+			<material>IPA/Grey2</material>
 		</gazebo>
 		<gazebo reference="${name}_thumb_1_link">
@@ -96,5 +96,5 @@
 				</controller:gazebo_ros_bumper>
 			</sensor:contact>
-			<material>Gazebo/Red</material>
+			<material>IPA/Grey1</material>
 			<turnGravityOff>false</turnGravityOff>
 		</gazebo>
@@ -112,5 +112,5 @@
 				</controller:gazebo_ros_bumper>
 			</sensor:contact>
-			<material>Gazebo/Blue</material>
+			<material>IPA/Grey2</material>
 		</gazebo>
 	</xacro:macro>

File: schunk_description/urdf/sdh/sdh.urdf.xacro (robot description, xacro)
@@ -97,5 +97,5 @@
 					<mesh filename="package://schunk_description/meshes/sdh/finger.stl" />
 				</geometry>
-			<material name="Red" />
+			<material name="Grey" />
 			</visual>
 			<collision>
@@ -126,5 +126,5 @@
 					<mesh filename="package://schunk_description/meshes/sdh/finger_tip.stl" />
 				</geometry>
-				<material name="Blue" />
+				<material name="Black" />
 			</visual>
 			<collision>
@@ -186,5 +186,5 @@
 					<mesh filename="package://schunk_description/meshes/sdh/finger.stl" />
 				</geometry>
-				<material name="Red" />
+				<material name="Grey" />
 			</visual>
 			<collision>
@@ -215,5 +215,5 @@
 					<mesh filename="package://schunk_description/meshes/sdh/finger_tip.stl" />
 				</geometry>
-				<material name="Blue" />
+				<material name="Black" />
 			</visual>
 			<collision>
@@ -271,5 +271,5 @@
 					<mesh filename="package://schunk_description/meshes/sdh/finger.stl" />
 				</geometry>
-				<material name="Red" />
+				<material name="Grey" />
 			</visual>
 			<collision>
@@ -300,5 +300,5 @@
 					<mesh filename="package://schunk_description/meshes/sdh/finger_tip.stl" />
 				</geometry>
-				<material name="Blue" />
+				<material name="Black" />
 			</visual>
 			<collision>
