Commit message: Redefined colors

File: schunk_description/urdf/lwa/lwa.gazebo.xacro (robot description, xacro)
@@ -6,33 +6,33 @@
 	<xacro:macro name="schunk_lwa_gazebo" params="name">
 		<gazebo reference="${name}_0_link">
-			<material value="IPA/DarkGolden" />
+			<material value="Schunk/DarkGolden" />
 			<turnGravityOff>false</turnGravityOff>
 		</gazebo>
 		<gazebo reference="${name}_1_link">
-			<material value="IPA/DarkGolden" />
+			<material value="Schunk/DarkGolden" />
 			<turnGravityOff>false</turnGravityOff>
 		</gazebo>
 		<gazebo reference="${name}_2_link">
-			<material value="IPA/DarkGolden" />
+			<material value="Schunk/DarkGolden" />
 			<turnGravityOff>false</turnGravityOff>
 		</gazebo>
 		<gazebo reference="${name}_3_link">
-			<material value="IPA/DarkGolden" />
+			<material value="Schunk/DarkGolden" />
 			<turnGravityOff>false</turnGravityOff>
 		</gazebo>
 		<gazebo reference="${name}_4_link">
-			<material value="IPA/DarkGolden" />
+			<material value="Schunk/DarkGolden" />
 			<turnGravityOff>false</turnGravityOff>
 		</gazebo>
 		<gazebo reference="${name}_5_link">
-			<material value="IPA/DarkGolden" />
+			<material value="Schunk/DarkGolden" />
 			<turnGravityOff>false</turnGravityOff>
 		</gazebo>
 		<gazebo reference="${name}_6_link">
-			<material value="IPA/DarkGolden" />
+			<material value="Schunk/DarkGolden" />
 			<turnGravityOff>false</turnGravityOff>
 		</gazebo>
 		<gazebo reference="${name}_7_link">
-			<material value="IPA/DarkGolden" />
+			<material value="Schunk/DarkGolden" />
 			<turnGravityOff>false</turnGravityOff>
 		</gazebo>

File: schunk_description/urdf/lwa_extended/lwa_extended.gazebo.xacro (robot description, xacro)
@@ -6,33 +6,33 @@
 	<xacro:macro name="schunk_lwa_extended_gazebo" params="name">
 		<gazebo reference="${name}_0_link">
-			<material value="PR2/Red" />
+			<material value="Schunk/DarkGolden" />
 			<turnGravityOff>false</turnGravityOff>
 		</gazebo>
 		<gazebo reference="${name}_1_link">
-			<material value="PR2/Blue" />
+			<material value="Schunk/DarkGolden" />
 			<turnGravityOff>false</turnGravityOff>
 		</gazebo>
 		<gazebo reference="${name}_2_link">
-			<material value="PR2/Red" />
+			<material value="Schunk/DarkGolden" />
 			<turnGravityOff>false</turnGravityOff>
 		</gazebo>
 		<gazebo reference="${name}_3_link">
-			<material value="PR2/Blue" />
+			<material value="Schunk/DarkGolden" />
 			<turnGravityOff>false</turnGravityOff>
 		</gazebo>
 		<gazebo reference="${name}_4_link">
-			<material value="PR2/Red" />
+			<material value="Schunk/DarkGolden" />
 			<turnGravityOff>false</turnGravityOff>
 		</gazebo>
 		<gazebo reference="${name}_5_link">
-			<material value="PR2/Blue" />
+			<material value="Schunk/DarkGolden" />
 			<turnGravityOff>false</turnGravityOff>
 		</gazebo>
 		<gazebo reference="${name}_6_link">
-			<material value="PR2/Red" />
+			<material value="Schunk/DarkGolden" />
 			<turnGravityOff>false</turnGravityOff>
 		</gazebo>
 		<gazebo reference="${name}_7_link">
-			<material value="PR2/Blue" />
+			<material value="Schunk/DarkGolden" />
 			<turnGravityOff>false</turnGravityOff>
 		</gazebo>

File: schunk_description/urdf/lwa_extended/lwa_extended.urdf.xacro (robot description, xacro)
@@ -24,5 +24,5 @@
 					<cylinder radius="0.045" length="0.08"/>
 				</geometry>
-				<material name="Red" />
+				<material name="Schunk/DarkGolden" />
 			</visual>
 			<collision>
@@ -56,5 +56,5 @@
 					<mesh filename="package://schunk_description/meshes/lwa/lwa1.stl" />
 				</geometry>
-				<material name="Blue" />
+				<material name="Schunk/DarkGolden" />
 			</visual>
 			<collision>
@@ -88,5 +88,5 @@
 					<mesh filename="package://schunk_description/meshes/lwa/lwa2.stl" />
 				</geometry>
-				<material name="Red" />
+				<material name="Schunk/DarkGolden" />
 			</visual>
 			<collision>
@@ -120,5 +120,5 @@
 					<mesh filename="package://schunk_description/meshes/lwa/lwa3.stl" />
 				</geometry>
-				<material name="Blue" />
+				<material name="Schunk/DarkGolden" />
 			</visual>
 			<collision>
@@ -152,5 +152,5 @@
 					<mesh filename="package://schunk_description/meshes/lwa/lwa4.stl" />
 				</geometry>
-				<material name="Red" />
+				<material name="Schunk/DarkGolden" />
 			</visual>
 			<collision>
@@ -183,5 +183,5 @@
 					<mesh filename="package://schunk_description/meshes/lwa/lwa5.stl" />
 				</geometry>
-				<material name="Blue" />
+				<material name="Schunk/DarkGolden" />
 			</visual>
 			<collision>
@@ -214,5 +214,5 @@
 					<mesh filename="package://schunk_description/meshes/lwa/lwa6.stl" />
 				</geometry>
-				<material name="Red" />
+				<material name="Schunk/DarkGolden" />
 			</visual>
 			<collision>
@@ -245,5 +245,5 @@
 					<mesh filename="package://schunk_description/meshes/lwa/lwa7.stl" />
 				</geometry>
-				<material name="Blue" />
+				<material name="Schunk/DarkGolden" />
 			</visual>
 			<collision>

File: schunk_description/urdf/materials.urdf.xacro (robot description, xacro)
@@ -1,26 +1,17 @@
 <?xml version="1.0"?>
 <robot>
-	<material name="Blue">
+	<material name="Schunk/Blue">
 		<color rgba="0.0 0.0 0.8 1.0"/>
 	</material>
-	<material name="Green">
-		<color rgba="0.0 0.8 0.0 1.0"/>
-	</material>
-	<material name="IPA/DarkGrey">
+	<material name="Schunk/DarkGrey">
 		<color rgba="0.7 0.7 0.7 1.0"/>
 	</material>
-	<material name="IPA/LightGrey">
+	<material name="Schunk/LightGrey">
 		<color rgba="0.81 0.81 0.81 1.0"/>
 	</material>
-	<material name="Red">
-		<color rgba="0.8 0.0 0.0 1.0"/>
-	</material>
-	<material name="White">
-		<color rgba="1.0 1.0 1.0 1.0"/>
-	</material>
-	<material name="IPA/Black">
+	<material name="Schunk/Black">
 		<color rgba="0.0 0.0 0.0 1.0"/>
 	</material>
-	<material name="IPA/Orange">
+	<material name="Schunk/Orange">
 		<color rgba="1.0 0.5 0.0 1.0"/>
 	</material>
@@ -28,15 +19,3 @@
 		<color rgba="0.72 0.5255 0.043 1.0"/>
 	</material>
-	<material name="Caster">
-		<texture filename="package://pr2_ogre/Media/materials/textures/pr2_caster_texture.png" />
-	</material>
-	<material name="Wheel_l">
-		<texture filename="package://pr2_ogre/Media/materials/textures/pr2_wheel_left.png" />
-	</material>
-	<material name="Wheel_r">
-		<texture filename="package://pr2_ogre/Media/materials/textures/pr2_wheel_right.png" />
-	</material>
-	<material name="RollLinks">
-		<texture filename="package://pr2_ogre/Media/materials/textures/pr2_wheel_left.png" />
-	</material>
 </robot>

File: schunk_description/urdf/powerball/powerball.gazebo.xacro (robot description, xacro)
@@ -6,35 +6,35 @@
 	<xacro:macro name="schunk_powerball_gazebo" params="name">
 		<gazebo reference="${name}_0_link">
-			<material value="Grey" />
+			<material value="Schunk/LightGrey" />
 			<turnGravityOff>false</turnGravityOff>
                         <selfCollide>true</selfCollide>
 		</gazebo>
 		<gazebo reference="${name}_1_link">
-			<material value="Gazebo/Blue" />
+			<material value="Schunk/Blue" />
 			<turnGravityOff>false</turnGravityOff>
                         <selfCollide>true</selfCollide>
 		</gazebo>
 		<gazebo reference="${name}_2_link">
-			<material value="Grey" />
+			<material value="Schunk/LightGrey" />
 			<turnGravityOff>false</turnGravityOff>
                         <selfCollide>true</selfCollide>
 		</gazebo>
 		<gazebo reference="${name}_3_link">
-			<material value="Gazebo/Blue" />
+			<material value="Schunk/Blue" />
 			<turnGravityOff>false</turnGravityOff>
                         <selfCollide>true</selfCollide>
 		</gazebo>
 		<gazebo reference="${name}_4_link">
-			<material value="Grey" />
+			<material value="Schunk/LightGrey" />
 			<turnGravityOff>false</turnGravityOff>
                         <selfCollide>true</selfCollide>
 		</gazebo>
 		<gazebo reference="${name}_5_link">
-			<material value="Gazebo/Blue" />
+			<material value="Schunk/Blue" />
 			<turnGravityOff>false</turnGravityOff>
                         <selfCollide>true</selfCollide>
 		</gazebo>
 		<gazebo reference="${name}_6_link">
-			<material value="Grey" />
+			<material value="Schunk/LightGrey" />
 			<turnGravityOff>false</turnGravityOff>
                         <selfCollide>true</selfCollide>

File: schunk_description/urdf/powerball/powerball.urdf.xacro (robot description, xacro)
@@ -24,5 +24,5 @@
 					<mesh filename="package://schunk_description/meshes/powerball/arm_0_link.stl" />
 				</geometry>
-				<material name="IPA/LightGrey" />
+				<material name="Schunk/LightGrey" />
 			</visual>
 			<collision>
@@ -55,5 +55,5 @@
 					<mesh filename="package://schunk_description/meshes/powerball/arm_1_link.stl" />
 				</geometry>
-				<material name="Blue" />
+				<material name="Schunk/Blue" />
 			</visual>
 			<collision>
@@ -86,5 +86,5 @@
 					<mesh filename="package://schunk_description/meshes/powerball/arm_2_link.stl" />
 				</geometry>
-				<material name="IPA/LightGrey" />
+				<material name="Schunk/LightGrey" />
 			</visual>
 			<collision>
@@ -117,5 +117,5 @@
 					<mesh filename="package://schunk_description/meshes/powerball/arm_3_link.stl" />
 				</geometry>
-				<material name="Blue" />
+				<material name="Schunk/Blue" />
 			</visual>
 			<collision>
@@ -148,5 +148,5 @@
 					<mesh filename="package://schunk_description/meshes/powerball/arm_4_link.stl" />
 				</geometry>
-				<material name="IPA/LightGrey" />
+				<material name="Schunk/LightGrey" />
 			</visual>
 			<collision>
@@ -179,5 +179,5 @@
 					<mesh filename="package://schunk_description/meshes/powerball/arm_5_link.stl" />
 				</geometry>
-				<material name="Blue" />
+				<material name="Schunk/Blue" />
 			</visual>
 			<collision>
@@ -210,5 +210,5 @@
 					<mesh filename="package://schunk_description/meshes/powerball/arm_6_link.stl" />
 				</geometry>
-				<material name="IPA/LightGrey" />
+				<material name="Schunk/LightGrey" />
 			</visual>
 			<collision>

File: schunk_description/urdf/sdh/sdh.gazebo.xacro (robot description, xacro)
@@ -6,9 +6,9 @@
 	<xacro:macro name="schunk_sdh_gazebo" params="name">
 		<gazebo reference="${name}_palm_link">
-			<material>Gazebo/Grey</material>
+			<material>Schunk/LightGrey</material>
 			<turnGravityOff>false</turnGravityOff>
 		</gazebo>
 		<gazebo reference="${name}_finger_11_link">
-			<material>Gazebo/Black</material>
+			<material>Schunk/Black</material>
 			<turnGravityOff>false</turnGravityOff>
 		</gazebo>
@@ -26,5 +26,5 @@
 				</controller:gazebo_ros_bumper>
 			</sensor:contact>
-			<material>IPA/Grey1</material>
+			<material>Schunk/LightGrey</material>
 			<turnGravityOff>false</turnGravityOff>
 		</gazebo>
@@ -42,8 +42,8 @@
 				</controller:gazebo_ros_bumper>
 			</sensor:contact>
-			<material>IPA/Grey2</material>
+			<material>Schunk/LightGrey</material>
 		</gazebo>
 		<gazebo reference="${name}_finger_21_link">
-			<material>Gazebo/Black</material>
+			<material>Schunk/Black</material>
 			<turnGravityOff>false</turnGravityOff>
 		</gazebo>
@@ -61,5 +61,5 @@
 				</controller:gazebo_ros_bumper>
 			</sensor:contact>
-			<material>IPA/Grey1</material>
+			<material>Schunk/LightGrey</material>
 			<turnGravityOff>false</turnGravityOff>
 		</gazebo>
@@ -77,8 +77,8 @@
 				</controller:gazebo_ros_bumper>
 			</sensor:contact>
-			<material>IPA/Grey2</material>
+			<material>Schunk/LightGrey</material>
 		</gazebo>
 		<gazebo reference="${name}_thumb_1_link">
-			<material>Gazebo/Black</material>
+			<material>Schunk/Black</material>
 			<turnGravityOff>false</turnGravityOff>
 		</gazebo>
@@ -96,5 +96,5 @@
 				</controller:gazebo_ros_bumper>
 			</sensor:contact>
-			<material>IPA/Grey1</material>
+			<material>Schunk/LightGrey</material>
 			<turnGravityOff>false</turnGravityOff>
 		</gazebo>
@@ -112,5 +112,5 @@
 				</controller:gazebo_ros_bumper>
 			</sensor:contact>
-			<material>IPA/Grey2</material>
+			<material>Schunk/LightGrey</material>
 		</gazebo>
 	</xacro:macro>

File: schunk_description/urdf/sdh/sdh.urdf.xacro (robot description, xacro)
@@ -24,5 +24,5 @@
 					<mesh filename="package://schunk_description/meshes/sdh/palm.stl" />
 				</geometry>
-				<material name="IPA/DarkGrey" />
+				<material name="Schunk/DarkGrey" />
 			</visual>
 			<collision>
@@ -68,5 +68,5 @@
 					<mesh filename="package://schunk_description/meshes/sdh/knuckle.stl" />
 				</geometry>
-				<material name="IPA/Black" />
+				<material name="Schunk/Black" />
 			</visual>
 			<collision>
@@ -97,5 +97,5 @@
 					<mesh filename="package://schunk_description/meshes/sdh/finger.stl" />
 				</geometry>
-			<material name="IPA/DarkGrey" />
+			<material name="Schunk/DarkGrey" />
 			</visual>
 			<collision>
@@ -126,5 +126,5 @@
 					<mesh filename="package://schunk_description/meshes/sdh/finger_tip.stl" />
 				</geometry>
-				<material name="IPA/Black" />
+				<material name="Schunk/Black" />
 			</visual>
 			<collision>
@@ -157,5 +157,5 @@
 					<mesh filename="package://schunk_description/meshes/sdh/knuckle.stl" />
 				</geometry>
-				<material name="IPA/Black" />
+				<material name="Schunk/Black" />
 			</visual>
 			<collision>
@@ -186,5 +186,5 @@
 					<mesh filename="package://schunk_description/meshes/sdh/finger.stl" />
 				</geometry>
-				<material name="IPA/DarkGrey" />
+				<material name="Schunk/DarkGrey" />
 			</visual>
 			<collision>
@@ -215,5 +215,5 @@
 					<mesh filename="package://schunk_description/meshes/sdh/finger_tip.stl" />
 				</geometry>
-				<material name="IPA/Black" />
+				<material name="Schunk/Black" />
 			</visual>
 			<collision>
@@ -242,5 +242,5 @@
 					<mesh filename="package://schunk_description/meshes/sdh/knuckle.stl" />
 				</geometry>
-				<material name="IPA/Black" />
+				<material name="Schunk/Black" />
 			</visual>
 			<collision>
@@ -271,5 +271,5 @@
 					<mesh filename="package://schunk_description/meshes/sdh/finger.stl" />
 				</geometry>
-				<material name="IPA/DarkGrey" />
+				<material name="Schunk/DarkGrey" />
 			</visual>
 			<collision>
@@ -300,5 +300,5 @@
 					<mesh filename="package://schunk_description/meshes/sdh/finger_tip.stl" />
 				</geometry>
-				<material name="IPA/Black" />
+				<material name="Schunk/Black" />
 			</visual>
 			<collision>
