Commit message: consistency changes due to latest gazebo tag format

File: schunk_description/urdf/lwa/lwa.gazebo.xacro (robot description, xacro)
@@ -3,34 +3,42 @@
   <xacro:macro name="schunk_lwa_gazebo" params="name">
     <gazebo reference="${name}_0_link">
+      <gravity>true</gravity>
+      <self_collide>false</self_collide>
       <material value="Schunk/DarkGolden" />
-      <turnGravityOff>false</turnGravityOff>
     </gazebo>
     <gazebo reference="${name}_1_link">
+      <gravity>true</gravity>
+      <self_collide>false</self_collide>
       <material value="Schunk/DarkGolden" />
-      <turnGravityOff>false</turnGravityOff>
     </gazebo>
     <gazebo reference="${name}_2_link">
+      <gravity>true</gravity>
+      <self_collide>false</self_collide>
       <material value="Schunk/DarkGolden" />
-      <turnGravityOff>false</turnGravityOff>
     </gazebo>
     <gazebo reference="${name}_3_link">
+      <gravity>true</gravity>
+      <self_collide>false</self_collide>
       <material value="Schunk/DarkGolden" />
-      <turnGravityOff>false</turnGravityOff>
     </gazebo>
     <gazebo reference="${name}_4_link">
+      <gravity>true</gravity>
+      <self_collide>false</self_collide>
       <material value="Schunk/DarkGolden" />
-      <turnGravityOff>false</turnGravityOff>
     </gazebo>
     <gazebo reference="${name}_5_link">
+      <gravity>true</gravity>
+      <self_collide>false</self_collide>
       <material value="Schunk/DarkGolden" />
-      <turnGravityOff>false</turnGravityOff>
     </gazebo>
     <gazebo reference="${name}_6_link">
+      <gravity>true</gravity>
+      <self_collide>false</self_collide>
       <material value="Schunk/DarkGolden" />
-      <turnGravityOff>false</turnGravityOff>
     </gazebo>
     <gazebo reference="${name}_7_link">
+      <gravity>true</gravity>
+      <self_collide>false</self_collide>
       <material value="Schunk/DarkGolden" />
-      <turnGravityOff>false</turnGravityOff>
     </gazebo>
   </xacro:macro>

File: schunk_description/urdf/lwa4d/lwa4d.gazebo.xacro (robot description, xacro)
@@ -3,14 +3,16 @@
   <xacro:macro name="schunk_lwa4d_gazebo" params="name">
     <gazebo reference="${name}_0_link">
+      <gravity>true</gravity>
+      <self_collide>false</self_collide>
       <material value="Schunk/DarkGolden" />
-      <turnGravityOff>false</turnGravityOff>
     </gazebo>
     <gazebo reference="${name}_1_link">
-      <material value="Schunk/DarkGolden" />
-      <turnGravityOff>false</turnGravityOff>
+      <gravity>true</gravity>
+      <self_collide>false</self_collide>
     </gazebo>
     <gazebo reference="${name}_2_link">
+      <gravity>true</gravity>
+      <self_collide>false</self_collide>
       <material value="Schunk/DarkGolden" />
-      <turnGravityOff>false</turnGravityOff>
     </gazebo>
     <gazebo reference="${name}_3_link">
@@ -19,18 +21,22 @@
     </gazebo>
     <gazebo reference="${name}_4_link">
+      <gravity>true</gravity>
+      <self_collide>false</self_collide>
       <material value="Schunk/DarkGolden" />
-      <turnGravityOff>false</turnGravityOff>
     </gazebo>
     <gazebo reference="${name}_5_link">
+      <gravity>true</gravity>
+      <self_collide>false</self_collide>
       <material value="Schunk/DarkGolden" />
-      <turnGravityOff>false</turnGravityOff>
     </gazebo>
     <gazebo reference="${name}_6_link">
+      <gravity>true</gravity>
+      <self_collide>false</self_collide>
       <material value="Schunk/DarkGolden" />
-      <turnGravityOff>false</turnGravityOff>
     </gazebo>
     <gazebo reference="${name}_7_link">
+      <gravity>true</gravity>
+      <self_collide>false</self_collide>
       <material value="Schunk/DarkGolden" />
-      <turnGravityOff>false</turnGravityOff>
     </gazebo>
   </xacro:macro>

File: schunk_description/urdf/lwa4p/lwa4p.gazebo.xacro (robot description, xacro)
@@ -3,37 +3,37 @@
   <xacro:macro name="schunk_lwa4p_gazebo" params="name">
     <gazebo reference="${name}_0_link">
+      <gravity>true</gravity>
+      <self_collide>false</self_collide>
       <material value="Schunk/LightGrey" />
-      <turnGravityOff>false</turnGravityOff>
-                        <selfCollide>true</selfCollide>
     </gazebo>
     <gazebo reference="${name}_1_link">
+      <gravity>true</gravity>
+      <self_collide>false</self_collide>
       <material value="Schunk/Blue" />
-      <turnGravityOff>false</turnGravityOff>
-                        <selfCollide>true</selfCollide>
     </gazebo>
     <gazebo reference="${name}_2_link">
+      <gravity>true</gravity>
+      <self_collide>false</self_collide>
       <material value="Schunk/LightGrey" />
-      <turnGravityOff>false</turnGravityOff>
-                        <selfCollide>true</selfCollide>
     </gazebo>
     <gazebo reference="${name}_3_link">
+      <gravity>true</gravity>
+      <self_collide>false</self_collide>
       <material value="Schunk/Blue" />
-      <turnGravityOff>false</turnGravityOff>
-                        <selfCollide>true</selfCollide>
     </gazebo>
     <gazebo reference="${name}_4_link">
+      <gravity>true</gravity>
+      <self_collide>false</self_collide>
       <material value="Schunk/LightGrey" />
-      <turnGravityOff>false</turnGravityOff>
-                        <selfCollide>true</selfCollide>
     </gazebo>
     <gazebo reference="${name}_5_link">
+      <gravity>true</gravity>
+      <self_collide>false</self_collide>
       <material value="Schunk/Blue" />
-      <turnGravityOff>false</turnGravityOff>
-                        <selfCollide>true</selfCollide>
     </gazebo>
     <gazebo reference="${name}_6_link">
+      <gravity>true</gravity>
+      <self_collide>false</self_collide>
       <material value="Schunk/LightGrey" />
-      <turnGravityOff>false</turnGravityOff>
-                        <selfCollide>true</selfCollide>
     </gazebo>
   </xacro:macro>

File: schunk_description/urdf/lwa4p_extended/lwa4p_extended.gazebo.xacro (robot description, xacro)
@@ -3,27 +3,35 @@
   <xacro:macro name="schunk_lwa4p_extended_gazebo" params="name">
     <gazebo reference="${name}_base_link">
-      <selfCollide>true</selfCollide>
+      <gravity>true</gravity>
+      <self_collide>false</self_collide>
     </gazebo>
     <gazebo reference="${name}_1_link">
-      <selfCollide>true</selfCollide>
+      <gravity>true</gravity>
+      <self_collide>false</self_collide>
     </gazebo>
     <gazebo reference="${name}_2_link">
-      <selfCollide>true</selfCollide>
+      <gravity>true</gravity>
+      <self_collide>false</self_collide>
     </gazebo>
     <gazebo reference="${name}_3_link">
-      <selfCollide>true</selfCollide>
+      <gravity>true</gravity>
+      <self_collide>false</self_collide>
     </gazebo>
     <gazebo reference="${name}_4_link">
-      <selfCollide>true</selfCollide>
+      <gravity>true</gravity>
+      <self_collide>false</self_collide>
     </gazebo>
     <gazebo reference="${name}_5_link">
-      <selfCollide>true</selfCollide>
+      <gravity>true</gravity>
+      <self_collide>false</self_collide>
     </gazebo>
     <gazebo reference="${name}_6_link">
-      <selfCollide>true</selfCollide>
+      <gravity>true</gravity>
+      <self_collide>false</self_collide>
     </gazebo>
     <gazebo reference="${name}_7_link">
+      <gravity>true</gravity>
+      <self_collide>false</self_collide>
       <material value="Schunk/LightGrey" />
-      <selfCollide>true</selfCollide>
     </gazebo>
   </xacro:macro>

File: schunk_description/urdf/lwa_extended/lwa_extended.gazebo.xacro (robot description, xacro)
@@ -3,34 +3,42 @@
   <xacro:macro name="schunk_lwa_extended_gazebo" params="name">
     <gazebo reference="${name}_0_link">
+      <gravity>true</gravity>
+      <self_collide>false</self_collide>
       <material value="Schunk/DarkGolden" />
-      <turnGravityOff>false</turnGravityOff>
     </gazebo>
     <gazebo reference="${name}_1_link">
+      <gravity>true</gravity>
+      <self_collide>false</self_collide>
       <material value="Schunk/DarkGolden" />
-      <turnGravityOff>false</turnGravityOff>
     </gazebo>
     <gazebo reference="${name}_2_link">
+      <gravity>true</gravity>
+      <self_collide>false</self_collide>
       <material value="Schunk/DarkGolden" />
-      <turnGravityOff>false</turnGravityOff>
     </gazebo>
     <gazebo reference="${name}_3_link">
+      <gravity>true</gravity>
+      <self_collide>false</self_collide>
       <material value="Schunk/DarkGolden" />
-      <turnGravityOff>false</turnGravityOff>
     </gazebo>
     <gazebo reference="${name}_4_link">
+      <gravity>true</gravity>
+      <self_collide>false</self_collide>
       <material value="Schunk/DarkGolden" />
-      <turnGravityOff>false</turnGravityOff>
     </gazebo>
     <gazebo reference="${name}_5_link">
+      <gravity>true</gravity>
+      <self_collide>false</self_collide>
       <material value="Schunk/DarkGolden" />
-      <turnGravityOff>false</turnGravityOff>
     </gazebo>
     <gazebo reference="${name}_6_link">
+      <gravity>true</gravity>
+      <self_collide>false</self_collide>
       <material value="Schunk/DarkGolden" />
-      <turnGravityOff>false</turnGravityOff>
     </gazebo>
     <gazebo reference="${name}_7_link">
+      <gravity>true</gravity>
+      <self_collide>false</self_collide>
       <material value="Schunk/DarkGolden" />
-      <turnGravityOff>false</turnGravityOff>
     </gazebo>
   </xacro:macro>

File: schunk_description/urdf/pg70/pg70.gazebo.xacro (robot description, xacro)
@@ -3,6 +3,7 @@
   <xacro:macro name="schunk_pg70_gazebo" params="name">
     <gazebo reference="${name}_palm_link">
+      <gravity>true</gravity>
+      <self_collide>false</self_collide>
       <material>Schunk/LightGrey</material>
-      <turnGravityOff>false</turnGravityOff>
     </gazebo>
     <gazebo reference="${name}_finger_1_link">
@@ -11,6 +12,7 @@
     </gazebo>
     <gazebo reference="${name}_finger_2_link">
+      <gravity>true</gravity>
+      <self_collide>false</self_collide>
       <material>Schunk/LightGrey</material>
-      <turnGravityOff>false</turnGravityOff>
     </gazebo>
   </xacro:macro>

File: schunk_description/urdf/sdh/sdh.gazebo.xacro (robot description, xacro)
@@ -3,13 +3,18 @@
   <xacro:macro name="schunk_sdh_gazebo" params="name">
     <gazebo reference="${name}_palm_link">
+      <gravity>true</gravity>
+      <self_collide>false</self_collide>
       <material>Schunk/LightGrey</material>
-      <turnGravityOff>false</turnGravityOff>
     </gazebo>
     <gazebo reference="${name}_finger_11_link">
+      <gravity>true</gravity>
+      <self_collide>false</self_collide>
       <material>Schunk/LightGrey</material>
-      <turnGravityOff>false</turnGravityOff>
     </gazebo>
-    <!--gazebo reference="${name}_finger_12_link">
-      <selfCollide>true</selfCollide>
+    <gazebo reference="${name}_finger_12_link">
+      <gravity>true</gravity>
+      <self_collide>false</self_collide>
+      <material>Schunk/LightGrey</material>
+<!--
       <sensor name='${name}_finger_12_contact_sensor' type='contact'>
         <always_on>true</always_on>
@@ -25,9 +30,11 @@
         </plugin>
       </sensor>
+-->
+    </gazebo>
+    <gazebo reference="${name}_finger_13_link">
+      <gravity>true</gravity>
+      <self_collide>false</self_collide>
       <material>Schunk/LightGrey</material>
-      <turnGravityOff>false</turnGravityOff>
-    </gazebo-->
-    <!--gazebo reference="${name}_finger_13_link">
-      <selfCollide>true</selfCollide>
+<!--
       <sensor name='${name}_finger_13_contact_sensor' type='contact'>
         <always_on>true</always_on>
@@ -43,16 +50,20 @@
         </plugin>
       </sensor>
+-->
+    </gazebo>
+    <gazebo reference="${name}_finger_21_link">
+      <gravity>true</gravity>
+      <self_collide>false</self_collide>
       <material>Schunk/LightGrey</material>
-    </gazebo-->
-    <gazebo reference="${name}_finger_21_link">
-      <material>Schunk/LightGrey</material>
-      <turnGravityOff>true</turnGravityOff>
-      <mu1 value="500" />
+      <!--mu1 value="500" />
       <mu2 value="500" />
       <kp value="1000000.0" />
-      <kd value="1.0" />
+      <kd value="1.0" /-->
     </gazebo>
-    <!--gazebo reference="${name}_finger_22_link">
-      <selfCollide>true</selfCollide>
+    <gazebo reference="${name}_finger_22_link">
+      <gravity>true</gravity>
+      <self_collide>false</self_collide>
+      <material>Schunk/LightGrey</material>
+<!--
       <sensor name='${name}_finger_22_contact_sensor' type='contact'>
         <always_on>true</always_on>
@@ -68,9 +79,11 @@
         </plugin>
       </sensor>
+-->
+    </gazebo>
+    <gazebo reference="${name}_finger_23_link">
+      <gravity>true</gravity>
+      <self_collide>false</self_collide>
       <material>Schunk/LightGrey</material>
-      <turnGravityOff>false</turnGravityOff>
-    </gazebo-->
-    <!--gazebo reference="${name}_finger_23_link">
-      <selfCollide>true</selfCollide>
+<!--
       <sensor name='${name}_finger_23_contact_sensor' type='contact'>
         <always_on>true</always_on>
@@ -86,12 +99,16 @@
         </plugin>
       </sensor>
+-->
+    </gazebo>
+    <gazebo reference="${name}_thumb_1_link">
+      <gravity>true</gravity>
+      <self_collide>false</self_collide>
       <material>Schunk/LightGrey</material>
-    </gazebo-->
-    <gazebo reference="${name}_thumb_1_link">
+    </gazebo>
+    <gazebo reference="${name}_thumb_2_link">
+      <gravity>true</gravity>
+      <self_collide>false</self_collide>
       <material>Schunk/LightGrey</material>
-      <turnGravityOff>false</turnGravityOff>
-    </gazebo>
-    <!--gazebo reference="${name}_thumb_2_link">
-      <selfCollide>true</selfCollide>
+<!--
       <sensor name='${name}_thumb_2_contact_sensor' type='contact'>
         <always_on>true</always_on>
@@ -107,9 +124,11 @@
         </plugin>
       </sensor>
+-->
+    </gazebo>
+    <gazebo reference="${name}_thumb_3_link">
+      <gravity>true</gravity>
+      <self_collide>false</self_collide>
       <material>Schunk/LightGrey</material>
-      <turnGravityOff>false</turnGravityOff>
-    </gazebo-->
-    <!--gazebo reference="${name}_thumb_3_link">
-      <selfCollide>true</selfCollide>
+<!--
       <sensor name='${name}_thumb_3_contact_sensor' type='contact'>
         <always_on>true</always_on>
@@ -125,12 +144,12 @@
         </plugin>
       </sensor>
-      <material>Schunk/LightGrey</material>
-    </gazebo-->
-    <gazebo reference="${name}_finger_21_joint">
+-->
+    </gazebo>
+    <!--gazebo reference="${name}_finger_21_joint">
       <stopKd value='1.0' />
       <stopKp value='10000000' />
       <fudgeFactor value='1.0' />
       <provideFeedback value="true"/>
-    </gazebo>
+    </gazebo-->
   </xacro:macro>
 </robot>
