Commit message: fix lwa

File: schunk_description/urdf/lwa/lwa.urdf.xacro (robot description, xacro)
@@ -54,12 +54,12 @@
 				<origin xyz="0 0 0" rpy="0 0 0" />
 				<geometry>
-					<mesh filename="package://schunk_description/meshes/lwa/arm1.stl" />
-				</geometry>
-				<material name="Blue" />
-			</visual>
-			<collision>
-				<origin xyz="0 0 0" rpy="0 0 0" />
-				<geometry>
-					<mesh filename="package://schunk_description/meshes/lwa/arm1.stlb" />
+					<mesh filename="package://schunk_description/meshes/lwa/lwa1.stl" />
+				</geometry>
+				<material name="Blue" />
+			</visual>
+			<collision>
+				<origin xyz="0 0 0" rpy="0 0 0" />
+				<geometry>
+					<mesh filename="package://schunk_description/meshes/lwa/lwa1.stlb" />
 				</geometry>
 			</collision>
@@ -86,12 +86,12 @@
 				<origin xyz="0 0 0" rpy="0 0 0" />
 				<geometry>
-					<mesh filename="package://schunk_description/meshes/lwa/arm2.stl" />
-				</geometry>
-				<material name="Red" />
-			</visual>
-			<collision>
-				<origin xyz="0 0 0" rpy="0 0 0" />
-				<geometry>
-					<mesh filename="package://schunk_description/meshes/lwa/arm2.stlb"/>
+					<mesh filename="package://schunk_description/meshes/lwa/lwa2.stl" />
+				</geometry>
+				<material name="Red" />
+			</visual>
+			<collision>
+				<origin xyz="0 0 0" rpy="0 0 0" />
+				<geometry>
+					<mesh filename="package://schunk_description/meshes/lwa/lwa2.stlb"/>
 				</geometry>
 			</collision>
@@ -118,12 +118,12 @@
 				<origin xyz="0 0 0" rpy="0 0 0" />
 				<geometry>
-					<mesh filename="package://schunk_description/meshes/lwa/arm3.stl" />
-				</geometry>
-				<material name="Blue" />
-			</visual>
-			<collision>
-				<origin xyz="0 0 0" rpy="0 0 0" />
-				<geometry>
-					<mesh filename="package://schunk_description/meshes/lwa/arm3.stlb"/>
+					<mesh filename="package://schunk_description/meshes/lwa/lwa3.stl" />
+				</geometry>
+				<material name="Blue" />
+			</visual>
+			<collision>
+				<origin xyz="0 0 0" rpy="0 0 0" />
+				<geometry>
+					<mesh filename="package://schunk_description/meshes/lwa/lwa3.stlb"/>
 				</geometry>
 			</collision>
@@ -150,12 +150,12 @@
 				<origin xyz="0 0 0" rpy="0 0 0" />
 				<geometry>
-					<mesh filename="package://schunk_description/meshes/lwa/arm4.stl" />
-				</geometry>
-				<material name="Red" />
-			</visual>
-			<collision>
-				<origin xyz="0 0 0" rpy="0 0 0" />
-				<geometry>
-					<mesh filename="package://schunk_description/meshes/lwa/arm4.stlb"/>
+					<mesh filename="package://schunk_description/meshes/lwa/lwa4.stl" />
+				</geometry>
+				<material name="Red" />
+			</visual>
+			<collision>
+				<origin xyz="0 0 0" rpy="0 0 0" />
+				<geometry>
+					<mesh filename="package://schunk_description/meshes/lwa/lwa4.stlb"/>
 				</geometry>
 			</collision>
@@ -181,12 +181,12 @@
 				<origin xyz="0 0 0" rpy="0 0 0" />
 				<geometry>
-					<mesh filename="package://schunk_description/meshes/lwa/arm5.stl" />
-				</geometry>
-				<material name="Blue" />
-			</visual>
-			<collision>
-				<origin xyz="0 0 0" rpy="0 0 0" />
-				<geometry>
-					<mesh filename="package://schunk_description/meshes/lwa/arm5.stlb"/>
+					<mesh filename="package://schunk_description/meshes/lwa/lwa5.stl" />
+				</geometry>
+				<material name="Blue" />
+			</visual>
+			<collision>
+				<origin xyz="0 0 0" rpy="0 0 0" />
+				<geometry>
+					<mesh filename="package://schunk_description/meshes/lwa/lwa5.stlb"/>
 				</geometry>
 			</collision>
@@ -212,12 +212,12 @@
 				<origin xyz="0 0 0" rpy="0 0 0" />
 				<geometry>
-					<mesh filename="package://schunk_description/meshes/lwa/arm6.stl" />
-				</geometry>
-				<material name="Red" />
-			</visual>
-			<collision>
-				<origin xyz="0 0 0" rpy="0 0 0" />
-				<geometry>
-					<mesh filename="package://schunk_description/meshes/lwa/arm6.stlb"/>
+					<mesh filename="package://schunk_description/meshes/lwa/lwa6.stl" />
+				</geometry>
+				<material name="Red" />
+			</visual>
+			<collision>
+				<origin xyz="0 0 0" rpy="0 0 0" />
+				<geometry>
+					<mesh filename="package://schunk_description/meshes/lwa/lwa6.stlb"/>
 				</geometry>
 			</collision>
@@ -243,12 +243,12 @@
 				<origin xyz="0 0 0" rpy="0 0 0" />
 				<geometry>
-					<mesh filename="package://schunk_description/meshes/lwa/arm7.stl" />
-				</geometry>
-				<material name="Blue" />
-			</visual>
-			<collision>
-				<origin xyz="0 0 0" rpy="0 0 0" />
-				<geometry>
-					<mesh filename="package://schunk_description/meshes/lwa/arm7.stlb"/>
+					<mesh filename="package://schunk_description/meshes/lwa/lwa7.stl" />
+				</geometry>
+				<material name="Blue" />
+			</visual>
+			<collision>
+				<origin xyz="0 0 0" rpy="0 0 0" />
+				<geometry>
+					<mesh filename="package://schunk_description/meshes/lwa/lwa7.stlb"/>
 				</geometry>
 			</collision>

Commit message: changed stlb links to stl

File: schunk_description/urdf/lwa/lwa.urdf.xacro (robot description, xacro)
@@ -61,5 +61,5 @@
 				<origin xyz="0 0 0" rpy="0 0 0" />
 				<geometry>
-					<mesh filename="package://schunk_description/meshes/lwa/lwa1.stlb" />
+					<mesh filename="package://schunk_description/meshes/lwa/lwa1.stl" />
 				</geometry>
 			</collision>
@@ -93,5 +93,5 @@
 				<origin xyz="0 0 0" rpy="0 0 0" />
 				<geometry>
-					<mesh filename="package://schunk_description/meshes/lwa/lwa2.stlb"/>
+					<mesh filename="package://schunk_description/meshes/lwa/lwa2.stl"/>
 				</geometry>
 			</collision>
@@ -125,5 +125,5 @@
 				<origin xyz="0 0 0" rpy="0 0 0" />
 				<geometry>
-					<mesh filename="package://schunk_description/meshes/lwa/lwa3.stlb"/>
+					<mesh filename="package://schunk_description/meshes/lwa/lwa3.stl"/>
 				</geometry>
 			</collision>
@@ -157,5 +157,5 @@
 				<origin xyz="0 0 0" rpy="0 0 0" />
 				<geometry>
-					<mesh filename="package://schunk_description/meshes/lwa/lwa4.stlb"/>
+					<mesh filename="package://schunk_description/meshes/lwa/lwa4.stl"/>
 				</geometry>
 			</collision>
@@ -188,5 +188,5 @@
 				<origin xyz="0 0 0" rpy="0 0 0" />
 				<geometry>
-					<mesh filename="package://schunk_description/meshes/lwa/lwa5.stlb"/>
+					<mesh filename="package://schunk_description/meshes/lwa/lwa5.stl"/>
 				</geometry>
 			</collision>
@@ -219,5 +219,5 @@
 				<origin xyz="0 0 0" rpy="0 0 0" />
 				<geometry>
-					<mesh filename="package://schunk_description/meshes/lwa/lwa6.stlb"/>
+					<mesh filename="package://schunk_description/meshes/lwa/lwa6.stl"/>
 				</geometry>
 			</collision>
@@ -250,5 +250,5 @@
 				<origin xyz="0 0 0" rpy="0 0 0" />
 				<geometry>
-					<mesh filename="package://schunk_description/meshes/lwa/lwa7.stlb"/>
+					<mesh filename="package://schunk_description/meshes/lwa/lwa7.stl"/>
 				</geometry>
 			</collision>

File: schunk_description/urdf/sdh/sdh.urdf.xacro (robot description, xacro)
@@ -29,5 +29,5 @@
 				<origin xyz="0 0 0" rpy="0 0 0" />
 				<geometry>
-					<mesh filename="package://schunk_description/meshes/sdh/palm.stlb"/>
+					<mesh filename="package://schunk_description/meshes/sdh/palm.stl"/>
 				</geometry>
 			</collision>
@@ -73,5 +73,5 @@
 				<origin xyz="0 0 0" rpy="0 0 0" />
 				<geometry>
-				<mesh filename="package://schunk_description/meshes/sdh/knuckle.stlb"/>
+				<mesh filename="package://schunk_description/meshes/sdh/knuckle.stl"/>
 				</geometry>
 			</collision>
@@ -102,5 +102,5 @@
 				<origin xyz="0 0 0" rpy="0 0 0" />
 				<geometry>
-					<mesh filename="package://schunk_description/meshes/sdh/finger.stlb"/>
+					<mesh filename="package://schunk_description/meshes/sdh/finger.stl"/>
 				</geometry>
 			</collision>
@@ -131,5 +131,5 @@
 				<origin xyz="0 0 0" rpy="0 0 0" />
 				<geometry>
-					<mesh filename="package://schunk_description/meshes/sdh/finger_tip.stlb"/>
+					<mesh filename="package://schunk_description/meshes/sdh/finger_tip.stl"/>
 				</geometry>
 			</collision>
@@ -162,5 +162,5 @@
 				<origin xyz="0 0 0" rpy="0 0 0" />
 				<geometry>
-					<mesh filename="package://schunk_description/meshes/sdh/knuckle.stlb"/>
+					<mesh filename="package://schunk_description/meshes/sdh/knuckle.stl"/>
 				</geometry>
 			</collision>
@@ -191,5 +191,5 @@
 				<origin xyz="0 0 0" rpy="0 0 0" />
 				<geometry>
-					<mesh filename="package://schunk_description/meshes/sdh/finger.stlb"/>
+					<mesh filename="package://schunk_description/meshes/sdh/finger.stl"/>
 				</geometry>
 			</collision>
@@ -220,5 +220,5 @@
 				<origin xyz="0 0 0" rpy="0 0 0" />
 				<geometry>
-					<mesh filename="package://schunk_description/meshes/sdh/finger_tip.stlb"/>
+					<mesh filename="package://schunk_description/meshes/sdh/finger_tip.stl"/>
 				</geometry>
 			</collision>
@@ -247,5 +247,5 @@
 				<origin xyz="0 0 0" rpy="0 0 0" />
 				<geometry>
-					<mesh filename="package://schunk_description/meshes/sdh/knuckle.stlb"/>
+					<mesh filename="package://schunk_description/meshes/sdh/knuckle.stl"/>
 				</geometry>
 			</collision>
@@ -276,5 +276,5 @@
 				<origin xyz="0 0 0" rpy="0 0 0" />
 				<geometry>
-					<mesh filename="package://schunk_description/meshes/sdh/finger.stlb"/>
+					<mesh filename="package://schunk_description/meshes/sdh/finger.stl"/>
 				</geometry>
 			</collision>
@@ -305,5 +305,5 @@
 				<origin xyz="0 0 0" rpy="0 0 0" />
 				<geometry>
-					<mesh filename="package://schunk_description/meshes/sdh/finger_tip.stlb"/>
+					<mesh filename="package://schunk_description/meshes/sdh/finger_tip.stl"/>
 				</geometry>
 			</collision>

Commit message: Renamed the colors

File: schunk_description/urdf/lwa/lwa.urdf.xacro (robot description, xacro)
@@ -24,5 +24,5 @@
 					<cylinder radius="0.045" length="0.08"/>
 				</geometry>
-				<material name="DarkGolden" />
+				<material name="Schunk/DarkGolden" />
 			</visual>
 			<collision>
@@ -56,5 +56,5 @@
 					<mesh filename="package://schunk_description/meshes/lwa/lwa1.stl" />
 				</geometry>
-				<material name="DarkGolden" />
+				<material name="Schunk/DarkGolden" />
 			</visual>
 			<collision>
@@ -88,5 +88,5 @@
 					<mesh filename="package://schunk_description/meshes/lwa/lwa2.stl" />
 				</geometry>
-				<material name="DarkGolden" />
+				<material name="Schunk/DarkGolden" />
 			</visual>
 			<collision>
@@ -120,5 +120,5 @@
 					<mesh filename="package://schunk_description/meshes/lwa/lwa3.stl" />
 				</geometry>
-				<material name="DarkGolden" />
+				<material name="Schunk/DarkGolden" />
 			</visual>
 			<collision>
@@ -152,5 +152,5 @@
 					<mesh filename="package://schunk_description/meshes/lwa/lwa4.stl" />
 				</geometry>
-				<material name="DarkGolden" />
+				<material name="Schunk/DarkGolden" />
 			</visual>
 			<collision>
@@ -183,5 +183,5 @@
 					<mesh filename="package://schunk_description/meshes/lwa/lwa5.stl" />
 				</geometry>
-				<material name="DarkGolden" />
+				<material name="Schunk/DarkGolden" />
 			</visual>
 			<collision>
@@ -214,5 +214,5 @@
 					<mesh filename="package://schunk_description/meshes/lwa/lwa6.stl" />
 				</geometry>
-				<material name="DarkGolden" />
+				<material name="Schunk/DarkGolden" />
 			</visual>
 			<collision>
@@ -245,5 +245,5 @@
 					<mesh filename="package://schunk_description/meshes/lwa/lwa7.stl" />
 				</geometry>
-				<material name="DarkGolden" />
+				<material name="Schunk/DarkGolden" />
 			</visual>
 			<collision>

File: schunk_description/urdf/powerball/powerball.urdf.xacro (robot description, xacro)
@@ -24,5 +24,5 @@
 					<mesh filename="package://schunk_description/meshes/powerball/arm_0_link.stl" />
 				</geometry>
-				<material name="Grey" />
+				<material name="IPA/LightGrey" />
 			</visual>
 			<collision>
@@ -86,5 +86,5 @@
 					<mesh filename="package://schunk_description/meshes/powerball/arm_2_link.stl" />
 				</geometry>
-				<material name="Grey" />
+				<material name="IPA/LightGrey" />
 			</visual>
 			<collision>
@@ -148,5 +148,5 @@
 					<mesh filename="package://schunk_description/meshes/powerball/arm_4_link.stl" />
 				</geometry>
-				<material name="Grey" />
+				<material name="IPA/LightGrey" />
 			</visual>
 			<collision>
@@ -210,5 +210,5 @@
 					<mesh filename="package://schunk_description/meshes/powerball/arm_6_link.stl" />
 				</geometry>
-				<material name="Grey" />
+				<material name="IPA/LightGrey" />
 			</visual>
 			<collision>

File: schunk_description/urdf/sdh/sdh.urdf.xacro (robot description, xacro)
@@ -24,5 +24,5 @@
 					<mesh filename="package://schunk_description/meshes/sdh/palm.stl" />
 				</geometry>
-				<material name="Grey" />
+				<material name="IPA/DarkGrey" />
 			</visual>
 			<collision>
@@ -68,5 +68,5 @@
 					<mesh filename="package://schunk_description/meshes/sdh/knuckle.stl" />
 				</geometry>
-				<material name="Black" />
+				<material name="IPA/Black" />
 			</visual>
 			<collision>
@@ -97,5 +97,5 @@
 					<mesh filename="package://schunk_description/meshes/sdh/finger.stl" />
 				</geometry>
-			<material name="Grey" />
+			<material name="IPA/DarkGrey" />
 			</visual>
 			<collision>
@@ -126,5 +126,5 @@
 					<mesh filename="package://schunk_description/meshes/sdh/finger_tip.stl" />
 				</geometry>
-				<material name="Black" />
+				<material name="IPA/Black" />
 			</visual>
 			<collision>
@@ -157,5 +157,5 @@
 					<mesh filename="package://schunk_description/meshes/sdh/knuckle.stl" />
 				</geometry>
-				<material name="Black" />
+				<material name="IPA/Black" />
 			</visual>
 			<collision>
@@ -186,5 +186,5 @@
 					<mesh filename="package://schunk_description/meshes/sdh/finger.stl" />
 				</geometry>
-				<material name="Grey" />
+				<material name="IPA/DarkGrey" />
 			</visual>
 			<collision>
@@ -215,5 +215,5 @@
 					<mesh filename="package://schunk_description/meshes/sdh/finger_tip.stl" />
 				</geometry>
-				<material name="Black" />
+				<material name="IPA/Black" />
 			</visual>
 			<collision>
@@ -242,5 +242,5 @@
 					<mesh filename="package://schunk_description/meshes/sdh/knuckle.stl" />
 				</geometry>
-				<material name="Black" />
+				<material name="IPA/Black" />
 			</visual>
 			<collision>
@@ -271,5 +271,5 @@
 					<mesh filename="package://schunk_description/meshes/sdh/finger.stl" />
 				</geometry>
-				<material name="Grey" />
+				<material name="IPA/DarkGrey" />
 			</visual>
 			<collision>
@@ -300,5 +300,5 @@
 					<mesh filename="package://schunk_description/meshes/sdh/finger_tip.stl" />
 				</geometry>
-				<material name="Black" />
+				<material name="IPA/Black" />
 			</visual>
 			<collision>

Commit message: update limits for lwa

File: schunk_description/urdf/lwa/lwa.urdf.xacro (robot description, xacro)
@@ -73,6 +73,6 @@
 			<calibration rising="${arm_2_ref}"/>
 			<dynamics damping="10" />
-			<limit effort="370" velocity="2.0" lower="-2.0943951" upper="2.0943951"/>
-			<safety_controller k_position="20" k_velocity="50" soft_lower_limit="${-2.0943 + 0.01}" 	soft_upper_limit="${2.0943 - 0.01}" />
+			<limit effort="370" velocity="2.0" lower="-1.97" upper="1.97"/>
+			<safety_controller k_position="20" k_velocity="50" soft_lower_limit="${-1.97 + 0.01}" 	soft_upper_limit="${1.97 - 0.01}" />
 		</joint>
 		<link name="${name}_2_link">
@@ -137,6 +137,6 @@
 			<calibration rising="${arm_4_ref}"/>
 			<dynamics damping="5" />
-			<limit effort="176" velocity="2.0" lower="-2.0943951" upper="2.0943951"/>
-			<safety_controller k_position="20" k_velocity="25" soft_lower_limit="${-2.0943951 + 0.01}" soft_upper_limit="${2.0943951 - 0.01}" />
+			<limit effort="176" velocity="2.0" lower="-2.08208" upper="2.08208"/>
+			<safety_controller k_position="20" k_velocity="25" soft_lower_limit="${-2.08208 + 0.01}" soft_upper_limit="${2.08208 - 0.01}" />
 		</joint>
 		<link name="${name}_4_link">
@@ -200,6 +200,6 @@
 			<calibration rising="${arm_6_ref}"/>
 			<dynamics damping="5" />
-			<limit effort="20.1" velocity="2.0" lower="-2.0943951" upper="2.0943951" />
-			<safety_controller k_position="20" k_velocity="25" soft_lower_limit="${-2.0943951 + 0.01}" soft_upper_limit="${2.0943951 - 0.01}" />
+			<limit effort="20.1" velocity="2.0" lower="-1.8" upper="1.8" />
+			<safety_controller k_position="20" k_velocity="25" soft_lower_limit="${-1.8 + 0.01}" soft_upper_limit="${1.8 - 0.01}" />
 		</joint>
 		<link name="${name}_6_link">
