Commit message: adapt limits for lwa and lwa_extended

File: schunk_description/urdf/lwa/lwa.urdf.xacro (robot description, xacro)
@@ -41,6 +41,6 @@
 			<calibration rising="${arm_1_ref}"/>
 			<dynamics damping="10" />
-			<limit effort="370" velocity="2.0" lower="-6.2831853" upper="6.2831853"/>
-			<safety_controller k_position="20" k_velocity="50" soft_lower_limit="${-6.2831853 + 0.01}" soft_upper_limit="${6.2831853 - 0.01}" />
+			<limit effort="370" velocity="2.0" lower="-6.25" upper="6.25"/>
+			<safety_controller k_position="20" k_velocity="50" soft_lower_limit="${-6.25 + 0.01}" soft_upper_limit="${6.25 - 0.01}" />
 		</joint>
 		<link name="${name}_1_link">
@@ -105,6 +105,6 @@
 			<calibration rising="${arm_3_ref}"/>
 			<dynamics damping="5" />
-			<limit effort="176" velocity="2.0" lower="-6.2831853" upper="6.2831853"/>
-			<safety_controller k_position="20" k_velocity="25" soft_lower_limit="${-6.2831853 + 0.01}" soft_upper_limit="${6.2831853 - 0.01}" />
+			<limit effort="176" velocity="2.0" lower="-6.25" upper="6.25"/>
+			<safety_controller k_position="20" k_velocity="25" soft_lower_limit="${-6.25 + 0.01}" soft_upper_limit="${6.25 - 0.01}" />
 		</joint>
 		<link name="${name}_3_link">
@@ -137,6 +137,6 @@
 			<calibration rising="${arm_4_ref}"/>
 			<dynamics damping="5" />
-			<limit effort="176" velocity="2.0" lower="-2.08208" upper="2.08208"/>
-			<safety_controller k_position="20" k_velocity="25" soft_lower_limit="${-2.08208 + 0.01}" soft_upper_limit="${2.08208 - 0.01}" />
+			<limit effort="176" velocity="2.0" lower="-1.97" upper="1.97"/>
+			<safety_controller k_position="20" k_velocity="25" soft_lower_limit="${-1.97 + 0.01}" soft_upper_limit="${1.97 - 0.01}" />
 		</joint>
 		<link name="${name}_4_link">
@@ -169,6 +169,6 @@
 			<calibration rising="${arm_5_ref}"/>
 			<dynamics damping="5" />
-			<limit effort="41.6" velocity="2.0" lower="-6.2831853" upper="6.2831853" />
-			<safety_controller k_position="20" k_velocity="25" soft_lower_limit="${-6.2831853 + 0.01}" soft_upper_limit="${6.2831853 - 0.01}" />
+			<limit effort="41.6" velocity="2.0" lower="-6.25" upper="6.25" />
+			<safety_controller k_position="20" k_velocity="25" soft_lower_limit="${-6.25 + 0.01}" soft_upper_limit="${6.25 - 0.01}" />
 		</joint>
 		<link name="${name}_5_link">
@@ -200,6 +200,6 @@
 			<calibration rising="${arm_6_ref}"/>
 			<dynamics damping="5" />
-			<limit effort="20.1" velocity="2.0" lower="-1.8" upper="1.8" />
-			<safety_controller k_position="20" k_velocity="25" soft_lower_limit="${-1.8 + 0.01}" soft_upper_limit="${1.8 - 0.01}" />
+			<limit effort="20.1" velocity="2.0" lower="-1.97" upper="1.97" />
+			<safety_controller k_position="20" k_velocity="25" soft_lower_limit="${-1.97 + 0.01}" soft_upper_limit="${1.97 - 0.01}" />
 		</joint>
 		<link name="${name}_6_link">
@@ -231,6 +231,6 @@
 			<calibration rising="${arm_7_ref}"/>
 			<dynamics damping="5" />
-			<limit effort="9.6" velocity="2.0" lower="-6.2831853" upper="6.2831853" />
-			<safety_controller k_position="20" k_velocity="25" soft_lower_limit="${-6.2831853 + 0.01}" soft_upper_limit="${6.2831853 - 0.01}" />
+			<limit effort="9.6" velocity="2.0" lower="-6.25" upper="6.25" />
+			<safety_controller k_position="20" k_velocity="25" soft_lower_limit="${-6.25 + 0.01}" soft_upper_limit="${6.25 - 0.01}" />
 		</joint>
 		<link name="${name}_7_link">

File: schunk_description/urdf/lwa_extended/lwa_extended.urdf.xacro (robot description, xacro)
@@ -41,6 +41,6 @@
 			<calibration rising="${arm_1_ref}"/>
 			<dynamics damping="10" />
-			<limit effort="370" velocity="2.0" lower="-6.2831853" upper="6.2831853"/>
-			<safety_controller k_position="20" k_velocity="50" soft_lower_limit="${-6.2831853 + 0.01}" soft_upper_limit="${6.2831853 - 0.01}" />
+			<limit effort="370" velocity="2.0" lower="-6.25" upper="6.25"/>
+			<safety_controller k_position="20" k_velocity="50" soft_lower_limit="${-6.25 + 0.01}" soft_upper_limit="${6.25 - 0.01}" />
 		</joint>
 		<link name="${name}_1_link">
@@ -73,6 +73,6 @@
 			<calibration rising="${arm_2_ref}"/>
 			<dynamics damping="10" />
-			<limit effort="370" velocity="2.0" lower="-2.0943951" upper="2.0943951"/>
-			<safety_controller k_position="20" k_velocity="50" soft_lower_limit="${-2.0943 + 0.01}" 	soft_upper_limit="${2.0943 - 0.01}" />
+			<limit effort="370" velocity="2.0" lower="-1.97" upper="1.97"/>
+			<safety_controller k_position="20" k_velocity="50" soft_lower_limit="${-1.97 + 0.01}" 	soft_upper_limit="${1.97 - 0.01}" />
 		</joint>
 		<link name="${name}_2_link">
@@ -105,6 +105,6 @@
 			<calibration rising="${arm_3_ref}"/>
 			<dynamics damping="5" />
-			<limit effort="176" velocity="2.0" lower="-6.2831853" upper="6.2831853"/>
-			<safety_controller k_position="20" k_velocity="25" soft_lower_limit="${-6.2831853 + 0.01}" soft_upper_limit="${6.2831853 - 0.01}" />
+			<limit effort="176" velocity="2.0" lower="-6.25" upper="6.25"/>
+			<safety_controller k_position="20" k_velocity="25" soft_lower_limit="${-6.25 + 0.01}" soft_upper_limit="${6.25 - 0.01}" />
 		</joint>
 		<link name="${name}_3_link">
@@ -137,6 +137,6 @@
 			<calibration rising="${arm_4_ref}"/>
 			<dynamics damping="5" />
-			<limit effort="176" velocity="2.0" lower="-2.0943951" upper="2.0943951"/>
-			<safety_controller k_position="20" k_velocity="25" soft_lower_limit="${-2.0943951 + 0.01}" soft_upper_limit="${2.0943951 - 0.01}" />
+			<limit effort="176" velocity="2.0" lower="-1.97" upper="1.97"/>
+			<safety_controller k_position="20" k_velocity="25" soft_lower_limit="${-1.97 + 0.01}" soft_upper_limit="${1.97 - 0.01}" />
 		</joint>
 		<link name="${name}_4_link">
@@ -169,6 +169,6 @@
 			<calibration rising="${arm_5_ref}"/>
 			<dynamics damping="5" />
-			<limit effort="41.6" velocity="2.0" lower="-6.2831853" upper="6.2831853" />
-			<safety_controller k_position="20" k_velocity="25" soft_lower_limit="${-6.2831853 + 0.01}" soft_upper_limit="${6.2831853 - 0.01}" />
+			<limit effort="41.6" velocity="2.0" lower="-6.25" upper="6.25" />
+			<safety_controller k_position="20" k_velocity="25" soft_lower_limit="${-6.25 + 0.01}" soft_upper_limit="${6.25 - 0.01}" />
 		</joint>
 		<link name="${name}_5_link">
@@ -200,6 +200,6 @@
 			<calibration rising="${arm_6_ref}"/>
 			<dynamics damping="5" />
-			<limit effort="20.1" velocity="2.0" lower="-2.0943951" upper="2.0943951" />
-			<safety_controller k_position="20" k_velocity="25" soft_lower_limit="${-2.0943951 + 0.01}" soft_upper_limit="${2.0943951 - 0.01}" />
+			<limit effort="20.1" velocity="2.0" lower="-1.97" upper="1.97" />
+			<safety_controller k_position="20" k_velocity="25" soft_lower_limit="${-1.97 + 0.01}" soft_upper_limit="${1.97 - 0.01}" />
 		</joint>
 		<link name="${name}_6_link">
@@ -231,6 +231,6 @@
 			<calibration rising="${arm_7_ref}"/>
 			<dynamics damping="5" />
-			<limit effort="9.6" velocity="2.0" lower="-6.2831853" upper="6.2831853" />
-			<safety_controller k_position="20" k_velocity="25" soft_lower_limit="${-6.2831853 + 0.01}" soft_upper_limit="${6.2831853 - 0.01}" />
+			<limit effort="9.6" velocity="2.0" lower="-6.25" upper="6.25" />
+			<safety_controller k_position="20" k_velocity="25" soft_lower_limit="${-6.25 + 0.01}" soft_upper_limit="${6.25 - 0.01}" />
 		</joint>
 		<link name="${name}_7_link">

Commit message: reduce joint limits for moveit

File: schunk_description/urdf/lwa/lwa.urdf.xacro (robot description, xacro)
@@ -34,5 +34,6 @@
       <calibration rising="${arm_1_ref}"/>
       <dynamics damping="10" />
-      <limit effort="370" velocity="2.0" lower="-6.25" upper="6.25"/>
+      <limit effort="370" velocity="2.0" lower="-3.1415" upper="3.1415"/>
+      <!--limit effort="370" velocity="2.0" lower="-6.25" upper="6.25"/-->
       <!--safety_controller k_position="20" k_velocity="50" soft_lower_limit="${-6.25 + 0.01}" soft_upper_limit="${6.25 - 0.01}" /-->
     </joint>
@@ -88,5 +89,6 @@
       <calibration rising="${arm_3_ref}"/>
       <dynamics damping="5" />
-      <limit effort="176" velocity="2.0" lower="-6.25" upper="6.25"/>
+      <limit effort="176" velocity="2.0" lower="-3.1415" upper="3.1415"/>
+      <!--limit effort="176" velocity="2.0" lower="-6.25" upper="6.25"/-->
       <!--safety_controller k_position="20" k_velocity="25" soft_lower_limit="${-6.25 + 0.01}" soft_upper_limit="${6.25 - 0.01}" /-->
     </joint>
@@ -142,5 +144,6 @@
       <calibration rising="${arm_5_ref}"/>
       <dynamics damping="5" />
-      <limit effort="41.6" velocity="2.0" lower="-6.25" upper="6.25" />
+      <limit effort="41.6" velocity="2.0" lower="-3.1415" upper="3.1415" />
+      <!--limit effort="41.6" velocity="2.0" lower="-6.25" upper="6.25" /-->
       <!--safety_controller k_position="20" k_velocity="25" soft_lower_limit="${-6.25 + 0.01}" soft_upper_limit="${6.25 - 0.01}" /-->
     </joint>
@@ -196,5 +199,6 @@
       <calibration rising="${arm_7_ref}"/>
       <dynamics damping="5" />
-      <limit effort="9.6" velocity="2.0" lower="-6.25" upper="6.25" />
+      <limit effort="9.6" velocity="2.0" lower="-3.1415" upper="3.1415" />
+      <!--limit effort="9.6" velocity="2.0" lower="-6.25" upper="6.25" /-->
       <!--safety_controller k_position="20" k_velocity="25" soft_lower_limit="${-6.25 + 0.01}" soft_upper_limit="${6.25 - 0.01}" /-->
     </joint>
