Commit message: update transmission for schunk components

File: schunk_description/urdf/lwa/lwa.transmission.xacro (robot description, xacro)
@@ -2,38 +2,59 @@
 <robot xmlns:xacro="http://www.ros.org/wiki/xacro">
   <xacro:macro name="schunk_lwa_transmission" params="name">
-    <transmission name="${name}_1_trans" type="pr2_mechanism_model/SimpleTransmission">
-      <actuator name="${name}_1_motor"/>
+    <transmission name="${name}_1_trans">
+      <type>transmission_interface/SimpleTransmission</type>
       <joint name="${name}_1_joint"/>
-      <mechanicalReduction>1</mechanicalReduction>
+      <actuator name="${name}_1_motor">
+        <hardwareInterface>EffortJointInterface</hardwareInterface>
+        <mechanicalReduction>1</mechanicalReduction>
+      </actuator>
     </transmission>
-    <transmission name="${name}_2_trans" type="pr2_mechanism_model/SimpleTransmission">
-      <actuator name="${name}_2_motor"/>
+    <transmission name="${name}_2_trans">
+      <type>transmission_interface/SimpleTransmission</type>
       <joint name="${name}_2_joint"/>
-      <mechanicalReduction>1</mechanicalReduction>
+      <actuator name="${name}_2_motor">
+        <hardwareInterface>EffortJointInterface</hardwareInterface>
+        <mechanicalReduction>1</mechanicalReduction>
+      </actuator>
     </transmission>
-    <transmission name="${name}_3_trans" type="pr2_mechanism_model/SimpleTransmission">
-      <actuator name="${name}_3_motor"/>
+    <transmission name="${name}_3_trans">
+      <type>transmission_interface/SimpleTransmission</type>
       <joint name="${name}_3_joint"/>
-      <mechanicalReduction>1</mechanicalReduction>
+      <actuator name="${name}_3_motor">
+        <hardwareInterface>EffortJointInterface</hardwareInterface>
+        <mechanicalReduction>1</mechanicalReduction>
+      </actuator>
     </transmission>
-    <transmission name="${name}_4_trans" type="pr2_mechanism_model/SimpleTransmission">
-      <actuator name="${name}_4_motor"/>
+    <transmission name="${name}_4_trans">
+      <type>transmission_interface/SimpleTransmission</type>
       <joint name="${name}_4_joint"/>
-      <mechanicalReduction>1</mechanicalReduction>
+      <actuator name="${name}_4_motor">
+        <hardwareInterface>EffortJointInterface</hardwareInterface>
+        <mechanicalReduction>1</mechanicalReduction>
+      </actuator>
     </transmission>
-    <transmission name="${name}_5_trans" type="pr2_mechanism_model/SimpleTransmission">
-      <actuator name="${name}_5_motor"/>
+    <transmission name="${name}_5_trans">
+      <type>transmission_interface/SimpleTransmission</type>
       <joint name="${name}_5_joint"/>
-      <mechanicalReduction>1</mechanicalReduction>
+      <actuator name="${name}_5_motor">
+        <hardwareInterface>EffortJointInterface</hardwareInterface>
+        <mechanicalReduction>1</mechanicalReduction>
+      </actuator>
     </transmission>
-    <transmission name="${name}_6_trans" type="pr2_mechanism_model/SimpleTransmission">
-      <actuator name="${name}_6_motor"/>
+    <transmission name="${name}_6_trans">
+      <type>transmission_interface/SimpleTransmission</type>
       <joint name="${name}_6_joint"/>
-      <mechanicalReduction>1</mechanicalReduction>
+      <actuator name="${name}_6_motor">
+        <hardwareInterface>EffortJointInterface</hardwareInterface>
+        <mechanicalReduction>1</mechanicalReduction>
+      </actuator>
     </transmission>
-    <transmission name="${name}_7_trans" type="pr2_mechanism_model/SimpleTransmission">
-      <actuator name="${name}_7_motor"/>
+    <transmission name="${name}_7_trans">
+      <type>transmission_interface/SimpleTransmission</type>
       <joint name="${name}_7_joint"/>
-      <mechanicalReduction>1</mechanicalReduction>
+      <actuator name="${name}_7_motor">
+        <hardwareInterface>EffortJointInterface</hardwareInterface>
+        <mechanicalReduction>1</mechanicalReduction>
+      </actuator>
     </transmission>
   </xacro:macro>

File: schunk_description/urdf/lwa4d/lwa4d.transmission.xacro (robot description, xacro)
@@ -2,38 +2,59 @@
 <robot xmlns:xacro="http://www.ros.org/wiki/xacro">
   <xacro:macro name="schunk_lwa_transmission" params="name">
-    <transmission name="${name}_1_trans" type="pr2_mechanism_model/SimpleTransmission">
-      <actuator name="${name}_1_motor"/>
+    <transmission name="${name}_1_trans">
+      <type>transmission_interface/SimpleTransmission</type>
       <joint name="${name}_1_joint"/>
-      <mechanicalReduction>1</mechanicalReduction>
+      <actuator name="${name}_1_motor">
+        <hardwareInterface>EffortJointInterface</hardwareInterface>
+        <mechanicalReduction>1</mechanicalReduction>
+      </actuator>
     </transmission>
-    <transmission name="${name}_2_trans" type="pr2_mechanism_model/SimpleTransmission">
-      <actuator name="${name}_2_motor"/>
+    <transmission name="${name}_2_trans">
+      <type>transmission_interface/SimpleTransmission</type>
       <joint name="${name}_2_joint"/>
-      <mechanicalReduction>1</mechanicalReduction>
+      <actuator name="${name}_2_motor">
+        <hardwareInterface>EffortJointInterface</hardwareInterface>
+        <mechanicalReduction>1</mechanicalReduction>
+      </actuator>
     </transmission>
-    <transmission name="${name}_3_trans" type="pr2_mechanism_model/SimpleTransmission">
-      <actuator name="${name}_3_motor"/>
+    <transmission name="${name}_3_trans">
+      <type>transmission_interface/SimpleTransmission</type>
       <joint name="${name}_3_joint"/>
-      <mechanicalReduction>1</mechanicalReduction>
+      <actuator name="${name}_3_motor">
+        <hardwareInterface>EffortJointInterface</hardwareInterface>
+        <mechanicalReduction>1</mechanicalReduction>
+      </actuator>
     </transmission>
-    <transmission name="${name}_4_trans" type="pr2_mechanism_model/SimpleTransmission">
-      <actuator name="${name}_4_motor"/>
+    <transmission name="${name}_4_trans">
+      <type>transmission_interface/SimpleTransmission</type>
       <joint name="${name}_4_joint"/>
-      <mechanicalReduction>1</mechanicalReduction>
+      <actuator name="${name}_4_motor">
+        <hardwareInterface>EffortJointInterface</hardwareInterface>
+        <mechanicalReduction>1</mechanicalReduction>
+      </actuator>
     </transmission>
-    <transmission name="${name}_5_trans" type="pr2_mechanism_model/SimpleTransmission">
-      <actuator name="${name}_5_motor"/>
+    <transmission name="${name}_5_trans">
+      <type>transmission_interface/SimpleTransmission</type>
       <joint name="${name}_5_joint"/>
-      <mechanicalReduction>1</mechanicalReduction>
+      <actuator name="${name}_5_motor">
+        <hardwareInterface>EffortJointInterface</hardwareInterface>
+        <mechanicalReduction>1</mechanicalReduction>
+      </actuator>
     </transmission>
-    <transmission name="${name}_6_trans" type="pr2_mechanism_model/SimpleTransmission">
-      <actuator name="${name}_6_motor"/>
+    <transmission name="${name}_6_trans">
+      <type>transmission_interface/SimpleTransmission</type>
       <joint name="${name}_6_joint"/>
-      <mechanicalReduction>1</mechanicalReduction>
+      <actuator name="${name}_6_motor">
+        <hardwareInterface>EffortJointInterface</hardwareInterface>
+        <mechanicalReduction>1</mechanicalReduction>
+      </actuator>
     </transmission>
-    <transmission name="${name}_7_trans" type="pr2_mechanism_model/SimpleTransmission">
-      <actuator name="${name}_7_motor"/>
+    <transmission name="${name}_7_trans">
+      <type>transmission_interface/SimpleTransmission</type>
       <joint name="${name}_7_joint"/>
-      <mechanicalReduction>1</mechanicalReduction>
+      <actuator name="${name}_7_motor">
+        <hardwareInterface>EffortJointInterface</hardwareInterface>
+        <mechanicalReduction>1</mechanicalReduction>
+      </actuator>
     </transmission>
   </xacro:macro>

File: schunk_description/urdf/lwa4p/lwa4p.transmission.xacro (robot description, xacro)
@@ -2,33 +2,51 @@
 <robot xmlns:xacro="http://www.ros.org/wiki/xacro">
   <xacro:macro name="schunk_lwa4p_transmission" params="name">
-    <transmission name="${name}_1_trans" type="pr2_mechanism_model/SimpleTransmission">
-      <actuator name="${name}_1_motor"/>
+    <transmission name="${name}_1_trans">
+      <type>transmission_interface/SimpleTransmission</type>
       <joint name="${name}_1_joint"/>
-      <mechanicalReduction>1</mechanicalReduction>
+      <actuator name="${name}_1_motor">
+        <hardwareInterface>EffortJointInterface</hardwareInterface>
+        <mechanicalReduction>1</mechanicalReduction>
+      </actuator>
     </transmission>
-    <transmission name="${name}_2_trans" type="pr2_mechanism_model/SimpleTransmission">
-      <actuator name="${name}_2_motor"/>
+    <transmission name="${name}_2_trans">
+      <type>transmission_interface/SimpleTransmission</type>
       <joint name="${name}_2_joint"/>
-      <mechanicalReduction>1</mechanicalReduction>
+      <actuator name="${name}_2_motor">
+        <hardwareInterface>EffortJointInterface</hardwareInterface>
+        <mechanicalReduction>1</mechanicalReduction>
+      </actuator>
     </transmission>
-    <transmission name="${name}_3_trans" type="pr2_mechanism_model/SimpleTransmission">
-      <actuator name="${name}_3_motor"/>
+    <transmission name="${name}_3_trans">
+      <type>transmission_interface/SimpleTransmission</type>
       <joint name="${name}_3_joint"/>
-      <mechanicalReduction>1</mechanicalReduction>
+      <actuator name="${name}_3_motor">
+        <hardwareInterface>EffortJointInterface</hardwareInterface>
+        <mechanicalReduction>1</mechanicalReduction>
+      </actuator>
     </transmission>
-    <transmission name="${name}_4_trans" type="pr2_mechanism_model/SimpleTransmission">
-      <actuator name="${name}_4_motor"/>
+    <transmission name="${name}_4_trans">
+      <type>transmission_interface/SimpleTransmission</type>
       <joint name="${name}_4_joint"/>
-      <mechanicalReduction>1</mechanicalReduction>
+      <actuator name="${name}_4_motor">
+        <hardwareInterface>EffortJointInterface</hardwareInterface>
+        <mechanicalReduction>1</mechanicalReduction>
+      </actuator>
     </transmission>
-    <transmission name="${name}_5_trans" type="pr2_mechanism_model/SimpleTransmission">
-      <actuator name="${name}_5_motor"/>
+    <transmission name="${name}_5_trans">
+      <type>transmission_interface/SimpleTransmission</type>
       <joint name="${name}_5_joint"/>
-      <mechanicalReduction>1</mechanicalReduction>
+      <actuator name="${name}_5_motor">
+        <hardwareInterface>EffortJointInterface</hardwareInterface>
+        <mechanicalReduction>1</mechanicalReduction>
+      </actuator>
     </transmission>
-    <transmission name="${name}_6_trans" type="pr2_mechanism_model/SimpleTransmission">
-      <actuator name="${name}_6_motor"/>
+    <transmission name="${name}_6_trans">
+      <type>transmission_interface/SimpleTransmission</type>
       <joint name="${name}_6_joint"/>
-      <mechanicalReduction>1</mechanicalReduction>
+      <actuator name="${name}_6_motor">
+        <hardwareInterface>EffortJointInterface</hardwareInterface>
+        <mechanicalReduction>1</mechanicalReduction>
+      </actuator>
     </transmission>
   </xacro:macro>

File: schunk_description/urdf/lwa_extended/lwa_extended.transmission.xacro (robot description, xacro)
@@ -2,38 +2,59 @@
 <robot xmlns:xacro="http://www.ros.org/wiki/xacro">
   <xacro:macro name="schunk_lwa_extended_transmission" params="name">
-    <transmission name="${name}_1_trans" type="pr2_mechanism_model/SimpleTransmission">
-      <actuator name="${name}_1_motor"/>
+    <transmission name="${name}_1_trans">
+      <type>transmission_interface/SimpleTransmission</type>
       <joint name="${name}_1_joint"/>
-      <mechanicalReduction>1</mechanicalReduction>
+      <actuator name="${name}_1_motor">
+        <hardwareInterface>EffortJointInterface</hardwareInterface>
+        <mechanicalReduction>1</mechanicalReduction>
+      </actuator>
     </transmission>
-    <transmission name="${name}_2_trans" type="pr2_mechanism_model/SimpleTransmission">
-      <actuator name="${name}_2_motor"/>
+    <transmission name="${name}_2_trans">
+      <type>transmission_interface/SimpleTransmission</type>
       <joint name="${name}_2_joint"/>
-      <mechanicalReduction>1</mechanicalReduction>
+      <actuator name="${name}_2_motor">
+        <hardwareInterface>EffortJointInterface</hardwareInterface>
+        <mechanicalReduction>1</mechanicalReduction>
+      </actuator>
     </transmission>
-    <transmission name="${name}_3_trans" type="pr2_mechanism_model/SimpleTransmission">
-      <actuator name="${name}_3_motor"/>
+    <transmission name="${name}_3_trans">
+      <type>transmission_interface/SimpleTransmission</type>
       <joint name="${name}_3_joint"/>
-      <mechanicalReduction>1</mechanicalReduction>
+      <actuator name="${name}_3_motor">
+        <hardwareInterface>EffortJointInterface</hardwareInterface>
+        <mechanicalReduction>1</mechanicalReduction>
+      </actuator>
     </transmission>
-    <transmission name="${name}_4_trans" type="pr2_mechanism_model/SimpleTransmission">
-      <actuator name="${name}_4_motor"/>
+    <transmission name="${name}_4_trans">
+      <type>transmission_interface/SimpleTransmission</type>
       <joint name="${name}_4_joint"/>
-      <mechanicalReduction>1</mechanicalReduction>
+      <actuator name="${name}_4_motor">
+        <hardwareInterface>EffortJointInterface</hardwareInterface>
+        <mechanicalReduction>1</mechanicalReduction>
+      </actuator>
     </transmission>
-    <transmission name="${name}_5_trans" type="pr2_mechanism_model/SimpleTransmission">
-      <actuator name="${name}_5_motor"/>
+    <transmission name="${name}_5_trans">
+      <type>transmission_interface/SimpleTransmission</type>
       <joint name="${name}_5_joint"/>
-      <mechanicalReduction>1</mechanicalReduction>
+      <actuator name="${name}_5_motor">
+        <hardwareInterface>EffortJointInterface</hardwareInterface>
+        <mechanicalReduction>1</mechanicalReduction>
+      </actuator>
     </transmission>
-    <transmission name="${name}_6_trans" type="pr2_mechanism_model/SimpleTransmission">
-      <actuator name="${name}_6_motor"/>
+    <transmission name="${name}_6_trans">
+      <type>transmission_interface/SimpleTransmission</type>
       <joint name="${name}_6_joint"/>
-      <mechanicalReduction>1</mechanicalReduction>
+      <actuator name="${name}_6_motor">
+        <hardwareInterface>EffortJointInterface</hardwareInterface>
+        <mechanicalReduction>1</mechanicalReduction>
+      </actuator>
     </transmission>
-    <transmission name="${name}_7_trans" type="pr2_mechanism_model/SimpleTransmission">
-      <actuator name="${name}_7_motor"/>
+    <transmission name="${name}_7_trans">
+      <type>transmission_interface/SimpleTransmission</type>
       <joint name="${name}_7_joint"/>
-      <mechanicalReduction>1</mechanicalReduction>
+      <actuator name="${name}_7_motor">
+        <hardwareInterface>EffortJointInterface</hardwareInterface>
+        <mechanicalReduction>1</mechanicalReduction>
+      </actuator>
     </transmission>
   </xacro:macro>

File: schunk_description/urdf/sdh/sdh.transmission.xacro (robot description, xacro)
@@ -3,69 +3,69 @@
   <xacro:macro name="schunk_sdh_transmission" params="name">
     <transmission name="${name}_knuckle_trans">
-    <type>transmission_interface/SimpleTransmission</type>
-    <actuator name="${name}_knuckle_motor">
-      <hardwareInterface>EffortJointInterface</hardwareInterface>
-            <mechanicalReduction>1</mechanicalReduction>
-          </actuator>
+      <type>transmission_interface/SimpleTransmission</type>
       <joint name="${name}_finger_21_joint"/>
+      <actuator name="${name}_knuckle_motor">
+        <hardwareInterface>EffortJointInterface</hardwareInterface>
+        <mechanicalReduction>1</mechanicalReduction>
+      </actuator>
     </transmission>
     <transmission name="${name}_knuckle_trans">
-    <type>transmission_interface/SimpleTransmission</type>
+      <type>transmission_interface/SimpleTransmission</type>
+      <joint name="${name}_knuckle_joint"/>
       <actuator name="${name}_knuckle_motor">
         <hardwareInterface>EffortJointInterface</hardwareInterface>
-            <mechanicalReduction>1</mechanicalReduction>
-          </actuator>
-      <joint name="${name}_knuckle_joint"/>
+        <mechanicalReduction>1</mechanicalReduction>
+      </actuator>
     </transmission>
     <!-- finger1 -->
     <transmission name="${name}_finger_12_trans">
-    <type>transmission_interface/SimpleTransmission</type>
+      <type>transmission_interface/SimpleTransmission</type>
+      <joint name="${name}_finger_12_joint"/>
       <actuator name="${name}_finger_12_motor">
-      <hardwareInterface>EffortJointInterface</hardwareInterface>
-            <mechanicalReduction>1</mechanicalReduction>
-          </actuator>
-      <joint name="${name}_finger_12_joint"/>
+        <hardwareInterface>EffortJointInterface</hardwareInterface>
+        <mechanicalReduction>1</mechanicalReduction>
+      </actuator>
     </transmission>
     <transmission name="${name}_finger_13_trans">
-    <type>transmission_interface/SimpleTransmission</type>
+      <type>transmission_interface/SimpleTransmission</type>
+      <joint name="${name}_finger_13_joint"/>
       <actuator name="${name}_finger_13_motor">
-      <hardwareInterface>EffortJointInterface</hardwareInterface>
-            <mechanicalReduction>1</mechanicalReduction>
-          </actuator>
-      <joint name="${name}_finger_13_joint"/>
+        <hardwareInterface>EffortJointInterface</hardwareInterface>
+        <mechanicalReduction>1</mechanicalReduction>
+      </actuator>
     </transmission>
     <!-- finger2 -->
     <transmission name="${name}_finger_22_trans">
-    <type>transmission_interface/SimpleTransmission</type>
+      <type>transmission_interface/SimpleTransmission</type>
+      <joint name="${name}_finger_22_joint"/>
       <actuator name="${name}_finger_22_motor">
-      <hardwareInterface>EffortJointInterface</hardwareInterface>
-            <mechanicalReduction>1</mechanicalReduction>
-          </actuator>
-      <joint name="${name}_finger_22_joint"/>
+        <hardwareInterface>EffortJointInterface</hardwareInterface>
+        <mechanicalReduction>1</mechanicalReduction>
+      </actuator>
     </transmission>
     <transmission name="${name}_finger_23_trans">
-    <type>transmission_interface/SimpleTransmission</type>
+      <type>transmission_interface/SimpleTransmission</type>
+      <joint name="${name}_finger_23_joint"/>
       <actuator name="${name}_finger_23_motor">
-      <hardwareInterface>EffortJointInterface</hardwareInterface>
-            <mechanicalReduction>1</mechanicalReduction>
-          </actuator>
-      <joint name="${name}_finger_23_joint"/>
+        <hardwareInterface>EffortJointInterface</hardwareInterface>
+        <mechanicalReduction>1</mechanicalReduction>
+      </actuator>
     </transmission>
     <!-- thumb -->
     <transmission name="${name}_thumb_2_trans">
-    <type>transmission_interface/SimpleTransmission</type>
+      <type>transmission_interface/SimpleTransmission</type>
+      <joint name="${name}_thumb_2_joint"/>
       <actuator name="${name}_thumb_2_motor">
-      <hardwareInterface>EffortJointInterface</hardwareInterface>
-            <mechanicalReduction>1</mechanicalReduction>
-          </actuator>
-      <joint name="${name}_thumb_2_joint"/>
+        <hardwareInterface>EffortJointInterface</hardwareInterface>
+        <mechanicalReduction>1</mechanicalReduction>
+      </actuator>
     </transmission>
     <transmission name="${name}_thumb_3_trans">
-    <type>transmission_interface/SimpleTransmission</type>
+      <type>transmission_interface/SimpleTransmission</type>
+      <joint name="${name}_thumb_3_joint"/>
       <actuator name="${name}_thumb_3_motor">
-      <hardwareInterface>EffortJointInterface</hardwareInterface>
-            <mechanicalReduction>1</mechanicalReduction>
-          </actuator>
-      <joint name="${name}_thumb_3_joint"/>
+        <hardwareInterface>EffortJointInterface</hardwareInterface>
+        <mechanicalReduction>1</mechanicalReduction>
+      </actuator>
     </transmission>
   </xacro:macro>
