Commit message: modifications in tranmissions, removing of bumpers and small cleanups

File: schunk_description/urdf/lwa/lwa.transmission.xacro (robot description, xacro)
@@ -4,5 +4,7 @@
     <transmission name="${name}_1_trans">
       <type>transmission_interface/SimpleTransmission</type>
-      <joint name="${name}_1_joint"/>
+      <joint name="${name}_1_joint">
+        <hardwareInterface>EffortJointInterface</hardwareInterface>
+      </joint>
       <actuator name="${name}_1_motor">
         <hardwareInterface>EffortJointInterface</hardwareInterface>
@@ -12,5 +14,7 @@
     <transmission name="${name}_2_trans">
       <type>transmission_interface/SimpleTransmission</type>
-      <joint name="${name}_2_joint"/>
+      <joint name="${name}_2_joint">
+        <hardwareInterface>EffortJointInterface</hardwareInterface>
+      </joint>
       <actuator name="${name}_2_motor">
         <hardwareInterface>EffortJointInterface</hardwareInterface>
@@ -20,5 +24,7 @@
     <transmission name="${name}_3_trans">
       <type>transmission_interface/SimpleTransmission</type>
-      <joint name="${name}_3_joint"/>
+      <joint name="${name}_3_joint">
+        <hardwareInterface>EffortJointInterface</hardwareInterface>
+      </joint>
       <actuator name="${name}_3_motor">
         <hardwareInterface>EffortJointInterface</hardwareInterface>
@@ -28,5 +34,7 @@
     <transmission name="${name}_4_trans">
       <type>transmission_interface/SimpleTransmission</type>
-      <joint name="${name}_4_joint"/>
+      <joint name="${name}_4_joint">
+        <hardwareInterface>EffortJointInterface</hardwareInterface>
+      </joint>
       <actuator name="${name}_4_motor">
         <hardwareInterface>EffortJointInterface</hardwareInterface>
@@ -36,5 +44,7 @@
     <transmission name="${name}_5_trans">
       <type>transmission_interface/SimpleTransmission</type>
-      <joint name="${name}_5_joint"/>
+      <joint name="${name}_5_joint">
+        <hardwareInterface>EffortJointInterface</hardwareInterface>
+      </joint>
       <actuator name="${name}_5_motor">
         <hardwareInterface>EffortJointInterface</hardwareInterface>
@@ -44,5 +54,7 @@
     <transmission name="${name}_6_trans">
       <type>transmission_interface/SimpleTransmission</type>
-      <joint name="${name}_6_joint"/>
+      <joint name="${name}_6_joint">
+        <hardwareInterface>EffortJointInterface</hardwareInterface>
+      </joint>
       <actuator name="${name}_6_motor">
         <hardwareInterface>EffortJointInterface</hardwareInterface>
@@ -52,5 +64,7 @@
     <transmission name="${name}_7_trans">
       <type>transmission_interface/SimpleTransmission</type>
-      <joint name="${name}_7_joint"/>
+      <joint name="${name}_7_joint">
+        <hardwareInterface>EffortJointInterface</hardwareInterface>
+      </joint>
       <actuator name="${name}_7_motor">
         <hardwareInterface>EffortJointInterface</hardwareInterface>

File: schunk_description/urdf/lwa4d/lwa4d.transmission.xacro (robot description, xacro)
@@ -4,5 +4,7 @@
     <transmission name="${name}_1_trans">
       <type>transmission_interface/SimpleTransmission</type>
-      <joint name="${name}_1_joint"/>
+      <joint name="${name}_1_joint">
+        <hardwareInterface>EffortJointInterface</hardwareInterface>
+      </joint>
       <actuator name="${name}_1_motor">
         <hardwareInterface>EffortJointInterface</hardwareInterface>
@@ -12,5 +14,7 @@
     <transmission name="${name}_2_trans">
       <type>transmission_interface/SimpleTransmission</type>
-      <joint name="${name}_2_joint"/>
+      <joint name="${name}_2_joint">
+        <hardwareInterface>EffortJointInterface</hardwareInterface>
+      </joint>
       <actuator name="${name}_2_motor">
         <hardwareInterface>EffortJointInterface</hardwareInterface>
@@ -20,5 +24,7 @@
     <transmission name="${name}_3_trans">
       <type>transmission_interface/SimpleTransmission</type>
-      <joint name="${name}_3_joint"/>
+      <joint name="${name}_3_joint">
+        <hardwareInterface>EffortJointInterface</hardwareInterface>
+      </joint>
       <actuator name="${name}_3_motor">
         <hardwareInterface>EffortJointInterface</hardwareInterface>
@@ -28,5 +34,7 @@
     <transmission name="${name}_4_trans">
       <type>transmission_interface/SimpleTransmission</type>
-      <joint name="${name}_4_joint"/>
+      <joint name="${name}_4_joint">
+        <hardwareInterface>EffortJointInterface</hardwareInterface>
+      </joint>
       <actuator name="${name}_4_motor">
         <hardwareInterface>EffortJointInterface</hardwareInterface>
@@ -36,5 +44,7 @@
     <transmission name="${name}_5_trans">
       <type>transmission_interface/SimpleTransmission</type>
-      <joint name="${name}_5_joint"/>
+      <joint name="${name}_5_joint">
+        <hardwareInterface>EffortJointInterface</hardwareInterface>
+      </joint>
       <actuator name="${name}_5_motor">
         <hardwareInterface>EffortJointInterface</hardwareInterface>
@@ -44,5 +54,7 @@
     <transmission name="${name}_6_trans">
       <type>transmission_interface/SimpleTransmission</type>
-      <joint name="${name}_6_joint"/>
+      <joint name="${name}_6_joint">
+        <hardwareInterface>EffortJointInterface</hardwareInterface>
+      </joint>
       <actuator name="${name}_6_motor">
         <hardwareInterface>EffortJointInterface</hardwareInterface>
@@ -52,5 +64,7 @@
     <transmission name="${name}_7_trans">
       <type>transmission_interface/SimpleTransmission</type>
-      <joint name="${name}_7_joint"/>
+      <joint name="${name}_7_joint">
+        <hardwareInterface>EffortJointInterface</hardwareInterface>
+      </joint>
       <actuator name="${name}_7_motor">
         <hardwareInterface>EffortJointInterface</hardwareInterface>

File: schunk_description/urdf/lwa4p/lwa4p.transmission.xacro (robot description, xacro)
@@ -4,5 +4,7 @@
     <transmission name="${name}_1_trans">
       <type>transmission_interface/SimpleTransmission</type>
-      <joint name="${name}_1_joint"/>
+      <joint name="${name}_1_joint">
+        <hardwareInterface>EffortJointInterface</hardwareInterface>
+      </joint>
       <actuator name="${name}_1_motor">
         <hardwareInterface>EffortJointInterface</hardwareInterface>
@@ -12,5 +14,7 @@
     <transmission name="${name}_2_trans">
       <type>transmission_interface/SimpleTransmission</type>
-      <joint name="${name}_2_joint"/>
+      <joint name="${name}_2_joint">
+        <hardwareInterface>EffortJointInterface</hardwareInterface>
+      </joint>
       <actuator name="${name}_2_motor">
         <hardwareInterface>EffortJointInterface</hardwareInterface>
@@ -20,5 +24,7 @@
     <transmission name="${name}_3_trans">
       <type>transmission_interface/SimpleTransmission</type>
-      <joint name="${name}_3_joint"/>
+      <joint name="${name}_3_joint">
+        <hardwareInterface>EffortJointInterface</hardwareInterface>
+      </joint>
       <actuator name="${name}_3_motor">
         <hardwareInterface>EffortJointInterface</hardwareInterface>
@@ -28,5 +34,7 @@
     <transmission name="${name}_4_trans">
       <type>transmission_interface/SimpleTransmission</type>
-      <joint name="${name}_4_joint"/>
+      <joint name="${name}_4_joint">
+        <hardwareInterface>EffortJointInterface</hardwareInterface>
+      </joint>
       <actuator name="${name}_4_motor">
         <hardwareInterface>EffortJointInterface</hardwareInterface>
@@ -36,5 +44,7 @@
     <transmission name="${name}_5_trans">
       <type>transmission_interface/SimpleTransmission</type>
-      <joint name="${name}_5_joint"/>
+      <joint name="${name}_5_joint">
+        <hardwareInterface>EffortJointInterface</hardwareInterface>
+      </joint>
       <actuator name="${name}_5_motor">
         <hardwareInterface>EffortJointInterface</hardwareInterface>
@@ -44,5 +54,7 @@
     <transmission name="${name}_6_trans">
       <type>transmission_interface/SimpleTransmission</type>
-      <joint name="${name}_6_joint"/>
+      <joint name="${name}_6_joint">
+        <hardwareInterface>EffortJointInterface</hardwareInterface>
+      </joint>
       <actuator name="${name}_6_motor">
         <hardwareInterface>EffortJointInterface</hardwareInterface>

File: schunk_description/urdf/lwa4p_extended/lwa4p_extended.transmission.xacro (robot description, xacro)
@@ -4,5 +4,7 @@
     <transmission name="${name}_1_trans">
       <type>transmission_interface/SimpleTransmission</type>
-      <joint name="${name}_1_joint"/>
+      <joint name="${name}_1_joint">
+        <hardwareInterface>EffortJointInterface</hardwareInterface>
+      </joint>
       <actuator name="${name}_1_motor">
         <hardwareInterface>EffortJointInterface</hardwareInterface>
@@ -12,5 +14,7 @@
     <transmission name="${name}_2_trans">
       <type>transmission_interface/SimpleTransmission</type>
-      <joint name="${name}_2_joint"/>
+      <joint name="${name}_2_joint">
+        <hardwareInterface>EffortJointInterface</hardwareInterface>
+      </joint>
       <actuator name="${name}_2_motor">
         <hardwareInterface>EffortJointInterface</hardwareInterface>
@@ -20,5 +24,7 @@
     <transmission name="${name}_3_trans">
       <type>transmission_interface/SimpleTransmission</type>
-      <joint name="${name}_3_joint"/>
+      <joint name="${name}_3_joint">
+        <hardwareInterface>EffortJointInterface</hardwareInterface>
+      </joint>
       <actuator name="${name}_3_motor">
         <hardwareInterface>EffortJointInterface</hardwareInterface>
@@ -28,5 +34,7 @@
     <transmission name="${name}_4_trans">
       <type>transmission_interface/SimpleTransmission</type>
-      <joint name="${name}_4_joint"/>
+      <joint name="${name}_4_joint">
+        <hardwareInterface>EffortJointInterface</hardwareInterface>
+      </joint>
       <actuator name="${name}_4_motor">
         <hardwareInterface>EffortJointInterface</hardwareInterface>
@@ -36,5 +44,7 @@
     <transmission name="${name}_5_trans">
       <type>transmission_interface/SimpleTransmission</type>
-      <joint name="${name}_5_joint"/>
+      <joint name="${name}_5_joint">
+        <hardwareInterface>EffortJointInterface</hardwareInterface>
+      </joint>
       <actuator name="${name}_5_motor">
         <hardwareInterface>EffortJointInterface</hardwareInterface>
@@ -44,5 +54,7 @@
     <transmission name="${name}_6_trans">
       <type>transmission_interface/SimpleTransmission</type>
-      <joint name="${name}_6_joint"/>
+      <joint name="${name}_6_joint">
+        <hardwareInterface>EffortJointInterface</hardwareInterface>
+      </joint>
       <actuator name="${name}_6_motor">
         <hardwareInterface>EffortJointInterface</hardwareInterface>
@@ -52,5 +64,7 @@
     <transmission name="${name}_7_trans">
       <type>transmission_interface/SimpleTransmission</type>
-      <joint name="${name}_7_joint"/>
+      <joint name="${name}_7_joint">
+        <hardwareInterface>EffortJointInterface</hardwareInterface>
+      </joint>
       <actuator name="${name}_7_motor">
         <hardwareInterface>EffortJointInterface</hardwareInterface>

File: schunk_description/urdf/lwa_extended/lwa_extended.transmission.xacro (robot description, xacro)
@@ -4,5 +4,7 @@
     <transmission name="${name}_1_trans">
       <type>transmission_interface/SimpleTransmission</type>
-      <joint name="${name}_1_joint"/>
+      <joint name="${name}_1_joint">
+        <hardwareInterface>EffortJointInterface</hardwareInterface>
+      </joint>
       <actuator name="${name}_1_motor">
         <hardwareInterface>EffortJointInterface</hardwareInterface>
@@ -12,5 +14,7 @@
     <transmission name="${name}_2_trans">
       <type>transmission_interface/SimpleTransmission</type>
-      <joint name="${name}_2_joint"/>
+      <joint name="${name}_2_joint">
+        <hardwareInterface>EffortJointInterface</hardwareInterface>
+      </joint>
       <actuator name="${name}_2_motor">
         <hardwareInterface>EffortJointInterface</hardwareInterface>
@@ -20,5 +24,7 @@
     <transmission name="${name}_3_trans">
       <type>transmission_interface/SimpleTransmission</type>
-      <joint name="${name}_3_joint"/>
+      <joint name="${name}_3_joint">
+        <hardwareInterface>EffortJointInterface</hardwareInterface>
+      </joint>
       <actuator name="${name}_3_motor">
         <hardwareInterface>EffortJointInterface</hardwareInterface>
@@ -28,5 +34,7 @@
     <transmission name="${name}_4_trans">
       <type>transmission_interface/SimpleTransmission</type>
-      <joint name="${name}_4_joint"/>
+      <joint name="${name}_4_joint">
+        <hardwareInterface>EffortJointInterface</hardwareInterface>
+      </joint>
       <actuator name="${name}_4_motor">
         <hardwareInterface>EffortJointInterface</hardwareInterface>
@@ -36,5 +44,7 @@
     <transmission name="${name}_5_trans">
       <type>transmission_interface/SimpleTransmission</type>
-      <joint name="${name}_5_joint"/>
+      <joint name="${name}_5_joint">
+        <hardwareInterface>EffortJointInterface</hardwareInterface>
+      </joint>
       <actuator name="${name}_5_motor">
         <hardwareInterface>EffortJointInterface</hardwareInterface>
@@ -44,5 +54,7 @@
     <transmission name="${name}_6_trans">
       <type>transmission_interface/SimpleTransmission</type>
-      <joint name="${name}_6_joint"/>
+      <joint name="${name}_6_joint">
+        <hardwareInterface>EffortJointInterface</hardwareInterface>
+      </joint>
       <actuator name="${name}_6_motor">
         <hardwareInterface>EffortJointInterface</hardwareInterface>
@@ -52,5 +64,7 @@
     <transmission name="${name}_7_trans">
       <type>transmission_interface/SimpleTransmission</type>
-      <joint name="${name}_7_joint"/>
+      <joint name="${name}_7_joint">
+        <hardwareInterface>EffortJointInterface</hardwareInterface>
+      </joint>
       <actuator name="${name}_7_motor">
         <hardwareInterface>EffortJointInterface</hardwareInterface>

File: schunk_description/urdf/pg70/pg70.transmission.xacro (robot description, xacro)
@@ -5,5 +5,7 @@
     <transmission name="${name}_finger_trans">
       <type>transmission_interface/SimpleTransmission</type>
-      <joint name="${name}_finger_joint"/>
+      <joint name="${name}_finger_joint">
+        <hardwareInterface>EffortJointInterface</hardwareInterface>
+      </joint>
       <actuator name="${name}_finger_motor">
         <hardwareInterface>EffortJointInterface</hardwareInterface>
@@ -14,5 +16,7 @@
     <transmission name="${name}_finger_mimic_trans">
       <type>transmission_interface/SimpleTransmission</type>
-      <joint name="${name}_finger_mimic_joint"/>
+      <joint name="${name}_finger_mimic_joint">
+        <hardwareInterface>EffortJointInterface</hardwareInterface>
+      </joint>
       <actuator name="${name}_finger_mimic_motor">
         <hardwareInterface>EffortJointInterface</hardwareInterface>

File: schunk_description/urdf/sdh/sdh.gazebo.xacro (robot description, xacro)
@@ -10,5 +10,5 @@
       <turnGravityOff>false</turnGravityOff>
     </gazebo>
-    <gazebo reference="${name}_finger_12_link">
+    <!--gazebo reference="${name}_finger_12_link">
       <selfCollide>true</selfCollide>
       <sensor name='${name}_finger_12_contact_sensor' type='contact'>
@@ -27,6 +27,6 @@
       <material>Schunk/LightGrey</material>
       <turnGravityOff>false</turnGravityOff>
-    </gazebo>
-    <gazebo reference="${name}_finger_13_link">
+    </gazebo-->
+    <!--gazebo reference="${name}_finger_13_link">
       <selfCollide>true</selfCollide>
       <sensor name='${name}_finger_13_contact_sensor' type='contact'>
@@ -44,5 +44,5 @@
       </sensor>
       <material>Schunk/LightGrey</material>
-    </gazebo>
+    </gazebo-->
     <gazebo reference="${name}_finger_21_link">
       <material>Schunk/LightGrey</material>
@@ -53,5 +53,5 @@
       <kd value="1.0" />
     </gazebo>
-    <gazebo reference="${name}_finger_22_link">
+    <!--gazebo reference="${name}_finger_22_link">
       <selfCollide>true</selfCollide>
       <sensor name='${name}_finger_22_contact_sensor' type='contact'>
@@ -70,6 +70,6 @@
       <material>Schunk/LightGrey</material>
       <turnGravityOff>false</turnGravityOff>
-    </gazebo>
-    <gazebo reference="${name}_finger_23_link">
+    </gazebo-->
+    <!--gazebo reference="${name}_finger_23_link">
       <selfCollide>true</selfCollide>
       <sensor name='${name}_finger_23_contact_sensor' type='contact'>
@@ -87,10 +87,10 @@
       </sensor>
       <material>Schunk/LightGrey</material>
-    </gazebo>
+    </gazebo-->
     <gazebo reference="${name}_thumb_1_link">
       <material>Schunk/LightGrey</material>
       <turnGravityOff>false</turnGravityOff>
     </gazebo>
-    <gazebo reference="${name}_thumb_2_link">
+    <!--gazebo reference="${name}_thumb_2_link">
       <selfCollide>true</selfCollide>
       <sensor name='${name}_thumb_2_contact_sensor' type='contact'>
@@ -109,6 +109,6 @@
       <material>Schunk/LightGrey</material>
       <turnGravityOff>false</turnGravityOff>
-    </gazebo>
-    <gazebo reference="${name}_thumb_3_link">
+    </gazebo-->
+    <!--gazebo reference="${name}_thumb_3_link">
       <selfCollide>true</selfCollide>
       <sensor name='${name}_thumb_3_contact_sensor' type='contact'>
@@ -126,5 +126,5 @@
       </sensor>
       <material>Schunk/LightGrey</material>
-    </gazebo>
+    </gazebo-->
     <gazebo reference="${name}_finger_21_joint">
       <stopKd value='1.0' />

File: schunk_description/urdf/sdh/sdh.transmission.xacro (robot description, xacro)
@@ -4,5 +4,7 @@
     <transmission name="${name}_knuckle_trans">
       <type>transmission_interface/SimpleTransmission</type>
-      <joint name="${name}_finger_21_joint"/>
+      <joint name="${name}_finger_21_joint">
+        <hardwareInterface>EffortJointInterface</hardwareInterface>
+      </joint>
       <actuator name="${name}_knuckle_motor">
         <hardwareInterface>EffortJointInterface</hardwareInterface>
@@ -12,5 +14,7 @@
     <transmission name="${name}_knuckle_trans">
       <type>transmission_interface/SimpleTransmission</type>
-      <joint name="${name}_knuckle_joint"/>
+      <joint name="${name}_knuckle_joint">
+        <hardwareInterface>EffortJointInterface</hardwareInterface>
+      </joint>
       <actuator name="${name}_knuckle_motor">
         <hardwareInterface>EffortJointInterface</hardwareInterface>
@@ -21,5 +25,7 @@
     <transmission name="${name}_finger_12_trans">
       <type>transmission_interface/SimpleTransmission</type>
-      <joint name="${name}_finger_12_joint"/>
+      <joint name="${name}_finger_12_joint">
+        <hardwareInterface>EffortJointInterface</hardwareInterface>
+      </joint>
       <actuator name="${name}_finger_12_motor">
         <hardwareInterface>EffortJointInterface</hardwareInterface>
@@ -29,5 +35,7 @@
     <transmission name="${name}_finger_13_trans">
       <type>transmission_interface/SimpleTransmission</type>
-      <joint name="${name}_finger_13_joint"/>
+      <joint name="${name}_finger_13_joint">
+        <hardwareInterface>EffortJointInterface</hardwareInterface>
+      </joint>
       <actuator name="${name}_finger_13_motor">
         <hardwareInterface>EffortJointInterface</hardwareInterface>
@@ -38,5 +46,7 @@
     <transmission name="${name}_finger_22_trans">
       <type>transmission_interface/SimpleTransmission</type>
-      <joint name="${name}_finger_22_joint"/>
+      <joint name="${name}_finger_22_joint">
+        <hardwareInterface>EffortJointInterface</hardwareInterface>
+      </joint>
       <actuator name="${name}_finger_22_motor">
         <hardwareInterface>EffortJointInterface</hardwareInterface>
@@ -46,5 +56,7 @@
     <transmission name="${name}_finger_23_trans">
       <type>transmission_interface/SimpleTransmission</type>
-      <joint name="${name}_finger_23_joint"/>
+      <joint name="${name}_finger_23_joint">
+        <hardwareInterface>EffortJointInterface</hardwareInterface>
+      </joint>
       <actuator name="${name}_finger_23_motor">
         <hardwareInterface>EffortJointInterface</hardwareInterface>
@@ -55,5 +67,7 @@
     <transmission name="${name}_thumb_2_trans">
       <type>transmission_interface/SimpleTransmission</type>
-      <joint name="${name}_thumb_2_joint"/>
+      <joint name="${name}_thumb_2_joint">
+        <hardwareInterface>EffortJointInterface</hardwareInterface>
+      </joint>
       <actuator name="${name}_thumb_2_motor">
         <hardwareInterface>EffortJointInterface</hardwareInterface>
@@ -63,5 +77,7 @@
     <transmission name="${name}_thumb_3_trans">
       <type>transmission_interface/SimpleTransmission</type>
-      <joint name="${name}_thumb_3_joint"/>
+      <joint name="${name}_thumb_3_joint">
+        <hardwareInterface>EffortJointInterface</hardwareInterface>
+      </joint>
       <actuator name="${name}_thumb_3_motor">
         <hardwareInterface>EffortJointInterface</hardwareInterface>
