Commit message: consistency changes due to new transmission format

File: schunk_description/urdf/lwa/lwa.transmission.xacro (robot description, xacro)
@@ -8,5 +8,4 @@
       </joint>
       <actuator name="${name}_1_motor">
-        <hardwareInterface>EffortJointInterface</hardwareInterface>
         <mechanicalReduction>1</mechanicalReduction>
       </actuator>
@@ -18,5 +17,4 @@
       </joint>
       <actuator name="${name}_2_motor">
-        <hardwareInterface>EffortJointInterface</hardwareInterface>
         <mechanicalReduction>1</mechanicalReduction>
       </actuator>
@@ -28,5 +26,4 @@
       </joint>
       <actuator name="${name}_3_motor">
-        <hardwareInterface>EffortJointInterface</hardwareInterface>
         <mechanicalReduction>1</mechanicalReduction>
       </actuator>
@@ -38,5 +35,4 @@
       </joint>
       <actuator name="${name}_4_motor">
-        <hardwareInterface>EffortJointInterface</hardwareInterface>
         <mechanicalReduction>1</mechanicalReduction>
       </actuator>
@@ -48,5 +44,4 @@
       </joint>
       <actuator name="${name}_5_motor">
-        <hardwareInterface>EffortJointInterface</hardwareInterface>
         <mechanicalReduction>1</mechanicalReduction>
       </actuator>
@@ -58,5 +53,4 @@
       </joint>
       <actuator name="${name}_6_motor">
-        <hardwareInterface>EffortJointInterface</hardwareInterface>
         <mechanicalReduction>1</mechanicalReduction>
       </actuator>
@@ -68,5 +62,4 @@
       </joint>
       <actuator name="${name}_7_motor">
-        <hardwareInterface>EffortJointInterface</hardwareInterface>
         <mechanicalReduction>1</mechanicalReduction>
       </actuator>

File: schunk_description/urdf/lwa4d/lwa4d.transmission.xacro (robot description, xacro)
@@ -8,5 +8,4 @@
       </joint>
       <actuator name="${name}_1_motor">
-        <hardwareInterface>EffortJointInterface</hardwareInterface>
         <mechanicalReduction>1</mechanicalReduction>
       </actuator>
@@ -18,5 +17,4 @@
       </joint>
       <actuator name="${name}_2_motor">
-        <hardwareInterface>EffortJointInterface</hardwareInterface>
         <mechanicalReduction>1</mechanicalReduction>
       </actuator>
@@ -28,5 +26,4 @@
       </joint>
       <actuator name="${name}_3_motor">
-        <hardwareInterface>EffortJointInterface</hardwareInterface>
         <mechanicalReduction>1</mechanicalReduction>
       </actuator>
@@ -38,5 +35,4 @@
       </joint>
       <actuator name="${name}_4_motor">
-        <hardwareInterface>EffortJointInterface</hardwareInterface>
         <mechanicalReduction>1</mechanicalReduction>
       </actuator>
@@ -48,5 +44,4 @@
       </joint>
       <actuator name="${name}_5_motor">
-        <hardwareInterface>EffortJointInterface</hardwareInterface>
         <mechanicalReduction>1</mechanicalReduction>
       </actuator>
@@ -58,5 +53,4 @@
       </joint>
       <actuator name="${name}_6_motor">
-        <hardwareInterface>EffortJointInterface</hardwareInterface>
         <mechanicalReduction>1</mechanicalReduction>
       </actuator>
@@ -68,5 +62,4 @@
       </joint>
       <actuator name="${name}_7_motor">
-        <hardwareInterface>EffortJointInterface</hardwareInterface>
         <mechanicalReduction>1</mechanicalReduction>
       </actuator>

File: schunk_description/urdf/lwa4p/lwa4p.transmission.xacro (robot description, xacro)
@@ -8,5 +8,4 @@
       </joint>
       <actuator name="${name}_1_motor">
-        <hardwareInterface>EffortJointInterface</hardwareInterface>
         <mechanicalReduction>1</mechanicalReduction>
       </actuator>
@@ -18,5 +17,4 @@
       </joint>
       <actuator name="${name}_2_motor">
-        <hardwareInterface>EffortJointInterface</hardwareInterface>
         <mechanicalReduction>1</mechanicalReduction>
       </actuator>
@@ -28,5 +26,4 @@
       </joint>
       <actuator name="${name}_3_motor">
-        <hardwareInterface>EffortJointInterface</hardwareInterface>
         <mechanicalReduction>1</mechanicalReduction>
       </actuator>
@@ -38,5 +35,4 @@
       </joint>
       <actuator name="${name}_4_motor">
-        <hardwareInterface>EffortJointInterface</hardwareInterface>
         <mechanicalReduction>1</mechanicalReduction>
       </actuator>
@@ -48,5 +44,4 @@
       </joint>
       <actuator name="${name}_5_motor">
-        <hardwareInterface>EffortJointInterface</hardwareInterface>
         <mechanicalReduction>1</mechanicalReduction>
       </actuator>
@@ -58,5 +53,4 @@
       </joint>
       <actuator name="${name}_6_motor">
-        <hardwareInterface>EffortJointInterface</hardwareInterface>
         <mechanicalReduction>1</mechanicalReduction>
       </actuator>

File: schunk_description/urdf/lwa4p_extended/lwa4p_extended.transmission.xacro (robot description, xacro)
@@ -4,7 +4,8 @@
     <transmission name="${jname}_${number}_trans">
       <type>transmission_interface/SimpleTransmission</type>
-      <joint name="${jname}_${number}_joint"/>
+      <joint name="${jname}_${number}_joint">
+        <hardwareInterface>EffortJointInterface</hardwareInterface>
+      </joint>
       <actuator name="${jname}_${number}_motor">
-        <hardwareInterface>EffortJointInterface</hardwareInterface>
         <mechanicalReduction>1</mechanicalReduction>
       </actuator>

File: schunk_description/urdf/lwa_extended/lwa_extended.transmission.xacro (robot description, xacro)
@@ -8,5 +8,4 @@
       </joint>
       <actuator name="${name}_1_motor">
-        <hardwareInterface>EffortJointInterface</hardwareInterface>
         <mechanicalReduction>1</mechanicalReduction>
       </actuator>
@@ -18,5 +17,4 @@
       </joint>
       <actuator name="${name}_2_motor">
-        <hardwareInterface>EffortJointInterface</hardwareInterface>
         <mechanicalReduction>1</mechanicalReduction>
       </actuator>
@@ -28,5 +26,4 @@
       </joint>
       <actuator name="${name}_3_motor">
-        <hardwareInterface>EffortJointInterface</hardwareInterface>
         <mechanicalReduction>1</mechanicalReduction>
       </actuator>
@@ -38,5 +35,4 @@
       </joint>
       <actuator name="${name}_4_motor">
-        <hardwareInterface>EffortJointInterface</hardwareInterface>
         <mechanicalReduction>1</mechanicalReduction>
       </actuator>
@@ -48,5 +44,4 @@
       </joint>
       <actuator name="${name}_5_motor">
-        <hardwareInterface>EffortJointInterface</hardwareInterface>
         <mechanicalReduction>1</mechanicalReduction>
       </actuator>
@@ -58,5 +53,4 @@
       </joint>
       <actuator name="${name}_6_motor">
-        <hardwareInterface>EffortJointInterface</hardwareInterface>
         <mechanicalReduction>1</mechanicalReduction>
       </actuator>
@@ -68,5 +62,4 @@
       </joint>
       <actuator name="${name}_7_motor">
-        <hardwareInterface>EffortJointInterface</hardwareInterface>
         <mechanicalReduction>1</mechanicalReduction>
       </actuator>

File: schunk_description/urdf/pg70/pg70.transmission.xacro (robot description, xacro)
@@ -9,5 +9,4 @@
       </joint>
       <actuator name="${name}_finger_motor">
-        <hardwareInterface>EffortJointInterface</hardwareInterface>
         <mechanicalReduction>1</mechanicalReduction>
       </actuator>
@@ -20,5 +19,4 @@
       </joint>
       <actuator name="${name}_finger_mimic_motor">
-        <hardwareInterface>EffortJointInterface</hardwareInterface>
         <mechanicalReduction>1</mechanicalReduction>
       </actuator>

File: schunk_description/urdf/sdh/sdh.transmission.xacro (robot description, xacro)
@@ -8,5 +8,4 @@
       </joint>
       <actuator name="${name}_knuckle_motor">
-        <hardwareInterface>EffortJointInterface</hardwareInterface>
         <mechanicalReduction>1</mechanicalReduction>
       </actuator>
@@ -18,5 +17,4 @@
       </joint>
       <actuator name="${name}_knuckle_motor">
-        <hardwareInterface>EffortJointInterface</hardwareInterface>
         <mechanicalReduction>1</mechanicalReduction>
       </actuator>
@@ -29,5 +27,4 @@
       </joint>
       <actuator name="${name}_finger_12_motor">
-        <hardwareInterface>EffortJointInterface</hardwareInterface>
         <mechanicalReduction>1</mechanicalReduction>
       </actuator>
@@ -39,5 +36,4 @@
       </joint>
       <actuator name="${name}_finger_13_motor">
-        <hardwareInterface>EffortJointInterface</hardwareInterface>
         <mechanicalReduction>1</mechanicalReduction>
       </actuator>
@@ -50,5 +46,4 @@
       </joint>
       <actuator name="${name}_finger_22_motor">
-        <hardwareInterface>EffortJointInterface</hardwareInterface>
         <mechanicalReduction>1</mechanicalReduction>
       </actuator>
@@ -60,5 +55,4 @@
       </joint>
       <actuator name="${name}_finger_23_motor">
-        <hardwareInterface>EffortJointInterface</hardwareInterface>
         <mechanicalReduction>1</mechanicalReduction>
       </actuator>
@@ -71,5 +65,4 @@
       </joint>
       <actuator name="${name}_thumb_2_motor">
-        <hardwareInterface>EffortJointInterface</hardwareInterface>
         <mechanicalReduction>1</mechanicalReduction>
       </actuator>
@@ -81,5 +74,4 @@
       </joint>
       <actuator name="${name}_thumb_3_motor">
-        <hardwareInterface>EffortJointInterface</hardwareInterface>
         <mechanicalReduction>1</mechanicalReduction>
       </actuator>

Commit message: allow cob3 components to be used with PositionJointInterface

File: schunk_description/urdf/lwa/lwa.transmission.xacro (robot description, xacro)
@@ -5,5 +5,5 @@
       <type>transmission_interface/SimpleTransmission</type>
       <joint name="${name}_1_joint">
-        <hardwareInterface>EffortJointInterface</hardwareInterface>
+        <hardwareInterface>PositionJointInterface</hardwareInterface>
       </joint>
       <actuator name="${name}_1_motor">
@@ -14,5 +14,5 @@
       <type>transmission_interface/SimpleTransmission</type>
       <joint name="${name}_2_joint">
-        <hardwareInterface>EffortJointInterface</hardwareInterface>
+        <hardwareInterface>PositionJointInterface</hardwareInterface>
       </joint>
       <actuator name="${name}_2_motor">
@@ -23,5 +23,5 @@
       <type>transmission_interface/SimpleTransmission</type>
       <joint name="${name}_3_joint">
-        <hardwareInterface>EffortJointInterface</hardwareInterface>
+        <hardwareInterface>PositionJointInterface</hardwareInterface>
       </joint>
       <actuator name="${name}_3_motor">
@@ -32,5 +32,5 @@
       <type>transmission_interface/SimpleTransmission</type>
       <joint name="${name}_4_joint">
-        <hardwareInterface>EffortJointInterface</hardwareInterface>
+        <hardwareInterface>PositionJointInterface</hardwareInterface>
       </joint>
       <actuator name="${name}_4_motor">
@@ -41,5 +41,5 @@
       <type>transmission_interface/SimpleTransmission</type>
       <joint name="${name}_5_joint">
-        <hardwareInterface>EffortJointInterface</hardwareInterface>
+        <hardwareInterface>PositionJointInterface</hardwareInterface>
       </joint>
       <actuator name="${name}_5_motor">
@@ -50,5 +50,5 @@
       <type>transmission_interface/SimpleTransmission</type>
       <joint name="${name}_6_joint">
-        <hardwareInterface>EffortJointInterface</hardwareInterface>
+        <hardwareInterface>PositionJointInterface</hardwareInterface>
       </joint>
       <actuator name="${name}_6_motor">
@@ -59,5 +59,5 @@
       <type>transmission_interface/SimpleTransmission</type>
       <joint name="${name}_7_joint">
-        <hardwareInterface>EffortJointInterface</hardwareInterface>
+        <hardwareInterface>PositionJointInterface</hardwareInterface>
       </joint>
       <actuator name="${name}_7_motor">

File: schunk_description/urdf/lwa/lwa.urdf.xacro (robot description, xacro)
@@ -5,15 +5,11 @@
   <xacro:macro name="schunk_lwa" params="parent name *origin">
     <!-- joint between base_link and arm_0_link -->
-    <joint name="${name}_0_joint" type="fixed" >
+    <joint name="${name}_base_joint" type="fixed" >
       <insert_block name="origin" />
       <parent link="${parent}" />
-      <child link="${name}_0_link" />
-    </joint>
-    <link name="${name}_0_link">
-      <inertial>
-        <origin xyz="0 0 0" rpy="0 0 0"/>
-        <mass value="1.0"/>
-        <inertia ixx="0.01" ixy="0" ixz="0" iyy="0.01" iyz="0" izz="0.01" />
-      </inertial>
+      <child link="${name}_base_link" />
+    </joint>
+    <link name="${name}_base_link">
+      <xacro:default_inertial/>
       <visual>
         <origin xyz="0 0 0.004" rpy="0 0 0" />
@@ -33,5 +29,5 @@
     <joint name="${name}_1_joint" type="revolute">
       <origin xyz="0 0 -0.250" rpy="0 0 3.1415926"/>
-      <parent link="${name}_0_link"/>
+      <parent link="${name}_base_link"/>
       <child link="${name}_1_link"/>
       <axis xyz="0 0 1"/>
@@ -39,13 +35,8 @@
       <dynamics damping="10" />
       <limit effort="370" velocity="2.0" lower="-6.25" upper="6.25"/>
-      <safety_controller k_position="20" k_velocity="50" soft_lower_limit="${-6.25 + 0.01}" soft_upper_limit="${6.25 - 0.01}" />
+      <!--safety_controller k_position="20" k_velocity="50" soft_lower_limit="${-6.25 + 0.01}" soft_upper_limit="${6.25 - 0.01}" /-->
     </joint>
     <link name="${name}_1_link">
-      <inertial>
-        <origin xyz="0 0 0" rpy="0 0 0" />
-        <!--mass value="5.9907"/-->
-        <mass value="2.0"/>
-        <inertia ixx="0.01" ixy="0" ixz="0" iyy="0.01" iyz="0" izz="0.01" />
-      </inertial>
+      <xacro:default_inertial/>
       <visual>
         <origin xyz="0 0 0" rpy="0 0 0" />
@@ -71,13 +62,8 @@
       <dynamics damping="10" />
       <limit effort="370" velocity="2.0" lower="-1.97" upper="1.97"/>
-      <safety_controller k_position="20" k_velocity="50" soft_lower_limit="${-1.97 + 0.01}"   soft_upper_limit="${1.97 - 0.01}" />
+      <!--safety_controller k_position="20" k_velocity="50" soft_lower_limit="${-1.97 + 0.01}"   soft_upper_limit="${1.97 - 0.01}" /-->
     </joint>
     <link name="${name}_2_link">
-      <inertial>
-        <origin xyz="0 0 0" rpy="0 0 0"/>
-        <!--mass value="5.734939"/-->
-        <mass value="2.0"/>
-        <inertia ixx="0.03" ixy="0" ixz="0" iyy="0.03" iyz="0" izz="0.03" />
-      </inertial>
+      <xacro:default_inertial/>
       <visual>
         <origin xyz="0 0 0" rpy="0 0 0" />
@@ -103,13 +89,8 @@
       <dynamics damping="5" />
       <limit effort="176" velocity="2.0" lower="-6.25" upper="6.25"/>
-      <safety_controller k_position="20" k_velocity="25" soft_lower_limit="${-6.25 + 0.01}" soft_upper_limit="${6.25 - 0.01}" />
+      <!--safety_controller k_position="20" k_velocity="25" soft_lower_limit="${-6.25 + 0.01}" soft_upper_limit="${6.25 - 0.01}" /-->
     </joint>
     <link name="${name}_3_link">
-      <inertial>
-        <origin xyz="0 0 0" rpy="0 0 0"/>
-        <!--mass value="4.214668"/-->
-        <mass value="2.0"/>
-        <inertia ixx="0.03" ixy="0" ixz="0" iyy="0.03" iyz="0" izz="0.03" />
-      </inertial>
+      <xacro:default_inertial/>
       <visual>
         <origin xyz="0 0 0" rpy="0 0 0" />
@@ -135,13 +116,8 @@
       <dynamics damping="5" />
       <limit effort="176" velocity="2.0" lower="-1.97" upper="1.97"/>
-      <safety_controller k_position="20" k_velocity="25" soft_lower_limit="${-1.97 + 0.01}" soft_upper_limit="${1.97 - 0.01}" />
+      <!--safety_controller k_position="20" k_velocity="25" soft_lower_limit="${-1.97 + 0.01}" soft_upper_limit="${1.97 - 0.01}" /-->
     </joint>
     <link name="${name}_4_link">
-      <inertial>
-        <origin xyz="0 0 0" rpy="0 0 0"/>
-        <!--mass value="3.669819"/-->
-        <mass value="2.0"/>
-        <inertia ixx="0.03" ixy="0" ixz="0" iyy="0.03" iyz="0" izz="0.03" />
-      </inertial>
+      <xacro:default_inertial/>
       <visual>
         <origin xyz="0 0 0" rpy="0 0 0" />
@@ -167,12 +143,8 @@
       <dynamics damping="5" />
       <limit effort="41.6" velocity="2.0" lower="-6.25" upper="6.25" />
-      <safety_controller k_position="20" k_velocity="25" soft_lower_limit="${-6.25 + 0.01}" soft_upper_limit="${6.25 - 0.01}" />
+      <!--safety_controller k_position="20" k_velocity="25" soft_lower_limit="${-6.25 + 0.01}" soft_upper_limit="${6.25 - 0.01}" /-->
     </joint>
     <link name="${name}_5_link">
-      <inertial>
-        <origin xyz="0 0 0" rpy="0 0 0"/>
-        <mass value="2.313272"/>
-        <inertia ixx="0.03" ixy="0" ixz="0" iyy="0.03" iyz="0" izz="0.03" />
-      </inertial>
+      <xacro:default_inertial/>
       <visual>
         <origin xyz="0 0 0" rpy="0 0 0" />
@@ -198,12 +170,8 @@
       <dynamics damping="5" />
       <limit effort="20.1" velocity="2.0" lower="-1.97" upper="1.97" />
-      <safety_controller k_position="20" k_velocity="25" soft_lower_limit="${-1.97 + 0.01}" soft_upper_limit="${1.97 - 0.01}" />
+      <!--safety_controller k_position="20" k_velocity="25" soft_lower_limit="${-1.97 + 0.01}" soft_upper_limit="${1.97 - 0.01}" /-->
     </joint>
     <link name="${name}_6_link">
-      <inertial>
-        <origin xyz="0 0 0" rpy="0 0 0"/>
-        <mass value="2.057856"/>
-        <inertia ixx="0.01" ixy="0" ixz="0" iyy="0.01" iyz="0" izz="0.01" />
-      </inertial>
+      <xacro:default_inertial/>
       <visual>
         <origin xyz="0 0 0" rpy="0 0 0" />
@@ -229,12 +197,8 @@
       <dynamics damping="5" />
       <limit effort="9.6" velocity="2.0" lower="-6.25" upper="6.25" />
-      <safety_controller k_position="20" k_velocity="25" soft_lower_limit="${-6.25 + 0.01}" soft_upper_limit="${6.25 - 0.01}" />
+      <!--safety_controller k_position="20" k_velocity="25" soft_lower_limit="${-6.25 + 0.01}" soft_upper_limit="${6.25 - 0.01}" /-->
     </joint>
     <link name="${name}_7_link">
-      <inertial>
-        <origin xyz="0 0 0" rpy="0 0 0"/>
-        <mass value="1.120198"/>
-        <inertia ixx="0.01" ixy="0" ixz="0" iyy="0.01" iyz="0" izz="0.01" />
-      </inertial>
+      <xacro:default_inertial/>
       <visual>
         <origin xyz="0 0 0" rpy="0 0 0" />

File: schunk_description/urdf/sdh/sdh.transmission.xacro (robot description, xacro)
@@ -5,5 +5,5 @@
       <type>transmission_interface/SimpleTransmission</type>
       <joint name="${name}_finger_21_joint">
-        <hardwareInterface>EffortJointInterface</hardwareInterface>
+        <hardwareInterface>PositionJointInterface</hardwareInterface>
       </joint>
       <actuator name="${name}_knuckle_motor">
@@ -14,5 +14,5 @@
       <type>transmission_interface/SimpleTransmission</type>
       <joint name="${name}_knuckle_joint">
-        <hardwareInterface>EffortJointInterface</hardwareInterface>
+        <hardwareInterface>PositionJointInterface</hardwareInterface>
       </joint>
       <actuator name="${name}_knuckle_motor">
@@ -24,5 +24,5 @@
       <type>transmission_interface/SimpleTransmission</type>
       <joint name="${name}_finger_12_joint">
-        <hardwareInterface>EffortJointInterface</hardwareInterface>
+        <hardwareInterface>PositionJointInterface</hardwareInterface>
       </joint>
       <actuator name="${name}_finger_12_motor">
@@ -33,5 +33,5 @@
       <type>transmission_interface/SimpleTransmission</type>
       <joint name="${name}_finger_13_joint">
-        <hardwareInterface>EffortJointInterface</hardwareInterface>
+        <hardwareInterface>PositionJointInterface</hardwareInterface>
       </joint>
       <actuator name="${name}_finger_13_motor">
@@ -43,5 +43,5 @@
       <type>transmission_interface/SimpleTransmission</type>
       <joint name="${name}_finger_22_joint">
-        <hardwareInterface>EffortJointInterface</hardwareInterface>
+        <hardwareInterface>PositionJointInterface</hardwareInterface>
       </joint>
       <actuator name="${name}_finger_22_motor">
@@ -52,5 +52,5 @@
       <type>transmission_interface/SimpleTransmission</type>
       <joint name="${name}_finger_23_joint">
-        <hardwareInterface>EffortJointInterface</hardwareInterface>
+        <hardwareInterface>PositionJointInterface</hardwareInterface>
       </joint>
       <actuator name="${name}_finger_23_motor">
@@ -62,5 +62,5 @@
       <type>transmission_interface/SimpleTransmission</type>
       <joint name="${name}_thumb_2_joint">
-        <hardwareInterface>EffortJointInterface</hardwareInterface>
+        <hardwareInterface>PositionJointInterface</hardwareInterface>
       </joint>
       <actuator name="${name}_thumb_2_motor">
@@ -71,5 +71,5 @@
       <type>transmission_interface/SimpleTransmission</type>
       <joint name="${name}_thumb_3_joint">
-        <hardwareInterface>EffortJointInterface</hardwareInterface>
+        <hardwareInterface>PositionJointInterface</hardwareInterface>
       </joint>
       <actuator name="${name}_thumb_3_motor">
