Commit message: More changes from powerball to lwa4d

File: schunk_description/urdf/lwa4d/lwa4d.gazebo.xacro (robot description, xacro)
@@ -4,39 +4,36 @@
        xmlns:interface="http://playerstage.sourceforge.net/gazebo/xmlschema/#interface"
        xmlns:xacro="http://ros.org/wiki/xacro">
-	<xacro:macro name="schunk_powerball_gazebo" params="name">
+	<xacro:macro name="schunk_lwa_gazebo" params="name">
 		<gazebo reference="${name}_0_link">
-			<material value="Schunk/LightGrey" />
+			<material value="Schunk/DarkGolden" />
 			<turnGravityOff>false</turnGravityOff>
-                        <selfCollide>true</selfCollide>
 		</gazebo>
 		<gazebo reference="${name}_1_link">
-			<material value="Schunk/Blue" />
+			<material value="Schunk/DarkGolden" />
 			<turnGravityOff>false</turnGravityOff>
-                        <selfCollide>true</selfCollide>
 		</gazebo>
 		<gazebo reference="${name}_2_link">
-			<material value="Schunk/LightGrey" />
+			<material value="Schunk/DarkGolden" />
 			<turnGravityOff>false</turnGravityOff>
-                        <selfCollide>true</selfCollide>
 		</gazebo>
 		<gazebo reference="${name}_3_link">
-			<material value="Schunk/Blue" />
+			<material value="Schunk/DarkGolden" />
 			<turnGravityOff>false</turnGravityOff>
-                        <selfCollide>true</selfCollide>
 		</gazebo>
 		<gazebo reference="${name}_4_link">
-			<material value="Schunk/LightGrey" />
+			<material value="Schunk/DarkGolden" />
 			<turnGravityOff>false</turnGravityOff>
-                        <selfCollide>true</selfCollide>
 		</gazebo>
 		<gazebo reference="${name}_5_link">
-			<material value="Schunk/Blue" />
+			<material value="Schunk/DarkGolden" />
 			<turnGravityOff>false</turnGravityOff>
-                        <selfCollide>true</selfCollide>
 		</gazebo>
 		<gazebo reference="${name}_6_link">
-			<material value="Schunk/LightGrey" />
+			<material value="Schunk/DarkGolden" />
 			<turnGravityOff>false</turnGravityOff>
-                        <selfCollide>true</selfCollide>
+		</gazebo>
+		<gazebo reference="${name}_7_link">
+			<material value="Schunk/DarkGolden" />
+			<turnGravityOff>false</turnGravityOff>
 		</gazebo>
 	</xacro:macro>

File: schunk_description/urdf/lwa4d/lwa4d.transmission.xacro (robot description, xacro)
@@ -4,5 +4,5 @@
        xmlns:interface="http://playerstage.sourceforge.net/gazebo/xmlschema/#interface"
        xmlns:xacro="http://ros.org/wiki/xacro">
-	<xacro:macro name="schunk_powerball_transmission" params="name">
+	<xacro:macro name="schunk_lwa_transmission" params="name">
 		<transmission name="${name}_1_trans" type="pr2_mechanism_model/SimpleTransmission">
 			<actuator name="${name}_1_motor"/>
@@ -35,4 +35,9 @@
 			<mechanicalReduction>1</mechanicalReduction>
 		</transmission>
+		<transmission name="${name}_7_trans" type="pr2_mechanism_model/SimpleTransmission">
+			<actuator name="${name}_7_motor"/>
+			<joint name="${name}_7_joint"/>
+			<mechanicalReduction>1</mechanicalReduction>
+		</transmission>
 	</xacro:macro>
 </robot>

File: schunk_description/urdf/lwa4d/lwa4d.urdf.xacro (robot description, xacro)
@@ -4,7 +4,7 @@
        xmlns:interface="http://playerstage.sourceforge.net/gazebo/xmlschema/#interface"
        xmlns:xacro="http://ros.org/wiki/xacro">
-	<include filename="$(find schunk_description)/urdf/powerball/powerball.gazebo.xacro" />
-	<include filename="$(find schunk_description)/urdf/powerball/powerball.transmission.xacro" />
-	<xacro:macro name="schunk_powerball" params="parent name *origin">
+	<include filename="$(find schunk_description)/urdf/lwa/lwa.gazebo.xacro" />
+	<include filename="$(find schunk_description)/urdf/lwa/lwa.transmission.xacro" />
+	<xacro:macro name="schunk_lwa" params="parent name *origin">
 		<!-- joint between base_link and arm_0_link -->
 		<joint name="${name}_0_joint" type="fixed" >
@@ -15,19 +15,19 @@
 		<link name="${name}_0_link">
 			<inertial>
-				<origin xyz="0 0 0" rpy="0 0 0" />
-				<mass value="0.29364"/>
-				<inertia ixx="0.01" ixy="0" ixz="0" iyy="0.01" iyz="0" izz="0.01" />
-			</inertial>
-			<visual>
-				<origin xyz="0 0 0" rpy="0 0 0" />
-				<geometry>
-					<mesh filename="package://schunk_description/meshes/powerball/arm_0_link.stl" />
-				</geometry>
-				<material name="Schunk/LightGrey" />
-			</visual>
-			<collision>
-				<origin xyz="0 0 0" rpy="0 0 0" />
-				<geometry>
-					<mesh filename="package://schunk_description/meshes/powerball/arm_0_link.stl" />
+				<origin xyz="0 0 0" rpy="0 0 0"/>
+				<mass value="1.0"/>
+				<inertia ixx="0.01" ixy="0" ixz="0" iyy="0.01" iyz="0" izz="0.01" />
+			</inertial>
+			<visual>
+				<origin xyz="0 0 0.004" rpy="0 0 0" />
+				<geometry>
+					<cylinder radius="0.045" length="0.08"/>
+				</geometry>
+				<material name="Schunk/DarkGolden" />
+			</visual>
+			<collision>
+				<origin xyz="0 0 0.005" rpy="0 0 0" />
+				<geometry>
+					<box size="0.01 0.01 0.01"/>
 				</geometry>
 			</collision>
@@ -35,5 +35,5 @@
 		<!-- joint between arm_0_link and arm_1_link -->
 		<joint name="${name}_1_joint" type="revolute">
-			<origin xyz="0 0 0.11" rpy="0 0 0"/>
+			<origin xyz="0 0 -0.250" rpy="0 0 3.1415926"/>
 			<parent link="${name}_0_link"/>
 			<child link="${name}_1_link"/>
@@ -47,18 +47,19 @@
 			<inertial>
 				<origin xyz="0 0 0" rpy="0 0 0" />
-				<mass value="0.29364"/>
-				<inertia ixx="0.01" ixy="0" ixz="0" iyy="0.01" iyz="0" izz="0.01" />
-			</inertial>
-			<visual>
-				<origin xyz="0 0 0" rpy="0 0 0" />
-				<geometry>
-					<mesh filename="package://schunk_description/meshes/powerball/arm_1_link.stl" />
-				</geometry>
-				<material name="Schunk/Blue" />
-			</visual>
-			<collision>
-				<origin xyz="0 0 0" rpy="0 0 0" />
-				<geometry>
-					<mesh filename="package://schunk_description/meshes/powerball/arm_1_link.stl" />
+				<!--mass value="5.9907"/-->
+				<mass value="2.0"/>
+				<inertia ixx="0.01" ixy="0" ixz="0" iyy="0.01" iyz="0" izz="0.01" />
+			</inertial>
+			<visual>
+				<origin xyz="0 0 0" rpy="0 0 0" />
+				<geometry>
+					<mesh filename="package://schunk_description/meshes/lwa/lwa1.stl" />
+				</geometry>
+				<material name="Schunk/DarkGolden" />
+			</visual>
+			<collision>
+				<origin xyz="0 0 0" rpy="0 0 0" />
+				<geometry>
+					<mesh filename="package://schunk_description/meshes/lwa/lwa1.stl" />
 				</geometry>
 			</collision>
@@ -72,24 +73,25 @@
 			<calibration rising="${arm_2_ref}"/>
 			<dynamics damping="10" />
-			<limit effort="370" velocity="2.0" lower="-2.0943951" upper="2.0943951"/>
-			<safety_controller k_position="20" k_velocity="50" soft_lower_limit="${-2.0943 + 0.01}" soft_upper_limit="${2.0943 - 0.01}" />
+			<limit effort="370" velocity="2.0" lower="-1.97" upper="1.97"/>
+			<safety_controller k_position="20" k_velocity="50" soft_lower_limit="${-1.97 + 0.01}" 	soft_upper_limit="${1.97 - 0.01}" />
 		</joint>
 		<link name="${name}_2_link">
 			<inertial>
 				<origin xyz="0 0 0" rpy="0 0 0"/>
-				<mass value="1.68311"/>
-				<inertia ixx="0.03" ixy="0" ixz="0" iyy="0.03" iyz="0" izz="0.03" />
-			</inertial>
-			<visual>
-				<origin xyz="0 0 0" rpy="0 0 0" />
-				<geometry>
-					<mesh filename="package://schunk_description/meshes/powerball/arm_2_link.stl" />
-				</geometry>
-				<material name="Schunk/LightGrey" />
-			</visual>
-			<collision>
-				<origin xyz="0 0 0" rpy="0 0 0" />
-				<geometry>
-					<mesh filename="package://schunk_description/meshes/powerball/arm_2_link.stl" />
+				<!--mass value="5.734939"/-->
+				<mass value="2.0"/>
+				<inertia ixx="0.03" ixy="0" ixz="0" iyy="0.03" iyz="0" izz="0.03" />
+			</inertial>
+			<visual>
+				<origin xyz="0 0 0" rpy="0 0 0" />
+				<geometry>
+					<mesh filename="package://schunk_description/meshes/lwa/lwa2.stl" />
+				</geometry>
+				<material name="Schunk/DarkGolden" />
+			</visual>
+			<collision>
+				<origin xyz="0 0 0" rpy="0 0 0" />
+				<geometry>
+					<mesh filename="package://schunk_description/meshes/lwa/lwa2.stl"/>
 				</geometry>
 			</collision>
@@ -97,5 +99,5 @@
 		<!-- joint between arm_2_link and arm_3_link -->
 		<joint name="${name}_3_joint" type="revolute">
-			<origin xyz="0 0.350 0" rpy="0 3.14159 0"/>
+			<origin xyz="0 -0.408 0" rpy="-1.5708 0 0"/>
 			<parent link="${name}_2_link"/>
 			<child link="${name}_3_link"/>
@@ -109,18 +111,19 @@
 			<inertial>
 				<origin xyz="0 0 0" rpy="0 0 0"/>
-				<mass value="2.1"/>
-				<inertia ixx="0.03" ixy="0" ixz="0" iyy="0.03" iyz="0" izz="0.03" />
-			</inertial>
-			<visual>
-				<origin xyz="0 0 0" rpy="0 0 0" />
-				<geometry>
-					<mesh filename="package://schunk_description/meshes/powerball/arm_3_link.stl" />
-				</geometry>
-				<material name="Schunk/Blue" />
-			</visual>
-			<collision>
-				<origin xyz="0 0 0" rpy="0 0 0" />
-				<geometry>
-					<mesh filename="package://schunk_description/meshes/powerball/arm_3_link.stl" />
+				<!--mass value="4.214668"/-->
+				<mass value="2.0"/>
+				<inertia ixx="0.03" ixy="0" ixz="0" iyy="0.03" iyz="0" izz="0.03" />
+			</inertial>
+			<visual>
+				<origin xyz="0 0 0" rpy="0 0 0" />
+				<geometry>
+					<mesh filename="package://schunk_description/meshes/lwa/lwa3.stl" />
+				</geometry>
+				<material name="Schunk/DarkGolden" />
+			</visual>
+			<collision>
+				<origin xyz="0 0 0" rpy="0 0 0" />
+				<geometry>
+					<mesh filename="package://schunk_description/meshes/lwa/lwa3.stl"/>
 				</geometry>
 			</collision>
@@ -128,5 +131,5 @@
 		<!-- joint between arm_3_link and arm_4_link -->
 		<joint name="${name}_4_joint" type="revolute">
-			<origin xyz="0 0 0" rpy="-1.5708 3.14159 0" />
+			<origin xyz="0 0 0" rpy="1.5708 0 0" />
 			<parent link="${name}_3_link"/>
 			<child link="${name}_4_link"/>
@@ -134,24 +137,25 @@
 			<calibration rising="${arm_4_ref}"/>
 			<dynamics damping="5" />
-			<limit effort="176" velocity="2.0" lower="-2.0943951" upper="2.0943951"/>
-			<safety_controller k_position="20" k_velocity="25" soft_lower_limit="${-2.0943951 + 0.01}" soft_upper_limit="${2.0943951 - 0.01}" />
+			<limit effort="176" velocity="2.0" lower="-2.08208" upper="2.08208"/>
+			<safety_controller k_position="20" k_velocity="25" soft_lower_limit="${-2.08208 + 0.01}" soft_upper_limit="${2.08208 - 0.01}" />
 		</joint>
 		<link name="${name}_4_link">
 			<inertial>
 				<origin xyz="0 0 0" rpy="0 0 0"/>
-				<mass value="1.68311"/>
-				<inertia ixx="0.03" ixy="0" ixz="0" iyy="0.03" iyz="0" izz="0.03" />
-			</inertial>
-			<visual>
-				<origin xyz="0 0 0" rpy="0 0 0" />
-				<geometry>
-					<mesh filename="package://schunk_description/meshes/powerball/arm_4_link.stl" />
-				</geometry>
-				<material name="Schunk/LightGrey" />
-			</visual>
-			<collision>
-				<origin xyz="0 0 0" rpy="0 0 0" />
-				<geometry>
-					<mesh filename="package://schunk_description/meshes/powerball/arm_4_link.stl" />
+				<!--mass value="3.669819"/-->
+				<mass value="2.0"/>
+				<inertia ixx="0.03" ixy="0" ixz="0" iyy="0.03" iyz="0" izz="0.03" />
+			</inertial>
+			<visual>
+				<origin xyz="0 0 0" rpy="0 0 0" />
+				<geometry>
+					<mesh filename="package://schunk_description/meshes/lwa/lwa4.stl" />
+				</geometry>
+				<material name="Schunk/DarkGolden" />
+			</visual>
+			<collision>
+				<origin xyz="0 0 0" rpy="0 0 0" />
+				<geometry>
+					<mesh filename="package://schunk_description/meshes/lwa/lwa4.stl"/>
 				</geometry>
 			</collision>
@@ -159,5 +163,5 @@
 		<!-- joint between arm_4_link and arm_5_link -->
 		<joint name="${name}_5_joint" type="revolute">
-			<origin xyz="0 0.005263 0.365" rpy="1.5708 0 3.14159" />
+			<origin xyz="0 -0.3165 0" rpy="-1.5708 0 0" />
 			<parent link="${name}_4_link"/>
 			<child link="${name}_5_link"/>
@@ -171,18 +175,18 @@
 			<inertial>
 				<origin xyz="0 0 0" rpy="0 0 0"/>
-				<mass value="0.807"/>
-				<inertia ixx="0.03" ixy="0" ixz="0" iyy="0.03" iyz="0" izz="0.03" />
-			</inertial>
-			<visual>
-				<origin xyz="0 0 0" rpy="0 0 0" />
-				<geometry>
-					<mesh filename="package://schunk_description/meshes/powerball/arm_5_link.stl" />
-				</geometry>
-				<material name="Schunk/Blue" />
-			</visual>
-			<collision>
-				<origin xyz="0 0 0" rpy="0 0 0" />
-				<geometry>
-					<mesh filename="package://schunk_description/meshes/powerball/arm_5_link.stl" />
+				<mass value="2.313272"/>
+				<inertia ixx="0.03" ixy="0" ixz="0" iyy="0.03" iyz="0" izz="0.03" />
+			</inertial>
+			<visual>
+				<origin xyz="0 0 0" rpy="0 0 0" />
+				<geometry>
+					<mesh filename="package://schunk_description/meshes/lwa/lwa5.stl" />
+				</geometry>
+				<material name="Schunk/DarkGolden" />
+			</visual>
+			<collision>
+				<origin xyz="0 0 0" rpy="0 0 0" />
+				<geometry>
+					<mesh filename="package://schunk_description/meshes/lwa/lwa5.stl"/>
 				</geometry>
 			</collision>
@@ -190,5 +194,5 @@
 		<!-- joint between arm_5_link and arm_6_link -->
 		<joint name="${name}_6_joint" type="revolute">
-			<origin xyz="0 0 0" rpy="-1.5708 0 0" />
+			<origin xyz="0 0 0" rpy="1.5708 0 0" />
 			<parent link="${name}_5_link"/>
 			<child link="${name}_6_link"/>
@@ -196,30 +200,61 @@
 			<calibration rising="${arm_6_ref}"/>
 			<dynamics damping="5" />
-			<limit effort="20.1" velocity="2.0" lower="-2.0943951" upper="2.0943951" />
-			<safety_controller k_position="20" k_velocity="25" soft_lower_limit="${-2.0943951 + 0.01}" soft_upper_limit="${2.0943951 - 0.01}" />
+			<limit effort="20.1" velocity="2.0" lower="-1.8" upper="1.8" />
+			<safety_controller k_position="20" k_velocity="25" soft_lower_limit="${-1.8 + 0.01}" soft_upper_limit="${1.8 - 0.01}" />
 		</joint>
 		<link name="${name}_6_link">
 			<inertial>
 				<origin xyz="0 0 0" rpy="0 0 0"/>
-				<mass value="0.819"/>
-				<inertia ixx="0.01" ixy="0" ixz="0" iyy="0.01" iyz="0" izz="0.01" />
-			</inertial>
-			<visual>
-				<origin xyz="0 0 0" rpy="0 0 0" />
-				<geometry>
-					<mesh filename="package://schunk_description/meshes/powerball/arm_6_link.stl" />
-				</geometry>
-				<material name="Schunk/LightGrey" />
-			</visual>
-			<collision>
-				<origin xyz="0 0 0" rpy="0 0 0" />
-				<geometry>
-					<mesh filename="package://schunk_description/meshes/powerball/arm_6_link.stl" />
+				<mass value="2.057856"/>
+				<inertia ixx="0.01" ixy="0" ixz="0" iyy="0.01" iyz="0" izz="0.01" />
+			</inertial>
+			<visual>
+				<origin xyz="0 0 0" rpy="0 0 0" />
+				<geometry>
+					<mesh filename="package://schunk_description/meshes/lwa/lwa6.stl" />
+				</geometry>
+				<material name="Schunk/DarkGolden" />
+			</visual>
+			<collision>
+				<origin xyz="0 0 0" rpy="0 0 0" />
+				<geometry>
+					<mesh filename="package://schunk_description/meshes/lwa/lwa6.stl"/>
+				</geometry>
+			</collision>
+		</link>
+		<!-- joint between arm_6_link and arm_7_link -->
+		<joint name="${name}_7_joint" type="revolute">
+			<origin xyz="0 -0.1927 0" rpy="-1.5708 0 0" />
+			<parent link="${name}_6_link"/>
+			<child link="${name}_7_link"/>
+			<axis xyz="0 0 1" />
+			<calibration rising="${arm_7_ref}"/>
+			<dynamics damping="5" />
+			<limit effort="9.6" velocity="2.0" lower="-6.2831853" upper="6.2831853" />
+			<safety_controller k_position="20" k_velocity="25" soft_lower_limit="${-6.2831853 + 0.01}" soft_upper_limit="${6.2831853 - 0.01}" />
+		</joint>
+		<link name="${name}_7_link">
+			<inertial>
+				<origin xyz="0 0 0" rpy="0 0 0"/>
+				<mass value="1.120198"/>
+				<inertia ixx="0.01" ixy="0" ixz="0" iyy="0.01" iyz="0" izz="0.01" />
+			</inertial>
+			<visual>
+				<origin xyz="0 0 0" rpy="0 0 0" />
+				<geometry>
+					<mesh filename="package://schunk_description/meshes/lwa/lwa7.stl" />
+				</geometry>
+				<material name="Schunk/DarkGolden" />
+			</visual>
+			<collision>
+				<origin xyz="0 0 0" rpy="0 0 0" />
+				<geometry>
+					<mesh filename="package://schunk_description/meshes/lwa/lwa7.stl"/>
 				</geometry>
 			</collision>
 		</link>
 		<!-- extensions -->
-		<xacro:schunk_powerball_gazebo name="${name}" />
-		<xacro:schunk_powerball_transmission name="${name}" />
+		<xacro:schunk_lwa_gazebo name="${name}" />
+		<xacro:schunk_lwa_transmission name="${name}" />
 	</xacro:macro>
 </robot>
