Commit message: Created lwa4d urdf model

File: schunk_description/urdf/lwa4d/lwa4d.gazebo.xacro (robot description, xacro)
@@ -4,35 +4,35 @@
        xmlns:interface="http://playerstage.sourceforge.net/gazebo/xmlschema/#interface"
        xmlns:xacro="http://ros.org/wiki/xacro">
-	<xacro:macro name="schunk_lwa_gazebo" params="name">
+	<xacro:macro name="schunk_lwa4d_gazebo" params="name">
 		<gazebo reference="${name}_0_link">
-			<material value="Schunk/DarkGolden" />
+			<material value="Schunk/Black" />
 			<turnGravityOff>false</turnGravityOff>
 		</gazebo>
 		<gazebo reference="${name}_1_link">
-			<material value="Schunk/DarkGolden" />
+			<material value="Schunk/LightGrey" />
 			<turnGravityOff>false</turnGravityOff>
 		</gazebo>
 		<gazebo reference="${name}_2_link">
-			<material value="Schunk/DarkGolden" />
+			<material value="Schunk/Black" />
 			<turnGravityOff>false</turnGravityOff>
 		</gazebo>
 		<gazebo reference="${name}_3_link">
-			<material value="Schunk/DarkGolden" />
+			<material value="Schunk/LightGrey" />
 			<turnGravityOff>false</turnGravityOff>
 		</gazebo>
 		<gazebo reference="${name}_4_link">
-			<material value="Schunk/DarkGolden" />
+			<material value="Schunk/Black" />
 			<turnGravityOff>false</turnGravityOff>
 		</gazebo>
 		<gazebo reference="${name}_5_link">
-			<material value="Schunk/DarkGolden" />
+			<material value="Schunk/LightGrey" />
 			<turnGravityOff>false</turnGravityOff>
 		</gazebo>
 		<gazebo reference="${name}_6_link">
-			<material value="Schunk/DarkGolden" />
+			<material value="Schunk/Black" />
 			<turnGravityOff>false</turnGravityOff>
 		</gazebo>
 		<gazebo reference="${name}_7_link">
-			<material value="Schunk/DarkGolden" />
+			<material value="Schunk/LightGrey" />
 			<turnGravityOff>false</turnGravityOff>
 		</gazebo>

File: schunk_description/urdf/lwa4d/lwa4d.transmission.xacro (robot description, xacro)
@@ -4,5 +4,5 @@
        xmlns:interface="http://playerstage.sourceforge.net/gazebo/xmlschema/#interface"
        xmlns:xacro="http://ros.org/wiki/xacro">
-	<xacro:macro name="schunk_lwa_transmission" params="name">
+	<xacro:macro name="schunk_lwa4d_transmission" params="name">
 		<transmission name="${name}_1_trans" type="pr2_mechanism_model/SimpleTransmission">
 			<actuator name="${name}_1_motor"/>

File: schunk_description/urdf/lwa4d/lwa4d.urdf.xacro (robot description, xacro)
@@ -4,7 +4,7 @@
        xmlns:interface="http://playerstage.sourceforge.net/gazebo/xmlschema/#interface"
        xmlns:xacro="http://ros.org/wiki/xacro">
-	<include filename="$(find schunk_description)/urdf/lwa/lwa.gazebo.xacro" />
-	<include filename="$(find schunk_description)/urdf/lwa/lwa.transmission.xacro" />
-	<xacro:macro name="schunk_lwa" params="parent name *origin">
+	<include filename="$(find schunk_description)/urdf/lwa4d/lwa4d.gazebo.xacro" />
+	<include filename="$(find schunk_description)/urdf/lwa4d/lwa4d.transmission.xacro" />
+	<xacro:macro name="schunk_lwa4d" params="parent name *origin">
 		<!-- joint between base_link and arm_0_link -->
 		<joint name="${name}_0_joint" type="fixed" >
@@ -24,5 +24,5 @@
 					<cylinder radius="0.045" length="0.08"/>
 				</geometry>
-				<material name="Schunk/DarkGolden" />
+				<material name="Schunk/Black" />
 			</visual>
 			<collision>
@@ -35,5 +35,5 @@
 		<!-- joint between arm_0_link and arm_1_link -->
 		<joint name="${name}_1_joint" type="revolute">
-			<origin xyz="0 0 -0.250" rpy="0 0 3.1415926"/>
+			<origin xyz="0 0 0.15" rpy="0 0 0"/>
 			<parent link="${name}_0_link"/>
 			<child link="${name}_1_link"/>
@@ -52,14 +52,14 @@
 			</inertial>
 			<visual>
-				<origin xyz="0 0 0" rpy="0 0 0" />
-				<geometry>
-					<mesh filename="package://schunk_description/meshes/lwa/lwa1.stl" />
-				</geometry>
-				<material name="Schunk/DarkGolden" />
-			</visual>
-			<collision>
-				<origin xyz="0 0 0" rpy="0 0 0" />
-				<geometry>
-					<mesh filename="package://schunk_description/meshes/lwa/lwa1.stl" />
+				<origin xyz="0 0 0.15" rpy="0 3.14 0" />
+				<geometry>
+					<mesh filename="package://schunk_description/meshes/lwa4d/arm_1_link.stl" />
+				</geometry>
+				<material name="Schunk/LightGrey" />
+			</visual>
+			<collision>
+				<origin xyz="0 0 0.15" rpy="0 3.14 0" />
+				<geometry>
+					<mesh filename="package://schunk_description/meshes/lwa4d/arm_1_link.stl" />
 				</geometry>
 			</collision>
@@ -67,5 +67,5 @@
 		<!-- joint between arm_1_link and arm_2_link -->
 		<joint name="${name}_2_joint" type="revolute">
-			<origin xyz="0 0 0" rpy="1.5708 0 0"/>
+			<origin xyz="0 0 0.15" rpy="-1.57 0 0"/>
 			<parent link="${name}_1_link"/>
 			<child link="${name}_2_link"/>
@@ -84,14 +84,14 @@
 			</inertial>
 			<visual>
-				<origin xyz="0 0 0" rpy="0 0 0" />
-				<geometry>
-					<mesh filename="package://schunk_description/meshes/lwa/lwa2.stl" />
-				</geometry>
-				<material name="Schunk/DarkGolden" />
-			</visual>
-			<collision>
-				<origin xyz="0 0 0" rpy="0 0 0" />
-				<geometry>
-					<mesh filename="package://schunk_description/meshes/lwa/lwa2.stl"/>
+				<origin xyz="0 0 0" rpy="0 3.14159 0" />
+				<geometry>
+					<mesh filename="package://schunk_description/meshes/lwa4d/arm_2_link.stl" />
+				</geometry>
+				<material name="Schunk/Black" />
+			</visual>
+			<collision>
+				<origin xyz="0 0 0" rpy="0 3.14159 0" />
+				<geometry>
+					<mesh filename="package://schunk_description/meshes/lwa4d/arm_2_link.stl"/>
 				</geometry>
 			</collision>
@@ -99,5 +99,5 @@
 		<!-- joint between arm_2_link and arm_3_link -->
 		<joint name="${name}_3_joint" type="revolute">
-			<origin xyz="0 -0.408 0" rpy="-1.5708 0 0"/>
+			<origin xyz="0 0 0" rpy="1.5708 0 0"/>
 			<parent link="${name}_2_link"/>
 			<child link="${name}_3_link"/>
@@ -116,14 +116,14 @@
 			</inertial>
 			<visual>
-				<origin xyz="0 0 0" rpy="0 0 0" />
-				<geometry>
-					<mesh filename="package://schunk_description/meshes/lwa/lwa3.stl" />
-				</geometry>
-				<material name="Schunk/DarkGolden" />
-			</visual>
-			<collision>
-				<origin xyz="0 0 0" rpy="0 0 0" />
-				<geometry>
-					<mesh filename="package://schunk_description/meshes/lwa/lwa3.stl"/>
+				<origin xyz="0 0 0.328" rpy="0 3.1415 0" />
+				<geometry>
+					<mesh filename="package://schunk_description/meshes/lwa4d/arm_3_link.stl" />
+				</geometry>
+				<material name="Schunk/LightGrey" />
+			</visual>
+			<collision>
+				<origin xyz="0 0 0.328" rpy="0 3.1415 0" />
+				<geometry>
+					<mesh filename="package://schunk_description/meshes/lwa4d/arm_3_link.stl"/>
 				</geometry>
 			</collision>
@@ -131,5 +131,5 @@
 		<!-- joint between arm_3_link and arm_4_link -->
 		<joint name="${name}_4_joint" type="revolute">
-			<origin xyz="0 0 0" rpy="1.5708 0 0" />
+			<origin xyz="0 0 0.328" rpy="-1.5708 0 0"/>
 			<parent link="${name}_3_link"/>
 			<child link="${name}_4_link"/>
@@ -148,14 +148,14 @@
 			</inertial>
 			<visual>
-				<origin xyz="0 0 0" rpy="0 0 0" />
-				<geometry>
-					<mesh filename="package://schunk_description/meshes/lwa/lwa4.stl" />
-				</geometry>
-				<material name="Schunk/DarkGolden" />
-			</visual>
-			<collision>
-				<origin xyz="0 0 0" rpy="0 0 0" />
-				<geometry>
-					<mesh filename="package://schunk_description/meshes/lwa/lwa4.stl"/>
+				<origin xyz="0 0 0" rpy="0 3.14159 0" />
+				<geometry>
+					<mesh filename="package://schunk_description/meshes/lwa4d/arm_4_link.stl" />
+				</geometry>
+				<material name="Schunk/Black" />
+			</visual>
+			<collision>
+				<origin xyz="0 0 0" rpy="0 3.14159 0" />
+				<geometry>
+					<mesh filename="package://schunk_description/meshes/lwa4d/arm_4_link.stl"/>
 				</geometry>
 			</collision>
@@ -163,5 +163,5 @@
 		<!-- joint between arm_4_link and arm_5_link -->
 		<joint name="${name}_5_joint" type="revolute">
-			<origin xyz="0 -0.3165 0" rpy="-1.5708 0 0" />
+			<origin xyz="0 0 0" rpy="1.5708 0 0" />
 			<parent link="${name}_4_link"/>
 			<child link="${name}_5_link"/>
@@ -179,14 +179,14 @@
 			</inertial>
 			<visual>
-				<origin xyz="0 0 0" rpy="0 0 0" />
-				<geometry>
-					<mesh filename="package://schunk_description/meshes/lwa/lwa5.stl" />
-				</geometry>
-				<material name="Schunk/DarkGolden" />
-			</visual>
-			<collision>
-				<origin xyz="0 0 0" rpy="0 0 0" />
-				<geometry>
-					<mesh filename="package://schunk_description/meshes/lwa/lwa5.stl"/>
+				<origin xyz="0 0 0.323" rpy="0 3.14159 0" />
+				<geometry>
+					<mesh filename="package://schunk_description/meshes/lwa4d/arm_5_link.stl" />
+				</geometry>
+				<material name="Schunk/LightGrey" />
+			</visual>
+			<collision>
+				<origin xyz="0 0 0.323" rpy="0 3.14159 0" />
+				<geometry>
+					<mesh filename="package://schunk_description/meshes/lwa4d/arm_5_link.stl"/>
 				</geometry>
 			</collision>
@@ -194,5 +194,5 @@
 		<!-- joint between arm_5_link and arm_6_link -->
 		<joint name="${name}_6_joint" type="revolute">
-			<origin xyz="0 0 0" rpy="1.5708 0 0" />
+			<origin xyz="0 0 0.323" rpy="-1.5708 0 0" />
 			<parent link="${name}_5_link"/>
 			<child link="${name}_6_link"/>
@@ -210,14 +210,14 @@
 			</inertial>
 			<visual>
-				<origin xyz="0 0 0" rpy="0 0 0" />
-				<geometry>
-					<mesh filename="package://schunk_description/meshes/lwa/lwa6.stl" />
-				</geometry>
-				<material name="Schunk/DarkGolden" />
-			</visual>
-			<collision>
-				<origin xyz="0 0 0" rpy="0 0 0" />
-				<geometry>
-					<mesh filename="package://schunk_description/meshes/lwa/lwa6.stl"/>
+				<origin xyz="0 0 0" rpy="0 0 3.14159" />
+				<geometry>
+					<mesh filename="package://schunk_description/meshes/lwa4d/arm_6_link.stl" />
+				</geometry>
+				<material name="Schunk/Black" />
+			</visual>
+			<collision>
+				<origin xyz="0 0 0" rpy="0 0 3.14159" />
+				<geometry>
+					<mesh filename="package://schunk_description/meshes/lwa4d/arm_6_link.stl"/>
 				</geometry>
 			</collision>
@@ -225,5 +225,5 @@
 		<!-- joint between arm_6_link and arm_7_link -->
 		<joint name="${name}_7_joint" type="revolute">
-			<origin xyz="0 -0.1927 0" rpy="-1.5708 0 0" />
+			<origin xyz="0 -0.075 0" rpy="1.5708 0 0" />
 			<parent link="${name}_6_link"/>
 			<child link="${name}_7_link"/>
@@ -241,20 +241,20 @@
 			</inertial>
 			<visual>
-				<origin xyz="0 0 0" rpy="0 0 0" />
-				<geometry>
-					<mesh filename="package://schunk_description/meshes/lwa/lwa7.stl" />
-				</geometry>
-				<material name="Schunk/DarkGolden" />
-			</visual>
-			<collision>
-				<origin xyz="0 0 0" rpy="0 0 0" />
-				<geometry>
-					<mesh filename="package://schunk_description/meshes/lwa/lwa7.stl"/>
+				<origin xyz="0 0 -0.075" rpy="0 0 0" />
+				<geometry>
+					<mesh filename="package://schunk_description/meshes/lwa4d/arm_7_link.stl" />
+				</geometry>
+				<material name="Schunk/LightGrey" />
+			</visual>
+			<collision>
+				<origin xyz="0 0 -0.075" rpy="0 0 0" />
+				<geometry>
+					<mesh filename="package://schunk_description/meshes/lwa4d/arm_7_link.stl"/>
 				</geometry>
 			</collision>
 		</link>
 		<!-- extensions -->
-		<xacro:schunk_lwa_gazebo name="${name}" />
-		<xacro:schunk_lwa_transmission name="${name}" />
+		<xacro:schunk_lwa4d_gazebo name="${name}" />
+		<xacro:schunk_lwa4d_transmission name="${name}" />
 	</xacro:macro>
 </robot>

Commit message: Fixed arm_7_joint position

File: schunk_description/urdf/lwa4d/lwa4d.gazebo.xacro (robot description, xacro)
@@ -37,4 +37,9 @@
 			<turnGravityOff>false</turnGravityOff>
 		</gazebo>
+		<!--<gazebo reference="${name}_gripper">
+			<material value="Schunk/LightGrey" />
+			<turnGravityOff>false</turnGravityOff>
+		</gazebo>
+                -->
 	</xacro:macro>
 </robot>

File: schunk_description/urdf/lwa4d/lwa4d.urdf.xacro (robot description, xacro)
@@ -223,5 +223,5 @@
 		<!-- joint between arm_6_link and arm_7_link -->
 		<joint name="${name}_7_joint" type="revolute">
-			<origin xyz="0 -0.075 0" rpy="-${M_PI/2} 0 0" />
+			<origin xyz="0 -0.075 0" rpy="${M_PI/2} 0 0" />
 			<parent link="${name}_6_link"/>
 			<child link="${name}_7_link"/>
@@ -239,5 +239,5 @@
 			</inertial>
 			<visual>
-				<origin xyz="0 0 0.075" rpy="0 ${M_PI} 0" />
+				<origin xyz="0 0 -0.075" rpy="0 0 0" />
 				<geometry>
 					<mesh filename="package://schunk_description/meshes/lwa4d/arm_7_link.stl" />
@@ -246,5 +246,5 @@
 			</visual>
 			<collision>
-				<origin xyz="0 0 0.075" rpy="0 ${M_PI} 0" />
+				<origin xyz="0 0 -0.075" rpy="0 0 0" />
 				<geometry>
 					<mesh filename="package://schunk_description/meshes/lwa4d/arm_7_link.stl"/>
@@ -252,4 +252,24 @@
 			</collision>
 		</link>
+		<!--<joint name="${name}_gripper_joint" type="fixed">
+   			 <origin rpy="0 0 0" xyz="0 0 0.06"/>
+   				 <parent link="${name}_7_link"/>
+  				  <child link="${name}_gripper"/>
+ 		 </joint>
+		<link name="${name}_gripper">
+  		  <visual>
+     			 <origin rpy="0 0 0" xyz="0 0 0" />
+     			 <geometry>
+     				   <mesh filename="package://schunk_description/meshes/lwa4d/arm_gripper.stl" />
+     			 </geometry>
+     			<material name="Schunk/LightGrey" />
+   		 </visual>
+   		 <collision>
+    			  <origin xyz="0 0 0" rpy="0 0 0" />
+    			  <geometry>
+    			    <mesh filename="package://schunk_description/meshes/lwa4d/arm_gripper.stl" />
+    			  </geometry>
+   		 </collision>
+	       </link>-->
 		<!-- extensions -->
 		<xacro:schunk_lwa4d_gazebo name="${name}" />

Commit message: tested on real arm

File: schunk_description/urdf/lwa4d/lwa4d.gazebo.xacro (robot description, xacro)
@@ -37,9 +37,4 @@
 			<turnGravityOff>false</turnGravityOff>
 		</gazebo>
-		<!--<gazebo reference="${name}_gripper">
-			<material value="Schunk/LightGrey" />
-			<turnGravityOff>false</turnGravityOff>
-		</gazebo>
-                -->
 	</xacro:macro>
 </robot>

File: schunk_description/urdf/lwa4d/lwa4d.urdf.xacro (robot description, xacro)
@@ -252,24 +252,4 @@
 			</collision>
 		</link>
-		<!--<joint name="${name}_gripper_joint" type="fixed">
-   			 <origin rpy="0 0 0" xyz="0 0 0.06"/>
-   				 <parent link="${name}_7_link"/>
-  				  <child link="${name}_gripper"/>
- 		 </joint>
-		<link name="${name}_gripper">
-  		  <visual>
-     			 <origin rpy="0 0 0" xyz="0 0 0" />
-     			 <geometry>
-     				   <mesh filename="package://schunk_description/meshes/lwa4d/arm_gripper.stl" />
-     			 </geometry>
-     			<material name="Schunk/LightGrey" />
-   		 </visual>
-   		 <collision>
-    			  <origin xyz="0 0 0" rpy="0 0 0" />
-    			  <geometry>
-    			    <mesh filename="package://schunk_description/meshes/lwa4d/arm_gripper.stl" />
-    			  </geometry>
-   		 </collision>
-	       </link>-->
 		<!-- extensions -->
 		<xacro:schunk_lwa4d_gazebo name="${name}" />

Commit message: cleaning up

File: schunk_description/urdf/lwa4d/lwa4d.gazebo.xacro (robot description, xacro)
@@ -2,5 +2,5 @@
 <robot xmlns:xacro="http://www.ros.org/wiki/xacro">
   <xacro:macro name="schunk_lwa4d_gazebo" params="name">
-    <gazebo reference="${name}_0_link">
+    <gazebo reference="${name}_base_link">
       <gravity>true</gravity>
       <self_collide>false</self_collide>

File: schunk_description/urdf/lwa4d/lwa4d.urdf.xacro (robot description, xacro)
@@ -3,10 +3,10 @@
   <xacro:include filename="$(find schunk_description)/urdf/lwa4d/lwa4d.gazebo.xacro" />
   <xacro:include filename="$(find schunk_description)/urdf/lwa4d/lwa4d.transmission.xacro" />
-  <xacro:macro name="schunk_lwa4d" params="parent name *origin">
-    <!-- joint between base_link and arm_0_link -->
-    <joint name="${name}_0_joint" type="fixed" >
+  <xacro:macro name="schunk_lwa4p_extended" params="parent name *origin arm_1_ref arm_2_ref arm_3_ref arm_4_ref arm_5_ref arm_6_ref arm_7_ref">
+    <!-- joint between base_link and arm_base_link -->
+    <joint name="${name}_base_joint" type="fixed">
       <insert_block name="origin" />
-      <parent link="${parent}" />
-      <child link="${name}_base_link" />
+      <parent link="${parent}"/>
+      <child link="${name}_base_link"/>
     </joint>
     <link name="${name}_base_link">
@@ -90,4 +90,5 @@
       <calibration rising="${arm_3_ref}"/>
       <limit effort="81.5" velocity="0.4189" lower="-${M_PI}" upper="${M_PI}"/>
+    </joint>
     <link name="${name}_3_link">
       <xacro:cylinder_inertial radius="0.056" length="0.134" mass="2.0">
