Commit message: beautification

File: schunk_description/urdf/lwa4d/lwa4d.gazebo.xacro (robot description, xacro)
@@ -5,38 +5,40 @@
       <gravity>true</gravity>
       <self_collide>false</self_collide>
-      <material value="Schunk/DarkGolden" />
+      <material value="Schunk/Black"/>
     </gazebo>
     <gazebo reference="${name}_1_link">
       <gravity>true</gravity>
       <self_collide>false</self_collide>
+      <material value="Schunk/LightGrey"/>
     </gazebo>
     <gazebo reference="${name}_2_link">
       <gravity>true</gravity>
       <self_collide>false</self_collide>
-      <material value="Schunk/DarkGolden" />
+      <material value="Schunk/Black"/>
     </gazebo>
     <gazebo reference="${name}_3_link">
-      <material value="Schunk/DarkGolden" />
-      <turnGravityOff>false</turnGravityOff>
+      <gravity>true</gravity>
+      <self_collide>false</self_collide>
+      <material value="Schunk/LightGrey"/>
     </gazebo>
     <gazebo reference="${name}_4_link">
       <gravity>true</gravity>
       <self_collide>false</self_collide>
-      <material value="Schunk/DarkGolden" />
+      <material value="Schunk/Black"/>
     </gazebo>
     <gazebo reference="${name}_5_link">
       <gravity>true</gravity>
       <self_collide>false</self_collide>
-      <material value="Schunk/DarkGolden" />
+      <material value="Schunk/LightGrey"/>
     </gazebo>
     <gazebo reference="${name}_6_link">
       <gravity>true</gravity>
       <self_collide>false</self_collide>
-      <material value="Schunk/DarkGolden" />
+      <material value="Schunk/Black"/>
     </gazebo>
     <gazebo reference="${name}_7_link">
       <gravity>true</gravity>
       <self_collide>false</self_collide>
-      <material value="Schunk/DarkGolden" />
+      <material value="Schunk/LightGrey"/>
     </gazebo>
   </xacro:macro>

File: schunk_description/urdf/lwa4d/lwa4d.urdf.xacro (robot description, xacro)
@@ -1,10 +1,10 @@
 <?xml version="1.0"?>
 <robot xmlns:xacro="http://www.ros.org/wiki/xacro">
-  <xacro:include filename="$(find schunk_description)/urdf/lwa4d/lwa4d.gazebo.xacro" />
-  <xacro:include filename="$(find schunk_description)/urdf/lwa4d/lwa4d.transmission.xacro" />
+  <xacro:include filename="$(find schunk_description)/urdf/lwa4d/lwa4d.gazebo.xacro"/>
+  <xacro:include filename="$(find schunk_description)/urdf/lwa4d/lwa4d.transmission.xacro"/>
   <xacro:macro name="schunk_lwa4d" params="parent name *origin arm_1_ref arm_2_ref arm_3_ref arm_4_ref arm_5_ref arm_6_ref arm_7_ref">
     <!-- joint between base_link and arm_base_link -->
     <joint name="${name}_base_joint" type="fixed">
-      <insert_block name="origin" />
+      <insert_block name="origin"/>
       <parent link="${parent}"/>
       <child link="${name}_base_link"/>
@@ -12,15 +12,15 @@
     <link name="${name}_base_link">
       <xacro:cylinder_inertial radius="0.06" length="0.156" mass="3.6">
-        <origin xyz="0 0 ${0.09}" rpy="0 0 0" />
-      </xacro:cylinder_inertial>
-      <visual>
-        <origin xyz="0 0 0.004" rpy="0 0 0" />
+        <origin xyz="0 0 ${0.09}" rpy="0 0 0"/>
+      </xacro:cylinder_inertial>
+      <visual>
+        <origin xyz="0 0 0.004" rpy="0 0 0"/>
         <geometry>
           <cylinder radius="0.045" length="0.08"/>
         </geometry>
-        <material name="Schunk/Black" />
-      </visual>
-      <collision>
-        <origin xyz="0 0 0.005" rpy="0 0 0" />
+        <material name="Schunk/Black"/>
+      </visual>
+      <collision>
+        <origin xyz="0 0 0.005" rpy="0 0 0"/>
         <geometry>
           <box size="0.01 0.01 0.01"/>
@@ -39,17 +39,17 @@
     <link name="${name}_1_link">
       <xacro:cylinder_inertial radius="0.06" length="0.156" mass="3.6">
-          <origin xyz="0 0.02 ${-0.15}" rpy="0 0 0" />
-      </xacro:cylinder_inertial>
-      <visual>
-        <origin xyz="0 0 -0.15" rpy="0 0 ${M_PI}" />
-        <geometry>
-          <mesh filename="package://schunk_description/meshes/lwa4d/arm_1_link.stl" />
-        </geometry>
-        <material name="Schunk/LightGrey" />
-      </visual>
-      <collision>
-        <origin xyz="0 0 -0.15" rpy="0 0 ${M_PI}" />
-        <geometry>
-          <mesh filename="package://schunk_description/meshes/lwa4d/arm_1_link.stl" />
+          <origin xyz="0 0.02 ${-0.15}" rpy="0 0 0"/>
+      </xacro:cylinder_inertial>
+      <visual>
+        <origin xyz="0 0 -0.15" rpy="0 0 ${M_PI}"/>
+        <geometry>
+          <mesh filename="package://schunk_description/meshes/lwa4d/arm_1_link.stl"/>
+        </geometry>
+        <material name="Schunk/LightGrey"/>
+      </visual>
+      <collision>
+        <origin xyz="0 0 -0.15" rpy="0 0 ${M_PI}"/>
+        <geometry>
+          <mesh filename="package://schunk_description/meshes/lwa4d/arm_1_link.stl"/>
         </geometry>
       </collision>
@@ -66,17 +66,17 @@
     <link name="${name}_2_link">
       <xacro:cylinder_inertial radius="0.056" length="0.134" mass="2.0">
-        <origin xyz="0 0.15 0" rpy="0 0 0" />
-      </xacro:cylinder_inertial>
-      <visual>
-        <origin xyz="0 0 0" rpy="0 0 ${M_PI}" />
-        <geometry>
-          <mesh filename="package://schunk_description/meshes/lwa4d/arm_2_link.stl" />
-        </geometry>
-        <material name="Schunk/Black" />
-      </visual>
-      <collision>
-        <origin xyz="0 0 0" rpy="0 0 ${M_PI}" />
-        <geometry>
-          <mesh filename="package://schunk_description/meshes/lwa4d/arm_2_link.stl" />
+        <origin xyz="0 0.15 0" rpy="0 0 0"/>
+      </xacro:cylinder_inertial>
+      <visual>
+        <origin xyz="0 0 0" rpy="0 0 ${M_PI}"/>
+        <geometry>
+          <mesh filename="package://schunk_description/meshes/lwa4d/arm_2_link.stl"/>
+        </geometry>
+        <material name="Schunk/Black"/>
+      </visual>
+      <collision>
+        <origin xyz="0 0 0" rpy="0 0 ${M_PI}"/>
+        <geometry>
+          <mesh filename="package://schunk_description/meshes/lwa4d/arm_2_link.stl"/>
         </geometry>
       </collision>
@@ -93,17 +93,17 @@
     <link name="${name}_3_link">
       <xacro:cylinder_inertial radius="0.056" length="0.134" mass="2.0">
-        <origin xyz="0.0 0.03 ${-0.39}" rpy="0 0 0" />
-      </xacro:cylinder_inertial>
-      <visual>
-        <origin xyz="0 0 -0.39" rpy="0 0 ${M_PI}" />
-        <geometry>
-          <mesh filename="package://schunk_description/meshes/lwa4d/arm_3_link.stl" />
-        </geometry>
-        <material name="Schunk/LightGrey" />
-      </visual>
-      <collision>
-        <origin xyz="0 0 -0.39" rpy="0 0 ${M_PI}" />
-        <geometry>
-          <mesh filename="package://schunk_description/meshes/lwa4d/arm_3_link.stl" />
+        <origin xyz="0.0 0.03 ${-0.39}" rpy="0 0 0"/>
+      </xacro:cylinder_inertial>
+      <visual>
+        <origin xyz="0 0 -0.39" rpy="0 0 ${M_PI}"/>
+        <geometry>
+          <mesh filename="package://schunk_description/meshes/lwa4d/arm_3_link.stl"/>
+        </geometry>
+        <material name="Schunk/LightGrey"/>
+      </visual>
+      <collision>
+        <origin xyz="0 0 -0.39" rpy="0 0 ${M_PI}"/>
+        <geometry>
+          <mesh filename="package://schunk_description/meshes/lwa4d/arm_3_link.stl"/>
         </geometry>
       </collision>
@@ -114,22 +114,22 @@
       <parent link="${name}_3_link"/>
       <child link="${name}_4_link"/>
-      <axis xyz="0 0 1" />
+      <axis xyz="0 0 1"/>
       <limit effort="81.5" velocity="0.4189" lower="-${M_PI}" upper="${M_PI}"/>
     </joint>
     <link name="${name}_4_link">
       <xacro:cylinder_inertial radius="0.056" length="0.134" mass="2.0">
-        <origin xyz="0 0.15 0.0" rpy="0 0 0" />
-      </xacro:cylinder_inertial>
-      <visual>
-        <origin xyz="0 0 0" rpy="0 0 ${M_PI}" />
-        <geometry>
-          <mesh filename="package://schunk_description/meshes/lwa4d/arm_4_link.stl" />
-        </geometry>
-        <material name="Schunk/Black" />
-      </visual>
-      <collision>
-        <origin xyz="0 0 0" rpy="0 0 ${M_PI}" />
-        <geometry>
-          <mesh filename="package://schunk_description/meshes/lwa4d/arm_4_link.stl" />
+        <origin xyz="0 0.15 0.0" rpy="0 0 0"/>
+      </xacro:cylinder_inertial>
+      <visual>
+        <origin xyz="0 0 0" rpy="0 0 ${M_PI}"/>
+        <geometry>
+          <mesh filename="package://schunk_description/meshes/lwa4d/arm_4_link.stl"/>
+        </geometry>
+        <material name="Schunk/Black"/>
+      </visual>
+      <collision>
+        <origin xyz="0 0 0" rpy="0 0 ${M_PI}"/>
+        <geometry>
+          <mesh filename="package://schunk_description/meshes/lwa4d/arm_4_link.stl"/>
         </geometry>
       </collision>
@@ -137,8 +137,8 @@
     <!-- joint between arm_4_link and arm_5_link -->
     <joint name="${name}_5_joint" type="revolute">
-      <origin xyz="0 0 0" rpy="${M_PI/2} 0 0" />
+      <origin xyz="0 0 0" rpy="${M_PI/2} 0 0"/>
       <parent link="${name}_4_link"/>
       <child link="${name}_5_link"/>
-      <axis xyz="0 0 1" />
+      <axis xyz="0 0 1"/>
       <calibration rising="${arm_5_ref}"/>
       <limit effort="20.7" velocity="0.43633" lower="-${M_PI}" upper="${M_PI}"/>
@@ -146,17 +146,17 @@
     <link name="${name}_5_link">
       <xacro:cylinder_inertial radius="0.0445" length="0.052" mass="0.4">
-        <origin xyz="0 0.05 -0.24" rpy="0 0 0" />
-      </xacro:cylinder_inertial>
-      <visual>
-        <origin xyz="0 0 -0.323" rpy="0 0 ${M_PI}" />
-        <geometry>
-          <mesh filename="package://schunk_description/meshes/lwa4d/arm_5_link.stl" />
-        </geometry>
-        <material name="Schunk/LightGrey" />
-      </visual>
-      <collision>
-        <origin xyz="0 0 -0.323" rpy="0 0 ${M_PI}" />
-        <geometry>
-          <mesh filename="package://schunk_description/meshes/lwa4d/arm_5_link.stl" />
+        <origin xyz="0 0.05 -0.24" rpy="0 0 0"/>
+      </xacro:cylinder_inertial>
+      <visual>
+        <origin xyz="0 0 -0.323" rpy="0 0 ${M_PI}"/>
+        <geometry>
+          <mesh filename="package://schunk_description/meshes/lwa4d/arm_5_link.stl"/>
+        </geometry>
+        <material name="Schunk/LightGrey"/>
+      </visual>
+      <collision>
+        <origin xyz="0 0 -0.323" rpy="0 0 ${M_PI}"/>
+        <geometry>
+          <mesh filename="package://schunk_description/meshes/lwa4d/arm_5_link.stl"/>
         </geometry>
       </collision>
@@ -164,10 +164,10 @@
     <!-- joint between arm_5_link and arm_6_link -->
     <joint name="${name}_6_joint" type="revolute">
-      <origin xyz="0 0 -0.323" rpy="-${M_PI/2} 0 0" />
+      <origin xyz="0 0 -0.323" rpy="-${M_PI/2} 0 0"/>
       <parent link="${name}_5_link"/>
       <child link="${name}_6_link"/>
-      <axis xyz="0 0 1" />
+      <axis xyz="0 0 1"/>
       <calibration rising="${arm_6_ref}"/>
-      <limit effort="15" velocity="1.2566" lower="-2.0943951" upper="2.0943951" />
+      <limit effort="15" velocity="1.2566" lower="-2.0943951" upper="2.0943951"/>
     </joint>
     <link name="${name}_6_link">
@@ -175,17 +175,17 @@
         <origin xyz="0 -0.012 -0.013" rpy="0 0 0"/>
         <mass value="1.9"/>
-        <inertia ixx="0.002750" ixy="0" ixz="0" iyy="0.004002" iyz="0" izz="0.002830" />
+        <inertia ixx="0.002750" ixy="0" ixz="0" iyy="0.004002" iyz="0" izz="0.002830"/>
       </inertial>
       <visual>
-        <origin xyz="0 0 0" rpy="0 ${M_PI} 0" />
-        <geometry>
-          <mesh filename="package://schunk_description/meshes/lwa4d/arm_6_link.stl" />
-        </geometry>
-        <material name="Schunk/Black" />
-      </visual>
-      <collision>
-        <origin xyz="0 0 0" rpy="0 ${M_PI} 0" />
-        <geometry>
-          <mesh filename="package://schunk_description/meshes/lwa4d/arm_6_link.stl" />
+        <origin xyz="0 0 0" rpy="0 ${M_PI} 0"/>
+        <geometry>
+          <mesh filename="package://schunk_description/meshes/lwa4d/arm_6_link.stl"/>
+        </geometry>
+        <material name="Schunk/Black"/>
+      </visual>
+      <collision>
+        <origin xyz="0 0 0" rpy="0 ${M_PI} 0"/>
+        <geometry>
+          <mesh filename="package://schunk_description/meshes/lwa4d/arm_6_link.stl"/>
         </geometry>
       </collision>
@@ -193,24 +193,24 @@
     <!-- joint between arm_6_link and arm_7_link -->
     <joint name="${name}_7_joint" type="revolute">
-      <origin xyz="0 0 0" rpy="-${M_PI/2} 0 0" />
+      <origin xyz="0 0 0" rpy="-${M_PI/2} 0 0"/>
       <parent link="${name}_6_link"/>
       <child link="${name}_7_link"/>
-      <axis xyz="0 0 1" />
+      <axis xyz="0 0 1"/>
       <calibration rising="${arm_7_ref}"/>
-      <limit effort="15" velocity="1.2566" lower="-2.0943951" upper="2.0943951" />
+      <limit effort="15" velocity="1.2566" lower="-2.0943951" upper="2.0943951"/>
     </joint>
     <link name="${name}_7_link">
       <xacro:cylinder_inertial radius="0.03" length="0.035" mass="0.005">
-        <origin xyz="0 0 0.06" rpy="0 0 0" />
-      </xacro:cylinder_inertial>
-      <visual>
-        <origin xyz="0 0 0" rpy="0 0 0" />
-        <geometry>
-          <mesh filename="package://schunk_description/meshes/lwa4d/arm_7_link.stl" />
-        </geometry>
-        <material name="Schunk/LightGrey" />
-      </visual>
-      <collision>
-        <origin xyz="0 0 0.06" rpy="0 0 0" />
+        <origin xyz="0 0 0.06" rpy="0 0 0"/>
+      </xacro:cylinder_inertial>
+      <visual>
+        <origin xyz="0 0 0" rpy="0 0 0"/>
+        <geometry>
+          <mesh filename="package://schunk_description/meshes/lwa4d/arm_7_link.stl"/>
+        </geometry>
+        <material name="Schunk/LightGrey"/>
+      </visual>
+      <collision>
+        <origin xyz="0 0 0.06" rpy="0 0 0"/>
         <geometry>
           <cylinder radius="0.03" length="0.035"/>
@@ -219,6 +219,6 @@
     </link>
     <!-- extensions -->
-    <xacro:schunk_lwa4d_gazebo name="${name}" />
-    <xacro:schunk_lwa4d_transmission name="${name}" />
+    <xacro:schunk_lwa4d_gazebo name="${name}"/>
+    <xacro:schunk_lwa4d_transmission name="${name}"/>
   </xacro:macro>
 </robot>
