Commit message: added inertias and limits for lwa4d

File: schunk_description/urdf/lwa4d/lwa4d.transmission.xacro (robot description, xacro)
@@ -6,5 +6,5 @@
       <joint name="${name}_1_joint"/>
       <actuator name="${name}_1_motor">
-        <hardwareInterface>EffortJointInterface</hardwareInterface>
+        <hardwareInterface>VelocityJointInterface</hardwareInterface>
         <mechanicalReduction>1</mechanicalReduction>
       </actuator>
@@ -14,5 +14,5 @@
       <joint name="${name}_2_joint"/>
       <actuator name="${name}_2_motor">
-        <hardwareInterface>EffortJointInterface</hardwareInterface>
+        <hardwareInterface>VelocityJointInterface</hardwareInterface>
         <mechanicalReduction>1</mechanicalReduction>
       </actuator>
@@ -22,5 +22,5 @@
       <joint name="${name}_3_joint"/>
       <actuator name="${name}_3_motor">
-        <hardwareInterface>EffortJointInterface</hardwareInterface>
+        <hardwareInterface>VelocityJointInterface</hardwareInterface>
         <mechanicalReduction>1</mechanicalReduction>
       </actuator>
@@ -30,5 +30,5 @@
       <joint name="${name}_4_joint"/>
       <actuator name="${name}_4_motor">
-        <hardwareInterface>EffortJointInterface</hardwareInterface>
+        <hardwareInterface>VelocityJointInterface</hardwareInterface>
         <mechanicalReduction>1</mechanicalReduction>
       </actuator>
@@ -38,5 +38,5 @@
       <joint name="${name}_5_joint"/>
       <actuator name="${name}_5_motor">
-        <hardwareInterface>EffortJointInterface</hardwareInterface>
+        <hardwareInterface>VelocityJointInterface</hardwareInterface>
         <mechanicalReduction>1</mechanicalReduction>
       </actuator>
@@ -46,5 +46,5 @@
       <joint name="${name}_6_joint"/>
       <actuator name="${name}_6_motor">
-        <hardwareInterface>EffortJointInterface</hardwareInterface>
+        <hardwareInterface>VelocityJointInterface</hardwareInterface>
         <mechanicalReduction>1</mechanicalReduction>
       </actuator>
@@ -54,5 +54,5 @@
       <joint name="${name}_7_joint"/>
       <actuator name="${name}_7_motor">
-        <hardwareInterface>EffortJointInterface</hardwareInterface>
+        <hardwareInterface>VelocityJointInterface</hardwareInterface>
         <mechanicalReduction>1</mechanicalReduction>
       </actuator>

File: schunk_description/urdf/lwa4d/lwa4d.urdf.xacro (robot description, xacro)
@@ -11,9 +11,7 @@
     </joint>
     <link name="${name}_0_link">
-      <inertial>
-        <origin xyz="0 0 0" rpy="0 0 0"/>
-        <mass value="1.0"/>
-        <inertia ixx="0.01" ixy="0" ixz="0" iyy="0.01" iyz="0" izz="0.01" />
-      </inertial>
+      <xacro:cylinder_inertial radius="0.06" length="0.156" mass="3.6">
+        <origin xyz="0 0 ${0.09}" rpy="0 0 0" />
+      </xacro:cylinder_inertial>
       <visual>
         <origin xyz="0 0 0.004" rpy="0 0 0" />
@@ -37,15 +35,10 @@
       <axis xyz="0 0 1"/>
       <calibration rising="${arm_1_ref}"/>
-      <dynamics damping="10" />
-      <limit effort="370" velocity="2.0" lower="-6.2831853" upper="6.2831853"/>
-      <safety_controller k_position="20" k_velocity="50" soft_lower_limit="${-6.2831853 + 0.01}" soft_upper_limit="${6.2831853 - 0.01}" />
+      <limit effort="216" velocity="0.43633" lower="-${M_PI}" upper="${M_PI}"/>
     </joint>
     <link name="${name}_1_link">
-      <inertial>
-        <origin xyz="0 0 0" rpy="0 0 0" />
-        <!--mass value="5.9907"/-->
-        <mass value="2.0"/>
-        <inertia ixx="0.01" ixy="0" ixz="0" iyy="0.01" iyz="0" izz="0.01" />
-      </inertial>
+      <xacro:cylinder_inertial radius="0.06" length="0.156" mass="3.6">
+          <origin xyz="0 0.02 ${-0.15}" rpy="0 0 0" />
+      </xacro:cylinder_inertial>
       <visual>
         <origin xyz="0 0 -0.15" rpy="0 0 ${M_PI}" />
@@ -69,14 +62,10 @@
       <axis xyz="0 0 1"/>
       <calibration rising="${arm_2_ref}"/>
-      <dynamics damping="10" />
-      <limit effort="370" velocity="2.0" lower="-1.97" upper="1.97"/>
-      <safety_controller k_position="20" k_velocity="50" soft_lower_limit="${-1.97 + 0.01}"   soft_upper_limit="${1.97 - 0.01}" />
+      <limit effort="216" velocity="0.43633" lower="-${M_PI}" upper="${M_PI}"/>
     </joint>
     <link name="${name}_2_link">
-      <inertial>
-        <origin xyz="0 0 0" rpy="0 0 0"/>
-        <mass value="2.0"/>
-        <inertia ixx="0.03" ixy="0" ixz="0" iyy="0.03" iyz="0" izz="0.03" />
-      </inertial>
+      <xacro:cylinder_inertial radius="0.056" length="0.134" mass="2.0">
+        <origin xyz="0 0.15 0" rpy="0 0 0" />
+      </xacro:cylinder_inertial>
       <visual>
         <origin xyz="0 0 0" rpy="0 0 ${M_PI}" />
@@ -100,16 +89,12 @@
       <axis xyz="0 0 1"/>
       <calibration rising="${arm_3_ref}"/>
-      <dynamics damping="5" />
-      <limit effort="176" velocity="2.0" lower="-6.2831853" upper="6.2831853"/>
-      <safety_controller k_position="20" k_velocity="25" soft_lower_limit="${-6.2831853 + 0.01}" soft_upper_limit="${6.2831853 - 0.01}" />
+      <limit effort="81.5" velocity="0.4189" lower="-${M_PI}" upper="${M_PI}"/>
     </joint>
     <link name="${name}_3_link">
-      <inertial>
-        <origin xyz="0 0 0" rpy="0 0 0"/>
-        <mass value="2.0"/>
-        <inertia ixx="0.03" ixy="0" ixz="0" iyy="0.03" iyz="0" izz="0.03" />
-      </inertial>
-      <visual>
-        <origin xyz="0 0 -0.328" rpy="0 0 ${M_PI}" />
+      <xacro:cylinder_inertial radius="0.056" length="0.134" mass="2.0">
+        <origin xyz="0.0 0.03 ${-0.39}" rpy="0 0 0" />
+      </xacro:cylinder_inertial>
+      <visual>
+        <origin xyz="0 0 -0.39" rpy="0 0 ${M_PI}" />
         <geometry>
           <mesh filename="package://schunk_description/meshes/lwa4d/arm_3_link.stl" />
@@ -118,5 +103,5 @@
       </visual>
       <collision>
-        <origin xyz="0 0 -0.328" rpy="0 0 ${M_PI}" />
+        <origin xyz="0 0 -0.39" rpy="0 0 ${M_PI}" />
         <geometry>
           <mesh filename="package://schunk_description/meshes/lwa4d/arm_3_link.stl" />
@@ -126,19 +111,14 @@
     <!-- joint between arm_3_link and arm_4_link -->
     <joint name="${name}_4_joint" type="revolute">
-      <origin xyz="0 0 -0.328" rpy="-${M_PI/2} 0 0"/>
+      <origin xyz="0 0 -0.39" rpy="-${M_PI/2} 0 0"/>
       <parent link="${name}_3_link"/>
       <child link="${name}_4_link"/>
       <axis xyz="0 0 1" />
-      <calibration rising="${arm_4_ref}"/>
-      <dynamics damping="5" />
-      <limit effort="176" velocity="2.0" lower="-2.08208" upper="2.08208"/>
-      <safety_controller k_position="20" k_velocity="25" soft_lower_limit="${-2.08208 + 0.01}" soft_upper_limit="${2.08208 - 0.01}" />
+      <limit effort="81.5" velocity="0.4189" lower="-${M_PI}" upper="${M_PI}"/>
     </joint>
     <link name="${name}_4_link">
-      <inertial>
-        <origin xyz="0 0 0" rpy="0 0 0"/>
-        <mass value="2.0"/>
-        <inertia ixx="0.03" ixy="0" ixz="0" iyy="0.03" iyz="0" izz="0.03" />
-      </inertial>
+      <xacro:cylinder_inertial radius="0.056" length="0.134" mass="2.0">
+        <origin xyz="0 0.15 0.0" rpy="0 0 0" />
+      </xacro:cylinder_inertial>
       <visual>
         <origin xyz="0 0 0" rpy="0 0 ${M_PI}" />
@@ -162,14 +142,10 @@
       <axis xyz="0 0 1" />
       <calibration rising="${arm_5_ref}"/>
-      <dynamics damping="5" />
-      <limit effort="41.6" velocity="2.0" lower="-6.2831853" upper="6.2831853" />
-      <safety_controller k_position="20" k_velocity="25" soft_lower_limit="${-6.2831853 + 0.01}" soft_upper_limit="${6.2831853 - 0.01}" />
+      <limit effort="20.7" velocity="0.43633" lower="-${M_PI}" upper="${M_PI}"/>
     </joint>
     <link name="${name}_5_link">
-      <inertial>
-        <origin xyz="0 0 0" rpy="0 0 0"/>
-        <mass value="2.313272"/>
-        <inertia ixx="0.03" ixy="0" ixz="0" iyy="0.03" iyz="0" izz="0.03" />
-      </inertial>
+      <xacro:cylinder_inertial radius="0.0445" length="0.052" mass="0.4">
+        <origin xyz="0 0.05 -0.24" rpy="0 0 0" />
+      </xacro:cylinder_inertial>
       <visual>
         <origin xyz="0 0 -0.323" rpy="0 0 ${M_PI}" />
@@ -193,13 +169,11 @@
       <axis xyz="0 0 1" />
       <calibration rising="${arm_6_ref}"/>
-      <dynamics damping="5" />
-      <limit effort="20.1" velocity="2.0" lower="-1.8" upper="1.8" />
-      <safety_controller k_position="20" k_velocity="25" soft_lower_limit="${-1.8 + 0.01}" soft_upper_limit="${1.8 - 0.01}" />
+      <limit effort="15" velocity="1.2566" lower="-2.0943951" upper="2.0943951" />
     </joint>
     <link name="${name}_6_link">
       <inertial>
-        <origin xyz="0 0 0" rpy="0 0 0"/>
-        <mass value="2.057856"/>
-        <inertia ixx="0.01" ixy="0" ixz="0" iyy="0.01" iyz="0" izz="0.01" />
+        <origin xyz="0 -0.012 -0.013" rpy="0 0 0"/>
+        <mass value="1.9"/>
+        <inertia ixx="0.002750" ixy="0" ixz="0" iyy="0.004002" iyz="0" izz="0.002830" />
       </inertial>
       <visual>
@@ -224,14 +198,10 @@
       <axis xyz="0 0 1" />
       <calibration rising="${arm_7_ref}"/>
-      <dynamics damping="5" />
-      <limit effort="9.6" velocity="2.0" lower="-6.2831853" upper="6.2831853" />
-      <safety_controller k_position="20" k_velocity="25" soft_lower_limit="${-6.2831853 + 0.01}" soft_upper_limit="${6.2831853 - 0.01}" />
+      <limit effort="15" velocity="1.2566" lower="-2.0943951" upper="2.0943951" />
     </joint>
     <link name="${name}_7_link">
-      <inertial>
-        <origin xyz="0 0 0" rpy="0 0 0"/>
-        <mass value="1.120198"/>
-        <inertia ixx="0.01" ixy="0" ixz="0" iyy="0.01" iyz="0" izz="0.01" />
-      </inertial>
+      <xacro:cylinder_inertial radius="0.03" length="0.035" mass="0.005">
+        <origin xyz="0 0 0.06" rpy="0 0 0" />
+      </xacro:cylinder_inertial>
       <visual>
         <origin xyz="0 0 0" rpy="0 0 0" />
@@ -242,7 +212,7 @@
       </visual>
       <collision>
-        <origin xyz="0 0 0" rpy="0 0 0" />
-        <geometry>
-          <mesh filename="package://schunk_description/meshes/lwa4d/arm_7_link.stl" />
+        <origin xyz="0 0 0.06" rpy="0 0 0" />
+        <geometry>
+          <cylinder radius="0.03" length="0.035"/>
         </geometry>
       </collision>

Commit message: use velocity interface, fix link name

File: schunk_description/urdf/lwa4d/lwa4d.transmission.xacro (robot description, xacro)
@@ -5,5 +5,5 @@
       <type>transmission_interface/SimpleTransmission</type>
       <joint name="${name}_1_joint">
-        <hardwareInterface>EffortJointInterface</hardwareInterface>
+        <hardwareInterface>VelocityJointInterface</hardwareInterface>
       </joint>
       <actuator name="${name}_1_motor">
@@ -14,5 +14,5 @@
       <type>transmission_interface/SimpleTransmission</type>
       <joint name="${name}_2_joint">
-        <hardwareInterface>EffortJointInterface</hardwareInterface>
+        <hardwareInterface>VelocityJointInterface</hardwareInterface>
       </joint>
       <actuator name="${name}_2_motor">
@@ -23,5 +23,5 @@
       <type>transmission_interface/SimpleTransmission</type>
       <joint name="${name}_3_joint">
-        <hardwareInterface>EffortJointInterface</hardwareInterface>
+        <hardwareInterface>VelocityJointInterface</hardwareInterface>
       </joint>
       <actuator name="${name}_3_motor">
@@ -32,5 +32,5 @@
       <type>transmission_interface/SimpleTransmission</type>
       <joint name="${name}_4_joint">
-        <hardwareInterface>EffortJointInterface</hardwareInterface>
+        <hardwareInterface>VelocityJointInterface</hardwareInterface>
       </joint>
       <actuator name="${name}_4_motor">
@@ -41,5 +41,5 @@
       <type>transmission_interface/SimpleTransmission</type>
       <joint name="${name}_5_joint">
-        <hardwareInterface>EffortJointInterface</hardwareInterface>
+        <hardwareInterface>VelocityJointInterface</hardwareInterface>
       </joint>
       <actuator name="${name}_5_motor">
@@ -50,5 +50,5 @@
       <type>transmission_interface/SimpleTransmission</type>
       <joint name="${name}_6_joint">
-        <hardwareInterface>EffortJointInterface</hardwareInterface>
+        <hardwareInterface>VelocityJointInterface</hardwareInterface>
       </joint>
       <actuator name="${name}_6_motor">
@@ -59,5 +59,5 @@
       <type>transmission_interface/SimpleTransmission</type>
       <joint name="${name}_7_joint">
-        <hardwareInterface>EffortJointInterface</hardwareInterface>
+        <hardwareInterface>VelocityJointInterface</hardwareInterface>
       </joint>
       <actuator name="${name}_7_motor">

File: schunk_description/urdf/lwa4d/lwa4d.urdf.xacro (robot description, xacro)
@@ -8,7 +8,7 @@
       <insert_block name="origin" />
       <parent link="${parent}" />
-      <child link="${name}_0_link" />
-    </joint>
-    <link name="${name}_0_link">
+      <child link="${name}_base_link" />
+    </joint>
+    <link name="${name}_base_link">
       <inertial>
         <origin xyz="0 0 0" rpy="0 0 0"/>
@@ -33,5 +33,5 @@
     <joint name="${name}_1_joint" type="revolute">
       <origin xyz="0 0 0.15" rpy="0 -${M_PI} 0"/>
-      <parent link="${name}_0_link"/>
+      <parent link="${name}_base_link"/>
       <child link="${name}_1_link"/>
       <axis xyz="0 0 1"/>

Commit message: added velocity and position controllers

File: schunk_description/urdf/lwa4d/lwa4d.transmission.xacro (robot description, xacro)
@@ -1,75 +1,24 @@
 <?xml version="1.0"?>
 <robot xmlns:xacro="http://www.ros.org/wiki/xacro">
-  <xacro:macro name="schunk_lwa4d_transmission" params="name">
-    <transmission name="${name}_1_trans">
+  <xacro:macro name="schunk_lwa4d_SimpleTransmission" params="jname number">
+    <transmission name="${jname}_${number}_trans">
       <type>transmission_interface/SimpleTransmission</type>
-      <joint name="${name}_1_joint">
+      <joint name="${jname}_${number}_joint">
         <hardwareInterface>PositionJointInterface</hardwareInterface>
         <hardwareInterface>VelocityJointInterface</hardwareInterface>
       </joint>
-      <actuator name="${name}_1_motor">
-        <mechanicalReduction>1</mechanicalReduction>
-      </actuator>
-    </transmission>
-    <transmission name="${name}_2_trans">
-      <type>transmission_interface/SimpleTransmission</type>
-      <joint name="${name}_2_joint">
-        <hardwareInterface>PositionJointInterface</hardwareInterface>
-        <hardwareInterface>VelocityJointInterface</hardwareInterface>
-      </joint>
-      <actuator name="${name}_2_motor">
-        <mechanicalReduction>1</mechanicalReduction>
-      </actuator>
-    </transmission>
-    <transmission name="${name}_3_trans">
-      <type>transmission_interface/SimpleTransmission</type>
-      <joint name="${name}_3_joint">
-        <hardwareInterface>PositionJointInterface</hardwareInterface>
-        <hardwareInterface>VelocityJointInterface</hardwareInterface>
-      </joint>
-      <actuator name="${name}_3_motor">
-        <mechanicalReduction>1</mechanicalReduction>
-      </actuator>
-    </transmission>
-    <transmission name="${name}_4_trans">
-      <type>transmission_interface/SimpleTransmission</type>
-      <joint name="${name}_4_joint">
-        <hardwareInterface>PositionJointInterface</hardwareInterface>
-        <hardwareInterface>VelocityJointInterface</hardwareInterface>
-      </joint>
-      <actuator name="${name}_4_motor">
-        <mechanicalReduction>1</mechanicalReduction>
-      </actuator>
-    </transmission>
-    <transmission name="${name}_5_trans">
-      <type>transmission_interface/SimpleTransmission</type>
-      <joint name="${name}_5_joint">
-        <hardwareInterface>PositionJointInterface</hardwareInterface>
-        <hardwareInterface>VelocityJointInterface</hardwareInterface>
-      </joint>
-      <actuator name="${name}_5_motor">
-        <mechanicalReduction>1</mechanicalReduction>
-      </actuator>
-    </transmission>
-    <transmission name="${name}_6_trans">
-      <type>transmission_interface/SimpleTransmission</type>
-      <joint name="${name}_6_joint">
-        <hardwareInterface>PositionJointInterface</hardwareInterface>
-        <hardwareInterface>VelocityJointInterface</hardwareInterface>
-      </joint>
-      <actuator name="${name}_6_motor">
-        <mechanicalReduction>1</mechanicalReduction>
-      </actuator>
-    </transmission>
-    <transmission name="${name}_7_trans">
-      <type>transmission_interface/SimpleTransmission</type>
-      <joint name="${name}_7_joint">
-        <hardwareInterface>PositionJointInterface</hardwareInterface>
-        <hardwareInterface>VelocityJointInterface</hardwareInterface>
-      </joint>
-      <actuator name="${name}_7_motor">
+      <actuator name="${jname}_${number}_motor">
         <mechanicalReduction>1</mechanicalReduction>
       </actuator>
     </transmission>
   </xacro:macro>
+  <xacro:macro name="schunk_lwa4d_transmission" params="name">
+    <xacro:schunk_lwa4d_SimpleTransmission jname="${name}" number="1"></xacro:schunk_lwa4d_SimpleTransmission>
+    <xacro:schunk_lwa4d_SimpleTransmission jname="${name}" number="2"></xacro:schunk_lwa4d_SimpleTransmission>
+    <xacro:schunk_lwa4d_SimpleTransmission jname="${name}" number="3"></xacro:schunk_lwa4d_SimpleTransmission>
+    <xacro:schunk_lwa4d_SimpleTransmission jname="${name}" number="4"></xacro:schunk_lwa4d_SimpleTransmission>
+    <xacro:schunk_lwa4d_SimpleTransmission jname="${name}" number="5"></xacro:schunk_lwa4d_SimpleTransmission>
+    <xacro:schunk_lwa4d_SimpleTransmission jname="${name}" number="6"></xacro:schunk_lwa4d_SimpleTransmission>
+    <xacro:schunk_lwa4d_SimpleTransmission jname="${name}" number="7"></xacro:schunk_lwa4d_SimpleTransmission>
+  </xacro:macro>
 </robot>

File: schunk_description/urdf/pg70/pg70.transmission.xacro (robot description, xacro)
@@ -7,4 +7,6 @@
       <joint name="${name}_finger_left_joint">
         <hardwareInterface>EffortJointInterface</hardwareInterface>
+        <hardwareInterface>PositionJointInterface</hardwareInterface>
+        <hardwareInterface>VelocityJointInterface</hardwareInterface>
       </joint>
       <actuator name="${name}_finger_left_motor">
@@ -17,4 +19,6 @@
       <joint name="${name}_finger_right_joint">
         <hardwareInterface>EffortJointInterface</hardwareInterface>
+        <hardwareInterface>PositionJointInterface</hardwareInterface>
+        <hardwareInterface>VelocityJointInterface</hardwareInterface>
       </joint>
       <actuator name="${name}_finger_right_motor">
