Commit message: Updated lwa4d description

File: schunk_description/urdf/lwa4d/lwa4d.urdf.xacro (robot description, xacro)
@@ -26,4 +26,5 @@
 				<material name="Schunk/Black" />
 			</visual>
+n
 			<collision>
 				<origin xyz="0 0 0.005" rpy="0 0 0" />
@@ -35,5 +36,5 @@
 		<!-- joint between arm_0_link and arm_1_link -->
 		<joint name="${name}_1_joint" type="revolute">
-			<origin xyz="0 0 0.15" rpy="0 0 0"/>
+			<origin xyz="0 0 0.15" rpy="0 -${M_PI} 0"/>
 			<parent link="${name}_0_link"/>
 			<child link="${name}_1_link"/>
@@ -52,5 +53,5 @@
 			</inertial>
 			<visual>
-				<origin xyz="0 0 0.15" rpy="0 3.14 0" />
+				<origin xyz="0 0 -0.15" rpy="0 0 ${M_PI}" />
 				<geometry>
 					<mesh filename="package://schunk_description/meshes/lwa4d/arm_1_link.stl" />
@@ -59,5 +60,5 @@
 			</visual>
 			<collision>
-				<origin xyz="0 0 0.15" rpy="0 3.14 0" />
+				<origin xyz="0 0 -0.15" rpy="0 0 ${M_PI}" />
 				<geometry>
 					<mesh filename="package://schunk_description/meshes/lwa4d/arm_1_link.stl" />
@@ -67,5 +68,5 @@
 		<!-- joint between arm_1_link and arm_2_link -->
 		<joint name="${name}_2_joint" type="revolute">
-			<origin xyz="0 0 0.15" rpy="-1.57 0 0"/>
+			<origin xyz="0 0 -0.15" rpy="-${M_PI/2} 0 0"/>
 			<parent link="${name}_1_link"/>
 			<child link="${name}_2_link"/>
@@ -79,10 +80,9 @@
 			<inertial>
 				<origin xyz="0 0 0" rpy="0 0 0"/>
-				<!--mass value="5.734939"/-->
-				<mass value="2.0"/>
-				<inertia ixx="0.03" ixy="0" ixz="0" iyy="0.03" iyz="0" izz="0.03" />
-			</inertial>
-			<visual>
-				<origin xyz="0 0 0" rpy="0 3.14159 0" />
+				<mass value="2.0"/>
+				<inertia ixx="0.03" ixy="0" ixz="0" iyy="0.03" iyz="0" izz="0.03" />
+			</inertial>
+			<visual>
+				<origin xyz="0 0 0" rpy="0 0 ${M_PI}" />
 				<geometry>
 					<mesh filename="package://schunk_description/meshes/lwa4d/arm_2_link.stl" />
@@ -91,5 +91,5 @@
 			</visual>
 			<collision>
-				<origin xyz="0 0 0" rpy="0 3.14159 0" />
+				<origin xyz="0 0 0" rpy="0 0 ${M_PI}" />
 				<geometry>
 					<mesh filename="package://schunk_description/meshes/lwa4d/arm_2_link.stl"/>
@@ -99,5 +99,5 @@
 		<!-- joint between arm_2_link and arm_3_link -->
 		<joint name="${name}_3_joint" type="revolute">
-			<origin xyz="0 0 0" rpy="1.5708 0 0"/>
+			<origin xyz="0 0 0" rpy="${M_PI/2} 0 0"/>
 			<parent link="${name}_2_link"/>
 			<child link="${name}_3_link"/>
@@ -111,10 +111,9 @@
 			<inertial>
 				<origin xyz="0 0 0" rpy="0 0 0"/>
-				<!--mass value="4.214668"/-->
-				<mass value="2.0"/>
-				<inertia ixx="0.03" ixy="0" ixz="0" iyy="0.03" iyz="0" izz="0.03" />
-			</inertial>
-			<visual>
-				<origin xyz="0 0 0.328" rpy="0 3.1415 0" />
+				<mass value="2.0"/>
+				<inertia ixx="0.03" ixy="0" ixz="0" iyy="0.03" iyz="0" izz="0.03" />
+			</inertial>
+			<visual>
+				<origin xyz="0 0 -0.328" rpy="0 0 ${M_PI}" />
 				<geometry>
 					<mesh filename="package://schunk_description/meshes/lwa4d/arm_3_link.stl" />
@@ -123,5 +122,5 @@
 			</visual>
 			<collision>
-				<origin xyz="0 0 0.328" rpy="0 3.1415 0" />
+				<origin xyz="0 0 -0.328" rpy="0 0 ${M_PI}" />
 				<geometry>
 					<mesh filename="package://schunk_description/meshes/lwa4d/arm_3_link.stl"/>
@@ -131,5 +130,5 @@
 		<!-- joint between arm_3_link and arm_4_link -->
 		<joint name="${name}_4_joint" type="revolute">
-			<origin xyz="0 0 0.328" rpy="-1.5708 0 0"/>
+			<origin xyz="0 0 -0.328" rpy="-${M_PI/2} 0 0"/>
 			<parent link="${name}_3_link"/>
 			<child link="${name}_4_link"/>
@@ -143,10 +142,9 @@
 			<inertial>
 				<origin xyz="0 0 0" rpy="0 0 0"/>
-				<!--mass value="3.669819"/-->
-				<mass value="2.0"/>
-				<inertia ixx="0.03" ixy="0" ixz="0" iyy="0.03" iyz="0" izz="0.03" />
-			</inertial>
-			<visual>
-				<origin xyz="0 0 0" rpy="0 3.14159 0" />
+				<mass value="2.0"/>
+				<inertia ixx="0.03" ixy="0" ixz="0" iyy="0.03" iyz="0" izz="0.03" />
+			</inertial>
+			<visual>
+				<origin xyz="0 0 0" rpy="0 0 ${M_PI}" />
 				<geometry>
 					<mesh filename="package://schunk_description/meshes/lwa4d/arm_4_link.stl" />
@@ -155,5 +153,5 @@
 			</visual>
 			<collision>
-				<origin xyz="0 0 0" rpy="0 3.14159 0" />
+				<origin xyz="0 0 0" rpy="0 0 ${M_PI}" />
 				<geometry>
 					<mesh filename="package://schunk_description/meshes/lwa4d/arm_4_link.stl"/>
@@ -163,5 +161,5 @@
 		<!-- joint between arm_4_link and arm_5_link -->
 		<joint name="${name}_5_joint" type="revolute">
-			<origin xyz="0 0 0" rpy="1.5708 0 0" />
+			<origin xyz="0 0 0" rpy="${M_PI/2} 0 0" />
 			<parent link="${name}_4_link"/>
 			<child link="${name}_5_link"/>
@@ -179,5 +177,5 @@
 			</inertial>
 			<visual>
-				<origin xyz="0 0 0.323" rpy="0 3.14159 0" />
+				<origin xyz="0 0 -0.323" rpy="0 0 ${M_PI}" />
 				<geometry>
 					<mesh filename="package://schunk_description/meshes/lwa4d/arm_5_link.stl" />
@@ -186,5 +184,5 @@
 			</visual>
 			<collision>
-				<origin xyz="0 0 0.323" rpy="0 3.14159 0" />
+				<origin xyz="0 0 -0.323" rpy="0 0 ${M_PI}" />
 				<geometry>
 					<mesh filename="package://schunk_description/meshes/lwa4d/arm_5_link.stl"/>
@@ -194,5 +192,5 @@
 		<!-- joint between arm_5_link and arm_6_link -->
 		<joint name="${name}_6_joint" type="revolute">
-			<origin xyz="0 0 0.323" rpy="-1.5708 0 0" />
+			<origin xyz="0 0 -0.323" rpy="-${M_PI/2} 0 0" />
 			<parent link="${name}_5_link"/>
 			<child link="${name}_6_link"/>
@@ -210,5 +208,5 @@
 			</inertial>
 			<visual>
-				<origin xyz="0 0 0" rpy="0 0 3.14159" />
+				<origin xyz="0 0 0" rpy="0 ${M_PI} 0" />
 				<geometry>
 					<mesh filename="package://schunk_description/meshes/lwa4d/arm_6_link.stl" />
@@ -217,5 +215,5 @@
 			</visual>
 			<collision>
-				<origin xyz="0 0 0" rpy="0 0 3.14159" />
+				<origin xyz="0 0 0" rpy="0 ${M_PI} 0" />
 				<geometry>
 					<mesh filename="package://schunk_description/meshes/lwa4d/arm_6_link.stl"/>
@@ -225,5 +223,5 @@
 		<!-- joint between arm_6_link and arm_7_link -->
 		<joint name="${name}_7_joint" type="revolute">
-			<origin xyz="0 -0.075 0" rpy="1.5708 0 0" />
+			<origin xyz="0 0.075 0" rpy="${M_PI/2} 0 0" />
 			<parent link="${name}_6_link"/>
 			<child link="${name}_7_link"/>
@@ -241,5 +239,5 @@
 			</inertial>
 			<visual>
-				<origin xyz="0 0 -0.075" rpy="0 0 0" />
+				<origin xyz="0 0 0.075" rpy="0 ${M_PI} 0" />
 				<geometry>
 					<mesh filename="package://schunk_description/meshes/lwa4d/arm_7_link.stl" />
@@ -248,5 +246,5 @@
 			</visual>
 			<collision>
-				<origin xyz="0 0 -0.075" rpy="0 0 0" />
+				<origin xyz="0 0 0.075" rpy="0 ${M_PI} 0" />
 				<geometry>
 					<mesh filename="package://schunk_description/meshes/lwa4d/arm_7_link.stl"/>

Commit message: add pg70 gripper

File: schunk_description/urdf/lwa4d/lwa4d.urdf.xacro (robot description, xacro)
@@ -4,7 +4,7 @@
        xmlns:interface="http://playerstage.sourceforge.net/gazebo/xmlschema/#interface"
        xmlns:xacro="http://ros.org/wiki/xacro">
-	<include filename="$(find schunk_description)/urdf/lwa/lwa.gazebo.xacro" />
-	<include filename="$(find schunk_description)/urdf/lwa/lwa.transmission.xacro" />
-	<xacro:macro name="schunk_lwa" params="parent name *origin">
+	<include filename="$(find schunk_description)/urdf/lwa4d/lwa4d.gazebo.xacro" />
+	<include filename="$(find schunk_description)/urdf/lwa4d/lwa4d.transmission.xacro" />
+	<xacro:macro name="schunk_lwa4d" params="parent name *origin">
 		<!-- joint between base_link and arm_0_link -->
 		<joint name="${name}_0_joint" type="fixed" >

Commit message: fix arm_6_joint

File: schunk_description/urdf/lwa4d/lwa4d.urdf.xacro (robot description, xacro)
@@ -192,5 +192,5 @@
 		<!-- joint between arm_5_link and arm_6_link -->
 		<joint name="${name}_6_joint" type="revolute">
-			<origin xyz="0 0 -0.323" rpy="-${M_PI/2} 0 0" />
+			<origin xyz="0 0 -0.323" rpy="${M_PI/2} 0 0" />
 			<parent link="${name}_5_link"/>
 			<child link="${name}_6_link"/>
@@ -208,5 +208,5 @@
 			</inertial>
 			<visual>
-				<origin xyz="0 0 0" rpy="0 ${M_PI} 0" />
+				<origin xyz="0 0 0" rpy="0 0 ${M_PI}" />
 				<geometry>
 					<mesh filename="package://schunk_description/meshes/lwa4d/arm_6_link.stl" />
@@ -215,5 +215,5 @@
 			</visual>
 			<collision>
-				<origin xyz="0 0 0" rpy="0 ${M_PI} 0" />
+				<origin xyz="0 0 0" rpy="0 0 ${M_PI}" />
 				<geometry>
 					<mesh filename="package://schunk_description/meshes/lwa4d/arm_6_link.stl"/>
@@ -223,5 +223,5 @@
 		<!-- joint between arm_6_link and arm_7_link -->
 		<joint name="${name}_7_joint" type="revolute">
-			<origin xyz="0 0.075 0" rpy="${M_PI/2} 0 0" />
+			<origin xyz="0 -0.075 0" rpy="-${M_PI/2} 0 0" />
 			<parent link="${name}_6_link"/>
 			<child link="${name}_7_link"/>

Commit message: update lwa4d description

File: schunk_description/urdf/lwa4d/lwa4d.urdf.xacro (robot description, xacro)
@@ -53,5 +53,5 @@
 			</inertial>
 			<visual>
-				<origin xyz="0 0 -0.15" rpy="0 0 ${M_PI}" />
+				<origin xyz="0 0 0" rpy="0 0 0" />
 				<geometry>
 					<mesh filename="package://schunk_description/meshes/lwa4d/arm_1_link.stl" />
@@ -60,5 +60,5 @@
 			</visual>
 			<collision>
-				<origin xyz="0 0 -0.15" rpy="0 0 ${M_PI}" />
+				<origin xyz="0 0 0" rpy="0 0 0" />
 				<geometry>
 					<mesh filename="package://schunk_description/meshes/lwa4d/arm_1_link.stl" />
@@ -84,5 +84,5 @@
 			</inertial>
 			<visual>
-				<origin xyz="0 0 0" rpy="0 0 ${M_PI}" />
+				<origin xyz="0 0 0" rpy="0 0 0" />
 				<geometry>
 					<mesh filename="package://schunk_description/meshes/lwa4d/arm_2_link.stl" />
@@ -91,5 +91,5 @@
 			</visual>
 			<collision>
-				<origin xyz="0 0 0" rpy="0 0 ${M_PI}" />
+				<origin xyz="0 0 0" rpy="0 0 0" />
 				<geometry>
 					<mesh filename="package://schunk_description/meshes/lwa4d/arm_2_link.stl"/>
@@ -115,5 +115,5 @@
 			</inertial>
 			<visual>
-				<origin xyz="0 0 -0.328" rpy="0 0 ${M_PI}" />
+				<origin xyz="0 0 0" rpy="0 0 0" />
 				<geometry>
 					<mesh filename="package://schunk_description/meshes/lwa4d/arm_3_link.stl" />
@@ -122,5 +122,5 @@
 			</visual>
 			<collision>
-				<origin xyz="0 0 -0.328" rpy="0 0 ${M_PI}" />
+				<origin xyz="0 0 0" rpy="0 0 0" />
 				<geometry>
 					<mesh filename="package://schunk_description/meshes/lwa4d/arm_3_link.stl"/>
@@ -146,5 +146,5 @@
 			</inertial>
 			<visual>
-				<origin xyz="0 0 0" rpy="0 0 ${M_PI}" />
+				<origin xyz="0 0 0" rpy="0 0 0" />
 				<geometry>
 					<mesh filename="package://schunk_description/meshes/lwa4d/arm_4_link.stl" />
@@ -153,5 +153,5 @@
 			</visual>
 			<collision>
-				<origin xyz="0 0 0" rpy="0 0 ${M_PI}" />
+				<origin xyz="0 0 0" rpy="0 0 0" />
 				<geometry>
 					<mesh filename="package://schunk_description/meshes/lwa4d/arm_4_link.stl"/>
@@ -177,5 +177,5 @@
 			</inertial>
 			<visual>
-				<origin xyz="0 0 -0.323" rpy="0 0 ${M_PI}" />
+				<origin xyz="0 0 0" rpy="0 0 0" />
 				<geometry>
 					<mesh filename="package://schunk_description/meshes/lwa4d/arm_5_link.stl" />
@@ -184,5 +184,5 @@
 			</visual>
 			<collision>
-				<origin xyz="0 0 -0.323" rpy="0 0 ${M_PI}" />
+				<origin xyz="0 0 0" rpy="0 0 0" />
 				<geometry>
 					<mesh filename="package://schunk_description/meshes/lwa4d/arm_5_link.stl"/>
@@ -208,5 +208,5 @@
 			</inertial>
 			<visual>
-				<origin xyz="0 0 0" rpy="0 0 ${M_PI}" />
+				<origin xyz="0 0 0" rpy="0 0 0" />
 				<geometry>
 					<mesh filename="package://schunk_description/meshes/lwa4d/arm_6_link.stl" />
@@ -215,5 +215,5 @@
 			</visual>
 			<collision>
-				<origin xyz="0 0 0" rpy="0 0 ${M_PI}" />
+				<origin xyz="0 0 0" rpy="0 0 0" />
 				<geometry>
 					<mesh filename="package://schunk_description/meshes/lwa4d/arm_6_link.stl"/>
@@ -239,5 +239,5 @@
 			</inertial>
 			<visual>
-				<origin xyz="0 0 0.075" rpy="0 ${M_PI} 0" />
+				<origin xyz="0 0 0" rpy="0 0 0" />
 				<geometry>
 					<mesh filename="package://schunk_description/meshes/lwa4d/arm_7_link.stl" />
@@ -246,5 +246,5 @@
 			</visual>
 			<collision>
-				<origin xyz="0 0 0.075" rpy="0 ${M_PI} 0" />
+				<origin xyz="0 0 0" rpy="0 0 0" />
 				<geometry>
 					<mesh filename="package://schunk_description/meshes/lwa4d/arm_7_link.stl"/>

Commit message: Fix mesh files for lwa4d

File: schunk_description/urdf/lwa4d/lwa4d.urdf.xacro (robot description, xacro)
@@ -36,5 +36,5 @@
 		<!-- joint between arm_0_link and arm_1_link -->
 		<joint name="${name}_1_joint" type="revolute">
-			<origin xyz="0 0 0.15" rpy="0 -${M_PI} 0"/>
+			<origin xyz="0 0 0.1" rpy="0 -${M_PI} 0"/>
 			<parent link="${name}_0_link"/>
 			<child link="${name}_1_link"/>
@@ -68,5 +68,5 @@
 		<!-- joint between arm_1_link and arm_2_link -->
 		<joint name="${name}_2_joint" type="revolute">
-			<origin xyz="0 0 -0.15" rpy="-${M_PI/2} 0 0"/>
+			<origin xyz="0 0 -0.18" rpy="-${M_PI/2} 0 0"/>
 			<parent link="${name}_1_link"/>
 			<child link="${name}_2_link"/>

Commit message: new meshes

File: schunk_description/urdf/lwa4d/lwa4d.urdf.xacro (robot description, xacro)
@@ -223,5 +223,5 @@
 		<!-- joint between arm_6_link and arm_7_link -->
 		<joint name="${name}_7_joint" type="revolute">
-			<origin xyz="0 -0.075 0" rpy="-${M_PI/2} 0 0" />
+			<origin xyz="0 -0.075 0" rpy="${M_PI/2} 0 0" />
 			<parent link="${name}_6_link"/>
 			<child link="${name}_7_link"/>

Commit message: 27.02. current status

File: schunk_description/urdf/lwa4d/lwa4d.urdf.xacro (robot description, xacro)
@@ -36,5 +36,5 @@
 		<!-- joint between arm_0_link and arm_1_link -->
 		<joint name="${name}_1_joint" type="revolute">
-			<origin xyz="0 0 0.1" rpy="0 -${M_PI} 0"/>
+			<origin xyz="0 0 0.15" rpy="0 -${M_PI} 0"/>
 			<parent link="${name}_0_link"/>
 			<child link="${name}_1_link"/>
@@ -53,5 +53,5 @@
 			</inertial>
 			<visual>
-				<origin xyz="0 0 0" rpy="0 0 0" />
+				<origin xyz="0 0 -0.15" rpy="0 0 ${M_PI}" />
 				<geometry>
 					<mesh filename="package://schunk_description/meshes/lwa4d/arm_1_link.stl" />
@@ -60,5 +60,5 @@
 			</visual>
 			<collision>
-				<origin xyz="0 0 0" rpy="0 0 0" />
+				<origin xyz="0 0 -0.15" rpy="0 0 ${M_PI}" />
 				<geometry>
 					<mesh filename="package://schunk_description/meshes/lwa4d/arm_1_link.stl" />
@@ -68,5 +68,5 @@
 		<!-- joint between arm_1_link and arm_2_link -->
 		<joint name="${name}_2_joint" type="revolute">
-			<origin xyz="0 0 -0.18" rpy="-${M_PI/2} 0 0"/>
+			<origin xyz="0 0 -0.15" rpy="-${M_PI/2} 0 0"/>
 			<parent link="${name}_1_link"/>
 			<child link="${name}_2_link"/>
@@ -84,5 +84,5 @@
 			</inertial>
 			<visual>
-				<origin xyz="0 0 0" rpy="0 0 0" />
+				<origin xyz="0 0 0" rpy="0 0 ${M_PI}" />
 				<geometry>
 					<mesh filename="package://schunk_description/meshes/lwa4d/arm_2_link.stl" />
@@ -91,5 +91,5 @@
 			</visual>
 			<collision>
-				<origin xyz="0 0 0" rpy="0 0 0" />
+				<origin xyz="0 0 0" rpy="0 0 ${M_PI}" />
 				<geometry>
 					<mesh filename="package://schunk_description/meshes/lwa4d/arm_2_link.stl"/>
@@ -115,5 +115,5 @@
 			</inertial>
 			<visual>
-				<origin xyz="0 0 0" rpy="0 0 0" />
+				<origin xyz="0 0 -0.328" rpy="0 0 ${M_PI}" />
 				<geometry>
 					<mesh filename="package://schunk_description/meshes/lwa4d/arm_3_link.stl" />
@@ -122,5 +122,5 @@
 			</visual>
 			<collision>
-				<origin xyz="0 0 0" rpy="0 0 0" />
+				<origin xyz="0 0 -0.328" rpy="0 0 ${M_PI}" />
 				<geometry>
 					<mesh filename="package://schunk_description/meshes/lwa4d/arm_3_link.stl"/>
@@ -146,5 +146,5 @@
 			</inertial>
 			<visual>
-				<origin xyz="0 0 0" rpy="0 0 0" />
+				<origin xyz="0 0 0" rpy="0 0 ${M_PI}" />
 				<geometry>
 					<mesh filename="package://schunk_description/meshes/lwa4d/arm_4_link.stl" />
@@ -153,5 +153,5 @@
 			</visual>
 			<collision>
-				<origin xyz="0 0 0" rpy="0 0 0" />
+				<origin xyz="0 0 0" rpy="0 0 ${M_PI}" />
 				<geometry>
 					<mesh filename="package://schunk_description/meshes/lwa4d/arm_4_link.stl"/>
@@ -177,5 +177,5 @@
 			</inertial>
 			<visual>
-				<origin xyz="0 0 0" rpy="0 0 0" />
+				<origin xyz="0 0 -0.323" rpy="0 0 ${M_PI}" />
 				<geometry>
 					<mesh filename="package://schunk_description/meshes/lwa4d/arm_5_link.stl" />
@@ -184,5 +184,5 @@
 			</visual>
 			<collision>
-				<origin xyz="0 0 0" rpy="0 0 0" />
+				<origin xyz="0 0 -0.323" rpy="0 0 ${M_PI}" />
 				<geometry>
 					<mesh filename="package://schunk_description/meshes/lwa4d/arm_5_link.stl"/>
@@ -208,5 +208,5 @@
 			</inertial>
 			<visual>
-				<origin xyz="0 0 0" rpy="0 0 0" />
+				<origin xyz="0 0 0" rpy="0 0 ${M_PI}" />
 				<geometry>
 					<mesh filename="package://schunk_description/meshes/lwa4d/arm_6_link.stl" />
@@ -215,5 +215,5 @@
 			</visual>
 			<collision>
-				<origin xyz="0 0 0" rpy="0 0 0" />
+				<origin xyz="0 0 0" rpy="0 0 ${M_PI}" />
 				<geometry>
 					<mesh filename="package://schunk_description/meshes/lwa4d/arm_6_link.stl"/>
@@ -239,5 +239,5 @@
 			</inertial>
 			<visual>
-				<origin xyz="0 0 0" rpy="0 0 0" />
+				<origin xyz="0 0 -0.075" rpy="0 0 0" />
 				<geometry>
 					<mesh filename="package://schunk_description/meshes/lwa4d/arm_7_link.stl" />
@@ -246,5 +246,5 @@
 			</visual>
 			<collision>
-				<origin xyz="0 0 0" rpy="0 0 0" />
+				<origin xyz="0 0 -0.075" rpy="0 0 0" />
 				<geometry>
 					<mesh filename="package://schunk_description/meshes/lwa4d/arm_7_link.stl"/>
@@ -252,4 +252,24 @@
 			</collision>
 		</link>
+		<!--<joint name="${name}_gripper_joint" type="fixed">
+   			 <origin rpy="0 0 0" xyz="0 0 0.06"/>
+   				 <parent link="${name}_7_link"/>
+  				  <child link="${name}_gripper"/>
+ 		 </joint>
+		<link name="${name}_gripper">
+  		  <visual>
+     			 <origin rpy="0 0 0" xyz="0 0 0" />
+     			 <geometry>
+     				   <mesh filename="package://schunk_description/meshes/lwa4d/arm_gripper.stl" />
+     			 </geometry>
+     			<material name="Schunk/LightGrey" />
+   		 </visual>
+   		 <collision>
+    			  <origin xyz="0 0 0" rpy="0 0 0" />
+    			  <geometry>
+    			    <mesh filename="package://schunk_description/meshes/lwa4d/arm_gripper.stl" />
+    			  </geometry>
+   		 </collision>
+	       </link>-->
 		<!-- extensions -->
 		<xacro:schunk_lwa4d_gazebo name="${name}" />

Commit message: lwa4d: fixed offsets error

File: schunk_description/urdf/lwa4d/lwa4d.urdf.xacro (robot description, xacro)
@@ -219,5 +219,5 @@
     <!-- joint between arm_6_link and arm_7_link -->
     <joint name="${name}_7_joint" type="revolute">
-      <origin xyz="0 -0.075 0" rpy="-${M_PI/2} 0 0" />
+      <origin xyz="0 0 0" rpy="${M_PI/2} 0 0" />
       <parent link="${name}_6_link"/>
       <child link="${name}_7_link"/>
@@ -235,5 +235,5 @@
       </inertial>
       <visual>
-        <origin xyz="0 0 -0.075" rpy="0 0 0" />
+        <origin xyz="0 0 0" rpy="0 0 0" />
         <geometry>
           <mesh filename="package://schunk_description/meshes/lwa4d/arm_7_link.stl" />
@@ -242,5 +242,5 @@
       </visual>
       <collision>
-        <origin xyz="0 0 -0.075" rpy="0 0 0" />
+        <origin xyz="0 0 0" rpy="0 0 0" />
         <geometry>
           <mesh filename="package://schunk_description/meshes/lwa4d/arm_7_link.stl" />
