Commit message: pg70 description and fixed origins for lwa4d

File: schunk_description/urdf/lwa4d/lwa4d.urdf.xacro (robot description, xacro)
@@ -188,5 +188,5 @@
     <!-- joint between arm_5_link and arm_6_link -->
     <joint name="${name}_6_joint" type="revolute">
-      <origin xyz="0 0 -0.323" rpy="${M_PI/2} 0 0" />
+      <origin xyz="0 0 -0.323" rpy="-${M_PI/2} 0 0" />
       <parent link="${name}_5_link"/>
       <child link="${name}_6_link"/>
@@ -204,5 +204,5 @@
       </inertial>
       <visual>
-        <origin xyz="0 0 0" rpy="0 0 ${M_PI}" />
+        <origin xyz="0 0 0" rpy="0 ${M_PI} 0" />
         <geometry>
           <mesh filename="package://schunk_description/meshes/lwa4d/arm_6_link.stl" />
@@ -211,5 +211,5 @@
       </visual>
       <collision>
-        <origin xyz="0 0 0" rpy="0 0 ${M_PI}" />
+        <origin xyz="0 0 0" rpy="0 ${M_PI} 0" />
         <geometry>
           <mesh filename="package://schunk_description/meshes/lwa4d/arm_6_link.stl" />
@@ -219,5 +219,5 @@
     <!-- joint between arm_6_link and arm_7_link -->
     <joint name="${name}_7_joint" type="revolute">
-      <origin xyz="0 0 0" rpy="${M_PI/2} 0 0" />
+      <origin xyz="0 0 0" rpy="-${M_PI/2} 0 0" />
       <parent link="${name}_6_link"/>
       <child link="${name}_7_link"/>

File: schunk_description/urdf/pg70/pg70.gazebo.xacro (robot description, xacro)
@@ -6,9 +6,9 @@
       <turnGravityOff>false</turnGravityOff>
     </gazebo>
-    <gazebo reference="${name}_finger_1_link">
+    <gazebo reference="${name}_finger_left_link">
       <material>Schunk/LightGrey</material>
       <turnGravityOff>false</turnGravityOff>
     </gazebo>
-    <gazebo reference="${name}_finger_2_link">
+    <gazebo reference="${name}_finger_right_link">
       <material>Schunk/LightGrey</material>
       <turnGravityOff>false</turnGravityOff>

File: schunk_description/urdf/pg70/pg70.transmission.xacro (robot description, xacro)
@@ -5,5 +5,5 @@
     <transmission name="${name}_finger_trans">
       <type>transmission_interface/SimpleTransmission</type>
-      <joint name="${name}_finger_joint"/>
+      <joint name="${name}_finger_left_joint"/>
       <actuator name="${name}_finger_motor">
         <hardwareInterface>EffortJointInterface</hardwareInterface>
@@ -14,5 +14,5 @@
     <transmission name="${name}_finger_mimic_trans">
       <type>transmission_interface/SimpleTransmission</type>
-      <joint name="${name}_finger_mimic_joint"/>
+      <joint name="${name}_finger_right_joint"/>
       <actuator name="${name}_finger_mimic_motor">
         <hardwareInterface>EffortJointInterface</hardwareInterface>

File: schunk_description/urdf/pg70/pg70.urdf.xacro (robot description, xacro)
@@ -4,95 +4,83 @@
   <xacro:include filename="$(find schunk_description)/urdf/pg70/pg70.transmission.xacro" />
   <xacro:macro name="schunk_pg70" params="parent name *origin">
-    <!-- joint between arm_7_link and pg70_palm_link -->
-    <joint name="${name}_palm_joint" type="fixed" >
-      <insert_block name="origin" />
-      <parent link="${parent}" />
-      <child link="${name}_palm_link" />
-    </joint>
-    <link name="${name}_palm_link">
-      <inertial>
-        <origin xyz="0 0 0" rpy="0 0 0"/>
-        <mass value="1.0"/>
-        <inertia ixx="0.01" ixy="0" ixz="0" iyy="0.01" iyz="0" izz="0.01" />
-      </inertial>
-      <visual>
-        <origin xyz="0 0 0" rpy="0 0 0" />
-        <geometry>
-          <mesh filename="package://schunk_description/meshes/pg70/pg70.dae" />
-        </geometry>
-      </visual>
-      <collision>
-        <origin xyz="0 0 0.0425" rpy="0 0 0" />
-        <geometry>
-          <box size="0.075 0.095 0.085"/>
-        </geometry>
-      </collision>
-    </link>
-    <!-- finger1 -->
-    <!-- joint between pg70_palm_link and pg70_finger_1_link -->
-    <joint name="${name}_finger_joint" type="prismatic">
-      <origin xyz="0.0 0.03 0.077" rpy="0 0 0" />
-      <parent link="${name}_palm_link"/>
-      <child link="${name}_finger_1_link"/>
-      <calibration rising="${pg70_finger_1_ref}"/>
-      <axis xyz="0 1 0" />
-      <dynamics damping="1" />
-      <limit effort="100" lower="-0.1" upper="1.1" velocity="5"/>
-    </joint>
-    <link name="${name}_finger_1_link">
-      <inertial>
-        <origin xyz="0 0 0" rpy="0 0 0"/>
-        <mass value="0.1"/>
-        <inertia ixx="0.01" ixy="0" ixz="0" iyy="0.01" iyz="0" izz="0.01" />
-      </inertial>
-      <visual>
-        <origin xyz="0 0 0.03" rpy="0 0 0" />
-        <geometry>
-          <box size="0.03 0.01 0.060"/>
-        </geometry>
-        <material name="Schunk/LightGrey" />
-      </visual>
-      <collision>
-        <origin xyz="0 0 0.03" rpy="0 0 0" />
-        <geometry>
-          <box size="0.025 0.005 0.055"/>
-        </geometry>
-      </collision>
-    </link>
-    <!-- finger2 -->
-    <!-- joint between pg70_palm_link and pg70_finger_2_link -->
-    <joint name="${name}_finger_mimic_joint" type="prismatic">
-      <!--mimic joint="${name}_finger_joint" multiplier="1" offset="0"/-->
-      <origin xyz="0.0 -0.03 0.077" rpy="0 0 3.14" />
-      <parent link="${name}_palm_link"/>
-      <child link="${name}_finger_2_link"/>
-      <calibration rising="${pg70_finger_2_ref}"/>
-      <axis xyz="0 1 0" />
-      <dynamics damping="1" />
-      <limit effort="100" lower="-0.1" upper="1.1" velocity="5"/>
-    </joint>
-    <link name="${name}_finger_2_link">
-      <inertial>
-        <origin xyz="0 0 0" rpy="0 0 0"/>
-        <mass value="0.1"/>
-        <inertia ixx="0.01" ixy="0" ixz="0" iyy="0.01" iyz="0" izz="0.01" />
-      </inertial>
-      <visual>
-        <origin xyz="0 0 0.03" rpy="0 0 0" />
-        <geometry>
-          <box size="0.03 0.01 0.059"/>
-        </geometry>
-        <material name="Schunk/LightGrey" />
-      </visual>
-      <collision>
-        <origin xyz="0 0 0.03" rpy="0 0 0" />
-        <geometry>
-          <box size="0.025 0.005 0.055"/>
-        </geometry>
-      </collision>
-    </link>
+        <joint name="${name}_gripper_joint" type="fixed" >
+            <parent link="${parent}" />
+            <child link="${name}_gripper_link" />
+            <xacro:insert_block name="origin" />
+        </joint>
+        <link name="${name}_gripper_link">
+                <visual>
+                    <geometry>
+                        <mesh filename="package://schunk_description/meshes/pg70/pg70.dae" />
+                    </geometry>
+                    <material name="blue">
+                        <color rgba="0 0 1 1"/>
+                    </material>
+                </visual>
+                <collision>
+                    <geometry>
+                        <mesh filename="package://schunk_description/meshes/pg70/pg70.dae" />
+                    </geometry>
+                    <material name="blue">
+                        <color rgba="0 0 1 1"/>
+                    </material>
+                </collision>
+        </link>
+        <joint name="${name}_finger_left_joint" type="prismatic" >
+                <parent link="${name}_gripper_link" />
+                <child link="${name}_finger_left_link" />
+                <limit effort="100" lower="-0.001" upper="0.0345" velocity="2.0"/>
+                <calibration rising="${pg70_finger_left_ref}"/>
+                <origin xyz="0 0.0105 0.0789" rpy="0 0 0"/>
+                <axis xyz="0 1 0" />
+        </joint>
+        <link name="${name}_finger_left_link">
+                <visual>
+                    <geometry>
+                        <box size="0.03 0.01 0.01"/>
+                    </geometry>
+                    <material name="black">
+                        <color rgba="0 0 0 1"/>
+                    </material>
+                </visual>
+                <collision>
+                    <geometry>
+                        <box size="0.03 0.01 0.01"/>
+                    </geometry>
+                    <material name="black">
+                        <color rgba="0 0 0 1"/>
+                    </material>
+                </collision>
+        </link>
+        <joint name="${name}_finger_right_joint" type="prismatic" >
+                <mimic joint="${name}_gripper_left_joint" multiplier="1" offset="0"/>
+                <parent link="${name}_gripper_link" />
+                <child link="${name}_finger_right_link" />
+                <limit effort="100" lower="-0.001" upper="0.0345" velocity="2.0"/>
+                <calibration rising="${pg70_finger_right_ref}"/>
+                <origin xyz="0 -0.0105 0.0789" rpy="-0 0 0"/>
+                <axis xyz="0 -1 0" />
+        </joint>
+        <link name="${name}_finger_right_link">
+                <visual>
+                    <geometry>
+                        <box size="0.03 0.01 0.01"/>
+                    </geometry>
+                    <material name="black">
+                        <color rgba="0 0 0 1"/>
+                    </material>
+                </visual>
+                <collision>
+                    <geometry>
+                        <box size="0.03 0.01 0.01"/>
+                    </geometry>
+                    <material name="black">
+                        <color rgba="0 0 0 1"/>
+                    </material>
+                </collision>
+        </link>
     <!-- extensions -->
     <xacro:schunk_pg70_gazebo name="${name}" />
     <xacro:schunk_pg70_transmission name="${name}" />
-  </xacro:macro>
+    </xacro:macro>
 </robot>

Commit message: fix bad merge

File: schunk_description/urdf/lwa4d/lwa4d.urdf.xacro (robot description, xacro)
@@ -3,5 +3,5 @@
   <xacro:include filename="$(find schunk_description)/urdf/lwa4d/lwa4d.gazebo.xacro" />
   <xacro:include filename="$(find schunk_description)/urdf/lwa4d/lwa4d.transmission.xacro" />
-  <xacro:macro name="schunk_lwa4p_extended" params="parent name *origin arm_1_ref arm_2_ref arm_3_ref arm_4_ref arm_5_ref arm_6_ref arm_7_ref">
+  <xacro:macro name="schunk_lwa4d" params="parent name *origin arm_1_ref arm_2_ref arm_3_ref arm_4_ref arm_5_ref arm_6_ref arm_7_ref">
     <!-- joint between base_link and arm_base_link -->
     <joint name="${name}_base_joint" type="fixed">

Commit message: fixed center of mass and inertias

File: schunk_description/urdf/lwa4d/lwa4d.urdf.xacro (robot description, xacro)
@@ -90,4 +90,5 @@
       <calibration rising="${arm_3_ref}"/>
       <limit effort="81.5" velocity="0.4189" lower="-${M_PI}" upper="${M_PI}"/>
+    </joint>
     <link name="${name}_3_link">
       <xacro:cylinder_inertial radius="0.056" length="0.134" mass="2.0">
@@ -117,5 +118,5 @@
     </joint>
     <link name="${name}_4_link">
-      <xacro:cylinder_inertial radius="0.056" length="0.134" mass="2.0">
+      <xacro:cylinder_inertial radius="0.0445" length="0.1125" mass="1.2">
         <origin xyz="0 0.15 0.0" rpy="0 0 0" />
       </xacro:cylinder_inertial>
@@ -144,5 +145,5 @@
     </joint>
     <link name="${name}_5_link">
-      <xacro:cylinder_inertial radius="0.0445" length="0.052" mass="0.4">
+      <xacro:cylinder_inertial radius="0.0445" length="0.032" mass="0.2">
         <origin xyz="0 0.05 -0.24" rpy="0 0 0" />
       </xacro:cylinder_inertial>
@@ -172,5 +173,5 @@
     <link name="${name}_6_link">
       <inertial>
-        <origin xyz="0 -0.012 -0.013" rpy="0 0 0"/>
+        <origin xyz="0 0.012 0.017" rpy="0 0 0"/>
         <mass value="1.9"/>
         <inertia ixx="0.002750" ixy="0" ixz="0" iyy="0.004002" iyz="0" izz="0.002830" />

File: schunk_description/urdf/lwa4p_extended/lwa4p_extended.urdf.xacro (robot description, xacro)
@@ -43,5 +43,5 @@
     <link name="${name}_1_link">
       <inertial>
-        <origin xyz="0.0 -0.0662 -0.0473" rpy="0 0 0"/>
+        <origin xyz="0.0 0.0662 0.0473" rpy="0 0 0"/>
         <mass value="0.8"/>
         <inertia ixx="0.002034" ixy="0.0" ixz="0.0" iyy="0.001437" iyz="0.000784" izz="0.00161" />

Commit message: improve model - velocity error <0.01

File: schunk_description/urdf/lwa4d/lwa4d.urdf.xacro (robot description, xacro)
@@ -10,21 +10,21 @@
       <child link="${name}_base_link"/>
     </joint>
-    <link name="${name}_base_link">
-      <xacro:cylinder_inertial radius="0.06" length="0.156" mass="3.6">
-        <origin xyz="0 0 ${0.09}" rpy="0 0 0"/>
-      </xacro:cylinder_inertial>
-      <visual>
-        <origin xyz="0 0 0.004" rpy="0 0 0"/>
-        <geometry>
-          <cylinder radius="0.045" length="0.08"/>
-        </geometry>
-        <material name="Schunk/Black"/>
-      </visual>
-      <collision>
-        <origin xyz="0 0 0.005" rpy="0 0 0"/>
-        <geometry>
-          <box size="0.01 0.01 0.01"/>
-        </geometry>
-      </collision>
+     <link name="${name}_base_link">
+      <xacro:cylinder_inertial radius="0.045" length="0.03" mass="3.6">
+        <origin xyz="0 0 0.015" rpy="0 0 0"/>
+       </xacro:cylinder_inertial>
+       <visual>
+        <origin xyz="0 0 0.015" rpy="0 0 0"/>
+         <geometry>
+          <cylinder radius="0.045" length="0.03"/>
+         </geometry>
+         <material name="Schunk/Black"/>
+       </visual>
+       <collision>
+        <origin xyz="0 0 0.015" rpy="0 0 0"/>
+         <geometry>
+          <cylinder radius="0.045" length="0.03"/>
+         </geometry>
+       </collision>
     </link>
     <!-- joint between arm_0_link and arm_1_link -->
@@ -38,6 +38,6 @@
     </joint>
     <link name="${name}_1_link">
-      <xacro:cylinder_inertial radius="0.06" length="0.156" mass="3.6">
-          <origin xyz="0 0.02 ${-0.15}" rpy="0 0 0"/>
+      <xacro:cylinder_inertial radius="0.06" length="0.150" mass="3.6">
+          <origin xyz="0 0 0.02" rpy="0 0 0"/>
       </xacro:cylinder_inertial>
       <visual>
@@ -65,6 +65,6 @@
     </joint>
     <link name="${name}_2_link">
-      <xacro:cylinder_inertial radius="0.056" length="0.134" mass="2.0">
-        <origin xyz="0 0.15 0" rpy="0 0 0"/>
+      <xacro:cylinder_inertial radius="0.06" length="0.150" mass="2.0">
+        <origin xyz="0 0 0" rpy="0 0 0"/>
       </xacro:cylinder_inertial>
       <visual>
@@ -78,5 +78,5 @@
         <origin xyz="0 0 0" rpy="0 0 ${M_PI}"/>
         <geometry>
-          <mesh filename="package://schunk_description/meshes/lwa4d/arm_2_link.stl"/>
+          <mesh filename="package://schunk_description/meshes/lwa4d/arm_2_link_collision.stl"/>
         </geometry>
       </collision>
@@ -92,6 +92,6 @@
     </joint>
     <link name="${name}_3_link">
-      <xacro:cylinder_inertial radius="0.056" length="0.134" mass="2.0">
-        <origin xyz="0.0 0.03 ${-0.39}" rpy="0 0 0"/>
+      <xacro:cylinder_inertial radius="0.06" length="0.2" mass="2.0">
+        <origin xyz="0.0 0 -0.2" rpy="0 0 0"/>
       </xacro:cylinder_inertial>
       <visual>
@@ -105,5 +105,5 @@
         <origin xyz="0 0 -0.39" rpy="0 0 ${M_PI}"/>
         <geometry>
-          <mesh filename="package://schunk_description/meshes/lwa4d/arm_3_link.stl"/>
+          <mesh filename="package://schunk_description/meshes/lwa4d/arm_3_link_collision.stl"/>
         </geometry>
       </collision>
@@ -115,9 +115,10 @@
       <child link="${name}_4_link"/>
       <axis xyz="0 0 1"/>
+      <calibration rising="${arm_4_ref}"/>
       <limit effort="81.5" velocity="0.4189" lower="-${M_PI}" upper="${M_PI}"/>
     </joint>
     <link name="${name}_4_link">
-      <xacro:cylinder_inertial radius="0.0445" length="0.1125" mass="1.2">
-        <origin xyz="0 0.15 0.0" rpy="0 0 0"/>
+      <xacro:cylinder_inertial radius="0.06" length="0.150" mass="1.2">
+        <origin xyz="0 0 0" rpy="0 0 0"/>
       </xacro:cylinder_inertial>
       <visual>
@@ -131,5 +132,5 @@
         <origin xyz="0 0 0" rpy="0 0 ${M_PI}"/>
         <geometry>
-          <mesh filename="package://schunk_description/meshes/lwa4d/arm_4_link.stl"/>
+          <mesh filename="package://schunk_description/meshes/lwa4d/arm_4_link_collision.stl"/>
         </geometry>
       </collision>
@@ -145,6 +146,6 @@
     </joint>
     <link name="${name}_5_link">
-      <xacro:cylinder_inertial radius="0.0445" length="0.032" mass="0.2">
-        <origin xyz="0 0.05 -0.24" rpy="0 0 0"/>
+      <xacro:cylinder_inertial radius="0.06" length="0.15" mass="1.2">
+        <origin xyz="0 0 -0.18" rpy="0 0 0"/>
       </xacro:cylinder_inertial>
       <visual>
@@ -158,5 +159,5 @@
         <origin xyz="0 0 -0.323" rpy="0 0 ${M_PI}"/>
         <geometry>
-          <mesh filename="package://schunk_description/meshes/lwa4d/arm_5_link.stl"/>
+          <mesh filename="package://schunk_description/meshes/lwa4d/arm_5_link_collision.stl"/>
         </geometry>
       </collision>
@@ -172,9 +173,7 @@
     </joint>
     <link name="${name}_6_link">
-      <inertial>
-        <origin xyz="0 0.012 0.017" rpy="0 0 0"/>
-        <mass value="1.9"/>
-        <inertia ixx="0.002750" ixy="0" ixz="0" iyy="0.004002" iyz="0" izz="0.002830"/>
-      </inertial>
+      <xacro:sphere_inertial radius="0.05" mass="1.9">
+        <origin xyz="0 0 0" rpy="0 0 0"/>
+      </xacro:sphere_inertial>
       <visual>
         <origin xyz="0 0 0" rpy="0 ${M_PI} 0"/>
@@ -187,5 +186,5 @@
         <origin xyz="0 0 0" rpy="0 ${M_PI} 0"/>
         <geometry>
-          <mesh filename="package://schunk_description/meshes/lwa4d/arm_6_link.stl"/>
+          <mesh filename="package://schunk_description/meshes/lwa4d/arm_6_link_collision.stl"/>
         </geometry>
       </collision>
@@ -201,11 +200,11 @@
     </joint>
     <link name="${name}_7_link">
-      <xacro:cylinder_inertial radius="0.03" length="0.035" mass="0.005">
+      <xacro:cylinder_inertial radius="0.03" length="0.035" mass="0.05">
         <origin xyz="0 0 0.06" rpy="0 0 0"/>
       </xacro:cylinder_inertial>
       <visual>
-        <origin xyz="0 0 0" rpy="0 0 0"/>
-        <geometry>
-          <mesh filename="package://schunk_description/meshes/lwa4d/arm_7_link.stl"/>
+        <origin xyz="0 0 0.06" rpy="0 0 0"/>
+        <geometry>
+          <cylinder radius="0.03" length="0.035"/>
         </geometry>
         <material name="Schunk/LightGrey"/>
