Commit message: inertia go to hell

File: schunk_description/urdf/lwa4d/lwa4d.urdf.xacro (robot description, xacro)
@@ -11,7 +11,10 @@
     </joint>
      <link name="${name}_base_link">
+      <xacro:default_inertial/>
+<!--
       <xacro:cylinder_inertial radius="0.045" length="0.03" mass="3.6">
         <origin xyz="0 0 0.015" rpy="0 0 0"/>
        </xacro:cylinder_inertial>
+-->
        <visual>
         <origin xyz="0 0 0.015" rpy="0 0 0"/>
@@ -38,7 +41,10 @@
     </joint>
     <link name="${name}_1_link">
+      <xacro:default_inertial/>
+<!--
       <xacro:cylinder_inertial radius="0.06" length="0.150" mass="3.6">
           <origin xyz="0 0 0.02" rpy="0 0 0"/>
       </xacro:cylinder_inertial>
+-->
       <visual>
         <origin xyz="0 0 -0.15" rpy="0 0 ${M_PI}"/>
@@ -65,7 +71,10 @@
     </joint>
     <link name="${name}_2_link">
+      <xacro:default_inertial/>
+<!--
       <xacro:cylinder_inertial radius="0.06" length="0.150" mass="2.0">
         <origin xyz="0 0 0" rpy="0 0 0"/>
       </xacro:cylinder_inertial>
+-->
       <visual>
         <origin xyz="0 0 0" rpy="0 0 ${M_PI}"/>
@@ -92,7 +101,10 @@
     </joint>
     <link name="${name}_3_link">
+      <xacro:default_inertial/>
+<!--
       <xacro:cylinder_inertial radius="0.06" length="0.2" mass="2.0">
         <origin xyz="0.0 0 -0.2" rpy="0 0 0"/>
       </xacro:cylinder_inertial>
+-->
       <visual>
         <origin xyz="0 0 -0.39" rpy="0 0 ${M_PI}"/>
@@ -119,7 +131,10 @@
     </joint>
     <link name="${name}_4_link">
+      <xacro:default_inertial/>
+<!--
       <xacro:cylinder_inertial radius="0.06" length="0.150" mass="1.2">
         <origin xyz="0 0 0" rpy="0 0 0"/>
       </xacro:cylinder_inertial>
+-->
       <visual>
         <origin xyz="0 0 0" rpy="0 0 ${M_PI}"/>
@@ -146,7 +161,10 @@
     </joint>
     <link name="${name}_5_link">
+      <xacro:default_inertial/>
+<!--
       <xacro:cylinder_inertial radius="0.06" length="0.15" mass="1.2">
         <origin xyz="0 0 -0.18" rpy="0 0 0"/>
       </xacro:cylinder_inertial>
+-->
       <visual>
         <origin xyz="0 0 -0.323" rpy="0 0 ${M_PI}"/>
@@ -173,7 +191,10 @@
     </joint>
     <link name="${name}_6_link">
+      <xacro:default_inertial/>
+<!--
       <xacro:sphere_inertial radius="0.05" mass="1.9">
         <origin xyz="0 0 0" rpy="0 0 0"/>
       </xacro:sphere_inertial>
+-->
       <visual>
         <origin xyz="0 0 0" rpy="0 ${M_PI} 0"/>
@@ -200,7 +221,10 @@
     </joint>
     <link name="${name}_7_link">
+      <xacro:default_inertial/>
+<!--
       <xacro:cylinder_inertial radius="0.03" length="0.035" mass="0.05">
         <origin xyz="0 0 0.06" rpy="0 0 0"/>
       </xacro:cylinder_inertial>
+-->
       <visual>
         <origin xyz="0 0 0.06" rpy="0 0 0"/>

File: schunk_description/urdf/lwa4p_extended/lwa4p_extended.urdf.xacro (robot description, xacro)
@@ -12,7 +12,10 @@
     <!-- static part of PRL100 -->
     <link name="${name}_base_link">
-      <xacro:cylinder_inertial radius="0.056" length="0.134" mass="2.0">
-        <origin xyz="0 0 ${0.134/2}" rpy="0 0 0" />
+      <xacro:default_inertial/>
+<!--
+      <xacro:cylinder_inertial radius="0.056" length="0.12" mass="2.0">
+        <origin xyz="0 0 ${0.12/2}" rpy="0 0 0" />
       </xacro:cylinder_inertial>
+-->
       <visual>
         <origin xyz="0 0 0" rpy="0 0 0" />
@@ -36,5 +39,4 @@
       <calibration rising="${arm_1_ref}"/>
       <dynamics damping="0" friction="0"/>
-      <!--limit effort="81.5" velocity="0.42" lower="-6.2831853" upper="6.2831853"/-->
       <limit effort="81.5" velocity="0.42" lower="-${M_PI}" upper="${M_PI}"/>
       <!--safety_controller k_position="20" k_velocity="50" soft_lower_limit="${-M_PI + 0.01}" soft_upper_limit="${M_PI - 0.01}" /-->
@@ -42,4 +44,6 @@
     <!-- prl100 rotor + shoulder flansh -->
     <link name="${name}_1_link">
+      <xacro:default_inertial/>
+<!--
       <inertial>
         <origin xyz="0.0 0.0662 0.0473" rpy="0 0 0"/>
@@ -47,4 +51,5 @@
         <inertia ixx="0.002034" ixy="0.0" ixz="0.0" iyy="0.001437" iyz="0.000784" izz="0.00161" />
       </inertial>
+-->
       <visual>
         <origin xyz="0 0 0" rpy="0 0 0" />
@@ -72,4 +77,6 @@
     </joint>
     <link name="${name}_2_link">
+      <xacro:default_inertial/>
+<!--
       <inertial>
         <origin xyz="0 0.018 -0.018" rpy="0 0 0"/>
@@ -77,4 +84,5 @@
         <inertia ixx="0.009780" ixy="0.0" ixz="0.0" iyy="0.013300" iyz="0.0" izz="0.009780" />
       </inertial>
+-->
       <visual>
         <origin xyz="0 0 0" rpy="0 0 0" />
@@ -86,5 +94,5 @@
         <origin xyz="0 0 0" rpy="0 0 0" />
         <geometry>
-          <mesh filename="package://schunk_description/meshes/lwa4p_extended/arm_2_link.dae" />
+          <mesh filename="package://schunk_description/meshes/lwa4p_extended/arm_2_collision.stl" />
         </geometry>
       </collision>
@@ -98,9 +106,10 @@
       <calibration rising="${arm_3_ref}"/>
       <dynamics damping="0" friction="0"/>
-      <!--limit effort="48" velocity="1.2566" lower="-6.2831853" upper="6.2831853"/-->
       <limit effort="48" velocity="1.2566" lower="-${M_PI}" upper="${M_PI}"/>
       <!--safety_controller k_position="20" k_velocity="25" soft_lower_limit="${-M_PI + 0.01}" soft_upper_limit="${M_PI - 0.01}" /-->
     </joint>
     <link name="${name}_3_link">
+      <xacro:default_inertial/>
+<!--
       <inertial>
         <origin xyz="0.0 0.06247 0.23425" rpy="0 0 0"/>
@@ -108,4 +117,5 @@
         <inertia ixx="0.0344" ixy="0.0" ixz="0.0077" iyy="0.0362" iyz="0.0" izz="0.0052" />
       </inertial>
+-->
       <visual>
         <origin xyz="0 0 0" rpy="0 0 0" />
@@ -133,4 +143,6 @@
     </joint>
     <link name="${name}_4_link">
+      <xacro:default_inertial/>
+<!--
       <inertial>
         <origin xyz="0 0.018 -0.018" rpy="0 0 0"/>
@@ -138,4 +150,5 @@
         <inertia ixx="0.009780" ixy="0.0" ixz="0.0" iyy="0.013300" iyz="0.0" izz="0.009780" />
       </inertial>
+-->
       <visual>
         <origin xyz="0 0 0" rpy="0 0 0" />
@@ -147,5 +160,5 @@
         <origin xyz="0 0 0" rpy="0 0 0" />
         <geometry>
-          <mesh filename="package://schunk_description/meshes/lwa4p_extended/arm_4_link.dae" />
+          <mesh filename="package://schunk_description/meshes/lwa4p_extended/arm_4_collision.stl" />
         </geometry>
       </collision>
@@ -159,9 +172,10 @@
       <calibration rising="${arm_5_ref}"/>
       <dynamics damping="0" friction="0"/>
-      <!--limit effort="48" velocity="1.2566" lower="-6.2831853" upper="6.2831853" /-->
       <limit effort="48" velocity="1.2566" lower="-${M_PI}" upper="${M_PI}" />
       <!--safety_controller k_position="20" k_velocity="25" soft_lower_limit="${-M_PI + 0.01}" soft_upper_limit="${M_PI - 0.01}" /-->
     </joint>
     <link name="${name}_5_link">
+      <xacro:default_inertial/>
+<!--
       <inertial>
         <origin xyz="0.0 0.04175 0.17026" rpy="0 0 0"/>
@@ -169,4 +183,5 @@
         <inertia ixx="0.01" ixy="0.0" ixz="-0.0031" iyy="0.0111" iyz="0.0" izz="0.0031" />
       </inertial>
+-->
       <visual>
         <origin xyz="0 0 0" rpy="0 0 0" />
@@ -194,4 +209,6 @@
     </joint>
     <link name="${name}_6_link">
+      <xacro:default_inertial/>
+<!--
       <inertial>
         <origin xyz="0 0.012 -0.012" rpy="0 0 0"/>
@@ -199,4 +216,5 @@
         <inertia ixx="0.002750" ixy="0.0" ixz="0.0" iyy="0.004002" iyz="0.0" izz="0.002830" />
       </inertial>
+-->
       <visual>
         <origin xyz="0 0 0" rpy="0 0 0" />
@@ -208,5 +226,5 @@
         <origin xyz="0 0 0" rpy="0 0 0" />
         <geometry>
-          <mesh filename="package://schunk_description/meshes/lwa4p_extended/arm_6_link.dae" />
+          <mesh filename="package://schunk_description/meshes/lwa4p_extended/arm_6_collision.stl" />
         </geometry>
       </collision>
@@ -224,7 +242,23 @@
     </joint>
     <link name="${name}_7_link">
-      <xacro:box_inertial x="0.01" y="0.01" z="0.01" mass="0.01">
-        <origin xyz="0 0 0.1" rpy="0 0 0" />
-      </xacro:box_inertial>
+      <xacro:default_inertial/>
+<!--
+      <xacro:cylinder_inertial radius="0.03" length="0.035" mass="0.05">
+        <origin xyz="0 0 0.06" rpy="0 0 0"/>
+      </xacro:cylinder_inertial>
+-->
+      <visual>
+        <origin xyz="0 0 0.06" rpy="0 0 0"/>
+        <geometry>
+          <cylinder radius="0.03" length="0.035"/>
+        </geometry>
+        <material name="Schunk/LightGrey"/>
+      </visual>
+      <collision>
+        <origin xyz="0 0 0.06" rpy="0 0 0"/>
+        <geometry>
+          <cylinder radius="0.03" length="0.035"/>
+        </geometry>
+      </collision>
     </link>
     <!-- extensions -->

Commit message: Update lwa4d.urdf.xacro
According to HW limits

File: schunk_description/urdf/lwa4d/lwa4d.urdf.xacro (robot description, xacro)
@@ -68,5 +68,5 @@
       <axis xyz="0 0 1"/>
       <calibration rising="${arm_2_ref}"/>
-      <limit effort="216" velocity="0.43633" lower="-${M_PI}" upper="${M_PI}"/>
+      <limit effort="216" velocity="0.43633" lower="-2.14" upper="2.14"/>
     </joint>
     <link name="${name}_2_link">
@@ -128,5 +128,5 @@
       <axis xyz="0 0 1"/>
       <calibration rising="${arm_4_ref}"/>
-      <limit effort="81.5" velocity="0.4189" lower="-${M_PI}" upper="${M_PI}"/>
+      <limit effort="81.5" velocity="0.4189" lower="-2.18" upper="2.18"/>
     </joint>
     <link name="${name}_4_link">
@@ -188,5 +188,5 @@
       <axis xyz="0 0 1"/>
       <calibration rising="${arm_6_ref}"/>
-      <limit effort="15" velocity="1.2566" lower="-2.0943951" upper="2.0943951"/>
+      <limit effort="15" velocity="1.2566" lower="-2.0" upper="2.0"/>
     </joint>
     <link name="${name}_6_link">

Commit message: updated schunk_lwa4d description

File: schunk_description/urdf/lwa4d/lwa4d.urdf.xacro (robot description, xacro)
@@ -1,6 +1,5 @@
 <?xml version="1.0"?>
 <robot xmlns:xacro="http://www.ros.org/wiki/xacro">
-  <xacro:include filename="$(find schunk_description)/urdf/lwa4d/lwa4d.gazebo.xacro"/>
-  <xacro:include filename="$(find schunk_description)/urdf/lwa4d/lwa4d.transmission.xacro"/>
+  <xacro:include filename="$(find schunk_description)/urdf/lwa4d/lwa4d_without_base.urdf.xacro"/>
   <xacro:macro name="schunk_lwa4d" params="parent name *origin arm_1_ref arm_2_ref arm_3_ref arm_4_ref arm_5_ref arm_6_ref arm_7_ref">
     <!-- joint between base_link and arm_base_link -->
@@ -31,217 +30,14 @@
        </collision>
     </link>
-    <!-- joint between arm_0_link and arm_1_link -->
-    <joint name="${name}_1_joint" type="revolute">
-      <origin xyz="0 0 0.15" rpy="0 -${M_PI} 0"/>
-      <parent link="${name}_base_link"/>
-      <child link="${name}_1_link"/>
-      <axis xyz="0 0 1"/>
-      <calibration rising="${arm_1_ref}"/>
-      <limit effort="216" velocity="0.43633" lower="-${M_PI}" upper="${M_PI}"/>
-    </joint>
-    <link name="${name}_1_link">
-      <xacro:default_inertial/>
-<!--
-      <xacro:cylinder_inertial radius="0.06" length="0.150" mass="3.6">
-          <origin xyz="0 0 0.02" rpy="0 0 0"/>
-      </xacro:cylinder_inertial>
--->
-      <visual>
-        <origin xyz="0 0 -0.15" rpy="0 0 ${M_PI}"/>
-        <geometry>
-          <mesh filename="package://schunk_description/meshes/lwa4d/arm_1_link.stl"/>
-        </geometry>
-        <material name="Schunk/LightGrey"/>
-      </visual>
-      <collision>
-        <origin xyz="0 0 -0.15" rpy="0 0 ${M_PI}"/>
-        <geometry>
-          <mesh filename="package://schunk_description/meshes/lwa4d/arm_1_link.stl"/>
-        </geometry>
-      </collision>
-    </link>
-    <!-- joint between arm_1_link and arm_2_link -->
-    <joint name="${name}_2_joint" type="revolute">
-      <origin xyz="0 0 -0.15" rpy="-${M_PI/2} 0 0"/>
-      <parent link="${name}_1_link"/>
-      <child link="${name}_2_link"/>
-      <axis xyz="0 0 1"/>
-      <calibration rising="${arm_2_ref}"/>
-      <limit effort="216" velocity="0.43633" lower="-${M_PI}" upper="${M_PI}"/>
-    </joint>
-    <link name="${name}_2_link">
-      <xacro:default_inertial/>
-<!--
-      <xacro:cylinder_inertial radius="0.06" length="0.150" mass="2.0">
-        <origin xyz="0 0 0" rpy="0 0 0"/>
-      </xacro:cylinder_inertial>
--->
-      <visual>
-        <origin xyz="0 0 0" rpy="0 0 ${M_PI}"/>
-        <geometry>
-          <mesh filename="package://schunk_description/meshes/lwa4d/arm_2_link.stl"/>
-        </geometry>
-        <material name="Schunk/Black"/>
-      </visual>
-      <collision>
-        <origin xyz="0 0 0" rpy="0 0 ${M_PI}"/>
-        <geometry>
-          <mesh filename="package://schunk_description/meshes/lwa4d/arm_2_link_collision.stl"/>
-        </geometry>
-      </collision>
-    </link>
-    <!-- joint between arm_2_link and arm_3_link -->
-    <joint name="${name}_3_joint" type="revolute">
-      <origin xyz="0 0 0" rpy="${M_PI/2} 0 0"/>
-      <parent link="${name}_2_link"/>
-      <child link="${name}_3_link"/>
-      <axis xyz="0 0 1"/>
-      <calibration rising="${arm_3_ref}"/>
-      <limit effort="81.5" velocity="0.4189" lower="-${M_PI}" upper="${M_PI}"/>
-    </joint>
-    <link name="${name}_3_link">
-      <xacro:default_inertial/>
-<!--
-      <xacro:cylinder_inertial radius="0.06" length="0.2" mass="2.0">
-        <origin xyz="0.0 0 -0.2" rpy="0 0 0"/>
-      </xacro:cylinder_inertial>
--->
-      <visual>
-        <origin xyz="0 0 -0.39" rpy="0 0 ${M_PI}"/>
-        <geometry>
-          <mesh filename="package://schunk_description/meshes/lwa4d/arm_3_link.stl"/>
-        </geometry>
-        <material name="Schunk/LightGrey"/>
-      </visual>
-      <collision>
-        <origin xyz="0 0 -0.39" rpy="0 0 ${M_PI}"/>
-        <geometry>
-          <mesh filename="package://schunk_description/meshes/lwa4d/arm_3_link_collision.stl"/>
-        </geometry>
-      </collision>
-    </link>
-    <!-- joint between arm_3_link and arm_4_link -->
-    <joint name="${name}_4_joint" type="revolute">
-      <origin xyz="0 0 -0.39" rpy="-${M_PI/2} 0 0"/>
-      <parent link="${name}_3_link"/>
-      <child link="${name}_4_link"/>
-      <axis xyz="0 0 1"/>
-      <calibration rising="${arm_4_ref}"/>
-      <limit effort="81.5" velocity="0.4189" lower="-${M_PI}" upper="${M_PI}"/>
-    </joint>
-    <link name="${name}_4_link">
-      <xacro:default_inertial/>
-<!--
-      <xacro:cylinder_inertial radius="0.06" length="0.150" mass="1.2">
-        <origin xyz="0 0 0" rpy="0 0 0"/>
-      </xacro:cylinder_inertial>
--->
-      <visual>
-        <origin xyz="0 0 0" rpy="0 0 ${M_PI}"/>
-        <geometry>
-          <mesh filename="package://schunk_description/meshes/lwa4d/arm_4_link.stl"/>
-        </geometry>
-        <material name="Schunk/Black"/>
-      </visual>
-      <collision>
-        <origin xyz="0 0 0" rpy="0 0 ${M_PI}"/>
-        <geometry>
-          <mesh filename="package://schunk_description/meshes/lwa4d/arm_4_link_collision.stl"/>
-        </geometry>
-      </collision>
-    </link>
-    <!-- joint between arm_4_link and arm_5_link -->
-    <joint name="${name}_5_joint" type="revolute">
-      <origin xyz="0 0 0" rpy="${M_PI/2} 0 0"/>
-      <parent link="${name}_4_link"/>
-      <child link="${name}_5_link"/>
-      <axis xyz="0 0 1"/>
-      <calibration rising="${arm_5_ref}"/>
-      <limit effort="20.7" velocity="0.43633" lower="-${M_PI}" upper="${M_PI}"/>
-    </joint>
-    <link name="${name}_5_link">
-      <xacro:default_inertial/>
-<!--
-      <xacro:cylinder_inertial radius="0.06" length="0.15" mass="1.2">
-        <origin xyz="0 0 -0.18" rpy="0 0 0"/>
-      </xacro:cylinder_inertial>
--->
-      <visual>
-        <origin xyz="0 0 -0.323" rpy="0 0 ${M_PI}"/>
-        <geometry>
-          <mesh filename="package://schunk_description/meshes/lwa4d/arm_5_link.stl"/>
-        </geometry>
-        <material name="Schunk/LightGrey"/>
-      </visual>
-      <collision>
-        <origin xyz="0 0 -0.323" rpy="0 0 ${M_PI}"/>
-        <geometry>
-          <mesh filename="package://schunk_description/meshes/lwa4d/arm_5_link_collision.stl"/>
-        </geometry>
-      </collision>
-    </link>
-    <!-- joint between arm_5_link and arm_6_link -->
-    <joint name="${name}_6_joint" type="revolute">
-      <origin xyz="0 0 -0.323" rpy="-${M_PI/2} 0 0"/>
-      <parent link="${name}_5_link"/>
-      <child link="${name}_6_link"/>
-      <axis xyz="0 0 1"/>
-      <calibration rising="${arm_6_ref}"/>
-      <limit effort="15" velocity="1.2566" lower="-2.0943951" upper="2.0943951"/>
-    </joint>
-    <link name="${name}_6_link">
-      <xacro:default_inertial/>
-<!--
-      <xacro:sphere_inertial radius="0.05" mass="1.9">
-        <origin xyz="0 0 0" rpy="0 0 0"/>
-      </xacro:sphere_inertial>
--->
-      <visual>
-        <origin xyz="0 0 0" rpy="0 ${M_PI} 0"/>
-        <geometry>
-          <mesh filename="package://schunk_description/meshes/lwa4d/arm_6_link.stl"/>
-        </geometry>
-        <material name="Schunk/Black"/>
-      </visual>
-      <collision>
-        <origin xyz="0 0 0" rpy="0 ${M_PI} 0"/>
-        <geometry>
-          <mesh filename="package://schunk_description/meshes/lwa4d/arm_6_link_collision.stl"/>
-        </geometry>
-      </collision>
-    </link>
-    <!-- joint between arm_6_link and arm_7_link -->
-    <joint name="${name}_7_joint" type="revolute">
-      <origin xyz="0 0 0" rpy="-${M_PI/2} 0 0"/>
-      <parent link="${name}_6_link"/>
-      <child link="${name}_7_link"/>
-      <axis xyz="0 0 1"/>
-      <calibration rising="${arm_7_ref}"/>
-      <limit effort="15" velocity="1.2566" lower="-2.0943951" upper="2.0943951"/>
-    </joint>
-    <link name="${name}_7_link">
-      <xacro:default_inertial/>
-<!--
-      <xacro:cylinder_inertial radius="0.03" length="0.035" mass="0.05">
-        <origin xyz="0 0 0.06" rpy="0 0 0"/>
-      </xacro:cylinder_inertial>
--->
-      <visual>
-        <origin xyz="0 0 0.06" rpy="0 0 0"/>
-        <geometry>
-          <cylinder radius="0.03" length="0.035"/>
-        </geometry>
-        <material name="Schunk/LightGrey"/>
-      </visual>
-      <collision>
-        <origin xyz="0 0 0.06" rpy="0 0 0"/>
-        <geometry>
-          <cylinder radius="0.03" length="0.035"/>
-        </geometry>
-      </collision>
-    </link>
-    <!-- extensions -->
-    <xacro:schunk_lwa4d_gazebo name="${name}"/>
-    <xacro:schunk_lwa4d_transmission name="${name}"/>
+  <xacro:schunk_lwa4d_without_base name="arm" parent="${name}_base_link"
+          arm_1_ref="${arm_1_ref}"
+          arm_2_ref="${arm_2_ref}"
+          arm_3_ref="${arm_3_ref}"
+          arm_4_ref="${arm_4_ref}"
+          arm_5_ref="${arm_5_ref}"
+          arm_6_ref="${arm_6_ref}"
+          arm_7_ref="${arm_7_ref}">
+    <origin xyz="0 0 0.15" rpy="0 -${M_PI} 0" />
+  </xacro:schunk_lwa4d_without_base>
   </xacro:macro>
 </robot>

File: schunk_description/urdf/lwa4d/lwa4d_without_base.urdf.xacro (robot description, xacro)
@@ -3,18 +3,9 @@
   <xacro:include filename="$(find schunk_description)/urdf/lwa4d/lwa4d.gazebo.xacro"/>
   <xacro:include filename="$(find schunk_description)/urdf/lwa4d/lwa4d.transmission.xacro"/>
-  <xacro:macro name="schunk_lwa4d" params="parent name *origin arm_1_ref arm_2_ref arm_3_ref arm_4_ref arm_5_ref arm_6_ref arm_7_ref">
-    <!-- joint between base_link and arm_base_link -->
-    <joint name="${name}_base_joint" type="fixed">
+  <xacro:macro name="schunk_lwa4d_without_base" params="parent name *origin arm_1_ref arm_2_ref arm_3_ref arm_4_ref arm_5_ref arm_6_ref arm_7_ref">
+    <!-- joint between arm_0_link and arm_1_link -->
+    <joint name="${name}_1_joint" type="revolute">
       <insert_block name="origin"/>
       <parent link="${parent}"/>
-      <child link="${name}_base_link"/>
-    </joint>
-     <link name="${name}_base_link">
-      <xacro:default_inertial/>
-    </link>
-    <!-- joint between arm_0_link and arm_1_link -->
-    <joint name="${name}_1_joint" type="revolute">
-      <origin xyz="0 0 0" rpy="0 -${M_PI} 0"/>
-      <parent link="${name}_base_link"/>
       <child link="${name}_1_link"/>
       <axis xyz="0 0 1"/>
