Commit message: new urdf structure

File: schunk_description/urdf/lwa4p_extended/lwa4p_extended.urdf.xacro (robot description, xacro)
@@ -1,20 +1,51 @@
 <?xml version="1.0"?>
 <robot xmlns:xacro="http://www.ros.org/wiki/xacro">
-  <xacro:include filename="$(find schunk_description)/urdf/lwa4p_extended/lwa4p_extended_without_base.urdf.xacro" />
-  <xacro:macro name="schunk_lwa4p_extended" params="parent name *origin arm_1_ref arm_2_ref arm_3_ref arm_4_ref arm_5_ref arm_6_ref arm_7_ref">
-    <!-- joint between base_link and lwa4p_extended_connector_link -->
-    <joint name="${name}_base_joint" type="fixed">
-      <insert_block name="origin" />
-      <parent link="${parent}"/>
-      <child link="${name}_base_link"/>
-    </joint>
+  <xacro:include filename="$(find schunk_description)/urdf/lwa4p_extended/lwa4p_extended.gazebo.xacro" />
+  <xacro:include filename="$(find schunk_description)/urdf/lwa4p_extended/lwa4p_extended.transmission.xacro" />
+  <xacro:macro name="schunk_lwa4p_extended" params="parent name *origin arm_1_ref arm_2_ref arm_3_ref arm_4_ref arm_5_ref arm_6_ref arm_7_ref has_podest">
+    <xacro:if value="${has_podest}">
+      <!-- joint between base_link and lwa4p_extended_connector_link -->
+      <joint name="${name}_podest_joint" type="fixed">
+        <insert_block name="origin" />
+        <parent link="${parent}"/>
+        <child link="${name}_podest_link"/>
+      </joint>
+      <link name="${name}_podest_link">
+        <xacro:default_inertial/>
+        <visual>
+          <origin xyz="0 0 0" rpy="0 0 0" />
+          <geometry>
+            <cylinder radius="0.03" length="0.05"/>
+          </geometry>
+        </visual>
+        <collision>
+          <origin xyz="0 0 0" rpy="0 0 0" />
+          <geometry>
+            <cylinder radius="0.03" length="0.05"/>
+          </geometry>
+        </collision>
+      </link>
+      <joint name="${name}_base_joint" type="fixed">
+        <origin xyz="0 0 0.025" rpy="0 0 0" />
+        <parent link="${name}_podest_link"/>
+        <child link="${name}_base_link"/>
+      </joint>
+    </xacro:if>
+    <xacro:unless value="${has_podest}">
+      <!-- joint between base_link and lwa4p_extended_connector_link -->
+      <joint name="${name}_base_joint" type="fixed">
+        <insert_block name="origin" />
+        <parent link="${parent}"/>
+        <child link="${name}_base_link"/>
+      </joint>
+    </xacro:unless>
     <!-- static part of PRL100 -->
     <link name="${name}_base_link">
       <xacro:default_inertial/>
-<!--
+  <!--
       <xacro:cylinder_inertial radius="0.056" length="0.12" mass="2.0">
         <origin xyz="0 0 ${0.12/2}" rpy="0 0 0" />
       </xacro:cylinder_inertial>
--->
+  -->
       <visual>
         <origin xyz="0 0 0" rpy="0 0 0" />
@@ -30,14 +61,238 @@
       </collision>
     </link>
-  <xacro:schunk_lwa4p_extended_without_base name="${name}" parent="${name}_base_link"
-          arm_1_ref="${arm_1_ref}"
-          arm_2_ref="${arm_2_ref}"
-          arm_3_ref="${arm_3_ref}"
-          arm_4_ref="${arm_4_ref}"
-          arm_5_ref="${arm_5_ref}"
-          arm_6_ref="${arm_6_ref}"
-          arm_7_ref="${arm_7_ref}">
-    <origin xyz="0 0 0.139" rpy="0 0 0" />
-  </xacro:schunk_lwa4p_extended_without_base>
+    <!-- joint between arm_base_link and arm_1_link -->
+    <joint name="${name}_1_joint" type="revolute">
+      <origin xyz="0 0 0.139" rpy="0 0 0" />
+      <parent link="${name}_base_link"/>
+      <child link="${name}_1_link" />
+      <axis xyz="0 0 1"/>
+      <calibration rising="${arm_1_ref}"/>
+      <dynamics damping="0" friction="0"/>
+      <limit effort="81.5" velocity="0.42" lower="-4.712" upper="4.712"/>   <!--Theoricarl limit +/-270 , Real Limit +/- 270-->
+      <!--safety_controller k_position="20" k_velocity="50" soft_lower_limit="${-M_PI + 0.01}" soft_upper_limit="${M_PI - 0.01}" /-->
+    </joint>
+    <!-- prl100 rotor + shoulder flansh -->
+    <link name="${name}_1_link">
+      <xacro:default_inertial/>
+<!--
+      <inertial>
+        <origin xyz="0.0 0.0662 0.0473" rpy="0 0 0"/>
+        <mass value="0.8"/>
+        <inertia ixx="0.002034" ixy="0.0" ixz="0.0" iyy="0.001437" iyz="0.000784" izz="0.00161" />
+      </inertial>
+-->
+      <visual>
+        <origin xyz="0 0 0" rpy="0 0 0" />
+        <geometry>
+          <mesh filename="package://schunk_description/meshes/lwa4p_extended/arm_1_link.dae" />
+        </geometry>
+      </visual>
+      <collision>
+        <origin xyz="0 0 0" rpy="0 0 0" />
+        <geometry>
+          <mesh filename="package://schunk_description/meshes/lwa4p_extended/arm_1_collision.stl" />
+        </geometry>
+      </collision>
+    </link>
+    <!-- joint between arm_1_link and arm_2_link -->
+    <joint name="${name}_2_joint" type="revolute">
+      <origin xyz="0 0 0.0915" rpy="1.5708 0 0"/>
+      <parent link="${name}_1_link"/>
+      <child link="${name}_2_link"/>
+      <axis xyz="0 0 1"/>
+      <calibration rising="${arm_2_ref}"/>
+      <dynamics damping="0" friction="0"/>
+      <limit effort="48" velocity="1.2566" lower="-1.92" upper="1.92"/>   <!--Theoricarl limit +/-170 , Real Limit +/- 110 (self collision)-->
+      <!--safety_controller k_position="20" k_velocity="50" soft_lower_limit="${-2.0943 + 0.01}" soft_upper_limit="${2.0943 - 0.01}" /-->
+    </joint>
+    <link name="${name}_2_link">
+      <xacro:default_inertial/>
+<!--
+      <inertial>
+        <origin xyz="0 0.018 -0.018" rpy="0 0 0"/>
+        <mass value="3.9"/>
+        <inertia ixx="0.009780" ixy="0.0" ixz="0.0" iyy="0.013300" iyz="0.0" izz="0.009780" />
+      </inertial>
+-->
+      <visual>
+        <origin xyz="0 0 0" rpy="0 0 0" />
+        <geometry>
+          <mesh filename="package://schunk_description/meshes/lwa4p_extended/arm_2_link.dae" />
+        </geometry>
+      </visual>
+      <collision>
+        <origin xyz="0 0 0" rpy="0 0 0" />
+        <geometry>
+          <mesh filename="package://schunk_description/meshes/lwa4p_extended/arm_2_collision.stl" />
+        </geometry>
+      </collision>
+    </link>
+    <!-- joint between arm_2_link and arm_3_link -->
+    <joint name="${name}_3_joint" type="revolute">
+      <origin xyz="0 0 0" rpy="-1.5708 0 0"/>
+      <parent link="${name}_2_link"/>
+      <child link="${name}_3_link"/>
+      <axis xyz="0 0 1"/>
+      <calibration rising="${arm_3_ref}"/>
+      <dynamics damping="0" friction="0"/>
+      <limit effort="48" velocity="1.2566" lower="-2.967" upper="2.967"/>   <!--Theoricarl limit +/-170 , Real Limit +/- 170-->
+      <!--safety_controller k_position="20" k_velocity="25" soft_lower_limit="${-M_PI + 0.01}" soft_upper_limit="${M_PI - 0.01}" /-->
+    </joint>
+    <link name="${name}_3_link">
+      <xacro:default_inertial/>
+<!--
+      <inertial>
+        <origin xyz="0.0 0.06247 0.23425" rpy="0 0 0"/>
+        <mass value="1.94533"/>
+        <inertia ixx="0.0344" ixy="0.0" ixz="0.0077" iyy="0.0362" iyz="0.0" izz="0.0052" />
+      </inertial>
+-->
+      <visual>
+        <origin xyz="0 0 0" rpy="0 0 0" />
+        <geometry>
+          <mesh filename="package://schunk_description/meshes/lwa4p_extended/arm_3_link.dae" />
+        </geometry>
+      </visual>
+      <collision>
+        <origin xyz="0 0 0" rpy="0 0 0" />
+        <geometry>
+          <mesh filename="package://schunk_description/meshes/lwa4p_extended/arm_3_collision.stl" />
+        </geometry>
+      </collision>
+    </link>
+    <!-- joint between arm_3_link and arm_4_link -->
+    <joint name="${name}_4_joint" type="revolute">
+      <origin xyz="0 0 0.45360" rpy="1.5708 0 0" />
+      <parent link="${name}_3_link"/>
+      <child link="${name}_4_link"/>
+      <axis xyz="0 0 1" />
+      <calibration rising="${arm_4_ref}"/>
+      <dynamics damping="0" friction="0"/>
+      <limit effort="48" velocity="1.2566" lower="-2.618" upper="2.618"/>   <!--Theoricarl limit +/-170 , Real Limit +/- 150 (self collision)-->
+      <!--safety_controller k_position="20" k_velocity="25" soft_lower_limit="${-2.0943951 + 0.01}" soft_upper_limit="${2.0943951 - 0.01}" /-->
+    </joint>
+    <link name="${name}_4_link">
+      <xacro:default_inertial/>
+<!--
+      <inertial>
+        <origin xyz="0 0.018 -0.018" rpy="0 0 0"/>
+        <mass value="3.9"/>
+        <inertia ixx="0.009780" ixy="0.0" ixz="0.0" iyy="0.013300" iyz="0.0" izz="0.009780" />
+      </inertial>
+-->
+      <visual>
+        <origin xyz="0 0 0" rpy="0 0 0" />
+        <geometry>
+          <mesh filename="package://schunk_description/meshes/lwa4p_extended/arm_4_link.dae" />
+        </geometry>
+      </visual>
+      <collision>
+        <origin xyz="0 0 0" rpy="0 0 0" />
+        <geometry>
+          <mesh filename="package://schunk_description/meshes/lwa4p_extended/arm_4_collision.stl" />
+        </geometry>
+      </collision>
+    </link>
+    <!-- joint between arm_4_link and arm_5_link -->
+    <joint name="${name}_5_joint" type="revolute">
+      <origin xyz="0 0 0" rpy="-1.5708 0 0" />
+      <parent link="${name}_4_link"/>
+      <child link="${name}_5_link"/>
+      <axis xyz="0 0 1" />
+      <calibration rising="${arm_5_ref}"/>
+      <dynamics damping="0" friction="0"/>
+      <limit effort="48" velocity="1.2566" lower="-2.967" upper="2.967"/>   <!--Theoricarl limit +/-170 , Real Limit +/- 170-->
+      <!--safety_controller k_position="20" k_velocity="25" soft_lower_limit="${-M_PI + 0.01}" soft_upper_limit="${M_PI - 0.01}" /-->
+    </joint>
+    <link name="${name}_5_link">
+      <xacro:default_inertial/>
+<!--
+      <inertial>
+        <origin xyz="0.0 0.04175 0.17026" rpy="0 0 0"/>
+        <mass value="1.3297"/>
+        <inertia ixx="0.01" ixy="0.0" ixz="-0.0031" iyy="0.0111" iyz="0.0" izz="0.0031" />
+      </inertial>
+-->
+      <visual>
+        <origin xyz="0 0 0" rpy="0 0 0" />
+        <geometry>
+          <mesh filename="package://schunk_description/meshes/lwa4p_extended/arm_5_link.dae" />
+        </geometry>
+      </visual>
+      <collision>
+        <origin xyz="0 0 0" rpy="0 0 0" />
+        <geometry>
+          <mesh filename="package://schunk_description/meshes/lwa4p_extended/arm_5_collision.stl" />
+        </geometry>
+      </collision>
+    </link>
+    <!-- joint between arm_5_link and arm_6_link -->
+    <joint name="${name}_6_joint" type="revolute">
+      <origin xyz="0 0 0.2986" rpy="1.5708 0 0" />
+      <parent link="${name}_5_link"/>
+      <child link="${name}_6_link"/>
+      <axis xyz="0 0 1" />
+      <calibration rising="${arm_6_ref}"/>
+      <dynamics damping="0" friction="0"/>
+      <limit effort="15" velocity="1.2566" lower="-2.443" upper="2.967"/>   <!--Theoricarl limit +/-170 , Real Limit -140/+170 (self collision)-->
+      <!--safety_controller k_position="20" k_velocity="25" soft_lower_limit="${-2.0943951 + 0.01}" soft_upper_limit="${2.0943951 - 0.01}" /-->
+    </joint>
+    <link name="${name}_6_link">
+      <xacro:default_inertial/>
+<!--
+      <inertial>
+        <origin xyz="0 0.012 -0.012" rpy="0 0 0"/>
+        <mass value="1.9"/>
+        <inertia ixx="0.002750" ixy="0.0" ixz="0.0" iyy="0.004002" iyz="0.0" izz="0.002830" />
+      </inertial>
+-->
+      <visual>
+        <origin xyz="0 0 0" rpy="0 0 0" />
+        <geometry>
+          <mesh filename="package://schunk_description/meshes/lwa4p_extended/arm_6_link.dae" />
+        </geometry>
+      </visual>
+      <collision>
+        <origin xyz="0 0 0" rpy="0 0 0" />
+        <geometry>
+          <mesh filename="package://schunk_description/meshes/lwa4p_extended/arm_6_collision.stl" />
+        </geometry>
+      </collision>
+    </link>
+    <!-- joint between arm_6_link and arm_7_link -->
+    <joint name="${name}_7_joint" type="revolute">
+      <origin xyz="0 0 0" rpy="-1.5708 0 0" />
+      <parent link="${name}_6_link"/>
+      <child link="${name}_7_link"/>
+      <axis xyz="0 0 1" />
+      <calibration rising="${arm_7_ref}"/>
+      <dynamics damping="0" friction="0"/>
+      <limit effort="15" velocity="1.2566" lower="-2.967" upper="2.967"/>   <!--Theoricarl limit +/-170 , Real Limit +/- 170-->
+      <!--safety_controller k_position="20" k_velocity="25" soft_lower_limit="${-2.0943951 + 0.01}" soft_upper_limit="${2.0943951 - 0.01}" /-->
+    </joint>
+    <link name="${name}_7_link">
+      <xacro:default_inertial/>
+<!--
+      <xacro:cylinder_inertial radius="0.03" length="0.035" mass="0.05">
+        <origin xyz="0 0 0.06" rpy="0 0 0"/>
+      </xacro:cylinder_inertial>
+-->
+      <visual>
+        <origin xyz="0 0 0.06" rpy="0 0 0"/>
+        <geometry>
+          <cylinder radius="0.03" length="0.035"/>
+        </geometry>
+        <material name="Schunk/LightGrey"/>
+      </visual>
+      <collision>
+        <origin xyz="0 0 0.06" rpy="0 0 0"/>
+        <geometry>
+          <cylinder radius="0.03" length="0.035"/>
+        </geometry>
+      </collision>
+    </link>
+    <!-- extensions -->
+    <xacro:schunk_lwa4p_extended_gazebo name="${name}" />
+    <xacro:schunk_lwa4p_extended_transmission name="${name}" />
   </xacro:macro>
 </robot>

Commit message: Fixes the limits for the lwa4d

File: schunk_description/urdf/lwa4d/lwa4d.urdf.xacro (robot description, xacro)
@@ -80,5 +80,5 @@
       <axis xyz="0 0 1"/>
       <calibration rising="${arm_2_ref}"/>
-      <limit effort="216" velocity="0.43633" lower="-${M_PI}" upper="${M_PI}"/>
+      <limit effort="216" velocity="0.43633" lower="-2.14" upper="2.14"/>
     </joint>
     <link name="${name}_2_link">
@@ -140,5 +140,5 @@
       <axis xyz="0 0 1"/>
       <calibration rising="${arm_4_ref}"/>
-      <limit effort="81.5" velocity="0.4189" lower="-${M_PI}" upper="${M_PI}"/>
+      <limit effort="81.5" velocity="0.4189" lower="-2.18" upper="2.18"/>
     </joint>
     <link name="${name}_4_link">
@@ -200,5 +200,5 @@
       <axis xyz="0 0 1"/>
       <calibration rising="${arm_6_ref}"/>
-      <limit effort="15" velocity="1.2566" lower="-2.0943951" upper="2.0943951"/>
+      <limit effort="15" velocity="1.2566" lower="-2.0" upper="2.0"/>
     </joint>
     <link name="${name}_6_link">

Commit message: Safety_offset

File: schunk_description/urdf/lwa4d/lwa4d.urdf.xacro (robot description, xacro)
@@ -4,4 +4,5 @@
   <xacro:include filename="$(find schunk_description)/urdf/lwa4d/lwa4d.transmission.xacro"/>
   <xacro:macro name="schunk_lwa4d" params="parent name *origin arm_1_ref arm_2_ref arm_3_ref arm_4_ref arm_5_ref arm_6_ref arm_7_ref has_podest">
+    <property name="safety_offset" value="0.01"/>
     <xacro:if value="${has_podest}">
       <!-- joint between base_link and lwa4p_extended_connector_link -->
@@ -50,5 +51,5 @@
       <axis xyz="0 0 1"/>
       <calibration rising="${arm_1_ref}"/>
-      <limit effort="216" velocity="0.43633" lower="-${M_PI}" upper="${M_PI}"/>
+      <limit effort="216" velocity="0.43633" lower="${-M_PI+safety_offset}" upper="${M_PI-safety_offset}"/>
     </joint>
     <link name="${name}_1_link">
@@ -80,5 +81,5 @@
       <axis xyz="0 0 1"/>
       <calibration rising="${arm_2_ref}"/>
-      <limit effort="216" velocity="0.43633" lower="-2.14" upper="2.14"/>
+      <limit effort="216" velocity="0.43633" lower="${-2.14 + safety_offset}" upper="${2.14 - safety_offset}"/>
     </joint>
     <link name="${name}_2_link">
@@ -110,5 +111,5 @@
       <axis xyz="0 0 1"/>
       <calibration rising="${arm_3_ref}"/>
-      <limit effort="81.5" velocity="0.4189" lower="-${M_PI}" upper="${M_PI}"/>
+      <limit effort="81.5" velocity="0.4189" lower="${-M_PI + safety_offset}" upper="${M_PI - safety_offset}"/>
     </joint>
     <link name="${name}_3_link">
@@ -140,5 +141,5 @@
       <axis xyz="0 0 1"/>
       <calibration rising="${arm_4_ref}"/>
-      <limit effort="81.5" velocity="0.4189" lower="-2.18" upper="2.18"/>
+      <limit effort="81.5" velocity="0.4189" lower="${-2.18 + safety_offset}" upper="${2.18 - safety_offset}"/>
     </joint>
     <link name="${name}_4_link">
@@ -170,5 +171,5 @@
       <axis xyz="0 0 1"/>
       <calibration rising="${arm_5_ref}"/>
-      <limit effort="20.7" velocity="0.43633" lower="-${M_PI}" upper="${M_PI}"/>
+      <limit effort="20.7" velocity="0.43633" lower="${-M_PI + safety_offset}" upper="${M_PI - safety_offset}"/>
     </joint>
     <link name="${name}_5_link">
@@ -200,5 +201,5 @@
       <axis xyz="0 0 1"/>
       <calibration rising="${arm_6_ref}"/>
-      <limit effort="15" velocity="1.2566" lower="-2.0" upper="2.0"/>
+      <limit effort="15" velocity="1.2566" lower="${-2.0 + safety_offset}" upper="${2.0 - safety_offset}"/>
     </joint>
     <link name="${name}_6_link">
@@ -230,5 +231,5 @@
       <axis xyz="0 0 1"/>
       <calibration rising="${arm_7_ref}"/>
-      <limit effort="15" velocity="1.2566" lower="-2.0943951" upper="2.0943951"/>
+      <limit effort="15" velocity="1.2566" lower="${-2.0943951 + safety_offset}" upper="${2.0943951 - safety_offset}"/>
     </joint>
     <link name="${name}_7_link">

File: schunk_description/urdf/lwa4p/lwa4p.urdf.xacro (robot description, xacro)
@@ -4,4 +4,5 @@
   <xacro:include filename="$(find schunk_description)/urdf/lwa4p/lwa4p.transmission.xacro" />
   <xacro:macro name="schunk_lwa4p" params="parent name *origin arm_1_ref arm_2_ref arm_3_ref arm_4_ref arm_5_ref arm_6_ref has_podest">
+    <property name="safety_offset" value="0.01"/>
     <xacro:if value="${has_podest}">
       <!-- joint between base_link and lwa4p_extended_connector_link -->
@@ -50,5 +51,5 @@
       <axis xyz="0 0 1"/>
       <calibration rising="${arm_1_ref}"/>
-      <limit effort="370" velocity="2.0" lower="-6.2831853" upper="6.2831853"/>
+      <limit effort="370" velocity="2.0" lower="${-6.2831853 + safety_offset}" upper="${6.2831853 - safety_offset}"/>
       <!--safety_controller k_position="20" k_velocity="50" soft_lower_limit="${-6.2831853 + 0.01}" soft_upper_limit="${6.2831853 - 0.01}" /-->
     </joint>
@@ -83,5 +84,5 @@
       <axis xyz="0 0 1"/>
       <calibration rising="${arm_2_ref}"/>
-      <limit effort="370" velocity="2.0" lower="-2.0943951" upper="2.0943951"/>
+      <limit effort="370" velocity="2.0" lower="${-2.0943951 + safety_offset}" upper="${2.0943951 - safety_offset}"/>
       <!--safety_controller k_position="20" k_velocity="50" soft_lower_limit="${-2.0943 + 0.01}" soft_upper_limit="${2.0943 - 0.01}" /-->
     </joint>
@@ -116,5 +117,5 @@
       <axis xyz="0 0 1"/>
       <calibration rising="${arm_3_ref}"/>
-      <limit effort="176" velocity="2.0" lower="-6.2831853" upper="6.2831853"/>
+      <limit effort="176" velocity="2.0" lower="${-6.2831853 + safety_offset}" upper="${6.2831853 - safety_offset}"/>
       <!--safety_controller k_position="20" k_velocity="25" soft_lower_limit="${-6.2831853 + 0.01}" soft_upper_limit="${6.2831853 - 0.01}" /-->
     </joint>
@@ -149,5 +150,5 @@
       <axis xyz="0 0 1" />
       <calibration rising="${arm_4_ref}"/>
-      <limit effort="176" velocity="2.0" lower="-2.0943951" upper="2.0943951"/>
+      <limit effort="176" velocity="2.0" lower="${-2.0943951 + safety_offset}" upper="${2.0943951 - safety_offset}"/>
       <!--safety_controller k_position="20" k_velocity="25" soft_lower_limit="${-2.0943951 + 0.01}" soft_upper_limit="${2.0943951 - 0.01}" /-->
     </joint>
@@ -182,5 +183,5 @@
       <axis xyz="0 0 1" />
       <calibration rising="${arm_5_ref}"/>
-      <limit effort="41.6" velocity="2.0" lower="-6.2831853" upper="6.2831853" />
+      <limit effort="41.6" velocity="2.0" lower="${-6.2831853 + safety_offset}" upper="${6.2831853 - safety_offset}" />
       <!--safety_controller k_position="20" k_velocity="25" soft_lower_limit="${-6.2831853 + 0.01}" soft_upper_limit="${6.2831853 - 0.01}" /-->
     </joint>
@@ -215,5 +216,5 @@
       <axis xyz="0 0 1" />
       <calibration rising="${arm_6_ref}"/>
-      <limit effort="20.1" velocity="2.0" lower="-2.0943951" upper="2.0943951" />
+      <limit effort="20.1" velocity="2.0" lower="${-2.0943951 + safety_offset}" upper="${2.0943951 - safety_offset}" />
       <!--safety_controller k_position="20" k_velocity="25" soft_lower_limit="${-2.0943951 + 0.01}" soft_upper_limit="${2.0943951 - 0.01}" /-->
     </joint>

Commit message: proper rounding of joint_limits for lwa4d

File: schunk_description/urdf/lwa4d/lwa4d.urdf.xacro (robot description, xacro)
@@ -1,5 +1,5 @@
 <?xml version="1.0"?>
 <robot xmlns:xacro="http://www.ros.org/wiki/xacro">
-  <property name="safety_offset" value="0.01"/>
+  <property name="safety_offset" value="0.02"/>
   <xacro:include filename="$(find schunk_description)/urdf/lwa4d/lwa4d.gazebo.xacro"/>
   <xacro:include filename="$(find schunk_description)/urdf/lwa4d/lwa4d.transmission.xacro"/>
@@ -201,5 +201,5 @@
       <axis xyz="0 0 1"/>
       <calibration rising="${arm_6_ref}"/>
-      <limit effort="15" velocity="1.2566" lower="${-2.0 + safety_offset}" upper="${2.0 - safety_offset}"/>
+      <limit effort="15" velocity="1.2566" lower="${-2.09 + safety_offset}" upper="${2.09 - safety_offset}"/>
     </joint>
     <link name="${name}_6_link">
@@ -231,5 +231,5 @@
       <axis xyz="0 0 1"/>
       <calibration rising="${arm_7_ref}"/>
-      <limit effort="15" velocity="1.2566" lower="${-2.0943951 + safety_offset}" upper="${2.0943951 - safety_offset}"/>
+      <limit effort="15" velocity="1.2566" lower="${-2.96 + safety_offset}" upper="${2.96 - safety_offset}"/>
     </joint>
     <link name="${name}_7_link">
