Commit message: remove unsupported calibration_rising

File: schunk_description/urdf/lwa4d/lwa4d.urdf.xacro (robot description, xacro)
@@ -4,5 +4,5 @@
   <xacro:include filename="$(find schunk_description)/urdf/lwa4d/lwa4d.gazebo.xacro"/>
   <xacro:include filename="$(find schunk_description)/urdf/lwa4d/lwa4d.transmission.xacro"/>
-  <xacro:macro name="schunk_lwa4d" params="parent name *origin arm_1_ref arm_2_ref arm_3_ref arm_4_ref arm_5_ref arm_6_ref arm_7_ref has_podest">
+  <xacro:macro name="schunk_lwa4d" params="parent name *origin has_podest">
     <xacro:if value="${has_podest}">
       <!-- joint between base_link and lwa4p_extended_connector_link -->
@@ -50,5 +50,4 @@
       <child link="${name}_1_link"/>
       <axis xyz="0 0 1"/>
-      <calibration rising="${arm_1_ref}"/>
       <limit effort="216" velocity="0.43633" lower="${-M_PI+safety_offset}" upper="${M_PI-safety_offset}"/>
     </joint>
@@ -80,5 +79,4 @@
       <child link="${name}_2_link"/>
       <axis xyz="0 0 1"/>
-      <calibration rising="${arm_2_ref}"/>
       <limit effort="216" velocity="0.43633" lower="${-2.14 + safety_offset}" upper="${2.14 - safety_offset}"/>
     </joint>
@@ -110,5 +108,4 @@
       <child link="${name}_3_link"/>
       <axis xyz="0 0 1"/>
-      <calibration rising="${arm_3_ref}"/>
       <limit effort="81.5" velocity="0.4189" lower="${-M_PI + safety_offset}" upper="${M_PI - safety_offset}"/>
     </joint>
@@ -140,5 +137,4 @@
       <child link="${name}_4_link"/>
       <axis xyz="0 0 1"/>
-      <calibration rising="${arm_4_ref}"/>
       <limit effort="81.5" velocity="0.4189" lower="${-2.18 + safety_offset}" upper="${2.18 - safety_offset}"/>
     </joint>
@@ -170,5 +166,4 @@
       <child link="${name}_5_link"/>
       <axis xyz="0 0 1"/>
-      <calibration rising="${arm_5_ref}"/>
       <limit effort="20.7" velocity="0.43633" lower="${-M_PI + safety_offset}" upper="${M_PI - safety_offset}"/>
     </joint>
@@ -200,5 +195,4 @@
       <child link="${name}_6_link"/>
       <axis xyz="0 0 1"/>
-      <calibration rising="${arm_6_ref}"/>
       <limit effort="15" velocity="1.2566" lower="${-2.09 + safety_offset}" upper="${2.09 - safety_offset}"/>
     </joint>
@@ -230,5 +224,4 @@
       <child link="${name}_7_link"/>
       <axis xyz="0 0 1"/>
-      <calibration rising="${arm_7_ref}"/>
       <limit effort="15" velocity="1.2566" lower="${-2.96 + safety_offset}" upper="${2.96 - safety_offset}"/>
     </joint>

File: schunk_description/urdf/pg70/pg70.urdf.xacro (robot description, xacro)
@@ -3,5 +3,5 @@
   <xacro:include filename="$(find schunk_description)/urdf/pg70/pg70.gazebo.xacro" />
   <xacro:include filename="$(find schunk_description)/urdf/pg70/pg70.transmission.xacro" />
-  <xacro:macro name="schunk_pg70" params="parent name *origin pg70_finger_left_ref pg70_finger_right_ref">
+  <xacro:macro name="schunk_pg70" params="parent name *origin">
     <joint name="${name}_palm_joint" type="fixed" >
       <parent link="${parent}" />
@@ -36,5 +36,4 @@
       <child link="${name}_finger_left_link" />
       <limit effort="100" lower="-0.001" upper="0.061" velocity="2.0"/>
-      <calibration rising="${pg70_finger_left_ref}"/>
       <origin xyz="0 0 0.0789" rpy="0 0 0"/>
       <axis xyz="0 1 0" />
@@ -68,5 +67,4 @@
       <child link="${name}_finger_right_link" />
       <limit effort="100" lower="-0.001" upper="0.061" velocity="2.0"/>
-      <calibration rising="${pg70_finger_right_ref}"/>
       <origin xyz="0 0 0.0789" rpy="-0 0 0"/>
       <axis xyz="0 -1 0" />

Commit message: fix lwa4d urdf - joint orientation according to convention

File: schunk_description/urdf/lwa4d/lwa4d.urdf.xacro (robot description, xacro)
@@ -15,18 +15,17 @@
         <xacro:default_inertial/>
         <visual>
-          <origin xyz="0 0 0" rpy="0 0 0" />
           <geometry>
-            <cylinder radius="0.03" length="0.05"/>
+            <mesh filename="package://schunk_description/meshes/lwa4d/arm_podest_link.stl"/>
           </geometry>
+          <material name="Schunk/LightGrey"/>
         </visual>
         <collision>
-          <origin xyz="0 0 0" rpy="0 0 0" />
           <geometry>
-            <cylinder radius="0.03" length="0.05"/>
+            <mesh filename="package://schunk_description/meshes/lwa4d/arm_podest_link.stl"/>
           </geometry>
         </collision>
       </link>
       <joint name="${name}_base_joint" type="fixed">
-        <origin xyz="0 0 0.175" rpy="0 ${M_PI} 0" />
+        <origin xyz="0 0 0.140" rpy="0 0 0" />
         <parent link="${name}_podest_link"/>
         <child link="${name}_base_link"/>
@@ -60,5 +59,4 @@
 -->
       <visual>
-        <origin xyz="0 0 -0.15" rpy="0 0 ${M_PI}"/>
         <geometry>
           <mesh filename="package://schunk_description/meshes/lwa4d/arm_1_link.stl"/>
@@ -67,5 +65,4 @@
       </visual>
       <collision>
-        <origin xyz="0 0 -0.15" rpy="0 0 ${M_PI}"/>
         <geometry>
           <mesh filename="package://schunk_description/meshes/lwa4d/arm_1_link.stl"/>
@@ -75,5 +72,5 @@
     <!-- joint between arm_1_link and arm_2_link -->
     <joint name="${name}_2_joint" type="revolute">
-      <origin xyz="0 0 -0.15" rpy="-${M_PI/2} 0 0"/>
+      <origin xyz="0 0 0.240" rpy="-${M_PI/2} -${M_PI/2} 0"/>
       <parent link="${name}_1_link"/>
       <child link="${name}_2_link"/>
@@ -89,5 +86,4 @@
 -->
       <visual>
-        <origin xyz="0 0 0" rpy="0 0 ${M_PI}"/>
         <geometry>
           <mesh filename="package://schunk_description/meshes/lwa4d/arm_2_link.stl"/>
@@ -96,5 +92,4 @@
       </visual>
       <collision>
-        <origin xyz="0 0 0" rpy="0 0 ${M_PI}"/>
         <geometry>
           <mesh filename="package://schunk_description/meshes/lwa4d/arm_2_link_collision.stl"/>
@@ -104,5 +99,5 @@
     <!-- joint between arm_2_link and arm_3_link -->
     <joint name="${name}_3_joint" type="revolute">
-      <origin xyz="0 0 0" rpy="${M_PI/2} 0 0"/>
+      <origin xyz="0 0 0" rpy="${M_PI/2} 0 ${M_PI/2}"/>
       <parent link="${name}_2_link"/>
       <child link="${name}_3_link"/>
@@ -118,5 +113,4 @@
 -->
       <visual>
-        <origin xyz="0 0 -0.39" rpy="0 0 ${M_PI}"/>
         <geometry>
           <mesh filename="package://schunk_description/meshes/lwa4d/arm_3_link.stl"/>
@@ -125,5 +119,4 @@
       </visual>
       <collision>
-        <origin xyz="0 0 -0.39" rpy="0 0 ${M_PI}"/>
         <geometry>
           <mesh filename="package://schunk_description/meshes/lwa4d/arm_3_link_collision.stl"/>
@@ -133,5 +126,5 @@
     <!-- joint between arm_3_link and arm_4_link -->
     <joint name="${name}_4_joint" type="revolute">
-      <origin xyz="0 0 -0.39" rpy="-${M_PI/2} 0 0"/>
+      <origin xyz="0 0 0.328" rpy="-${M_PI/2} -${M_PI/2} 0"/>
       <parent link="${name}_3_link"/>
       <child link="${name}_4_link"/>
@@ -147,5 +140,4 @@
 -->
       <visual>
-        <origin xyz="0 0 0" rpy="0 0 ${M_PI}"/>
         <geometry>
           <mesh filename="package://schunk_description/meshes/lwa4d/arm_4_link.stl"/>
@@ -154,5 +146,4 @@
       </visual>
       <collision>
-        <origin xyz="0 0 0" rpy="0 0 ${M_PI}"/>
         <geometry>
           <mesh filename="package://schunk_description/meshes/lwa4d/arm_4_link_collision.stl"/>
@@ -162,5 +153,5 @@
     <!-- joint between arm_4_link and arm_5_link -->
     <joint name="${name}_5_joint" type="revolute">
-      <origin xyz="0 0 0" rpy="${M_PI/2} 0 0"/>
+      <origin xyz="0 0 0" rpy="${M_PI/2} 0 ${M_PI/2}"/>
       <parent link="${name}_4_link"/>
       <child link="${name}_5_link"/>
@@ -176,5 +167,4 @@
 -->
       <visual>
-        <origin xyz="0 0 -0.323" rpy="0 0 ${M_PI}"/>
         <geometry>
           <mesh filename="package://schunk_description/meshes/lwa4d/arm_5_link.stl"/>
@@ -183,5 +173,4 @@
       </visual>
       <collision>
-        <origin xyz="0 0 -0.323" rpy="0 0 ${M_PI}"/>
         <geometry>
           <mesh filename="package://schunk_description/meshes/lwa4d/arm_5_link_collision.stl"/>
@@ -191,5 +180,5 @@
     <!-- joint between arm_5_link and arm_6_link -->
     <joint name="${name}_6_joint" type="revolute">
-      <origin xyz="0 0 -0.323" rpy="-${M_PI/2} 0 0"/>
+      <origin xyz="0 0 0.323" rpy="-${M_PI/2} -${M_PI/2} 0"/>
       <parent link="${name}_5_link"/>
       <child link="${name}_6_link"/>
@@ -205,5 +194,4 @@
 -->
       <visual>
-        <origin xyz="0 0 0" rpy="0 ${M_PI} 0"/>
         <geometry>
           <mesh filename="package://schunk_description/meshes/lwa4d/arm_6_link.stl"/>
@@ -212,5 +200,4 @@
       </visual>
       <collision>
-        <origin xyz="0 0 0" rpy="0 ${M_PI} 0"/>
         <geometry>
           <mesh filename="package://schunk_description/meshes/lwa4d/arm_6_link_collision.stl"/>
@@ -220,5 +207,5 @@
     <!-- joint between arm_6_link and arm_7_link -->
     <joint name="${name}_7_joint" type="revolute">
-      <origin xyz="0 0 0" rpy="-${M_PI/2} 0 0"/>
+      <origin xyz="0 0 0" rpy="${M_PI/2} 0 ${M_PI/2}"/>
       <parent link="${name}_6_link"/>
       <child link="${name}_7_link"/>
@@ -234,16 +221,22 @@
 -->
       <visual>
-        <origin xyz="0 0 0.06" rpy="0 0 0"/>
-        <geometry>
-          <cylinder radius="0.03" length="0.035"/>
-        </geometry>
-        <material name="Schunk/LightGrey"/>
-      </visual>
-      <collision>
-        <origin xyz="0 0 0.06" rpy="0 0 0"/>
-        <geometry>
-          <cylinder radius="0.03" length="0.035"/>
-        </geometry>
-      </collision>
+        <geometry>
+          <mesh filename="package://schunk_description/meshes/lwa4d/arm_7_link.stl"/>
+        </geometry>
+        <material name="Schunk/LightGrey"/>
+      </visual>
+      <collision>
+        <geometry>
+          <mesh filename="package://schunk_description/meshes/lwa4d/arm_7_link.stl"/>
+        </geometry>
+      </collision>
+    </link>
+    <joint name="${name}_ee_joint" type="fixed">
+      <origin xyz="0 0 0.0824" rpy="0 0 0"/>
+      <parent link="${name}_7_link"/>
+      <child link="${name}_ee_link"/>
+    </joint>
+    <link name="${name}_ee_link">
+      <xacro:default_inertial/>
     </link>
     <!-- extensions -->

Commit message: added 'invert' paramter to lwa4d xacro description, default value matches DH params, -1 matches default hardware configuration

File: schunk_description/urdf/lwa4d/lwa4d.urdf.xacro (robot description, xacro)
@@ -4,5 +4,5 @@
   <xacro:include filename="$(find schunk_description)/urdf/lwa4d/lwa4d.gazebo.xacro"/>
   <xacro:include filename="$(find schunk_description)/urdf/lwa4d/lwa4d.transmission.xacro"/>
-  <xacro:macro name="schunk_lwa4d" params="parent name *origin has_podest">
+  <xacro:macro name="schunk_lwa4d" params="parent name *origin has_podest invert:=1">
     <xacro:if value="${has_podest}">
       <!-- joint between base_link and lwa4p_extended_connector_link -->
@@ -48,5 +48,5 @@
       <parent link="${name}_base_link"/>
       <child link="${name}_1_link"/>
-      <axis xyz="0 0 1"/>
+      <axis xyz="0 0 ${invert}"/>
       <limit effort="216" velocity="0.43633" lower="${-M_PI+safety_offset}" upper="${M_PI-safety_offset}"/>
     </joint>
@@ -75,5 +75,5 @@
       <parent link="${name}_1_link"/>
       <child link="${name}_2_link"/>
-      <axis xyz="0 0 1"/>
+      <axis xyz="0 0 ${invert}"/>
       <limit effort="216" velocity="0.43633" lower="${-2.14 + safety_offset}" upper="${2.14 - safety_offset}"/>
     </joint>
@@ -102,5 +102,5 @@
       <parent link="${name}_2_link"/>
       <child link="${name}_3_link"/>
-      <axis xyz="0 0 1"/>
+      <axis xyz="0 0 ${invert}"/>
       <limit effort="81.5" velocity="0.4189" lower="${-M_PI + safety_offset}" upper="${M_PI - safety_offset}"/>
     </joint>
@@ -129,5 +129,5 @@
       <parent link="${name}_3_link"/>
       <child link="${name}_4_link"/>
-      <axis xyz="0 0 1"/>
+      <axis xyz="0 0 ${invert}"/>
       <limit effort="81.5" velocity="0.4189" lower="${-2.18 + safety_offset}" upper="${2.18 - safety_offset}"/>
     </joint>
@@ -156,5 +156,5 @@
       <parent link="${name}_4_link"/>
       <child link="${name}_5_link"/>
-      <axis xyz="0 0 1"/>
+      <axis xyz="0 0 ${invert}"/>
       <limit effort="20.7" velocity="0.43633" lower="${-M_PI + safety_offset}" upper="${M_PI - safety_offset}"/>
     </joint>

Commit message: added axis invert macro and set up parameters for each joint -- defaults to dh convention

File: schunk_description/urdf/lwa4d/lwa4d.urdf.xacro (robot description, xacro)
@@ -4,5 +4,13 @@
   <xacro:include filename="$(find schunk_description)/urdf/lwa4d/lwa4d.gazebo.xacro"/>
   <xacro:include filename="$(find schunk_description)/urdf/lwa4d/lwa4d.transmission.xacro"/>
-  <xacro:macro name="schunk_lwa4d" params="parent name *origin has_podest invert:=1">
+  <xacro:macro name="axis_config" params="invert">
+    <xacro:if value="${invert}">
+      <axis xyz="0 0 1" />
+    </xacro:if>
+    <xacro:unless value="${invert}">
+      <axis xyz="0 0 -1" />
+    </xacro:unless>
+  </xacro:macro>
+  <xacro:macro name="schunk_lwa4d" params="parent name *origin has_podest invert_j1:=true invert_j2:=true invert_j3:=true invert_j4:=true invert_j5:=true invert_j6:=true invert_j7:=true">
     <xacro:if value="${has_podest}">
       <!-- joint between base_link and lwa4p_extended_connector_link -->
@@ -48,5 +56,5 @@
       <parent link="${name}_base_link"/>
       <child link="${name}_1_link"/>
-      <axis xyz="0 0 ${invert}"/>
+      <xacro:axis_config invert="${invert_j1}"/>
       <limit effort="216" velocity="0.43633" lower="${-M_PI+safety_offset}" upper="${M_PI-safety_offset}"/>
     </joint>
@@ -75,5 +83,5 @@
       <parent link="${name}_1_link"/>
       <child link="${name}_2_link"/>
-      <axis xyz="0 0 ${invert}"/>
+      <xacro:axis_config invert="${invert_j2}"/>
       <limit effort="216" velocity="0.43633" lower="${-2.14 + safety_offset}" upper="${2.14 - safety_offset}"/>
     </joint>
@@ -102,5 +110,5 @@
       <parent link="${name}_2_link"/>
       <child link="${name}_3_link"/>
-      <axis xyz="0 0 ${invert}"/>
+      <xacro:axis_config invert="${invert_j3}"/>
       <limit effort="81.5" velocity="0.4189" lower="${-M_PI + safety_offset}" upper="${M_PI - safety_offset}"/>
     </joint>
@@ -129,5 +137,5 @@
       <parent link="${name}_3_link"/>
       <child link="${name}_4_link"/>
-      <axis xyz="0 0 ${invert}"/>
+      <xacro:axis_config invert="${invert_j4}"/>
       <limit effort="81.5" velocity="0.4189" lower="${-2.18 + safety_offset}" upper="${2.18 - safety_offset}"/>
     </joint>
@@ -156,5 +164,5 @@
       <parent link="${name}_4_link"/>
       <child link="${name}_5_link"/>
-      <axis xyz="0 0 ${invert}"/>
+      <xacro:axis_config invert="${invert_j5}"/>
       <limit effort="20.7" velocity="0.43633" lower="${-M_PI + safety_offset}" upper="${M_PI - safety_offset}"/>
     </joint>
@@ -183,5 +191,5 @@
       <parent link="${name}_5_link"/>
       <child link="${name}_6_link"/>
-      <axis xyz="0 0 1"/>
+      <xacro:axis_config invert="${invert_j6}"/>
       <limit effort="15" velocity="1.2566" lower="${-2.09 + safety_offset}" upper="${2.09 - safety_offset}"/>
     </joint>
@@ -210,5 +218,5 @@
       <parent link="${name}_6_link"/>
       <child link="${name}_7_link"/>
-      <axis xyz="0 0 1"/>
+      <xacro:axis_config invert="${invert_j7}"/>
       <limit effort="15" velocity="1.2566" lower="${-2.96 + safety_offset}" upper="${2.96 - safety_offset}"/>
     </joint>

Commit message: added schunk_lwa4d_custom macro and changed setting to use_factory_settings to make it easier to add default/DH config

File: schunk_description/urdf/lwa4d/lwa4d.urdf.xacro (robot description, xacro)
@@ -13,8 +13,8 @@
   </xacro:macro>
   <!-- invert_* is a xacro parameter to be used to adapt the urdf according to your hardware setup.
-       use invert_*:=true if you configured your hardware to follow DH-convention, i.e. motors have been inverted in the firmware.
-       use invert_*:=false if you are using factory settings, i.e. motors are not inverted in the firmware.
-       The default follows the DH-convention -->
-  <xacro:macro name="schunk_lwa4d" params="parent name *origin has_podest invert_j1:=true invert_j2:=true invert_j3:=true invert_j4:=true invert_j5:=true invert_j6:=true invert_j7:=true">
+       use invert_*:=true if  motors are inverted in the firmware.
+       use invert_*:=false if motors are not inverted in the firmware.
+  -->
+  <xacro:macro name="schunk_lwa4d_custom" params="parent name *origin has_podest invert_j1 invert_j2 invert_j3 invert_j4 invert_j5 invert_j6 invert_j7">
     <xacro:if value="${has_podest}">
       <!-- joint between base_link and lwa4p_extended_connector_link -->
@@ -256,3 +256,20 @@
     <xacro:schunk_lwa4d_transmission name="${name}"/>
   </xacro:macro>
+  <!-- use_factory_setings is a xacro parameter to be used to adapt the urdf according to your hardware setup.
+       use_factory_settings:=true if you have not modified the schunk firmware.
+       use_factory_settings:=false if you have modified the schunk firmware to follow DH parameters (you have inverted the PRL+ motors j1-j5)
+       if you are using custom firmware settings, use schunk_lwa4d_custom
+  -->
+  <xacro:macro name="schunk_lwa4d" params="parent name *origin has_podest use_factory_settings:=false">
+    <xacro:if value="${use_factory_settings}">
+      <xacro:schunk_lwa4d_custom parent="${parent}" name="${name}" has_podest="${has_podest}" invert_j1="false" invert_j2="false" invert_j3="false" invert_j4="false" invert_j5="false" invert_j6="true" invert_j7="true">
+        <xacro:insert_block name="origin" />
+      </xacro:schunk_lwa4d_custom>
+    </xacro:if>
+    <xacro:unless value="${use_factory_settings}">
+      <xacro:schunk_lwa4d_custom parent="${parent}" name="${name}" has_podest="${has_podest}" invert_j1="true" invert_j2="true" invert_j3="true" invert_j4="true" invert_j5="true" invert_j6="true" invert_j7="true">
+        <xacro:insert_block name="origin" />
+      </xacro:schunk_lwa4d_custom>
+    </xacro:unless>
+  </xacro:macro>
 </robot>

Commit message: python True/False

File: schunk_description/urdf/lwa4d/lwa4d.urdf.xacro (robot description, xacro)
@@ -14,6 +14,6 @@
   </xacro:macro>
   <!-- invert_* is a xacro parameter to be used to adapt the urdf according to your hardware setup.
-       use invert_*:=true if  motors are inverted in the firmware.
-       use invert_*:=false if motors are not inverted in the firmware.
+       use invert_*:=True if  motors are inverted in the firmware.
+       use invert_*:=False if motors are not inverted in the firmware.
   -->
   <xacro:macro name="schunk_lwa4d_custom" params="parent name *origin has_podest invert_j1 invert_j2 invert_j3 invert_j4 invert_j5 invert_j6 invert_j7">
@@ -265,16 +265,16 @@
   </xacro:macro>
   <!-- use_factory_setings is a xacro parameter to be used to adapt the urdf according to your hardware setup.
-       use_factory_settings:=true if you have not modified the schunk firmware.
-       use_factory_settings:=false if you have modified the schunk firmware to follow DH parameters (you have inverted the PRL+ motors j1-j5)
+       use_factory_settings:=True if you have not modified the schunk firmware.
+       use_factory_settings:=False if you have modified the schunk firmware to follow DH parameters (you have inverted the PRL+ motors j1-j5)
        if you are using custom firmware settings, use schunk_lwa4d_custom
   -->
-  <xacro:macro name="schunk_lwa4d" params="parent name *origin has_podest use_factory_settings:=false">
+  <xacro:macro name="schunk_lwa4d" params="parent name *origin has_podest use_factory_settings:=False">
     <xacro:if value="${use_factory_settings}">
-      <xacro:schunk_lwa4d_custom parent="${parent}" name="${name}" has_podest="${has_podest}" invert_j1="false" invert_j2="false" invert_j3="false" invert_j4="false" invert_j5="false" invert_j6="true" invert_j7="true">
+      <xacro:schunk_lwa4d_custom parent="${parent}" name="${name}" has_podest="${has_podest}" invert_j1="False" invert_j2="False" invert_j3="False" invert_j4="False" invert_j5="False" invert_j6="True" invert_j7="True">
         <xacro:insert_block name="origin" />
       </xacro:schunk_lwa4d_custom>
     </xacro:if>
     <xacro:unless value="${use_factory_settings}">
-      <xacro:schunk_lwa4d_custom parent="${parent}" name="${name}" has_podest="${has_podest}" invert_j1="true" invert_j2="true" invert_j3="true" invert_j4="true" invert_j5="true" invert_j6="true" invert_j7="true">
+      <xacro:schunk_lwa4d_custom parent="${parent}" name="${name}" has_podest="${has_podest}" invert_j1="True" invert_j2="True" invert_j3="True" invert_j4="True" invert_j5="True" invert_j6="True" invert_j7="True">
         <xacro:insert_block name="origin" />
       </xacro:schunk_lwa4d_custom>
