Commit message: Revert "python True/False"
This reverts commit 28ee3a0bca4514baef065d4e2744b73ca7bd35f9.

File: schunk_description/urdf/lwa4d/lwa4d.urdf.xacro (robot description, xacro)
@@ -14,6 +14,6 @@
   </xacro:macro>
   <!-- invert_* is a xacro parameter to be used to adapt the urdf according to your hardware setup.
-       use invert_*:=True if  motors are inverted in the firmware.
-       use invert_*:=False if motors are not inverted in the firmware.
+       use invert_*:=true if  motors are inverted in the firmware.
+       use invert_*:=false if motors are not inverted in the firmware.
   -->
   <xacro:macro name="schunk_lwa4d_custom" params="parent name *origin has_podest invert_j1 invert_j2 invert_j3 invert_j4 invert_j5 invert_j6 invert_j7">
@@ -265,16 +265,16 @@
   </xacro:macro>
   <!-- use_factory_setings is a xacro parameter to be used to adapt the urdf according to your hardware setup.
-       use_factory_settings:=True if you have not modified the schunk firmware.
-       use_factory_settings:=False if you have modified the schunk firmware to follow DH parameters (you have inverted the PRL+ motors j1-j5)
+       use_factory_settings:=true if you have not modified the schunk firmware.
+       use_factory_settings:=false if you have modified the schunk firmware to follow DH parameters (you have inverted the PRL+ motors j1-j5)
        if you are using custom firmware settings, use schunk_lwa4d_custom
   -->
-  <xacro:macro name="schunk_lwa4d" params="parent name *origin has_podest use_factory_settings:=False">
+  <xacro:macro name="schunk_lwa4d" params="parent name *origin has_podest use_factory_settings:=false">
     <xacro:if value="${use_factory_settings}">
-      <xacro:schunk_lwa4d_custom parent="${parent}" name="${name}" has_podest="${has_podest}" invert_j1="False" invert_j2="False" invert_j3="False" invert_j4="False" invert_j5="False" invert_j6="True" invert_j7="True">
+      <xacro:schunk_lwa4d_custom parent="${parent}" name="${name}" has_podest="${has_podest}" invert_j1="false" invert_j2="false" invert_j3="false" invert_j4="false" invert_j5="false" invert_j6="true" invert_j7="true">
         <xacro:insert_block name="origin" />
       </xacro:schunk_lwa4d_custom>
     </xacro:if>
     <xacro:unless value="${use_factory_settings}">
-      <xacro:schunk_lwa4d_custom parent="${parent}" name="${name}" has_podest="${has_podest}" invert_j1="True" invert_j2="True" invert_j3="True" invert_j4="True" invert_j5="True" invert_j6="True" invert_j7="True">
+      <xacro:schunk_lwa4d_custom parent="${parent}" name="${name}" has_podest="${has_podest}" invert_j1="true" invert_j2="true" invert_j3="true" invert_j4="true" invert_j5="true" invert_j6="true" invert_j7="true">
         <xacro:insert_block name="origin" />
       </xacro:schunk_lwa4d_custom>
