Commit message: change to light grey

File: schunk_description/urdf/sdh/sdh.gazebo.xacro (robot description, xacro)
@@ -10,5 +10,5 @@
 		</gazebo>
 		<gazebo reference="${name}_finger_11_link">
-			<material>Schunk/Black</material>
+			<material>Schunk/LightGrey</material>
 			<turnGravityOff>false</turnGravityOff>
 		</gazebo>
@@ -45,5 +45,5 @@
 		</gazebo>
 		<gazebo reference="${name}_finger_21_link">
-			<material>Schunk/Black</material>
+			<material>Schunk/LightGrey</material>
 			<turnGravityOff>false</turnGravityOff>
 		</gazebo>
@@ -80,5 +80,5 @@
 		</gazebo>
 		<gazebo reference="${name}_thumb_1_link">
-			<material>Schunk/Black</material>
+			<material>Schunk/LightGrey</material>
 			<turnGravityOff>false</turnGravityOff>
 		</gazebo>

File: schunk_description/urdf/sdh/sdh.urdf.xacro (robot description, xacro)
@@ -24,5 +24,5 @@
 					<mesh filename="package://schunk_description/meshes/sdh/palm.stl" />
 				</geometry>
-				<material name="Schunk/DarkGrey" />
+				<material name="Schunk/LightGrey" />
 			</visual>
 			<collision>
@@ -68,5 +68,5 @@
 					<mesh filename="package://schunk_description/meshes/sdh/knuckle.stl" />
 				</geometry>
-				<material name="Schunk/Black" />
+				<material name="Schunk/LightGrey" />
 			</visual>
 			<collision>
@@ -97,5 +97,5 @@
 					<mesh filename="package://schunk_description/meshes/sdh/finger.stl" />
 				</geometry>
-			<material name="Schunk/DarkGrey" />
+			<material name="Schunk/LightGrey" />
 			</visual>
 			<collision>
@@ -126,5 +126,5 @@
 					<mesh filename="package://schunk_description/meshes/sdh/finger_tip.stl" />
 				</geometry>
-				<material name="Schunk/Black" />
+				<material name="Schunk/LightGrey" />
 			</visual>
 			<collision>
@@ -157,5 +157,5 @@
 					<mesh filename="package://schunk_description/meshes/sdh/knuckle.stl" />
 				</geometry>
-				<material name="Schunk/Black" />
+				<material name="Schunk/LightGrey" />
 			</visual>
 			<collision>
@@ -186,5 +186,5 @@
 					<mesh filename="package://schunk_description/meshes/sdh/finger.stl" />
 				</geometry>
-				<material name="Schunk/DarkGrey" />
+				<material name="Schunk/LightGrey" />
 			</visual>
 			<collision>
@@ -215,5 +215,5 @@
 					<mesh filename="package://schunk_description/meshes/sdh/finger_tip.stl" />
 				</geometry>
-				<material name="Schunk/Black" />
+				<material name="Schunk/LightGrey" />
 			</visual>
 			<collision>
@@ -242,5 +242,5 @@
 					<mesh filename="package://schunk_description/meshes/sdh/knuckle.stl" />
 				</geometry>
-				<material name="Schunk/Black" />
+				<material name="Schunk/LightGrey" />
 			</visual>
 			<collision>
@@ -271,5 +271,5 @@
 					<mesh filename="package://schunk_description/meshes/sdh/finger.stl" />
 				</geometry>
-				<material name="Schunk/DarkGrey" />
+				<material name="Schunk/LightGrey" />
 			</visual>
 			<collision>
@@ -300,5 +300,5 @@
 					<mesh filename="package://schunk_description/meshes/sdh/finger_tip.stl" />
 				</geometry>
-				<material name="Schunk/Black" />
+				<material name="Schunk/LightGrey" />
 			</visual>
 			<collision>

Commit message: fix sdh description according to new gazebo format

File: schunk_description/urdf/sdh/sdh.gazebo.xacro (robot description, xacro)
@@ -15,4 +15,10 @@
 		<gazebo reference="${name}_finger_12_link">
 			<selfCollide>true</selfCollide>
+			<sensor name='${name}_finger_12_contact_sensor' type='contact'>
+				<contact>
+					<collision>${name}_finger_12_link_geom</collision>
+				</contact>
+			</sensor>
+<!--
 			<sensor:contact name="${name}_finger_12_contact_sensor">
 				<geom>${name}_finger_12_link_geom</geom>
@@ -26,4 +32,5 @@
 				</controller:gazebo_ros_bumper>
 			</sensor:contact>
+-->
 			<material>Schunk/LightGrey</material>
 			<turnGravityOff>false</turnGravityOff>
@@ -31,4 +38,10 @@
 		<gazebo reference="${name}_finger_13_link">
 			<selfCollide>true</selfCollide>
+			<sensor name='${name}_finger_13_contact_sensor' type='contact'>
+				<contact>
+					<collision>${name}_finger_13_link_geom</collision>
+				</contact>
+			</sensor>
+<!--
 			<sensor:contact name="${name}_finger_13_contact_sensor">
 				<geom>${name}_finger_13_link_geom</geom>
@@ -42,4 +55,5 @@
 				</controller:gazebo_ros_bumper>
 			</sensor:contact>
+-->
 			<material>Schunk/LightGrey</material>
 		</gazebo>
@@ -49,5 +63,11 @@
 		</gazebo>
 		<gazebo reference="${name}_finger_22_link">
-		<selfCollide>true</selfCollide>
+			<selfCollide>true</selfCollide>
+			<sensor name='${name}_finger_22_contact_sensor' type='contact'>
+				<contact>
+					<collision>${name}_finger_22_link_geom</collision>
+				</contact>
+			</sensor>
+<!--
 			<sensor:contact name="${name}_finger_22_contact_sensor">
 				<geom>${name}_finger_22_link_geom</geom>
@@ -61,4 +81,5 @@
 				</controller:gazebo_ros_bumper>
 			</sensor:contact>
+-->
 			<material>Schunk/LightGrey</material>
 			<turnGravityOff>false</turnGravityOff>
@@ -66,4 +87,10 @@
 		<gazebo reference="${name}_finger_23_link">
 			<selfCollide>true</selfCollide>
+			<sensor name='${name}_finger_23_contact_sensor' type='contact'>
+				<contact>
+					<collision>${name}_finger_23_link_geom</collision>
+				</contact>
+			</sensor>
+<!--
 			<sensor:contact name="${name}_finger_23_contact_sensor">
 				<geom>${name}_finger_23_link_geom</geom>
@@ -77,4 +104,5 @@
 				</controller:gazebo_ros_bumper>
 			</sensor:contact>
+-->
 			<material>Schunk/LightGrey</material>
 		</gazebo>
@@ -85,4 +113,10 @@
 		<gazebo reference="${name}_thumb_2_link">
 			<selfCollide>true</selfCollide>
+			<sensor name='${name}_thumb_2_contact_sensor' type='contact'>
+				<contact>
+					<collision>${name}_thumb_2_link_geom</collision>
+				</contact>
+			</sensor>
+<!--
 			<sensor:contact name="${name}_thumb_2_contact_sensor">
 				<geom>${name}_thumb_2_link_geom</geom>
@@ -96,4 +130,5 @@
 				</controller:gazebo_ros_bumper>
 			</sensor:contact>
+-->
 			<material>Schunk/LightGrey</material>
 			<turnGravityOff>false</turnGravityOff>
@@ -101,4 +136,10 @@
 		<gazebo reference="${name}_thumb_3_link">
 			<selfCollide>true</selfCollide>
+			<sensor name='${name}_thumb_3_contact_sensor' type='contact'>
+				<contact>
+					<collision>${name}_thumb_3_link_geom</collision>
+				</contact>
+			</sensor>
+<!--
 			<sensor:contact name="${name}_thumb_3_contact_sensor">
 				<geom>${name}_thumb_3_link_geom</geom>
@@ -112,4 +153,5 @@
 				</controller:gazebo_ros_bumper>
 			</sensor:contact>
+-->
 			<material>Schunk/LightGrey</material>
 		</gazebo>

Commit message: fix bumper plugins

File: schunk_description/urdf/sdh/sdh.gazebo.xacro (robot description, xacro)
@@ -16,19 +16,16 @@
       <self_collide>false</self_collide>
       <material>Schunk/LightGrey</material>
-<!--
       <sensor name='${name}_finger_12_contact_sensor' type='contact'>
-        <always_on>true</always_on>
+        <always_on>1</always_on>
         <update_rate>100</update_rate>
         <contact>
-          <collision>${name}_finger_12_link_geom</collision>
+          <collision>${name}_finger_12_link_collision</collision>
+          <topic>${name}_finger_12_bumper</topic>
         </contact>
         <plugin name="${name}_finger_12_gazebo_ros_bumper_controller" filename="libgazebo_ros_bumper.so">
-          <alwaysOn>true</alwaysOn>
-          <updateRate>100.0</updateRate>
           <frameName>${name}_finger_12_link</frameName>
           <bumperTopicName>${name}_finger_12_bumper</bumperTopicName>
         </plugin>
       </sensor>
--->
     </gazebo>
     <gazebo reference="${name}_finger_13_link">
@@ -36,19 +33,16 @@
       <self_collide>false</self_collide>
       <material>Schunk/LightGrey</material>
-<!--
       <sensor name='${name}_finger_13_contact_sensor' type='contact'>
-        <always_on>true</always_on>
+        <always_on>1</always_on>
         <update_rate>100</update_rate>
         <contact>
-          <collision>${name}_finger_13_link_geom</collision>
+          <collision>${name}_finger_13_link_collision</collision>
+          <topic>${name}_finger_13_bumper</topic>
         </contact>
         <plugin name="${name}_finger_13_gazebo_ros_bumper_controller" filename="libgazebo_ros_bumper.so">
-          <alwaysOn>true</alwaysOn>
-          <updateRate>100.0</updateRate>
           <frameName>${name}_finger_13_link</frameName>
           <bumperTopicName>${name}_finger_13_bumper</bumperTopicName>
         </plugin>
       </sensor>
--->
     </gazebo>
     <gazebo reference="${name}_finger_21_link">
@@ -65,19 +59,16 @@
       <self_collide>false</self_collide>
       <material>Schunk/LightGrey</material>
-<!--
       <sensor name='${name}_finger_22_contact_sensor' type='contact'>
-        <always_on>true</always_on>
+        <always_on>1</always_on>
         <update_rate>100</update_rate>
         <contact>
-          <collision>${name}_finger_22_link_geom</collision>
+          <collision>${name}_finger_22_link_collision</collision>
+          <topic>${name}_finger_22_bumper</topic>
         </contact>
         <plugin name="${name}_finger_22_gazebo_ros_bumper_controller" filename="libgazebo_ros_bumper.so">
-          <alwaysOn>true</alwaysOn>
-          <updateRate>100.0</updateRate>
           <frameName>${name}_finger_22_link</frameName>
           <bumperTopicName>${name}_finger_22_bumper</bumperTopicName>
         </plugin>
       </sensor>
--->
     </gazebo>
     <gazebo reference="${name}_finger_23_link">
@@ -85,19 +76,16 @@
       <self_collide>false</self_collide>
       <material>Schunk/LightGrey</material>
-<!--
       <sensor name='${name}_finger_23_contact_sensor' type='contact'>
-        <always_on>true</always_on>
+        <always_on>1</always_on>
         <update_rate>100</update_rate>
         <contact>
-          <collision>${name}_finger_23_link_geom</collision>
+          <collision>${name}_finger_23_link_collision</collision>
+          <topic>${name}_finger_23_bumper</topic>
         </contact>
         <plugin name="${name}_finger_23_gazebo_ros_bumper_controller" filename="libgazebo_ros_bumper.so">
-          <alwaysOn>true</alwaysOn>
-          <updateRate>100.0</updateRate>
           <frameName>${name}_finger_23_link</frameName>
           <bumperTopicName>${name}_finger_23_bumper</bumperTopicName>
         </plugin>
       </sensor>
--->
     </gazebo>
     <gazebo reference="${name}_thumb_1_link">
@@ -110,19 +98,16 @@
       <self_collide>false</self_collide>
       <material>Schunk/LightGrey</material>
-<!--
       <sensor name='${name}_thumb_2_contact_sensor' type='contact'>
-        <always_on>true</always_on>
+        <always_on>1</always_on>
         <update_rate>100</update_rate>
         <contact>
-          <collision>${name}_thumb_2_link_geom</collision>
+          <collision>${name}_thumb_2_link_collision</collision>
+          <topic>${name}_thumb_2_bumper</topic>
         </contact>
         <plugin name="${name}_thumb_2_gazebo_ros_bumper_controller" filename="libgazebo_ros_bumper.so">
-          <alwaysOn>true</alwaysOn>
-          <updateRate>100.0</updateRate>
           <frameName>${name}_thumb_2_link</frameName>
           <bumperTopicName>${name}_thumb_2_bumper</bumperTopicName>
         </plugin>
       </sensor>
--->
     </gazebo>
     <gazebo reference="${name}_thumb_3_link">
@@ -130,19 +115,16 @@
       <self_collide>false</self_collide>
       <material>Schunk/LightGrey</material>
-<!--
       <sensor name='${name}_thumb_3_contact_sensor' type='contact'>
-        <always_on>true</always_on>
+        <always_on>1</always_on>
         <update_rate>100</update_rate>
         <contact>
-          <collision>${name}_thumb_3_link_geom</collision>
+          <collision>${name}_thumb_3_link_collision</collision>
+          <topic>${name}_thumb_3_bumper</topic>
         </contact>
         <plugin name="${name}_thumb_3_gazebo_ros_bumper_controller" filename="libgazebo_ros_bumper.so">
-          <alwaysOn>true</alwaysOn>
-          <updateRate>100.0</updateRate>
           <frameName>${name}_thumb_3_link</frameName>
           <bumperTopicName>${name}_thumb_3_bumper</bumperTopicName>
         </plugin>
       </sensor>
--->
     </gazebo>
     <!--gazebo reference="${name}_finger_21_joint">
