Commit message: 2DOF Hack for finger

File: schunk_description/urdf/pg70/pg70.transmission.xacro (robot description, xacro)
@@ -6,13 +6,13 @@
 	<xacro:macro name="schunk_pg70_transmission" params="name">
 		<!-- finger1 -->
-		<transmission name="${name}_finger_1_trans" type="pr2_mechanism_model/SimpleTransmission">
-			<actuator name="${name}_finger_1_motor"/>
-			<joint name="${name}_finger_1_joint"/>
+		<transmission name="${name}_finger_trans" type="pr2_mechanism_model/SimpleTransmission">
+			<actuator name="${name}_finger_motor"/>
+			<joint name="${name}_finger_joint"/>
 			<mechanicalReduction>1</mechanicalReduction>
 		</transmission>
 		<!-- finger2 -->
-		<transmission name="${name}_finger_2_trans" type="pr2_mechanism_model/SimpleTransmission">
-			<actuator name="${name}_finger_2_motor"/>
-			<joint name="${name}_finger_2_joint"/>
+		<transmission name="${name}_finger_mimic_trans" type="pr2_mechanism_model/SimpleTransmission">
+			<actuator name="${name}_finger_mimic_motor"/>
+			<joint name="${name}_finger_mimic_joint"/>
 			<mechanicalReduction>1</mechanicalReduction>
 		</transmission>

File: schunk_description/urdf/pg70/pg70.urdf.xacro (robot description, xacro)
@@ -17,5 +17,5 @@
 			<inertial>
 				<origin xyz="0 0 0" rpy="0 0 0"/>
-				<mass value="1.4"/>
+				<mass value="1.0"/>
 				<inertia ixx="0.01" ixy="0" ixz="0" iyy="0.01" iyz="0" izz="0.01" />
 			</inertial>
@@ -30,5 +30,5 @@
 				<origin xyz="0 0 0.0465" rpy="0 0 0" />
 				<geometry>
-					<box size="0.08 0.10 0.093"/>
+					<box size="0.075 0.095 0.085"/>
 				</geometry>
 			</collision>
@@ -36,5 +36,5 @@
 		<!-- finger1 -->
 		<!-- joint between pg70_palm_link and pg70_finger_1_link -->
-		<joint name="${name}_finger_1_joint" type="prismatic">
+		<joint name="${name}_finger_joint" type="prismatic">
 			<origin xyz="0.0 0.03 0.093" rpy="0 0 0" />
 			<parent link="${name}_palm_link"/>
@@ -47,5 +47,5 @@
 			<inertial>
 				<origin xyz="0 0 0" rpy="0 0 0"/>
-				<mass value="0.01"/>
+				<mass value="0.1"/>
 				<inertia ixx="0.01" ixy="0" ixz="0" iyy="0.01" iyz="0" izz="0.01" />
 			</inertial>
@@ -53,5 +53,5 @@
 				<origin xyz="0 0 0.03" rpy="0 0 0" />
 				<geometry>
-					<box size="0.03 0.01 0.06"/>
+					<box size="0.03 0.01 0.060"/>
 				</geometry>
 				<material name="Schunk/LightGrey" />
@@ -60,5 +60,5 @@
 				<origin xyz="0 0 0.03" rpy="0 0 0" />
 				<geometry>
-					<box size="0.03 0.01 0.06"/>
+					<box size="0.025 0.005 0.055"/>
 				</geometry>
 			</collision>
@@ -66,10 +66,10 @@
 		<!-- finger2 -->
 		<!-- joint between pg70_palm_link and pg70_finger_2_link -->
-		<joint name="${name}_finger_2_joint" type="prismatic">
-			<mimic joint="${name}_finger_1_joint" multiplier="1" offset="0"/>
-			<origin xyz="0.0 -0.03 0.093" rpy="0 0 0" />
+		<joint name="${name}_finger_mimic_joint" type="prismatic">
+			<!--mimic joint="${name}_finger_joint" multiplier="1" offset="0"/-->
+			<origin xyz="0.0 -0.03 0.093" rpy="0 0 3.14" />
 			<parent link="${name}_palm_link"/>
 			<child link="${name}_finger_2_link"/>
-			<axis xyz="0 -1 0" />
+			<axis xyz="0 1 0" />
 			<dynamics damping="1" />
 			<limit effort="100" lower="0" upper="0.034" velocity="5"/>
@@ -78,5 +78,5 @@
 			<inertial>
 				<origin xyz="0 0 0" rpy="0 0 0"/>
-				<mass value="0.01"/>
+				<mass value="0.1"/>
 				<inertia ixx="0.01" ixy="0" ixz="0" iyy="0.01" iyz="0" izz="0.01" />
 			</inertial>
@@ -84,5 +84,5 @@
 				<origin xyz="0 0 0.03" rpy="0 0 0" />
 				<geometry>
-					<box size="0.03 0.01 0.06"/>
+					<box size="0.03 0.01 0.059"/>
 				</geometry>
 				<material name="Schunk/LightGrey" />
@@ -91,5 +91,5 @@
 				<origin xyz="0 0 0.03" rpy="0 0 0" />
 				<geometry>
-					<box size="0.03 0.01 0.06"/>
+					<box size="0.025 0.005 0.055"/>
 				</geometry>
 			</collision>

Commit message: lwad description without base

File: schunk_description/urdf/pg70/pg70.transmission.xacro (robot description, xacro)
@@ -11,5 +11,5 @@
       </joint>
       <actuator name="${name}_finger_left_motor">
-        <mechanicalReduction>1</mechanicalReduction>
+        <mechanicalReduction>0.5</mechanicalReduction>
       </actuator>
     </transmission>
@@ -23,5 +23,5 @@
       </joint>
       <actuator name="${name}_finger_right_motor">
-        <mechanicalReduction>1</mechanicalReduction>
+        <mechanicalReduction>0.5</mechanicalReduction>
       </actuator>
     </transmission>

File: schunk_description/urdf/pg70/pg70.urdf.xacro (robot description, xacro)
@@ -35,7 +35,7 @@
       <parent link="${name}_palm_link" />
       <child link="${name}_finger_left_link" />
-      <limit effort="100" lower="-0.001" upper="0.0345" velocity="2.0"/>
+      <limit effort="100" lower="-0.001" upper="0.061" velocity="2.0"/>
       <calibration rising="${pg70_finger_left_ref}"/>
-      <origin xyz="0 0.0105 0.0789" rpy="0 0 0"/>
+      <origin xyz="0 0.0 0.0789" rpy="0 0 0"/>
       <axis xyz="0 1 0" />
     </joint>
@@ -67,7 +67,7 @@
       <parent link="${name}_palm_link" />
       <child link="${name}_finger_right_link" />
-      <limit effort="100" lower="-0.001" upper="0.0345" velocity="2.0"/>
+      <limit effort="100" lower="-0.001" upper="0.061" velocity="2.0"/>
       <calibration rising="${pg70_finger_right_ref}"/>
-      <origin xyz="0 -0.0105 0.0789" rpy="-0 0 0"/>
+      <origin xyz="0 0.0 0.0789" rpy="-0 0 0"/>
       <axis xyz="0 -1 0" />
     </joint>
