Commit message: fix pg70

File: schunk_description/urdf/pg70/pg70.gazebo.xacro (robot description, xacro)
@@ -5,15 +5,12 @@
       <gravity>true</gravity>
       <self_collide>false</self_collide>
-      <material>Schunk/LightGrey</material>
     </gazebo>
     <gazebo reference="${name}_finger_left_link">
       <gravity>true</gravity>
       <self_collide>false</self_collide>
-      <material>Schunk/LightGrey</material>
     </gazebo>
     <gazebo reference="${name}_finger_right_link">
       <gravity>true</gravity>
       <self_collide>false</self_collide>
-      <material>Schunk/LightGrey</material>
     </gazebo>
   </xacro:macro>

File: schunk_description/urdf/pg70/pg70.transmission.xacro (robot description, xacro)
@@ -6,10 +6,10 @@
       <type>transmission_interface/SimpleTransmission</type>
       <joint name="${name}_finger_left_joint">
-        <hardwareInterface>EffortJointInterface</hardwareInterface>
         <hardwareInterface>PositionJointInterface</hardwareInterface>
         <hardwareInterface>VelocityJointInterface</hardwareInterface>
+        <hardwareInterface>EffortJointInterface</hardwareInterface>
       </joint>
       <actuator name="${name}_finger_left_motor">
-        <mechanicalReduction>0.5</mechanicalReduction>
+        <mechanicalReduction>1</mechanicalReduction>
       </actuator>
     </transmission>
@@ -18,10 +18,10 @@
       <type>transmission_interface/SimpleTransmission</type>
       <joint name="${name}_finger_right_joint">
-        <hardwareInterface>EffortJointInterface</hardwareInterface>
         <hardwareInterface>PositionJointInterface</hardwareInterface>
         <hardwareInterface>VelocityJointInterface</hardwareInterface>
+        <hardwareInterface>EffortJointInterface</hardwareInterface>
       </joint>
       <actuator name="${name}_finger_right_motor">
-        <mechanicalReduction>0.5</mechanicalReduction>
+        <mechanicalReduction>1</mechanicalReduction>
       </actuator>
     </transmission>

File: schunk_description/urdf/pg70/pg70.urdf.xacro (robot description, xacro)
@@ -19,23 +19,17 @@
           <mesh filename="package://schunk_description/meshes/pg70/pg70.dae" />
         </geometry>
-        <material name="blue">
-          <color rgba="0 0 1 1"/>
-        </material>
       </visual>
       <collision>
         <geometry>
-          <mesh filename="package://schunk_description/meshes/pg70/pg70.dae" />
+          <mesh filename="package://schunk_description/meshes/pg70/pg70.stl" />
         </geometry>
-        <material name="blue">
-          <color rgba="0 0 1 1"/>
-        </material>
       </collision>
     </link>
     <joint name="${name}_finger_left_joint" type="prismatic" >
+      <origin xyz="0 0 0.0789" rpy="0 0 0"/>
       <parent link="${name}_palm_link" />
       <child link="${name}_finger_left_link" />
-      <limit effort="100" lower="-0.001" upper="0.061" velocity="2.0"/>
-      <origin xyz="0 0 0.0789" rpy="0 0 0"/>
       <axis xyz="0 1 0" />
+      <limit effort="10" lower="-0.001" upper="0.061" velocity="2.0"/>
     </joint>
     <link name="${name}_finger_left_link">
@@ -63,10 +57,10 @@
     </link>
     <joint name="${name}_finger_right_joint" type="prismatic" >
-      <mimic joint="${name}_finger_left_joint" multiplier="1" offset="0"/>
+      <origin xyz="0 0 0.0789" rpy="-0 0 0"/>
       <parent link="${name}_palm_link" />
       <child link="${name}_finger_right_link" />
-      <limit effort="100" lower="-0.001" upper="0.061" velocity="2.0"/>
-      <origin xyz="0 0 0.0789" rpy="-0 0 0"/>
       <axis xyz="0 -1 0" />
+      <mimic joint="${name}_finger_left_joint" multiplier="1" offset="0"/>
+      <limit effort="10" lower="-0.001" upper="0.061" velocity="2.0"/>
     </joint>
     <link name="${name}_finger_right_link">
