Commit message: update pg70

File: schunk_description/urdf/pg70/pg70.urdf.xacro (robot description, xacro)
@@ -21,5 +21,5 @@
 			</inertial>
 			<visual>
-				<origin xyz="0 0 0" rpy="0 0 0" />
+				<origin xyz="0.04 0 0" rpy="0 0 0" />
 				<geometry>
 					<box size="0.08 0.10 0.093"/>
@@ -28,5 +28,5 @@
 			</visual>
 			<collision>
-				<origin xyz="0 0 0" rpy="0 0 0" />
+				<origin xyz="0.04 0 0" rpy="0 0 0" />
 				<geometry>
 					<box size="0.08 0.10 0.093"/>

Commit message: fix fingers

File: schunk_description/urdf/pg70/pg70.urdf.xacro (robot description, xacro)
@@ -21,5 +21,5 @@
 			</inertial>
 			<visual>
-				<origin xyz="0.04 0 0" rpy="0 0 0" />
+				<origin xyz="0 0 0.0465" rpy="0 0 0" />
 				<geometry>
 					<box size="0.08 0.10 0.093"/>
@@ -28,5 +28,5 @@
 			</visual>
 			<collision>
-				<origin xyz="0.04 0 0" rpy="0 0 0" />
+				<origin xyz="0 0 0.0465" rpy="0 0 0" />
 				<geometry>
 					<box size="0.08 0.10 0.093"/>
@@ -37,10 +37,10 @@
 		<!-- joint between pg70_palm_link and pg70_finger_1_link -->
 		<joint name="${name}_finger_1_joint" type="prismatic">
-			<origin xyz="0.0 0.03 0.06" rpy="0 0 0" />
+			<origin xyz="0.0 0.03 0.093" rpy="0 0 0" />
 			<parent link="${name}_palm_link"/>
 			<child link="${name}_finger_1_link"/>
 			<axis xyz="0 1 0" />
 			<dynamics damping="1" />
-			<limit effort="100" lower="0" upper="1.570796327" velocity="5"/>
+			<limit effort="100" lower="0" upper="0.034" velocity="5"/>
 		</joint>
 		<link name="${name}_finger_1_link">
@@ -51,5 +51,5 @@
 			</inertial>
 			<visual>
-				<origin xyz="0 0 0" rpy="0 0 0" />
+				<origin xyz="0 0 0.03" rpy="0 0 0" />
 				<geometry>
 					<box size="0.03 0.01 0.06"/>
@@ -58,5 +58,5 @@
 			</visual>
 			<collision>
-				<origin xyz="0 0 0" rpy="0 0 0" />
+				<origin xyz="0 0 0.03" rpy="0 0 0" />
 				<geometry>
 					<box size="0.03 0.01 0.06"/>
@@ -68,10 +68,10 @@
 		<joint name="${name}_finger_2_joint" type="prismatic">
 			<mimic joint="${name}_finger_1_joint" multiplier="1" offset="0"/>
-			<origin xyz="0.0 -0.03 0.06" rpy="0 0 0" />
+			<origin xyz="0.0 -0.03 0.093" rpy="0 0 0" />
 			<parent link="${name}_palm_link"/>
 			<child link="${name}_finger_2_link"/>
 			<axis xyz="0 -1 0" />
 			<dynamics damping="1" />
-			<limit effort="100" lower="0" upper="1.570796327" velocity="5"/>
+			<limit effort="100" lower="0" upper="0.034" velocity="5"/>
 		</joint>
 		<link name="${name}_finger_2_link">
@@ -82,5 +82,5 @@
 			</inertial>
 			<visual>
-				<origin xyz="0 0 0" rpy="0 0 0" />
+				<origin xyz="0 0 0.03" rpy="0 0 0" />
 				<geometry>
 					<box size="0.03 0.01 0.06"/>
@@ -89,5 +89,5 @@
 			</visual>
 			<collision>
-				<origin xyz="0 0 0" rpy="0 0 0" />
+				<origin xyz="0 0 0.03" rpy="0 0 0" />
 				<geometry>
 					<box size="0.03 0.01 0.06"/>

Commit message: pg70 collada model

File: schunk_description/urdf/pg70/pg70.urdf.xacro (robot description, xacro)
@@ -17,12 +17,11 @@
       </inertial>
       <visual>
-        <origin xyz="0 0 0.0465" rpy="0 0 0" />
+        <origin xyz="0 0 0" rpy="0 0 0" />
         <geometry>
-          <box size="0.08 0.10 0.093"/>
+          <mesh filename="package://schunk_description/meshes/pg70/pg70.dae" />
         </geometry>
-        <material name="Schunk/LightGrey" />
       </visual>
       <collision>
-        <origin xyz="0 0 0.0465" rpy="0 0 0" />
+        <origin xyz="0 0 0" rpy="0 0 0" />
         <geometry>
           <box size="0.075 0.095 0.085"/>
@@ -33,5 +32,5 @@
     <!-- joint between pg70_palm_link and pg70_finger_1_link -->
     <joint name="${name}_finger_joint" type="prismatic">
-      <origin xyz="0.0 0.03 0.093" rpy="0 0 0" />
+      <origin xyz="0.0 0.03 0.077" rpy="0 0 0" />
       <parent link="${name}_palm_link"/>
       <child link="${name}_finger_1_link"/>
@@ -64,5 +63,5 @@
     <joint name="${name}_finger_mimic_joint" type="prismatic">
       <!--mimic joint="${name}_finger_joint" multiplier="1" offset="0"/-->
-      <origin xyz="0.0 -0.03 0.093" rpy="0 0 3.14" />
+      <origin xyz="0.0 -0.03 0.077" rpy="0 0 3.14" />
       <parent link="${name}_palm_link"/>
       <child link="${name}_finger_2_link"/>

Commit message: origin for collision model is in the center of the box

File: schunk_description/urdf/pg70/pg70.urdf.xacro (robot description, xacro)
@@ -23,5 +23,5 @@
       </visual>
       <collision>
-        <origin xyz="0 0 0" rpy="0 0 0" />
+        <origin xyz="0 0 0.0425" rpy="0 0 0" />
         <geometry>
           <box size="0.075 0.095 0.085"/>

Commit message: pg70 setup

File: schunk_description/urdf/pg70/pg70.urdf.xacro (robot description, xacro)
@@ -35,7 +35,8 @@
       <parent link="${name}_palm_link"/>
       <child link="${name}_finger_1_link"/>
+      <calibration rising="${pg70_finger_1_ref}"/>
       <axis xyz="0 1 0" />
       <dynamics damping="1" />
-      <limit effort="100" lower="0" upper="0.034" velocity="5"/>
+      <limit effort="100" lower="-0.1" upper="1.1" velocity="5"/>
     </joint>
     <link name="${name}_finger_1_link">
@@ -66,7 +67,8 @@
       <parent link="${name}_palm_link"/>
       <child link="${name}_finger_2_link"/>
+      <calibration rising="${pg70_finger_2_ref}"/>
       <axis xyz="0 1 0" />
       <dynamics damping="1" />
-      <limit effort="100" lower="0" upper="0.034" velocity="5"/>
+      <limit effort="100" lower="-0.1" upper="1.1" velocity="5"/>
     </joint>
     <link name="${name}_finger_2_link">

Commit message: fix pg70 property name

File: schunk_description/urdf/pg70/pg70.urdf.xacro (robot description, xacro)
@@ -3,5 +3,5 @@
   <xacro:include filename="$(find schunk_description)/urdf/pg70/pg70.gazebo.xacro" />
   <xacro:include filename="$(find schunk_description)/urdf/pg70/pg70.transmission.xacro" />
-  <xacro:macro name="schunk_pg70" params="parent name *origin">
+  <xacro:macro name="schunk_pg70" params="parent name *origin pg70_finger_left_ref pg70_finger_right_ref">
     <!-- joint between arm_7_link and pg70_palm_link -->
     <joint name="${name}_palm_joint" type="fixed" >
@@ -35,5 +35,5 @@
       <parent link="${name}_palm_link"/>
       <child link="${name}_finger_1_link"/>
-      <calibration rising="${pg70_finger_1_ref}"/>
+      <calibration rising="${pg70_finger_left_ref}"/>
       <axis xyz="0 1 0" />
       <dynamics damping="1" />
@@ -67,5 +67,5 @@
       <parent link="${name}_palm_link"/>
       <child link="${name}_finger_2_link"/>
-      <calibration rising="${pg70_finger_2_ref}"/>
+      <calibration rising="${pg70_finger_right_ref}"/>
       <axis xyz="0 1 0" />
       <dynamics damping="1" />

Commit message: Update pg70.urdf.xacro

File: schunk_description/urdf/pg70/pg70.urdf.xacro (robot description, xacro)
@@ -37,5 +37,5 @@
       <limit effort="100" lower="-0.001" upper="0.061" velocity="2.0"/>
       <calibration rising="${pg70_finger_left_ref}"/>
-      <origin xyz="0 0.0 0.0789" rpy="0 0 0"/>
+      <origin xyz="0 0 0.0789" rpy="0 0 0"/>
       <axis xyz="0 1 0" />
     </joint>
@@ -69,5 +69,5 @@
       <limit effort="100" lower="-0.001" upper="0.061" velocity="2.0"/>
       <calibration rising="${pg70_finger_right_ref}"/>
-      <origin xyz="0 0.0 0.0789" rpy="-0 0 0"/>
+      <origin xyz="0 0 0.0789" rpy="-0 0 0"/>
       <axis xyz="0 -1 0" />
     </joint>

Commit message: new package schunk_pg70

File: schunk_description/urdf/pg70/pg70.urdf.xacro (robot description, xacro)
@@ -3,10 +3,39 @@
   <xacro:include filename="$(find schunk_description)/urdf/pg70/pg70.gazebo.xacro" />
   <xacro:include filename="$(find schunk_description)/urdf/pg70/pg70.transmission.xacro" />
-  <xacro:macro name="schunk_pg70" params="parent name *origin">
-    <joint name="${name}_palm_joint" type="fixed" >
-      <parent link="${parent}" />
-      <child link="${name}_palm_link" />
-      <xacro:insert_block name="origin" />
-    </joint>
+  <xacro:macro name="schunk_pg70" params="parent name *origin has_podest">
+    <xacro:if value="${has_podest}">
+      <joint name="${name}_podest_joint" type="fixed">
+        <insert_block name="origin" />
+        <parent link="${parent}"/>
+        <child link="${name}_podest_link"/>
+      </joint>
+      <link name="${name}_podest_link">
+        <xacro:default_inertial/>
+        <visual>
+          <origin xyz="0 0 0" rpy="0 ${M_PI} 0" />
+          <geometry>
+          <mesh filename="package://schunk_description/meshes/lwa4p/arm_base_link.stl" />
+          </geometry>
+        </visual>
+        <collision>
+          <origin xyz="0 0 0" rpy="0 ${M_PI} 0" />
+          <geometry>
+          <mesh filename="package://schunk_description/meshes/lwa4p/arm_base_link.stl" />
+          </geometry>
+        </collision>
+      </link>
+      <joint name="${name}_palm_joint" type="fixed">
+        <origin xyz="0 0 0.10" rpy="0 0 0" />
+        <parent link="${name}_podest_link"/>
+        <child link="${name}_palm_link"/>
+      </joint>
+    </xacro:if>
+    <xacro:unless value="${has_podest}">
+      <joint name="${name}_palm_joint" type="fixed">
+        <insert_block name="origin" />
+        <parent link="${parent}"/>
+        <child link="${name}_palm_link" />
+      </joint>
+    </xacro:unless>
     <link name="${name}_palm_link">
       <inertial>

Commit message: fix limits and simplify collision model
The gripper fingers both can move 30mm according to the datasheet
to give a distance of 60mm between the fingers.
The _finger_palm_link can be easily simplified as a box geometry
for faster collision checking.

File: schunk_description/urdf/pg70/pg70.urdf.xacro (robot description, xacro)
@@ -51,6 +51,7 @@
       </visual>
       <collision>
+        <origin xyz="0 0 ${0.040-0.5*0.0171}" rpy="0 0 0" />
         <geometry>
-          <mesh filename="package://schunk_description/meshes/pg70/pg70.stl" />
+          <box size="0.082 0.114 0.080" />
         </geometry>
       </collision>
@@ -61,5 +62,5 @@
       <child link="${name}_finger_left_link" />
       <axis xyz="0 1 0" />
-      <limit effort="10" lower="-0.001" upper="0.061" velocity="2.0"/>
+      <limit effort="10" lower="-0.001" upper="0.0301" velocity="0.041"/>
     </joint>
     <link name="${name}_finger_left_link">
@@ -92,5 +93,5 @@
       <axis xyz="0 -1 0" />
       <mimic joint="${name}_finger_left_joint" multiplier="1" offset="0"/>
-      <limit effort="10" lower="-0.001" upper="0.061" velocity="2.0"/>
+      <limit effort="10" lower="-0.001" upper="0.0301" velocity="0.041"/>
     </joint>
     <link name="${name}_finger_right_link">
