Commit message: wrong lenght

File: schunk_description/urdf/lwa4p/lwa4p.urdf.xacro (robot description, xacro)
@@ -156,5 +156,5 @@
     <!-- joint between arm_4_link and arm_5_link -->
     <joint name="${name}_5_joint" type="revolute">
-      <origin xyz="0 0.005263 0.365" rpy="1.5708 0 3.14159" />
+      <origin xyz="0 0.005263 0.305" rpy="1.5708 0 3.14159" />
       <parent link="${name}_4_link"/>
       <child link="${name}_5_link"/>

Commit message: prepare lwa4p for VelocityInterface

File: schunk_description/urdf/lwa4p/lwa4p.urdf.xacro (robot description, xacro)
@@ -11,4 +11,6 @@
     </joint>
     <link name="${name}_0_link">
+      <xacro:default_inertial/>
+<!--
       <inertial>
         <origin xyz="0 0 0" rpy="0 0 0" />
@@ -16,4 +18,5 @@
         <inertia ixx="0.01" ixy="0" ixz="0" iyy="0.01" iyz="0" izz="0.01" />
       </inertial>
+-->
       <visual>
         <origin xyz="0 0 0" rpy="0 0 0" />
@@ -37,9 +40,10 @@
       <axis xyz="0 0 1"/>
       <calibration rising="${arm_1_ref}"/>
-      <dynamics damping="10" />
       <limit effort="370" velocity="2.0" lower="-6.2831853" upper="6.2831853"/>
-      <safety_controller k_position="20" k_velocity="50" soft_lower_limit="${-6.2831853 + 0.01}" soft_upper_limit="${6.2831853 - 0.01}" />
+      <!--safety_controller k_position="20" k_velocity="50" soft_lower_limit="${-6.2831853 + 0.01}" soft_upper_limit="${6.2831853 - 0.01}" /-->
     </joint>
     <link name="${name}_1_link">
+      <xacro:default_inertial/>
+<!--
       <inertial>
         <origin xyz="0 0 0" rpy="0 0 0" />
@@ -47,4 +51,5 @@
         <inertia ixx="0.01" ixy="0" ixz="0" iyy="0.01" iyz="0" izz="0.01" />
       </inertial>
+-->
       <visual>
         <origin xyz="0 0 0" rpy="0 0 0" />
@@ -68,9 +73,10 @@
       <axis xyz="0 0 1"/>
       <calibration rising="${arm_2_ref}"/>
-      <dynamics damping="10" />
       <limit effort="370" velocity="2.0" lower="-2.0943951" upper="2.0943951"/>
-      <safety_controller k_position="20" k_velocity="50" soft_lower_limit="${-2.0943 + 0.01}" soft_upper_limit="${2.0943 - 0.01}" />
+      <!--safety_controller k_position="20" k_velocity="50" soft_lower_limit="${-2.0943 + 0.01}" soft_upper_limit="${2.0943 - 0.01}" /-->
     </joint>
     <link name="${name}_2_link">
+      <xacro:default_inertial/>
+<!--
       <inertial>
         <origin xyz="0 0 0" rpy="0 0 0"/>
@@ -78,4 +84,5 @@
         <inertia ixx="0.03" ixy="0" ixz="0" iyy="0.03" iyz="0" izz="0.03" />
       </inertial>
+-->
       <visual>
         <origin xyz="0 0 0" rpy="0 0 0" />
@@ -99,9 +106,10 @@
       <axis xyz="0 0 1"/>
       <calibration rising="${arm_3_ref}"/>
-      <dynamics damping="5" />
       <limit effort="176" velocity="2.0" lower="-6.2831853" upper="6.2831853"/>
-      <safety_controller k_position="20" k_velocity="25" soft_lower_limit="${-6.2831853 + 0.01}" soft_upper_limit="${6.2831853 - 0.01}" />
+      <!--safety_controller k_position="20" k_velocity="25" soft_lower_limit="${-6.2831853 + 0.01}" soft_upper_limit="${6.2831853 - 0.01}" /-->
     </joint>
     <link name="${name}_3_link">
+      <xacro:default_inertial/>
+<!--
       <inertial>
         <origin xyz="0 0 0" rpy="0 0 0"/>
@@ -109,4 +117,5 @@
         <inertia ixx="0.03" ixy="0" ixz="0" iyy="0.03" iyz="0" izz="0.03" />
       </inertial>
+-->
       <visual>
         <origin xyz="0 0 0" rpy="0 0 0" />
@@ -130,9 +139,10 @@
       <axis xyz="0 0 1" />
       <calibration rising="${arm_4_ref}"/>
-      <dynamics damping="5" />
       <limit effort="176" velocity="2.0" lower="-2.0943951" upper="2.0943951"/>
-      <safety_controller k_position="20" k_velocity="25" soft_lower_limit="${-2.0943951 + 0.01}" soft_upper_limit="${2.0943951 - 0.01}" />
+      <!--safety_controller k_position="20" k_velocity="25" soft_lower_limit="${-2.0943951 + 0.01}" soft_upper_limit="${2.0943951 - 0.01}" /-->
     </joint>
     <link name="${name}_4_link">
+      <xacro:default_inertial/>
+<!--
       <inertial>
         <origin xyz="0 0 0" rpy="0 0 0"/>
@@ -140,4 +150,5 @@
         <inertia ixx="0.03" ixy="0" ixz="0" iyy="0.03" iyz="0" izz="0.03" />
       </inertial>
+-->
       <visual>
         <origin xyz="0 0 0" rpy="0 0 0" />
@@ -161,9 +172,10 @@
       <axis xyz="0 0 1" />
       <calibration rising="${arm_5_ref}"/>
-      <dynamics damping="5" />
       <limit effort="41.6" velocity="2.0" lower="-6.2831853" upper="6.2831853" />
-      <safety_controller k_position="20" k_velocity="25" soft_lower_limit="${-6.2831853 + 0.01}" soft_upper_limit="${6.2831853 - 0.01}" />
+      <!--safety_controller k_position="20" k_velocity="25" soft_lower_limit="${-6.2831853 + 0.01}" soft_upper_limit="${6.2831853 - 0.01}" /-->
     </joint>
     <link name="${name}_5_link">
+      <xacro:default_inertial/>
+<!--
       <inertial>
         <origin xyz="0 0 0" rpy="0 0 0"/>
@@ -171,4 +183,5 @@
         <inertia ixx="0.03" ixy="0" ixz="0" iyy="0.03" iyz="0" izz="0.03" />
       </inertial>
+-->
       <visual>
         <origin xyz="0 0 0" rpy="0 0 0" />
@@ -192,9 +205,10 @@
       <axis xyz="0 0 1" />
       <calibration rising="${arm_6_ref}"/>
-      <dynamics damping="5" />
       <limit effort="20.1" velocity="2.0" lower="-2.0943951" upper="2.0943951" />
-      <safety_controller k_position="20" k_velocity="25" soft_lower_limit="${-2.0943951 + 0.01}" soft_upper_limit="${2.0943951 - 0.01}" />
+      <!--safety_controller k_position="20" k_velocity="25" soft_lower_limit="${-2.0943951 + 0.01}" soft_upper_limit="${2.0943951 - 0.01}" /-->
     </joint>
     <link name="${name}_6_link">
+      <xacro:default_inertial/>
+<!--
       <inertial>
         <origin xyz="0 0 0" rpy="0 0 0"/>
@@ -202,4 +216,5 @@
         <inertia ixx="0.01" ixy="0" ixz="0" iyy="0.01" iyz="0" izz="0.01" />
       </inertial>
+-->
       <visual>
         <origin xyz="0 0 0" rpy="0 0 0" />

Commit message: unify all schunk urdfs

File: schunk_description/urdf/lwa4p/lwa4p.urdf.xacro (robot description, xacro)
@@ -3,10 +3,10 @@
   <xacro:include filename="$(find schunk_description)/urdf/lwa4p/lwa4p.gazebo.xacro" />
   <xacro:include filename="$(find schunk_description)/urdf/lwa4p/lwa4p.transmission.xacro" />
-  <xacro:macro name="schunk_lwa4p" params="parent name *origin">
+  <xacro:macro name="schunk_lwa4p" params="parent name *origin arm_1_ref arm_2_ref arm_3_ref arm_4_ref arm_5_ref arm_6_ref">
     <!-- joint between base_link and arm_0_link -->
-    <joint name="${name}_0_joint" type="fixed" >
+    <joint name="${name}_0_joint" type="fixed">
       <insert_block name="origin" />
-      <parent link="${parent}" />
-      <child link="${name}_0_link" />
+      <parent link="${parent}"/>
+      <child link="${name}_0_link"/>
     </joint>
     <link name="${name}_0_link">
