Commit message: new without_base descriptions

File: schunk_description/urdf/lwa4p/lwa4p.urdf.xacro (robot description, xacro)
@@ -1,14 +1,13 @@
 <?xml version="1.0"?>
 <robot xmlns:xacro="http://www.ros.org/wiki/xacro">
-  <xacro:include filename="$(find schunk_description)/urdf/lwa4p/lwa4p.gazebo.xacro" />
-  <xacro:include filename="$(find schunk_description)/urdf/lwa4p/lwa4p.transmission.xacro" />
+  <xacro:include filename="$(find schunk_description)/urdf/lwa4p/lwa4p_without_base.urdf.xacro" />
   <xacro:macro name="schunk_lwa4p" params="parent name *origin arm_1_ref arm_2_ref arm_3_ref arm_4_ref arm_5_ref arm_6_ref">
-    <!-- joint between base_link and arm_0_link -->
-    <joint name="${name}_0_joint" type="fixed">
+    <!-- joint between base_link and arm_base_link -->
+    <joint name="${name}_base_joint" type="fixed">
       <insert_block name="origin" />
       <parent link="${parent}"/>
-      <child link="${name}_0_link"/>
+      <child link="${name}_base_link"/>
     </joint>
-    <link name="${name}_0_link">
+    <link name="${name}_base_link">
       <xacro:default_inertial/>
 <!--
@@ -22,5 +21,5 @@
         <origin xyz="0 0 0" rpy="0 0 0" />
         <geometry>
-          <mesh filename="package://schunk_description/meshes/lwa4p/arm_0_link.stl" />
+          <mesh filename="package://schunk_description/meshes/lwa4p/arm_base_link.stl" />
         </geometry>
         <material name="Schunk/LightGrey" />
@@ -29,209 +28,17 @@
         <origin xyz="0 0 0" rpy="0 0 0" />
         <geometry>
-          <mesh filename="package://schunk_description/meshes/lwa4p/arm_0_link.stl" />
+          <mesh filename="package://schunk_description/meshes/lwa4p/arm_base_link.stl" />
         </geometry>
       </collision>
     </link>
-    <!-- joint between arm_0_link and arm_1_link -->
-    <joint name="${name}_1_joint" type="revolute">
-      <origin xyz="0 0 0.11" rpy="0 0 0"/>
-      <parent link="${name}_0_link"/>
-      <child link="${name}_1_link"/>
-      <axis xyz="0 0 1"/>
-      <calibration rising="${arm_1_ref}"/>
-      <limit effort="370" velocity="2.0" lower="-6.2831853" upper="6.2831853"/>
-      <!--safety_controller k_position="20" k_velocity="50" soft_lower_limit="${-6.2831853 + 0.01}" soft_upper_limit="${6.2831853 - 0.01}" /-->
-    </joint>
-    <link name="${name}_1_link">
-      <xacro:default_inertial/>
-<!--
-      <inertial>
-        <origin xyz="0 0 0" rpy="0 0 0" />
-        <mass value="0.29364"/>
-        <inertia ixx="0.01" ixy="0" ixz="0" iyy="0.01" iyz="0" izz="0.01" />
-      </inertial>
--->
-      <visual>
-        <origin xyz="0 0 0" rpy="0 0 0" />
-        <geometry>
-          <mesh filename="package://schunk_description/meshes/lwa4p/arm_1_link.stl" />
-        </geometry>
-        <material name="Schunk/Blue" />
-      </visual>
-      <collision>
-        <origin xyz="0 0 0" rpy="0 0 0" />
-        <geometry>
-          <mesh filename="package://schunk_description/meshes/lwa4p/arm_1_link.stl" />
-        </geometry>
-      </collision>
-    </link>
-    <!-- joint between arm_1_link and arm_2_link -->
-    <joint name="${name}_2_joint" type="revolute">
-      <origin xyz="0 0 0" rpy="1.5708 0 0"/>
-      <parent link="${name}_1_link"/>
-      <child link="${name}_2_link"/>
-      <axis xyz="0 0 1"/>
-      <calibration rising="${arm_2_ref}"/>
-      <limit effort="370" velocity="2.0" lower="-2.0943951" upper="2.0943951"/>
-      <!--safety_controller k_position="20" k_velocity="50" soft_lower_limit="${-2.0943 + 0.01}" soft_upper_limit="${2.0943 - 0.01}" /-->
-    </joint>
-    <link name="${name}_2_link">
-      <xacro:default_inertial/>
-<!--
-      <inertial>
-        <origin xyz="0 0 0" rpy="0 0 0"/>
-        <mass value="1.68311"/>
-        <inertia ixx="0.03" ixy="0" ixz="0" iyy="0.03" iyz="0" izz="0.03" />
-      </inertial>
--->
-      <visual>
-        <origin xyz="0 0 0" rpy="0 0 0" />
-        <geometry>
-          <mesh filename="package://schunk_description/meshes/lwa4p/arm_2_link.stl" />
-        </geometry>
-        <material name="Schunk/LightGrey" />
-      </visual>
-      <collision>
-        <origin xyz="0 0 0" rpy="0 0 0" />
-        <geometry>
-          <mesh filename="package://schunk_description/meshes/lwa4p/arm_2_link.stl" />
-        </geometry>
-      </collision>
-    </link>
-    <!-- joint between arm_2_link and arm_3_link -->
-    <joint name="${name}_3_joint" type="revolute">
-      <origin xyz="0 0.350 0" rpy="0 3.14159 0"/>
-      <parent link="${name}_2_link"/>
-      <child link="${name}_3_link"/>
-      <axis xyz="0 0 1"/>
-      <calibration rising="${arm_3_ref}"/>
-      <limit effort="176" velocity="2.0" lower="-6.2831853" upper="6.2831853"/>
-      <!--safety_controller k_position="20" k_velocity="25" soft_lower_limit="${-6.2831853 + 0.01}" soft_upper_limit="${6.2831853 - 0.01}" /-->
-    </joint>
-    <link name="${name}_3_link">
-      <xacro:default_inertial/>
-<!--
-      <inertial>
-        <origin xyz="0 0 0" rpy="0 0 0"/>
-        <mass value="2.1"/>
-        <inertia ixx="0.03" ixy="0" ixz="0" iyy="0.03" iyz="0" izz="0.03" />
-      </inertial>
--->
-      <visual>
-        <origin xyz="0 0 0" rpy="0 0 0" />
-        <geometry>
-          <mesh filename="package://schunk_description/meshes/lwa4p/arm_3_link.stl" />
-        </geometry>
-        <material name="Schunk/Blue" />
-      </visual>
-      <collision>
-        <origin xyz="0 0 0" rpy="0 0 0" />
-        <geometry>
-          <mesh filename="package://schunk_description/meshes/lwa4p/arm_3_link.stl" />
-        </geometry>
-      </collision>
-    </link>
-    <!-- joint between arm_3_link and arm_4_link -->
-    <joint name="${name}_4_joint" type="revolute">
-      <origin xyz="0 0 0" rpy="-1.5708 3.14159 0" />
-      <parent link="${name}_3_link"/>
-      <child link="${name}_4_link"/>
-      <axis xyz="0 0 1" />
-      <calibration rising="${arm_4_ref}"/>
-      <limit effort="176" velocity="2.0" lower="-2.0943951" upper="2.0943951"/>
-      <!--safety_controller k_position="20" k_velocity="25" soft_lower_limit="${-2.0943951 + 0.01}" soft_upper_limit="${2.0943951 - 0.01}" /-->
-    </joint>
-    <link name="${name}_4_link">
-      <xacro:default_inertial/>
-<!--
-      <inertial>
-        <origin xyz="0 0 0" rpy="0 0 0"/>
-        <mass value="1.68311"/>
-        <inertia ixx="0.03" ixy="0" ixz="0" iyy="0.03" iyz="0" izz="0.03" />
-      </inertial>
--->
-      <visual>
-        <origin xyz="0 0 0" rpy="0 0 0" />
-        <geometry>
-          <mesh filename="package://schunk_description/meshes/lwa4p/arm_4_link.stl" />
-        </geometry>
-        <material name="Schunk/LightGrey" />
-      </visual>
-      <collision>
-        <origin xyz="0 0 0" rpy="0 0 0" />
-        <geometry>
-          <mesh filename="package://schunk_description/meshes/lwa4p/arm_4_link.stl" />
-        </geometry>
-      </collision>
-    </link>
-    <!-- joint between arm_4_link and arm_5_link -->
-    <joint name="${name}_5_joint" type="revolute">
-      <origin xyz="0 0.005263 0.305" rpy="1.5708 0 3.14159" />
-      <parent link="${name}_4_link"/>
-      <child link="${name}_5_link"/>
-      <axis xyz="0 0 1" />
-      <calibration rising="${arm_5_ref}"/>
-      <limit effort="41.6" velocity="2.0" lower="-6.2831853" upper="6.2831853" />
-      <!--safety_controller k_position="20" k_velocity="25" soft_lower_limit="${-6.2831853 + 0.01}" soft_upper_limit="${6.2831853 - 0.01}" /-->
-    </joint>
-    <link name="${name}_5_link">
-      <xacro:default_inertial/>
-<!--
-      <inertial>
-        <origin xyz="0 0 0" rpy="0 0 0"/>
-        <mass value="0.807"/>
-        <inertia ixx="0.03" ixy="0" ixz="0" iyy="0.03" iyz="0" izz="0.03" />
-      </inertial>
--->
-      <visual>
-        <origin xyz="0 0 0" rpy="0 0 0" />
-        <geometry>
-          <mesh filename="package://schunk_description/meshes/lwa4p/arm_5_link.stl" />
-        </geometry>
-        <material name="Schunk/Blue" />
-      </visual>
-      <collision>
-        <origin xyz="0 0 0" rpy="0 0 0" />
-        <geometry>
-          <mesh filename="package://schunk_description/meshes/lwa4p/arm_5_link.stl" />
-        </geometry>
-      </collision>
-    </link>
-    <!-- joint between arm_5_link and arm_6_link -->
-    <joint name="${name}_6_joint" type="revolute">
-      <origin xyz="0 0 0" rpy="-1.5708 0 0" />
-      <parent link="${name}_5_link"/>
-      <child link="${name}_6_link"/>
-      <axis xyz="0 0 1" />
-      <calibration rising="${arm_6_ref}"/>
-      <limit effort="20.1" velocity="2.0" lower="-2.0943951" upper="2.0943951" />
-      <!--safety_controller k_position="20" k_velocity="25" soft_lower_limit="${-2.0943951 + 0.01}" soft_upper_limit="${2.0943951 - 0.01}" /-->
-    </joint>
-    <link name="${name}_6_link">
-      <xacro:default_inertial/>
-<!--
-      <inertial>
-        <origin xyz="0 0 0" rpy="0 0 0"/>
-        <mass value="0.819"/>
-        <inertia ixx="0.01" ixy="0" ixz="0" iyy="0.01" iyz="0" izz="0.01" />
-      </inertial>
--->
-      <visual>
-        <origin xyz="0 0 0" rpy="0 0 0" />
-        <geometry>
-          <mesh filename="package://schunk_description/meshes/lwa4p/arm_6_link.stl" />
-        </geometry>
-        <material name="Schunk/LightGrey" />
-      </visual>
-      <collision>
-        <origin xyz="0 0 0" rpy="0 0 0" />
-        <geometry>
-          <mesh filename="package://schunk_description/meshes/lwa4p/arm_6_link.stl" />
-        </geometry>
-      </collision>
-    </link>
-    <!-- extensions -->
-    <xacro:schunk_lwa4p_gazebo name="${name}" />
-    <xacro:schunk_lwa4p_transmission name="${name}" />
+  <xacro:schunk_lwa4p_without_base name="${name}" parent="${name}_base_link"
+          arm_1_ref="${arm_1_ref}"
+          arm_2_ref="${arm_2_ref}"
+          arm_3_ref="${arm_3_ref}"
+          arm_4_ref="${arm_4_ref}"
+          arm_5_ref="${arm_5_ref}"
+          arm_6_ref="${arm_6_ref}">
+    <origin xyz="0 0 0.11" rpy="0 0 0" />
+  </xacro:schunk_lwa4p_without_base>
   </xacro:macro>
 </robot>

File: schunk_description/urdf/lwa4p_extended/lwa4p_extended.urdf.xacro (robot description, xacro)
@@ -1,6 +1,5 @@
 <?xml version="1.0"?>
 <robot xmlns:xacro="http://www.ros.org/wiki/xacro">
-  <xacro:include filename="$(find schunk_description)/urdf/lwa4p_extended/lwa4p_extended.gazebo.xacro" />
-  <xacro:include filename="$(find schunk_description)/urdf/lwa4p_extended/lwa4p_extended.transmission.xacro" />
+  <xacro:include filename="$(find schunk_description)/urdf/lwa4p_extended/lwa4p_extended_without_base.urdf.xacro" />
   <xacro:macro name="schunk_lwa4p_extended" params="parent name *origin arm_1_ref arm_2_ref arm_3_ref arm_4_ref arm_5_ref arm_6_ref arm_7_ref">
     <!-- joint between base_link and lwa4p_extended_connector_link -->
@@ -31,238 +30,14 @@
       </collision>
     </link>
-    <!-- joint between arm_base_link and arm_1_link -->
-    <joint name="${name}_1_joint" type="revolute">
-      <origin xyz="0 0 ${0.134+0.005}" rpy="0 0 0" />
-      <parent link="${name}_base_link" />
-      <child link="${name}_1_link" />
-      <axis xyz="0 0 1"/>
-      <calibration rising="${arm_1_ref}"/>
-      <dynamics damping="0" friction="0"/>
-      <limit effort="81.5" velocity="0.42" lower="-4.712" upper="4.712"/>   <!--Theoricarl limit +/-270 , Real Limit +/- 270-->
-      <!--safety_controller k_position="20" k_velocity="50" soft_lower_limit="${-M_PI + 0.01}" soft_upper_limit="${M_PI - 0.01}" /-->
-    </joint>
-    <!-- prl100 rotor + shoulder flansh -->
-    <link name="${name}_1_link">
-      <xacro:default_inertial/>
-<!--
-      <inertial>
-        <origin xyz="0.0 0.0662 0.0473" rpy="0 0 0"/>
-        <mass value="0.8"/>
-        <inertia ixx="0.002034" ixy="0.0" ixz="0.0" iyy="0.001437" iyz="0.000784" izz="0.00161" />
-      </inertial>
--->
-      <visual>
-        <origin xyz="0 0 0" rpy="0 0 0" />
-        <geometry>
-          <mesh filename="package://schunk_description/meshes/lwa4p_extended/arm_1_link.dae" />
-        </geometry>
-      </visual>
-      <collision>
-        <origin xyz="0 0 0" rpy="0 0 0" />
-        <geometry>
-          <mesh filename="package://schunk_description/meshes/lwa4p_extended/arm_1_collision.stl" />
-        </geometry>
-      </collision>
-    </link>
-    <!-- joint between arm_1_link and arm_2_link -->
-    <joint name="${name}_2_joint" type="revolute">
-      <origin xyz="0 0 0.0915" rpy="1.5708 0 0"/>
-      <parent link="${name}_1_link"/>
-      <child link="${name}_2_link"/>
-      <axis xyz="0 0 1"/>
-      <calibration rising="${arm_2_ref}"/>
-      <dynamics damping="0" friction="0"/>
-      <limit effort="48" velocity="1.2566" lower="-1.92" upper="1.92"/>   <!--Theoricarl limit +/-170 , Real Limit +/- 110 (self collision)-->
-      <!--safety_controller k_position="20" k_velocity="50" soft_lower_limit="${-2.0943 + 0.01}" soft_upper_limit="${2.0943 - 0.01}" /-->
-    </joint>
-    <link name="${name}_2_link">
-      <xacro:default_inertial/>
-<!--
-      <inertial>
-        <origin xyz="0 0.018 -0.018" rpy="0 0 0"/>
-        <mass value="3.9"/>
-        <inertia ixx="0.009780" ixy="0.0" ixz="0.0" iyy="0.013300" iyz="0.0" izz="0.009780" />
-      </inertial>
--->
-      <visual>
-        <origin xyz="0 0 0" rpy="0 0 0" />
-        <geometry>
-          <mesh filename="package://schunk_description/meshes/lwa4p_extended/arm_2_link.dae" />
-        </geometry>
-      </visual>
-      <collision>
-        <origin xyz="0 0 0" rpy="0 0 0" />
-        <geometry>
-          <mesh filename="package://schunk_description/meshes/lwa4p_extended/arm_2_collision.stl" />
-        </geometry>
-      </collision>
-    </link>
-    <!-- joint between arm_2_link and arm_3_link -->
-    <joint name="${name}_3_joint" type="revolute">
-      <origin xyz="0 0 0" rpy="-1.5708 0 0"/>
-      <parent link="${name}_2_link"/>
-      <child link="${name}_3_link"/>
-      <axis xyz="0 0 1"/>
-      <calibration rising="${arm_3_ref}"/>
-      <dynamics damping="0" friction="0"/>
-      <limit effort="48" velocity="1.2566" lower="-2.967" upper="2.967"/>   <!--Theoricarl limit +/-170 , Real Limit +/- 170-->
-      <!--safety_controller k_position="20" k_velocity="25" soft_lower_limit="${-M_PI + 0.01}" soft_upper_limit="${M_PI - 0.01}" /-->
-    </joint>
-    <link name="${name}_3_link">
-      <xacro:default_inertial/>
-<!--
-      <inertial>
-        <origin xyz="0.0 0.06247 0.23425" rpy="0 0 0"/>
-        <mass value="1.94533"/>
-        <inertia ixx="0.0344" ixy="0.0" ixz="0.0077" iyy="0.0362" iyz="0.0" izz="0.0052" />
-      </inertial>
--->
-      <visual>
-        <origin xyz="0 0 0" rpy="0 0 0" />
-        <geometry>
-          <mesh filename="package://schunk_description/meshes/lwa4p_extended/arm_3_link.dae" />
-        </geometry>
-      </visual>
-      <collision>
-        <origin xyz="0 0 0" rpy="0 0 0" />
-        <geometry>
-          <mesh filename="package://schunk_description/meshes/lwa4p_extended/arm_3_collision.stl" />
-        </geometry>
-      </collision>
-    </link>
-    <!-- joint between arm_3_link and arm_4_link -->
-    <joint name="${name}_4_joint" type="revolute">
-      <origin xyz="0 0 0.45360" rpy="1.5708 0 0" />
-      <parent link="${name}_3_link"/>
-      <child link="${name}_4_link"/>
-      <axis xyz="0 0 1" />
-      <calibration rising="${arm_4_ref}"/>
-      <dynamics damping="0" friction="0"/>
-      <limit effort="48" velocity="1.2566" lower="-2.618" upper="2.618"/>   <!--Theoricarl limit +/-170 , Real Limit +/- 150 (self collision)-->
-      <!--safety_controller k_position="20" k_velocity="25" soft_lower_limit="${-2.0943951 + 0.01}" soft_upper_limit="${2.0943951 - 0.01}" /-->
-    </joint>
-    <link name="${name}_4_link">
-      <xacro:default_inertial/>
-<!--
-      <inertial>
-        <origin xyz="0 0.018 -0.018" rpy="0 0 0"/>
-        <mass value="3.9"/>
-        <inertia ixx="0.009780" ixy="0.0" ixz="0.0" iyy="0.013300" iyz="0.0" izz="0.009780" />
-      </inertial>
--->
-      <visual>
-        <origin xyz="0 0 0" rpy="0 0 0" />
-        <geometry>
-          <mesh filename="package://schunk_description/meshes/lwa4p_extended/arm_4_link.dae" />
-        </geometry>
-      </visual>
-      <collision>
-        <origin xyz="0 0 0" rpy="0 0 0" />
-        <geometry>
-          <mesh filename="package://schunk_description/meshes/lwa4p_extended/arm_4_collision.stl" />
-        </geometry>
-      </collision>
-    </link>
-    <!-- joint between arm_4_link and arm_5_link -->
-    <joint name="${name}_5_joint" type="revolute">
-      <origin xyz="0 0 0" rpy="-1.5708 0 0" />
-      <parent link="${name}_4_link"/>
-      <child link="${name}_5_link"/>
-      <axis xyz="0 0 1" />
-      <calibration rising="${arm_5_ref}"/>
-      <dynamics damping="0" friction="0"/>
-      <limit effort="48" velocity="1.2566" lower="-2.967" upper="2.967"/>   <!--Theoricarl limit +/-170 , Real Limit +/- 170-->
-      <!--safety_controller k_position="20" k_velocity="25" soft_lower_limit="${-M_PI + 0.01}" soft_upper_limit="${M_PI - 0.01}" /-->
-    </joint>
-    <link name="${name}_5_link">
-      <xacro:default_inertial/>
-<!--
-      <inertial>
-        <origin xyz="0.0 0.04175 0.17026" rpy="0 0 0"/>
-        <mass value="1.3297"/>
-        <inertia ixx="0.01" ixy="0.0" ixz="-0.0031" iyy="0.0111" iyz="0.0" izz="0.0031" />
-      </inertial>
--->
-      <visual>
-        <origin xyz="0 0 0" rpy="0 0 0" />
-        <geometry>
-          <mesh filename="package://schunk_description/meshes/lwa4p_extended/arm_5_link.dae" />
-        </geometry>
-      </visual>
-      <collision>
-        <origin xyz="0 0 0" rpy="0 0 0" />
-        <geometry>
-          <mesh filename="package://schunk_description/meshes/lwa4p_extended/arm_5_collision.stl" />
-        </geometry>
-      </collision>
-    </link>
-    <!-- joint between arm_5_link and arm_6_link -->
-    <joint name="${name}_6_joint" type="revolute">
-      <origin xyz="0 0 0.2986" rpy="1.5708 0 0" />
-      <parent link="${name}_5_link"/>
-      <child link="${name}_6_link"/>
-      <axis xyz="0 0 1" />
-      <calibration rising="${arm_6_ref}"/>
-      <dynamics damping="0" friction="0"/>
-      <limit effort="15" velocity="1.2566" lower="-2.443" upper="2.967"/>   <!--Theoricarl limit +/-170 , Real Limit -140/+170 (self collision)-->
-      <!--safety_controller k_position="20" k_velocity="25" soft_lower_limit="${-2.0943951 + 0.01}" soft_upper_limit="${2.0943951 - 0.01}" /-->
-    </joint>
-    <link name="${name}_6_link">
-      <xacro:default_inertial/>
-<!--
-      <inertial>
-        <origin xyz="0 0.012 -0.012" rpy="0 0 0"/>
-        <mass value="1.9"/>
-        <inertia ixx="0.002750" ixy="0.0" ixz="0.0" iyy="0.004002" iyz="0.0" izz="0.002830" />
-      </inertial>
--->
-      <visual>
-        <origin xyz="0 0 0" rpy="0 0 0" />
-        <geometry>
-          <mesh filename="package://schunk_description/meshes/lwa4p_extended/arm_6_link.dae" />
-        </geometry>
-      </visual>
-      <collision>
-        <origin xyz="0 0 0" rpy="0 0 0" />
-        <geometry>
-          <mesh filename="package://schunk_description/meshes/lwa4p_extended/arm_6_collision.stl" />
-        </geometry>
-      </collision>
-    </link>
-    <!-- joint between arm_6_link and arm_7_link -->
-    <joint name="${name}_7_joint" type="revolute">
-      <origin xyz="0 0 0" rpy="-1.5708 0 0" />
-      <parent link="${name}_6_link"/>
-      <child link="${name}_7_link"/>
-      <axis xyz="0 0 1" />
-      <calibration rising="${arm_7_ref}"/>
-      <dynamics damping="0" friction="0"/>
-      <limit effort="15" velocity="1.2566" lower="-2.967" upper="2.967"/>   <!--Theoricarl limit +/-170 , Real Limit +/- 170-->
-      <!--safety_controller k_position="20" k_velocity="25" soft_lower_limit="${-2.0943951 + 0.01}" soft_upper_limit="${2.0943951 - 0.01}" /-->
-    </joint>
-    <link name="${name}_7_link">
-      <xacro:default_inertial/>
-<!--
-      <xacro:cylinder_inertial radius="0.03" length="0.035" mass="0.05">
-        <origin xyz="0 0 0.06" rpy="0 0 0"/>
-      </xacro:cylinder_inertial>
--->
-      <visual>
-        <origin xyz="0 0 0.06" rpy="0 0 0"/>
-        <geometry>
-          <cylinder radius="0.03" length="0.035"/>
-        </geometry>
-        <material name="Schunk/LightGrey"/>
-      </visual>
-      <collision>
-        <origin xyz="0 0 0.06" rpy="0 0 0"/>
-        <geometry>
-          <cylinder radius="0.03" length="0.035"/>
-        </geometry>
-      </collision>
-    </link>
-    <!-- extensions -->
-    <xacro:schunk_lwa4p_extended_gazebo name="${name}" />
-    <xacro:schunk_lwa4p_extended_transmission name="${name}" />
+  <xacro:schunk_lwa4p_extended_without_base name="${name}" parent="${name}_base_link"
+          arm_1_ref="${arm_1_ref}"
+          arm_2_ref="${arm_2_ref}"
+          arm_3_ref="${arm_3_ref}"
+          arm_4_ref="${arm_4_ref}"
+          arm_5_ref="${arm_5_ref}"
+          arm_6_ref="${arm_6_ref}"
+          arm_7_ref="${arm_7_ref}">
+    <origin xyz="0 0 0.139" rpy="0 0 0" />
+  </xacro:schunk_lwa4p_extended_without_base>
   </xacro:macro>
 </robot>
