Commit message: Updated lwa4p urdf with manufacturer's specified joint limits.

File: schunk_description/urdf/lwa4p/lwa4p.urdf.xacro (robot description, xacro)
@@ -50,5 +50,5 @@
       <child link="${name}_1_link"/>
       <axis xyz="0 0 1"/>
-      <limit effort="370" velocity="2.0" lower="${-6.28 + safety_offset}" upper="${6.28 - safety_offset}"/>
+      <limit effort="370" velocity="2.0" lower="${-2.967 + safety_offset}" upper="${2.967 - safety_offset}"/>
       <!--safety_controller k_position="20" k_velocity="50" soft_lower_limit="${-6.28 + 0.01}" soft_upper_limit="${6.28 - 0.01}" /-->
     </joint>
@@ -82,5 +82,5 @@
       <child link="${name}_2_link"/>
       <axis xyz="0 0 1"/>
-      <limit effort="370" velocity="2.0" lower="${-2.09 + safety_offset}" upper="${2.09 - safety_offset}"/>
+      <limit effort="370" velocity="2.0" lower="${-2.967 + safety_offset}" upper="${2.967 - safety_offset}"/>
       <!--safety_controller k_position="20" k_velocity="50" soft_lower_limit="${-2.09 + 0.01}" soft_upper_limit="${2.09 - 0.01}" /-->
     </joint>
@@ -114,5 +114,5 @@
       <child link="${name}_3_link"/>
       <axis xyz="0 0 1"/>
-      <limit effort="176" velocity="2.0" lower="${-6.28 + safety_offset}" upper="${6.28 - safety_offset}"/>
+      <limit effort="176" velocity="2.0" lower="${-2.714 + safety_offset}" upper="${2.714 - safety_offset}"/>
       <!--safety_controller k_position="20" k_velocity="25" soft_lower_limit="${-6.28 + 0.01}" soft_upper_limit="${6.28 - 0.01}" /-->
     </joint>
@@ -146,5 +146,5 @@
       <child link="${name}_4_link"/>
       <axis xyz="0 0 1" />
-      <limit effort="176" velocity="2.0" lower="${-2.09 + safety_offset}" upper="${2.09 - safety_offset}"/>
+      <limit effort="176" velocity="2.0" lower="${-2.967 + safety_offset}" upper="${2.967 - safety_offset}"/>
       <!--safety_controller k_position="20" k_velocity="25" soft_lower_limit="${-2.09 + 0.01}" soft_upper_limit="${2.09 - 0.01}" /-->
     </joint>
@@ -178,5 +178,5 @@
       <child link="${name}_5_link"/>
       <axis xyz="0 0 1" />
-      <limit effort="41.6" velocity="2.0" lower="${-6.28 + safety_offset}" upper="${6.28 - safety_offset}" />
+      <limit effort="41.6" velocity="2.0" lower="${-2.967 + safety_offset}" upper="${2.967 - safety_offset}" />
       <!--safety_controller k_position="20" k_velocity="25" soft_lower_limit="${-6.28 + 0.01}" soft_upper_limit="${6.28 - 0.01}" /-->
     </joint>
@@ -210,5 +210,5 @@
       <child link="${name}_6_link"/>
       <axis xyz="0 0 1" />
-      <limit effort="20.1" velocity="2.0" lower="${-2.09 + safety_offset}" upper="${2.09 - safety_offset}" />
+      <limit effort="20.1" velocity="2.0" lower="${-2.967 + safety_offset}" upper="${2.967 - safety_offset}" />
       <!--safety_controller k_position="20" k_velocity="25" soft_lower_limit="${-2.09 + 0.01}" soft_upper_limit="${2.09 - 0.01}" /-->
     </joint>

Commit message: Update lwa4p.urdf.xacro with joint speed limits.

File: schunk_description/urdf/lwa4p/lwa4p.urdf.xacro (robot description, xacro)
@@ -50,5 +50,5 @@
       <child link="${name}_1_link"/>
       <axis xyz="0 0 1"/>
-      <limit effort="370" velocity="2.0" lower="${-2.967 + safety_offset}" upper="${2.967 - safety_offset}"/>
+      <limit effort="370" velocity="1.26" lower="${-2.967 + safety_offset}" upper="${2.967 - safety_offset}"/>
       <!--safety_controller k_position="20" k_velocity="50" soft_lower_limit="${-6.28 + 0.01}" soft_upper_limit="${6.28 - 0.01}" /-->
     </joint>
@@ -82,5 +82,5 @@
       <child link="${name}_2_link"/>
       <axis xyz="0 0 1"/>
-      <limit effort="370" velocity="2.0" lower="${-2.967 + safety_offset}" upper="${2.967 - safety_offset}"/>
+      <limit effort="370" velocity="1.26" lower="${-2.967 + safety_offset}" upper="${2.967 - safety_offset}"/>
       <!--safety_controller k_position="20" k_velocity="50" soft_lower_limit="${-2.09 + 0.01}" soft_upper_limit="${2.09 - 0.01}" /-->
     </joint>
@@ -114,5 +114,5 @@
       <child link="${name}_3_link"/>
       <axis xyz="0 0 1"/>
-      <limit effort="176" velocity="2.0" lower="${-2.714 + safety_offset}" upper="${2.714 - safety_offset}"/>
+      <limit effort="176" velocity="1.26" lower="${-2.714 + safety_offset}" upper="${2.714 - safety_offset}"/>
       <!--safety_controller k_position="20" k_velocity="25" soft_lower_limit="${-6.28 + 0.01}" soft_upper_limit="${6.28 - 0.01}" /-->
     </joint>
@@ -146,5 +146,5 @@
       <child link="${name}_4_link"/>
       <axis xyz="0 0 1" />
-      <limit effort="176" velocity="2.0" lower="${-2.967 + safety_offset}" upper="${2.967 - safety_offset}"/>
+      <limit effort="176" velocity="1.26" lower="${-2.967 + safety_offset}" upper="${2.967 - safety_offset}"/>
       <!--safety_controller k_position="20" k_velocity="25" soft_lower_limit="${-2.09 + 0.01}" soft_upper_limit="${2.09 - 0.01}" /-->
     </joint>
@@ -178,5 +178,5 @@
       <child link="${name}_5_link"/>
       <axis xyz="0 0 1" />
-      <limit effort="41.6" velocity="2.0" lower="${-2.967 + safety_offset}" upper="${2.967 - safety_offset}" />
+      <limit effort="41.6" velocity="1.26" lower="${-2.967 + safety_offset}" upper="${2.967 - safety_offset}" />
       <!--safety_controller k_position="20" k_velocity="25" soft_lower_limit="${-6.28 + 0.01}" soft_upper_limit="${6.28 - 0.01}" /-->
     </joint>
@@ -210,5 +210,5 @@
       <child link="${name}_6_link"/>
       <axis xyz="0 0 1" />
-      <limit effort="20.1" velocity="2.0" lower="${-2.967 + safety_offset}" upper="${2.967 - safety_offset}" />
+      <limit effort="20.1" velocity="1.26" lower="${-2.967 + safety_offset}" upper="${2.967 - safety_offset}" />
       <!--safety_controller k_position="20" k_velocity="25" soft_lower_limit="${-2.09 + 0.01}" soft_upper_limit="${2.09 - 0.01}" /-->
     </joint>

Commit message: Added new xacro file created by A. Heilig

File: schunk_description/urdf/lwa4p/lwa4p.urdf.xacro (robot description, xacro)
@@ -14,16 +14,56 @@
       <link name="${name}_podest_link">
         <xacro:default_inertial/>
-        <visual>
-          <origin xyz="0 0 0" rpy="0 ${M_PI} 0" />
-          <geometry>
-          <mesh filename="package://schunk_description/meshes/lwa4p/arm_base_link.stl" />
-          </geometry>
-        </visual>
-        <collision>
-          <origin xyz="0 0 0" rpy="0 ${M_PI} 0" />
-          <geometry>
-          <mesh filename="package://schunk_description/meshes/lwa4p/arm_base_link.stl" />
-          </geometry>
-        </collision>
+     <visual>
+          <origin xyz="0 0 0" rpy="0 0 ${-M_PI/2}" />
+      <geometry>
+        <mesh filename="package://industrial_kuka_ros/robot_description/meshes/LWA4P/A0_1.stl" scale="0.001 0.001 0.001" />
+      </geometry>
+        <material name="Schunk/LightGrey" />
+    </visual>
+    <collision>
+          <origin xyz="0 0 0" rpy="0 0 ${-M_PI/2}" />
+      <geometry>
+        <mesh filename="package://industrial_kuka_ros/robot_description/meshes/LWA4P/A0_1.stl" scale="0.001 0.001 0.001" />
+      </geometry>
+    </collision>
+    <visual>
+          <origin xyz="0 0 0" rpy="0 0 ${-M_PI/2}" />
+      <geometry>
+        <mesh filename="package://industrial_kuka_ros/robot_description/meshes/LWA4P/A0_2.stl" scale="0.001 0.001 0.001" />
+      </geometry>
+        <material name="Schunk/LightGrey" />
+    </visual>
+    <collision>
+          <origin xyz="0 0 0" rpy="0 0 ${-M_PI/2}" />
+      <geometry>
+        <mesh filename="package://industrial_kuka_ros/robot_description/meshes/LWA4P/A0_2.stl" scale="0.001 0.001 0.001" />
+      </geometry>
+    </collision>
+    <visual>
+          <origin xyz="0 0 0" rpy="0 0 ${-M_PI/2}" />
+      <geometry>
+        <mesh filename="package://industrial_kuka_ros/robot_description/meshes/LWA4P/A0_3.stl" scale="0.001 0.001 0.001" />
+      </geometry>
+        <material name="Schunk/LightGrey" />
+    </visual>
+    <collision>
+          <origin xyz="0 0 0" rpy="0 0 ${-M_PI/2}" />
+      <geometry>
+        <mesh filename="package://industrial_kuka_ros/robot_description/meshes/LWA4P/A0_3.stl" scale="0.001 0.001 0.001" />
+      </geometry>
+    </collision>
+    <visual>
+          <origin xyz="0 0 0" rpy="0 0 ${-M_PI/2}" />
+      <geometry>
+        <mesh filename="package://industrial_kuka_ros/robot_description/meshes/LWA4P/A0_4.stl" scale="0.001 0.001 0.001" />
+      </geometry>
+        <material name="Schunk/LightGrey" />
+    </visual>
+    <collision>
+          <origin xyz="0 0 0" rpy="0 0 0" />
+      <geometry>
+        <mesh filename="package://industrial_kuka_ros/robot_description/meshes/LWA4P/A0_4.stl" scale="0.001 0.001 0.001" />
+      </geometry>
+    </collision>
       </link>
       <joint name="${name}_base_joint" type="fixed">
@@ -46,5 +86,5 @@
     <!-- joint between arm_0_link and arm_1_link -->
     <joint name="${name}_1_joint" type="revolute">
-      <origin xyz="0 0 0" rpy="0 0 0" />
+      <origin xyz="0 0 0.1053" rpy="0 0 0" />
       <parent link="${name}_base_link"/>
       <child link="${name}_1_link"/>
@@ -62,21 +102,21 @@
       </inertial>
 -->
-      <visual>
-        <origin xyz="0 0 0" rpy="0 0 0" />
-        <geometry>
-          <mesh filename="package://schunk_description/meshes/lwa4p/arm_1_link.stl" />
-        </geometry>
-        <material name="Schunk/Blue" />
-      </visual>
-      <collision>
-        <origin xyz="0 0 0" rpy="0 0 0" />
-        <geometry>
-          <mesh filename="package://schunk_description/meshes/lwa4p/arm_1_link.stl" />
-        </geometry>
-      </collision>
+    <visual>
+      <origin rpy="0 0 -1.57079632679" xyz="0 0 -0.2053"/>
+      <geometry>
+        <mesh filename="package://industrial_kuka_ros/robot_description/meshes/LWA4P/A1.stl" scale="0.001 0.001 0.001" />
+      </geometry>
+       <material name="Schunk/Blue" />
+    </visual>
+    <collision>
+      <origin rpy="0 0 -1.57079632679" xyz="0 0 -0.2053"/>
+      <geometry>
+        <mesh filename="package://industrial_kuka_ros/robot_description/meshes/LWA4P/A1.stl" scale="0.001 0.001 0.001" />
+      </geometry>
+    </collision>
     </link>
     <!-- joint between arm_1_link and arm_2_link -->
     <joint name="${name}_2_joint" type="revolute">
-      <origin xyz="0 0 0" rpy="1.5708 0 0"/>
+      <origin xyz="0 0 0" rpy="${-M_PI/2} 0 0"/>
       <parent link="${name}_1_link"/>
       <child link="${name}_2_link"/>
@@ -94,21 +134,47 @@
       </inertial>
 -->
-      <visual>
-        <origin xyz="0 0 0" rpy="0 0 0" />
-        <geometry>
-          <mesh filename="package://schunk_description/meshes/lwa4p/arm_2_link.stl" />
-        </geometry>
-        <material name="Schunk/LightGrey" />
-      </visual>
-      <collision>
-        <origin xyz="0 0 0" rpy="0 0 0" />
-        <geometry>
-          <mesh filename="package://schunk_description/meshes/lwa4p/arm_2_link.stl" />
-        </geometry>
-      </collision>
+    <visual>
+      <origin rpy="0 1.57079632679 0" xyz="-0.2053 0 0"/>
+      <geometry>
+        <mesh filename="package://industrial_kuka_ros/robot_description/meshes/LWA4P/A2_1.stl" scale="0.001 0.001 0.001" />
+      </geometry>
+        <material name="Schunk/LightGrey" />
+    </visual>
+    <collision>
+      <origin rpy="0 1.57079632679 0" xyz="-0.2053 0 0"/>
+     <geometry>
+        <mesh filename="package://industrial_kuka_ros/robot_description/meshes/LWA4P/A2_1.stl" scale="0.001 0.001 0.001" />
+      </geometry>
+    </collision>
+    <visual>
+      <origin rpy="1.57079632679 1.57079632679 0" xyz="0 0.2053 0"/>
+      <geometry>
+        <mesh filename="package://industrial_kuka_ros/robot_description/meshes/LWA4P/A2_2.stl" scale="0.001 0.001 0.001" />
+      </geometry>
+        <material name="Schunk/LightGrey" />
+    </visual>
+    <collision>
+      <origin rpy="1.57079632679 1.57079632679 0" xyz="0 0.2053 0"/>
+     <geometry>
+        <mesh filename="package://industrial_kuka_ros/robot_description/meshes/LWA4P/A2_2.stl" scale="0.001 0.001 0.001" />
+      </geometry>
+    </collision>
+    <visual>
+      <origin rpy="1.57079632679 1.57079632679 0" xyz="0 0.2053 0"/>
+      <geometry>
+        <mesh filename="package://industrial_kuka_ros/robot_description/meshes/LWA4P/A2_3.stl" scale="0.001 0.001 0.001" />
+      </geometry>
+        <material name="Schunk/LightGrey" />
+    </visual>
+    <collision>
+      <origin rpy="1.57079632679 1.57079632679 0" xyz="0 0.2053 0"/>
+     <geometry>
+        <mesh filename="package://industrial_kuka_ros/robot_description/meshes/LWA4P/A2_3.stl" scale="0.001 0.001 0.001" />
+      </geometry>
+    </collision>
     </link>
     <!-- joint between arm_2_link and arm_3_link -->
     <joint name="${name}_3_joint" type="revolute">
-      <origin xyz="0 0.350 0" rpy="0 3.14159 0"/>
+      <origin xyz="0 -0.350 0" rpy="0 0 0"/>
       <parent link="${name}_2_link"/>
       <child link="${name}_3_link"/>
@@ -126,21 +192,21 @@
       </inertial>
 -->
-      <visual>
-        <origin xyz="0 0 0" rpy="0 0 0" />
-        <geometry>
-          <mesh filename="package://schunk_description/meshes/lwa4p/arm_3_link.stl" />
-        </geometry>
+    <visual>
+       <origin rpy="0 1.57079632679 -1.57079632679" xyz="0 0.5553 0 "/>
+      <geometry>
+        <mesh filename="package://industrial_kuka_ros/robot_description/meshes/LWA4P/A3.stl" scale="0.001 0.001 0.001" />
+      </geometry>
         <material name="Schunk/Blue" />
-      </visual>
-      <collision>
-        <origin xyz="0 0 0" rpy="0 0 0" />
-        <geometry>
-          <mesh filename="package://schunk_description/meshes/lwa4p/arm_3_link.stl" />
-        </geometry>
-      </collision>
+    </visual>
+    <collision>
+       <origin rpy="0 1.57079632679 -1.57079632679" xyz="0 0.5553 0 "/>
+      <geometry>
+        <mesh filename="package://industrial_kuka_ros/robot_description/meshes/LWA4P/A3.stl" scale="0.001 0.001 0.001" />
+      </geometry>
+    </collision>
     </link>
     <!-- joint between arm_3_link and arm_4_link -->
     <joint name="${name}_4_joint" type="revolute">
-      <origin xyz="0 0 0" rpy="-1.5708 3.14159 0" />
+      <origin xyz="0 0 0" rpy="${-M_PI/2} 0 0" />
       <parent link="${name}_3_link"/>
       <child link="${name}_4_link"/>
@@ -158,21 +224,47 @@
       </inertial>
 -->
-      <visual>
-        <origin xyz="0 0 0" rpy="0 0 0" />
-        <geometry>
-          <mesh filename="package://schunk_description/meshes/lwa4p/arm_4_link.stl" />
-        </geometry>
-        <material name="Schunk/LightGrey" />
-      </visual>
-      <collision>
-        <origin xyz="0 0 0" rpy="0 0 0" />
-        <geometry>
-          <mesh filename="package://schunk_description/meshes/lwa4p/arm_4_link.stl" />
-        </geometry>
-      </collision>
+    <visual>
+      <origin rpy="0 3.14159265359 0" xyz="0 0 0.5553"/>
+      <geometry>
+        <mesh filename="package://industrial_kuka_ros/robot_description/meshes/LWA4P/A4_1.stl" scale="0.001 0.001 0.001" />
+      </geometry>
+        <material name="Schunk/LightGrey" />
+    </visual>
+    <collision>
+      <origin rpy="0 3.14159265359 0" xyz="0 0 0.5553"/>
+      <geometry>
+        <mesh filename="package://industrial_kuka_ros/robot_description/meshes/LWA4P/A4_1.stl" scale="0.001 0.001 0.001" />
+      </geometry>
+    </collision>
+    <visual>
+      <origin rpy="0 3.14159265359 -1.57079632679" xyz="0 0 0.5553"/>
+      <geometry>
+        <mesh filename="package://industrial_kuka_ros/robot_description/meshes/LWA4P/A4_2.stl" scale="0.001 0.001 0.001" />
+      </geometry>
+        <material name="Schunk/LightGrey" />
+    </visual>
+    <collision>
+      <origin rpy="0 3.14159265359 -1.57079632679" xyz="0 0 0"/>
+      <geometry>
+        <mesh filename="package://industrial_kuka_ros/robot_description/meshes/LWA4P/A4_2.stl" scale="0.001 0.001 0.001" />
+      </geometry>
+    </collision>
+    <visual>
+      <origin rpy="0 3.14159265359 -1.57079632679" xyz="0 0 0.5553"/>
+      <geometry>
+        <mesh filename="package://industrial_kuka_ros/robot_description/meshes/LWA4P/A4_3.stl" scale="0.001 0.001 0.001" />
+      </geometry>
+        <material name="Schunk/LightGrey" />
+    </visual>
+    <collision>
+      <origin rpy="0 3.14159265359 -1.57079632679" xyz="0 0 0.5553"/>
+      <geometry>
+        <mesh filename="package://industrial_kuka_ros/robot_description/meshes/LWA4P/A4_3.stl" scale="0.001 0.001 0.001" />
+      </geometry>
+    </collision>
     </link>
     <!-- joint between arm_4_link and arm_5_link -->
     <joint name="${name}_5_joint" type="revolute">
-      <origin xyz="0 0.005263 0.305" rpy="1.5708 0 3.14159" />
+      <origin xyz="0 0 -0.3049" rpy="${M_PI/2} 0 0" />
       <parent link="${name}_4_link"/>
       <child link="${name}_5_link"/>
@@ -190,21 +282,21 @@
       </inertial>
 -->
-      <visual>
-        <origin xyz="0 0 0" rpy="0 0 0" />
-        <geometry>
-          <mesh filename="package://schunk_description/meshes/lwa4p/arm_5_link.stl" />
-        </geometry>
+    <visual>
+       <origin rpy="0 1.57079632679 -1.57079632679" xyz="0 0.8602 0"/>
+      <geometry>
+        <mesh filename="package://industrial_kuka_ros/robot_description/meshes/LWA4P/A5.stl" scale="0.001 0.001 0.001" />
+      </geometry>
         <material name="Schunk/Blue" />
-      </visual>
-      <collision>
-        <origin xyz="0 0 0" rpy="0 0 0" />
-        <geometry>
-          <mesh filename="package://schunk_description/meshes/lwa4p/arm_5_link.stl" />
-        </geometry>
-      </collision>
+    </visual>
+    <collision>
+       <origin rpy="0 1.57079632679 -1.57079632679" xyz="0 0.8602 0"/>
+      <geometry>
+        <mesh filename="package://industrial_kuka_ros/robot_description/meshes/LWA4P/A5.stl" scale="0.001 0.001 0.001" />
+      </geometry>
+    </collision>
     </link>
     <!-- joint between arm_5_link and arm_6_link -->
     <joint name="${name}_6_joint" type="revolute">
-      <origin xyz="0 0 0" rpy="-1.5708 0 0" />
+      <origin xyz="0 0 0" rpy="${-M_PI/2} 0 0" />
       <parent link="${name}_5_link"/>
       <child link="${name}_6_link"/>
@@ -222,17 +314,62 @@
       </inertial>
 -->
-      <visual>
-        <origin xyz="0 0 0" rpy="0 0 0" />
-        <geometry>
-          <mesh filename="package://schunk_description/meshes/lwa4p/arm_6_link.stl" />
-        </geometry>
-        <material name="Schunk/LightGrey" />
-      </visual>
-      <collision>
-        <origin xyz="0 0 0" rpy="0 0 0" />
-        <geometry>
-          <mesh filename="package://schunk_description/meshes/lwa4p/arm_6_link.stl" />
-        </geometry>
-      </collision>
+    <visual>
+      <origin rpy="0 3.14159265359 0" xyz="0 0 0.8602"/>
+      <geometry>
+        <mesh filename="package://industrial_kuka_ros/robot_description/meshes/LWA4P/A6_1.stl" scale="0.001 0.001 0.001" />
+      </geometry>
+        <material name="Schunk/LightGrey" />
+    </visual>
+    <collision>
+      <origin rpy="0 3.14159265359 0" xyz="0 0 0.8602"/>
+      <geometry>
+        <mesh filename="package://industrial_kuka_ros/robot_description/meshes/LWA4P/A6_1.stl" scale="0.001 0.001 0.001" />
+      </geometry>
+    </collision>
+    <visual>
+      <origin rpy="0 3.14159265359 0" xyz="0 0 0.8602"/>
+      <geometry>
+        <mesh filename="package://industrial_kuka_ros/robot_description/meshes/LWA4P/A6_2.stl" scale="0.001 0.001 0.001" />
+      </geometry>
+        <material name="Schunk/LightGrey" />
+    </visual>
+    <collision>
+      <origin rpy="0 3.14159265359 0" xyz="0 0 0.8602"/>
+      <geometry>
+        <mesh filename="package://industrial_kuka_ros/robot_description/meshes/LWA4P/A6_2.stl" scale="0.001 0.001 0.001" />
+      </geometry>
+    </collision>
+    <visual>
+      <origin rpy="0 3.14159265359 0" xyz="0 0 0.8602"/>
+      <geometry>
+        <mesh filename="package://industrial_kuka_ros/robot_description/meshes/LWA4P/A6_3.stl" scale="0.001 0.001 0.001" />
+      </geometry>
+        <material name="Schunk/LightGrey" />
+    </visual>
+    <collision>
+      <origin rpy="0 3.14159265359 0" xyz="0 0 0.8602"/>
+      <geometry>
+        <mesh filename="package://industrial_kuka_ros/robot_description/meshes/LWA4P/A6_3.stl" scale="0.001 0.001 0.001" />
+      </geometry>
+    </collision>
+    </link>
+ <!-- flange -->
+    <joint name="${name}_7_joint" type="fixed">
+      <origin xyz="0 0 -0.0751" rpy="${M_PI} 0 0" />
+      <parent link="${name}_6_link"/>
+      <child link="${name}_7_link"/>
+      <axis xyz="0 0 1" />
+      <limit effort="20.1" velocity="1.26" lower="${-2.967 + safety_offset}" upper="${2.967 - safety_offset}" />
+      <!--safety_controller k_position="20" k_velocity="25" soft_lower_limit="${-2.09 + 0.01}" soft_upper_limit="${2.09 - 0.01}" /-->
+    </joint>
+    <link name="${name}_7_link">
+      <xacro:default_inertial/>
+<!--
+      <inertial>
+        <origin xyz="0 0 0" rpy="0 0 0"/>
+        <mass value="0.819"/>
+        <inertia ixx="0.01" ixy="0" ixz="0" iyy="0.01" iyz="0" izz="0.01" />
+      </inertial>
+-->
     </link>
     <!-- extensions -->
