Commit message: New stl files and corrected path to this files

File: schunk_description/urdf/lwa4p/lwa4p.urdf.xacro (robot description, xacro)
@@ -17,44 +17,44 @@
           <origin xyz="0 0 0" rpy="0 0 ${-M_PI/2}" />
       <geometry>
-        <mesh filename="package://industrial_kuka_ros/robot_description/meshes/LWA4P/A0_1.stl" scale="0.001 0.001 0.001" />
-      </geometry>
-        <material name="Schunk/LightGrey" />
-    </visual>
-    <collision>
-          <origin xyz="0 0 0" rpy="0 0 ${-M_PI/2}" />
-      <geometry>
-        <mesh filename="package://industrial_kuka_ros/robot_description/meshes/LWA4P/A0_1.stl" scale="0.001 0.001 0.001" />
-      </geometry>
-    </collision>
-    <visual>
-          <origin xyz="0 0 0" rpy="0 0 ${-M_PI/2}" />
-      <geometry>
-        <mesh filename="package://industrial_kuka_ros/robot_description/meshes/LWA4P/A0_2.stl" scale="0.001 0.001 0.001" />
-      </geometry>
-        <material name="Schunk/LightGrey" />
-    </visual>
-    <collision>
-          <origin xyz="0 0 0" rpy="0 0 ${-M_PI/2}" />
-      <geometry>
-        <mesh filename="package://industrial_kuka_ros/robot_description/meshes/LWA4P/A0_2.stl" scale="0.001 0.001 0.001" />
-      </geometry>
-    </collision>
-    <visual>
-          <origin xyz="0 0 0" rpy="0 0 ${-M_PI/2}" />
-      <geometry>
-        <mesh filename="package://industrial_kuka_ros/robot_description/meshes/LWA4P/A0_3.stl" scale="0.001 0.001 0.001" />
-      </geometry>
-        <material name="Schunk/LightGrey" />
-    </visual>
-    <collision>
-          <origin xyz="0 0 0" rpy="0 0 ${-M_PI/2}" />
-      <geometry>
-        <mesh filename="package://industrial_kuka_ros/robot_description/meshes/LWA4P/A0_3.stl" scale="0.001 0.001 0.001" />
-      </geometry>
-    </collision>
-    <visual>
-          <origin xyz="0 0 0" rpy="0 0 ${-M_PI/2}" />
-      <geometry>
-        <mesh filename="package://industrial_kuka_ros/robot_description/meshes/LWA4P/A0_4.stl" scale="0.001 0.001 0.001" />
+        <mesh filename="package://schunk_description/meshes/lwa4p/A0_1.stl" scale="0.001 0.001 0.001" />
+      </geometry>
+        <material name="Schunk/LightGrey" />
+    </visual>
+    <collision>
+          <origin xyz="0 0 0" rpy="0 0 ${-M_PI/2}" />
+      <geometry>
+        <mesh filename="package://schunk_description/meshes/lwa4p/A0_1.stl" scale="0.001 0.001 0.001" />
+      </geometry>
+    </collision>
+    <visual>
+          <origin xyz="0 0 0" rpy="0 0 ${-M_PI/2}" />
+      <geometry>
+        <mesh filename="package://schunk_description/meshes/lwa4p/A0_2.stl" scale="0.001 0.001 0.001" />
+      </geometry>
+        <material name="Schunk/LightGrey" />
+    </visual>
+    <collision>
+          <origin xyz="0 0 0" rpy="0 0 ${-M_PI/2}" />
+      <geometry>
+        <mesh filename="package://schunk_description/meshes/lwa4p/A0_2.stl" scale="0.001 0.001 0.001" />
+      </geometry>
+    </collision>
+    <visual>
+          <origin xyz="0 0 0" rpy="0 0 ${-M_PI/2}" />
+      <geometry>
+        <mesh filename="package://schunk_description/meshes/lwa4p/A0_3.stl" scale="0.001 0.001 0.001" />
+      </geometry>
+        <material name="Schunk/LightGrey" />
+    </visual>
+    <collision>
+          <origin xyz="0 0 0" rpy="0 0 ${-M_PI/2}" />
+      <geometry>
+        <mesh filename="package://schunk_description/meshes/lwa4p/A0_3.stl" scale="0.001 0.001 0.001" />
+      </geometry>
+    </collision>
+    <visual>
+          <origin xyz="0 0 0" rpy="0 0 ${-M_PI/2}" />
+      <geometry>
+        <mesh filename="package://schunk_description/meshes/lwa4p/A0_4.stl" scale="0.001 0.001 0.001" />
       </geometry>
         <material name="Schunk/LightGrey" />
@@ -63,5 +63,5 @@
           <origin xyz="0 0 0" rpy="0 0 0" />
       <geometry>
-        <mesh filename="package://industrial_kuka_ros/robot_description/meshes/LWA4P/A0_4.stl" scale="0.001 0.001 0.001" />
+        <mesh filename="package://schunk_description/meshes/lwa4p/A0_4.stl" scale="0.001 0.001 0.001" />
       </geometry>
     </collision>
@@ -105,5 +105,5 @@
       <origin rpy="0 0 -1.57079632679" xyz="0 0 -0.2053"/>
       <geometry>
-        <mesh filename="package://industrial_kuka_ros/robot_description/meshes/LWA4P/A1.stl" scale="0.001 0.001 0.001" />
+        <mesh filename="package://schunk_description/meshes/lwa4p/A1.stl" scale="0.001 0.001 0.001" />
       </geometry>
        <material name="Schunk/Blue" />
@@ -112,5 +112,5 @@
       <origin rpy="0 0 -1.57079632679" xyz="0 0 -0.2053"/>
       <geometry>
-        <mesh filename="package://industrial_kuka_ros/robot_description/meshes/LWA4P/A1.stl" scale="0.001 0.001 0.001" />
+        <mesh filename="package://schunk_description/meshes/lwa4p/A1.stl" scale="0.001 0.001 0.001" />
       </geometry>
     </collision>
@@ -137,5 +137,5 @@
       <origin rpy="0 1.57079632679 0" xyz="-0.2053 0 0"/>
       <geometry>
-        <mesh filename="package://industrial_kuka_ros/robot_description/meshes/LWA4P/A2_1.stl" scale="0.001 0.001 0.001" />
+        <mesh filename="package://schunk_description/meshes/lwa4p/A2_1.stl" scale="0.001 0.001 0.001" />
       </geometry>
         <material name="Schunk/LightGrey" />
@@ -144,5 +144,5 @@
       <origin rpy="0 1.57079632679 0" xyz="-0.2053 0 0"/>
      <geometry>
-        <mesh filename="package://industrial_kuka_ros/robot_description/meshes/LWA4P/A2_1.stl" scale="0.001 0.001 0.001" />
+        <mesh filename="package://schunk_description/meshes/lwa4p/A2_1.stl" scale="0.001 0.001 0.001" />
       </geometry>
     </collision>
@@ -150,5 +150,5 @@
       <origin rpy="1.57079632679 1.57079632679 0" xyz="0 0.2053 0"/>
       <geometry>
-        <mesh filename="package://industrial_kuka_ros/robot_description/meshes/LWA4P/A2_2.stl" scale="0.001 0.001 0.001" />
+        <mesh filename="package://schunk_description/meshes/lwa4p/A2_2.stl" scale="0.001 0.001 0.001" />
       </geometry>
         <material name="Schunk/LightGrey" />
@@ -157,5 +157,5 @@
       <origin rpy="1.57079632679 1.57079632679 0" xyz="0 0.2053 0"/>
      <geometry>
-        <mesh filename="package://industrial_kuka_ros/robot_description/meshes/LWA4P/A2_2.stl" scale="0.001 0.001 0.001" />
+        <mesh filename="package://schunk_description/meshes/lwa4p/A2_2.stl" scale="0.001 0.001 0.001" />
       </geometry>
     </collision>
@@ -163,5 +163,5 @@
       <origin rpy="1.57079632679 1.57079632679 0" xyz="0 0.2053 0"/>
       <geometry>
-        <mesh filename="package://industrial_kuka_ros/robot_description/meshes/LWA4P/A2_3.stl" scale="0.001 0.001 0.001" />
+        <mesh filename="package://schunk_description/meshes/lwa4p/A2_3.stl" scale="0.001 0.001 0.001" />
       </geometry>
         <material name="Schunk/LightGrey" />
@@ -170,5 +170,5 @@
       <origin rpy="1.57079632679 1.57079632679 0" xyz="0 0.2053 0"/>
      <geometry>
-        <mesh filename="package://industrial_kuka_ros/robot_description/meshes/LWA4P/A2_3.stl" scale="0.001 0.001 0.001" />
+        <mesh filename="package://schunk_description/meshes/lwa4p/A2_3.stl" scale="0.001 0.001 0.001" />
       </geometry>
     </collision>
@@ -195,5 +195,5 @@
        <origin rpy="0 1.57079632679 -1.57079632679" xyz="0 0.5553 0 "/>
       <geometry>
-        <mesh filename="package://industrial_kuka_ros/robot_description/meshes/LWA4P/A3.stl" scale="0.001 0.001 0.001" />
+        <mesh filename="package://schunk_description/meshes/lwa4p/A3.stl" scale="0.001 0.001 0.001" />
       </geometry>
         <material name="Schunk/Blue" />
@@ -202,5 +202,5 @@
        <origin rpy="0 1.57079632679 -1.57079632679" xyz="0 0.5553 0 "/>
       <geometry>
-        <mesh filename="package://industrial_kuka_ros/robot_description/meshes/LWA4P/A3.stl" scale="0.001 0.001 0.001" />
+        <mesh filename="package://schunk_description/meshes/lwa4p/A3.stl" scale="0.001 0.001 0.001" />
       </geometry>
     </collision>
@@ -227,5 +227,5 @@
       <origin rpy="0 3.14159265359 0" xyz="0 0 0.5553"/>
       <geometry>
-        <mesh filename="package://industrial_kuka_ros/robot_description/meshes/LWA4P/A4_1.stl" scale="0.001 0.001 0.001" />
+        <mesh filename="package://schunk_description/meshes/lwa4p/A4_1.stl" scale="0.001 0.001 0.001" />
       </geometry>
         <material name="Schunk/LightGrey" />
@@ -234,5 +234,5 @@
       <origin rpy="0 3.14159265359 0" xyz="0 0 0.5553"/>
       <geometry>
-        <mesh filename="package://industrial_kuka_ros/robot_description/meshes/LWA4P/A4_1.stl" scale="0.001 0.001 0.001" />
+        <mesh filename="package://schunk_description/meshes/lwa4p/A4_1.stl" scale="0.001 0.001 0.001" />
       </geometry>
     </collision>
@@ -240,5 +240,5 @@
       <origin rpy="0 3.14159265359 -1.57079632679" xyz="0 0 0.5553"/>
       <geometry>
-        <mesh filename="package://industrial_kuka_ros/robot_description/meshes/LWA4P/A4_2.stl" scale="0.001 0.001 0.001" />
+        <mesh filename="package://schunk_description/meshes/lwa4p/A4_2.stl" scale="0.001 0.001 0.001" />
       </geometry>
         <material name="Schunk/LightGrey" />
@@ -247,5 +247,5 @@
       <origin rpy="0 3.14159265359 -1.57079632679" xyz="0 0 0"/>
       <geometry>
-        <mesh filename="package://industrial_kuka_ros/robot_description/meshes/LWA4P/A4_2.stl" scale="0.001 0.001 0.001" />
+        <mesh filename="package://schunk_description/meshes/lwa4p/A4_2.stl" scale="0.001 0.001 0.001" />
       </geometry>
     </collision>
@@ -253,5 +253,5 @@
       <origin rpy="0 3.14159265359 -1.57079632679" xyz="0 0 0.5553"/>
       <geometry>
-        <mesh filename="package://industrial_kuka_ros/robot_description/meshes/LWA4P/A4_3.stl" scale="0.001 0.001 0.001" />
+        <mesh filename="package://schunk_description/meshes/lwa4p/A4_3.stl" scale="0.001 0.001 0.001" />
       </geometry>
         <material name="Schunk/LightGrey" />
@@ -260,5 +260,5 @@
       <origin rpy="0 3.14159265359 -1.57079632679" xyz="0 0 0.5553"/>
       <geometry>
-        <mesh filename="package://industrial_kuka_ros/robot_description/meshes/LWA4P/A4_3.stl" scale="0.001 0.001 0.001" />
+        <mesh filename="package://schunk_description/meshes/lwa4p/A4_3.stl" scale="0.001 0.001 0.001" />
       </geometry>
     </collision>
@@ -285,5 +285,5 @@
        <origin rpy="0 1.57079632679 -1.57079632679" xyz="0 0.8602 0"/>
       <geometry>
-        <mesh filename="package://industrial_kuka_ros/robot_description/meshes/LWA4P/A5.stl" scale="0.001 0.001 0.001" />
+        <mesh filename="package://schunk_description/meshes/lwa4p/A5.stl" scale="0.001 0.001 0.001" />
       </geometry>
         <material name="Schunk/Blue" />
@@ -292,5 +292,5 @@
        <origin rpy="0 1.57079632679 -1.57079632679" xyz="0 0.8602 0"/>
       <geometry>
-        <mesh filename="package://industrial_kuka_ros/robot_description/meshes/LWA4P/A5.stl" scale="0.001 0.001 0.001" />
+        <mesh filename="package://schunk_description/meshes/lwa4p/A5.stl" scale="0.001 0.001 0.001" />
       </geometry>
     </collision>
@@ -317,38 +317,38 @@
       <origin rpy="0 3.14159265359 0" xyz="0 0 0.8602"/>
       <geometry>
-        <mesh filename="package://industrial_kuka_ros/robot_description/meshes/LWA4P/A6_1.stl" scale="0.001 0.001 0.001" />
-      </geometry>
-        <material name="Schunk/LightGrey" />
-    </visual>
-    <collision>
-      <origin rpy="0 3.14159265359 0" xyz="0 0 0.8602"/>
-      <geometry>
-        <mesh filename="package://industrial_kuka_ros/robot_description/meshes/LWA4P/A6_1.stl" scale="0.001 0.001 0.001" />
-      </geometry>
-    </collision>
-    <visual>
-      <origin rpy="0 3.14159265359 0" xyz="0 0 0.8602"/>
-      <geometry>
-        <mesh filename="package://industrial_kuka_ros/robot_description/meshes/LWA4P/A6_2.stl" scale="0.001 0.001 0.001" />
-      </geometry>
-        <material name="Schunk/LightGrey" />
-    </visual>
-    <collision>
-      <origin rpy="0 3.14159265359 0" xyz="0 0 0.8602"/>
-      <geometry>
-        <mesh filename="package://industrial_kuka_ros/robot_description/meshes/LWA4P/A6_2.stl" scale="0.001 0.001 0.001" />
-      </geometry>
-    </collision>
-    <visual>
-      <origin rpy="0 3.14159265359 0" xyz="0 0 0.8602"/>
-      <geometry>
-        <mesh filename="package://industrial_kuka_ros/robot_description/meshes/LWA4P/A6_3.stl" scale="0.001 0.001 0.001" />
-      </geometry>
-        <material name="Schunk/LightGrey" />
-    </visual>
-    <collision>
-      <origin rpy="0 3.14159265359 0" xyz="0 0 0.8602"/>
-      <geometry>
-        <mesh filename="package://industrial_kuka_ros/robot_description/meshes/LWA4P/A6_3.stl" scale="0.001 0.001 0.001" />
+        <mesh filename="package://schunk_description/meshes/lwa4p/A6_1.stl" scale="0.001 0.001 0.001" />
+      </geometry>
+        <material name="Schunk/LightGrey" />
+    </visual>
+    <collision>
+      <origin rpy="0 3.14159265359 0" xyz="0 0 0.8602"/>
+      <geometry>
+        <mesh filename="package://schunk_description/meshes/lwa4p/A6_1.stl" scale="0.001 0.001 0.001" />
+      </geometry>
+    </collision>
+    <visual>
+      <origin rpy="0 3.14159265359 0" xyz="0 0 0.8602"/>
+      <geometry>
+        <mesh filename="package://schunk_description/meshes/lwa4p/A6_2.stl" scale="0.001 0.001 0.001" />
+      </geometry>
+        <material name="Schunk/LightGrey" />
+    </visual>
+    <collision>
+      <origin rpy="0 3.14159265359 0" xyz="0 0 0.8602"/>
+      <geometry>
+        <mesh filename="package://schunk_description/meshes/lwa4p/A6_2.stl" scale="0.001 0.001 0.001" />
+      </geometry>
+    </collision>
+    <visual>
+      <origin rpy="0 3.14159265359 0" xyz="0 0 0.8602"/>
+      <geometry>
+        <mesh filename="package://schunk_description/meshes/lwa4p/A6_3.stl" scale="0.001 0.001 0.001" />
+      </geometry>
+        <material name="Schunk/LightGrey" />
+    </visual>
+    <collision>
+      <origin rpy="0 3.14159265359 0" xyz="0 0 0.8602"/>
+      <geometry>
+        <mesh filename="package://schunk_description/meshes/lwa4p/A6_3.stl" scale="0.001 0.001 0.001" />
       </geometry>
     </collision>

Commit message: Correct description

File: schunk_description/urdf/lwa4p/lwa4p.urdf.xacro (robot description, xacro)
@@ -121,5 +121,5 @@
       <parent link="${name}_1_link"/>
       <child link="${name}_2_link"/>
-      <axis xyz="0 0 1"/>
+      <axis xyz="0 0 -1"/>
       <limit effort="370" velocity="1.26" lower="${-2.967 + safety_offset}" upper="${2.967 - safety_offset}"/>
       <!--safety_controller k_position="20" k_velocity="50" soft_lower_limit="${-2.09 + 0.01}" soft_upper_limit="${2.09 - 0.01}" /-->
@@ -211,5 +211,5 @@
       <parent link="${name}_3_link"/>
       <child link="${name}_4_link"/>
-      <axis xyz="0 0 1" />
+      <axis xyz="0 0 -1" />
       <limit effort="176" velocity="1.26" lower="${-2.967 + safety_offset}" upper="${2.967 - safety_offset}"/>
       <!--safety_controller k_position="20" k_velocity="25" soft_lower_limit="${-2.09 + 0.01}" soft_upper_limit="${2.09 - 0.01}" /-->
@@ -301,5 +301,5 @@
       <parent link="${name}_5_link"/>
       <child link="${name}_6_link"/>
-      <axis xyz="0 0 1" />
+      <axis xyz="0 0 -1" />
       <limit effort="20.1" velocity="1.26" lower="${-2.967 + safety_offset}" upper="${2.967 - safety_offset}" />
       <!--safety_controller k_position="20" k_velocity="25" soft_lower_limit="${-2.09 + 0.01}" soft_upper_limit="${2.09 - 0.01}" /-->

Commit message: rename 7_link to tool_link

File: schunk_description/urdf/lwa4p/lwa4p.urdf.xacro (robot description, xacro)
@@ -354,14 +354,14 @@
     </collision>
     </link>
- <!-- flange -->
-    <joint name="${name}_7_joint" type="fixed">
+    <!-- flange -->
+    <joint name="${name}_tool_joint" type="fixed">
       <origin xyz="0 0 -0.0751" rpy="${M_PI} 0 0" />
       <parent link="${name}_6_link"/>
-      <child link="${name}_7_link"/>
+      <child link="${name}_tool_link"/>
       <axis xyz="0 0 1" />
       <limit effort="20.1" velocity="1.26" lower="${-2.967 + safety_offset}" upper="${2.967 - safety_offset}" />
       <!--safety_controller k_position="20" k_velocity="25" soft_lower_limit="${-2.09 + 0.01}" soft_upper_limit="${2.09 - 0.01}" /-->
     </joint>
-    <link name="${name}_7_link">
+    <link name="${name}_tool_link">
       <xacro:default_inertial/>
 <!--
