Commit message: Updated description of Powerball and added new materials

File: schunk_description/urdf/lwa4p/lwa4p.urdf.xacro (robot description, xacro)
@@ -19,5 +19,5 @@
         <mesh filename="package://schunk_description/meshes/lwa4p/A0_1.stl" scale="0.001 0.001 0.001" />
       </geometry>
-        <material name="Schunk/LightGrey" />
+        <material name="Schunk/DarkGrey" />
     </visual>
     <collision>
@@ -32,5 +32,5 @@
         <mesh filename="package://schunk_description/meshes/lwa4p/A0_2.stl" scale="0.001 0.001 0.001" />
       </geometry>
-        <material name="Schunk/LightGrey" />
+        <material name="Schunk/DarkGrey" />
     </visual>
     <collision>
@@ -45,5 +45,5 @@
         <mesh filename="package://schunk_description/meshes/lwa4p/A0_3.stl" scale="0.001 0.001 0.001" />
       </geometry>
-        <material name="Schunk/LightGrey" />
+        <material name="Schunk/DarkGrey" />
     </visual>
     <collision>
@@ -58,5 +58,5 @@
         <mesh filename="package://schunk_description/meshes/lwa4p/A0_4.stl" scale="0.001 0.001 0.001" />
       </geometry>
-        <material name="Schunk/LightGrey" />
+        <material name="Schunk/DarkGrey" />
     </visual>
     <collision>
@@ -107,5 +107,5 @@
         <mesh filename="package://schunk_description/meshes/lwa4p/A1.stl" scale="0.001 0.001 0.001" />
       </geometry>
-       <material name="Schunk/Blue" />
+       <material name="Schunk/DarkGrey" />
     </visual>
     <collision>
@@ -139,5 +139,5 @@
         <mesh filename="package://schunk_description/meshes/lwa4p/A2_1.stl" scale="0.001 0.001 0.001" />
       </geometry>
-        <material name="Schunk/LightGrey" />
+        <material name="Schunk/DarkBlue" />
     </visual>
     <collision>
@@ -152,5 +152,5 @@
         <mesh filename="package://schunk_description/meshes/lwa4p/A2_2.stl" scale="0.001 0.001 0.001" />
       </geometry>
-        <material name="Schunk/LightGrey" />
+        <material name="Schunk/DarkBlue" />
     </visual>
     <collision>
@@ -165,5 +165,5 @@
         <mesh filename="package://schunk_description/meshes/lwa4p/A2_3.stl" scale="0.001 0.001 0.001" />
       </geometry>
-        <material name="Schunk/LightGrey" />
+        <material name="Schunk/DarkBlue" />
     </visual>
     <collision>
@@ -197,5 +197,5 @@
         <mesh filename="package://schunk_description/meshes/lwa4p/A3.stl" scale="0.001 0.001 0.001" />
       </geometry>
-        <material name="Schunk/Blue" />
+        <material name="Schunk/DarkGrey" />
     </visual>
     <collision>
@@ -225,12 +225,12 @@
 -->
     <visual>
-      <origin rpy="0 3.14159265359 0" xyz="0 0 0.5553"/>
+      <origin rpy="0 ${M_PI} 0" xyz="0 0 0.5553"/>
       <geometry>
         <mesh filename="package://schunk_description/meshes/lwa4p/A4_1.stl" scale="0.001 0.001 0.001" />
       </geometry>
-        <material name="Schunk/LightGrey" />
-    </visual>
-    <collision>
-      <origin rpy="0 3.14159265359 0" xyz="0 0 0.5553"/>
+        <material name="Schunk/DarkBlue" />
+    </visual>
+    <collision>
+      <origin rpy="0 ${M_PI} 0" xyz="0 0 0.5553"/>
       <geometry>
         <mesh filename="package://schunk_description/meshes/lwa4p/A4_1.stl" scale="0.001 0.001 0.001" />
@@ -238,12 +238,12 @@
     </collision>
     <visual>
-      <origin rpy="0 3.14159265359 -1.57079632679" xyz="0 0 0.5553"/>
+      <origin rpy="0 ${M_PI} -1.57079632679" xyz="0 0 0.5553"/>
       <geometry>
         <mesh filename="package://schunk_description/meshes/lwa4p/A4_2.stl" scale="0.001 0.001 0.001" />
       </geometry>
-        <material name="Schunk/LightGrey" />
-    </visual>
-    <collision>
-      <origin rpy="0 3.14159265359 -1.57079632679" xyz="0 0 0"/>
+        <material name="Schunk/DarkBlue" />
+    </visual>
+    <collision>
+      <origin rpy="0 ${M_PI} -1.57079632679" xyz="0 0 0"/>
       <geometry>
         <mesh filename="package://schunk_description/meshes/lwa4p/A4_2.stl" scale="0.001 0.001 0.001" />
@@ -251,12 +251,12 @@
     </collision>
     <visual>
-      <origin rpy="0 3.14159265359 -1.57079632679" xyz="0 0 0.5553"/>
+      <origin rpy="0 ${M_PI} -1.57079632679" xyz="0 0 0.5553"/>
       <geometry>
         <mesh filename="package://schunk_description/meshes/lwa4p/A4_3.stl" scale="0.001 0.001 0.001" />
       </geometry>
-        <material name="Schunk/LightGrey" />
-    </visual>
-    <collision>
-      <origin rpy="0 3.14159265359 -1.57079632679" xyz="0 0 0.5553"/>
+        <material name="Schunk/DarkBlue" />
+    </visual>
+    <collision>
+      <origin rpy="0 ${M_PI} -1.57079632679" xyz="0 0 0.5553"/>
       <geometry>
         <mesh filename="package://schunk_description/meshes/lwa4p/A4_3.stl" scale="0.001 0.001 0.001" />
@@ -287,5 +287,5 @@
         <mesh filename="package://schunk_description/meshes/lwa4p/A5.stl" scale="0.001 0.001 0.001" />
       </geometry>
-        <material name="Schunk/Blue" />
+        <material name="Schunk/DarkGrey" />
     </visual>
     <collision>
@@ -314,62 +314,39 @@
       </inertial>
 -->
-    <visual>
-      <origin rpy="0 3.14159265359 0" xyz="0 0 0.8602"/>
-      <geometry>
-        <mesh filename="package://schunk_description/meshes/lwa4p/A6_1.stl" scale="0.001 0.001 0.001" />
-      </geometry>
-        <material name="Schunk/LightGrey" />
-    </visual>
-    <collision>
-      <origin rpy="0 3.14159265359 0" xyz="0 0 0.8602"/>
-      <geometry>
-        <mesh filename="package://schunk_description/meshes/lwa4p/A6_1.stl" scale="0.001 0.001 0.001" />
-      </geometry>
-    </collision>
-    <visual>
-      <origin rpy="0 3.14159265359 0" xyz="0 0 0.8602"/>
-      <geometry>
-        <mesh filename="package://schunk_description/meshes/lwa4p/A6_2.stl" scale="0.001 0.001 0.001" />
-      </geometry>
-        <material name="Schunk/LightGrey" />
-    </visual>
-    <collision>
-      <origin rpy="0 3.14159265359 0" xyz="0 0 0.8602"/>
-      <geometry>
-        <mesh filename="package://schunk_description/meshes/lwa4p/A6_2.stl" scale="0.001 0.001 0.001" />
-      </geometry>
-    </collision>
-    <visual>
-      <origin rpy="0 3.14159265359 0" xyz="0 0 0.8602"/>
-      <geometry>
-        <mesh filename="package://schunk_description/meshes/lwa4p/A6_3.stl" scale="0.001 0.001 0.001" />
-      </geometry>
-        <material name="Schunk/LightGrey" />
-    </visual>
-    <collision>
-      <origin rpy="0 3.14159265359 0" xyz="0 0 0.8602"/>
-      <geometry>
-        <mesh filename="package://schunk_description/meshes/lwa4p/A6_3.stl" scale="0.001 0.001 0.001" />
-      </geometry>
-    </collision>
+        <visual>
+        <origin rpy="0 ${M_PI} 0" xyz="0 0 0.8602"/>
+        <geometry>
+            <mesh filename="package://schunk_description/meshes/lwa4p/A6_1.stl" scale="0.001 0.001 0.001" />
+        </geometry>
+        <material name="Schunk/DarkGrey" />
+        </visual>
+        <collision>
+        <origin rpy="0 ${M_PI} 0" xyz="0 0 0.8602"/>
+        <geometry>
+            <mesh filename="package://schunk_description/meshes/lwa4p/A6_1.stl" scale="0.001 0.001 0.001" />
+        </geometry>
+        </collision>
+        <visual>
+        <origin rpy="0 ${M_PI} 0" xyz="0 0 0.8602"/>
+        <geometry>
+            <mesh filename="package://schunk_description/meshes/lwa4p/A6_2.stl" scale="0.001 0.001 0.001" />
+        </geometry>
+        <material name="Schunk/Black" />
+        </visual>
+        <collision>
+        <origin rpy="0 ${M_PI} 0" xyz="0 0 0.8602"/>
+        <geometry>
+            <mesh filename="package://schunk_description/meshes/lwa4p/A6_2.stl" scale="0.001 0.001 0.001" />
+        </geometry>
+        </collision>
     </link>
     <!-- flange -->
     <joint name="${name}_tool_joint" type="fixed">
-      <origin xyz="0 0 -0.0751" rpy="${M_PI} 0 0" />
+      <origin xyz="0 0 -0.0748" rpy="${M_PI} 0 0" />
       <parent link="${name}_6_link"/>
       <child link="${name}_tool_link"/>
-      <axis xyz="0 0 1" />
-      <limit effort="20.1" velocity="1.26" lower="${-2.967 + safety_offset}" upper="${2.967 - safety_offset}" />
-      <!--safety_controller k_position="20" k_velocity="25" soft_lower_limit="${-2.09 + 0.01}" soft_upper_limit="${2.09 - 0.01}" /-->
     </joint>
     <link name="${name}_tool_link">
       <xacro:default_inertial/>
-<!--
-      <inertial>
-        <origin xyz="0 0 0" rpy="0 0 0"/>
-        <mass value="0.819"/>
-        <inertia ixx="0.01" ixy="0" ixz="0" iyy="0.01" iyz="0" izz="0.01" />
-      </inertial>
--->
     </link>
     <!-- extensions -->

File: schunk_description/urdf/materials.urdf.xacro (robot description, xacro)
@@ -16,3 +16,6 @@
     <color rgba="0.0 0.0 0.8 1.0"/>
   </material>
+  <material name="Schunk/DarkBlue">
+      <color rgba="0.05 0.0 0.4 1.0"/>
+  </material>
 </robot>

Commit message: Updated description

File: schunk_description/urdf/lwa4p/lwa4p.urdf.xacro (robot description, xacro)
@@ -103,5 +103,5 @@
 -->
     <visual>
-      <origin rpy="0 0 -1.57079632679" xyz="0 0 -0.2053"/>
+      <origin rpy="0 0 ${-M_PI/2}" xyz="0 0 -0.2053"/>
       <geometry>
         <mesh filename="package://schunk_description/meshes/lwa4p/A1.stl" scale="0.001 0.001 0.001" />
@@ -110,5 +110,5 @@
     </visual>
     <collision>
-      <origin rpy="0 0 -1.57079632679" xyz="0 0 -0.2053"/>
+      <origin rpy="0 0 ${-M_PI/2}" xyz="0 0 -0.2053"/>
       <geometry>
         <mesh filename="package://schunk_description/meshes/lwa4p/A1.stl" scale="0.001 0.001 0.001" />
@@ -135,5 +135,5 @@
 -->
     <visual>
-      <origin rpy="0 1.57079632679 0" xyz="-0.2053 0 0"/>
+      <origin rpy="0 ${M_PI/2} 0" xyz="-0.2053 0 0"/>
       <geometry>
         <mesh filename="package://schunk_description/meshes/lwa4p/A2_1.stl" scale="0.001 0.001 0.001" />
@@ -142,5 +142,5 @@
     </visual>
     <collision>
-      <origin rpy="0 1.57079632679 0" xyz="-0.2053 0 0"/>
+      <origin rpy="0 ${M_PI/2} 0" xyz="-0.2053 0 0"/>
      <geometry>
         <mesh filename="package://schunk_description/meshes/lwa4p/A2_1.stl" scale="0.001 0.001 0.001" />
@@ -148,5 +148,5 @@
     </collision>
     <visual>
-      <origin rpy="1.57079632679 1.57079632679 0" xyz="0 0.2053 0"/>
+      <origin rpy="${M_PI/2} ${M_PI/2} 0" xyz="0 0.2053 0"/>
       <geometry>
         <mesh filename="package://schunk_description/meshes/lwa4p/A2_2.stl" scale="0.001 0.001 0.001" />
@@ -155,5 +155,5 @@
     </visual>
     <collision>
-      <origin rpy="1.57079632679 1.57079632679 0" xyz="0 0.2053 0"/>
+      <origin rpy="${M_PI/2} ${M_PI/2} 0" xyz="0 0.2053 0"/>
      <geometry>
         <mesh filename="package://schunk_description/meshes/lwa4p/A2_2.stl" scale="0.001 0.001 0.001" />
@@ -161,5 +161,5 @@
     </collision>
     <visual>
-      <origin rpy="1.57079632679 1.57079632679 0" xyz="0 0.2053 0"/>
+      <origin rpy="${M_PI/2} ${M_PI/2} 0" xyz="0 0.2053 0"/>
       <geometry>
         <mesh filename="package://schunk_description/meshes/lwa4p/A2_3.stl" scale="0.001 0.001 0.001" />
@@ -168,5 +168,5 @@
     </visual>
     <collision>
-      <origin rpy="1.57079632679 1.57079632679 0" xyz="0 0.2053 0"/>
+      <origin rpy="${M_PI/2} ${M_PI/2} 0" xyz="0 0.2053 0"/>
      <geometry>
         <mesh filename="package://schunk_description/meshes/lwa4p/A2_3.stl" scale="0.001 0.001 0.001" />
@@ -193,5 +193,5 @@
 -->
     <visual>
-       <origin rpy="0 1.57079632679 -1.57079632679" xyz="0 0.5553 0 "/>
+       <origin rpy="0 ${M_PI/2} ${-M_PI/2}" xyz="0 0.5553 0 "/>
       <geometry>
         <mesh filename="package://schunk_description/meshes/lwa4p/A3.stl" scale="0.001 0.001 0.001" />
@@ -200,5 +200,5 @@
     </visual>
     <collision>
-       <origin rpy="0 1.57079632679 -1.57079632679" xyz="0 0.5553 0 "/>
+       <origin rpy="0 ${M_PI/2} ${-M_PI/2}" xyz="0 0.5553 0 "/>
       <geometry>
         <mesh filename="package://schunk_description/meshes/lwa4p/A3.stl" scale="0.001 0.001 0.001" />
@@ -238,5 +238,5 @@
     </collision>
     <visual>
-      <origin rpy="0 ${M_PI} -1.57079632679" xyz="0 0 0.5553"/>
+      <origin rpy="0 ${M_PI} ${-M_PI/2}" xyz="0 0 0.5553"/>
       <geometry>
         <mesh filename="package://schunk_description/meshes/lwa4p/A4_2.stl" scale="0.001 0.001 0.001" />
@@ -245,5 +245,5 @@
     </visual>
     <collision>
-      <origin rpy="0 ${M_PI} -1.57079632679" xyz="0 0 0"/>
+      <origin rpy="0 ${M_PI} ${-M_PI/2}" xyz="0 0 0"/>
       <geometry>
         <mesh filename="package://schunk_description/meshes/lwa4p/A4_2.stl" scale="0.001 0.001 0.001" />
@@ -251,5 +251,5 @@
     </collision>
     <visual>
-      <origin rpy="0 ${M_PI} -1.57079632679" xyz="0 0 0.5553"/>
+      <origin rpy="0 ${M_PI} ${-M_PI/2}" xyz="0 0 0.5553"/>
       <geometry>
         <mesh filename="package://schunk_description/meshes/lwa4p/A4_3.stl" scale="0.001 0.001 0.001" />
@@ -258,5 +258,5 @@
     </visual>
     <collision>
-      <origin rpy="0 ${M_PI} -1.57079632679" xyz="0 0 0.5553"/>
+      <origin rpy="0 ${M_PI} ${-M_PI/2}" xyz="0 0 0.5553"/>
       <geometry>
         <mesh filename="package://schunk_description/meshes/lwa4p/A4_3.stl" scale="0.001 0.001 0.001" />
@@ -283,5 +283,5 @@
 -->
     <visual>
-       <origin rpy="0 1.57079632679 -1.57079632679" xyz="0 0.8602 0"/>
+       <origin rpy="0 ${M_PI/2} ${-M_PI/2}" xyz="0 0.8602 0"/>
       <geometry>
         <mesh filename="package://schunk_description/meshes/lwa4p/A5.stl" scale="0.001 0.001 0.001" />
@@ -290,5 +290,5 @@
     </visual>
     <collision>
-       <origin rpy="0 1.57079632679 -1.57079632679" xyz="0 0.8602 0"/>
+       <origin rpy="0 ${M_PI/2} ${-M_PI/2}" xyz="0 0.8602 0"/>
       <geometry>
         <mesh filename="package://schunk_description/meshes/lwa4p/A5.stl" scale="0.001 0.001 0.001" />
