Commit message: Indentation is corrected. Using M_PI insted of nummbers

File: schunk_description/urdf/lwa4p/lwa4p.urdf.xacro (robot description, xacro)
@@ -14,56 +14,56 @@
       <link name="${name}_podest_link">
         <xacro:default_inertial/>
-     <visual>
-          <origin xyz="0 0 0" rpy="0 0 ${-M_PI/2}" />
-      <geometry>
-        <mesh filename="package://schunk_description/meshes/lwa4p/A0_1.stl" scale="0.001 0.001 0.001" />
-      </geometry>
-        <material name="Schunk/DarkGrey" />
-    </visual>
-    <collision>
-          <origin xyz="0 0 0" rpy="0 0 ${-M_PI/2}" />
-      <geometry>
-        <mesh filename="package://schunk_description/meshes/lwa4p/A0_1.stl" scale="0.001 0.001 0.001" />
-      </geometry>
-    </collision>
-    <visual>
-          <origin xyz="0 0 0" rpy="0 0 ${-M_PI/2}" />
-      <geometry>
-        <mesh filename="package://schunk_description/meshes/lwa4p/A0_2.stl" scale="0.001 0.001 0.001" />
-      </geometry>
-        <material name="Schunk/DarkGrey" />
-    </visual>
-    <collision>
-          <origin xyz="0 0 0" rpy="0 0 ${-M_PI/2}" />
-      <geometry>
-        <mesh filename="package://schunk_description/meshes/lwa4p/A0_2.stl" scale="0.001 0.001 0.001" />
-      </geometry>
-    </collision>
-    <visual>
-          <origin xyz="0 0 0" rpy="0 0 ${-M_PI/2}" />
-      <geometry>
-        <mesh filename="package://schunk_description/meshes/lwa4p/A0_3.stl" scale="0.001 0.001 0.001" />
-      </geometry>
-        <material name="Schunk/DarkGrey" />
-    </visual>
-    <collision>
-          <origin xyz="0 0 0" rpy="0 0 ${-M_PI/2}" />
-      <geometry>
-        <mesh filename="package://schunk_description/meshes/lwa4p/A0_3.stl" scale="0.001 0.001 0.001" />
-      </geometry>
-    </collision>
-    <visual>
-          <origin xyz="0 0 0" rpy="0 0 ${-M_PI/2}" />
-      <geometry>
-        <mesh filename="package://schunk_description/meshes/lwa4p/A0_4.stl" scale="0.001 0.001 0.001" />
-      </geometry>
-        <material name="Schunk/DarkGrey" />
-    </visual>
-    <collision>
+        <visual>
+          <origin xyz="0 0 0" rpy="0 0 ${-M_PI/2}" />
+          <geometry>
+            <mesh filename="package://schunk_description/meshes/lwa4p/A0_1.stl" scale="0.001 0.001 0.001" />
+          </geometry>
+          <material name="Schunk/DarkGrey" />
+        </visual>
+        <collision>
+          <origin xyz="0 0 0" rpy="0 0 ${-M_PI/2}" />
+          <geometry>
+            <mesh filename="package://schunk_description/meshes/lwa4p/A0_1.stl" scale="0.001 0.001 0.001" />
+          </geometry>
+        </collision>
+        <visual>
+          <origin xyz="0 0 0" rpy="0 0 ${-M_PI/2}" />
+          <geometry>
+            <mesh filename="package://schunk_description/meshes/lwa4p/A0_2.stl" scale="0.001 0.001 0.001" />
+          </geometry>
+          <material name="Schunk/DarkGrey" />
+        </visual>
+        <collision>
+          <origin xyz="0 0 0" rpy="0 0 ${-M_PI/2}" />
+          <geometry>
+            <mesh filename="package://schunk_description/meshes/lwa4p/A0_2.stl" scale="0.001 0.001 0.001" />
+          </geometry>
+        </collision>
+        <visual>
+          <origin xyz="0 0 0" rpy="0 0 ${-M_PI/2}" />
+          <geometry>
+            <mesh filename="package://schunk_description/meshes/lwa4p/A0_3.stl" scale="0.001 0.001 0.001" />
+          </geometry>
+            <material name="Schunk/DarkGrey" />
+        </visual>
+        <collision>
+            <origin xyz="0 0 0" rpy="0 0 ${-M_PI/2}" />
+            <geometry>
+              <mesh filename="package://schunk_description/meshes/lwa4p/A0_3.stl" scale="0.001 0.001 0.001" />
+            </geometry>
+        </collision>
+        <visual>
+          <origin xyz="0 0 0" rpy="0 0 ${-M_PI/2}" />
+          <geometry>
+            <mesh filename="package://schunk_description/meshes/lwa4p/A0_4.stl" scale="0.001 0.001 0.001" />
+          </geometry>
+          <material name="Schunk/DarkGrey" />
+        </visual>
+        <collision>
           <origin xyz="0 0 0" rpy="0 0 0" />
-      <geometry>
-        <mesh filename="package://schunk_description/meshes/lwa4p/A0_4.stl" scale="0.001 0.001 0.001" />
-      </geometry>
-    </collision>
+          <geometry>
+            <mesh filename="package://schunk_description/meshes/lwa4p/A0_4.stl" scale="0.001 0.001 0.001" />
+          </geometry>
+        </collision>
       </link>
       <joint name="${name}_base_joint" type="fixed">
@@ -102,17 +102,17 @@
       </inertial>
 -->
-    <visual>
-      <origin rpy="0 0 ${-M_PI/2}" xyz="0 0 -0.2053"/>
-      <geometry>
-        <mesh filename="package://schunk_description/meshes/lwa4p/A1.stl" scale="0.001 0.001 0.001" />
-      </geometry>
-       <material name="Schunk/DarkGrey" />
-    </visual>
-    <collision>
-      <origin rpy="0 0 ${-M_PI/2}" xyz="0 0 -0.2053"/>
-      <geometry>
-        <mesh filename="package://schunk_description/meshes/lwa4p/A1.stl" scale="0.001 0.001 0.001" />
-      </geometry>
-    </collision>
+      <visual>
+        <origin xyz="0 0 -0.2053" rpy="0 0 ${-M_PI/2}"/>
+        <geometry>
+          <mesh filename="package://schunk_description/meshes/lwa4p/A1.stl" scale="0.001 0.001 0.001" />
+        </geometry>
+        <material name="Schunk/DarkGrey" />
+      </visual>
+      <collision>
+        <origin xyz="0 0 -0.2053" rpy="0 0 ${-M_PI/2}"/>
+        <geometry>
+          <mesh filename="package://schunk_description/meshes/lwa4p/A1.stl" scale="0.001 0.001 0.001" />
+        </geometry>
+      </collision>
     </link>
     <!-- joint between arm_1_link and arm_2_link -->
@@ -134,43 +134,43 @@
       </inertial>
 -->
-    <visual>
-      <origin rpy="0 ${M_PI/2} 0" xyz="-0.2053 0 0"/>
-      <geometry>
-        <mesh filename="package://schunk_description/meshes/lwa4p/A2_1.stl" scale="0.001 0.001 0.001" />
-      </geometry>
-        <material name="Schunk/DarkBlue" />
-    </visual>
-    <collision>
-      <origin rpy="0 ${M_PI/2} 0" xyz="-0.2053 0 0"/>
-     <geometry>
-        <mesh filename="package://schunk_description/meshes/lwa4p/A2_1.stl" scale="0.001 0.001 0.001" />
-      </geometry>
-    </collision>
-    <visual>
-      <origin rpy="${M_PI/2} ${M_PI/2} 0" xyz="0 0.2053 0"/>
-      <geometry>
-        <mesh filename="package://schunk_description/meshes/lwa4p/A2_2.stl" scale="0.001 0.001 0.001" />
-      </geometry>
-        <material name="Schunk/DarkBlue" />
-    </visual>
-    <collision>
-      <origin rpy="${M_PI/2} ${M_PI/2} 0" xyz="0 0.2053 0"/>
-     <geometry>
-        <mesh filename="package://schunk_description/meshes/lwa4p/A2_2.stl" scale="0.001 0.001 0.001" />
-      </geometry>
-    </collision>
-    <visual>
-      <origin rpy="${M_PI/2} ${M_PI/2} 0" xyz="0 0.2053 0"/>
-      <geometry>
-        <mesh filename="package://schunk_description/meshes/lwa4p/A2_3.stl" scale="0.001 0.001 0.001" />
-      </geometry>
-        <material name="Schunk/DarkBlue" />
-    </visual>
-    <collision>
-      <origin rpy="${M_PI/2} ${M_PI/2} 0" xyz="0 0.2053 0"/>
-     <geometry>
-        <mesh filename="package://schunk_description/meshes/lwa4p/A2_3.stl" scale="0.001 0.001 0.001" />
-      </geometry>
-    </collision>
+      <visual>
+        <origin xyz="-0.2053 0 0" rpy="0 ${M_PI/2} 0"/>
+        <geometry>
+          <mesh filename="package://schunk_description/meshes/lwa4p/A2_1.stl" scale="0.001 0.001 0.001" />
+        </geometry>
+        <material name="Schunk/DarkBlue" />
+      </visual>
+      <collision>
+        <origin xyz="-0.2053 0 0" rpy="0 ${M_PI/2} 0"/>
+        <geometry>
+          <mesh filename="package://schunk_description/meshes/lwa4p/A2_1.stl" scale="0.001 0.001 0.001" />
+        </geometry>
+      </collision>
+      <visual>
+        <origin xyz="0 0.2053 0" rpy="${M_PI/2} ${M_PI/2} 0"/>
+        <geometry>
+          <mesh filename="package://schunk_description/meshes/lwa4p/A2_2.stl" scale="0.001 0.001 0.001" />
+        </geometry>
+        <material name="Schunk/DarkBlue" />
+      </visual>
+      <collision>
+        <origin xyz="0 0.2053 0" rpy="${M_PI/2} ${M_PI/2} 0"/>
+        <geometry>
+          <mesh filename="package://schunk_description/meshes/lwa4p/A2_2.stl" scale="0.001 0.001 0.001" />
+        </geometry>
+      </collision>
+      <visual>
+        <origin xyz="0 0.2053 0" rpy="${M_PI/2} ${M_PI/2} 0"/>
+        <geometry>
+          <mesh filename="package://schunk_description/meshes/lwa4p/A2_3.stl" scale="0.001 0.001 0.001" />
+        </geometry>
+        <material name="Schunk/DarkBlue" />
+      </visual>
+      <collision>
+        <origin xyz="0 0.2053 0" rpy="${M_PI/2} ${M_PI/2} 0"/>
+        <geometry>
+          <mesh filename="package://schunk_description/meshes/lwa4p/A2_3.stl" scale="0.001 0.001 0.001" />
+        </geometry>
+      </collision>
     </link>
     <!-- joint between arm_2_link and arm_3_link -->
@@ -192,17 +192,17 @@
       </inertial>
 -->
-    <visual>
-       <origin rpy="0 ${M_PI/2} ${-M_PI/2}" xyz="0 0.5553 0 "/>
-      <geometry>
-        <mesh filename="package://schunk_description/meshes/lwa4p/A3.stl" scale="0.001 0.001 0.001" />
-      </geometry>
+      <visual>
+        <origin xyz="0 0.5553 0" rpy="0 ${M_PI/2} ${-M_PI/2}"/>
+        <geometry>
+          <mesh filename="package://schunk_description/meshes/lwa4p/A3.stl" scale="0.001 0.001 0.001" />
+        </geometry>
         <material name="Schunk/DarkGrey" />
-    </visual>
-    <collision>
-       <origin rpy="0 ${M_PI/2} ${-M_PI/2}" xyz="0 0.5553 0 "/>
-      <geometry>
-        <mesh filename="package://schunk_description/meshes/lwa4p/A3.stl" scale="0.001 0.001 0.001" />
-      </geometry>
-    </collision>
+      </visual>
+      <collision>
+        <origin xyz="0 0.5553 0" rpy="0 ${M_PI/2} ${-M_PI/2}"/>
+        <geometry>
+          <mesh filename="package://schunk_description/meshes/lwa4p/A3.stl" scale="0.001 0.001 0.001" />
+        </geometry>
+      </collision>
     </link>
     <!-- joint between arm_3_link and arm_4_link -->
@@ -224,43 +224,43 @@
       </inertial>
 -->
-    <visual>
-      <origin rpy="0 ${M_PI} 0" xyz="0 0 0.5553"/>
-      <geometry>
-        <mesh filename="package://schunk_description/meshes/lwa4p/A4_1.stl" scale="0.001 0.001 0.001" />
-      </geometry>
-        <material name="Schunk/DarkBlue" />
-    </visual>
-    <collision>
-      <origin rpy="0 ${M_PI} 0" xyz="0 0 0.5553"/>
-      <geometry>
-        <mesh filename="package://schunk_description/meshes/lwa4p/A4_1.stl" scale="0.001 0.001 0.001" />
-      </geometry>
-    </collision>
-    <visual>
-      <origin rpy="0 ${M_PI} ${-M_PI/2}" xyz="0 0 0.5553"/>
-      <geometry>
-        <mesh filename="package://schunk_description/meshes/lwa4p/A4_2.stl" scale="0.001 0.001 0.001" />
-      </geometry>
-        <material name="Schunk/DarkBlue" />
-    </visual>
-    <collision>
-      <origin rpy="0 ${M_PI} ${-M_PI/2}" xyz="0 0 0"/>
-      <geometry>
-        <mesh filename="package://schunk_description/meshes/lwa4p/A4_2.stl" scale="0.001 0.001 0.001" />
-      </geometry>
-    </collision>
-    <visual>
-      <origin rpy="0 ${M_PI} ${-M_PI/2}" xyz="0 0 0.5553"/>
-      <geometry>
-        <mesh filename="package://schunk_description/meshes/lwa4p/A4_3.stl" scale="0.001 0.001 0.001" />
-      </geometry>
-        <material name="Schunk/DarkBlue" />
-    </visual>
-    <collision>
-      <origin rpy="0 ${M_PI} ${-M_PI/2}" xyz="0 0 0.5553"/>
-      <geometry>
-        <mesh filename="package://schunk_description/meshes/lwa4p/A4_3.stl" scale="0.001 0.001 0.001" />
-      </geometry>
-    </collision>
+      <visual>
+        <origin xyz="0 0 0.5553" rpy="0 ${M_PI} 0"/>
+        <geometry>
+          <mesh filename="package://schunk_description/meshes/lwa4p/A4_1.stl" scale="0.001 0.001 0.001" />
+        </geometry>
+        <material name="Schunk/DarkBlue" />
+      </visual>
+      <collision>
+        <origin xyz="0 0 0.5553" rpy="0 ${M_PI} 0"/>
+        <geometry>
+          <mesh filename="package://schunk_description/meshes/lwa4p/A4_1.stl" scale="0.001 0.001 0.001" />
+        </geometry>
+      </collision>
+      <visual>
+        <origin xyz="0 0 0.5553" rpy="0 ${M_PI} ${-M_PI/2}"/>
+        <geometry>
+          <mesh filename="package://schunk_description/meshes/lwa4p/A4_2.stl" scale="0.001 0.001 0.001" />
+        </geometry>
+        <material name="Schunk/DarkBlue" />
+      </visual>
+      <collision>
+        <origin xyz="0 0 0" rpy="0 ${M_PI} ${-M_PI/2}"/>
+        <geometry>
+          <mesh filename="package://schunk_description/meshes/lwa4p/A4_2.stl" scale="0.001 0.001 0.001" />
+        </geometry>
+      </collision>
+      <visual>
+        <origin xyz="0 0 0.5553" rpy="0 ${M_PI} ${-M_PI/2}"/>
+        <geometry>
+          <mesh filename="package://schunk_description/meshes/lwa4p/A4_3.stl" scale="0.001 0.001 0.001" />
+        </geometry>
+        <material name="Schunk/DarkBlue" />
+      </visual>
+      <collision>
+        <origin xyz="0 0 0.5553" rpy="0 ${M_PI} ${-M_PI/2}"/>
+        <geometry>
+          <mesh filename="package://schunk_description/meshes/lwa4p/A4_3.stl" scale="0.001 0.001 0.001" />
+        </geometry>
+      </collision>
     </link>
     <!-- joint between arm_4_link and arm_5_link -->
@@ -282,17 +282,17 @@
       </inertial>
 -->
-    <visual>
-       <origin rpy="0 ${M_PI/2} ${-M_PI/2}" xyz="0 0.8602 0"/>
-      <geometry>
-        <mesh filename="package://schunk_description/meshes/lwa4p/A5.stl" scale="0.001 0.001 0.001" />
-      </geometry>
+      <visual>
+        <origin xyz="0 0.8602 0" rpy="0 ${M_PI/2} ${-M_PI/2}"/>
+        <geometry>
+          <mesh filename="package://schunk_description/meshes/lwa4p/A5.stl" scale="0.001 0.001 0.001" />
+        </geometry>
         <material name="Schunk/DarkGrey" />
-    </visual>
-    <collision>
-       <origin rpy="0 ${M_PI/2} ${-M_PI/2}" xyz="0 0.8602 0"/>
-      <geometry>
-        <mesh filename="package://schunk_description/meshes/lwa4p/A5.stl" scale="0.001 0.001 0.001" />
-      </geometry>
-    </collision>
+      </visual>
+      <collision>
+        <origin xyz="0 0.8602 0" rpy="0 ${M_PI/2} ${-M_PI/2}"/>
+        <geometry>
+          <mesh filename="package://schunk_description/meshes/lwa4p/A5.stl" scale="0.001 0.001 0.001" />
+        </geometry>
+      </collision>
     </link>
     <!-- joint between arm_5_link and arm_6_link -->
@@ -314,30 +314,30 @@
       </inertial>
 -->
-        <visual>
-        <origin rpy="0 ${M_PI} 0" xyz="0 0 0.8602"/>
-        <geometry>
-            <mesh filename="package://schunk_description/meshes/lwa4p/A6_1.stl" scale="0.001 0.001 0.001" />
+      <visual>
+        <origin xyz="0 0 0.8602" rpy="0 ${M_PI} 0"/>
+        <geometry>
+          <mesh filename="package://schunk_description/meshes/lwa4p/A6_1.stl" scale="0.001 0.001 0.001" />
         </geometry>
         <material name="Schunk/DarkGrey" />
-        </visual>
-        <collision>
-        <origin rpy="0 ${M_PI} 0" xyz="0 0 0.8602"/>
-        <geometry>
-            <mesh filename="package://schunk_description/meshes/lwa4p/A6_1.stl" scale="0.001 0.001 0.001" />
-        </geometry>
-        </collision>
-        <visual>
-        <origin rpy="0 ${M_PI} 0" xyz="0 0 0.8602"/>
-        <geometry>
-            <mesh filename="package://schunk_description/meshes/lwa4p/A6_2.stl" scale="0.001 0.001 0.001" />
+      </visual>
+      <collision>
+        <origin xyz="0 0 0.8602" rpy="0 ${M_PI} 0"/>
+        <geometry>
+          <mesh filename="package://schunk_description/meshes/lwa4p/A6_1.stl" scale="0.001 0.001 0.001" />
+        </geometry>
+      </collision>
+      <visual>
+        <origin xyz="0 0 0.8602" rpy="0 ${M_PI} 0"/>
+        <geometry>
+          <mesh filename="package://schunk_description/meshes/lwa4p/A6_2.stl" scale="0.001 0.001 0.001" />
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