Commit message: Joint limits for pw70 added.

File: schunk_description/urdf/pw70/pw70.urdf.xacro (robot description, xacro)
@@ -29,5 +29,5 @@
       <child link="${name}_pan_link" />
       <axis xyz="0 0 1" />
-	  <!--<limit effort="10" lower="-0.001" upper="0.061" velocity="2.0"/>-->
+	  <limit effort="2.0" velocity="${2 * M_PI}" lower="${-7/3 * M_PI}" upper="${7/3 * M_PI}"/>
     </joint>
     <link name="${name}_pan_link">
@@ -51,6 +51,5 @@
       <child link="${name}_tilt_link" />
       <axis xyz="0 1 0" />
-	  <!--<mimic joint="${name}_finger_left_joint" multiplier="1" offset="0"/>
-	  <limit effort="10" lower="-0.001" upper="0.061" velocity="2.0"/>-->
+	  <limit effort="12.0" velocity="4.1" lower="${-4/6 * M_PI}" upper="${4/6 * M_PI}"/>
     </joint>
     <link name="${name}_tilt_link">

Commit message: removed tool joint

File: schunk_description/urdf/pw70/pw70.urdf.xacro (robot description, xacro)
@@ -68,10 +68,4 @@
 	  -->
     </link>
-	<joint name="${name}_tool_joint" type="fixed" >
-	  <origin xyz="0 0 0" rpy="0 0 0"/>
-      <parent link="${name}_tilt_joint" />
-      <child link="${name}_tool_link" />
-      <xacro:insert_block name="origin" />
-    </joint>
   <!-- extensions -->
   <xacro:schunk_pw70_gazebo name="${name}" />

Commit message: Added calibration offset in pw70 description.

File: schunk_description/urdf/pw70/pw70.urdf.xacro (robot description, xacro)
@@ -5,7 +5,7 @@
   <xacro:macro name="schunk_pw70" params="parent name *origin">
     <joint name="${name}_base_joint" type="fixed" >
+      <xacro:insert_block name="origin" />
       <parent link="${parent}" />
       <child link="${name}_base_link" />
-      <xacro:insert_block name="origin" />
     </joint>
     <link name="${name}_base_link">
@@ -29,5 +29,6 @@
       <child link="${name}_pan_link" />
       <axis xyz="0 0 1" />
-	  <limit effort="2.0" velocity="${2 * M_PI}" lower="${-7/3 * M_PI}" upper="${7/3 * M_PI}"/>
+	  <limit effort="200" velocity="${2 * M_PI}" lower="${-7/3 * M_PI}" upper="${7/3 * M_PI}"/>
+	  <calibration rising="0.0"/>
     </joint>
     <link name="${name}_pan_link">
@@ -52,4 +53,5 @@
       <axis xyz="0 1 0" />
 	  <limit effort="12.0" velocity="4.1" lower="${-4/6 * M_PI}" upper="${4/6 * M_PI}"/>
+	  <calibration rising="0.0"/>
     </joint>
     <link name="${name}_tilt_link">

Commit message: Added tool link. Advertising services in private namespace.

File: schunk_description/urdf/pw70/pw70.urdf.xacro (robot description, xacro)
@@ -70,4 +70,24 @@
 	  -->
     </link>
+	<joint name="${name}_tool_joint" type="fixed" >
+      <origin xyz="0 0 0" rpy="0 0 0"/>
+      <parent link="${name}_tilt_link" />
+      <child link="${name}_tool_link" />
+    </joint>
+    <link name="${name}_tool_link">
+      <xacro:default_inertial/>
+	  <!--
+      <visual>
+        <geometry>
+          <mesh filename="package://schunk_description/meshes/pw70/pw70_tilt.dae" />
+        </geometry>
+      </visual>
+      <collision>
+        <geometry>
+          <mesh filename="package://schunk_description/meshes/pw70/pw70_tilt.stl" />
+        </geometry>
+      </collision>
+	  -->
+    </link>
   <!-- extensions -->
   <xacro:schunk_pw70_gazebo name="${name}" />

Commit message: Updated description of powercube, now is how it should be when powercube is reverslly mounted.

File: schunk_description/urdf/pw70/pw70.urdf.xacro (robot description, xacro)
@@ -4,10 +4,10 @@
   <xacro:include filename="$(find schunk_description)/urdf/pw70/pw70.transmission.xacro" />
   <xacro:macro name="schunk_pw70" params="parent name *origin">
-    <joint name="${name}_base_joint" type="fixed" >
+    <joint name="${name}_joint" type="fixed" >
       <xacro:insert_block name="origin" />
       <parent link="${parent}" />
-      <child link="${name}_base_link" />
+      <child link="${name}_link" />
     </joint>
-    <link name="${name}_base_link">
+    <link name="${name}_link">
       <xacro:default_inertial/>
 	  <!--
@@ -26,7 +26,7 @@
     <joint name="${name}_pan_joint" type="revolute" >
       <origin xyz="0 0 0" rpy="0 0 0"/>
-      <parent link="${name}_base_link" />
+      <parent link="${name}_link" />
       <child link="${name}_pan_link" />
-      <axis xyz="0 0 1" />
+      <axis xyz="0 0 -1" />
 	  <limit effort="200" velocity="${2 * M_PI}" lower="${-7/3 * M_PI}" upper="${7/3 * M_PI}"/>
 	  <calibration rising="0.0"/>
@@ -48,8 +48,8 @@
     </link>
     <joint name="${name}_tilt_joint" type="revolute" >
-      <origin xyz="0 0 0" rpy="0 0 0"/>
+      <origin xyz="0 0 0.0951" rpy="0 0 0"/>
       <parent link="${name}_pan_link" />
       <child link="${name}_tilt_link" />
-      <axis xyz="0 1 0" />
+      <axis xyz="0 -1 0" />
 	  <limit effort="12.0" velocity="4.1" lower="${-4/6 * M_PI}" upper="${4/6 * M_PI}"/>
 	  <calibration rising="0.0"/>
@@ -71,5 +71,5 @@
     </link>
 	<joint name="${name}_tool_joint" type="fixed" >
-      <origin xyz="0 0 0" rpy="0 0 0"/>
+      <origin xyz="0 0 0.07" rpy="0 0 0"/>
       <parent link="${name}_tilt_link" />
       <child link="${name}_tool_link" />

Commit message: Added meshes of pw70 and updated urdf to support upsidedown pw70.

File: schunk_description/urdf/pw70/pw70.urdf.xacro (robot description, xacro)
@@ -3,94 +3,166 @@
   <xacro:include filename="$(find schunk_description)/urdf/pw70/pw70.gazebo.xacro" />
   <xacro:include filename="$(find schunk_description)/urdf/pw70/pw70.transmission.xacro" />
-  <xacro:macro name="schunk_pw70" params="parent name *origin">
-    <joint name="${name}_joint" type="fixed" >
-      <xacro:insert_block name="origin" />
-      <parent link="${parent}" />
-      <child link="${name}_link" />
-    </joint>
-    <link name="${name}_link">
-      <xacro:default_inertial/>
-	  <!--
-      <visual>
-        <geometry>
-          <mesh filename="package://schunk_description/meshes/pw70/pw70_base.dae" />
-        </geometry>
-      </visual>
-      <collision>
-        <geometry>
-          <mesh filename="package://schunk_description/meshes/pw70/pw70_base.stl" />
-        </geometry>
-      </collision>
-	  -->
-    </link>
-    <joint name="${name}_pan_joint" type="revolute" >
-      <origin xyz="0 0 0" rpy="0 0 0"/>
-      <parent link="${name}_link" />
-      <child link="${name}_pan_link" />
-      <axis xyz="0 0 -1" />
-	  <limit effort="200" velocity="${2 * M_PI}" lower="${-7/3 * M_PI}" upper="${7/3 * M_PI}"/>
-	  <calibration rising="0.0"/>
-    </joint>
-    <link name="${name}_pan_link">
-      <xacro:default_inertial/>
-      <!--
-      <visual>
-        <geometry>
-          <mesh filename="package://schunk_description/meshes/pw70/pw70_pan.dae" />
-        </geometry>
-      </visual>
-      <collision>
-        <geometry>
-          <mesh filename="package://schunk_description/meshes/pw70/pw70_pan.stl" />
-        </geometry>
-      </collision>
-	  -->
-    </link>
-    <joint name="${name}_tilt_joint" type="revolute" >
-      <origin xyz="0 0 0.0951" rpy="0 0 0"/>
-      <parent link="${name}_pan_link" />
-      <child link="${name}_tilt_link" />
-      <axis xyz="0 -1 0" />
-	  <limit effort="12.0" velocity="4.1" lower="${-4/6 * M_PI}" upper="${4/6 * M_PI}"/>
-	  <calibration rising="0.0"/>
-    </joint>
-    <link name="${name}_tilt_link">
-      <xacro:default_inertial/>
-	  <!--
-      <visual>
-        <geometry>
-          <mesh filename="package://schunk_description/meshes/pw70/pw70_tilt.dae" />
-        </geometry>
-      </visual>
-      <collision>
-        <geometry>
-          <mesh filename="package://schunk_description/meshes/pw70/pw70_tilt.stl" />
-        </geometry>
-      </collision>
-	  -->
-    </link>
-	<joint name="${name}_tool_joint" type="fixed" >
-      <origin xyz="0 0 0.07" rpy="0 0 0"/>
-      <parent link="${name}_tilt_link" />
-      <child link="${name}_tool_link" />
-    </joint>
-    <link name="${name}_tool_link">
-      <xacro:default_inertial/>
-	  <!--
-      <visual>
-        <geometry>
-          <mesh filename="package://schunk_description/meshes/pw70/pw70_tilt.dae" />
-        </geometry>
-      </visual>
-      <collision>
-        <geometry>
-          <mesh filename="package://schunk_description/meshes/pw70/pw70_tilt.stl" />
-        </geometry>
-      </collision>
-	  -->
-    </link>
-  <!-- extensions -->
-  <xacro:schunk_pw70_gazebo name="${name}" />
-  <xacro:schunk_pw70_transmission name="${name}" />
+  <xacro:macro name="schunk_pw70" params="parent name *origin is_upsidedown">
+    <xacro:unless value="${is_upsidedown}">
+      <joint name="${name}_joint" type="fixed" >
+        <xacro:insert_block name="origin" />
+        <parent link="${parent}" />
+        <child link="${name}_link" />
+      </joint>
+      <link name="${name}_link">
+        <xacro:default_inertial/>
+      </link>
+      <joint name="${name}_tilt_joint" type="revolute" >
+        <origin xyz="0 0 0.07" rpy="0 0 0"/>
+        <parent link="${name}_link" />
+        <child link="${name}_tilt_link" />
+        <axis xyz="0 1 0" />
+        <limit effort="12.0" velocity="4.1" lower="${-4/6 * M_PI}" upper="${4/6 * M_PI}"/>
+        <calibration rising="0.0"/>
+      </joint>
+      <link name="${name}_tilt_link">
+        <xacro:default_inertial/>
+        <visual>
+          <origin xyz="0 0 0" rpy="0 0 0" />
+          <geometry>
+            <mesh filename="package://schunk_description/meshes/pw70/pw70_tilt.dae" />
+          </geometry>
+        </visual>
+        <!--
+        <collision>
+          <geometry>
+            <mesh filename="package://schunk_description/meshes/pw70/pw70_tilt.stl" />
+          </geometry>
+        </collision>
+        -->
+      </link>
+      <joint name="${name}_pan_joint" type="revolute" >
+        <origin xyz="0 0 0.0951" rpy="0 0 0"/>
+        <parent link="${name}_tilt_joint" />
+        <child link="${name}_pan_link" />
+        <axis xyz="0 0 1" />
+        <limit effort="200" velocity="${2 * M_PI}" lower="${-7/3 * M_PI}" upper="${7/3 * M_PI}"/>
+        <calibration rising="0.0"/>
+      </joint>
+      <link name="${name}_pan_link">
+        <xacro:default_inertial/>
+        <visual>
+          <origin xyz="0 0 0" rpy="0 0 0" />
+          <geometry>
+            <mesh filename="package://schunk_description/meshes/pw70/pw70_pan.dae" />
+          </geometry>
+        </visual>
+        <!--
+        <collision>
+          <geometry>
+            <mesh filename="package://schunk_description/meshes/pw70/pw70_pan.stl" />
+          </geometry>
+        </collision>
+        -->
+      </link>
+      <joint name="${name}_tool_joint" type="fixed" >
+        <origin xyz="0 0 0.07" rpy="0 0 0"/>
+        <parent link="${name}_pan_link" />
+        <child link="${name}_tool_link" />
+      </joint>
+      <link name="${name}_tool_link">
+        <xacro:default_inertial/>
+        <visual>
+          <origin xyz="0 0 0" rpy="0 0 0" />
+          <geometry>
+            <mesh filename="package://schunk_description/meshes/pw70/pw70_base.dae" />
+          </geometry>
+        </visual>
+        <!--
+        <collision>
+          <geometry>
+            <mesh filename="package://schunk_description/meshes/pw70/pw70_base.stl" />
+          </geometry>
+        </collision>
+        -->
+      </link>
+    </xacro:unless>
+    <xacro:if value="${is_upsidedown}">
+      <joint name="${name}_joint" type="fixed" >
+        <xacro:insert_block name="origin" />
+        <parent link="${parent}" />
+        <child link="${name}_link" />
+      </joint>
+      <link name="${name}_link">
+        <xacro:default_inertial/>
+        <visual>
+          <origin xyz="0 0 0" rpy="0 0 0" />
+          <geometry>
+            <mesh filename="package://schunk_description/meshes/pw70/pw70_base.dae" />
+          </geometry>
+        </visual>
+        <!--
+        <collision>
+          <geometry>
+            <mesh filename="package://schunk_description/meshes/pw70/pw70_base.stl" />
+          </geometry>
+        </collision>
+        -->
+      </link>
+      <joint name="${name}_pan_joint" type="revolute" >
+        <origin xyz="0 0 0" rpy="0 0 0"/>
+        <parent link="${name}_link" />
+        <child link="${name}_pan_link" />
+        <axis xyz="0 0 -1" />
+        <limit effort="200" velocity="${2 * M_PI}" lower="${-7/3 * M_PI}" upper="${7/3 * M_PI}"/>
+        <calibration rising="0.0"/>
+      </joint>
+      <link name="${name}_pan_link">
+        <xacro:default_inertial/>
+        <visual>
+          <origin xyz="0 0 0" rpy="0 0 0" />
+          <geometry>
+            <mesh filename="package://schunk_description/meshes/pw70/pw70_pan.dae" />
+          </geometry>
+        </visual>
+        <!--
+        <collision>
+          <geometry>
+            <mesh filename="package://schunk_description/meshes/pw70/pw70_pan.stl" />
+          </geometry>
+        </collision>
+        -->
+      </link>
+      <joint name="${name}_tilt_joint" type="revolute" >
+        <origin xyz="0 0 0.0951" rpy="0 0 0"/>
+        <parent link="${name}_pan_link" />
+        <child link="${name}_tilt_link" />
+        <axis xyz="0 -1 0" />
+        <limit effort="12.0" velocity="4.1" lower="${-4/6 * M_PI}" upper="${4/6 * M_PI}"/>
+        <calibration rising="0.0"/>
+      </joint>
+      <link name="${name}_tilt_link">
+        <xacro:default_inertial/>
+        <visual>
+          <origin xyz="0 0 0" rpy="0 0 0" />
+          <geometry>
+            <mesh filename="package://schunk_description/meshes/pw70/pw70_tilt.dae" />
+          </geometry>
+        </visual>
+        <!--
+        <collision>
+          <geometry>
+            <mesh filename="package://schunk_description/meshes/pw70/pw70_tilt.stl" />
+          </geometry>
+        </collision>
+        -->
+      </link>
+      <joint name="${name}_tool_joint" type="fixed" >
+        <origin xyz="0 0 0.07" rpy="0 0 0"/>
+        <parent link="${name}_tilt_link" />
+        <child link="${name}_tool_link" />
+      </joint>
+      <link name="${name}_tool_link">
+        <xacro:default_inertial/>
+      </link>
+    </xacro:if>
+    <!-- extensions -->
+    <xacro:schunk_pw70_gazebo name="${name}" />
+    <xacro:schunk_pw70_transmission name="${name}" />
   </xacro:macro>
 </robot>

Commit message: pw70 working

File: schunk_description/urdf/pw70/pw70.urdf.xacro (robot description, xacro)
@@ -12,4 +12,15 @@
       <link name="${name}_link">
         <xacro:default_inertial/>
+	<visual>
+          <origin xyz="0 0 0.07" rpy="0 0 0" />
+          <geometry>
+            <mesh filename="package://schunk_description/meshes/pw70/pw70_square_holder.stl" />
+          </geometry>
+        </visual>
+<!--        <collision>
+          <geometry>
+            <mesh filename="package://schunk_description/meshes/pw70/pw70_square_holder.stl" />
+          </geometry>
+        </collision>  -->
       </link>
       <joint name="${name}_tilt_joint" type="revolute" >
@@ -17,5 +28,5 @@
         <parent link="${name}_link" />
         <child link="${name}_tilt_link" />
-        <axis xyz="0 1 0" />
+        <axis xyz="-1 0  0" />
         <limit effort="12.0" velocity="4.1" lower="${-4/6 * M_PI}" upper="${4/6 * M_PI}"/>
         <calibration rising="0.0"/>
@@ -26,23 +37,21 @@
           <origin xyz="0 0 0" rpy="0 0 0" />
           <geometry>
-            <mesh filename="package://schunk_description/meshes/pw70/pw70_tilt.dae" />
+            <mesh filename="package://schunk_description/meshes/pw70/pw70_body.stl" />
           </geometry>
         </visual>
-        <!--
-        <collision>
+<!--        <collision>
           <geometry>
-            <mesh filename="package://schunk_description/meshes/pw70/pw70_tilt.stl" />
+            <mesh filename="package://schunk_description/meshes/pw70/pw70_body.stl" />
           </geometry>
-        </collision>
-        -->
+        </collision>-->
       </link>
       <joint name="${name}_pan_joint" type="revolute" >
-        <origin xyz="0 0 0.0951" rpy="0 0 0"/>
-        <parent link="${name}_tilt_joint" />
+        <origin xyz="0 0 0" rpy="0 0 0"/>
+        <parent link="${name}_tilt_link" />
         <child link="${name}_pan_link" />
         <axis xyz="0 0 1" />
         <limit effort="200" velocity="${2 * M_PI}" lower="${-7/3 * M_PI}" upper="${7/3 * M_PI}"/>
         <calibration rising="0.0"/>
-      </joint>
+     </joint>
       <link name="${name}_pan_link">
         <xacro:default_inertial/>
@@ -50,17 +59,15 @@
           <origin xyz="0 0 0" rpy="0 0 0" />
           <geometry>
-            <mesh filename="package://schunk_description/meshes/pw70/pw70_pan.dae" />
+            <mesh filename="package://schunk_description/meshes/pw70/pw70_round_holder.stl" />
           </geometry>
         </visual>
-        <!--
-        <collision>
+<!--        <collision>
           <geometry>
-            <mesh filename="package://schunk_description/meshes/pw70/pw70_pan.stl" />
+            <mesh filename="package://schunk_description/meshes/pw70/pw70_round_holder.stl" />
           </geometry>
-        </collision>
-        -->
+        </collision>-->
       </link>
       <joint name="${name}_tool_joint" type="fixed" >
-        <origin xyz="0 0 0.07" rpy="0 0 0"/>
+        <origin xyz="0 0 0.095" rpy="0 0 0"/>
         <parent link="${name}_pan_link" />
         <child link="${name}_tool_link" />
@@ -68,17 +75,4 @@
       <link name="${name}_tool_link">
         <xacro:default_inertial/>
-        <visual>
-          <origin xyz="0 0 0" rpy="0 0 0" />
-          <geometry>
-            <mesh filename="package://schunk_description/meshes/pw70/pw70_base.dae" />
-          </geometry>
-        </visual>
-        <!--
-        <collision>
-          <geometry>
-            <mesh filename="package://schunk_description/meshes/pw70/pw70_base.stl" />
-          </geometry>
-        </collision>
-        -->
       </link>
     </xacro:unless>
@@ -92,19 +86,17 @@
         <xacro:default_inertial/>
         <visual>
-          <origin xyz="0 0 0" rpy="0 0 0" />
+          <origin xyz="0 0 0.095" rpy="${M_PI} 0 0" />
           <geometry>
-            <mesh filename="package://schunk_description/meshes/pw70/pw70_base.dae" />
+            <mesh filename="package://schunk_description/meshes/pw70/pw70_round_holder.stl" />
           </geometry>
         </visual>
-        <!--
-        <collision>
+<!--        <collision>
           <geometry>
-            <mesh filename="package://schunk_description/meshes/pw70/pw70_base.stl" />
+            <mesh filename="package://schunk_description/meshes/pw70/pw70_round_holder.stl" />
           </geometry>
-        </collision>
-        -->
+        </collision>-->
       </link>
       <joint name="${name}_pan_joint" type="revolute" >
-        <origin xyz="0 0 0" rpy="0 0 0"/>
+        <origin xyz="0 0 0.095" rpy="0 0 0"/>
         <parent link="${name}_link" />
         <child link="${name}_pan_link" />
@@ -116,22 +108,20 @@
         <xacro:default_inertial/>
         <visual>
-          <origin xyz="0 0 0" rpy="0 0 0" />
+          <origin xyz="0 0 0" rpy="${M_PI} 0 0" />
           <geometry>
-            <mesh filename="package://schunk_description/meshes/pw70/pw70_pan.dae" />
+            <mesh filename="package://schunk_description/meshes/pw70/pw70_body.stl" />
           </geometry>
         </visual>
-        <!--
-        <collision>
+<!--        <collision>
           <geometry>
-            <mesh filename="package://schunk_description/meshes/pw70/pw70_pan.stl" />
+            <mesh filename="package://schunk_description/meshes/pw70/pw70_body.stl"/>
           </geometry>
-        </collision>
-        -->
+        </collision>   -->
       </link>
       <joint name="${name}_tilt_joint" type="revolute" >
-        <origin xyz="0 0 0.0951" rpy="0 0 0"/>
+        <origin xyz="0 0 0" rpy="0 0 0"/>
         <parent link="${name}_pan_link" />
         <child link="${name}_tilt_link" />
-        <axis xyz="0 -1 0" />
+        <axis xyz="-1 0 0" />
         <limit effort="12.0" velocity="4.1" lower="${-4/6 * M_PI}" upper="${4/6 * M_PI}"/>
         <calibration rising="0.0"/>
@@ -140,16 +130,14 @@
         <xacro:default_inertial/>
         <visual>
-          <origin xyz="0 0 0" rpy="0 0 0" />
+          <origin xyz="0 0 0" rpy="${M_PI} 0 0" />
           <geometry>
-            <mesh filename="package://schunk_description/meshes/pw70/pw70_tilt.dae" />
+            <mesh filename="package://schunk_description/meshes/pw70/pw70_square_holder.stl" />
           </geometry>
         </visual>
-        <!--
-        <collision>
+        <!--<collision>
           <geometry>
-            <mesh filename="package://schunk_description/meshes/pw70/pw70_tilt.stl" />
+            <mesh filename="package://schunk_description/meshes/pw70/pw70_square_holder.stl" />
           </geometry>
-        </collision>
-        -->
+        </collision>    -->
       </link>
       <joint name="${name}_tool_joint" type="fixed" >
