Commit message: Enabled collison

File: schunk_description/urdf/pw70/pw70.urdf.xacro (robot description, xacro)
@@ -12,5 +12,5 @@
       <link name="${name}_link">
         <xacro:default_inertial/>
-	<visual>
+        <visual>
           <origin xyz="0 0 0.07" rpy="0 0 0" />
           <geometry>
@@ -18,9 +18,9 @@
           </geometry>
         </visual>
-<!--        <collision>
+        <collision>
           <geometry>
             <mesh filename="package://schunk_description/meshes/pw70/pw70_square_holder.stl" />
           </geometry>
-        </collision>  -->
+        </collision>
       </link>
       <joint name="${name}_tilt_joint" type="revolute" >
@@ -40,9 +40,9 @@
           </geometry>
         </visual>
-<!--        <collision>
+        <collision>
           <geometry>
             <mesh filename="package://schunk_description/meshes/pw70/pw70_body.stl" />
           </geometry>
-        </collision>-->
+        </collision>
       </link>
       <joint name="${name}_pan_joint" type="revolute" >
@@ -62,9 +62,9 @@
           </geometry>
         </visual>
-<!--        <collision>
+        <collision>
           <geometry>
             <mesh filename="package://schunk_description/meshes/pw70/pw70_round_holder.stl" />
           </geometry>
-        </collision>-->
+        </collision>
       </link>
       <joint name="${name}_tool_joint" type="fixed" >
@@ -91,9 +91,9 @@
           </geometry>
         </visual>
-<!--        <collision>
+        <collision>
           <geometry>
             <mesh filename="package://schunk_description/meshes/pw70/pw70_round_holder.stl" />
           </geometry>
-        </collision>-->
+        </collision>
       </link>
       <joint name="${name}_pan_joint" type="revolute" >
@@ -113,9 +113,9 @@
           </geometry>
         </visual>
-<!--        <collision>
+        <collision>
           <geometry>
             <mesh filename="package://schunk_description/meshes/pw70/pw70_body.stl"/>
           </geometry>
-        </collision>   -->
+        </collision>
       </link>
       <joint name="${name}_tilt_joint" type="revolute" >
@@ -135,9 +135,9 @@
           </geometry>
         </visual>
-        <!--<collision>
+        <collision>
           <geometry>
             <mesh filename="package://schunk_description/meshes/pw70/pw70_square_holder.stl" />
           </geometry>
-        </collision>    -->
+        </collision>
       </link>
       <joint name="${name}_tool_joint" type="fixed" >
